Commit message: Changes to the single robot macros
Maybe these files should be deleted instead, but these trailing changes might be helpful at some point.

File: o2as_scene_description/urdf/ur10_joint_limited_robot.urdf.xacro (robot description, xacro)
@@ -2,4 +2,5 @@
 <robot xmlns:xacro="http://ros.org/wiki/xacro"
        name="ur10" >
+  <xacro:arg name="parent" default="world"/>
   <xacro:arg name="prefix" default=""/>
   <xacro:arg name="origin_xyz" default="0.0 0.0 0.0"/>
@@ -18,8 +19,8 @@
     wrist_3_lower_limit="${-pi}" wrist_3_upper_limit="${pi}"
   />
-  <link name="world" />
-  <joint name="world_joint" type="fixed">
-    <parent link="world" />
-    <child link = "$(arg prefix)base_link" />
+  <link name="$(arg parent)" />
+  <joint name="$(arg parent)_joint" type="fixed">
+    <parent link="$(arg parent)" />
+    <child link ="$(arg prefix)base_link" />
     <origin xyz="$(arg origin_xyz)" rpy="$(arg origin_rpy)" />
   </joint>

File: o2as_scene_description/urdf/ur10_robot.urdf.xacro (robot description, xacro)
@@ -2,4 +2,5 @@
 <robot xmlns:xacro="http://ros.org/wiki/xacro"
        name="ur10" >
+  <xacro:arg name="parent" default="world"/>
   <xacro:arg name="prefix" default=""/>
   <xacro:arg name="origin_xyz" default="0.0 0.0 0.0"/>
@@ -11,8 +12,8 @@
   <!-- arm -->
   <xacro:ur10_robot prefix="$(arg prefix)" joint_limited="false"/>
-  <link name="world" />
-  <joint name="world_joint" type="fixed">
-    <parent link="world" />
-    <child link = "$(arg prefix)base_link" />
+  <link name="$(arg parent)" />
+  <joint name="$(arg parent)_joint" type="fixed">
+    <parent link="$(arg parent)" />
+    <child link ="$(arg prefix)base_link" />
     <origin xyz="$(arg origin_xyz)" rpy="$(arg origin_rpy)" />
   </joint>

File: o2as_scene_description/urdf/ur3_joint_limited_robot.urdf.xacro (robot description, xacro)
@@ -2,4 +2,5 @@
 <robot xmlns:xacro="http://ros.org/wiki/xacro"
        name="ur3" >
+  <xacro:arg name="parent" default="world"/>
   <xacro:arg name="prefix" default=""/>
   <xacro:arg name="origin_xyz" default="0.0 0.0 0.0"/>
@@ -18,8 +19,8 @@
     wrist_3_lower_limit="${-pi}" wrist_3_upper_limit="${pi}"
   />
-  <link name="world" />
-  <joint name="world_joint" type="fixed">
-    <parent link="world" />
-    <child link = "$(arg prefix)base_link" />
+  <link name="$(arg parent)" />
+  <joint name="$(arg parent)_joint" type="fixed">
+    <parent link="$(arg parent)" />
+    <child link ="$(arg prefix)base_link" />
     <origin xyz="$(arg origin_xyz)" rpy="$(arg origin_rpy)" />
   </joint>

File: o2as_scene_description/urdf/ur3_robot.urdf.xacro (robot description, xacro)
@@ -2,4 +2,5 @@
 <robot xmlns:xacro="http://ros.org/wiki/xacro"
        name="ur3" >
+  <xacro:arg name="parent" default="world"/>
   <xacro:arg name="prefix" default=""/>
   <xacro:arg name="origin_xyz" default="0.0 0.0 0.0"/>
@@ -11,8 +12,8 @@
   <!-- arm -->
   <xacro:ur3_robot prefix="$(arg prefix)" joint_limited="false"/>
-  <link name="world" />
-  <joint name="world_joint" type="fixed">
-    <parent link="world" />
-    <child link = "$(arg prefix)base_link" />
+  <link name="$(arg parent)" />
+  <joint name="$(arg parent)_joint" type="fixed">
+    <parent link="$(arg parent)" />
+    <child link ="$(arg prefix)base_link" />
     <origin xyz="$(arg origin_xyz)" rpy="$(arg origin_rpy)" />
   </joint>

File: o2as_scene_description/urdf/ur5_joint_limited_robot.urdf.xacro (robot description, xacro)
@@ -2,4 +2,5 @@
 <robot xmlns:xacro="http://ros.org/wiki/xacro"
        name="ur5" >
+  <xacro:arg name="parent" default="world"/>
   <xacro:arg name="prefix" default=""/>
   <xacro:arg name="origin_xyz" default="0.0 0.0 0.0"/>
@@ -18,8 +19,8 @@
     wrist_3_lower_limit="${-pi}" wrist_3_upper_limit="${pi}"
   />
-  <link name="world" />
-  <joint name="world_joint" type="fixed">
-    <parent link="world" />
-    <child link = "$(arg prefix)base_link" />
+  <link name="$(arg parent)" />
+  <joint name="$(arg parent)_joint" type="fixed">
+    <parent link="$(arg parent)" />
+    <child link ="$(arg prefix)base_link" />
     <origin xyz="$(arg origin_xyz)" rpy="$(arg origin_rpy)" />
   </joint>

File: o2as_scene_description/urdf/ur5_robot.urdf.xacro (robot description, xacro)
@@ -2,4 +2,5 @@
 <robot xmlns:xacro="http://ros.org/wiki/xacro"
        name="ur5" >
+  <xacro:arg name="parent" default="world"/>
   <xacro:arg name="prefix" default=""/>
   <xacro:arg name="origin_xyz" default="0.0 0.0 0.0"/>
@@ -11,8 +12,8 @@
   <!-- arm -->
   <xacro:ur5_robot prefix="$(arg prefix)" joint_limited="false"/>
-  <link name="world" />
-  <joint name="world_joint" type="fixed">
-    <parent link="world" />
-    <child link = "$(arg prefix)base_link" />
+  <link name="$(arg parent)" />
+  <joint name="$(arg parent)_joint" type="fixed">
+    <parent link="$(arg parent)" />
+    <child link ="$(arg prefix)base_link" />
     <origin xyz="$(arg origin_xyz)" rpy="$(arg origin_rpy)" />
   </joint>
