Commit message: Fix kitting bin mesh in gazebo, + fix forgotten file
1) The mesh is loaded in gazebo but not in MoveIt now. 2) The last commit was missing changes in the gazebo launch file.

File: o2as_scene_description/urdf/kitting_bin.xacro (robot description, xacro)
@@ -3,6 +3,6 @@
   <xacro:macro name="kitting_bin" params="binname parent *origin">
   <!-- This creates a box with the origin in the bottom corner, connected to the world link. -->
-  <xacro:property name="mesh_file" value="$(find o2as_scene_description)/mesh/bin1_EA661CA-11.stl" />
-  <xacro:property name="mesh_file_col" value="$(find o2as_scene_description)/mesh/bin1_EA661CA-11.vhacd.obj" />
+  <xacro:property name="mesh_file" value="$(find o2as_scene_description)/meshes/bin1_EA661CA-11.stl" />
+  <xacro:property name="mesh_file_col" value="$(find o2as_scene_description)/meshes/bin1_EA661CA-11.vhacd.obj" />
   <link name="${binname}">
     <inertial>
@@ -12,8 +12,8 @@
     </inertial>
     <visual>
-      <origin rpy="1.5707 0 0" xyz="0 0 0"/>
+      <origin rpy="${pi/2} 0 ${pi/2}" xyz="0 0 0"/>
       <geometry>
-        <!-- <mesh filename="${mesh_file}" scale="0.001 0.001 0.001"/> -->
-        <mesh filename="package://ur_description/meshes/ur5/visual/shoulder.dae"/>
+        <mesh filename="${mesh_file}" scale="0.001 0.001 0.001"/>
+        <!-- <mesh filename="package://ur_description/meshes/ur5/visual/shoulder.dae"/> -->
       </geometry>
       <material name="white">
@@ -22,8 +22,8 @@
     </visual>
     <collision>
-      <origin rpy="1.5707 0 0" xyz="0 0 0"/>
+      <origin rpy="${pi/2} 0 ${pi/2}" xyz="0 0 0"/>
       <geometry>
-        <!-- <mesh filename="${mesh_file_col}" scale="0.001 0.001 0.001"/> -->
-        <mesh filename="package://ur_description/meshes/ur5/collision/shoulder.stl"/>
+        <mesh filename="${mesh_file_col}" scale="0.001 0.001 0.001"/>
+        <!-- <mesh filename="package://ur_description/meshes/ur5/collision/shoulder.stl"/> -->
       </geometry>
     </collision>

Commit message: Avoid a strange bug when reading in mesh files
Thanks to Yoshioka-san for finding it.

File: o2as_scene_description/urdf/kitting_bin.xacro (robot description, xacro)
@@ -3,6 +3,9 @@
   <xacro:macro name="kitting_bin" params="binname parent *origin">
   <!-- This creates a box with the origin in the bottom corner, connected to the world link. -->
-  <xacro:property name="mesh_file" value="$(find o2as_scene_description)/meshes/bin1_EA661CA-11.stl" />
-  <xacro:property name="mesh_file_col" value="$(find o2as_scene_description)/meshes/bin1_EA661CA-11.vhacd.obj" />
+  <!-- <xacro:property name="mesh_file" value="$(find o2as_scene_description)/meshes/bin1_EA661CA-11.stl" />
+  <xacro:property name="mesh_file_col" value="$(find o2as_scene_description)/meshes/bin1_EA661CA-11.vhacd.obj" /> -->
+  <!-- The lines above don't work, the lines below do. Why?? This seems like a bug. -->
+  <xacro:property name="mesh_file" value="package://o2as_scene_description/meshes/bin1_EA661CA-11.stl" />
+  <xacro:property name="mesh_file_col" value="package://o2as_scene_description/meshes/bin1_EA661CA-11.vhacd.obj" />
   <link name="${binname}">
     <inertial>

Commit message: Fix gazebo colors

File: o2as_scene_description/urdf/kitting_bin.xacro (robot description, xacro)
@@ -32,4 +32,7 @@
     </collision>
   </link>
+  <gazebo reference="${binname}">
+    <material>Gazebo/Orange</material>
+  </gazebo>
   <joint name="${binname}" type="fixed">
       <parent link="${parent}" />

File: o2as_scene_description/urdf/o2as_base.xacro (robot description, xacro)
@@ -30,8 +30,8 @@
           izz="0.0" />
       </inertial>
-      <!-- <gazebo reference="${boxname}">
-        <material>Gazebo/DarkGrey</material>
-      </gazebo> -->
     </link>
+    <gazebo reference="${boxname}">
+      <material>Gazebo/FlatBlack</material>
+    </gazebo>
     <joint name="${boxname}" type="fixed">
       <parent link="world" />

File: o2as_scene_description/urdf/o2as_box.xacro (robot description, xacro)
@@ -3,7 +3,4 @@
   <xacro:macro name="o2as_box" params="boxname box_w box_l box_h *origin">
     <!-- This creates a box with the origin in the bottom corner, fixed to the world link. -->
-    <!-- <gazebo reference="${boxname}">
-      <material>Gazebo/Gray</material>
-    </gazebo> -->
     <link name="${boxname}">
       <!-- w is in x, l is in y, h is in z -->
@@ -31,4 +28,7 @@
       </inertial>
     </link>
+    <gazebo reference="${boxname}">
+      <material>Gazebo/Grey</material>
+    </gazebo>
     <joint name="${boxname}" type="fixed">
       <parent link="world" />
