Commit message: add kitting scene.

File: o2as_scene_description/urdf/kit_task_scene.urdf.xacro (robot description, xacro)
@@ -1,5 +1,5 @@
 <?xml version="1.0"?>
 <robot xmlns:xacro="http://ros.org/wiki/xacro"
-       name="asm_task_scene" >
+       name="kit_task_scene" >
   <xacro:property name="a_bot_x" value="0.0"/>
   <xacro:property name="a_bot_y" value="0.5"/>
@@ -13,22 +13,20 @@
   <xacro:include filename="$(find ur_description)/urdf/common.gazebo.xacro" />
   <!-- robots -->
+  <xacro:include filename="$(find o2as_scene_description)/urdf/ur10.urdf.xacro" />
   <xacro:include filename="$(find o2as_scene_description)/urdf/ur5.urdf.xacro" />
   <xacro:include filename="$(find o2as_scene_description)/urdf/ur3.urdf.xacro" />
-  <!-- grippers -->
-  <!-- <xacro:include filename="$(find robotiq_c2_model_visualization)/urdf/robotiq_c2_model_macro.xacro" /> -->
   <!-- Scene items (trays, bins...) -->
   <xacro:include filename="$(find o2as_scene_description)/urdf/kitting_scene_1.xacro" />
   <!-- Robot bases -->
-  <xacro:property name="table_edge" value=".4" />
   <!-- Putting these at height 0.0 makes them intersect with the ground, so they are elevated. -->
   <!-- There are some instabilities when the box is big, for some reason. -->
   <xacro:include filename="$(find o2as_scene_description)/urdf/o2as_base.xacro" />
-  <xacro:o2as_base boxname="a_bot_base_smfl">
+  <xacro:o2as_base boxname="a_bot_base_smfl" parent="o2as_ground">
     <origin xyz="${a_bot_x-.65/2} ${a_bot_y-.65/2} 0.65" rpy="0 0 0" />
   </xacro:o2as_base>
-  <xacro:o2as_base boxname="b_bot_base_smfl">
+  <xacro:o2as_base boxname="b_bot_base_smfl" parent="o2as_ground">
     <origin xyz="${b_bot_x-.65/2} ${b_bot_y-.65/2} 0.65" rpy="0 0 0" />
   </xacro:o2as_base>
-  <xacro:o2as_base boxname="c_bot_base_smfl">
+  <xacro:o2as_base boxname="c_bot_base_smfl" parent="o2as_ground">
     <origin xyz="${c_bot_x-.65/2-.22} ${c_bot_y-.65/2-.22} 0.65" rpy="0 0 0" />
   </xacro:o2as_base>
@@ -38,10 +36,10 @@
   <xacro:property name="plate_w" value="0.8"/>
   <xacro:property name="plate_l" value="0.8"/>
-  <xacro:o2as_box boxname="workbox" box_w="${plate_w}" box_l="${plate_l}" box_h=".01">
+  <xacro:o2as_box boxname="workbox" box_w="${plate_w}" box_l="${plate_l}" box_h=".01" parent="o2as_ground">
     <origin xyz="${-plate_w/2} ${-plate_l/2} ${bots_z-.02}" rpy="0 0 0" />
   </xacro:o2as_box>
   <link name="workspace_center" />
   <joint name="world_to_workspace" type="fixed">
-    <parent link="world" />
+    <parent link="o2as_ground" />
     <child link="workspace_center" />
     <origin xyz="0.0 0.0 ${bots_z}" rpy="0.0 0.0 0.0" />
@@ -69,25 +67,37 @@
     wrist_2_lower_limit="${-pi}" wrist_2_upper_limit="${pi}"
     wrist_3_lower_limit="${-pi}" wrist_3_upper_limit="${pi}"/>
-  <link name="world" />
+  <link name="o2as_ground" />
   <joint name="world_a_bot_joint" type="fixed">
-    <parent link="world" />
+    <parent link="o2as_ground" />
     <child link="a_bot_base_link" />
     <origin xyz="${a_bot_x} ${a_bot_y} ${bots_z}" rpy="0.0 0.0 0.0" />
   </joint>
   <joint name="world_b_bot_joint" type="fixed">
-    <parent link="world" />
+    <parent link="o2as_ground" />
     <child link = "b_bot_base_link" />
     <origin xyz="${b_bot_x} ${b_bot_y} ${bots_z}" rpy="0.0 0.0 0.0" />
   </joint>
   <joint name="world_c_bot_joint" type="fixed">
-    <parent link="world" />
+    <parent link="o2as_ground" />
     <child link = "c_bot_base_link" />
     <origin xyz="${c_bot_x} ${c_bot_y} ${bots_z}" rpy="0.0 0.0 0.0" />
   </joint>
-  <!-- attach grippers -->
-    <!-- <joint name="a_bot_gripper_link" type="fixed">
-      <origin xyz="0 0 0" rpy="0 0 0" />
-      <parent link="a_bot_tool0" />
-      <child link="a_bot_eef_link" />
-    </joint> -->
+  <!-- spawn and attach grippers -->
+  <xacro:include filename="$(find o2as_scene_description)/urdf/robotiq_85_gripper.urdf.xacro" />
+  <xacro:robotiq_85_gripper_o2as prefix="a_bot_" parent = "a_bot_ee_link">
+    <origin xyz="0.0 0 0.0" rpy="0 0 0"/>
+  </xacro:robotiq_85_gripper_o2as>
+  <xacro:robotiq_85_gripper_o2as prefix="b_bot_" parent = "b_bot_ee_link">
+    <origin xyz="0.0 0 0.0" rpy="0 0 0"/>
+  </xacro:robotiq_85_gripper_o2as>
+  <xacro:robotiq_85_gripper_o2as prefix="c_bot_" parent = "c_bot_ee_link">
+    <origin xyz="0.0 0 0.0" rpy="0 0 0"/>
+  </xacro:robotiq_85_gripper_o2as>
+  <!-- I meant to remove the "world" link definition, but apparently it is necessary for Gazebo -->
+  <link name="world" />
+  <joint name="world_o2as_joint" type="fixed">
+    <parent link="world" />
+    <child link="o2as_ground" />
+    <origin xyz="0.0 0.0 0.0" rpy="0.0 0.0 0.0" />
+  </joint>
 </robot>

File: o2as_scene_description/urdf/kitting_scene_1.xacro (robot description, xacro)
@@ -1,7 +1,5 @@
 <?xml version="1.0"?>
 <robot xmlns:xacro="http://www.ros.org/wiki/xacro" name="kitting_scene">
-  <xacro:include filename="$(find o2as_scene_description)/urdf/kitting_bin1.xacro" />
-  <xacro:include filename="$(find o2as_scene_description)/urdf/kitting_bin2.xacro" />
-  <xacro:include filename="$(find o2as_scene_description)/urdf/kitting_bin3.xacro" />
+  <xacro:include filename="$(find o2as_scene_description)/urdf/kitting_bins.xacro" />
   <xacro:include filename="$(find o2as_scene_description)/urdf/kitting_tray.xacro" />
   <xacro:property name="bin1_width" value=".125"/>
@@ -18,19 +16,19 @@
   <xacro:property name="set1_y" value="${.32-bin1_width/2}"/>
   <xacro:property name="set1_z" value=".00" />
-  <xacro:kitting_bin1 binname="set1_bin1_1" parent="workspace_center">
+  <xacro:kitting_bin_1 binname="set1_bin1_1" parent="workspace_center">
     <origin xyz="${set1_x} ${set1_y} ${set1_z}" rpy="0 0 0" />
-  </xacro:kitting_bin1>
-  <xacro:kitting_bin1 binname="set1_bin1_2" parent="workspace_center">
+  </xacro:kitting_bin_1>
+  <xacro:kitting_bin_1 binname="set1_bin1_2" parent="workspace_center">
     <origin xyz="${set1_x} ${set1_y - bin1_width*1} ${set1_z}" rpy="0 0 0" />
-  </xacro:kitting_bin1>
-  <xacro:kitting_bin1 binname="set1_bin1_3" parent="workspace_center">
+  </xacro:kitting_bin_1>
+  <xacro:kitting_bin_1 binname="set1_bin1_3" parent="workspace_center">
     <origin xyz="${set1_x} ${set1_y - bin1_width*2} ${set1_z}" rpy="0 0 0" />
-  </xacro:kitting_bin1>
-  <xacro:kitting_bin1 binname="set1_bin1_4" parent="workspace_center">
+  </xacro:kitting_bin_1>
+  <xacro:kitting_bin_1 binname="set1_bin1_4" parent="workspace_center">
     <origin xyz="${set1_x} ${set1_y - bin1_width*3} ${set1_z}" rpy="0 0 0" />
-  </xacro:kitting_bin1>
-  <xacro:kitting_bin1 binname="set1_bin1_5" parent="workspace_center">
+  </xacro:kitting_bin_1>
+  <xacro:kitting_bin_1 binname="set1_bin1_5" parent="workspace_center">
     <origin xyz="${set1_x} ${set1_y - bin1_width*4} ${set1_z}" rpy="0 0 0" />
-  </xacro:kitting_bin1>
+  </xacro:kitting_bin_1>
   <!-- A row of bin2 and bin3 -->
   <xacro:property name="set2_x_bin3" value="${bin1_length/2+bin3_length/2}" />
@@ -38,19 +36,19 @@
   <xacro:property name="set2_y" value="${.32-bin3_width/2}" />
   <xacro:property name="set2_z" value=".00" />
-  <xacro:kitting_bin3 binname="set2_bin3" parent="workspace_center">
+  <xacro:kitting_bin_3 binname="set2_bin3" parent="workspace_center">
     <origin xyz="${set2_x_bin3} ${set2_y} ${set2_z}" rpy="0 0 0" />
-  </xacro:kitting_bin3>
-  <xacro:kitting_bin2 binname="set2_bin2_1" parent="workspace_center">
+  </xacro:kitting_bin_3>
+  <xacro:kitting_bin_2 binname="set2_bin2_1" parent="workspace_center">
     <origin xyz="${set2_x_bin2} ${set2_y-bin3_width/2-bin2_width/2*1} ${set2_z}" rpy="0 0 0" />
-  </xacro:kitting_bin2>
-  <xacro:kitting_bin2 binname="set2_bin2_2" parent="workspace_center">
+  </xacro:kitting_bin_2>
+  <xacro:kitting_bin_2 binname="set2_bin2_2" parent="workspace_center">
     <origin xyz="${set2_x_bin2} ${set2_y-bin3_width/2-bin2_width*3/2} ${set2_z}" rpy="0 0 0" />
-  </xacro:kitting_bin2>
-  <xacro:kitting_bin2 binname="set2_bin2_3" parent="workspace_center">
+  </xacro:kitting_bin_2>
+  <xacro:kitting_bin_2 binname="set2_bin2_3" parent="workspace_center">
     <origin xyz="${set2_x_bin2} ${set2_y-bin3_width/2-bin2_width*5/2} ${set2_z}" rpy="0 0 0" />
-  </xacro:kitting_bin2>
-  <xacro:kitting_bin2 binname="set2_bin2_4" parent="workspace_center">
+  </xacro:kitting_bin_2>
+  <xacro:kitting_bin_2 binname="set2_bin2_4" parent="workspace_center">
     <origin xyz="${set2_x_bin2} ${set2_y-bin3_width/2-bin2_width*7/2} ${set2_z}" rpy="0 0 0" />
-  </xacro:kitting_bin2>
+  </xacro:kitting_bin_2>
   <!-- A row of tray -->
   <xacro:property name="set3_x" value="${-(bin1_length/2+tray_length/2)}" />

Commit message: Add script to simulate reachable area on KITTing

File: o2as_scene_description/urdf/kit_task_scene.urdf.xacro (robot description, xacro)
@@ -34,8 +34,8 @@
   <!-- The surface is 0.01 m below the robot bases and the "workspace_center" frame. -->
   <xacro:include filename="$(find o2as_scene_description)/urdf/o2as_box.xacro" />
-  <xacro:property name="plate_w" value="0.8"/>
-  <xacro:property name="plate_l" value="0.8"/>
+  <xacro:property name="plate_w" value="0.84"/>
+  <xacro:property name="plate_l" value="0.62"/>
   <xacro:o2as_box boxname="workbox" box_w="${plate_w}" box_l="${plate_l}" box_h=".01" parent="o2as_ground">
-    <origin xyz="${-plate_w/2} ${-plate_l/2} ${bots_z-.02}" rpy="0 0 0" />
+    <origin xyz="${-plate_w/2} ${-plate_l/2} ${bots_z+.09}" rpy="0 0 0" />
   </xacro:o2as_box>
   <link name="workspace_center" />
@@ -43,5 +43,5 @@
     <parent link="o2as_ground" />
     <child link="workspace_center" />
-    <origin xyz="0.0 0.0 ${bots_z}" rpy="0.0 0.0 0.0" />
+    <origin xyz="0.0 0.0 ${bots_z+.1}" rpy="0.0 0.0 0.0" />
   </joint>
   <!-- robot arms -->
@@ -53,5 +53,5 @@
     wrist_2_lower_limit="${-pi}" wrist_2_upper_limit="${pi}"
     wrist_3_lower_limit="${-pi}" wrist_3_upper_limit="${pi}"/>
-  <xacro:ur5_robot prefix="b_bot_" joint_limited="true"
+  <!-- <xacro:ur5_robot prefix="b_bot_" joint_limited="true"
     shoulder_pan_lower_limit="${-pi}" shoulder_pan_upper_limit="${pi}"
     shoulder_lift_lower_limit="${-pi}" shoulder_lift_upper_limit="${pi}"
@@ -66,5 +66,5 @@
     wrist_1_lower_limit="${-pi}" wrist_1_upper_limit="${pi}"
     wrist_2_lower_limit="${-pi}" wrist_2_upper_limit="${pi}"
-    wrist_3_lower_limit="${-pi}" wrist_3_upper_limit="${pi}"/>
+    wrist_3_lower_limit="${-pi}" wrist_3_upper_limit="${pi}"/> -->
   <link name="o2as_ground" />
   <joint name="world_a_bot_joint" type="fixed">
@@ -73,5 +73,5 @@
     <origin xyz="${a_bot_x} ${a_bot_y} ${bots_z}" rpy="0.0 0.0 0.0" />
   </joint>
-  <joint name="world_b_bot_joint" type="fixed">
+  <!-- <joint name="world_b_bot_joint" type="fixed">
     <parent link="o2as_ground" />
     <child link = "b_bot_base_link" />
@@ -82,5 +82,5 @@
     <child link = "c_bot_base_link" />
     <origin xyz="${c_bot_x} ${c_bot_y} ${bots_z}" rpy="0.0 0.0 0.0" />
-  </joint>
+  </joint> -->
   <!-- spawn and attach grippers -->
   <xacro:include filename="$(find o2as_scene_description)/urdf/robotiq_85_gripper.urdf.xacro" />
@@ -88,10 +88,10 @@
     <origin xyz="0.0 0 0.0" rpy="0 0 0"/>
   </xacro:robotiq_85_gripper_o2as>
-  <xacro:robotiq_85_gripper_o2as prefix="b_bot_" parent = "b_bot_ee_link">
+  <!-- <xacro:robotiq_85_gripper_o2as prefix="b_bot_" parent = "b_bot_ee_link">
     <origin xyz="0.0 0 0.0" rpy="0 0 0"/>
   </xacro:robotiq_85_gripper_o2as>
   <xacro:robotiq_85_gripper_o2as prefix="c_bot_" parent = "c_bot_ee_link">
     <origin xyz="0.0 0 0.0" rpy="0 0 0"/>
-  </xacro:robotiq_85_gripper_o2as>
+  </xacro:robotiq_85_gripper_o2as> -->
   <!-- I meant to remove the "world" link definition, but apparently it is necessary for Gazebo -->
   <link name="world" />

Commit message: WIP: initial robot pose is occured collision.

File: o2as_scene_description/urdf/kit_task_scene.urdf.xacro (robot description, xacro)
@@ -53,5 +53,5 @@
     wrist_2_lower_limit="${-pi}" wrist_2_upper_limit="${pi}"
     wrist_3_lower_limit="${-pi}" wrist_3_upper_limit="${pi}"/>
-  <!-- <xacro:ur5_robot prefix="b_bot_" joint_limited="true"
+  <xacro:ur5_robot prefix="b_bot_" joint_limited="true"
     shoulder_pan_lower_limit="${-pi}" shoulder_pan_upper_limit="${pi}"
     shoulder_lift_lower_limit="${-pi}" shoulder_lift_upper_limit="${pi}"
@@ -66,5 +66,5 @@
     wrist_1_lower_limit="${-pi}" wrist_1_upper_limit="${pi}"
     wrist_2_lower_limit="${-pi}" wrist_2_upper_limit="${pi}"
-    wrist_3_lower_limit="${-pi}" wrist_3_upper_limit="${pi}"/> -->
+    wrist_3_lower_limit="${-pi}" wrist_3_upper_limit="${pi}"/>
   <link name="o2as_ground" />
   <joint name="world_a_bot_joint" type="fixed">
@@ -73,5 +73,5 @@
     <origin xyz="${a_bot_x} ${a_bot_y} ${bots_z}" rpy="0.0 0.0 0.0" />
   </joint>
-  <!-- <joint name="world_b_bot_joint" type="fixed">
+  <joint name="world_b_bot_joint" type="fixed">
     <parent link="o2as_ground" />
     <child link = "b_bot_base_link" />
@@ -82,5 +82,5 @@
     <child link = "c_bot_base_link" />
     <origin xyz="${c_bot_x} ${c_bot_y} ${bots_z}" rpy="0.0 0.0 0.0" />
-  </joint> -->
+  </joint>
   <!-- spawn and attach grippers -->
   <xacro:include filename="$(find o2as_scene_description)/urdf/robotiq_85_gripper.urdf.xacro" />
@@ -88,10 +88,10 @@
     <origin xyz="0.0 0 0.0" rpy="0 0 0"/>
   </xacro:robotiq_85_gripper_o2as>
-  <!-- <xacro:robotiq_85_gripper_o2as prefix="b_bot_" parent = "b_bot_ee_link">
+  <xacro:robotiq_85_gripper_o2as prefix="b_bot_" parent = "b_bot_ee_link">
     <origin xyz="0.0 0 0.0" rpy="0 0 0"/>
   </xacro:robotiq_85_gripper_o2as>
   <xacro:robotiq_85_gripper_o2as prefix="c_bot_" parent = "c_bot_ee_link">
     <origin xyz="0.0 0 0.0" rpy="0 0 0"/>
-  </xacro:robotiq_85_gripper_o2as> -->
+  </xacro:robotiq_85_gripper_o2as>
   <!-- I meant to remove the "world" link definition, but apparently it is necessary for Gazebo -->
   <link name="world" />

File: o2as_scene_description/urdf/kitting_scene_1.xacro (robot description, xacro)
@@ -16,16 +16,21 @@
   <xacro:property name="set1_y" value="${.32-bin1_width/2}"/>
   <xacro:property name="set1_z" value=".00" />
+  <!-- set1_bin1_1 -->
   <xacro:kitting_bin_1 binname="set1_bin1_1" parent="workspace_center">
     <origin xyz="${set1_x} ${set1_y} ${set1_z}" rpy="0 0 0" />
   </xacro:kitting_bin_1>
+  <!-- set1_bin1_2 -->
   <xacro:kitting_bin_1 binname="set1_bin1_2" parent="workspace_center">
     <origin xyz="${set1_x} ${set1_y - bin1_width*1} ${set1_z}" rpy="0 0 0" />
   </xacro:kitting_bin_1>
+  <!-- set1_bin1_3 -->
   <xacro:kitting_bin_1 binname="set1_bin1_3" parent="workspace_center">
     <origin xyz="${set1_x} ${set1_y - bin1_width*2} ${set1_z}" rpy="0 0 0" />
   </xacro:kitting_bin_1>
+  <!-- set1_bin1_4 -->
   <xacro:kitting_bin_1 binname="set1_bin1_4" parent="workspace_center">
     <origin xyz="${set1_x} ${set1_y - bin1_width*3} ${set1_z}" rpy="0 0 0" />
   </xacro:kitting_bin_1>
+  <!-- set1_bin1_5 -->
   <xacro:kitting_bin_1 binname="set1_bin1_5" parent="workspace_center">
     <origin xyz="${set1_x} ${set1_y - bin1_width*4} ${set1_z}" rpy="0 0 0" />
@@ -36,16 +41,21 @@
   <xacro:property name="set2_y" value="${.32-bin3_width/2}" />
   <xacro:property name="set2_z" value=".00" />
+  <!-- set2_bin3 -->
   <xacro:kitting_bin_3 binname="set2_bin3" parent="workspace_center">
     <origin xyz="${set2_x_bin3} ${set2_y} ${set2_z}" rpy="0 0 0" />
   </xacro:kitting_bin_3>
+  <!-- set2_bin2_1 -->
   <xacro:kitting_bin_2 binname="set2_bin2_1" parent="workspace_center">
     <origin xyz="${set2_x_bin2} ${set2_y-bin3_width/2-bin2_width/2*1} ${set2_z}" rpy="0 0 0" />
   </xacro:kitting_bin_2>
+  <!-- set2_bin2_2 -->
   <xacro:kitting_bin_2 binname="set2_bin2_2" parent="workspace_center">
     <origin xyz="${set2_x_bin2} ${set2_y-bin3_width/2-bin2_width*3/2} ${set2_z}" rpy="0 0 0" />
   </xacro:kitting_bin_2>
+  <!-- set2_bin2_3 -->
   <xacro:kitting_bin_2 binname="set2_bin2_3" parent="workspace_center">
     <origin xyz="${set2_x_bin2} ${set2_y-bin3_width/2-bin2_width*5/2} ${set2_z}" rpy="0 0 0" />
   </xacro:kitting_bin_2>
+  <!-- set2_bin2_4 -->
   <xacro:kitting_bin_2 binname="set2_bin2_4" parent="workspace_center">
     <origin xyz="${set2_x_bin2} ${set2_y-bin3_width/2-bin2_width*7/2} ${set2_z}" rpy="0 0 0" />
@@ -55,7 +65,9 @@
   <xacro:property name="set3_y" value="${.32-tray_width/2}" />
   <xacro:property name="set3_z" value=".00" />
+  <!-- set3_tray_1 -->
   <xacro:kitting_tray binname="set3_tray_1" parent="workspace_center">
     <origin xyz="${set3_x} ${set3_y} ${set3_z}" rpy="0 0 0" />
   </xacro:kitting_tray>
+  <!-- set3_tray_2 -->
   <xacro:kitting_tray binname="set3_tray_2" parent="workspace_center">
     <origin xyz="${set3_x} ${set3_y-tray_width} ${set3_z}" rpy="0 0 0" />
