Commit message: Add version without namespaces, all in single URDF file
I didn't know how to connect the previous commit to MoveIt, since it's not easy to work with namespaces. Current version spawns in gazebo and will be hopefully easier to integrate into MoveIt.

File: o2as_scene_description/urdf/asm_task_scene.urdf.xacro (robot description, xacro)
@@ -17,6 +17,5 @@
     wrist_1_lower_limit="${-pi}" wrist_1_upper_limit="${pi}"
     wrist_2_lower_limit="${-pi}" wrist_2_upper_limit="${pi}"
-    wrist_3_lower_limit="${-pi}" wrist_3_upper_limit="${pi}"
-  />
+    wrist_3_lower_limit="${-pi}" wrist_3_upper_limit="${pi}"/>
   <xacro:ur5_robot prefix="b_bot_" joint_limited="true"
     shoulder_pan_lower_limit="${-pi}" shoulder_pan_upper_limit="${pi}"
@@ -25,6 +24,5 @@
     wrist_1_lower_limit="${-pi}" wrist_1_upper_limit="${pi}"
     wrist_2_lower_limit="${-pi}" wrist_2_upper_limit="${pi}"
-    wrist_3_lower_limit="${-pi}" wrist_3_upper_limit="${pi}"
-  />
+    wrist_3_lower_limit="${-pi}" wrist_3_upper_limit="${pi}"/>
   <xacro:ur3_robot prefix="c_bot_" joint_limited="true"
     shoulder_pan_lower_limit="${-pi}" shoulder_pan_upper_limit="${pi}"
@@ -33,21 +31,20 @@
     wrist_1_lower_limit="${-pi}" wrist_1_upper_limit="${pi}"
     wrist_2_lower_limit="${-pi}" wrist_2_upper_limit="${pi}"
-    wrist_3_lower_limit="${-pi}" wrist_3_upper_limit="${pi}"
-  />
+    wrist_3_lower_limit="${-pi}" wrist_3_upper_limit="${pi}"/>
   <link name="world" />
-  <joint name="world_joint_A" type="fixed">
+  <joint name="world_a_bot_joint" type="fixed">
     <parent link="world" />
-    <child link = "a_bot_base_link" />
-    <origin xyz="0.0 0.8 0.0" rpy="0.0 0.0 0.0" />
+    <child link="a_bot_base_link" />
+    <origin xyz="0.0 0.5 0.5" rpy="0.0 0.0 0.0" />
   </joint>
-  <joint name="world_joint_B" type="fixed">
+  <joint name="world_b_bot_joint" type="fixed">
     <parent link="world" />
     <child link = "b_bot_base_link" />
-    <origin xyz="0.0 -0.5 0.0" rpy="0.0 0.0 0.0" />
+    <origin xyz="0.0 -0.5 0.5" rpy="0.0 0.0 0.0" />
   </joint>
-  <joint name="world_joint_C" type="fixed">
+  <joint name="world_c_bot_joint" type="fixed">
     <parent link="world" />
     <child link = "c_bot_base_link" />
-    <origin xyz="-0.8 0.0 0.0" rpy="0.0 0.0 0.0" />
+    <origin xyz="-0.5 0.0 0.5" rpy="0.0 0.0 0.0" />
   </joint>
   <!-- attach grippers -->

Commit message: Add robot bases and work plate
The frame "workspace_center" should be used as the main frame of reference. Colors do not work right in Gazebo. Waiting on a response to the issue I posted.

File: o2as_scene_description/urdf/asm_task_scene.urdf.xacro (robot description, xacro)
@@ -2,4 +2,11 @@
 <robot xmlns:xacro="http://ros.org/wiki/xacro"
        name="asm_task_scene" >
+  <xacro:property name="a_bot_x" value="0.0"/>
+  <xacro:property name="a_bot_y" value="0.5"/>
+  <xacro:property name="b_bot_x" value="0.0"/>
+  <xacro:property name="b_bot_y" value="-0.5"/>
+  <xacro:property name="c_bot_x" value="-0.5"/>
+  <xacro:property name="c_bot_y" value="0.0"/>
+  <xacro:property name="bots_z" value="0.75"/>
   <!-- common stuff -->
   <xacro:include filename="$(find ur_description)/urdf/common.gazebo.xacro" />
@@ -10,5 +17,34 @@
   <!-- grippers -->
   <!-- <xacro:include filename="$(find robotiq_c2_model_visualization)/urdf/robotiq_c2_model_macro.xacro" /> -->
-  <!-- arms -->
+  <!-- Scene items (trays, bins...) -->
+  <!-- <xacro:include filename="$(find o2as_scene_description)/urdf/kitting_scene.xacro" /> -->
+  <!-- Robot bases -->
+  <!-- Putting these at height 0.0 makes them intersect with the ground, so they are elevated. -->
+  <!-- There are some instabilities when the box is big, for some reason. -->
+  <xacro:include filename="$(find o2as_scene_description)/urdf/o2as_base.xacro" />
+  <xacro:o2as_base boxname="a_bot_base_smfl">
+    <origin xyz="${a_bot_x-.65/2} ${a_bot_y-.65/2} 0.65" rpy="0 0 0" />
+  </xacro:o2as_base>
+  <xacro:o2as_base boxname="b_bot_base_smfl">
+    <origin xyz="${b_bot_x-.65/2} ${b_bot_y-.65/2} 0.65" rpy="0 0 0" />
+  </xacro:o2as_base>
+  <xacro:o2as_base boxname="c_bot_base_smfl">
+    <origin xyz="${c_bot_x-.65/2-.22} ${c_bot_y-.65/2-.22} 0.65" rpy="0 0 0" />
+  </xacro:o2as_base>
+  <!-- Main workspace -->
+  <!-- The top surface is at 0.01 m below the robot bases. -->
+  <xacro:include filename="$(find o2as_scene_description)/urdf/o2as_box.xacro" />
+  <xacro:property name="plate_w" value="0.8"/>
+  <xacro:property name="plate_l" value="0.8"/>
+  <xacro:o2as_box boxname="workbox" box_w="${plate_w}" box_l="${plate_l}" box_h=".05">
+    <origin xyz="${-plate_w/2} ${-plate_l/2} ${bots_z-.06}" rpy="0 0 0" />
+  </xacro:o2as_box>
+  <link name="workspace_center" />
+  <joint name="world_to_workspace" type="fixed">
+    <parent link="world" />
+    <child link="workspace_center" />
+    <origin xyz="0.0 0.0 ${bots_z}" rpy="0.0 0.0 0.0" />
+  </joint>
+  <!-- robot arms -->
   <xacro:ur10_robot prefix="a_bot_" joint_limited="true"
     shoulder_pan_lower_limit="${-pi}" shoulder_pan_upper_limit="${pi}"
@@ -36,15 +72,15 @@
     <parent link="world" />
     <child link="a_bot_base_link" />
-    <origin xyz="0.0 0.5 0.5" rpy="0.0 0.0 0.0" />
+    <origin xyz="${a_bot_x} ${a_bot_y} ${bots_z}" rpy="0.0 0.0 0.0" />
   </joint>
   <joint name="world_b_bot_joint" type="fixed">
     <parent link="world" />
     <child link = "b_bot_base_link" />
-    <origin xyz="0.0 -0.5 0.5" rpy="0.0 0.0 0.0" />
+    <origin xyz="${b_bot_x} ${b_bot_y} ${bots_z}" rpy="0.0 0.0 0.0" />
   </joint>
   <joint name="world_c_bot_joint" type="fixed">
     <parent link="world" />
     <child link = "c_bot_base_link" />
-    <origin xyz="-0.5 0.0 0.5" rpy="0.0 0.0 0.0" />
+    <origin xyz="${c_bot_x} ${c_bot_y} ${bots_z}" rpy="0.0 0.0 0.0" />
   </joint>
   <!-- attach grippers -->

Commit message: WIP: Add kitting scene
It seems that the mesh files cannot be read. The current version has a UR part instead.

File: o2as_scene_description/urdf/asm_task_scene.urdf.xacro (robot description, xacro)
@@ -9,14 +9,15 @@
   <xacro:property name="c_bot_y" value="0.0"/>
   <xacro:property name="bots_z" value="0.75"/>
+  <!-- This is the main file defining our robot arrangement and physical environment. -->
   <!-- common stuff -->
   <xacro:include filename="$(find ur_description)/urdf/common.gazebo.xacro" />
   <!-- robots -->
-  <xacro:include filename="$(find o2as_scene_description)/urdf/ur3.urdf.xacro" />
   <xacro:include filename="$(find o2as_scene_description)/urdf/ur10.urdf.xacro" />
   <xacro:include filename="$(find o2as_scene_description)/urdf/ur5.urdf.xacro" />
+  <xacro:include filename="$(find o2as_scene_description)/urdf/ur3.urdf.xacro" />
   <!-- grippers -->
   <!-- <xacro:include filename="$(find robotiq_c2_model_visualization)/urdf/robotiq_c2_model_macro.xacro" /> -->
   <!-- Scene items (trays, bins...) -->
-  <!-- <xacro:include filename="$(find o2as_scene_description)/urdf/kitting_scene.xacro" /> -->
+  <xacro:include filename="$(find o2as_scene_description)/urdf/kitting_scene.xacro" />
   <!-- Robot bases -->
   <!-- Putting these at height 0.0 makes them intersect with the ground, so they are elevated. -->

File: o2as_scene_description/urdf/kitting_bin.xacro (robot description, xacro)
@@ -1,5 +1,5 @@
 <?xml version="1.0" ?>
 <robot xmlns:xacro="http://ros.org/wiki/xacro" name="kitting_bin">
-  <xacro:macro name="kitting_bin" params="binname *origin">
+  <xacro:macro name="kitting_bin" params="binname parent *origin">
   <!-- This creates a box with the origin in the bottom corner, connected to the world link. -->
   <xacro:property name="mesh_file" value="$(find o2as_scene_description)/mesh/bin1_EA661CA-11.stl" />
@@ -9,12 +9,13 @@
       <origin rpy="0 0 0" xyz="0 0 0"/>
       <mass value="1.0"/>
-      <inertia ixx="0" ixy="0" ixz="0" iyy="0" iyz="0" izz="0"/>
+      <inertia ixx="1.0" ixy="0" ixz="0" iyy="1.0" iyz="0" izz="1.0"/>
     </inertial>
     <visual>
       <origin rpy="1.5707 0 0" xyz="0 0 0"/>
       <geometry>
-        <mesh filename="${mesh_file}" scale="0.001 0.001 0.001"/>
+        <!-- <mesh filename="${mesh_file}" scale="0.001 0.001 0.001"/> -->
+        <mesh filename="package://ur_description/meshes/ur5/visual/shoulder.dae"/>
       </geometry>
-       <material name="white">
+      <material name="white">
         <color rgba="1 1 1 1"/>
       </material>
@@ -23,10 +24,11 @@
       <origin rpy="1.5707 0 0" xyz="0 0 0"/>
       <geometry>
-        <mesh filename="${mesh_file_col}" scale="0.001 0.001 0.001"/>
+        <!-- <mesh filename="${mesh_file_col}" scale="0.001 0.001 0.001"/> -->
+        <mesh filename="package://ur_description/meshes/ur5/collision/shoulder.stl"/>
       </geometry>
     </collision>
   </link>
   <joint name="${binname}" type="fixed">
-      <parent link="world" />
+      <parent link="${parent}" />
       <child link = "${binname}" />
       <xacro:insert_block name="origin"/>

File: o2as_scene_description/urdf/kitting_scene.xacro (robot description, xacro)
@@ -3,19 +3,33 @@
   <xacro:include filename="$(find o2as_scene_description)/urdf/kitting_bin.xacro" />
   <xacro:property name="bin_width" value=".15"/>
-  <!-- A few arranged bins -->
-  <xacro:property name="set1_x" value=".15"/>
-  <xacro:property name="set1_y" value="0"/>
-  <xacro:property name="set1_z" value=".95"/>
-  <xacro:kitting_bin binname="set1_bin1">
+  <!-- <xacro:include filename="$(find o2as_scene_description)/urdf/o2as_base.xacro" />
+  <xacro:o2as_base boxname="test_bot_base_smfl">
+    <origin xyz="0.0 0.0 0.2" rpy="0 0 0" />
+  </xacro:o2as_base> -->
+  <!-- A row of bins -->
+  <xacro:property name="set1_x" value=".25"/>
+  <xacro:property name="set1_y" value="${-bin_width}"/>
+  <xacro:property name="set1_z" value=".05"/>
+  <xacro:kitting_bin binname="set1_bin1" parent="workspace_center">
     <origin xyz="${set1_x} ${set1_y} ${set1_z}" rpy="0 0 0" />
   </xacro:kitting_bin>
-  <xacro:kitting_bin binname="set1_bin2">
+  <xacro:kitting_bin binname="set1_bin2" parent="workspace_center">
     <origin xyz="${set1_x} ${set1_y + bin_width*1} ${set1_z}" rpy="0 0 0" />
   </xacro:kitting_bin>
-  <xacro:kitting_bin binname="set1_bin3">
+  <xacro:kitting_bin binname="set1_bin3" parent="workspace_center">
     <origin xyz="${set1_x} ${set1_y + bin_width*2} ${set1_z}" rpy="0 0 0" />
   </xacro:kitting_bin>
-  <xacro:property name="set2_x" value=".25"/>
-  <xacro:property name="set2_y" value="0"/>
-  <xacro:property name="set2_z" value=".85"/>
+  <!-- Another row of bins -->
+  <xacro:property name="set2_x" value=".45"/>
+  <xacro:property name="set2_y" value="${-bin_width}"/>
+  <xacro:property name="set2_z" value=".15"/>
+  <xacro:kitting_bin binname="set2_bin1" parent="workspace_center">
+    <origin xyz="${set2_x} ${set2_y} ${set2_z}" rpy="0 0 0" />
+  </xacro:kitting_bin>
+  <xacro:kitting_bin binname="set2_bin2" parent="workspace_center">
+    <origin xyz="${set2_x} ${set2_y + bin_width*1} ${set2_z}" rpy="0 0 0" />
+  </xacro:kitting_bin>
+  <xacro:kitting_bin binname="set2_bin3" parent="workspace_center">
+    <origin xyz="${set2_x} ${set2_y + bin_width*2} ${set2_z}" rpy="0 0 0" />
+  </xacro:kitting_bin>
 </robot>

Commit message: Improvements to MoveIt defaults and kitting setup
Various usability and documentation improvements.

File: o2as_scene_description/urdf/asm_task_scene.urdf.xacro (robot description, xacro)
@@ -34,10 +34,10 @@
   </xacro:o2as_base>
   <!-- Main workspace -->
-  <!-- The top surface is at 0.01 m below the robot bases. -->
+  <!-- The surface is 0.01 m below the robot bases and the "workspace_center" frame. -->
   <xacro:include filename="$(find o2as_scene_description)/urdf/o2as_box.xacro" />
   <xacro:property name="plate_w" value="0.8"/>
   <xacro:property name="plate_l" value="0.8"/>
-  <xacro:o2as_box boxname="workbox" box_w="${plate_w}" box_l="${plate_l}" box_h=".05">
-    <origin xyz="${-plate_w/2} ${-plate_l/2} ${bots_z-.06}" rpy="0 0 0" />
+  <xacro:o2as_box boxname="workbox" box_w="${plate_w}" box_l="${plate_l}" box_h=".01">
+    <origin xyz="${-plate_w/2} ${-plate_l/2} ${bots_z-.02}" rpy="0 0 0" />
   </xacro:o2as_box>
   <link name="workspace_center" />
@@ -51,5 +51,5 @@
     shoulder_pan_lower_limit="${-pi}" shoulder_pan_upper_limit="${pi}"
     shoulder_lift_lower_limit="${-pi}" shoulder_lift_upper_limit="${pi}"
-    elbow_joint_lower_limit="${-pi}" elbow_joint_upper_limit="${pi}"
+    elbow_joint_lower_limit="0.0" elbow_joint_upper_limit="${pi}"
     wrist_1_lower_limit="${-pi}" wrist_1_upper_limit="${pi}"
     wrist_2_lower_limit="${-pi}" wrist_2_upper_limit="${pi}"
@@ -58,5 +58,5 @@
     shoulder_pan_lower_limit="${-pi}" shoulder_pan_upper_limit="${pi}"
     shoulder_lift_lower_limit="${-pi}" shoulder_lift_upper_limit="${pi}"
-    elbow_joint_lower_limit="${-pi}" elbow_joint_upper_limit="${pi}"
+    elbow_joint_lower_limit="0.0" elbow_joint_upper_limit="${pi}"
     wrist_1_lower_limit="${-pi}" wrist_1_upper_limit="${pi}"
     wrist_2_lower_limit="${-pi}" wrist_2_upper_limit="${pi}"
@@ -65,5 +65,5 @@
     shoulder_pan_lower_limit="${-pi}" shoulder_pan_upper_limit="${pi}"
     shoulder_lift_lower_limit="${-pi}" shoulder_lift_upper_limit="${pi}"
-    elbow_joint_lower_limit="${-pi}" elbow_joint_upper_limit="${pi}"
+    elbow_joint_lower_limit="0.0" elbow_joint_upper_limit="${pi}"
     wrist_1_lower_limit="${-pi}" wrist_1_upper_limit="${pi}"
     wrist_2_lower_limit="${-pi}" wrist_2_upper_limit="${pi}"

File: o2as_scene_description/urdf/kitting_scene.xacro (robot description, xacro)
@@ -2,5 +2,5 @@
 <robot xmlns:xacro="http://www.ros.org/wiki/xacro" name="kitting_scene">
   <xacro:include filename="$(find o2as_scene_description)/urdf/kitting_bin.xacro" />
-  <xacro:property name="bin_width" value=".15"/>
+  <xacro:property name="bin_width" value=".13"/>
   <!-- <xacro:include filename="$(find o2as_scene_description)/urdf/o2as_base.xacro" />
   <xacro:o2as_base boxname="test_bot_base_smfl">
@@ -21,7 +21,7 @@
   </xacro:kitting_bin>
   <!-- Another row of bins -->
-  <xacro:property name="set2_x" value=".45"/>
-  <xacro:property name="set2_y" value="${-bin_width}"/>
-  <xacro:property name="set2_z" value=".15"/>
+  <xacro:property name="set2_x" value=".4"/>
+  <xacro:property name="set2_y" value="${-bin_width*3/2}"/>
+  <xacro:property name="set2_z" value=".1"/>
   <xacro:kitting_bin binname="set2_bin1" parent="workspace_center">
     <origin xyz="${set2_x} ${set2_y} ${set2_z}" rpy="0 0 0" />
@@ -33,3 +33,6 @@
     <origin xyz="${set2_x} ${set2_y + bin_width*2} ${set2_z}" rpy="0 0 0" />
   </xacro:kitting_bin>
+  <xacro:kitting_bin binname="set2_bin4" parent="workspace_center">
+    <origin xyz="${set2_x} ${set2_y + bin_width*3} ${set2_z}" rpy="0 0 0" />
+  </xacro:kitting_bin>
 </robot>

Commit message: WIP: Set up gripper. This model does not seem to work.

File: o2as_scene_description/urdf/asm_task_scene.urdf.xacro (robot description, xacro)
@@ -16,6 +16,4 @@
   <xacro:include filename="$(find o2as_scene_description)/urdf/ur5.urdf.xacro" />
   <xacro:include filename="$(find o2as_scene_description)/urdf/ur3.urdf.xacro" />
-  <!-- grippers -->
-  <!-- <xacro:include filename="$(find robotiq_c2_model_visualization)/urdf/robotiq_c2_model_macro.xacro" /> -->
   <!-- Scene items (trays, bins...) -->
   <xacro:include filename="$(find o2as_scene_description)/urdf/kitting_scene.xacro" />
@@ -85,9 +83,11 @@
     <origin xyz="${c_bot_x} ${c_bot_y} ${bots_z}" rpy="0.0 0.0 0.0" />
   </joint>
-  <!-- attach grippers -->
-    <!-- <joint name="a_bot_gripper_link" type="fixed">
-      <origin xyz="0 0 0" rpy="0 0 0" />
-      <parent link="a_bot_tool0" />
-      <child link="a_bot_eef_link" />
-    </joint> -->
+  <!-- spawn and attach grippers -->
+  <xacro:include filename="$(find o2as_scene_description)/urdf/robotiq_c2_model_macro.xacro" />
+  <xacro:robotiq_c2_model prefix="a_bot_"/>
+  <joint name="a_bot_gripper_link" type="fixed">
+    <origin xyz="0 0 0" rpy="0 0 0" />
+    <parent link="a_bot_ee_link" />
+    <child link="a_bot_robotiq_85_adapter_link" />
+  </joint>
 </robot>

Commit message: Add gripper model from CRI repo
Uncommitted change to submodule: Removed openrave dependency. It still works fine.

File: o2as_scene_description/urdf/asm_task_scene.urdf.xacro (robot description, xacro)
@@ -84,10 +84,7 @@
   </joint>
   <!-- spawn and attach grippers -->
-  <xacro:include filename="$(find o2as_scene_description)/urdf/robotiq_c2_model_macro.xacro" />
-  <xacro:robotiq_c2_model prefix="a_bot_"/>
-  <joint name="a_bot_gripper_link" type="fixed">
-    <origin xyz="0 0 0" rpy="0 0 0" />
-    <parent link="a_bot_ee_link" />
-    <child link="a_bot_robotiq_85_adapter_link" />
-  </joint>
+  <xacro:include filename="$(find robotiq_description)/urdf/robotiq_85_gripper.urdf.xacro" />
+  <xacro:robotiq_85_gripper prefix="a_bot_" parent = "a_bot_ee_link">
+    <origin xyz="0.0 0 0.0" rpy="0 0 0"/>
+  </xacro:robotiq_85_gripper>
 </robot>

Commit message: Add 3 grippers, scene colors, o2as_ground link
The o2as_ground_link is now connected to world as a virtual joint in the MoveIt definition to avoid a warning. The colors are properly defined in gazebo and moveit. "Gray" vs "Grey" seems to be bugged in Gazebo.

File: o2as_scene_description/urdf/asm_task_scene.urdf.xacro (robot description, xacro)
@@ -22,11 +22,11 @@
   <!-- There are some instabilities when the box is big, for some reason. -->
   <xacro:include filename="$(find o2as_scene_description)/urdf/o2as_base.xacro" />
-  <xacro:o2as_base boxname="a_bot_base_smfl">
+  <xacro:o2as_base boxname="a_bot_base_smfl" parent="o2as_ground">
     <origin xyz="${a_bot_x-.65/2} ${a_bot_y-.65/2} 0.65" rpy="0 0 0" />
   </xacro:o2as_base>
-  <xacro:o2as_base boxname="b_bot_base_smfl">
+  <xacro:o2as_base boxname="b_bot_base_smfl" parent="o2as_ground">
     <origin xyz="${b_bot_x-.65/2} ${b_bot_y-.65/2} 0.65" rpy="0 0 0" />
   </xacro:o2as_base>
-  <xacro:o2as_base boxname="c_bot_base_smfl">
+  <xacro:o2as_base boxname="c_bot_base_smfl" parent="o2as_ground">
     <origin xyz="${c_bot_x-.65/2-.22} ${c_bot_y-.65/2-.22} 0.65" rpy="0 0 0" />
   </xacro:o2as_base>
@@ -36,15 +36,15 @@
   <xacro:property name="plate_w" value="0.8"/>
   <xacro:property name="plate_l" value="0.8"/>
-  <xacro:o2as_box boxname="workbox" box_w="${plate_w}" box_l="${plate_l}" box_h=".01">
+  <xacro:o2as_box boxname="workbox" box_w="${plate_w}" box_l="${plate_l}" box_h=".01" parent="o2as_ground">
     <origin xyz="${-plate_w/2} ${-plate_l/2} ${bots_z-.02}" rpy="0 0 0" />
   </xacro:o2as_box>
   <link name="workspace_center" />
   <joint name="world_to_workspace" type="fixed">
-    <parent link="world" />
+    <parent link="o2as_ground" />
     <child link="workspace_center" />
     <origin xyz="0.0 0.0 ${bots_z}" rpy="0.0 0.0 0.0" />
   </joint>
   <!-- robot arms -->
-  <xacro:ur10_robot prefix="a_bot_" joint_limited="true"
+  <xacro:ur5_robot prefix="a_bot_" joint_limited="true"
     shoulder_pan_lower_limit="${-pi}" shoulder_pan_upper_limit="${pi}"
     shoulder_lift_lower_limit="${-pi}" shoulder_lift_upper_limit="${pi}"
@@ -67,17 +67,17 @@
     wrist_2_lower_limit="${-pi}" wrist_2_upper_limit="${pi}"
     wrist_3_lower_limit="${-pi}" wrist_3_upper_limit="${pi}"/>
-  <link name="world" />
+  <link name="o2as_ground" />
   <joint name="world_a_bot_joint" type="fixed">
-    <parent link="world" />
+    <parent link="o2as_ground" />
     <child link="a_bot_base_link" />
     <origin xyz="${a_bot_x} ${a_bot_y} ${bots_z}" rpy="0.0 0.0 0.0" />
   </joint>
   <joint name="world_b_bot_joint" type="fixed">
-    <parent link="world" />
+    <parent link="o2as_ground" />
     <child link = "b_bot_base_link" />
     <origin xyz="${b_bot_x} ${b_bot_y} ${bots_z}" rpy="0.0 0.0 0.0" />
   </joint>
   <joint name="world_c_bot_joint" type="fixed">
-    <parent link="world" />
+    <parent link="o2as_ground" />
     <child link = "c_bot_base_link" />
     <origin xyz="${c_bot_x} ${c_bot_y} ${bots_z}" rpy="0.0 0.0 0.0" />
@@ -88,3 +88,16 @@
     <origin xyz="0.0 0 0.0" rpy="0 0 0"/>
   </xacro:robotiq_85_gripper>
+  <xacro:robotiq_85_gripper prefix="b_bot_" parent = "b_bot_ee_link">
+    <origin xyz="0.0 0 0.0" rpy="0 0 0"/>
+  </xacro:robotiq_85_gripper>
+  <xacro:robotiq_85_gripper prefix="c_bot_" parent = "c_bot_ee_link">
+    <origin xyz="0.0 0 0.0" rpy="0 0 0"/>
+  </xacro:robotiq_85_gripper>
+  <!-- I meant to remove the "world" link definition, but apparently it is necessary for Gazebo -->
+  <link name="world" />
+  <joint name="world_o2as_joint" type="fixed">
+    <parent link="world" />
+    <child link="o2as_ground" />
+    <origin xyz="0.0 0.0 0.0" rpy="0.0 0.0 0.0" />
+  </joint>
 </robot>

File: o2as_scene_description/urdf/kitting_bin.xacro (robot description, xacro)
@@ -20,6 +20,6 @@
         <!-- <mesh filename="package://ur_description/meshes/ur5/visual/shoulder.dae"/> -->
       </geometry>
-      <material name="white">
-        <color rgba="1 1 1 1"/>
+      <material name="orange">
+        <color rgba="1 0.5088 0.0468 1"/>
       </material>
     </visual>

File: o2as_scene_description/urdf/o2as_base.xacro (robot description, xacro)
@@ -1,5 +1,5 @@
 <?xml version="1.0"?>
 <robot xmlns:xacro="http://www.ros.org/wiki/xacro" name="o2as_base">
-  <xacro:macro name="o2as_base" params="boxname *origin">
+  <xacro:macro name="o2as_base" params="boxname parent *origin">
     <!-- This creates a box with the origin in the bottom corner, fixed to the world link. -->
     <xacro:property name="box_w" value=".65"/>
@@ -35,5 +35,5 @@
     </gazebo>
     <joint name="${boxname}" type="fixed">
-      <parent link="world" />
+      <parent link="${parent}" />
       <child link = "${boxname}" />
       <xacro:insert_block name="origin"/>

File: o2as_scene_description/urdf/o2as_box.xacro (robot description, xacro)
@@ -1,5 +1,5 @@
 <?xml version="1.0"?>
 <robot xmlns:xacro="http://www.ros.org/wiki/xacro" name="o2as_box">
-  <xacro:macro name="o2as_box" params="boxname box_w box_l box_h *origin">
+  <xacro:macro name="o2as_box" params="boxname box_w box_l box_h parent *origin">
     <!-- This creates a box with the origin in the bottom corner, fixed to the world link. -->
     <link name="${boxname}">
@@ -32,5 +32,5 @@
     </gazebo>
     <joint name="${boxname}" type="fixed">
-      <parent link="world" />
+      <parent link="${parent}" />
       <child link = "${boxname}" />
       <xacro:insert_block name="origin"/>
