Commit message: Add a camera to the scene, update Readme

File: o2as_scene_description/urdf/asm_task_scene.urdf.xacro (robot description, xacro)
@@ -12,4 +12,6 @@
   <!-- common stuff -->
   <xacro:include filename="$(find ur_description)/urdf/common.gazebo.xacro" />
+  <xacro:include filename="$(find o2as_scene_description)/urdf/asm_task_scene.gazebo" />
+  <xacro:include filename="$(find realsense2_camera)/urdf/_r410.urdf.xacro" />
   <!-- robots -->
   <xacro:include filename="$(find o2as_scene_description)/urdf/ur10.urdf.xacro" />
@@ -94,4 +96,14 @@
     <origin xyz="0.0 0 0.0" rpy="0 0 0"/>
   </xacro:robotiq_85_gripper_o2as>
+  <!-- Add cameras -->
+  <link name="b_bot_cam_holder_link" />
+  <joint name="b_bot_cam_holder_joint" type="fixed">
+    <parent link="b_bot_wrist_3_link" />
+    <child link = "b_bot_cam_holder_link" />
+    <origin xyz="0.0 -0.06 0.06" rpy="0.0 0.0 ${pi/2}" />
+  </joint>
+  <xacro:sensor_r410 prefix="b_bot_" parent = "b_bot_cam_holder_link">
+    <origin xyz="0 0.05 0" rpy="0 0 0"/>
+  </xacro:sensor_r410>
   <!-- I meant to remove the "world" link definition, but apparently it is necessary for Gazebo -->
   <link name="world" />

Commit message: Revert duplicated files

File: o2as_scene_description/urdf/asm_task_scene.urdf.xacro (robot description, xacro)
@@ -34,8 +34,8 @@
   <!-- The surface is 0.01 m below the robot bases and the "workspace_center" frame. -->
   <xacro:include filename="$(find o2as_scene_description)/urdf/o2as_box.xacro" />
-  <xacro:property name="plate_w" value="0.8"/>
-  <xacro:property name="plate_l" value="0.8"/>
+  <xacro:property name="plate_w" value="0.84"/>
+  <xacro:property name="plate_l" value="0.62"/>
   <xacro:o2as_box boxname="workbox" box_w="${plate_w}" box_l="${plate_l}" box_h=".01" parent="o2as_ground">
-    <origin xyz="${-plate_w/2} ${-plate_l/2} ${bots_z-.02}" rpy="0 0 0" />
+    <origin xyz="${-plate_w/2} ${-plate_l/2} ${bots_z+.09}" rpy="0 0 0" />
   </xacro:o2as_box>
   <link name="workspace_center" />
@@ -43,5 +43,5 @@
     <parent link="o2as_ground" />
     <child link="workspace_center" />
-    <origin xyz="0.0 0.0 ${bots_z}" rpy="0.0 0.0 0.0" />
+    <origin xyz="0.0 0.0 ${bots_z+.1}" rpy="0.0 0.0 0.0" />
   </joint>
   <!-- robot arms -->

File: o2as_scene_description/urdf/kitting_scene.xacro (robot description, xacro)
@@ -2,38 +2,74 @@
 <robot xmlns:xacro="http://www.ros.org/wiki/xacro" name="kitting_scene">
   <xacro:include filename="$(find o2as_scene_description)/urdf/kitting_bins.xacro" />
-  <xacro:property name="bin_width_1" value=".13"/>
-  <xacro:property name="bin_width_2" value=".12"/>
-  <!-- <xacro:include filename="$(find o2as_scene_description)/urdf/o2as_base.xacro" />
-  <xacro:o2as_base boxname="test_bot_base_smfl">
-    <origin xyz="0.0 0.0 0.2" rpy="0 0 0" />
-  </xacro:o2as_base> -->
-  <!-- A row of bins -->
-  <xacro:property name="set1_x" value=".25"/>
-  <xacro:property name="set1_y" value="${-bin_width_1}"/>
-  <xacro:property name="set1_z" value=".05"/>
-  <xacro:kitting_bin_1 binname="set1_bin1" parent="workspace_center">
+  <xacro:include filename="$(find o2as_scene_description)/urdf/kitting_tray.xacro" />
+  <xacro:property name="bin1_width" value=".125"/>
+  <xacro:property name="bin1_length" value=".128" />
+  <xacro:property name="bin2_width" value=".112" />
+  <xacro:property name="bin2_length" value=".201" />
+  <xacro:property name="bin3_width" value=".192" />
+  <xacro:property name="bin3_length" value=".285" />
+  <xacro:property name="tray_width" value=".300" />
+  <xacro:property name="tray_length" value=".210" />
+  <xacro:property name="rack_width" value=".640" />
+  <!-- A row of bin1 -->
+  <xacro:property name="set1_x" value=".00"/>
+  <xacro:property name="set1_y" value="${.32-bin1_width/2}"/>
+  <xacro:property name="set1_z" value=".00" />
+  <!-- set1_bin1_1 -->
+  <xacro:kitting_bin_1 binname="set1_bin1_1" parent="workspace_center">
     <origin xyz="${set1_x} ${set1_y} ${set1_z}" rpy="0 0 0" />
   </xacro:kitting_bin_1>
-  <xacro:kitting_bin_1 binname="set1_bin2" parent="workspace_center">
-    <origin xyz="${set1_x} ${set1_y + bin_width_1*1} ${set1_z}" rpy="0 0 0" />
+  <!-- set1_bin1_2 -->
+  <xacro:kitting_bin_1 binname="set1_bin1_2" parent="workspace_center">
+    <origin xyz="${set1_x} ${set1_y - bin1_width*1} ${set1_z}" rpy="0 0 0" />
   </xacro:kitting_bin_1>
-  <xacro:kitting_bin_1 binname="set1_bin3" parent="workspace_center">
-    <origin xyz="${set1_x} ${set1_y + bin_width_1*2} ${set1_z}" rpy="0 0 0" />
+  <!-- set1_bin1_3 -->
+  <xacro:kitting_bin_1 binname="set1_bin1_3" parent="workspace_center">
+    <origin xyz="${set1_x} ${set1_y - bin1_width*2} ${set1_z}" rpy="0 0 0" />
   </xacro:kitting_bin_1>
-  <!-- Another row of bins -->
-  <xacro:property name="set2_x" value=".4"/>
-  <xacro:property name="set2_y" value="${-bin_width_2*3/2}"/>
-  <xacro:property name="set2_z" value=".1"/>
-  <xacro:kitting_bin_2 binname="set2_bin1" parent="workspace_center">
-    <origin xyz="${set2_x} ${set2_y} ${set2_z}" rpy="0 0 0" />
+  <!-- set1_bin1_4 -->
+  <xacro:kitting_bin_1 binname="set1_bin1_4" parent="workspace_center">
+    <origin xyz="${set1_x} ${set1_y - bin1_width*3} ${set1_z}" rpy="0 0 0" />
+  </xacro:kitting_bin_1>
+  <!-- set1_bin1_5 -->
+  <xacro:kitting_bin_1 binname="set1_bin1_5" parent="workspace_center">
+    <origin xyz="${set1_x} ${set1_y - bin1_width*4} ${set1_z}" rpy="0 0 0" />
+  </xacro:kitting_bin_1>
+  <!-- A row of bin2 and bin3 -->
+  <xacro:property name="set2_x_bin3" value="${bin1_length/2+bin3_length/2}" />
+  <xacro:property name="set2_x_bin2" value="${bin1_length/2+bin2_length/2}" />
+  <xacro:property name="set2_y" value="${.32-bin3_width/2}" />
+  <xacro:property name="set2_z" value=".00" />
+  <!-- set2_bin3 -->
+  <xacro:kitting_bin_3 binname="set2_bin3" parent="workspace_center">
+    <origin xyz="${set2_x_bin3} ${set2_y} ${set2_z}" rpy="0 0 0" />
+  </xacro:kitting_bin_3>
+  <!-- set2_bin2_1 -->
+  <xacro:kitting_bin_2 binname="set2_bin2_1" parent="workspace_center">
+    <origin xyz="${set2_x_bin2} ${set2_y-bin3_width/2-bin2_width/2*1} ${set2_z}" rpy="0 0 0" />
   </xacro:kitting_bin_2>
-  <xacro:kitting_bin_2 binname="set2_bin2" parent="workspace_center">
-    <origin xyz="${set2_x} ${set2_y + bin_width_2*1} ${set2_z}" rpy="0 0 0" />
+  <!-- set2_bin2_2 -->
+  <xacro:kitting_bin_2 binname="set2_bin2_2" parent="workspace_center">
+    <origin xyz="${set2_x_bin2} ${set2_y-bin3_width/2-bin2_width*3/2} ${set2_z}" rpy="0 0 0" />
   </xacro:kitting_bin_2>
-  <xacro:kitting_bin_2 binname="set2_bin3" parent="workspace_center">
-    <origin xyz="${set2_x} ${set2_y + bin_width_2*2} ${set2_z}" rpy="0 0 0" />
+  <!-- set2_bin2_3 -->
+  <xacro:kitting_bin_2 binname="set2_bin2_3" parent="workspace_center">
+    <origin xyz="${set2_x_bin2} ${set2_y-bin3_width/2-bin2_width*5/2} ${set2_z}" rpy="0 0 0" />
   </xacro:kitting_bin_2>
-  <xacro:kitting_bin_2 binname="set2_bin4" parent="workspace_center">
-    <origin xyz="${set2_x} ${set2_y + bin_width_2*3} ${set2_z}" rpy="0 0 0" />
+  <!-- set2_bin2_4 -->
+  <xacro:kitting_bin_2 binname="set2_bin2_4" parent="workspace_center">
+    <origin xyz="${set2_x_bin2} ${set2_y-bin3_width/2-bin2_width*7/2} ${set2_z}" rpy="0 0 0" />
   </xacro:kitting_bin_2>
+  <!-- A row of tray -->
+  <xacro:property name="set3_x" value="${-(bin1_length/2+tray_length/2)}" />
+  <xacro:property name="set3_y" value="${.32-tray_width/2}" />
+  <xacro:property name="set3_z" value=".00" />
+  <!-- set3_tray_1 -->
+  <xacro:kitting_tray binname="set3_tray_1" parent="workspace_center">
+    <origin xyz="${set3_x} ${set3_y} ${set3_z}" rpy="0 0 0" />
+  </xacro:kitting_tray>
+  <!-- set3_tray_2 -->
+  <xacro:kitting_tray binname="set3_tray_2" parent="workspace_center">
+    <origin xyz="${set3_x} ${set3_y-tray_width} ${set3_z}" rpy="0 0 0" />
+  </xacro:kitting_tray>
 </robot>

Commit message: Change home pose, fix initial Gazebo pose

File: o2as_scene_description/urdf/asm_task_scene.urdf.xacro (robot description, xacro)
@@ -3,7 +3,7 @@
        name="asm_task_scene" >
   <xacro:property name="a_bot_x" value="0.0"/>
-  <xacro:property name="a_bot_y" value="0.5"/>
+  <xacro:property name="a_bot_y" value="-0.5"/>
   <xacro:property name="b_bot_x" value="0.0"/>
-  <xacro:property name="b_bot_y" value="-0.5"/>
+  <xacro:property name="b_bot_y" value="0.5"/>
   <xacro:property name="c_bot_x" value="-0.5"/>
   <xacro:property name="c_bot_y" value="0.0"/>
@@ -76,10 +76,10 @@
     <parent link="o2as_ground" />
     <child link = "b_bot_base_link" />
-    <origin xyz="${b_bot_x} ${b_bot_y} ${bots_z}" rpy="0.0 0.0 0.0" />
+    <origin xyz="${b_bot_x} ${b_bot_y} ${bots_z}" rpy="0.0 0.0 ${-pi}" />
   </joint>
   <joint name="world_c_bot_joint" type="fixed">
     <parent link="o2as_ground" />
     <child link = "c_bot_base_link" />
-    <origin xyz="${c_bot_x} ${c_bot_y} ${bots_z}" rpy="0.0 0.0 0.0" />
+    <origin xyz="${c_bot_x} ${c_bot_y} ${bots_z}" rpy="0.0 0.0 ${-pi/2}" />
   </joint>
   <!-- spawn and attach grippers -->
