Commit message: Cleanup

File: o2as_scene_description/urdf/walls.xacro (robot description, xacro)
@@ -21,15 +21,5 @@
         </geometry>
       </collision>
-      <!-- Tall objects seem to be instable in Gazebo, so we ignore the walls for the physical simulation. -->
-      <!-- <inertial>
-        <mass value="1.0" />
-        <inertia ixx="1.0" ixy="0.0" ixz="0.0"
-          iyy="1.0" iyz="0.0"
-          izz="1.0" />
-      </inertial> -->
     </link>
-    <!-- <gazebo reference="${wall_name}">
-      <material>Gazebo/Brick</material>
-    </gazebo> -->
     <joint name="${wall_name}" type="fixed">
       <parent link="world" />
@@ -39,6 +29,6 @@
   </xacro:macro>
   <!-- ############################# -->
-  <xacro:o2as_wall wall_name="wall_b" wall_w="${wall_width}" wall_l="${wall_thickness}" wall_h="${wall_height}">
-    <origin xyz="0.0 -1.0 0.0" rpy="0.0 0.0 0.0" />
+  <xacro:o2as_wall wall_name="wall_a" wall_w="${wall_width}" wall_l="${wall_thickness}" wall_h="${wall_height}">
+    <origin xyz="0.0 -1.2 0.0" rpy="0.0 0.0 0.0" />
   </xacro:o2as_wall>
   <xacro:o2as_wall wall_name="wall_c" wall_w="${wall_width}" wall_l="${wall_thickness}" wall_h="${wall_height}">
