Commit message: WIP: Change robotiq + screw tip link orientation
This will be reverted, it isn't necessary, just might avoid some conversion when sending commands to the robot.

File: o2as_scene_description/urdf/robotiq_85_gripper.urdf.xacro (robot description, xacro)
@@ -11,7 +11,20 @@
       <parent link="${prefix}robotiq_85_base_link"/>
       <child link="${prefix}robotiq_85_tip_link"/>
-      <origin rpy="0.0 0.0 0.0" xyz=".16 0.0 0.0"/>
+      <origin rpy="${-pi/2} 0.0 ${-pi/2}" xyz=".16 0.0 0.0"/>
     </joint>
     <link name="${prefix}robotiq_85_tip_link"/>
+    <!-- <joint name="${prefix}robotiq_85_m5_screw_tool_tip_joint" type="fixed">
+      <parent link="${prefix}robotiq_85_base_link"/>
+      <child link="${prefix}robotiq_85_m5_screw_tool_tip"/>
+      <origin rpy="${-pi/2} 0.0 ${-pi/2}" xyz=".14 0.0 -0.088"/>
+    </joint>
+    <link name="${prefix}robotiq_85_m5_screw_tool_tip"/> -->
+    <!-- Screw tool tip. Z-axis points along the screw into the hole. -->
+    <joint name="${prefix}robotiq_85_m5_screw_tool_tip_joint" type="fixed">
+      <parent link="${prefix}robotiq_85_tip_link"/>
+      <child link="${prefix}robotiq_85_m5_screw_tool_tip"/>
+      <origin rpy="${-pi/2} 0.0 0.0" xyz="0.0 0.088 -0.02"/>
+    </joint>
+    <link name="${prefix}robotiq_85_m5_screw_tool_tip"/>
   </xacro:macro>
 </robot>

Commit message: Change package name, cleanup

File: o2as_scene_description/urdf/robotiq_85_gripper.urdf.xacro (robot description, xacro)
@@ -8,10 +8,12 @@
         <xacro:insert_block name="origin"/>
     </xacro:robotiq_85_gripper>
+    <!-- Add additional links for us to plan with. Oriented like the UR frame. -->
     <joint name="${prefix}robotiq_85_tip_link_joint" type="fixed">
       <parent link="${prefix}robotiq_85_base_link"/>
       <child link="${prefix}robotiq_85_tip_link"/>
-      <origin rpy="${-pi/2} 0.0 ${-pi/2}" xyz=".16 0.0 0.0"/>
+      <origin rpy="0.0 0.0 0.0" xyz=".16 0.0 0.0"/>
     </joint>
     <link name="${prefix}robotiq_85_tip_link"/>
+    <!-- This orients the joint like the EE link of the robot -->
     <!-- <joint name="${prefix}robotiq_85_m5_screw_tool_tip_joint" type="fixed">
       <parent link="${prefix}robotiq_85_base_link"/>
@@ -23,8 +25,8 @@
     <joint name="${prefix}robotiq_85_m5_screw_tool_tip_joint" type="fixed">
       <parent link="${prefix}robotiq_85_tip_link"/>
-      <child link="${prefix}robotiq_85_m5_screw_tool_tip"/>
-      <origin rpy="${-pi/2} 0.0 0.0" xyz="0.0 0.088 -0.02"/>
+      <child link="${prefix}screw_tool_m5_tip_link"/>
+      <origin rpy="0.0 0.0 0.0" xyz="-0.02 0.0 -0.11 "/>
     </joint>
-    <link name="${prefix}robotiq_85_m5_screw_tool_tip"/>
+    <link name="${prefix}screw_tool_m5_tip_link"/>
   </xacro:macro>
 </robot>

File: o2as_scene_description/urdf/screw_feeder.xacro (robot description, xacro)
@@ -69,4 +69,10 @@
     <xacro:insert_block name="origin"/>
   </joint>
+  <joint name="${feedername}_outlet_joint" type="fixed">
+    <parent link="${feedername}_link"/>
+    <child link="${feedername}_outlet_link"/>
+    <origin rpy="0.0 0.0 0.0" xyz="${length-.01} ${width/2} ${height/2 + .02}"/>
+  </joint>
+  <link name="${feedername}_outlet_link"/>
   </xacro:macro>
 </robot>

Commit message: Comment demo, tune screw tool frame

File: o2as_scene_description/urdf/robotiq_85_gripper.urdf.xacro (robot description, xacro)
@@ -15,16 +15,9 @@
     </joint>
     <link name="${prefix}robotiq_85_tip_link"/>
-    <!-- This orients the joint like the EE link of the robot -->
-    <!-- <joint name="${prefix}robotiq_85_m5_screw_tool_tip_joint" type="fixed">
-      <parent link="${prefix}robotiq_85_base_link"/>
-      <child link="${prefix}robotiq_85_m5_screw_tool_tip"/>
-      <origin rpy="${-pi/2} 0.0 ${-pi/2}" xyz=".14 0.0 -0.088"/>
-    </joint>
-    <link name="${prefix}robotiq_85_m5_screw_tool_tip"/> -->
     <!-- Screw tool tip. Z-axis points along the screw into the hole. -->
     <joint name="${prefix}robotiq_85_m5_screw_tool_tip_joint" type="fixed">
       <parent link="${prefix}robotiq_85_tip_link"/>
       <child link="${prefix}screw_tool_m5_tip_link"/>
-      <origin rpy="0.0 0.0 0.0" xyz="-0.02 0.0 -0.11 "/>
+      <origin rpy="0.0 0.0 0.0" xyz="-0.03 0.0 -0.12 "/>
     </joint>
     <link name="${prefix}screw_tool_m5_tip_link"/>
