Commit message: Fix collisions, add gripper to moveit_config

File: o2as_scene_description/urdf/combined_gripper.xacro (robot description, xacro)
@@ -12,23 +12,28 @@
       <geometry>
         <mesh filename="${mesh_file}" scale="1 1 1"/>
-        <!-- <mesh filename="package://ur_description/meshes/ur5/visual/shoulder.dae"/> -->
       </geometry>
-      <material name="red">
-        <color rgba="1 0.5 0.5 1"/>
-      </material>
+        <material name="darkgrey">
+          <color rgba="0.1 0.1 0.1 1"/>
+        </material>
     </visual>
     <collision>
-      <origin rpy="0 0 0" xyz="0 0 0"/>
+      <origin rpy="0 0 0" xyz="-0.175 0 0"/>
       <geometry>
-        <mesh filename="${mesh_file}" scale="1 1 1"/>
-        <!-- <mesh filename="package://ur_description/meshes/ur5/collision/shoulder.stl"/> -->
+        <box size="0.35 0.15 0.1"/>
       </geometry>
     </collision>
   </link>
   <joint name="${prefix}${grippername}" type="fixed">
-      <parent link="${parent}" />
-      <child link = "${prefix}${grippername}" />
-      <xacro:insert_block name="origin"/>
-    </joint>
+    <parent link="${parent}" />
+    <child link = "${prefix}${grippername}" />
+    <xacro:insert_block name="origin"/>
+  </joint>
+  <!-- Add additional links for us to plan with.-->
+  <joint name="${prefix}${grippername}_tip_link_joint" type="fixed">
+    <parent link="${parent}"/>
+    <child link="${prefix}${grippername}_tip_link"/>
+    <origin rpy="0.0 ${-pi/2} 0.0" xyz="0.0 0.0 .35"/>
+  </joint>
+  <link name="${prefix}${grippername}_tip_link"/>
   </xacro:macro>
 </robot>
