Commit message: Finish taskboard & placement mat URDF

File: o2as_scene_description/urdf/kitting_tray.xacro (robot description, xacro)
@@ -16,5 +16,4 @@
       <geometry>
         <mesh filename="${mesh_file}" scale="0.001 0.001 0.001"/>
-        <!-- <mesh filename="package://ur_description/meshes/ur5/visual/shoulder.dae"/> -->
       </geometry>
       <material name="white">
@@ -26,5 +25,4 @@
       <geometry>
         <mesh filename="${mesh_file_col}" scale="0.001 0.001 0.001"/>
-        <!-- <mesh filename="package://ur_description/meshes/ur5/collision/shoulder.stl"/> -->
       </geometry>
     </collision>

File: o2as_scene_description/urdf/o2as_mat.xacro (robot description, xacro)
@@ -15,12 +15,40 @@
       </visual>
       <visual>
-        <origin xyz="${mat_w/2} ${mat_l/2} ${mat_h/2}+.0001" rpy="0 0 0"/>
+        <origin xyz="${mat_w-.01} ${mat_l/2} ${mat_h}" rpy="0 0 ${pi/2}"/>
         <geometry>
-          <box size="${mat_w} ${mat_l} ${mat_h}"/>
+          <box size=".38 .002 ${mat_h}"/>
         </geometry>
-        <material name="white">
-          <color rgba="1 1 1 1"/>
+        <material name="black">
+          <color rgba=".1 .1 .1 1"/>
         </material>
       </visual>
+      <visual>
+        <origin xyz=".01 ${mat_l/2} ${mat_h}" rpy="0 0 ${pi/2}"/>
+        <geometry>
+          <box size=".38 .002 ${mat_h}"/>
+        </geometry>
+        <material name="black">
+          <color rgba=".1 .1 .1 1"/>
+        </material>
+      </visual>
+      <visual>
+        <origin xyz="${mat_w/2} ${mat_l-.01} ${mat_h}" rpy="0 0 0"/>
+        <geometry>
+          <box size=".38 .002 ${mat_h}"/>
+        </geometry>
+        <material name="black">
+          <color rgba=".1 .1 .1 1"/>
+        </material>
+      </visual>
+      <visual>
+        <origin xyz="${mat_w/2} .01 ${mat_h}" rpy="0 0 0"/>
+        <geometry>
+          <box size=".38 .002 ${mat_h}"/>
+        </geometry>
+        <material name="black">
+          <color rgba=".1 .1 .1 1"/>
+        </material>
+      </visual>
+      <!-- Done with boundary drawing -->
       <collision>
         <geometry>

File: o2as_scene_description/urdf/task_board.xacro (robot description, xacro)
@@ -64,6 +64,14 @@
     <origin rpy="0.0 0.0 ${pi/2}" xyz="0.07 0.26 0.0045"/>
   </joint>
-  <link name="${boardname}_part5"/>
-  <!--  -->
+  <link name="${boardname}_part5">
+    <visual>
+      <origin xyz="0 0 -.00275" rpy="0 0 0"/>
+      <geometry>
+        <cylinder length=".0045" radius=".002"/>
+      </geometry>
+      <material name="grey"/>
+    </visual>
+  </link>
+  <!-- The pulleys for the belt -->
   <joint name="${boardname}_part6_small_pulley" type="fixed">
     <parent link="${boardname}_surface"/>
@@ -71,5 +79,13 @@
     <origin rpy="0.0 0.0 ${pi/2}" xyz="0.06 0.06 0.0085"/>
   </joint>
-  <link name="${boardname}_part6_small_pulley"/>
+  <link name="${boardname}_part6_small_pulley">
+    <visual>
+      <origin xyz="0 0 -.00475" rpy="0 0 0"/>
+      <geometry>
+        <cylinder length=".0085" radius=".016"/>
+      </geometry>
+      <material name="grey"/>
+    </visual>
+  </link>
   <joint name="${boardname}_part6_large_pulley" type="fixed">
     <parent link="${boardname}_surface"/>
@@ -77,7 +93,15 @@
     <origin rpy="0.0 0.0 ${pi/2}" xyz="0.188 0.06 0.0085"/>
   </joint>
-  <link name="${boardname}_part6_large_pulley"/>
-  <!--  -->
-  <!--  -->
+  <link name="${boardname}_part6_large_pulley">
+    <visual>
+      <origin xyz="0 0 -.00475" rpy="0 0 0"/>
+      <geometry>
+        <cylinder length=".0085" radius=".031"/>
+      </geometry>
+      <material name="grey"/>
+    </visual>
+  </link>
+  <!-- ======== -->
+  <!-- The nut and bolt on the metal sheet -->
   <joint name="${boardname}_part7a" type="fixed">
     <parent link="${boardname}_surface"/>
@@ -91,6 +115,14 @@
     <origin rpy="0.0 0.0 ${pi/2}" xyz="0.338 0.056 0.05"/>
   </joint>
-  <link name="${boardname}_part7b"/>
-  <!--  -->
+  <link name="${boardname}_part7b">
+    <visual>
+      <origin xyz="0 0.0015 -.015" rpy="0 0 0"/>
+      <geometry>
+        <box size=".015 0.003 .07"/>
+      </geometry>
+      <material name="grey"/>
+    </visual>
+  </link>
+  <!-- ======== -->
   <joint name="${boardname}_part8" type="fixed">
     <parent link="${boardname}_surface"/>
@@ -98,5 +130,13 @@
     <origin rpy="0.0 0.0 ${pi/2}" xyz="0.32 0.25 0.012"/>
   </joint>
-  <link name="${boardname}_part8"/>
+  <link name="${boardname}_part8">
+    <visual>
+      <origin xyz="0 0 -.006" rpy="0 0 0"/>
+      <geometry>
+        <cylinder length=".012" radius=".006"/>
+      </geometry>
+      <material name="grey"/>
+    </visual>
+  </link>
   <joint name="${boardname}_part9" type="fixed">
     <parent link="${boardname}_surface"/>
@@ -104,5 +144,13 @@
     <origin rpy="0.0 0.0 ${pi/2}" xyz="0.26 0.15 0.009"/>
   </joint>
-  <link name="${boardname}_part9"/>
+  <link name="${boardname}_part9">
+    <visual>
+      <origin xyz="0 0 -.0045" rpy="0 0 0"/>
+      <geometry>
+        <cylinder length=".009" radius=".0032"/>
+      </geometry>
+      <material name="grey"/>
+    </visual>
+  </link>
   <joint name="${boardname}_part10" type="fixed">
     <parent link="${boardname}_surface"/>
@@ -110,5 +158,13 @@
     <origin rpy="0.0 0.0 ${pi/2}" xyz="0.16 0.36 0.05"/>
   </joint>
-  <link name="${boardname}_part10"/>
+  <link name="${boardname}_part10">
+    <visual>
+      <origin xyz="0 0 -.025" rpy="0 0 0"/>
+      <geometry>
+        <cylinder length=".05" radius=".003"/>
+      </geometry>
+      <material name="grey"/>
+    </visual>
+  </link>
   <joint name="${boardname}_part11" type="fixed">
     <parent link="${boardname}_surface"/>
@@ -134,5 +190,13 @@
     <origin rpy="0.0 0.0 ${pi/2}" xyz="0.23 0.23 0.05"/>
   </joint>
-  <link name="${boardname}_part14"/>
+  <link name="${boardname}_part14">
+    <visual>
+      <origin xyz="0 0 -.025" rpy="0 0 0"/>
+      <geometry>
+        <cylinder length=".05" radius=".003"/>
+      </geometry>
+      <material name="grey"/>
+    </visual>
+  </link>
   <joint name="${boardname}_part15" type="fixed">
     <parent link="${boardname}_surface"/>
@@ -141,4 +205,5 @@
   </joint>
   <link name="${boardname}_part15"/>
+   <!-- The cylinder is already defined under part10 -->
   <joint name="${boardname}_corner1" type="fixed">
     <parent link="${boardname}_surface"/>
