Commit message: Fix gripper frame z-coordinate

File: o2as_scene_description/urdf/precision_gripper.xacro (robot description, xacro)
@@ -45,5 +45,5 @@
     <!-- Front part -->
     <collision>
-      <origin rpy="0 ${pi/2} 0" xyz="-0.16 0 0"/>
+      <origin rpy="0 ${pi/2} 0" xyz="-0.14 0 0"/>
       <geometry>
         <box size=".1 .08 .07"/>
@@ -60,5 +60,5 @@
     <parent link="${parent}"/>
     <child link="${prefix}${grippername}_tip_link"/>
-    <origin rpy="0.0 ${-pi/2} 0.0" xyz="0.0 0.0 .24"/>
+    <origin rpy="0.0 ${-pi/2} 0.0" xyz="0.0 0.0 .233"/>
   </joint>
   <link name="${prefix}${grippername}_tip_link"/>

Commit message: Set recalibrated gripper frame

File: o2as_scene_description/urdf/precision_gripper.xacro (robot description, xacro)
@@ -60,5 +60,6 @@
     <parent link="${parent}"/>
     <child link="${prefix}${grippername}_tip_link"/>
-    <origin rpy="0.0 ${-pi/2} 0.0" xyz="0.0 0.0 .233"/>
+    <!-- Hand-calibrated values from 14 August 2018 @ OSX (not very precise) -->
+    <origin rpy="0.0 ${-pi/2} 0.0" xyz="0.005 -0.003 .233"/>
   </joint>
   <link name="${prefix}${grippername}_tip_link"/>

Commit message: Update MoveIt config etc.

File: o2as_scene_description/urdf/precision_gripper.xacro (robot description, xacro)
@@ -18,13 +18,4 @@
     </visual>
     <!-- <visual>
-      <origin rpy="0 ${pi/2} 0" xyz="-0.16 0 0"/>
-      <geometry>
-        <box size=".1 .08 .07"/>
-      </geometry>
-      <material name="cyan2">
-        <color rgba="0.3 0.5 0.5 0.3"/>
-      </material>
-    </visual>
-    <visual>
       <origin rpy="0 ${pi/2} 0" xyz="-0.05 0 0"/>
       <geometry>
@@ -33,4 +24,13 @@
       <material name="green2">
         <color rgba="0.1 0.8 0.1 0.3"/>
+      </material>
+    </visual>
+    <visual>
+      <origin rpy="0 ${pi/2} 0" xyz="-0.14 0 0"/>
+      <geometry>
+        <box size=".1 .08 .07"/>
+      </geometry>
+      <material name="cyan2">
+        <color rgba="0.3 0.5 0.5 0.3"/>
       </material>
     </visual> -->

File: o2as_scene_description/urdf/task_board.xacro (robot description, xacro)
@@ -70,5 +70,7 @@
         <cylinder length=".0045" radius=".002"/>
       </geometry>
-      <material name="grey"/>
+      <material name="grey">
+        <color rgba=".3 .3 .3 1"/>
+      </material>
     </visual>
   </link>
@@ -85,5 +87,7 @@
         <cylinder length=".0085" radius=".016"/>
       </geometry>
-      <material name="grey"/>
+      <material name="grey">
+        <color rgba=".3 .3 .3 1"/>
+      </material>
     </visual>
   </link>
@@ -99,5 +103,7 @@
         <cylinder length=".0085" radius=".031"/>
       </geometry>
-      <material name="grey"/>
+      <material name="grey">
+        <color rgba=".3 .3 .3 1"/>
+      </material>
     </visual>
   </link>
@@ -121,5 +127,7 @@
         <box size=".015 0.003 .07"/>
       </geometry>
-      <material name="grey"/>
+      <material name="grey">
+        <color rgba=".3 .3 .3 1"/>
+      </material>
     </visual>
   </link>
@@ -136,5 +144,7 @@
         <cylinder length=".012" radius=".006"/>
       </geometry>
-      <material name="grey"/>
+      <material name="grey">
+        <color rgba=".3 .3 .3 1"/>
+      </material>
     </visual>
   </link>
@@ -150,5 +160,7 @@
         <cylinder length=".009" radius=".0032"/>
       </geometry>
-      <material name="grey"/>
+      <material name="grey">
+        <color rgba=".3 .3 .3 1"/>
+      </material>
     </visual>
   </link>
@@ -164,5 +176,7 @@
         <cylinder length=".05" radius=".003"/>
       </geometry>
-      <material name="grey"/>
+      <material name="grey">
+        <color rgba=".3 .3 .3 1"/>
+      </material>
     </visual>
   </link>
@@ -196,5 +210,7 @@
         <cylinder length=".05" radius=".003"/>
       </geometry>
-      <material name="grey"/>
+      <material name="grey">
+        <color rgba=".3 .3 .3 1"/>
+      </material>
     </visual>
   </link>

Commit message: Fix precision gripper driver & params

File: o2as_scene_description/urdf/precision_gripper.xacro (robot description, xacro)
@@ -61,5 +61,5 @@
     <child link="${prefix}${grippername}_tip_link"/>
     <!-- Hand-calibrated values from 14 August 2018 @ OSX (not very precise) -->
-    <origin rpy="0.0 ${-pi/2} 0.0" xyz="0.005 -0.003 .233"/>
+    <origin rpy="0.0 ${-pi/2} 0.0" xyz="0.0025 -0.002 .235"/>
   </joint>
   <link name="${prefix}${grippername}_tip_link"/>
