Commit message: finished test scene in Osaka

File: o2as_scene_description/urdf/o2as_osakabase_scene.urdf.xacro (robot description, xacro)
@@ -27,13 +27,13 @@
   <!-- Putting these at height 0.0 makes them intersect with the ground, so they are elevated. -->
   <!-- There are some instabilities when the box is big, for some reason. -->
-  <xacro:include filename="$(find o2as_scene_description)/urdf/o2as_base.xacro" />
+  <xacro:include filename="$(find o2as_scene_description)/urdf/o2as_osakabase.xacro" />
   <xacro:o2as_base boxname="a_bot_base_smfl" parent="o2as_ground">
-    <origin xyz="${a_bot_x-.65/2} ${a_bot_y-.65/2} ${bots_z-.06}" rpy="0 0 0" />
+    <origin xyz="${a_bot_x-.4/2} ${a_bot_y-.4/2} ${bots_z-.06}" rpy="0 0 0" />
   </xacro:o2as_base>
   <xacro:o2as_base boxname="b_bot_base_smfl" parent="o2as_ground">
-    <origin xyz="${b_bot_x-.65/2} ${b_bot_y-.65/2} ${bots_z-.06}" rpy="0 0 0" />
+    <origin xyz="${b_bot_x-.4/2} ${b_bot_y-.4/2} ${bots_z-.06}" rpy="0 0 0" />
   </xacro:o2as_base>
   <xacro:o2as_base boxname="c_bot_base_smfl" parent="o2as_ground">
-    <origin xyz="${c_bot_x-.65/2-.16} ${c_bot_y-.65/2-.1} ${bots_z-.06}" rpy="0 0 0" />
+    <origin xyz="${c_bot_x-.4/2-.16} ${c_bot_y-.4/2-.1} ${bots_z-.06}" rpy="0 0 0" />
   </xacro:o2as_base>
   <!-- Main workspace -->
@@ -43,5 +43,5 @@
   <xacro:property name="plate_l" value="0.75"/>
   <xacro:o2as_box boxname="workbox" box_w="${plate_w}" box_l="${plate_l}" box_h=".01" parent="o2as_ground">
-    <origin xyz="${-plate_w/2+.1} ${-plate_l/2} ${bots_z}" rpy="0 0 0" />
+    <origin xyz="${-plate_w/2+.1} ${-plate_l/2} ${bots_z-0.196}" rpy="0 0 0" />
   </xacro:o2as_box>
   <link name="workspace_center" />
@@ -49,8 +49,8 @@
     <parent link="o2as_ground" />
     <child link="workspace_center" />
-    <origin xyz="0.0 0.0 ${bots_z+.01}" rpy="0.0 0.0 0.0" />
+    <origin xyz="0.0 0.0 ${bots_z+.01-0.196}" rpy="0.0 0.0 0.0" />
   </joint>
   <!-- Screw holder & screw tool visual -->
-  <xacro:include filename="$(find o2as_scene_description)/urdf/screw_tools.xacro" />
+  <!-- <xacro:include filename="$(find o2as_scene_description)/urdf/screw_tools.xacro" /> -->
   <!-- Feeders -->
   <!-- <xacro:include filename="$(find o2as_scene_description)/urdf/screw_feeder.xacro" />

Commit message: add taskboard seq for part1 and part6

File: o2as_scene_description/urdf/o2as_osakabase_scene.urdf.xacro (robot description, xacro)
@@ -21,6 +21,6 @@
   <xacro:include filename="$(find o2as_scene_description)/urdf/ur3.urdf.xacro" />
   <!-- Scene items (trays, bins...) -->
-  <xacro:include filename="$(find o2as_scene_description)/urdf/taskboard_scene.xacro" />
-  <!-- <xacro:include filename="$(find o2as_scene_description)/urdf/kitting_scene.xacro" /> -->
+  <!-- <xacro:include filename="$(find o2as_scene_description)/urdf/taskboard_scene.xacro" /> -->
+  <xacro:include filename="$(find o2as_scene_description)/urdf/kitting_scene.xacro" />
   <!-- <xacro:include filename="$(find o2as_scene_description)/urdf/assembly_scene.xacro" /> -->
   <!-- Robot bases -->

File: o2as_scene_description/urdf/task_board.xacro (robot description, xacro)
@@ -41,4 +41,10 @@
   </joint>
   <link name="${boardname}_part1"/>
+  <joint name="${boardname}_tool" type="fixed">
+    <parent link="${boardname}_surface"/>
+    <child link="${boardname}_tool"/>
+    <origin rpy="0.0 0.0 ${pi/2}" xyz="-0.07 0.0 -0.02"/>
+  </joint>
+  <link name="${boardname}_tool"/>
   <joint name="${boardname}_part2" type="fixed">
     <parent link="${boardname}_surface"/>
