Commit message: Modify M5 screw tool for M3,M4,M6 and collision judgment

File: o2as_scene_description/urdf/robotiq_85_gripper_with_ft300.urdf.xacro (robot description, xacro)
@@ -36,8 +36,8 @@
     <joint name="${prefix}robotiq_85_m5_screw_tool_tip_joint" type="fixed">
       <parent link="${prefix}robotiq_85_tip_link"/>
-      <child link="${prefix}screw_tool_m5_tip_link"/>
+      <child link="${prefix}screw_tool_m6_tip_link"/>
       <origin rpy="0.0 0.0 0.0" xyz="-0.03 0.0 -0.12 "/>
     </joint>
-    <link name="${prefix}screw_tool_m5_tip_link"/>
+    <link name="${prefix}screw_tool_m6_tip_link"/>
   </xacro:macro>
 </robot>

File: o2as_scene_description/urdf/screw_tools.xacro (robot description, xacro)
@@ -29,5 +29,5 @@
   </joint>
   <!-- ++++++++++++++++++++++++++++ -->
-  <link name="screw_tool_m5_link">
+ <link name="screw_tool_m6_link">
     <inertial>
       <origin rpy="0 0 0" xyz="0 0 0"/>
@@ -38,5 +38,5 @@
       <origin rpy="0 0 0" xyz="0 0 0"/>
       <geometry>
-        <mesh filename="package://o2as_scene_description/meshes/screw_tool_m5_BC5-XL320-00.stl" scale="0.001 0.001 0.001"/>
+        <mesh filename="package://o2as_scene_description/meshes/screw_tool_m6_BC5-XL320-LG20-R_v2.stl" scale="0.001 0.001 0.001"/>
       </geometry>
       <material name="white">
@@ -51,7 +51,7 @@
     </collision>
   </link>
-  <joint name="screw_tool_m5_to_holder" type="fixed">
+  <joint name="screw_tool_m6_to_holder" type="fixed">
     <parent link="screw_tool_holder" />
-    <child link="screw_tool_m5_link" />
+    <child link="screw_tool_m6_link" />
     <origin xyz="0.1 0.0 0.0" rpy="0.0 0.0 0.0" />
   </joint>
@@ -65,5 +65,5 @@
       <origin rpy="0 0 0" xyz="0 0 0"/>
       <geometry>
-        <mesh filename="package://o2as_scene_description/meshes/screw_tool_m5_BC5-XL320-00.stl" scale="0.001 0.001 0.001"/>
+        <mesh filename="package://o2as_scene_description/meshes/screw_tool_m4_BC5-XL320-AY3.5-EH3R4.stl" scale="0.001 0.001 0.001"/>
       </geometry>
       <material name="white">
@@ -92,5 +92,5 @@
       <origin rpy="0 0 0" xyz="0 0 0"/>
       <geometry>
-        <mesh filename="package://o2as_scene_description/meshes/screw_tool_m5_BC5-XL320-00.stl" scale="0.001 0.001 0.001"/>
+        <mesh filename="package://o2as_scene_description/meshes/screw_tool_m3_BC5-XL320-R-AY2.6-EH2.stl" scale="0.001 0.001 0.001"/>
       </geometry>
       <material name="white">
@@ -123,8 +123,8 @@
     <origin xyz="0.0 0.0 0.0" rpy="0.0 0.0 ${-pi/2}" />
   </joint>
-  <link name="screw_tool_m5_helper_link"/>
-  <joint name="screw_tool_m5_helper_joint" type="fixed">
-    <parent link="screw_tool_m5_link" />
-    <child link="screw_tool_m5_helper_link" />
+  <link name="screw_tool_m6_helper_link"/>
+  <joint name="screw_tool_m6_helper_joint" type="fixed">
+    <parent link="screw_tool_m6_link" />
+    <child link="screw_tool_m6_helper_link" />
     <origin xyz="0.0 0.0 0.0" rpy="0.0 0.0 ${-pi/2}" />
   </joint>

Commit message: WIP: Cartesian path time parametrization

File: o2as_scene_description/urdf/robotiq_85_gripper_with_ft300.urdf.xacro (robot description, xacro)
@@ -35,11 +35,23 @@
     </joint>
     <link name="${prefix}robotiq_85_tip_link"/>
-    <!-- Screw tool tip. Z-axis points along the screw into the hole. -->
-    <joint name="${prefix}robotiq_85_m5_screw_tool_tip_joint" type="fixed">
+    <!-- Screw tool tips. X-axis points along the screw into the hole. -->
+    <joint name="${prefix}robotiq_85_m6_screw_tool_tip_joint" type="fixed">
       <parent link="${prefix}robotiq_85_tip_link"/>
       <child link="${prefix}screw_tool_m6_tip_link"/>
-      <origin rpy="0.0 0.0 0.0" xyz="-0.03 0.0 -0.12 "/>
+      <origin rpy="0.0 ${pi/2} 0.0" xyz="-0.03 0.0 -0.12 "/>
     </joint>
     <link name="${prefix}screw_tool_m6_tip_link"/>
+    <joint name="${prefix}robotiq_85_m4_screw_tool_tip_joint" type="fixed">
+      <parent link="${prefix}robotiq_85_tip_link"/>
+      <child link="${prefix}screw_tool_m4_tip_link"/>
+      <origin rpy="0.0 ${pi/2} 0.0" xyz="-0.03 0.0 -0.13 "/>
+    </joint>
+    <link name="${prefix}screw_tool_m4_tip_link"/>
+    <joint name="${prefix}robotiq_85_m3_screw_tool_tip_joint" type="fixed">
+      <parent link="${prefix}robotiq_85_tip_link"/>
+      <child link="${prefix}screw_tool_m3_tip_link"/>
+      <origin rpy="0.0 ${pi/2} 0.0" xyz="-0.03 0.0 -0.112 "/>
+    </joint>
+    <link name="${prefix}screw_tool_m3_tip_link"/>
   </xacro:macro>
 </robot>

File: o2as_scene_description/urdf/screw_tools.xacro (robot description, xacro)
@@ -44,10 +44,10 @@
       </material>
     </visual>
-    <collision>
+    <!-- <collision>
       <origin rpy="0 0 -.225" xyz="0 0 0"/>
       <geometry>
         <box size=".02 .04 .155"/>
       </geometry>
-    </collision>
+    </collision> -->
   </link>
   <joint name="screw_tool_m6_to_holder" type="fixed">
@@ -71,10 +71,10 @@
       </material>
     </visual>
-    <collision>
+    <!-- <collision>
       <origin rpy="0 0 -.225" xyz="0 0 0"/>
       <geometry>
         <box size=".02 .04 .155"/>
       </geometry>
-    </collision>
+    </collision> -->
   </link>
   <joint name="screw_tool_m4_to_holder" type="fixed">
@@ -98,10 +98,10 @@
       </material>
     </visual>
-    <collision>
+    <!-- <collision>
       <origin rpy="0 0 -.225" xyz="0 0 0"/>
       <geometry>
         <box size=".02 .04 .155"/>
       </geometry>
-    </collision>
+    </collision> -->
   </link>
   <joint name="screw_tool_m3_to_holder" type="fixed">
