Commit message: Fix incorrect collision box of robot bases

File: o2as_scene_description/urdf/o2as_base.xacro (robot description, xacro)
@@ -14,8 +14,9 @@
         </geometry>
         <material name="DarkGrey">
-          <color rgba="0.2 0.2 0.2 1.0"/>
+          <color rgba="0.4 0.4 0.4 1.0"/>
         </material>
       </visual>
       <collision>
+        <origin xyz="${box_w/2} ${box_l/2} ${box_h/2}" rpy="0 0 0"/>
         <geometry>
           <box size="${box_w} ${box_l} ${box_h}"/>

File: o2as_scene_description/urdf/o2as_box.xacro (robot description, xacro)
@@ -15,4 +15,5 @@
       </visual>
       <collision>
+        <origin xyz="${box_w/2} ${box_l/2} ${box_h/2}" rpy="0 0 0"/>
         <geometry>
           <box size="${box_w} ${box_l} ${box_h}"/>

Commit message: Clean up

File: o2as_scene_description/urdf/o2as_base.xacro (robot description, xacro)
@@ -1,4 +1,4 @@
 <?xml version="1.0"?>
-<robot xmlns:xacro="http://www.ros.org/wiki/xacro" name="o2as_base">
+<robot xmlns:xacro="http://www.ros.org/wiki/xacro">
   <xacro:macro name="o2as_base" params="boxname parent *origin">
     <!-- This creates a box with the origin in the bottom corner, fixed to the world link. -->

File: o2as_scene_description/urdf/o2as_base_scene.urdf.xacro (robot description, xacro)
@@ -1,4 +1,4 @@
 <?xml version="1.0"?>
-<robot xmlns:xacro="http://ros.org/wiki/xacro"
+<robot xmlns:xacro="http://www.ros.org/wiki/xacro"
        name="o2as_base_scene" >
   <!-- Calibration from 20 August 2018 -->

File: o2as_scene_description/urdf/o2as_box.xacro (robot description, xacro)
@@ -1,4 +1,4 @@
 <?xml version="1.0"?>
-<robot xmlns:xacro="http://www.ros.org/wiki/xacro" name="o2as_box">
+<robot xmlns:xacro="http://www.ros.org/wiki/xacro">
   <xacro:macro name="o2as_box" params="boxname box_w box_l box_h parent *origin">
     <!-- This creates a box with the origin in the bottom corner, fixed to the world link. -->

File: o2as_scene_description/urdf/o2as_osaka_scene.urdf.xacro (robot description, xacro)
@@ -1,4 +1,4 @@
 <?xml version="1.0"?>
-<robot xmlns:xacro="http://ros.org/wiki/xacro"
+<robot xmlns:xacro="http://www.ros.org/wiki/xacro"
        name="o2as_base_scene" >
   <!-- This is the main file defining our robot arrangement and physical environment. -->

File: o2as_scene_description/urdf/phoxi_m_camera.urdf.xacro (robot description, xacro)
@@ -1,4 +1,4 @@
 <?xml version="1.0"?>
-<robot name="phoxi_m_camera" xmlns:xacro="http://ros.org/wiki/xacro">
+<robot name="phoxi_m_camera" xmlns:xacro="http://www.ros.org/wiki/xacro">
   <xacro:macro name="phoxi_m_camera" params="prefix parent *origin">
     <xacro:include filename="$(find o2as_phoxi_camera)/urdf/PhoXi3Dscanner_values.xacro"/>

File: o2as_scene_description/urdf/screw_feeder.xacro (robot description, xacro)
@@ -1,4 +1,4 @@
 <?xml version="1.0" ?>
-<robot xmlns:xacro="http://ros.org/wiki/xacro" name="screw_feeder">
+<robot xmlns:xacro="http://www.ros.org/wiki/xacro" name="screw_feeder">
   <xacro:macro name="screw_feeder" params="feedername parent *origin">
   <!-- This creates a screw feeder (roughly) with the origin in the back right corner. -->

File: o2as_scene_description/urdf/screw_tools.xacro (robot description, xacro)
@@ -3,5 +3,5 @@
 <!-- The gripper center would be about 44 mm from the top, so the tip might be 111 mm further down -->
 <!-- The tip\axis seems to be 11.5 mm from the "front" side. The front side looks into the gripper -->
-<robot name="screw_tools">
+<robot xmlns:xacro="http://www.ros.org/wiki/xacro">
   <link name="screw_tool_holder">
     <inertial>
@@ -10,14 +10,28 @@
       <inertia ixx="1" ixy="0" ixz="0" iyy="1" iyz="0" izz="1"/>
     </inertial>
+    <!-- The horizontal plate -->
     <visual>
-      <origin rpy="0 0 0" xyz="0 -.05 0"/>
+      <origin rpy="0 0 0" xyz="-0.15 .0033 0.002"/>
       <geometry>
-        <box size=".3 .1 .004"/>
+        <box size=".3 .066 .004"/>
       </geometry>
     </visual>
     <collision>
-      <origin rpy="0 0 0" xyz="0 -.05 0"/>
+      <origin rpy="0 0 0" xyz="-0.15 .0033 0.002"/>
       <geometry>
-        <box size=".3 .1 .004"/>
+        <box size=".3 .066 .004"/>
+      </geometry>
+    </collision>
+    <!-- The vertical plate -->
+    <visual>
+      <origin rpy="0 0 0" xyz="-0.15 -.011 0.0179"/>
+      <geometry>
+        <box size=".3 .004 .035"/>
+      </geometry>
+    </visual>
+    <collision>
+      <origin rpy="0 0 0" xyz="-0.15 -.011 0.0179"/>
+      <geometry>
+        <box size=".3 .004 .035"/>
       </geometry>
     </collision>
@@ -26,8 +40,11 @@
     <parent link="c_bot_base_smfl" />
     <child link="screw_tool_holder" />
-    <origin xyz="0.45 0.7 0.06" rpy="0.0 0.0 0.0" />
+    <origin xyz="${0.65-0.045} ${0.65+.004} 0.06" rpy="0.0 0.0 0.0" />
   </joint>
   <!-- ++++++++++++++++++++++++++++ -->
- <link name="screw_tool_m6_link">
+  <xacro:property name="bit_cushion_to_axis" value="0.0285"/>
+  <xacro:property name="tool_offset" value="${-.005 + bit_cushion_to_axis}" />
+  <!-- The collision boxes of the tools only include the top part (not what is hanging underneath the holder) -->
+  <link name="screw_tool_m6_link">
     <inertial>
       <origin rpy="0 0 0" xyz="0 0 0"/>
@@ -44,15 +61,15 @@
       </material>
     </visual>
-    <!-- <collision>
-      <origin rpy="0 0 -.225" xyz="0 0 0"/>
+    <collision>
+      <origin rpy="0 0 0" xyz="0 ${bit_cushion_to_axis - .02} .0275"/>
       <geometry>
-        <box size=".02 .04 .155"/>
+        <box size=".026 .04 .055"/>
       </geometry>
-    </collision> -->
+    </collision>
   </link>
   <joint name="screw_tool_m6_to_holder" type="fixed">
     <parent link="screw_tool_holder" />
     <child link="screw_tool_m6_link" />
-    <origin xyz="0.1 0.0 0.0" rpy="0.0 0.0 0.0" />
+    <origin xyz="-0.05 ${tool_offset} 0.004" rpy="0.0 0.0 0.0" />
   </joint>
   <link name="screw_tool_m4_link">
@@ -71,15 +88,15 @@
       </material>
     </visual>
-    <!-- <collision>
-      <origin rpy="0 0 -.225" xyz="0 0 0"/>
+    <collision>
+      <origin rpy="0 0 0" xyz="0 ${bit_cushion_to_axis - .02} .0275"/>
       <geometry>
-        <box size=".02 .04 .155"/>
+        <box size=".026 .04 .055"/>
       </geometry>
-    </collision> -->
+    </collision>
   </link>
   <joint name="screw_tool_m4_to_holder" type="fixed">
     <parent link="screw_tool_holder" />
     <child link="screw_tool_m4_link" />
-    <origin xyz="0.0 0.0 0.0" rpy="0.0 0.0 0.0" />
+    <origin xyz="-0.15 ${tool_offset} 0.004" rpy="0.0 0.0 0.0" />
   </joint>
   <link name="screw_tool_m3_link">
@@ -98,17 +115,17 @@
       </material>
     </visual>
-    <!-- <collision>
-      <origin rpy="0 0 -.225" xyz="0 0 0"/>
+    <collision>
+      <origin rpy="0 0 0" xyz="0 ${bit_cushion_to_axis - .02} .0275"/>
       <geometry>
-        <box size=".02 .04 .155"/>
+        <box size=".026 .04 .055"/>
       </geometry>
-    </collision> -->
+    </collision>
   </link>
   <joint name="screw_tool_m3_to_holder" type="fixed">
     <parent link="screw_tool_holder" />
     <child link="screw_tool_m3_link" />
-    <origin xyz="-0.1 0.0 0.0" rpy="0.0 0.0 0.0" />
+    <origin xyz="-0.25 ${tool_offset} 0.004" rpy="0.0 0.0 0.0" />
   </joint>
-  <!-- Extra links to position the gripper more simply -->
+  <!-- Extra links to position the gripper more easily -->
   <link name="screw_tool_m3_helper_link"/>
   <joint name="screw_tool_m3_helper_joint" type="fixed">

Commit message: Fix collision boxes of several objects

File: o2as_scene_description/urdf/o2as_base.xacro (robot description, xacro)
@@ -18,4 +18,5 @@
       </visual>
       <collision>
+      <origin xyz="${box_w/2} ${box_l/2} ${box_h/2}" rpy="0 0 0"/>
         <geometry>
           <box size="${box_w} ${box_l} ${box_h}"/>

File: o2as_scene_description/urdf/o2as_box.xacro (robot description, xacro)
@@ -15,4 +15,5 @@
       </visual>
       <collision>
+        <origin xyz="${box_w/2} ${box_l/2} ${box_h/2}" rpy="0 0 0"/>
         <geometry>
           <box size="${box_w} ${box_l} ${box_h}"/>

File: o2as_scene_description/urdf/o2as_mat.xacro (robot description, xacro)
@@ -52,4 +52,5 @@
       <!-- Done with boundary drawing -->
       <collision>
+        <origin xyz="${mat_w/2} .01 ${mat_h}" rpy="0 0 0"/>
         <geometry>
           <box size="${mat_w} ${mat_l} ${mat_h}"/>
