Commit message: Fix more references

File: o2as_scene_description/urdf/o2as_osaka_scene.urdf.xacro (robot description, xacro)
@@ -1,5 +1,5 @@
 <?xml version="1.0"?>
 <robot xmlns:xacro="http://ros.org/wiki/xacro"
-       name="o2as_base_scene" >
+       name="o2as_osaka_scene" >
   <xacro:property name="a_bot_x" value="0.0"/>
   <xacro:property name="a_bot_y" value="-0.25"/>
@@ -19,15 +19,12 @@
   <xacro:include filename="$(find o2as_scene_description)/urdf/ur3.urdf.xacro" />
   <!-- Scene items (trays, bins...) -->
-  <xacro:include filename="$(find o2as_scene_description)/urdf/walls.xacro" />
   <xacro:include filename="$(find o2as_scene_description)/urdf/kitting_scene.xacro" />
-  <!-- Robot bases -->
-  <!-- Putting these at height 0.0 makes them intersect with the ground, so they are elevated. -->
-  <!-- There are some instabilities when the box is big, for some reason. -->
+  <!-- Robot base -->
   <xacro:include filename="$(find o2as_scene_description)/urdf/o2as_box.xacro" />
   <xacro:o2as_box boxname="bot_base_column" box_w=".1" box_l=".1" box_h="1.5" parent="o2as_ground">
-    <origin xyz="${-.05} ${-.05} .75" rpy="0 0 0" />
+    <origin xyz="${-.05} ${-.05} 0" rpy="0 0 0" />
   </xacro:o2as_box>
-  <xacro:o2as_box boxname="bot_base_tee" box_w=".1" box_l=".5" box_h=".1" parent="o2as_ground">
-    <origin xyz="${-.05} ${-.05} 1.6" rpy="0 0 0" />
+  <xacro:o2as_box boxname="bot_base_tee" box_w=".1" box_l=".4" box_h=".1" parent="o2as_ground">
+    <origin xyz="${-.05} ${-.2} 1.5" rpy="0 0 0" />
   </xacro:o2as_box>
   <!-- Main workspace -->
@@ -80,5 +77,5 @@
     <parent link="o2as_ground" />
     <child link = "c_bot_base_link" />
-    <origin xyz="${c_bot_x} ${c_bot_y} ${bots_z}" rpy="0.0 0.0 ${-pi/2}" />
+    <origin xyz="${c_bot_x} ${c_bot_y} 0" rpy="0.0 0.0 0.0" />
   </joint>
   <!-- spawn and attach grippers -->

Commit message: Almost in correct orientation

File: o2as_scene_description/urdf/o2as_osaka_scene.urdf.xacro (robot description, xacro)
@@ -2,7 +2,7 @@
 <robot xmlns:xacro="http://ros.org/wiki/xacro"
        name="o2as_osaka_scene" >
-  <xacro:property name="a_bot_x" value="0.0"/>
+  <xacro:property name="a_bot_x" value="-0.3"/>
   <xacro:property name="a_bot_y" value="-0.25"/>
-  <xacro:property name="b_bot_x" value="0.0"/>
+  <xacro:property name="b_bot_x" value="-0.3"/>
   <xacro:property name="b_bot_y" value="0.25"/>
   <xacro:property name="c_bot_x" value="-1.0"/>
@@ -23,8 +23,8 @@
   <xacro:include filename="$(find o2as_scene_description)/urdf/o2as_box.xacro" />
   <xacro:o2as_box boxname="bot_base_column" box_w=".1" box_l=".1" box_h="1.5" parent="o2as_ground">
-    <origin xyz="${-.05} ${-.05} 0" rpy="0 0 0" />
+    <origin xyz="${a_bot_x-.05} ${-.05} 0" rpy="0 0 0" />
   </xacro:o2as_box>
   <xacro:o2as_box boxname="bot_base_tee" box_w=".1" box_l=".4" box_h=".1" parent="o2as_ground">
-    <origin xyz="${-.05} ${-.2} 1.5" rpy="0 0 0" />
+    <origin xyz="${a_bot_x-.05} ${-.2} 1.5" rpy="0 0 0" />
   </xacro:o2as_box>
   <!-- Main workspace -->
@@ -33,5 +33,5 @@
   <xacro:property name="plate_l" value="0.62"/>
   <xacro:o2as_box boxname="workbox" box_w="${plate_w}" box_l="${plate_l}" box_h=".01" parent="o2as_ground">
-    <origin xyz="${-plate_w/2} ${-plate_l/2} ${bots_z-.4}" rpy="0 0 0" />
+    <origin xyz="${-plate_w/2} ${-plate_l/2} ${bots_z-.5}" rpy="0 0 0" />
   </xacro:o2as_box>
   <link name="workspace_center" />
@@ -39,5 +39,5 @@
     <parent link="o2as_ground" />
     <child link="workspace_center" />
-    <origin xyz="0.0 0.0 ${bots_z+.1}" rpy="0.0 0.0 0.0" />
+    <origin xyz="0.0 0.0 ${bots_z-.5}" rpy="0.0 0.0 0.0" />
   </joint>
   <!-- robot arms -->
@@ -67,10 +67,10 @@
     <parent link="o2as_ground" />
     <child link="a_bot_base_link" />
-    <origin xyz="${a_bot_x} ${a_bot_y} ${bots_z}" rpy="0.0 ${pi*3/2} 0.0" />
+    <origin xyz="${a_bot_x} ${a_bot_y} ${bots_z}" rpy="${-pi*1/4} ${pi*5/4} ${-pi}" />
   </joint>
   <joint name="world_b_bot_joint" type="fixed">
     <parent link="o2as_ground" />
     <child link = "b_bot_base_link" />
-    <origin xyz="${b_bot_x} ${b_bot_y} ${bots_z}" rpy="0.0 ${-pi*3/2} ${-pi}" />
+    <origin xyz="${b_bot_x} ${b_bot_y} ${bots_z}" rpy="${-pi*1/4} ${-pi*5/4} 0.0" />
   </joint>
   <joint name="world_c_bot_joint" type="fixed">

Commit message: Overall fixes

File: o2as_scene_description/urdf/o2as_osaka_scene.urdf.xacro (robot description, xacro)
@@ -33,5 +33,5 @@
   <xacro:property name="plate_l" value="0.62"/>
   <xacro:o2as_box boxname="workbox" box_w="${plate_w}" box_l="${plate_l}" box_h=".01" parent="o2as_ground">
-    <origin xyz="${-plate_w/2} ${-plate_l/2} ${bots_z-.5}" rpy="0 0 0" />
+    <origin xyz="${-plate_w/2} ${-plate_l/2} ${bots_z-.6}" rpy="0 0 0" />
   </xacro:o2as_box>
   <link name="workspace_center" />
@@ -42,5 +42,5 @@
   </joint>
   <!-- robot arms -->
-  <xacro:ur3_robot prefix="a_bot_" joint_limited="true"
+  <xacro:ur3_robot prefix="a_bot_" joint_limited="false"
     shoulder_pan_lower_limit="${-pi}" shoulder_pan_upper_limit="${pi}"
     shoulder_lift_lower_limit="${-pi}" shoulder_lift_upper_limit="${pi}"
@@ -49,5 +49,5 @@
     wrist_2_lower_limit="${-pi}" wrist_2_upper_limit="${pi}"
     wrist_3_lower_limit="${-pi}" wrist_3_upper_limit="${pi}"/>
-  <xacro:ur3_robot prefix="b_bot_" joint_limited="true"
+  <xacro:ur3_robot prefix="b_bot_" joint_limited="false"
     shoulder_pan_lower_limit="${-pi}" shoulder_pan_upper_limit="${pi}"
     shoulder_lift_lower_limit="${-pi}" shoulder_lift_upper_limit="${pi}"
@@ -56,5 +56,5 @@
     wrist_2_lower_limit="${-pi}" wrist_2_upper_limit="${pi}"
     wrist_3_lower_limit="${-pi}" wrist_3_upper_limit="${pi}"/>
-  <xacro:ur3_robot prefix="c_bot_" joint_limited="true"
+  <xacro:ur3_robot prefix="c_bot_" joint_limited="false"
     shoulder_pan_lower_limit="${-pi}" shoulder_pan_upper_limit="${pi}"
     shoulder_lift_lower_limit="${-pi}" shoulder_lift_upper_limit="${pi}"
@@ -67,10 +67,10 @@
     <parent link="o2as_ground" />
     <child link="a_bot_base_link" />
-    <origin xyz="${a_bot_x} ${a_bot_y} ${bots_z}" rpy="${-pi*1/4} ${pi*5/4} ${-pi}" />
+    <origin xyz="${a_bot_x} ${a_bot_y} ${bots_z}" rpy="${-pi*1/4} ${pi} ${-pi}" />
   </joint>
   <joint name="world_b_bot_joint" type="fixed">
     <parent link="o2as_ground" />
     <child link = "b_bot_base_link" />
-    <origin xyz="${b_bot_x} ${b_bot_y} ${bots_z}" rpy="${-pi*1/4} ${-pi*5/4} 0.0" />
+    <origin xyz="${b_bot_x} ${b_bot_y} ${bots_z}" rpy="${-pi*1/4} ${-pi} 0.0" />
   </joint>
   <joint name="world_c_bot_joint" type="fixed">

Commit message: Small adjustments

File: o2as_scene_description/urdf/o2as_osaka_scene.urdf.xacro (robot description, xacro)
@@ -19,5 +19,5 @@
   <xacro:include filename="$(find o2as_scene_description)/urdf/ur3.urdf.xacro" />
   <!-- Scene items (trays, bins...) -->
-  <xacro:include filename="$(find o2as_scene_description)/urdf/kitting_scene.xacro" />
+  <!-- <xacro:include filename="$(find o2as_scene_description)/urdf/kitting_scene.xacro" /> -->
   <!-- Robot base -->
   <xacro:include filename="$(find o2as_scene_description)/urdf/o2as_box.xacro" />
@@ -33,5 +33,5 @@
   <xacro:property name="plate_l" value="0.62"/>
   <xacro:o2as_box boxname="workbox" box_w="${plate_w}" box_l="${plate_l}" box_h=".01" parent="o2as_ground">
-    <origin xyz="${-plate_w/2} ${-plate_l/2} ${bots_z-.6}" rpy="0 0 0" />
+    <origin xyz="${-plate_w/2} ${-plate_l/2} ${bots_z-.5}" rpy="0 0 0" />
   </xacro:o2as_box>
   <link name="workspace_center" />
@@ -39,5 +39,5 @@
     <parent link="o2as_ground" />
     <child link="workspace_center" />
-    <origin xyz="0.0 0.0 ${bots_z-.5}" rpy="0.0 0.0 0.0" />
+    <origin xyz="0.0 0.0 ${bots_z-.4}" rpy="0.0 0.0 0.0" />
   </joint>
   <!-- robot arms -->

Commit message: Move MoveIt changes to o2as_osaka_config

File: o2as_scene_description/urdf/o2as_osaka_scene.urdf.xacro (robot description, xacro)
@@ -1,13 +1,15 @@
 <?xml version="1.0"?>
 <robot xmlns:xacro="http://ros.org/wiki/xacro"
-       name="o2as_osaka_scene" >
-  <xacro:property name="a_bot_x" value="-0.3"/>
-  <xacro:property name="a_bot_y" value="-0.25"/>
-  <xacro:property name="b_bot_x" value="-0.3"/>
-  <xacro:property name="b_bot_y" value="0.25"/>
-  <xacro:property name="c_bot_x" value="-1.0"/>
+       name="o2as_base_scene" >
+  <!-- This is the main file defining our robot arrangement and physical environment. -->
+  <!-- Calibration from 20 August 2018 -->
+  <!-- Calibration help: If the robot is not moving far enough to the calibration point, increase these distances -->
+  <xacro:property name="a_bot_x" value="-0.005"/>
+  <xacro:property name="a_bot_y" value="-0.543"/>
+  <xacro:property name="b_bot_x" value="0.001"/>
+  <xacro:property name="b_bot_y" value="0.529"/>
+  <xacro:property name="c_bot_x" value="-0.5"/>
   <xacro:property name="c_bot_y" value="0.0"/>
-  <xacro:property name="bots_z" value="1.5"/>
-  <!-- This is the main file defining our robot arrangement and physical environment. -->
+  <xacro:property name="bots_z" value="0.75"/>
   <!-- common stuff -->
   <xacro:include filename="$(find ur_description)/urdf/common.gazebo.xacro" />
@@ -19,19 +21,27 @@
   <xacro:include filename="$(find o2as_scene_description)/urdf/ur3.urdf.xacro" />
   <!-- Scene items (trays, bins...) -->
-  <!-- <xacro:include filename="$(find o2as_scene_description)/urdf/kitting_scene.xacro" /> -->
-  <!-- Robot base -->
-  <xacro:include filename="$(find o2as_scene_description)/urdf/o2as_box.xacro" />
-  <xacro:o2as_box boxname="bot_base_column" box_w=".1" box_l=".1" box_h="1.5" parent="o2as_ground">
-    <origin xyz="${a_bot_x-.05} ${-.05} 0" rpy="0 0 0" />
-  </xacro:o2as_box>
-  <xacro:o2as_box boxname="bot_base_tee" box_w=".1" box_l=".4" box_h=".1" parent="o2as_ground">
-    <origin xyz="${a_bot_x-.05} ${-.2} 1.5" rpy="0 0 0" />
-  </xacro:o2as_box>
+  <!-- <xacro:include filename="$(find o2as_scene_description)/urdf/taskboard_scene.xacro" /> -->
+  <xacro:include filename="$(find o2as_scene_description)/urdf/kitting_scene.xacro" />
+  <!-- <xacro:include filename="$(find o2as_scene_description)/urdf/assembly_scene.xacro" /> -->
+  <!-- Robot bases -->
+  <!-- Putting these at height 0.0 makes them intersect with the ground, so they are elevated. -->
+  <!-- There are some instabilities when the box is big, for some reason. -->
+  <xacro:include filename="$(find o2as_scene_description)/urdf/o2as_osakabase.xacro" />
+  <xacro:o2as_base boxname="a_bot_base_smfl" parent="o2as_ground">
+    <origin xyz="${a_bot_x-.4/2} ${a_bot_y-.4/2} ${bots_z-.06}" rpy="0 0 0" />
+  </xacro:o2as_base>
+  <xacro:o2as_base boxname="b_bot_base_smfl" parent="o2as_ground">
+    <origin xyz="${b_bot_x-.4/2} ${b_bot_y-.4/2} ${bots_z-.06}" rpy="0 0 0" />
+  </xacro:o2as_base>
+  <xacro:o2as_base boxname="c_bot_base_smfl" parent="o2as_ground">
+    <origin xyz="${c_bot_x-.4/2-.16} ${c_bot_y-.4/2-.1} ${bots_z-.06}" rpy="0 0 0" />
+  </xacro:o2as_base>
   <!-- Main workspace -->
   <!-- The surface is 0.01 m below the robot bases and the "workspace_center" frame. -->
-  <xacro:property name="plate_w" value="0.84"/>
-  <xacro:property name="plate_l" value="0.62"/>
+  <xacro:include filename="$(find o2as_scene_description)/urdf/o2as_box.xacro" />
+  <xacro:property name="plate_w" value="0.9"/>
+  <xacro:property name="plate_l" value="0.75"/>
   <xacro:o2as_box boxname="workbox" box_w="${plate_w}" box_l="${plate_l}" box_h=".01" parent="o2as_ground">
-    <origin xyz="${-plate_w/2} ${-plate_l/2} ${bots_z-.5}" rpy="0 0 0" />
+    <origin xyz="${-plate_w/2+.1} ${-plate_l/2} ${bots_z-0.196}" rpy="0 0 0" />
   </xacro:o2as_box>
   <link name="workspace_center" />
@@ -39,24 +49,37 @@
     <parent link="o2as_ground" />
     <child link="workspace_center" />
-    <origin xyz="0.0 0.0 ${bots_z-.4}" rpy="0.0 0.0 0.0" />
+    <origin xyz="0.0 0.0 ${bots_z+.01-0.196}" rpy="0.0 0.0 0.0" />
   </joint>
+  <!-- Screw holder & screw tool visual -->
+  <!-- <xacro:include filename="$(find o2as_scene_description)/urdf/screw_tools.xacro" /> -->
+  <!-- Feeders -->
+  <!-- <xacro:include filename="$(find o2as_scene_description)/urdf/screw_feeder.xacro" />
+  <xacro:screw_feeder feedername="m3_feeder" parent="a_bot_base_smfl">
+    <origin xyz=".1 .4 .05" rpy="0 0 ${pi/2}" />
+  </xacro:screw_feeder>
+  <xacro:screw_feeder feedername="m4_feeder" parent="c_bot_base_smfl">
+    <origin xyz=".45 .05 .05" rpy="0 0 0" />
+  </xacro:screw_feeder> -->
+  <!-- <xacro:screw_feeder feedername="m5_feeder" parent="c_bot_base_smfl">
+    <origin xyz=".45 .2 .05" rpy="0 0 0" />
+  </xacro:screw_feeder> -->
   <!-- robot arms -->
-  <xacro:ur3_robot prefix="a_bot_" joint_limited="false"
-    shoulder_pan_lower_limit="${-pi}" shoulder_pan_upper_limit="${pi}"
-    shoulder_lift_lower_limit="${-pi}" shoulder_lift_upper_limit="${pi}"
+  <xacro:ur5_robot prefix="a_bot_" joint_limited="true"
+    shoulder_pan_lower_limit="0.0" shoulder_pan_upper_limit="${pi}"
+    shoulder_lift_lower_limit="${-pi}" shoulder_lift_upper_limit="0.0"
     elbow_joint_lower_limit="0.0" elbow_joint_upper_limit="${pi}"
-    wrist_1_lower_limit="${-pi}" wrist_1_upper_limit="${pi}"
+    wrist_1_lower_limit="${-pi}" wrist_1_upper_limit="0.3"
     wrist_2_lower_limit="${-pi}" wrist_2_upper_limit="${pi}"
     wrist_3_lower_limit="${-pi}" wrist_3_upper_limit="${pi}"/>
-  <xacro:ur3_robot prefix="b_bot_" joint_limited="false"
+  <xacro:ur5_robot prefix="b_bot_" joint_limited="true"
     shoulder_pan_lower_limit="${-pi}" shoulder_pan_upper_limit="${pi}"
-    shoulder_lift_lower_limit="${-pi}" shoulder_lift_upper_limit="${pi}"
+    shoulder_lift_lower_limit="${-pi}" shoulder_lift_upper_limit="0.0"
     elbow_joint_lower_limit="0.0" elbow_joint_upper_limit="${pi}"
-    wrist_1_lower_limit="${-pi}" wrist_1_upper_limit="${pi}"
+    wrist_1_lower_limit="${-pi}" wrist_1_upper_limit="0.3"
     wrist_2_lower_limit="${-pi}" wrist_2_upper_limit="${pi}"
     wrist_3_lower_limit="${-pi}" wrist_3_upper_limit="${pi}"/>
-  <xacro:ur3_robot prefix="c_bot_" joint_limited="false"
-    shoulder_pan_lower_limit="${-pi}" shoulder_pan_upper_limit="${pi}"
-    shoulder_lift_lower_limit="${-pi}" shoulder_lift_upper_limit="${pi}"
+  <xacro:ur3_robot prefix="c_bot_" joint_limited="true"
+    shoulder_pan_lower_limit="0.0" shoulder_pan_upper_limit="${pi}"
+    shoulder_lift_lower_limit="${-pi}" shoulder_lift_upper_limit="0.0"
     elbow_joint_lower_limit="0.0" elbow_joint_upper_limit="${pi}"
     wrist_1_lower_limit="${-pi}" wrist_1_upper_limit="${pi}"
@@ -67,27 +90,24 @@
     <parent link="o2as_ground" />
     <child link="a_bot_base_link" />
-    <origin xyz="${a_bot_x} ${a_bot_y} ${bots_z}" rpy="${-pi*1/4} ${pi} ${-pi}" />
+    <origin xyz="${a_bot_x} ${a_bot_y} ${bots_z}" rpy="0.0 0.0 0.0" />
   </joint>
   <joint name="world_b_bot_joint" type="fixed">
     <parent link="o2as_ground" />
     <child link = "b_bot_base_link" />
-    <origin xyz="${b_bot_x} ${b_bot_y} ${bots_z}" rpy="${-pi*1/4} ${-pi} 0.0" />
+    <origin xyz="${b_bot_x} ${b_bot_y} ${bots_z}" rpy="0.0 0.0 ${-pi}" />
   </joint>
   <joint name="world_c_bot_joint" type="fixed">
     <parent link="o2as_ground" />
     <child link = "c_bot_base_link" />
-    <origin xyz="${c_bot_x} ${c_bot_y} 0" rpy="0.0 0.0 0.0" />
+    <origin xyz="${c_bot_x} ${c_bot_y} ${bots_z}" rpy="0.0 0.0 ${-pi/2}" />
   </joint>
   <!-- spawn and attach grippers -->
-  <xacro:include filename="$(find o2as_scene_description)/urdf/robotiq_85_gripper.urdf.xacro" />
-  <xacro:robotiq_85_gripper_o2as prefix="a_bot_" parent = "a_bot_ee_link">
-    <origin xyz="0.0 0 0.0" rpy="0 0 0"/>
-  </xacro:robotiq_85_gripper_o2as>
-  <xacro:robotiq_85_gripper_o2as prefix="b_bot_" parent = "b_bot_ee_link">
-    <origin xyz="0.0 0 0.0" rpy="0 0 0"/>
-  </xacro:robotiq_85_gripper_o2as>
-  <xacro:robotiq_85_gripper_o2as prefix="c_bot_" parent = "c_bot_ee_link">
-    <origin xyz="0.0 0 0.0" rpy="0 0 0"/>
-  </xacro:robotiq_85_gripper_o2as>
+  <xacro:include filename="$(find o2as_scene_description)/urdf/precision_gripper.xacro" />
+  <xacro:precision_gripper prefix="a_bot_"  grippername = "gripper" parent = "a_bot_tool0">
+    <origin xyz="0.0 0 0.04" rpy="0 ${pi/2} 0"/>
+  </xacro:precision_gripper>
+  <xacro:include filename="$(find o2as_scene_description)/urdf/robotiq_85_gripper_with_ft300.urdf.xacro" />
+  <xacro:robotiq_85_gripper_o2as prefix="b_bot_" parent = "b_bot_ee_link" />
+  <xacro:robotiq_85_gripper_o2as prefix="c_bot_" parent = "c_bot_ee_link"/>
   <!-- Add cameras -->
   <link name="b_bot_cam_holder_link" />
@@ -100,5 +120,5 @@
     <origin xyz="0 0 0" rpy="0 0 0"/>
   </xacro:sensor_d435>
-  <!-- I meant to remove the "world" link definition, but apparently it is necessary for Gazebo -->
+  <!-- I would like to remove the "world" link definition, but apparently it is necessary for Gazebo -->
   <link name="world" />
   <joint name="world_o2as_joint" type="fixed">

Commit message: Add belt_pick stub and change to taskbaord scene

File: o2as_scene_description/urdf/o2as_osaka_scene.urdf.xacro (robot description, xacro)
@@ -21,6 +21,6 @@
   <xacro:include filename="$(find o2as_scene_description)/urdf/ur3.urdf.xacro" />
   <!-- Scene items (trays, bins...) -->
-  <!-- <xacro:include filename="$(find o2as_scene_description)/urdf/taskboard_scene.xacro" /> -->
-  <xacro:include filename="$(find o2as_scene_description)/urdf/kitting_scene.xacro" />
+  <xacro:include filename="$(find o2as_scene_description)/urdf/taskboard_scene.xacro" />
+  <!-- <xacro:include filename="$(find o2as_scene_description)/urdf/kitting_scene.xacro" /> -->
   <!-- <xacro:include filename="$(find o2as_scene_description)/urdf/assembly_scene.xacro" /> -->
   <!-- Robot bases -->

File: o2as_scene_description/urdf/taskboard_scene.xacro (robot description, xacro)
@@ -5,6 +5,6 @@
   <xacro:include filename="$(find o2as_scene_description)/urdf/task_board.xacro" />
   <xacro:task_board boardname="taskboard" parent="workspace_center">
-    <!-- <origin xyz="-0.35 0.2 0.0" rpy="0 0 ${-pi/2}" />    -->
-    <origin xyz="-0.35 0.1 0.0" rpy="0 0 ${-pi/2}" />
+    <origin xyz="-0.35 0.2 0.0" rpy="0 0 ${-pi/2}" />
+    <!-- <origin xyz="-0.35 0.1 0.0" rpy="0 0 ${-pi/2}" />  -->
   </xacro:task_board>
   <!-- Placement mat -->

Commit message: add inner_open_slightly function to precision gripper

File: o2as_scene_description/urdf/o2as_osaka_scene.urdf.xacro (robot description, xacro)
@@ -52,13 +52,13 @@
   </joint>
   <!-- Screw holder & screw tool visual -->
-  <!-- <xacro:include filename="$(find o2as_scene_description)/urdf/screw_tools.xacro" /> -->
+  <xacro:include filename="$(find o2as_scene_description)/urdf/screw_tools.xacro" />
   <!-- Feeders -->
-  <!-- <xacro:include filename="$(find o2as_scene_description)/urdf/screw_feeder.xacro" />
+  <xacro:include filename="$(find o2as_scene_description)/urdf/screw_feeder.xacro" />
   <xacro:screw_feeder feedername="m3_feeder" parent="a_bot_base_smfl">
-    <origin xyz=".1 .4 .05" rpy="0 0 ${pi/2}" />
+    <origin xyz=".1 .4 -.01" rpy="0 0 ${pi/2}" />
   </xacro:screw_feeder>
-  <xacro:screw_feeder feedername="m4_feeder" parent="c_bot_base_smfl">
+  <!-- <xacro:screw_feeder feedername="m4_feeder" parent="c_bot_base_smfl">
     <origin xyz=".45 .05 .05" rpy="0 0 0" />
-  </xacro:screw_feeder> -->
+  </xacro:screw_feeder> --> -->
   <!-- <xacro:screw_feeder feedername="m5_feeder" parent="c_bot_base_smfl">
     <origin xyz=".45 .2 .05" rpy="0 0 0" />

Commit message: add the gripper and adjust the collision model

File: o2as_scene_description/urdf/o2as_osaka_scene.urdf.xacro (robot description, xacro)
@@ -17,10 +17,10 @@
   <xacro:include filename="$(find realsense2_camera)/urdf/_d435.urdf.xacro" />
   <!-- robots -->
-  <xacro:include filename="$(find o2as_scene_description)/urdf/ur10.urdf.xacro" />
+  <!-- <xacro:include filename="$(find o2as_scene_description)/urdf/ur10.urdf.xacro" /> -->
   <xacro:include filename="$(find o2as_scene_description)/urdf/ur5.urdf.xacro" />
   <xacro:include filename="$(find o2as_scene_description)/urdf/ur3.urdf.xacro" />
   <!-- Scene items (trays, bins...) -->
-  <xacro:include filename="$(find o2as_scene_description)/urdf/taskboard_scene.xacro" />
-  <!-- <xacro:include filename="$(find o2as_scene_description)/urdf/kitting_scene.xacro" /> -->
+  <!-- <xacro:include filename="$(find o2as_scene_description)/urdf/taskboard_scene.xacro" /> -->
+  <xacro:include filename="$(find o2as_scene_description)/urdf/kitting_scene_osaka.xacro" />
   <!-- <xacro:include filename="$(find o2as_scene_description)/urdf/assembly_scene.xacro" /> -->
   <!-- Robot bases -->
@@ -56,9 +56,9 @@
   <!-- <xacro:include filename="$(find o2as_scene_description)/urdf/screw_feeder.xacro" />
   <xacro:screw_feeder feedername="m3_feeder" parent="a_bot_base_smfl">
-    <origin xyz=".1 .4 -.01" rpy="0 0 ${pi/2}" />
+    <origin xyz=".1 .4 .05" rpy="0 0 ${pi/2}" />
+  </xacro:screw_feeder>
+  <xacro:screw_feeder feedername="m4_feeder" parent="c_bot_base_smfl">
+    <origin xyz=".45 .05 .05" rpy="0 0 0" />
   </xacro:screw_feeder> -->
-  <!-- <xacro:screw_feeder feedername="m4_feeder" parent="c_bot_base_smfl">
-    <origin xyz=".45 .05 .05" rpy="0 0 0" />
-  </xacro:screw_feeder> --> -->
   <!-- <xacro:screw_feeder feedername="m5_feeder" parent="c_bot_base_smfl">
     <origin xyz=".45 .2 .05" rpy="0 0 0" />
@@ -103,8 +103,12 @@
   </joint>
   <!-- spawn and attach grippers -->
-  <xacro:include filename="$(find o2as_scene_description)/urdf/precision_gripper.xacro" />
+  <!-- <xacro:include filename="$(find o2as_scene_description)/urdf/precision_gripper.xacro" />
   <xacro:precision_gripper prefix="a_bot_"  grippername = "gripper" parent = "a_bot_tool0">
     <origin xyz="0.0 0 0.04" rpy="0 ${pi/2} 0"/>
-  </xacro:precision_gripper>
+  </xacro:precision_gripper> -->
+  <xacro:include filename="$(find o2as_scene_description)/urdf/InnerOnlyGripper.xacro" />
+  <xacro:InnerOnlyGripper prefix="a_bot_"  grippername = "gripper" parent = "a_bot_tool0">
+    <origin xyz="0.0 0 0.0" rpy="0 0 0"/>
+  </xacro:InnerOnlyGripper>
   <xacro:include filename="$(find o2as_scene_description)/urdf/robotiq_85_gripper_with_ft300.urdf.xacro" />
   <xacro:robotiq_85_gripper_o2as prefix="b_bot_" parent = "b_bot_ee_link" />
