Commit message: Fixed bins origin.

File: o2as_scene_description/urdf/kitting_bin_macros.xacro (robot description, xacro)
@@ -12,5 +12,5 @@
       </inertial>
       <visual>
-        <origin rpy="${pi/2} 0 ${pi/2}" xyz="0 0 ${z_origin_offset}"/>
+        <origin rpy="${pi/2} 0 ${-pi/2}" xyz="0 0 ${z_origin_offset}"/>
         <geometry>
           <mesh filename="${mesh_file}" scale="0.001 0.001 0.001"/>
@@ -22,5 +22,5 @@
       </visual>
       <collision>
-        <origin rpy="${pi/2} 0 ${pi/2}" xyz="0 0 ${z_origin_offset}"/>
+        <origin rpy="${pi/2} 0 ${-pi/2}" xyz="0 0 ${z_origin_offset}"/>
         <geometry>
           <mesh filename="${mesh_file_col}" scale="0.001 0.001 0.001"/>

File: o2as_scene_description/urdf/kitting_bins.xacro (robot description, xacro)
@@ -17,50 +17,50 @@
  <xacro:property name="z_origin_offset_3" value="-.004" />
  <!-- A row of bin1 -->
- <xacro:property name="set1_x" value=".0"/>
+ <xacro:property name="set1_x" value=".1675"/>
  <xacro:property name="set1_y" value="0.33"/>
- <xacro:property name="set1_z" value=".01"/>
+ <xacro:property name="set1_z" value=".0"/>
  <!-- A row of bin2 -->
- <xacro:property name="set2_x" value=".20"/>
+ <xacro:property name="set2_x" value=".376"/>
  <xacro:property name="set2_y" value="0.33"/>
- <xacro:property name="set2_z" value=".00"/>
- <!--set1_bin1_1_-->
-  <xacro:kitting_bin_1 binname="set1_bin1_1" parent="workspace_center" z_origin_offset="-.008">
-      <origin xyz=".0 0.2675 0.018" rpy="0 0 0" />
+ <xacro:property name="set2_z" value=".0"/>
+ <!--set1_bin3_1_-->
+  <xacro:kitting_bin_3 binname="set1_bin3_1" parent="workspace_center" z_origin_offset="-.004">
+      <origin xyz=".1675 0.234 0.004" rpy="0 0 0" />
+  </xacro:kitting_bin_3>
+  <!--set1_bin2_1_-->
+  <xacro:kitting_bin_2 binname="set1_bin2_1" parent="workspace_center" z_origin_offset="-.009">
+      <origin xyz=".1675 0.082 0.009" rpy="0 0 0" />
+  </xacro:kitting_bin_2>
+  <!--set1_bin2_2_-->
+  <xacro:kitting_bin_2 binname="set1_bin2_2" parent="workspace_center" z_origin_offset="-.009">
+      <origin xyz=".1675 -0.03 0.009" rpy="0 0 0" />
+  </xacro:kitting_bin_2>
+  <!--set1_bin2_3_-->
+  <xacro:kitting_bin_2 binname="set1_bin2_3" parent="workspace_center" z_origin_offset="-.009">
+      <origin xyz=".1675 -0.142 0.009" rpy="0 0 0" />
+  </xacro:kitting_bin_2>
+  <!--set1_bin2_4_-->
+  <xacro:kitting_bin_2 binname="set1_bin2_4" parent="workspace_center" z_origin_offset="-.009">
+      <origin xyz=".1675 -0.254 0.009" rpy="0 0 0" />
+  </xacro:kitting_bin_2>
+  <!--set2_bin1_1_-->
+  <xacro:kitting_bin_1 binname="set2_bin1_1" parent="workspace_center" z_origin_offset="-.008">
+      <origin xyz=".376 0.2675 0.008" rpy="0 0 0" />
   </xacro:kitting_bin_1>
-  <!--set1_bin1_2_-->
-  <xacro:kitting_bin_1 binname="set1_bin1_2" parent="workspace_center" z_origin_offset="-.008">
-      <origin xyz=".0 0.1425 0.018" rpy="0 0 0" />
+  <!--set2_bin1_2_-->
+  <xacro:kitting_bin_1 binname="set2_bin1_2" parent="workspace_center" z_origin_offset="-.008">
+      <origin xyz=".376 0.1425 0.008" rpy="0 0 0" />
   </xacro:kitting_bin_1>
-  <!--set1_bin1_3_-->
-  <xacro:kitting_bin_1 binname="set1_bin1_3" parent="workspace_center" z_origin_offset="-.008">
-      <origin xyz=".0 0.0175 0.018" rpy="0 0 0" />
+  <!--set2_bin1_3_-->
+  <xacro:kitting_bin_1 binname="set2_bin1_3" parent="workspace_center" z_origin_offset="-.008">
+      <origin xyz=".376 0.0175 0.008" rpy="0 0 0" />
   </xacro:kitting_bin_1>
-  <!--set1_bin1_4_-->
-  <xacro:kitting_bin_1 binname="set1_bin1_4" parent="workspace_center" z_origin_offset="-.008">
-      <origin xyz=".0 -0.1075 0.018" rpy="0 0 0" />
+  <!--set2_bin1_4_-->
+  <xacro:kitting_bin_1 binname="set2_bin1_4" parent="workspace_center" z_origin_offset="-.008">
+      <origin xyz=".376 -0.1075 0.008" rpy="0 0 0" />
   </xacro:kitting_bin_1>
-  <!--set1_bin1_5_-->
-  <xacro:kitting_bin_1 binname="set1_bin1_5" parent="workspace_center" z_origin_offset="-.008">
-      <origin xyz=".0 -0.2325 0.018" rpy="0 0 0" />
+  <!--set2_bin1_5_-->
+  <xacro:kitting_bin_1 binname="set2_bin1_5" parent="workspace_center" z_origin_offset="-.008">
+      <origin xyz=".376 -0.2325 0.008" rpy="0 0 0" />
   </xacro:kitting_bin_1>
-  <!--set2_bin3_1_-->
-  <xacro:kitting_bin_3 binname="set2_bin3_1" parent="workspace_center" z_origin_offset="-.004">
-      <origin xyz=".20 0.234 0.004" rpy="0 0 0" />
-  </xacro:kitting_bin_3>
-  <!--set2_bin2_1_-->
-  <xacro:kitting_bin_2 binname="set2_bin2_1" parent="workspace_center" z_origin_offset="-.009">
-      <origin xyz=".20 0.082 0.009" rpy="0 0 0" />
-  </xacro:kitting_bin_2>
-  <!--set2_bin2_2_-->
-  <xacro:kitting_bin_2 binname="set2_bin2_2" parent="workspace_center" z_origin_offset="-.009">
-      <origin xyz=".20 -0.03 0.009" rpy="0 0 0" />
-  </xacro:kitting_bin_2>
-  <!--set2_bin2_3_-->
-  <xacro:kitting_bin_2 binname="set2_bin2_3" parent="workspace_center" z_origin_offset="-.009">
-      <origin xyz=".20 -0.142 0.009" rpy="0 0 0" />
-  </xacro:kitting_bin_2>
-  <!--set2_bin2_4_-->
-  <xacro:kitting_bin_2 binname="set2_bin2_4" parent="workspace_center" z_origin_offset="-.009">
-      <origin xyz=".20 -0.254 0.009" rpy="0 0 0" />
-  </xacro:kitting_bin_2>
 </robot>

File: o2as_scene_description/urdf/kitting_scene.xacro (robot description, xacro)
@@ -1,6 +1,6 @@
 <?xml version="1.0"?>
 <robot xmlns:xacro="http://www.ros.org/wiki/xacro" name="kitting_scene">
-  <!-- <xacro:include filename="$(find o2as_scene_description)/urdf/kitting_bins.xacro" /> -->
-  <!-- <xacro:include filename="$(find o2as_scene_description)/urdf/kitting_tray_with_partitions.xacro" /> -->
+  <xacro:include filename="$(find o2as_scene_description)/urdf/kitting_bins.xacro" />
+  <xacro:include filename="$(find o2as_scene_description)/urdf/kitting_tray_with_partitions.xacro" />
   <xacro:include filename="$(find realsense2_camera)/urdf/_d435.urdf.xacro" />
   <!-- spawn and attach dual suction grippers -->
@@ -23,5 +23,5 @@
   <!-- TODO: Deal with this camera? -->
   <!-- A row of tray -->
-  <!-- <xacro:property name="set3_x" value="${-.3}" />
+  <xacro:property name="set3_x" value="${-.3}" />
   <xacro:property name="set3_y" value="${0}" />
   <xacro:property name="set3_z" value=".00" />
@@ -31,4 +31,4 @@
   <xacro:kitting_tray2 trayname="set3_tray_2" parent="workspace_center">
     <origin xyz="${set3_x} ${set3_y-tray_width} ${set3_z}" rpy="0 0 0" />
-  </xacro:kitting_tray2> -->
+  </xacro:kitting_tray2>
 </robot>

Commit message: Update kitting scene

File: o2as_scene_description/urdf/kitting_bin_macros.xacro (robot description, xacro)
@@ -42,4 +42,10 @@
       <xacro:insert_block name="origin"/>
     </xacro:kitting_bin_internal>
+    <joint name="${binname}_top_left_corner_joint" type="fixed">
+      <parent link="${binname}"/>
+      <child link="${binname}_top_left_corner_link"/>
+      <origin rpy="0.0 0.0 0.0" xyz="0.1 0.1 -0.146 "/>
+    </joint>
+    <link name="${binname}_top_left_corner_link"/>
   </xacro:macro>
   <xacro:macro name="kitting_bin_2" params="binname parent z_origin_offset *origin">

File: o2as_scene_description/urdf/kitting_bins.xacro (robot description, xacro)
@@ -11,5 +11,5 @@
     <parent link="workspace_center" />
     <child link="rack_bins_center"/>
-    <origin xyz=".21 0 0.015" rpy="0 0 0"/>
+    <origin xyz=".26 0 0.015" rpy="0 0 0"/>
   </joint>
  <!-- space for bin -->
@@ -27,50 +27,50 @@
  <xacro:property name="z_origin_offset_3" value="-.004" />
  <!-- A row of bin1 -->
- <xacro:property name="set1_x" value=".1425"/>
+ <xacro:property name="set1_x" value=".2425"/>
  <xacro:property name="set1_y" value="0.245"/>
  <xacro:property name="set1_z" value="0.015"/>
  <!-- A row of bin2 -->
- <xacro:property name="set2_x" value=".349"/>
+ <xacro:property name="set2_x" value=".449"/>
  <xacro:property name="set2_y" value="0.245"/>
  <xacro:property name="set2_z" value="0.015"/>
  <!--set1_bin2_1_-->
   <xacro:kitting_bin_2 binname="set1_bin2_1" parent="workspace_center" z_origin_offset="-.009">
-      <origin xyz=".1425 0.189 0.024" rpy="0 0 0" />
+      <origin xyz=".2425 0.189 0.024" rpy="0 0 0" />
   </xacro:kitting_bin_2>
   <!--set1_bin2_2_-->
   <xacro:kitting_bin_2 binname="set1_bin2_2" parent="workspace_center" z_origin_offset="-.009">
-      <origin xyz=".1425 0.077 0.024" rpy="0 0 0" />
+      <origin xyz=".2425 0.077 0.024" rpy="0 0 0" />
   </xacro:kitting_bin_2>
   <!--set1_bin2_3_-->
   <xacro:kitting_bin_2 binname="set1_bin2_3" parent="workspace_center" z_origin_offset="-.009">
-      <origin xyz=".1425 -0.035 0.024" rpy="0 0 0" />
+      <origin xyz=".2425 -0.035 0.024" rpy="0 0 0" />
   </xacro:kitting_bin_2>
   <!--set1_bin2_4_-->
   <xacro:kitting_bin_2 binname="set1_bin2_4" parent="workspace_center" z_origin_offset="-.009">
-      <origin xyz=".1425 -0.147 0.024" rpy="0 0 0" />
+      <origin xyz=".2425 -0.147 0.024" rpy="0 0 0" />
   </xacro:kitting_bin_2>
   <!--set1_bin3_1_-->
   <xacro:kitting_bin_3 binname="set1_bin3_1" parent="workspace_center" z_origin_offset="-.004">
-      <origin xyz=".1425 -0.299 0.019" rpy="0 0 0" />
+      <origin xyz=".2425 -0.299 0.019" rpy="0 0 0" />
   </xacro:kitting_bin_3>
   <!--set2_bin1_1_-->
   <xacro:kitting_bin_1 binname="set2_bin1_1" parent="workspace_center" z_origin_offset="-.008">
-      <origin xyz=".349 0.1825 0.023" rpy="0 0 0" />
+      <origin xyz=".449 0.1825 0.023" rpy="0 0 0" />
   </xacro:kitting_bin_1>
   <!--set2_bin1_2_-->
   <xacro:kitting_bin_1 binname="set2_bin1_2" parent="workspace_center" z_origin_offset="-.008">
-      <origin xyz=".349 0.0575 0.023" rpy="0 0 0" />
+      <origin xyz=".449 0.0575 0.023" rpy="0 0 0" />
   </xacro:kitting_bin_1>
   <!--set2_bin1_3_-->
   <xacro:kitting_bin_1 binname="set2_bin1_3" parent="workspace_center" z_origin_offset="-.008">
-      <origin xyz=".349 -0.0675 0.023" rpy="0 0 0" />
+      <origin xyz=".449 -0.0675 0.023" rpy="0 0 0" />
   </xacro:kitting_bin_1>
   <!--set2_bin1_4_-->
   <xacro:kitting_bin_1 binname="set2_bin1_4" parent="workspace_center" z_origin_offset="-.008">
-      <origin xyz=".349 -0.1925 0.023" rpy="0 0 0" />
+      <origin xyz=".449 -0.1925 0.023" rpy="0 0 0" />
   </xacro:kitting_bin_1>
   <!--set2_bin1_5_-->
   <xacro:kitting_bin_1 binname="set2_bin1_5" parent="workspace_center" z_origin_offset="-.008">
-      <origin xyz=".349 -0.3175 0.023" rpy="0 0 0" />
+      <origin xyz=".449 -0.3175 0.023" rpy="0 0 0" />
   </xacro:kitting_bin_1>
 </robot>

File: o2as_scene_description/urdf/templates/o2as_bin_template_front.xacro (robot description, xacro)
@@ -11,4 +11,4 @@
     <parent link="workspace_center" />
     <child link="rack_bins_center"/>
-    <origin xyz=".21 0 0.015" rpy="0 0 0"/>
+    <origin xyz=".26 0 0.015" rpy="0 0 0"/>
   </joint>

Commit message: add frames in the corners of the set 2 bin

File: o2as_scene_description/urdf/kitting_bin_macros.xacro (robot description, xacro)
@@ -42,10 +42,52 @@
       <xacro:insert_block name="origin"/>
     </xacro:kitting_bin_internal>
-    <joint name="${binname}_top_left_corner_joint" type="fixed">
+    <joint name="${binname}_bottom_front_right_corner_joint" type="fixed">
       <parent link="${binname}"/>
-      <child link="${binname}_top_left_corner_link"/>
-      <origin rpy="0.0 0.0 0.0" xyz="0.1 0.1 -0.146 "/>
+      <child link="${binname}_bottom_front_right_corner"/>
+      <origin rpy="0.0 0.0 0.0" xyz="0.04 0.055 0.0 "/>
     </joint>
-    <link name="${binname}_top_left_corner_link"/>
+    <link name="${binname}_bottom_front_right_corner"/>
+    <joint name="${binname}_bottom_back_right_corner_joint" type="fixed">
+      <parent link="${binname}"/>
+      <child link="${binname}_bottom_back_right_corner"/>
+      <origin rpy="0.0 0.0 0.0" xyz="-0.055 0.055 0.0 "/>
+    </joint>
+    <link name="${binname}_bottom_back_right_corner"/>
+    <joint name="${binname}_bottom_back_left_corner_joint" type="fixed">
+      <parent link="${binname}"/>
+      <child link="${binname}_bottom_back_left_corner"/>
+      <origin rpy="0.0 0.0 0.0" xyz="-0.055 -0.055 0.0 "/>
+    </joint>
+    <link name="${binname}_bottom_back_left_corner"/>
+    <joint name="${binname}_bottom_front_left_corner_joint" type="fixed">
+      <parent link="${binname}"/>
+      <child link="${binname}_bottom_front_left_corner"/>
+      <origin rpy="0.0 0.0 0.0" xyz="0.04 -0.055 0.0 "/>
+    </joint>
+    <link name="${binname}_bottom_front_left_corner"/>
+    <joint name="${binname}_top_front_right_corner_joint" type="fixed">
+      <parent link="${binname}"/>
+      <child link="${binname}_top_front_right_corner"/>
+      <origin rpy="0.0 0.0 0.0" xyz="0.04 0.055 0.04 "/>
+    </joint>
+    <link name="${binname}_top_front_right_corner"/>
+    <joint name="${binname}_top_back_right_corner_joint" type="fixed">
+      <parent link="${binname}"/>
+      <child link="${binname}_top_back_right_corner"/>
+      <origin rpy="0.0 0.0 0.0" xyz="-0.055 0.055 0.04 "/>
+    </joint>
+    <link name="${binname}_top_back_right_corner"/>
+    <joint name="${binname}_top_back_left_corner_joint" type="fixed">
+      <parent link="${binname}"/>
+      <child link="${binname}_top_back_left_corner"/>
+      <origin rpy="0.0 0.0 0.0" xyz="-0.055 -0.055 0.04 "/>
+    </joint>
+    <link name="${binname}_top_back_left_corner"/>
+    <joint name="${binname}_top_front_left_corner_joint" type="fixed">
+      <parent link="${binname}"/>
+      <child link="${binname}_top_front_left_corner"/>
+      <origin rpy="0.0 0.0 0.0" xyz="0.04 -0.055 0.04 "/>
+    </joint>
+    <link name="${binname}_top_front_left_corner"/>
   </xacro:macro>
   <xacro:macro name="kitting_bin_2" params="binname parent z_origin_offset *origin">
