Commit message: Add bin corner calibration frames and functions

File: o2as_scene_description/urdf/kitting_bin_macros.xacro (robot description, xacro)
@@ -15,5 +15,4 @@
         <geometry>
           <mesh filename="${mesh_file}" scale="0.001 0.001 0.001"/>
-          <!-- <mesh filename="package://ur_description/meshes/ur5/visual/shoulder.dae"/> -->
         </geometry>
         <material name="orange">
@@ -25,5 +24,4 @@
         <geometry>
           <mesh filename="${mesh_file_col}" scale="0.001 0.001 0.001"/>
-          <!-- <mesh filename="package://ur_description/meshes/ur5/collision/shoulder.stl"/> -->
         </geometry>
       </collision>
@@ -42,10 +40,55 @@
       <xacro:insert_block name="origin"/>
     </xacro:kitting_bin_internal>
-    <joint name="${binname}_top_left_corner_joint" type="fixed">
-      <parent link="${binname}"/>
-      <child link="${binname}_top_left_corner_link"/>
-      <origin rpy="0.0 0.0 0.0" xyz="0.1 0.1 -0.146 "/>
-    </joint>
-    <link name="${binname}_top_left_corner_link"/>
+    <xacro:property name="bin1_half_width" value="0.055"/>
+    <xacro:property name="bin1_half_length" value="0.055"/>
+    <xacro:property name="bin1_height_internal" value=".05" />
+    <joint name="${binname}_bottom_front_right_corner_joint" type="fixed">
+      <parent link="${binname}"/>
+      <child link="${binname}_bottom_front_right_corner"/>
+      <origin rpy="0.0 0.0 0.0" xyz="${bin1_half_length-.015} ${bin1_half_width} 0.0 "/>
+    </joint>
+    <link name="${binname}_bottom_front_right_corner"/>
+    <joint name="${binname}_bottom_back_right_corner_joint" type="fixed">
+      <parent link="${binname}"/>
+      <child link="${binname}_bottom_back_right_corner"/>
+      <origin rpy="0.0 0.0 0.0" xyz="${-bin1_half_length} ${bin1_half_width} 0.0 "/>
+    </joint>
+    <link name="${binname}_bottom_back_right_corner"/>
+    <joint name="${binname}_bottom_back_left_corner_joint" type="fixed">
+      <parent link="${binname}"/>
+      <child link="${binname}_bottom_back_left_corner"/>
+      <origin rpy="0.0 0.0 0.0" xyz="${-bin1_half_length} ${-bin1_half_width} 0.0 "/>
+    </joint>
+    <link name="${binname}_bottom_back_left_corner"/>
+    <joint name="${binname}_bottom_front_left_corner_joint" type="fixed">
+      <parent link="${binname}"/>
+      <child link="${binname}_bottom_front_left_corner"/>
+      <origin rpy="0.0 0.0 0.0" xyz="${bin1_half_length-.015} ${-bin1_half_width} 0.0 "/>
+    </joint>
+    <link name="${binname}_bottom_front_left_corner"/>
+    <joint name="${binname}_top_front_right_corner_joint" type="fixed">
+      <parent link="${binname}"/>
+      <child link="${binname}_top_front_right_corner"/>
+      <origin rpy="0.0 0.0 0.0" xyz="${bin1_half_length -.015} ${bin1_half_width} ${bin1_height_internal} "/>
+    </joint>
+    <link name="${binname}_top_front_right_corner"/>
+    <joint name="${binname}_top_back_right_corner_joint" type="fixed">
+      <parent link="${binname}"/>
+      <child link="${binname}_top_back_right_corner"/>
+      <origin rpy="0.0 0.0 0.0" xyz="${-bin1_half_length} ${bin1_half_width} ${bin1_height_internal} "/>
+    </joint>
+    <link name="${binname}_top_back_right_corner"/>
+    <joint name="${binname}_top_back_left_corner_joint" type="fixed">
+      <parent link="${binname}"/>
+      <child link="${binname}_top_back_left_corner"/>
+      <origin rpy="0.0 0.0 0.0" xyz="${-bin1_half_length} ${-bin1_half_width} ${bin1_height_internal} "/>
+    </joint>
+    <link name="${binname}_top_back_left_corner"/>
+    <joint name="${binname}_top_front_left_corner_joint" type="fixed">
+      <parent link="${binname}"/>
+      <child link="${binname}_top_front_left_corner"/>
+      <origin rpy="0.0 0.0 0.0" xyz="${bin1_half_length-.015} ${-bin1_half_width} ${bin1_height_internal} "/>
+    </joint>
+    <link name="${binname}_top_front_left_corner"/>
   </xacro:macro>
   <xacro:macro name="kitting_bin_2" params="binname parent z_origin_offset *origin">
@@ -53,4 +96,55 @@
       <xacro:insert_block name="origin"/>
     </xacro:kitting_bin_internal>
+    <xacro:property name="bin2_half_width" value="0.045"/>
+    <xacro:property name="bin2_half_length" value="0.09"/>
+    <xacro:property name="bin2_height_internal" value=".07" />
+    <joint name="${binname}_bottom_front_right_corner_joint" type="fixed">
+      <parent link="${binname}"/>
+      <child link="${binname}_bottom_front_right_corner"/>
+      <origin rpy="0.0 0.0 0.0" xyz="${bin2_half_length-.02} ${bin2_half_width} 0.0 "/>
+    </joint>
+    <link name="${binname}_bottom_front_right_corner"/>
+    <joint name="${binname}_bottom_back_right_corner_joint" type="fixed">
+      <parent link="${binname}"/>
+      <child link="${binname}_bottom_back_right_corner"/>
+      <origin rpy="0.0 0.0 0.0" xyz="${-bin2_half_length} ${bin2_half_width} 0.0 "/>
+    </joint>
+    <link name="${binname}_bottom_back_right_corner"/>
+    <joint name="${binname}_bottom_back_left_corner_joint" type="fixed">
+      <parent link="${binname}"/>
+      <child link="${binname}_bottom_back_left_corner"/>
+      <origin rpy="0.0 0.0 0.0" xyz="${-bin2_half_length} ${-bin2_half_width} 0.0 "/>
+    </joint>
+    <link name="${binname}_bottom_back_left_corner"/>
+    <joint name="${binname}_bottom_front_left_corner_joint" type="fixed">
+      <parent link="${binname}"/>
+      <child link="${binname}_bottom_front_left_corner"/>
+      <origin rpy="0.0 0.0 0.0" xyz="${bin2_half_length-.02} ${-bin2_half_width} 0.0 "/>
+    </joint>
+    <link name="${binname}_bottom_front_left_corner"/>
+    <joint name="${binname}_top_front_right_corner_joint" type="fixed">
+      <parent link="${binname}"/>
+      <child link="${binname}_top_front_right_corner"/>
+      <origin rpy="0.0 0.0 0.0" xyz="${bin2_half_length-.02} ${bin2_half_width} ${bin2_height_internal} "/>
+    </joint>
+    <link name="${binname}_top_front_right_corner"/>
+    <joint name="${binname}_top_back_right_corner_joint" type="fixed">
+      <parent link="${binname}"/>
+      <child link="${binname}_top_back_right_corner"/>
+      <origin rpy="0.0 0.0 0.0" xyz="${-bin2_half_length} ${bin2_half_width} ${bin2_height_internal} "/>
+    </joint>
+    <link name="${binname}_top_back_right_corner"/>
+    <joint name="${binname}_top_back_left_corner_joint" type="fixed">
+      <parent link="${binname}"/>
+      <child link="${binname}_top_back_left_corner"/>
+      <origin rpy="0.0 0.0 0.0" xyz="${-bin2_half_length} ${-bin2_half_width} ${bin2_height_internal} "/>
+    </joint>
+    <link name="${binname}_top_back_left_corner"/>
+    <joint name="${binname}_top_front_left_corner_joint" type="fixed">
+      <parent link="${binname}"/>
+      <child link="${binname}_top_front_left_corner"/>
+      <origin rpy="0.0 0.0 0.0" xyz="${bin2_half_length-.02} ${-bin2_half_width} ${bin2_height_internal} "/>
+    </joint>
+    <link name="${binname}_top_front_left_corner"/>
   </xacro:macro>
   <xacro:macro name="kitting_bin_3" params="binname parent z_origin_offset *origin">
@@ -58,4 +152,55 @@
       <xacro:insert_block name="origin"/>
     </xacro:kitting_bin_internal>
+    <xacro:property name="bin3_half_width" value="0.078"/>
+    <xacro:property name="bin3_half_length" value="0.13"/>
+    <xacro:property name="bin3_height_internal" value=".09" />
+    <joint name="${binname}_bottom_front_right_corner_joint" type="fixed">
+      <parent link="${binname}"/>
+      <child link="${binname}_bottom_front_right_corner"/>
+      <origin rpy="0.0 0.0 0.0" xyz="${bin3_half_length-.045} ${bin3_half_width} 0.0 "/>
+    </joint>
+    <link name="${binname}_bottom_front_right_corner"/>
+    <joint name="${binname}_bottom_back_right_corner_joint" type="fixed">
+      <parent link="${binname}"/>
+      <child link="${binname}_bottom_back_right_corner"/>
+      <origin rpy="0.0 0.0 0.0" xyz="${-bin3_half_length} ${bin3_half_width} 0.0 "/>
+    </joint>
+    <link name="${binname}_bottom_back_right_corner"/>
+    <joint name="${binname}_bottom_back_left_corner_joint" type="fixed">
+      <parent link="${binname}"/>
+      <child link="${binname}_bottom_back_left_corner"/>
+      <origin rpy="0.0 0.0 0.0" xyz="${-bin3_half_length} ${-bin3_half_width} 0.0 "/>
+    </joint>
+    <link name="${binname}_bottom_back_left_corner"/>
+    <joint name="${binname}_bottom_front_left_corner_joint" type="fixed">
+      <parent link="${binname}"/>
+      <child link="${binname}_bottom_front_left_corner"/>
+      <origin rpy="0.0 0.0 0.0" xyz="${bin3_half_length-.045} ${-bin3_half_width} 0.0 "/>
+    </joint>
+    <link name="${binname}_bottom_front_left_corner"/>
+    <joint name="${binname}_top_front_right_corner_joint" type="fixed">
+      <parent link="${binname}"/>
+      <child link="${binname}_top_front_right_corner"/>
+      <origin rpy="0.0 0.0 0.0" xyz="${bin3_half_length-.045} ${bin3_half_width} ${bin3_height_internal} "/>
+    </joint>
+    <link name="${binname}_top_front_right_corner"/>
+    <joint name="${binname}_top_back_right_corner_joint" type="fixed">
+      <parent link="${binname}"/>
+      <child link="${binname}_top_back_right_corner"/>
+      <origin rpy="0.0 0.0 0.0" xyz="${-bin3_half_length} ${bin3_half_width} ${bin3_height_internal} "/>
+    </joint>
+    <link name="${binname}_top_back_right_corner"/>
+    <joint name="${binname}_top_back_left_corner_joint" type="fixed">
+      <parent link="${binname}"/>
+      <child link="${binname}_top_back_left_corner"/>
+      <origin rpy="0.0 0.0 0.0" xyz="${-bin3_half_length} ${-bin3_half_width} ${bin3_height_internal} "/>
+    </joint>
+    <link name="${binname}_top_back_left_corner"/>
+    <joint name="${binname}_top_front_left_corner_joint" type="fixed">
+      <parent link="${binname}"/>
+      <child link="${binname}_top_front_left_corner"/>
+      <origin rpy="0.0 0.0 0.0" xyz="${bin3_half_length-.045} ${-bin3_half_width} ${bin3_height_internal} "/>
+    </joint>
+    <link name="${binname}_top_front_left_corner"/>
   </xacro:macro>
 </robot>
