Commit message: Clean kitting bin definitions, update scene

File: o2as_scene_description/urdf/kitting_scene.xacro (robot description, xacro)
@@ -1,6 +1,7 @@
 <?xml version="1.0"?>
 <robot xmlns:xacro="http://www.ros.org/wiki/xacro" name="kitting_scene">
-  <xacro:include filename="$(find o2as_scene_description)/urdf/kitting_bin.xacro" />
-  <xacro:property name="bin_width" value=".13"/>
+  <xacro:include filename="$(find o2as_scene_description)/urdf/kitting_bins.xacro" />
+  <xacro:property name="bin_width_1" value=".13"/>
+  <xacro:property name="bin_width_2" value=".12"/>
   <!-- <xacro:include filename="$(find o2as_scene_description)/urdf/o2as_base.xacro" />
   <xacro:o2as_base boxname="test_bot_base_smfl">
@@ -9,30 +10,30 @@
   <!-- A row of bins -->
   <xacro:property name="set1_x" value=".25"/>
-  <xacro:property name="set1_y" value="${-bin_width}"/>
+  <xacro:property name="set1_y" value="${-bin_width_1}"/>
   <xacro:property name="set1_z" value=".05"/>
-  <xacro:kitting_bin binname="set1_bin1" parent="workspace_center">
+  <xacro:kitting_bin_1 binname="set1_bin1" parent="workspace_center">
     <origin xyz="${set1_x} ${set1_y} ${set1_z}" rpy="0 0 0" />
-  </xacro:kitting_bin>
-  <xacro:kitting_bin binname="set1_bin2" parent="workspace_center">
-    <origin xyz="${set1_x} ${set1_y + bin_width*1} ${set1_z}" rpy="0 0 0" />
-  </xacro:kitting_bin>
-  <xacro:kitting_bin binname="set1_bin3" parent="workspace_center">
-    <origin xyz="${set1_x} ${set1_y + bin_width*2} ${set1_z}" rpy="0 0 0" />
-  </xacro:kitting_bin>
+  </xacro:kitting_bin_1>
+  <xacro:kitting_bin_1 binname="set1_bin2" parent="workspace_center">
+    <origin xyz="${set1_x} ${set1_y + bin_width_1*1} ${set1_z}" rpy="0 0 0" />
+  </xacro:kitting_bin_1>
+  <xacro:kitting_bin_1 binname="set1_bin3" parent="workspace_center">
+    <origin xyz="${set1_x} ${set1_y + bin_width_1*2} ${set1_z}" rpy="0 0 0" />
+  </xacro:kitting_bin_1>
   <!-- Another row of bins -->
   <xacro:property name="set2_x" value=".4"/>
-  <xacro:property name="set2_y" value="${-bin_width*3/2}"/>
+  <xacro:property name="set2_y" value="${-bin_width_2*3/2}"/>
   <xacro:property name="set2_z" value=".1"/>
-  <xacro:kitting_bin binname="set2_bin1" parent="workspace_center">
+  <xacro:kitting_bin_2 binname="set2_bin1" parent="workspace_center">
     <origin xyz="${set2_x} ${set2_y} ${set2_z}" rpy="0 0 0" />
-  </xacro:kitting_bin>
-  <xacro:kitting_bin binname="set2_bin2" parent="workspace_center">
-    <origin xyz="${set2_x} ${set2_y + bin_width*1} ${set2_z}" rpy="0 0 0" />
-  </xacro:kitting_bin>
-  <xacro:kitting_bin binname="set2_bin3" parent="workspace_center">
-    <origin xyz="${set2_x} ${set2_y + bin_width*2} ${set2_z}" rpy="0 0 0" />
-  </xacro:kitting_bin>
-  <xacro:kitting_bin binname="set2_bin4" parent="workspace_center">
-    <origin xyz="${set2_x} ${set2_y + bin_width*3} ${set2_z}" rpy="0 0 0" />
-  </xacro:kitting_bin>
+  </xacro:kitting_bin_2>
+  <xacro:kitting_bin_2 binname="set2_bin2" parent="workspace_center">
+    <origin xyz="${set2_x} ${set2_y + bin_width_2*1} ${set2_z}" rpy="0 0 0" />
+  </xacro:kitting_bin_2>
+  <xacro:kitting_bin_2 binname="set2_bin3" parent="workspace_center">
+    <origin xyz="${set2_x} ${set2_y + bin_width_2*2} ${set2_z}" rpy="0 0 0" />
+  </xacro:kitting_bin_2>
+  <xacro:kitting_bin_2 binname="set2_bin4" parent="workspace_center">
+    <origin xyz="${set2_x} ${set2_y + bin_width_2*3} ${set2_z}" rpy="0 0 0" />
+  </xacro:kitting_bin_2>
 </robot>

Commit message: Partitions and a screw holder are attached to kitting trays.

File: o2as_scene_description/urdf/kitting_scene.xacro (robot description, xacro)
@@ -2,5 +2,7 @@
 <robot xmlns:xacro="http://www.ros.org/wiki/xacro" name="kitting_scene">
   <xacro:include filename="$(find o2as_scene_description)/urdf/kitting_bins.xacro" />
-  <xacro:include filename="$(find o2as_scene_description)/urdf/kitting_tray.xacro" />
+  <!-- <xacro:include filename="$(find o2as_scene_description)/urdf/kitting_tray.xacro" /> -->
+  <xacro:include filename="$(find o2as_scene_description)/urdf/kitting_tray1.xacro" />
+  <xacro:include filename="$(find o2as_scene_description)/urdf/kitting_tray2.xacro" />
   <xacro:property name="bin1_width" value=".125"/>
   <xacro:property name="bin1_length" value=".128" />
@@ -69,10 +71,16 @@
   <xacro:property name="set3_z" value=".007" />
   <!-- set3_tray_1 -->
-  <xacro:kitting_tray trayname="set3_tray_1" parent="workspace_center">
+  <!-- <xacro:kitting_tray trayname="set3_tray_1" parent="workspace_center"> -->
+  <!--   <origin xyz="${set3_x} ${set3_y} ${set3_z}" rpy="0 0 0" /> -->
+  <!-- </xacro:kitting_tray> -->
+  <xacro:kitting_tray1 trayname="set3_tray_1" parent="workspace_center">
     <origin xyz="${set3_x} ${set3_y} ${set3_z}" rpy="0 0 0" />
-  </xacro:kitting_tray>
+  </xacro:kitting_tray1>
   <!-- set3_tray_2 -->
-  <xacro:kitting_tray trayname="set3_tray_2" parent="workspace_center">
+  <!-- <xacro:kitting_tray trayname="set3_tray_2" parent="workspace_center"> -->
+  <!--   <origin xyz="${set3_x} ${set3_y-tray_width} ${set3_z}" rpy="0 0 0" /> -->
+  <!-- </xacro:kitting_tray> -->
+  <xacro:kitting_tray2 trayname="set3_tray_2" parent="workspace_center">
     <origin xyz="${set3_x} ${set3_y-tray_width} ${set3_z}" rpy="0 0 0" />
-  </xacro:kitting_tray>
+  </xacro:kitting_tray2>
 </robot>

File: o2as_scene_description/urdf/o2as_base_scene.urdf.xacro (robot description, xacro)
@@ -21,5 +21,6 @@
   <!-- Scene items (trays, bins...) -->
   <xacro:include filename="$(find o2as_scene_description)/urdf/walls.xacro" />
-  <xacro:include filename="$(find o2as_scene_description)/urdf/taskboard_scene.xacro" />
+  <!-- <xacro:include filename="$(find o2as_scene_description)/urdf/taskboard_scene.xacro" /> -->
+  <xacro:include filename="$(find o2as_scene_description)/urdf/kitting_scene.xacro" />
   <!-- Robot bases -->
   <!-- Putting these at height 0.0 makes them intersect with the ground, so they are elevated. -->

Commit message: WIP: update kitting scene.
I have a problem.
D435 'alminum is not unique'

File: o2as_scene_description/urdf/kitting_scene.xacro (robot description, xacro)
@@ -2,5 +2,7 @@
 <robot xmlns:xacro="http://www.ros.org/wiki/xacro" name="kitting_scene">
   <xacro:include filename="$(find o2as_scene_description)/urdf/kitting_bins.xacro" />
-  <xacro:include filename="$(find o2as_scene_description)/urdf/kitting_tray.xacro" />
+  <!-- <xacro:include filename="$(find o2as_scene_description)/urdf/kitting_tray.xacro" /> -->
+  <xacro:include filename="$(find o2as_scene_description)/urdf/kitting_tray_with_partitions.xacro" />
+    <xacro:include filename="$(find realsense2_camera)/urdf/_d435.urdf.xacro" />
   <xacro:property name="bin1_width" value=".125"/>
   <xacro:property name="bin1_length" value=".128" />
@@ -11,7 +13,7 @@
   <xacro:property name="tray_width" value=".300" />
   <xacro:property name="tray_length" value=".210" />
-  <xacro:property name="rack_width" value=".640" />
+  <!-- <xacro:property name="rack_width" value=".640" /> -->
   <!-- A row of bin1 -->
-  <xacro:property name="set1_x" value=".00"/>
+  <xacro:property name="set1_x" value="+0.05"/>
   <xacro:property name="set1_y" value="${.32-bin1_width/2}"/>
   <xacro:property name="set1_z" value=".01" />
@@ -38,6 +40,6 @@
   </xacro:kitting_bin_1>
   <!-- A row of bin2 and bin3 -->
-  <xacro:property name="set2_x_bin3" value="${bin1_length/2+bin3_length/2}" />
-  <xacro:property name="set2_x_bin2" value="${bin1_length/2+bin2_length/2}" />
+  <xacro:property name="set2_x_bin3" value="${bin1_length/2+bin3_length/2+0.05}" />
+  <xacro:property name="set2_x_bin2" value="${bin1_length/2+bin2_length/2+0.05}" />
   <xacro:property name="set2_y" value="${.32-bin3_width/2}" />
   <xacro:property name="set2_z" value=".00" />
@@ -64,15 +66,31 @@
     <origin xyz="${set2_x_bin2} ${set2_y-bin3_width/2-bin2_width*7/2} ${set2_z - z_origin_offset_2}" rpy="0 0 0" />
   </xacro:kitting_bin_2>
+  <!-- add camera for pose matching on the table -->
+  <link name="workspace_cam_holder_link" />
+  <joint name="workspace_cam_holder_joint" type="fixed">
+    <parent link="workspace_center" />
+    <child  link="workspace_cam_holder_link" />
+    <origin xyz="-0.05 0 0.0" rpy="0.0 -${pi/2} 0.0" />
+  </joint>
+  <xacro:sensor_d435 prefix="workspace_" parent="workspace_cam_holder_link">
+    <origin xyz="0 0 0" rpy="0 0 0"/>
+  </xacro:sensor_d435>
   <!-- A row of tray -->
-  <xacro:property name="set3_x" value="${-(bin1_length/2+tray_length/2)}" />
+  <xacro:property name="set3_x" value="${-(bin1_length/2+tray_length/2)-0.05}" />
   <xacro:property name="set3_y" value="${.32-tray_width/2}" />
   <xacro:property name="set3_z" value=".007" />
   <!-- set3_tray_1 -->
-  <xacro:kitting_tray trayname="set3_tray_1" parent="workspace_center">
+  <!-- <xacro:kitting_tray trayname="set3_tray_1" parent="workspace_center"> -->
+  <!--   <origin xyz="${set3_x} ${set3_y} ${set3_z}" rpy="0 0 0" /> -->
+  <!-- </xacro:kitting_tray> -->
+  <xacro:kitting_tray1 trayname="set3_tray_1" parent="workspace_center">
     <origin xyz="${set3_x} ${set3_y} ${set3_z}" rpy="0 0 0" />
-  </xacro:kitting_tray>
+  </xacro:kitting_tray1>
   <!-- set3_tray_2 -->
-  <xacro:kitting_tray trayname="set3_tray_2" parent="workspace_center">
+  <!-- <xacro:kitting_tray trayname="set3_tray_2" parent="workspace_center"> -->
+  <!--   <origin xyz="${set3_x} ${set3_y-tray_width} ${set3_z}" rpy="0 0 0" /> -->
+  <!-- </xacro:kitting_tray> -->
+  <xacro:kitting_tray2 trayname="set3_tray_2" parent="workspace_center">
     <origin xyz="${set3_x} ${set3_y-tray_width} ${set3_z}" rpy="0 0 0" />
-  </xacro:kitting_tray>
+  </xacro:kitting_tray2>
 </robot>

Commit message: Add bins generator for kitting task

File: o2as_scene_description/urdf/kitting_scene.xacro (robot description, xacro)
@@ -1,67 +1,70 @@
 <?xml version="1.0"?>
 <robot xmlns:xacro="http://www.ros.org/wiki/xacro" name="kitting_scene">
-  <xacro:include filename="$(find o2as_scene_description)/urdf/kitting_bins.xacro" />
+  <xacro:include filename="$(find o2as_scene_description)/urdf/kitting_bin.xacro" />
   <xacro:include filename="$(find o2as_scene_description)/urdf/kitting_tray.xacro" />
-  <xacro:property name="bin1_width" value=".125"/>
-  <xacro:property name="bin1_length" value=".128" />
-  <xacro:property name="bin2_width" value=".112" />
-  <xacro:property name="bin2_length" value=".201" />
-  <xacro:property name="bin3_width" value=".192" />
-  <xacro:property name="bin3_length" value=".285" />
+  <xacro:property name="rack_width" value=".640" />
   <xacro:property name="tray_width" value=".300" />
   <xacro:property name="tray_length" value=".210" />
-  <xacro:property name="rack_width" value=".640" />
-  <!-- A row of bin1 -->
-  <xacro:property name="set1_x" value=".00"/>
-  <xacro:property name="set1_y" value="${.32-bin1_width/2}"/>
-  <xacro:property name="set1_z" value=".01" />
-  <xacro:property name="z_origin_offset_1" value="-.008" />
-  <!-- set1_bin1_1 -->
-  <xacro:kitting_bin_1 binname="set1_bin1_1" parent="workspace_center" z_origin_offset="${z_origin_offset_1}">
-    <origin xyz="${set1_x} ${set1_y} ${set1_z - z_origin_offset_1}" rpy="0 0 0" />
+ <!-- space for bin -->
+ <!-- bin1_definition -->
+ <xacro:property name="bin1_width" value="0.125"/>
+ <xacro:property name="bin1_length" value="0.128"/>
+ <xacro:property name="z_origin_offset_1" value="-.008" />
+ <!-- bin2_definition -->
+ <xacro:property name="bin2_width" value="0.112"/>
+ <xacro:property name="bin2_length" value="0.201"/>
+ <xacro:property name="z_origin_offset_2" value="-.009" />
+ <!-- bin3_definition -->
+ <xacro:property name="bin3_width" value="0.192"/>
+ <xacro:property name="bin3_length" value="0.285"/>
+ <xacro:property name="z_origin_offset_3" value="-.004" />
+ <!-- A row of bin1 -->
+ <xacro:property name="set1_x" value=".0"/>
+ <xacro:property name="set1_y" value="0.36"/>
+ <xacro:property name="set1_z" value=".01"/>
+ <!-- A row of bin2 -->
+ <xacro:property name="set2_x" value=".20"/>
+ <xacro:property name="set2_y" value="0.36"/>
+ <xacro:property name="set2_z" value=".00"/>
+ <!--set1_bin1_1_-->
+  <xacro:kitting_bin_1 binname="set1_bin1_1" parent="workspace_center" z_origin_offset="-.008">
+      <origin xyz=".0 0.2975 0.018" rpy="0 0 0" />
   </xacro:kitting_bin_1>
-  <!-- set1_bin1_2 -->
-  <xacro:kitting_bin_1 binname="set1_bin1_2" parent="workspace_center" z_origin_offset="${z_origin_offset_1}">
-    <origin xyz="${set1_x} ${set1_y - bin1_width*1} ${set1_z - z_origin_offset_1}" rpy="0 0 0" />
+  <!--set1_bin1_2_-->
+  <xacro:kitting_bin_1 binname="set1_bin1_2" parent="workspace_center" z_origin_offset="-.008">
+      <origin xyz=".0 0.1725 0.018" rpy="0 0 0" />
   </xacro:kitting_bin_1>
-  <!-- set1_bin1_3 -->
-  <xacro:kitting_bin_1 binname="set1_bin1_3" parent="workspace_center" z_origin_offset="${z_origin_offset_1}">
-    <origin xyz="${set1_x} ${set1_y - bin1_width*2} ${set1_z - z_origin_offset_1}" rpy="0 0 0" />
+  <!--set1_bin1_3_-->
+  <xacro:kitting_bin_1 binname="set1_bin1_3" parent="workspace_center" z_origin_offset="-.008">
+      <origin xyz=".0 0.0475 0.018" rpy="0 0 0" />
   </xacro:kitting_bin_1>
-  <!-- set1_bin1_4 -->
-  <xacro:kitting_bin_1 binname="set1_bin1_4" parent="workspace_center" z_origin_offset="${z_origin_offset_1}">
-    <origin xyz="${set1_x} ${set1_y - bin1_width*3} ${set1_z - z_origin_offset_1}" rpy="0 0 0" />
+  <!--set1_bin1_4_-->
+  <xacro:kitting_bin_1 binname="set1_bin1_4" parent="workspace_center" z_origin_offset="-.008">
+      <origin xyz=".0 -0.0775 0.018" rpy="0 0 0" />
   </xacro:kitting_bin_1>
-  <!-- set1_bin1_5 -->
-  <xacro:kitting_bin_1 binname="set1_bin1_5" parent="workspace_center" z_origin_offset="${z_origin_offset_1}">
-    <origin xyz="${set1_x} ${set1_y - bin1_width*4} ${set1_z - z_origin_offset_1}" rpy="0 0 0" />
+  <!--set1_bin1_5_-->
+  <xacro:kitting_bin_1 binname="set1_bin1_5" parent="workspace_center" z_origin_offset="-.008">
+      <origin xyz=".0 -0.2025 0.018" rpy="0 0 0" />
   </xacro:kitting_bin_1>
-  <!-- A row of bin2 and bin3 -->
-  <xacro:property name="set2_x_bin3" value="${bin1_length/2+bin3_length/2}" />
-  <xacro:property name="set2_x_bin2" value="${bin1_length/2+bin2_length/2}" />
-  <xacro:property name="set2_y" value="${.32-bin3_width/2}" />
-  <xacro:property name="set2_z" value=".00" />
-  <xacro:property name="z_origin_offset_2" value="-.009" />
-  <xacro:property name="z_origin_offset_3" value="-.004" />
-  <!-- set2_bin3 -->
-  <xacro:kitting_bin_3 binname="set2_bin3" parent="workspace_center" z_origin_offset="${z_origin_offset_3}">
-    <origin xyz="${set2_x_bin3} ${set2_y} ${set2_z - z_origin_offset_3}" rpy="0 0 0" />
+  <!--set2_bin2_1_-->
+  <xacro:kitting_bin_2 binname="set2_bin2_1" parent="workspace_center" z_origin_offset="-.009">
+      <origin xyz=".20 0.304 0.009" rpy="0 0 0" />
+  </xacro:kitting_bin_2>
+  <!--set2_bin2_2_-->
+  <xacro:kitting_bin_2 binname="set2_bin2_2" parent="workspace_center" z_origin_offset="-.009">
+      <origin xyz=".20 0.192 0.009" rpy="0 0 0" />
+  </xacro:kitting_bin_2>
+  <!--set2_bin2_3_-->
+  <xacro:kitting_bin_2 binname="set2_bin2_3" parent="workspace_center" z_origin_offset="-.009">
+      <origin xyz=".20 0.08 0.009" rpy="0 0 0" />
+  </xacro:kitting_bin_2>
+  <!--set2_bin2_4_-->
+  <xacro:kitting_bin_2 binname="set2_bin2_4" parent="workspace_center" z_origin_offset="-.009">
+      <origin xyz=".20 -0.032 0.009" rpy="0 0 0" />
+  </xacro:kitting_bin_2>
+  <!--set2_bin3_1_-->
+  <xacro:kitting_bin_3 binname="set2_bin3_1" parent="workspace_center" z_origin_offset="-.004">
+      <origin xyz=".20 -0.184 0.004" rpy="0 0 0" />
   </xacro:kitting_bin_3>
-  <!-- set2_bin2_1 -->
-  <xacro:kitting_bin_2 binname="set2_bin2_1" parent="workspace_center" z_origin_offset="${z_origin_offset_2}">
-    <origin xyz="${set2_x_bin2} ${set2_y-bin3_width/2-bin2_width/2*1} ${set2_z - z_origin_offset_2}" rpy="0 0 0" />
-  </xacro:kitting_bin_2>
-  <!-- set2_bin2_2 -->
-  <xacro:kitting_bin_2 binname="set2_bin2_2" parent="workspace_center" z_origin_offset="${z_origin_offset_2}">
-    <origin xyz="${set2_x_bin2} ${set2_y-bin3_width/2-bin2_width*3/2} ${set2_z - z_origin_offset_2}" rpy="0 0 0" />
-  </xacro:kitting_bin_2>
-  <!-- set2_bin2_3 -->
-  <xacro:kitting_bin_2 binname="set2_bin2_3" parent="workspace_center" z_origin_offset="${z_origin_offset_2}">
-    <origin xyz="${set2_x_bin2} ${set2_y-bin3_width/2-bin2_width*5/2} ${set2_z - z_origin_offset_2}" rpy="0 0 0" />
-  </xacro:kitting_bin_2>
-  <!-- set2_bin2_4 -->
-  <xacro:kitting_bin_2 binname="set2_bin2_4" parent="workspace_center" z_origin_offset="${z_origin_offset_2}">
-    <origin xyz="${set2_x_bin2} ${set2_y-bin3_width/2-bin2_width*7/2} ${set2_z - z_origin_offset_2}" rpy="0 0 0" />
-  </xacro:kitting_bin_2>
   <!-- A row of tray -->
   <xacro:property name="set3_x" value="${-(bin1_length/2+tray_length/2)}" />

File: o2as_scene_description/urdf/o2as_base_scene.urdf.xacro (robot description, xacro)
@@ -21,5 +21,7 @@
   <!-- Scene items (trays, bins...) -->
   <xacro:include filename="$(find o2as_scene_description)/urdf/walls.xacro" />
-  <xacro:include filename="$(find o2as_scene_description)/urdf/taskboard_scene.xacro" />
+  <!-- <xacro:include filename="$(find o2as_scene_description)/urdf/taskboard_scene.xacro" /> -->
+  <xacro:include filename="$(find o2as_scene_description)/urdf/kitting_scene.xacro" />
+  <!-- <xacro:include filename="$(find o2as_scene_description)/urdf/kitting_scene_old.xacro" /> -->
   <!-- Robot bases -->
   <!-- Putting these at height 0.0 makes them intersect with the ground, so they are elevated. -->
@@ -59,7 +61,7 @@
     <origin xyz=".45 .05 .05" rpy="0 0 0" />
   </xacro:screw_feeder>
-  <!-- <xacro:screw_feeder feedername="m5_feeder" parent="c_bot_base_smfl">
+  <xacro:screw_feeder feedername="m5_feeder" parent="c_bot_base_smfl">
     <origin xyz=".45 .2 .05" rpy="0 0 0" />
-  </xacro:screw_feeder> -->
+  </xacro:screw_feeder>
   <!-- robot arms -->
   <xacro:ur5_robot prefix="a_bot_" joint_limited="true"
