Commit message: Update suction operation.

File: o2as_scene_description/urdf/kitting_scene.xacro (robot description, xacro)
@@ -13,57 +13,82 @@
   <xacro:property name="tray_width" value=".300" />
   <xacro:property name="tray_length" value=".210" />
-  <!-- <xacro:property name="rack_width" value=".640" /> -->
-  <!-- A row of bin1 -->
-  <xacro:property name="set1_x" value="+0.05"/>
+  <xacro:property name="z_origin_offset_1" value="-.008" />
+  <xacro:property name="z_origin_offset_2" value="-.009" />
+  <xacro:property name="z_origin_offset_3" value="-.004" />
+  <xacro:property name="set1_x" value="${bin3_length/2}" />
+  <xacro:property name="set1_y" value="${-.33 + bin3_width / 2}" />
+  <xacro:property name="set1_z" value="0.01" />
+  <xacro:kitting_bin_3 binname="part_6" parent="workspace_center" z_origin_offset="${z_origin_offset_3}">
+    <origin xyz="${set1_x} ${set1_y} ${set1_z - z_origin_offset_3}" rpy="0 0 ${pi}" />
+  </xacro:kitting_bin_3>
+  <xacro:kitting_bin_2 binname="part_4" parent="workspace_center" z_origin_offset="${z_origin_offset_2}">
+    <origin xyz="${set1_x} ${set1_y + bin3_width / 2 + bin2_width / 2} ${set1_z - z_origin_offset_2}" rpy="0 0 ${pi}" />
+  </xacro:kitting_bin_2>
+  <xacro:kitting_bin_2 binname="part_8" parent="workspace_center" z_origin_offset="${z_origin_offset_2}">
+    <origin xyz="${set1_x} ${set1_y + bin3_width / 2 + 3 * bin2_width / 2} ${set1_z - z_origin_offset_2}" rpy="0 0 ${pi}" />
+  </xacro:kitting_bin_2>
+  <xacro:kitting_bin_2 binname="part_11" parent="workspace_center" z_origin_offset="${z_origin_offset_2}">
+    <origin xyz="${set1_x} ${set1_y + bin3_width / 2 + 5 * bin2_width / 2} ${set1_z - z_origin_offset_2}" rpy="0 0 ${pi}" />
+  </xacro:kitting_bin_2>
+  <xacro:kitting_bin_2 binname="part_13" parent="workspace_center" z_origin_offset="${z_origin_offset_2}">
+    <origin xyz="${set1_x} ${set1_y + bin3_width / 2 + 7 * bin2_width / 2} ${set1_z - z_origin_offset_2}" rpy="0 0 ${pi}" />
+  </xacro:kitting_bin_2>
+  <xacro:property name="set2_x" value="${.42-bin1_length/2}" />
+  <xacro:property name="set2_y" value="0" />
+  <xacro:property name="set2_z" value="0.01" />
+  <xacro:kitting_bin_1 binname="part_9" parent="workspace_center" z_origin_offset="${z_origin_offset_1}">
+    <origin xyz="${set2_x} ${set2_y} ${set2_z - z_origin_offset_1}" rpy="0 0 ${pi}" />
+  </xacro:kitting_bin_1>
+  <xacro:kitting_bin_1 binname="part_12" parent="workspace_center" z_origin_offset="${z_origin_offset_1}">
+    <origin xyz="${set2_x} ${set2_y - bin1_width} ${set2_z - z_origin_offset_1}" rpy="0 0 ${pi}" />
+  </xacro:kitting_bin_1>
+  <xacro:kitting_bin_1 binname="part_16" parent="workspace_center" z_origin_offset="${z_origin_offset_1}">
+    <origin xyz="${set2_x} ${set2_y + bin1_width} ${set2_z - z_origin_offset_1}" rpy="0 0 ${pi}" />
+  </xacro:kitting_bin_1>
+  <xacro:kitting_bin_1 binname="part_17" parent="workspace_center" z_origin_offset="${z_origin_offset_1}">
+    <origin xyz="${set2_x} ${set2_y - 2 * bin1_width} ${set2_z - z_origin_offset_1}" rpy="0 0 ${pi}" />
+  </xacro:kitting_bin_1>
+  <xacro:kitting_bin_1 binname="part_18" parent="workspace_center" z_origin_offset="${z_origin_offset_1}">
+    <origin xyz="${set2_x} ${set2_y + 2 * bin1_width} ${set2_z - z_origin_offset_1}" rpy="0 0 ${pi}" />
+  </xacro:kitting_bin_1>
+  <!-- <xacro:property name="set1_x" value="+0.05"/>
   <xacro:property name="set1_y" value="${.32-bin1_width/2}"/>
   <xacro:property name="set1_z" value=".01" />
-  <xacro:property name="z_origin_offset_1" value="-.008" />
-  <!-- set1_bin1_1 -->
   <xacro:kitting_bin_1 binname="set1_bin1_1" parent="workspace_center" z_origin_offset="${z_origin_offset_1}">
     <origin xyz="${set1_x} ${set1_y} ${set1_z - z_origin_offset_1}" rpy="0 0 0" />
   </xacro:kitting_bin_1>
-  <!-- set1_bin1_2 -->
   <xacro:kitting_bin_1 binname="set1_bin1_2" parent="workspace_center" z_origin_offset="${z_origin_offset_1}">
     <origin xyz="${set1_x} ${set1_y - bin1_width*1} ${set1_z - z_origin_offset_1}" rpy="0 0 0" />
   </xacro:kitting_bin_1>
-  <!-- set1_bin1_3 -->
   <xacro:kitting_bin_1 binname="set1_bin1_3" parent="workspace_center" z_origin_offset="${z_origin_offset_1}">
     <origin xyz="${set1_x} ${set1_y - bin1_width*2} ${set1_z - z_origin_offset_1}" rpy="0 0 0" />
   </xacro:kitting_bin_1>
-  <!-- set1_bin1_4 -->
   <xacro:kitting_bin_1 binname="set1_bin1_4" parent="workspace_center" z_origin_offset="${z_origin_offset_1}">
     <origin xyz="${set1_x} ${set1_y - bin1_width*3} ${set1_z - z_origin_offset_1}" rpy="0 0 0" />
   </xacro:kitting_bin_1>
-  <!-- set1_bin1_5 -->
   <xacro:kitting_bin_1 binname="set1_bin1_5" parent="workspace_center" z_origin_offset="${z_origin_offset_1}">
     <origin xyz="${set1_x} ${set1_y - bin1_width*4} ${set1_z - z_origin_offset_1}" rpy="0 0 0" />
-  </xacro:kitting_bin_1>
+  </xacro:kitting_bin_1> -->
   <!-- A row of bin2 and bin3 -->
-  <xacro:property name="set2_x_bin3" value="${bin1_length/2+bin3_length/2+0.05}" />
+  <!-- <xacro:property name="set2_x_bin3" value="${bin1_length/2+bin3_length/2+0.05}" />
   <xacro:property name="set2_x_bin2" value="${bin1_length/2+bin2_length/2+0.05}" />
   <xacro:property name="set2_y" value="${.32-bin3_width/2}" />
   <xacro:property name="set2_z" value=".00" />
-  <xacro:property name="z_origin_offset_2" value="-.009" />
-  <xacro:property name="z_origin_offset_3" value="-.004" />
-  <!-- set2_bin3 -->
-  <xacro:kitting_bin_3 binname="set2_bin3" parent="workspace_center" z_origin_offset="${z_origin_offset_3}">
+   -->
+  <!-- <xacro:kitting_bin_3 binname="set2_bin3" parent="workspace_center" z_origin_offset="${z_origin_offset_3}">
     <origin xyz="${set2_x_bin3} ${set2_y} ${set2_z - z_origin_offset_3}" rpy="0 0 0" />
   </xacro:kitting_bin_3>
-  <!-- set2_bin2_1 -->
   <xacro:kitting_bin_2 binname="set2_bin2_1" parent="workspace_center" z_origin_offset="${z_origin_offset_2}">
     <origin xyz="${set2_x_bin2} ${set2_y-bin3_width/2-bin2_width/2*1} ${set2_z - z_origin_offset_2}" rpy="0 0 0" />
   </xacro:kitting_bin_2>
-  <!-- set2_bin2_2 -->
   <xacro:kitting_bin_2 binname="set2_bin2_2" parent="workspace_center" z_origin_offset="${z_origin_offset_2}">
     <origin xyz="${set2_x_bin2} ${set2_y-bin3_width/2-bin2_width*3/2} ${set2_z - z_origin_offset_2}" rpy="0 0 0" />
   </xacro:kitting_bin_2>
-  <!-- set2_bin2_3 -->
   <xacro:kitting_bin_2 binname="set2_bin2_3" parent="workspace_center" z_origin_offset="${z_origin_offset_2}">
     <origin xyz="${set2_x_bin2} ${set2_y-bin3_width/2-bin2_width*5/2} ${set2_z - z_origin_offset_2}" rpy="0 0 0" />
   </xacro:kitting_bin_2>
-  <!-- set2_bin2_4 -->
   <xacro:kitting_bin_2 binname="set2_bin2_4" parent="workspace_center" z_origin_offset="${z_origin_offset_2}">
     <origin xyz="${set2_x_bin2} ${set2_y-bin3_width/2-bin2_width*7/2} ${set2_z - z_origin_offset_2}" rpy="0 0 0" />
-  </xacro:kitting_bin_2>
+  </xacro:kitting_bin_2> -->
   <!-- add camera for pose matching on the table -->
   <link name="workspace_cam_holder_link" />

Commit message: WIP: various fixed to aist robots.

File: o2as_scene_description/urdf/kitting_scene.xacro (robot description, xacro)
@@ -8,5 +8,5 @@
   <xacro:include filename="$(find o2as_scene_description)/urdf/dual_suction_gripper.urdf.xacro" />
   <xacro:dual_suction_gripper_o2as prefix="b_bot_" parent = "b_bot_ee_link">
-    <origin xyz="0 0 0" rpy="0 0 0"/>
+    <origin xyz="0 0 0" rpy="${pi/2} 0 0"/>
   </xacro:dual_suction_gripper_o2as>
   <xacro:property name="tray_width" value=".300" />

File: o2as_scene_description/urdf/o2as_base_scene.urdf.xacro (robot description, xacro)
@@ -139,5 +139,5 @@
   <xacro:include filename="$(find o2as_scene_description)/urdf/phoxi_m_camera.urdf.xacro" />
   <xacro:phoxi_m_camera prefix="a_" parent="o2as_ground">
-    <origin xyz="0.46 0 ${bots_z + .1 + .8}" rpy="${-160*pi/180} 0 ${pi/2}"/>
+    <origin xyz="0.61696890577  0.17103542533 1.42309125675" rpy="-2.626594398897875 0.2001733992896885 1.5970042364211503"/>
   </xacro:phoxi_m_camera>
   <!-- I would like to remove the "world" link definition, but apparently it is necessary for Gazebo -->

Commit message: Add suction tool, kitting scene and rough calibration

File: o2as_scene_description/urdf/kitting_scene.xacro (robot description, xacro)
@@ -6,24 +6,13 @@
   <xacro:include filename="$(find o2as_scene_description)/urdf/o2as_box.xacro"/>
   <!-- spawn and attach dual suction grippers -->
-  <xacro:include filename="$(find o2as_scene_description)/urdf/dual_suction_gripper.urdf.xacro" />
+  <!-- <xacro:include filename="$(find o2as_scene_description)/urdf/dual_suction_gripper.urdf.xacro" />
   <xacro:dual_suction_gripper_o2as prefix="b_bot_" parent = "b_bot_ee_link">
     <origin xyz="0 0 0" rpy="${pi/2} 0 0"/>
-  </xacro:dual_suction_gripper_o2as>
+  </xacro:dual_suction_gripper_o2as> -->
   <xacro:property name="tray_width" value=".300" />
   <xacro:property name="tray_length" value=".210" />
-  <!-- add camera for pose matching on the table -->
-  <link name="workspace_cam_holder_link" />
-  <joint name="workspace_cam_holder_joint" type="fixed">
-    <parent link="workspace_center" />
-    <child  link="workspace_cam_holder_link" />
-    <origin xyz="0 0 0" rpy="0.0 -${pi/2} 0.0" />
-  </joint>
-  <xacro:sensor_d435 prefix="workspace_" parent="workspace_cam_holder_link">
-    <origin xyz="0 0 0" rpy="0 0 0"/>
-  </xacro:sensor_d435>
-  <!-- TODO: Deal with this camera? -->
   <!-- add tray rack -->
   <xacro:o2as_box boxname="rack_trays" box_w="0.21" box_l="0.60" box_h=".015" parent="workspace_center">
-    <origin xyz="-.26 -0.3 0" rpy="0 0 0" />
+    <origin xyz="-.33 -0.3 0" rpy="0 0 0" />
   </xacro:o2as_box>
   <link name="rack_trays_center" />
@@ -34,12 +23,11 @@
   </joint>
   <!-- add trays -->
-  <xacro:property name="set3_x" value="${-tray_length-.05}" />
-  <xacro:property name="set3_y" value="0" />
-  <xacro:property name="set3_z" value="0.015" />
-  <xacro:kitting_tray1 trayname="set3_tray_1" parent="workspace_center">
-    <origin xyz="${set3_x} ${set3_y} ${set3_z}" rpy="0 0 0" />
+  <xacro:property name="tray_x" value="${-tray_length+.01}" />
+  <xacro:property name="tray_y" value="0" />
+  <xacro:kitting_tray1 trayname="tray_1" parent="rack_trays_center">
+    <origin xyz="${tray_x} ${tray_y} 0" rpy="0 0 0" />
   </xacro:kitting_tray1>
-  <xacro:kitting_tray2 trayname="set3_tray_2" parent="workspace_center">
-    <origin xyz="${set3_x} ${set3_y-tray_width} ${set3_z}" rpy="0 0 0" />
+  <xacro:kitting_tray2 trayname="tray_2" parent="rack_trays_center">
+    <origin xyz="+.01 0 0" rpy="0 0 ${pi}" />
   </xacro:kitting_tray2>
 </robot>

File: o2as_scene_description/urdf/o2as_base_scene.urdf.xacro (robot description, xacro)
@@ -117,5 +117,5 @@
   <xacro:include filename="$(find o2as_scene_description)/urdf/robotiq_b_bot_gripper.urdf.xacro" />
   <xacro:include filename="$(find o2as_scene_description)/urdf/robotiq_c_bot_gripper.urdf.xacro" />
-  <!-- <xacro:o2as_b_bot_gripper prefix="b_bot_" parent = "b_bot_ee_link" /> -->
+  <xacro:o2as_b_bot_gripper prefix="b_bot_" parent = "b_bot_ee_link" />
   <xacro:o2as_c_bot_gripper prefix="c_bot_" parent = "c_bot_ee_link"/>
   <!-- Add cameras -->
@@ -135,14 +135,14 @@
   <!-- spawn and attach AR markers -->
   <xacro:include filename="$(find o2as_gazebo)/urdf/o2as_ar_marker.urdf.xacro"/>
-  <xacro:o2as_ar_marker prefix="a_bot_"
+  <!-- <xacro:o2as_ar_marker prefix="a_bot_"
 			parent="a_bot_ee_link"
 			marker_id="17">
     <origin xyz="0.25 0.0 0.047" rpy="0 0 0"/>
-  </xacro:o2as_ar_marker>
-  <xacro:o2as_ar_marker prefix="b_bot_"
+  </xacro:o2as_ar_marker> -->
+  <!-- <xacro:o2as_ar_marker prefix="b_bot_"
 			parent="b_bot_dual_suction_gripper_base_link"
 			marker_id="26">
     <origin xyz="0.063 0.0 0.0215" rpy="0 0 0"/>
-  </xacro:o2as_ar_marker>
+  </xacro:o2as_ar_marker> -->
   <!-- <xacro:o2as_ar_marker prefix="b_bot_" -->
   <!-- 			parent="b_bot_single_suction_gripper_base_link" -->
@@ -150,9 +150,9 @@
   <!--   <origin xyz="0.063 0.0 0.0215" rpy="0 0 0"/> -->
   <!-- </xacro:o2as_ar_marker> -->
-  <xacro:o2as_ar_marker prefix="c_bot_"
+  <!-- <xacro:o2as_ar_marker prefix="c_bot_"
 			parent="c_bot_robotiq_85_tip_link"
 			marker_id="256">
     <origin xyz="0.0 0.0 0.0185" rpy="0 0 0"/>
-  </xacro:o2as_ar_marker>
+  </xacro:o2as_ar_marker> -->
   <!-- Add PhoXi 3D scanners -->
   <xacro:include filename="$(find o2as_scene_description)/urdf/phoxi_m_camera.urdf.xacro" />

File: o2as_scene_description/urdf/robotiq_b_bot_gripper.urdf.xacro (robot description, xacro)
@@ -39,4 +39,16 @@
     </joint>
     <link name="${prefix}set_screw_tool_tip_link"/>
+    <joint name="${prefix}robotiq_85_suction_tool_tip_joint" type="fixed">
+      <parent link="${prefix}robotiq_85_tip_link"/>
+      <child link="${prefix}suction_tool_tip_link"/>
+      <origin rpy="0.0 ${pi/2} 0.0" xyz="${dx+.008} 0.0 -0.126 "/>
+    </joint>
+    <link name="${prefix}suction_tool_tip_link"/>
+    <joint name="${prefix}dual_suction_gripper_pad_joint" type="fixed">
+      <parent link="${prefix}suction_tool_tip_link"/>
+      <child link="${prefix}dual_suction_gripper_pad_link"/>
+      <origin rpy="0.0 0 0.0" xyz="0 0 0 "/>
+    </joint>
+    <link name="${prefix}dual_suction_gripper_pad_link"/>
   </xacro:macro>
 </robot>

File: o2as_scene_description/urdf/screw_tools.xacro (robot description, xacro)
@@ -101,4 +101,32 @@
     <origin xyz="-0.05 ${tool_offset} 0.004" rpy="0.0 0.0 0.0" />
   </joint>
+    <link name="suction_tool_link">
+    <inertial>
+      <origin rpy="0 0 0" xyz="0 0 0"/>
+      <mass value="1.0"/>
+      <inertia ixx="1" ixy="0" ixz="0" iyy="1" iyz="0" izz="1"/>
+    </inertial>
+    <visual>
+      <origin rpy="${pi/2} 0 ${-pi/2}" xyz=".03 0.04 -.104"/>
+      <!-- <origin rpy="0 0 0" xyz=".104 -.015 0"/> -->
+      <geometry>
+        <mesh filename="package://o2as_scene_description/meshes/single_suction_gripper.stl" scale="0.001 0.001 0.001"/>
+      </geometry>
+      <material name="white">
+        <color rgba=".9 .9 .9 1"/>
+      </material>
+    </visual>
+    <collision>
+      <origin rpy="0 0 0" xyz="0 ${bit_cushion_to_axis - .02} .0275"/>
+      <geometry>
+        <box size=".026 .04 .055"/>
+      </geometry>
+    </collision>
+  </link>
+  <joint name="suction_tool_to_holder" type="fixed">
+    <parent link="screw_tool_holder" />
+    <child link="suction_tool_link" />
+    <origin xyz="-0.05 ${tool_offset} 0.004" rpy="0.0 0.0 0.0" />
+  </joint>
   <link name="screw_tool_m4_link">
     <inertial>
@@ -180,3 +208,9 @@
     <origin xyz="0.0 0.0 0.0" rpy="0.0 0.0 ${-pi/2}" />
   </joint>
+  <link name="suction_tool_helper_link"/>
+  <joint name="suction_tool_helper_joint" type="fixed">
+    <parent link="suction_tool_link" />
+    <child link="suction_tool_helper_link" />
+    <origin xyz="0.0 0.0 0.0" rpy="0.0 0.0 ${-pi/2}" />
+  </joint>
 </robot>

Commit message: Fix kitting scene, add joint poses

File: o2as_scene_description/urdf/kitting_scene.xacro (robot description, xacro)
@@ -31,8 +31,8 @@
   </xacro:kitting_tray2>
   <xacro:kitting_tray2 trayname="set_3_tray_2" parent="rack_trays_center">
-    <origin xyz="+.01 ${tray_width} 0" rpy="0 0 ${pi}" />
+    <origin xyz="${tray_length+.01} ${tray_width} -.01" rpy="0 0 ${pi}" />
   </xacro:kitting_tray2>
   <xacro:kitting_tray1 trayname="set_1_tray_1" parent="rack_trays_center">
-    <origin xyz="+.01 0 -.01" rpy="0 0 0" />
+    <origin xyz="${-tray_length+.01} 0 0" rpy="0 0 0" />
   </xacro:kitting_tray1>
   <xacro:kitting_tray1 trayname="set_2_tray_1" parent="b_bot_base">

Commit message: Add kitting strategy
This should run completely in simulation.

File: o2as_scene_description/urdf/kitting_scene.xacro (robot description, xacro)
@@ -5,4 +5,12 @@
   <xacro:include filename="$(find realsense2_camera)/urdf/_d435.urdf.xacro" />
   <xacro:include filename="$(find o2as_scene_description)/urdf/o2as_box.xacro"/>
+  <!-- Screw feeders -->
+  <xacro:include filename="$(find o2as_scene_description)/urdf/screw_feeder.xacro" />
+  <xacro:screw_feeder feedername="m3_feeder" parent="c_bot_base_smfl">
+    <origin xyz=".66 -0.25 .065" rpy="0 0 ${pi/2}" />
+  </xacro:screw_feeder>
+  <xacro:screw_feeder feedername="m4_feeder" parent="c_bot_base_smfl">
+    <origin xyz=".52 -0.25 .065" rpy="0 0 ${pi/2}" />
+  </xacro:screw_feeder>
   <!-- spawn and attach dual suction grippers -->
   <!-- <xacro:include filename="$(find o2as_scene_description)/urdf/dual_suction_gripper.urdf.xacro" />
@@ -28,8 +36,8 @@
   </xacro:kitting_tray2>
   <xacro:kitting_tray2 trayname="set_2_tray_2" parent="rack_trays_center">
-    <origin xyz="${tray_length+.01} 0 -.01" rpy="0 0 ${pi}" />
+    <origin xyz="${tray_length+.01} 0 0" rpy="0 0 ${pi}" />
   </xacro:kitting_tray2>
   <xacro:kitting_tray2 trayname="set_3_tray_2" parent="rack_trays_center">
-    <origin xyz="${tray_length+.01} ${tray_width} -.01" rpy="0 0 ${pi}" />
+    <origin xyz="${tray_length+.01} ${tray_width} 0" rpy="0 0 ${pi}" />
   </xacro:kitting_tray2>
   <xacro:kitting_tray1 trayname="set_1_tray_1" parent="rack_trays_center">
@@ -37,8 +45,8 @@
   </xacro:kitting_tray1>
   <xacro:kitting_tray1 trayname="set_2_tray_1" parent="b_bot_base">
-    <origin xyz=".55 ${tray_length-.1} 0.01" rpy="0 0 ${pi/2}" />
+    <origin xyz=".55 -.1 0.01" rpy="0 0 ${pi/2}" />
   </xacro:kitting_tray1>
   <xacro:kitting_tray1 trayname="set_3_tray_1" parent="b_bot_base">
-    <origin xyz=".55 -.1 0.01" rpy="0 0 ${pi/2}" />
+    <origin xyz=".55 ${tray_length-.1} 0.01" rpy="0 0 ${pi/2}" />
   </xacro:kitting_tray1>
   <!-- <xacro:property name="tray_x" value="${-tray_length+.01}" />

File: o2as_scene_description/urdf/o2as_base_scene.urdf.xacro (robot description, xacro)
@@ -59,12 +59,4 @@
   <!-- Screw holder & screw tool visual -->
   <xacro:include filename="$(find o2as_scene_description)/urdf/screw_tools.xacro" />
-  <!-- Feeders -->
-  <xacro:include filename="$(find o2as_scene_description)/urdf/screw_feeder.xacro" />
-  <xacro:screw_feeder feedername="m3_feeder" parent="c_bot_base_smfl">
-    <origin xyz=".66 -0.25 .065" rpy="0 0 ${pi/2}" />
-  </xacro:screw_feeder>
-  <xacro:screw_feeder feedername="m4_feeder" parent="c_bot_base_smfl">
-    <origin xyz=".52 -0.25 .065" rpy="0 0 ${pi/2}" />
-  </xacro:screw_feeder>
   <!-- robot arms -->
   <xacro:ur5_robot prefix="a_bot_" joint_limited="false"

File: o2as_scene_description/urdf/screw_feeder.xacro (robot description, xacro)
@@ -72,9 +72,13 @@
     <parent link="${feedername}_link"/>
     <child link="${feedername}_outlet_link"/>
-    <!-- <origin rpy="0.0 0 0.0" xyz="${length-.01} ${width/2} ${height/2 + .02}"/> -->
-    <!-- <origin rpy="0.0 ${pi/2} 0.0" xyz="${-height/2 - .02} ${width/2} ${length-.01}"/> -->
     <origin rpy="0.0 ${pi/2} 0.0" xyz="${length-.01} ${width/2} ${height/2}"/>
   </joint>
   <link name="${feedername}_outlet_link"/>
+  <joint name="${feedername}_inlet_joint" type="fixed">
+    <parent link="${feedername}_link"/>
+    <child link="${feedername}_inlet_link"/>
+    <origin rpy="0.0 0.0 0.0" xyz="${length/3} ${width/3} ${height}"/>
+  </joint>
+  <link name="${feedername}_inlet_link"/>
   </xacro:macro>
 </robot>

Commit message: Add intermediate poses for suction

File: o2as_scene_description/urdf/kitting_scene.xacro (robot description, xacro)
@@ -36,11 +36,11 @@
   </xacro:kitting_tray2>
   <xacro:kitting_tray2 trayname="set_2_tray_2" parent="rack_trays_center">
-    <origin xyz="${tray_length+.01} 0 0" rpy="0 0 ${pi}" />
+    <origin xyz="${tray_length+.02} 0 -.01" rpy="0 0 ${pi}" />
   </xacro:kitting_tray2>
   <xacro:kitting_tray2 trayname="set_3_tray_2" parent="rack_trays_center">
-    <origin xyz="${tray_length+.01} ${tray_width} 0" rpy="0 0 ${pi}" />
+    <origin xyz="${tray_length+.02} ${tray_width} -.01" rpy="0 0 ${pi}" />
   </xacro:kitting_tray2>
   <xacro:kitting_tray1 trayname="set_1_tray_1" parent="rack_trays_center">
-    <origin xyz="${-tray_length+.01} 0 0" rpy="0 0 0" />
+    <origin xyz="${-tray_length+.02} 0 0" rpy="0 0 0" />
   </xacro:kitting_tray1>
   <xacro:kitting_tray1 trayname="set_2_tray_1" parent="b_bot_base">

File: o2as_scene_description/urdf/robotiq_b_bot_gripper.urdf.xacro (robot description, xacro)
@@ -42,5 +42,5 @@
       <parent link="${prefix}robotiq_85_tip_link"/>
       <child link="${prefix}suction_tool_tip_link"/>
-      <origin rpy="0.0 ${pi/2} 0.0" xyz="${dx+.013} 0.0 -0.131 "/>
+      <origin rpy="0.0 ${pi/2} 0.0" xyz="${dx+.008} 0.0 -0.131 "/>
     </joint>
     <link name="${prefix}suction_tool_tip_link"/>

Commit message: Improve kitting speed, fix bugs

File: o2as_scene_description/urdf/kitting_scene.xacro (robot description, xacro)
@@ -36,8 +36,8 @@
   </xacro:kitting_tray2>
   <xacro:kitting_tray2 trayname="set_2_tray_2" parent="rack_trays_center">
-    <origin xyz="${tray_length+.02} 0 -.01" rpy="0 0 ${pi}" />
+    <origin xyz="${tray_length+.02} 0 -.015" rpy="0 0 ${pi}" />
   </xacro:kitting_tray2>
   <xacro:kitting_tray2 trayname="set_3_tray_2" parent="rack_trays_center">
-    <origin xyz="${tray_length+.02} ${tray_width} -.01" rpy="0 0 ${pi}" />
+    <origin xyz="${tray_length+.02} ${tray_width} -.015" rpy="0 0 ${pi}" />
   </xacro:kitting_tray2>
   <xacro:kitting_tray1 trayname="set_1_tray_1" parent="rack_trays_center">
