Commit message: Misc + cleanup. Works, but LIN motion jumps

File: o2as_scene_description/urdf/screw_tools.xacro (robot description, xacro)
@@ -110,3 +110,22 @@
     <origin xyz="-0.1 0.0 0.0" rpy="0.0 0.0 0.0" />
   </joint>
+  <!-- Extra links to position the gripper more simply -->
+  <link name="screw_tool_m3_helper_link"/>
+  <joint name="screw_tool_m3_helper_joint" type="fixed">
+    <parent link="screw_tool_m3_link" />
+    <child link="screw_tool_m3_helper_link" />
+    <origin xyz="0.0 0.0 0.0" rpy="0.0 0.0 ${-pi/2}" />
+  </joint>
+  <link name="screw_tool_m4_helper_link"/>
+  <joint name="screw_tool_m4_helper_joint" type="fixed">
+    <parent link="screw_tool_m4_link" />
+    <child link="screw_tool_m4_helper_link" />
+    <origin xyz="0.0 0.0 0.0" rpy="0.0 0.0 ${-pi/2}" />
+  </joint>
+  <link name="screw_tool_m5_helper_link"/>
+  <joint name="screw_tool_m5_helper_joint" type="fixed">
+    <parent link="screw_tool_m5_link" />
+    <child link="screw_tool_m5_helper_link" />
+    <origin xyz="0.0 0.0 0.0" rpy="0.0 0.0 ${-pi/2}" />
+  </joint>
 </robot>

Commit message: Update suction tool model

File: o2as_scene_description/urdf/screw_tools.xacro (robot description, xacro)
@@ -108,8 +108,7 @@
     </inertial>
     <visual>
-      <origin rpy="${pi/2} 0 ${-pi/2}" xyz=".03 0.04 -.104"/>
-      <!-- <origin rpy="0 0 0" xyz=".104 -.015 0"/> -->
-      <geometry>
-        <mesh filename="package://o2as_scene_description/meshes/single_suction_gripper.stl" scale="0.001 0.001 0.001"/>
+      <origin rpy="${pi/2} 0 ${-pi/2}" xyz="0 0.009 0.047"/>
+      <geometry>
+        <mesh filename="package://o2as_scene_description/meshes/suction_tool_phi10.stl" scale="0.001 0.001 0.001"/>
       </geometry>
       <material name="white">

Commit message: WIP: Update suction tool holder

File: o2as_scene_description/urdf/screw_tools.xacro (robot description, xacro)
@@ -126,5 +126,5 @@
     <parent link="screw_tool_holder" />
     <child link="suction_tool_link" />
-    <origin xyz="-0.05 ${tool_offset} 0.004" rpy="0.0 0.0 0.0" />
+    <origin xyz="-0.355 ${tool_offset} 0.004" rpy="0.0 0.0 0.0" />
   </joint>
   <link name="screw_tool_m4_link">

Commit message: Fix bug, add set screw tool to skill server

File: o2as_scene_description/urdf/screw_tools.xacro (robot description, xacro)
@@ -101,5 +101,5 @@
     <origin xyz="-0.05 ${tool_offset} 0.004" rpy="0.0 0.0 0.0" />
   </joint>
-    <link name="suction_tool_link">
+  <link name="suction_tool_link">
     <inertial>
       <origin rpy="0 0 0" xyz="0 0 0"/>
@@ -127,4 +127,16 @@
     <child link="suction_tool_link" />
     <origin xyz="-0.355 ${tool_offset - .015} 0.004" rpy="0.0 0.0 0.0" />
+  </joint>
+  <link name="set_screw_tool_link">
+    <inertial>
+      <origin rpy="0 0 0" xyz="0 0 0"/>
+      <mass value="1.0"/>
+      <inertia ixx="1" ixy="0" ixz="0" iyy="1" iyz="0" izz="1"/>
+    </inertial>
+  </link>
+  <joint name="set_screw_tool_to_holder" type="fixed">
+    <parent link="screw_tool_holder" />
+    <child link="set_screw_tool_link" />
+    <origin xyz="-0.355 ${tool_offset- .015} 0.004" rpy="0.0 0.0 0.0" />
   </joint>
   <link name="screw_tool_m4_link">
@@ -213,3 +225,9 @@
     <origin xyz="0.0 0.0 0.0" rpy="0.0 0.0 ${-pi/2}" />
   </joint>
+  <link name="set_screw_tool_helper_link"/>
+  <joint name="set_screw_tool_helper_joint" type="fixed">
+    <parent link="set_screw_tool_link" />
+    <child link="set_screw_tool_helper_link" />
+    <origin xyz="0.0 0.0 0.0" rpy="0.0 0.0 ${-pi/2}" />
+  </joint>
 </robot>
