Commit message: Improved taskboard

File: o2as_scene_description/urdf/task_board.xacro (robot description, xacro)
@@ -28,8 +28,8 @@
   </link>
   <joint name="${boardname}" type="fixed">
-      <parent link="${parent}" />
-      <child link = "${boardname}" />
-      <xacro:insert_block name="origin"/>
-    </joint>
+    <parent link="${parent}" />
+    <child link = "${boardname}" />
+    <xacro:insert_block name="origin"/>
+  </joint>
   <joint name="${boardname}_part1" type="fixed">
     <parent link="${boardname}"/>
@@ -59,17 +59,39 @@
     <parent link="${boardname}"/>
     <child link="${boardname}_part5"/>
-    <origin rpy="0.0 0.0 ${pi/2}" xyz="0.07 0.26 0.01"/>
+    <origin rpy="0.0 0.0 ${pi/2}" xyz="0.07 0.26 0.0145"/>
   </joint>
   <link name="${boardname}_part5"/>
-  <joint name="${boardname}_part6" type="fixed">
+  <!--  -->
+  <joint name="${boardname}_part6_small_pulley" type="fixed">
     <parent link="${boardname}"/>
-    <child link="${boardname}_part6"/>
-    <origin rpy="0.0 0.0 ${pi/2}" xyz="0.2 0.2 0.01"/>
+    <child link="${boardname}_part6_small_pulley"/>
+    <origin rpy="0.0 0.0 ${pi/2}" xyz="0.06 0.06 0.0085"/>
   </joint>
-  <link name="${boardname}_part6"/>
+  <link name="${boardname}_part6_small_pulley"/>
+  <joint name="${boardname}_part6_large_pulley" type="fixed">
+    <parent link="${boardname}"/>
+    <child link="${boardname}_part6_large_pulley"/>
+    <origin rpy="0.0 0.0 ${pi/2}" xyz="0.188 0.06 0.0085"/>
+  </joint>
+  <link name="${boardname}_part6_large_pulley"/>
+  <!--  -->
+  <!--  -->
+  <joint name="${boardname}_part7a" type="fixed">
+    <parent link="${boardname}"/>
+    <child link="${boardname}_part7a"/>
+    <origin rpy="0.0 0.0 ${pi/2}" xyz="0.335 0.056 0.05"/>
+  </joint>
+  <link name="${boardname}_part7a"/>
+  <joint name="${boardname}_part7b" type="fixed">
+    <parent link="${boardname}"/>
+    <child link="${boardname}_part7b"/>
+    <origin rpy="0.0 0.0 ${pi/2}" xyz="0.338 0.056 0.05"/>
+  </joint>
+  <link name="${boardname}_part7b"/>
+  <!--  -->
   <joint name="${boardname}_part8" type="fixed">
     <parent link="${boardname}"/>
     <child link="${boardname}_part8"/>
-    <origin rpy="0.0 0.0 ${pi/2}" xyz="0.32 0.25 0.01"/>
+    <origin rpy="0.0 0.0 ${pi/2}" xyz="0.32 0.25 0.022"/>
   </joint>
   <link name="${boardname}_part8"/>
@@ -77,5 +99,5 @@
     <parent link="${boardname}"/>
     <child link="${boardname}_part9"/>
-    <origin rpy="0.0 0.0 ${pi/2}" xyz="0.26 0.15 0.01"/>
+    <origin rpy="0.0 0.0 ${pi/2}" xyz="0.26 0.15 0.019"/>
   </joint>
   <link name="${boardname}_part9"/>
@@ -83,5 +105,5 @@
     <parent link="${boardname}"/>
     <child link="${boardname}_part10"/>
-    <origin rpy="0.0 0.0 ${pi/2}" xyz="0.16 0.36 0.01"/>
+    <origin rpy="0.0 0.0 ${pi/2}" xyz="0.16 0.36 0.06"/>
   </joint>
   <link name="${boardname}_part10"/>
@@ -107,5 +129,5 @@
     <parent link="${boardname}"/>
     <child link="${boardname}_part14"/>
-    <origin rpy="0.0 0.0 ${pi/2}" xyz="0.23 0.23 0.01"/>
+    <origin rpy="0.0 0.0 ${pi/2}" xyz="0.23 0.23 0.06"/>
   </joint>
   <link name="${boardname}_part14"/>

Commit message: Add gripper calibration, fix offset problem

File: o2as_scene_description/urdf/task_board.xacro (robot description, xacro)
@@ -156,5 +156,5 @@
     <parent link="${boardname}_surface"/>
     <child link="${boardname}_part10"/>
-    <origin rpy="0.0 0.0 ${pi/2}" xyz="0.16 0.36 0.05"/>
+    <origin rpy="0.0 0.0 ${pi/2}" xyz="0.16 0.36 0.0515"/>
   </joint>
   <link name="${boardname}_part10">
@@ -188,5 +188,5 @@
     <parent link="${boardname}_surface"/>
     <child link="${boardname}_part14"/>
-    <origin rpy="0.0 0.0 ${pi/2}" xyz="0.23 0.23 0.05"/>
+    <origin rpy="0.0 0.0 ${pi/2}" xyz="0.23 0.23 0.0515"/>
   </joint>
   <link name="${boardname}_part14">

Commit message: Correct frame in taskboard

File: o2as_scene_description/urdf/task_board.xacro (robot description, xacro)
@@ -218,5 +218,5 @@
     <parent link="${boardname}_surface"/>
     <child link="${boardname}_part15"/>
-    <origin rpy="0.0 0.0 ${pi/2}" xyz="0.16 0.36 0.05"/>
+    <origin rpy="0.0 0.0 ${pi/2}" xyz="0.16 0.36 0.0515"/>
   </joint>
   <link name="${boardname}_part15"/>

Commit message: First successful belt insertion

File: o2as_scene_description/urdf/task_board.xacro (robot description, xacro)
@@ -41,10 +41,4 @@
   </joint>
   <link name="${boardname}_part1"/>
-  <joint name="${boardname}_tool" type="fixed">
-    <parent link="${boardname}_surface"/>
-    <child link="${boardname}_tool"/>
-    <origin rpy="0.0 0.0 ${pi/2}" xyz="-0.07 0.0 -0.02"/>
-  </joint>
-  <link name="${boardname}_tool"/>
   <joint name="${boardname}_part2" type="fixed">
     <parent link="${boardname}_surface"/>

File: o2as_scene_description/urdf/taskboard_scene.xacro (robot description, xacro)
@@ -15,3 +15,9 @@
     <origin xyz="0.0 0.41 0.0" rpy="0 0 0" />
   </xacro:o2as_mat>
+  <joint name="belt_placement_tool" type="fixed">
+    <parent link="taskboard"/>
+    <child link="belt_placement_tool"/>
+    <origin rpy="0.0 0.0 ${pi/2}" xyz="-0.07 0.0 0.0"/>
+  </joint>
+  <link name="belt_placement_tool"/>
 </robot>

Commit message: add seq 2,12,13. Left: 6,7,2(put the tool on the taskboard

File: o2as_scene_description/urdf/task_board.xacro (robot description, xacro)
@@ -114,5 +114,5 @@
     <parent link="${boardname}_surface"/>
     <child link="${boardname}_part7_1"/>
-    <origin rpy="0.0 0.0 ${pi/2}" xyz="0.362 0.056 0.05"/>
+    <origin rpy="0.0 0.0 0" xyz="0.362 0.056 0.05"/>
   </joint>
   <link name="${boardname}_part7_1"/>
@@ -120,9 +120,9 @@
     <parent link="${boardname}_surface"/>
     <child link="${boardname}_part7_2"/>
-    <origin rpy="0.0 0.0 ${pi/2}" xyz="0.365 0.056 0.05"/>
+    <origin rpy="0.0 0.0 ${pi}" xyz="0.365 0.056 0.05"/>
   </joint>
   <link name="${boardname}_part7_2">
     <visual>
-      <origin xyz="0 0.0015 -.015" rpy="0 0 0"/>
+      <origin xyz="0 0.0015 -.015" rpy="0 0 ${pi/2}"/>
       <geometry>
         <box size=".015 0.003 .07"/>
@@ -191,5 +191,5 @@
     <parent link="${boardname}_surface"/>
     <child link="${boardname}_part12"/>
-    <origin rpy="0.0 0.0 ${pi/2}" xyz="0.14 0.14 0.0"/>
+    <origin rpy="0.0 ${pi/2} ${pi/2}" xyz="0.14 0.14 0.0"/>
   </joint>
   <link name="${boardname}_part12"/>
@@ -197,5 +197,5 @@
     <parent link="${boardname}_surface"/>
     <child link="${boardname}_part13"/>
-    <origin rpy="0.0 0.0 ${pi/2}" xyz="0.07 0.26 0.078"/>
+    <origin rpy="0.0 ${pi/2} ${pi/2}" xyz="0.07 0.26 0.078"/>
   </joint>
   <link name="${boardname}_part13"/>

Commit message: WIP: Update taskboard definition

File: o2as_scene_description/urdf/task_board.xacro (robot description, xacro)
@@ -1,3 +1,2 @@
-<?xml version="1.0"?>
 <robot xmlns:xacro="http://www.ros.org/wiki/xacro" name="task_board">
   <xacro:macro name="task_board" params="boardname parent *origin">
@@ -36,4 +35,192 @@
   </joint>
   <link name="${boardname}_surface"/>
+  <joint name="${boardname}_part1" type="fixed">
+    <parent link="${boardname}_surface"/>
+    <child link="${boardname}_part1"/>
+    <origin rpy="0.0 0.0 ${pi/2}" xyz="0.34 0.34 0.0"/>
+  </joint>
+  <link name="${boardname}_part1"/>
+  <joint name="${boardname}_part2" type="fixed">
+    <parent link="${boardname}_surface"/>
+    <child link="${boardname}_part2"/>
+    <origin rpy="0.0 0.0 ${pi/2}" xyz="0.05 0.35 0.0"/>
+  </joint>
+  <link name="${boardname}_part2"/>
+  <joint name="${boardname}_part3" type="fixed">
+    <parent link="${boardname}_surface"/>
+    <child link="${boardname}_part3"/>
+    <origin rpy="0.0 0.0 ${pi/2}" xyz="0.08 0.31 0.0"/>
+  </joint>
+  <link name="${boardname}_part3"/>
+  <joint name="${boardname}_part4" type="fixed">
+    <parent link="${boardname}_surface"/>
+    <child link="${boardname}_part4"/>
+    <origin rpy="0.0 0.0 ${pi/2}" xyz="0.15 0.28 0.0"/>
+  </joint>
+  <link name="${boardname}_part4"/>
+  <joint name="${boardname}_part5" type="fixed">
+    <parent link="${boardname}_surface"/>
+    <child link="${boardname}_part5"/>
+    <origin rpy="0.0 0.0 ${pi/2}" xyz="0.07 0.26 0.002"/>
+  </joint>
+  <link name="${boardname}_part5">
+    <visual>
+      <origin xyz="0 0 .0375" rpy="0 0 0"/>
+      <geometry>
+        <!-- <cylinder length=".0045" radius=".002"/>  -->
+        <cylinder length=".075" radius=".005"/>
+      </geometry>
+      <material name="grey">
+        <color rgba=".3 .3 .3 1"/>
+      </material>
+    </visual>
+  </link>
+  <!-- The pulleys for the belt -->
+  <joint name="${boardname}_part6_small_pulley" type="fixed">
+    <parent link="${boardname}_surface"/>
+    <child link="${boardname}_part6_small_pulley"/>
+    <origin rpy="0.0 0.0 ${pi/2}" xyz="0.06 0.06 0.0085"/>
+  </joint>
+  <link name="${boardname}_part6_small_pulley">
+    <visual>
+      <origin xyz="0 0 -.00475" rpy="0 0 0"/>
+      <geometry>
+        <cylinder length=".0085" radius=".016"/>
+      </geometry>
+      <material name="grey">
+        <color rgba=".3 .3 .3 1"/>
+      </material>
+    </visual>
+  </link>
+  <joint name="${boardname}_part6_large_pulley" type="fixed">
+    <parent link="${boardname}_surface"/>
+    <child link="${boardname}_part6_large_pulley"/>
+    <origin rpy="0.0 0.0 ${pi/2}" xyz="0.188 0.06 0.0085"/>
+  </joint>
+  <link name="${boardname}_part6_large_pulley">
+    <visual>
+      <origin xyz="0 0 -.00475" rpy="0 0 0"/>
+      <geometry>
+        <cylinder length=".0085" radius=".031"/>
+      </geometry>
+      <material name="grey">
+        <color rgba=".3 .3 .3 1"/>
+      </material>
+    </visual>
+  </link>
+  <!-- ======== -->
+  <!-- The nut and bolt on the metal sheet -->
+  <joint name="${boardname}_part7_1" type="fixed">
+    <parent link="${boardname}_surface"/>
+    <child link="${boardname}_part7_1"/>
+    <origin rpy="0.0 0.0 0" xyz="0.362 0.056 0.05"/>
+  </joint>
+  <link name="${boardname}_part7_1"/>
+  <joint name="${boardname}_part7_2" type="fixed">
+    <parent link="${boardname}_surface"/>
+    <child link="${boardname}_part7_2"/>
+    <origin rpy="0.0 0.0 ${pi}" xyz="0.365 0.056 0.05"/>
+  </joint>
+  <link name="${boardname}_part7_2">
+    <visual>
+      <origin xyz="0 0.0015 -.015" rpy="0 0 ${pi/2}"/>
+      <geometry>
+        <box size=".015 0.003 .07"/>
+      </geometry>
+      <material name="grey">
+        <color rgba=".3 .3 .3 1"/>
+      </material>
+    </visual>
+  </link>
+  <!-- ======== -->
+  <joint name="${boardname}_part8" type="fixed">
+    <parent link="${boardname}_surface"/>
+    <child link="${boardname}_part8"/>
+    <origin rpy="0.0 0.0 ${pi/2}" xyz="0.32 0.25 0.012"/>
+  </joint>
+  <link name="${boardname}_part8">
+    <visual>
+      <origin xyz="0 0 -.006" rpy="0 0 0"/>
+      <geometry>
+        <cylinder length=".012" radius=".006"/>
+      </geometry>
+      <material name="grey">
+        <color rgba=".3 .3 .3 1"/>
+      </material>
+    </visual>
+  </link>
+  <joint name="${boardname}_part9" type="fixed">
+    <parent link="${boardname}_surface"/>
+    <child link="${boardname}_part9"/>
+    <origin rpy="0.0 0.0 ${pi/2}" xyz="0.26 0.15 0.009"/>
+  </joint>
+  <link name="${boardname}_part9">
+    <visual>
+      <origin xyz="0 0 -.0045" rpy="0 0 0"/>
+      <geometry>
+        <cylinder length=".009" radius=".0032"/>
+      </geometry>
+      <material name="grey">
+        <color rgba=".3 .3 .3 1"/>
+      </material>
+    </visual>
+  </link>
+  <joint name="${boardname}_part10" type="fixed">
+    <parent link="${boardname}_surface"/>
+    <child link="${boardname}_part10"/>
+    <origin rpy="0.0 0.0 ${pi/2}" xyz="0.16 0.36 0.0515"/>
+  </joint>
+  <link name="${boardname}_part10">
+    <visual>
+      <origin xyz="0 0 -.025" rpy="0 0 0"/>
+      <geometry>
+        <cylinder length=".05" radius=".003"/>
+      </geometry>
+      <material name="grey">
+        <color rgba=".3 .3 .3 1"/>
+      </material>
+    </visual>
+  </link>
+  <joint name="${boardname}_part11" type="fixed">
+    <parent link="${boardname}_surface"/>
+    <child link="${boardname}_part11"/>
+    <origin rpy="0.0 0.0 ${pi/2}" xyz="0.06 0.18 0.0"/>
+  </joint>
+  <link name="${boardname}_part11"/>
+  <joint name="${boardname}_part12" type="fixed">
+    <parent link="${boardname}_surface"/>
+    <child link="${boardname}_part12"/>
+    <origin rpy="0.0 ${pi/2} ${pi/2}" xyz="0.14 0.14 0.0"/>
+  </joint>
+  <link name="${boardname}_part12"/>
+  <joint name="${boardname}_part13" type="fixed">
+    <parent link="${boardname}_surface"/>
+    <child link="${boardname}_part13"/>
+    <origin rpy="0.0 ${pi/2} ${pi/2}" xyz="0.07 0.26 0.078"/>
+  </joint>
+  <link name="${boardname}_part13"/>
+  <joint name="${boardname}_part14" type="fixed">
+    <parent link="${boardname}_surface"/>
+    <child link="${boardname}_part14"/>
+    <origin rpy="0.0 0.0 ${pi/2}" xyz="0.23 0.23 0.0515"/>
+  </joint>
+  <link name="${boardname}_part14">
+    <visual>
+      <origin xyz="0 0 -.025" rpy="0 0 0"/>
+      <geometry>
+        <cylinder length=".05" radius=".003"/>
+      </geometry>
+      <material name="grey">
+        <color rgba=".3 .3 .3 1"/>
+      </material>
+    </visual>
+  </link>
+  <joint name="${boardname}_part15" type="fixed">
+    <parent link="${boardname}_surface"/>
+    <child link="${boardname}_part15"/>
+    <origin rpy="0.0 0.0 ${pi/2}" xyz="0.07 0.26 0.0772"/>
+  </joint>
+  <link name="${boardname}_part15"/>
+   <!-- The cylinder is already defined under part10 -->
   <joint name="${boardname}_corner1" type="fixed">
     <parent link="${boardname}_surface"/>
@@ -60,189 +247,4 @@
   </joint>
   <link name="${boardname}_corner4"/>
-  <joint name="${boardname}_part1" type="fixed">
-    <parent link="${boardname}_surface"/>
-    <child link="${boardname}_part1"/>
-    <origin rpy="0.0 0.0 ${pi*0.5}" xyz="0.34 0.34 0.0"/>
-  </joint>
-  <link name="${boardname}_part1"/>
-  <joint name="${boardname}_part2" type="fixed">
-    <parent link="${boardname}_surface"/>
-    <child link="${boardname}_part2"/>
-    <origin rpy="0.0 0.0 ${pi*0.5}" xyz="0.05 0.35 0.0"/>
-  </joint>
-  <link name="${boardname}_part2"/>
-  <joint name="${boardname}_part3" type="fixed">
-    <parent link="${boardname}_surface"/>
-    <child link="${boardname}_part3"/>
-    <origin rpy="0.0 0.0 ${pi*0.5}" xyz="0.08 0.31 0.0"/>
-  </joint>
-  <link name="${boardname}_part3"/>
-  <joint name="${boardname}_part4" type="fixed">
-    <parent link="${boardname}_surface"/>
-    <child link="${boardname}_part4"/>
-    <origin rpy="0.0 0.0 ${pi*0.5}" xyz="0.15 0.28 0.0"/>
-  </joint>
-  <link name="${boardname}_part4"/>
-  <joint name="${boardname}_part5" type="fixed">
-    <parent link="${boardname}_surface"/>
-    <child link="${boardname}_part5"/>
-    <origin rpy="0.0 0.0 ${pi*0.5}" xyz="0.07 0.26 0.0045"/>
-  </joint>
-  <link name="${boardname}_part5">
-    <visual>
-      <origin xyz="0 0 .0375" rpy="0 0 0"/>
-      <geometry>
-        <!-- <cylinder length=".0045" radius=".002"/>  -->
-        <cylinder length=".075" radius=".005"/>
-      </geometry>
-      <material name="grey">
-        <color rgba=".3 .3 .3 1"/>
-      </material>
-    </visual>
-  </link>
-  <joint name="${boardname}_part15" type="fixed">
-    <parent link="${boardname}_surface"/>
-    <child link="${boardname}_part15"/>
-    <origin rpy="0.0 0.0 ${pi*0.5}" xyz="0.07 0.26 0.0515"/>
-  </joint>
-  <link name="${boardname}_part15"/>
-  <joint name="${boardname}_part6_small_pulley" type="fixed">
-    <parent link="${boardname}_surface"/>
-    <child link="${boardname}_part6_small_pulley"/>
-    <origin rpy="0.0 0.0 ${pi*0.5}" xyz="0.06 0.06 0.0085"/>
-  </joint>
-  <link name="${boardname}_part6_small_pulley">
-    <visual>
-      <origin xyz="0 0 -.00475" rpy="0 0 0"/>
-      <geometry>
-        <cylinder length=".0085" radius=".016"/>
-      </geometry>
-      <material name="grey">
-        <color rgba=".3 .3 .3 1"/>
-      </material>
-    </visual>
-  </link>
-  <joint name="${boardname}_part7_1" type="fixed">
-    <parent link="${boardname}_surface"/>
-    <child link="${boardname}_part7_1"/>
-    <origin rpy="0.0 0.0 ${pi*0.5}" xyz="0.36 0.056 0.05"/>
-  </joint>
-  <link name="${boardname}_part7_1"/>
-  <joint name="${boardname}_part8" type="fixed">
-    <parent link="${boardname}_surface"/>
-    <child link="${boardname}_part8"/>
-    <origin rpy="0.0 0.0 ${pi*0.5}" xyz="0.32 0.25 0.012"/>
-  </joint>
-  <link name="${boardname}_part8">
-    <visual>
-      <origin xyz="0 0 -.006" rpy="0 0 0"/>
-      <geometry>
-        <cylinder length=".012" radius=".006"/>
-      </geometry>
-      <material name="grey">
-        <color rgba=".3 .3 .3 1"/>
-      </material>
-    </visual>
-  </link>
-  <joint name="${boardname}_part9" type="fixed">
-    <parent link="${boardname}_surface"/>
-    <child link="${boardname}_part9"/>
-    <origin rpy="0.0 0.0 ${pi*0.5}" xyz="0.26 0.15 0.009"/>
-  </joint>
-  <link name="${boardname}_part9">
-    <visual>
-      <origin xyz="0 0 -.0045" rpy="0 0 0"/>
-      <geometry>
-        <cylinder length=".009" radius=".0032"/>
-      </geometry>
-      <material name="grey">
-        <color rgba=".3 .3 .3 1"/>
-      </material>
-    </visual>
-  </link>
-  <joint name="${boardname}_part10" type="fixed">
-    <parent link="${boardname}_surface"/>
-    <child link="${boardname}_part10"/>
-    <origin rpy="0.0 0.0 ${pi*0.5}" xyz="0.16 0.36 0.0515"/>
-  </joint>
-  <link name="${boardname}_part10">
-    <visual>
-      <origin xyz="0 0 -.025" rpy="0 0 0"/>
-      <geometry>
-        <cylinder length=".05" radius=".003"/>
-      </geometry>
-      <material name="grey">
-        <color rgba=".3 .3 .3 1"/>
-      </material>
-    </visual>
-  </link>
-  <joint name="${boardname}_part11" type="fixed">
-    <parent link="${boardname}_surface"/>
-    <child link="${boardname}_part11"/>
-    <origin rpy="0.0 0.0 ${pi*0.5}" xyz="0.06 0.18 0.0"/>
-  </joint>
-  <link name="${boardname}_part11"/>
-  <joint name="${boardname}_part12" type="fixed">
-    <parent link="${boardname}_surface"/>
-    <child link="${boardname}_part12"/>
-    <origin rpy="0.0 0.0 ${pi*0.5}" xyz="0.14 0.14 0.0"/>
-  </joint>
-  <link name="${boardname}_part12"/>
-  <joint name="${boardname}_part13" type="fixed">
-    <parent link="${boardname}_surface"/>
-    <child link="${boardname}_part13"/>
-    <origin rpy="0.0 0.0 ${pi*0.5}" xyz="0.35 0.12 0.0"/>
-  </joint>
-  <link name="${boardname}_part13"/>
-  <joint name="${boardname}_part14" type="fixed">
-    <parent link="${boardname}_surface"/>
-    <child link="${boardname}_part14"/>
-    <origin rpy="0.0 0.0 ${pi*0.5}" xyz="0.23 0.23 0.0515"/>
-  </joint>
-  <link name="${boardname}_part14">
-    <visual>
-      <origin xyz="0 0 -.025" rpy="0 0 0"/>
-      <geometry>
-        <cylinder length=".05" radius=".003"/>
-      </geometry>
-      <material name="grey">
-        <color rgba=".3 .3 .3 1"/>
-      </material>
-    </visual>
-  </link>
-  <joint name="${boardname}_part6_large_pulley" type="fixed">
-    <parent link="${boardname}_part6_small_pulley"/>
-    <child link="${boardname}_part6_large_pulley"/>
-    <origin rpy="0.0 0.0 ${pi*0.0}" xyz="0.0 -0.128 0.0"/>
-  </joint>
-  <link name="${boardname}_part6_large_pulley">
-    <visual>
-      <origin xyz="0 0 -.00475" rpy="0 0 0"/>
-      <geometry>
-        <cylinder length=".0085" radius=".031"/>
-      </geometry>
-      <material name="grey">
-        <color rgba=".3 .3 .3 1"/>
-      </material>
-    </visual>
-  </link>
-  <!-- ======== -->
-  <joint name="${boardname}_part7_2" type="fixed">
-    <parent link="${boardname}_part7_1"/>
-    <child link="${boardname}_part7_2"/>
-    <origin rpy="0.0 0.0 ${pi*0.0}" xyz="0.0 -0.003 0.0"/>
-  </joint>
-  <link name="${boardname}_part7_2">
-    <visual>
-      <origin xyz="0 0.0015 -.015" rpy="0 0 0"/>
-      <geometry>
-        <box size=".015 0.003 .07"/>
-      </geometry>
-      <material name="grey">
-        <color rgba=".3 .3 .3 1"/>
-      </material>
-    </visual>
-  </link>
-  <!-- ======== -->
   </xacro:macro>
   <!-- Add additional links for us to plan with.-->

File: o2as_scene_description/urdf/templates/taskboard_part_template/o2as_taskboard_part_5_template_tail.xacro (robot description, xacro)
@@ -1,7 +1,7 @@
   <link name="${boardname}_part5">
     <visual>
-      <origin xyz="0 0 -.00275" rpy="0 0 0"/>
+      <origin xyz="0 0 .0375" rpy="0 0 0"/>
       <geometry>
-        <cylinder length=".0045" radius=".002"/>
+        <cylinder length=".075" radius=".005"/>
       </geometry>
       <material name="grey">

File: o2as_scene_description/urdf/templates/taskboard_part_template/o2as_taskboard_part_7_2_template_tail.xacro (robot description, xacro)
@@ -1,5 +1,5 @@
   <link name="${boardname}_part7_2">
     <visual>
-      <origin xyz="0 0.0015 -.015" rpy="0 0 0"/>
+      <origin xyz="0 0.0015 -.015" rpy="0 0 {pi/2}"/>
       <geometry>
         <box size=".015 0.003 .07"/>
