Commit message: Correct taskboard_generator and add competition layout

File: o2as_scene_description/urdf/task_board.xacro (robot description, xacro)
@@ -1,2 +1,3 @@
+<?xml version="1.0"?>
 <robot xmlns:xacro="http://www.ros.org/wiki/xacro" name="task_board">
   <xacro:macro name="task_board" params="boardname parent *origin">
@@ -35,8 +36,32 @@
   </joint>
   <link name="${boardname}_surface"/>
+  <joint name="${boardname}_corner1" type="fixed">
+    <parent link="${boardname}_surface"/>
+    <child link="${boardname}_corner1"/>
+    <origin rpy="0.0 0.0 ${pi/2}" xyz="0.01 0.39 0.0"/>
+  </joint>
+  <link name="${boardname}_corner1"/>
+  <joint name="${boardname}_corner2" type="fixed">
+    <parent link="${boardname}_surface"/>
+    <child link="${boardname}_corner2"/>
+    <origin rpy="0.0 0.0 ${pi/2}" xyz="0.39 0.39 0.0"/>
+  </joint>
+  <link name="${boardname}_corner2"/>
+  <joint name="${boardname}_corner3" type="fixed">
+    <parent link="${boardname}_surface"/>
+    <child link="${boardname}_corner3"/>
+    <origin rpy="0.0 0.0 ${pi/2}" xyz="0.39 0.01 0.0"/>
+  </joint>
+  <link name="${boardname}_corner3"/>
+  <joint name="${boardname}_corner4" type="fixed">
+    <parent link="${boardname}_surface"/>
+    <child link="${boardname}_corner4"/>
+    <origin rpy="0.0 0.0 ${pi/2}" xyz="0.01 0.01 0.0"/>
+  </joint>
+  <link name="${boardname}_corner4"/>
   <joint name="${boardname}_part1" type="fixed">
     <parent link="${boardname}_surface"/>
     <child link="${boardname}_part1"/>
-    <origin rpy="0.0 0.0 ${pi/2}" xyz="0.34 0.34 0.0"/>
+    <origin rpy="0.0 0.0 ${pi*0.5}" xyz="0.33 0.33 0.0"/>
   </joint>
   <link name="${boardname}_part1"/>
@@ -44,5 +69,5 @@
     <parent link="${boardname}_surface"/>
     <child link="${boardname}_part2"/>
-    <origin rpy="0.0 0.0 ${pi/2}" xyz="0.05 0.35 0.0"/>
+    <origin rpy="0.0 0.0 ${pi*0.5}" xyz="0.06 0.36 0.0"/>
   </joint>
   <link name="${boardname}_part2"/>
@@ -50,5 +75,5 @@
     <parent link="${boardname}_surface"/>
     <child link="${boardname}_part3"/>
-    <origin rpy="0.0 0.0 ${pi/2}" xyz="0.08 0.31 0.0"/>
+    <origin rpy="0.0 0.0 ${pi*0.5}" xyz="0.09 0.3 0.0"/>
   </joint>
   <link name="${boardname}_part3"/>
@@ -56,5 +81,5 @@
     <parent link="${boardname}_surface"/>
     <child link="${boardname}_part4"/>
-    <origin rpy="0.0 0.0 ${pi/2}" xyz="0.15 0.28 0.0"/>
+    <origin rpy="0.0 0.0 ${pi*0.5}" xyz="0.16 0.27 0.0"/>
   </joint>
   <link name="${boardname}_part4"/>
@@ -62,5 +87,5 @@
     <parent link="${boardname}_surface"/>
     <child link="${boardname}_part5"/>
-    <origin rpy="0.0 0.0 ${pi/2}" xyz="0.07 0.26 0.002"/>
+    <origin rpy="0.0 0.0 ${pi*0.5}" xyz="0.05 0.25 0.002"/>
   </joint>
   <link name="${boardname}_part5">
@@ -68,5 +93,4 @@
       <origin xyz="0 0 .0375" rpy="0 0 0"/>
       <geometry>
-        <!-- <cylinder length=".0045" radius=".002"/>  -->
         <cylinder length=".075" radius=".005"/>
       </geometry>
@@ -76,9 +100,14 @@
     </visual>
   </link>
-  <!-- The pulleys for the belt -->
+  <joint name="${boardname}_part15" type="fixed">
+    <parent link="${boardname}_surface"/>
+    <child link="${boardname}_part15"/>
+    <origin rpy="0.0 0.0 ${pi*0.5}" xyz="0.05 0.25 0.0772"/>
+  </joint>
+  <link name="${boardname}_part15"/>
   <joint name="${boardname}_part6_small_pulley" type="fixed">
     <parent link="${boardname}_surface"/>
     <child link="${boardname}_part6_small_pulley"/>
-    <origin rpy="0.0 0.0 ${pi/2}" xyz="0.06 0.06 0.0085"/>
+    <origin rpy="0.0 0.0 ${pi*0.5}" xyz="0.06 0.07 0.0085"/>
   </joint>
   <link name="${boardname}_part6_small_pulley">
@@ -93,49 +122,14 @@
     </visual>
   </link>
-  <joint name="${boardname}_part6_large_pulley" type="fixed">
-    <parent link="${boardname}_surface"/>
-    <child link="${boardname}_part6_large_pulley"/>
-    <origin rpy="0.0 0.0 ${pi/2}" xyz="0.188 0.06 0.0085"/>
-  </joint>
-  <link name="${boardname}_part6_large_pulley">
-    <visual>
-      <origin xyz="0 0 -.00475" rpy="0 0 0"/>
-      <geometry>
-        <cylinder length=".0085" radius=".031"/>
-      </geometry>
-      <material name="grey">
-        <color rgba=".3 .3 .3 1"/>
-      </material>
-    </visual>
-  </link>
-  <!-- ======== -->
-  <!-- The nut and bolt on the metal sheet -->
   <joint name="${boardname}_part7_1" type="fixed">
     <parent link="${boardname}_surface"/>
     <child link="${boardname}_part7_1"/>
-    <origin rpy="0.0 0.0 0" xyz="0.362 0.056 0.05"/>
+    <origin rpy="0.0 0.0 ${pi*0.0}" xyz="0.351 0.056 0.0505"/>
   </joint>
   <link name="${boardname}_part7_1"/>
-  <joint name="${boardname}_part7_2" type="fixed">
-    <parent link="${boardname}_surface"/>
-    <child link="${boardname}_part7_2"/>
-    <origin rpy="0.0 0.0 ${pi}" xyz="0.365 0.056 0.05"/>
-  </joint>
-  <link name="${boardname}_part7_2">
-    <visual>
-      <origin xyz="0 0.0015 -.015" rpy="0 0 ${pi/2}"/>
-      <geometry>
-        <box size=".015 0.003 .07"/>
-      </geometry>
-      <material name="grey">
-        <color rgba=".3 .3 .3 1"/>
-      </material>
-    </visual>
-  </link>
-  <!-- ======== -->
   <joint name="${boardname}_part8" type="fixed">
     <parent link="${boardname}_surface"/>
     <child link="${boardname}_part8"/>
-    <origin rpy="0.0 0.0 ${pi/2}" xyz="0.32 0.25 0.012"/>
+    <origin rpy="0.0 0.0 ${pi*0.5}" xyz="0.32 0.24 0.012"/>
   </joint>
   <link name="${boardname}_part8">
@@ -153,5 +147,5 @@
     <parent link="${boardname}_surface"/>
     <child link="${boardname}_part9"/>
-    <origin rpy="0.0 0.0 ${pi/2}" xyz="0.26 0.15 0.009"/>
+    <origin rpy="0.0 0.0 ${pi*0.5}" xyz="0.28 0.13 0.009"/>
   </joint>
   <link name="${boardname}_part9">
@@ -169,5 +163,5 @@
     <parent link="${boardname}_surface"/>
     <child link="${boardname}_part10"/>
-    <origin rpy="0.0 0.0 ${pi/2}" xyz="0.16 0.36 0.0515"/>
+    <origin rpy="0.0 0.0 ${pi*0.5}" xyz="0.19 0.34 0.0515"/>
   </joint>
   <link name="${boardname}_part10">
@@ -185,5 +179,5 @@
     <parent link="${boardname}_surface"/>
     <child link="${boardname}_part11"/>
-    <origin rpy="0.0 0.0 ${pi/2}" xyz="0.06 0.18 0.0"/>
+    <origin rpy="0.0 0.0 ${pi*0.5}" xyz="0.07 0.17 0.0"/>
   </joint>
   <link name="${boardname}_part11"/>
@@ -191,5 +185,5 @@
     <parent link="${boardname}_surface"/>
     <child link="${boardname}_part12"/>
-    <origin rpy="0.0 ${pi/2} ${pi/2}" xyz="0.14 0.14 0.0"/>
+    <origin rpy="0.0 0.0 ${pi*0.5}" xyz="0.15 0.15 0.0"/>
   </joint>
   <link name="${boardname}_part12"/>
@@ -197,5 +191,5 @@
     <parent link="${boardname}_surface"/>
     <child link="${boardname}_part13"/>
-    <origin rpy="0.0 ${pi/2} ${pi/2}" xyz="0.07 0.26 0.078"/>
+    <origin rpy="0.0 0.0 ${pi*0.5}" xyz="0.05 0.25 0.078"/>
   </joint>
   <link name="${boardname}_part13"/>
@@ -203,5 +197,5 @@
     <parent link="${boardname}_surface"/>
     <child link="${boardname}_part14"/>
-    <origin rpy="0.0 0.0 ${pi/2}" xyz="0.23 0.23 0.0515"/>
+    <origin rpy="0.0 0.0 ${pi*0.5}" xyz="0.22 0.22 0.0515"/>
   </joint>
   <link name="${boardname}_part14">
@@ -216,35 +210,38 @@
     </visual>
   </link>
-  <joint name="${boardname}_part15" type="fixed">
-    <parent link="${boardname}_surface"/>
-    <child link="${boardname}_part15"/>
-    <origin rpy="0.0 0.0 ${pi/2}" xyz="0.07 0.26 0.0772"/>
-  </joint>
-  <link name="${boardname}_part15"/>
-   <!-- The cylinder is already defined under part10 -->
-  <joint name="${boardname}_corner1" type="fixed">
-    <parent link="${boardname}_surface"/>
-    <child link="${boardname}_corner1"/>
-    <origin rpy="0.0 0.0 ${pi/2}" xyz="0.01 0.39 0.0"/>
-  </joint>
-  <link name="${boardname}_corner1"/>
-  <joint name="${boardname}_corner2" type="fixed">
-    <parent link="${boardname}_surface"/>
-    <child link="${boardname}_corner2"/>
-    <origin rpy="0.0 0.0 ${pi/2}" xyz="0.39 0.39 0.0"/>
-  </joint>
-  <link name="${boardname}_corner2"/>
-  <joint name="${boardname}_corner3" type="fixed">
-    <parent link="${boardname}_surface"/>
-    <child link="${boardname}_corner3"/>
-    <origin rpy="0.0 0.0 ${pi/2}" xyz="0.39 0.01 0.0"/>
-  </joint>
-  <link name="${boardname}_corner3"/>
-  <joint name="${boardname}_corner4" type="fixed">
-    <parent link="${boardname}_surface"/>
-    <child link="${boardname}_corner4"/>
-    <origin rpy="0.0 0.0 ${pi/2}" xyz="0.01 0.01 0.0"/>
-  </joint>
-  <link name="${boardname}_corner4"/>
+  <joint name="${boardname}_part6_large_pulley" type="fixed">
+    <parent link="${boardname}_part6_small_pulley"/>
+    <child link="${boardname}_part6_large_pulley"/>
+    <origin rpy="0.0 0.0 ${pi*0.0}" xyz="0.0 -0.128 0.0"/>
+  </joint>
+  <link name="${boardname}_part6_large_pulley">
+    <visual>
+      <origin xyz="0 0 -.00475" rpy="0 0 0"/>
+      <geometry>
+        <cylinder length=".0085" radius=".031"/>
+      </geometry>
+      <material name="grey">
+        <color rgba=".3 .3 .3 1"/>
+      </material>
+    </visual>
+  </link>
+  <!-- ======== -->
+  <joint name="${boardname}_part7_2" type="fixed">
+    <parent link="${boardname}_part7_1"/>
+    <child link="${boardname}_part7_2"/>
+    <origin rpy="0.0 0.0 ${pi*1.0}" xyz="0.003 0.0 0.0"/>
+  </joint>
+  <link name="${boardname}_part7_2">
+    <visual>
+      <origin xyz="0.0015 0 -0.0125" rpy="0 0 ${pi/2}"/>
+      <geometry>
+        <box size=".025 0.003 .076"/>
+      </geometry>
+      <material name="grey">
+        <color rgba=".3 .3 .3 1"/>
+      </material>
+    </visual>
+  </link>
+  <!-- ======== -->
   </xacro:macro>
   <!-- Add additional links for us to plan with.-->

File: o2as_scene_description/urdf/templates/taskboard_part_template/o2as_taskboard_part_7_2_template_tail.xacro (robot description, xacro)
@@ -1,7 +1,7 @@
   <link name="${boardname}_part7_2">
     <visual>
-      <origin xyz="0 0.0015 -.015" rpy="0 0 {pi/2}"/>
+      <origin xyz="0.0015 0 -0.0125" rpy="0 0 ${pi/2}"/>
       <geometry>
-        <box size=".015 0.003 .07"/>
+        <box size=".025 0.003 .076"/>
       </geometry>
       <material name="grey">

Commit message: Fix taskboard screw frames

File: o2as_scene_description/urdf/task_board.xacro (robot description, xacro)
@@ -63,5 +63,5 @@
     <parent link="${boardname}_surface"/>
     <child link="${boardname}_part1"/>
-    <origin rpy="0.0 0.0 ${pi*0.5}" xyz="0.33 0.33 0.0"/>
+    <origin rpy="0.0 0.0 ${pi*0.5}" xyz="0.34 0.06 0.0"/>
   </joint>
   <link name="${boardname}_part1"/>
@@ -69,5 +69,5 @@
     <parent link="${boardname}_surface"/>
     <child link="${boardname}_part2"/>
-    <origin rpy="0.0 0.0 ${pi*0.5}" xyz="0.06 0.36 0.0"/>
+    <origin rpy="0.0 0.0 ${pi*0.5}" xyz="0.35 0.35 0.0"/>
   </joint>
   <link name="${boardname}_part2"/>
@@ -75,5 +75,5 @@
     <parent link="${boardname}_surface"/>
     <child link="${boardname}_part3"/>
-    <origin rpy="0.0 0.0 ${pi*0.5}" xyz="0.09 0.3 0.0"/>
+    <origin rpy="0.0 0.0 ${pi*0.5}" xyz="0.31 0.32 0.0"/>
   </joint>
   <link name="${boardname}_part3"/>
@@ -81,5 +81,5 @@
     <parent link="${boardname}_surface"/>
     <child link="${boardname}_part4"/>
-    <origin rpy="0.0 0.0 ${pi*0.5}" xyz="0.16 0.27 0.0"/>
+    <origin rpy="0.0 0.0 ${pi*0.5}" xyz="0.28 0.25 0.0"/>
   </joint>
   <link name="${boardname}_part4"/>
@@ -87,5 +87,5 @@
     <parent link="${boardname}_surface"/>
     <child link="${boardname}_part5"/>
-    <origin rpy="0.0 0.0 ${pi*0.5}" xyz="0.05 0.25 0.002"/>
+    <origin rpy="0.0 0.0 ${pi*0.5}" xyz="0.26 0.33 0.002"/>
   </joint>
   <link name="${boardname}_part5">
@@ -103,5 +103,5 @@
     <parent link="${boardname}_surface"/>
     <child link="${boardname}_part15"/>
-    <origin rpy="0.0 0.0 ${pi*0.5}" xyz="0.05 0.25 0.0772"/>
+    <origin rpy="0.0 0.0 ${pi*0.5}" xyz="0.26 0.33 0.0772"/>
   </joint>
   <link name="${boardname}_part15"/>
@@ -109,5 +109,5 @@
     <parent link="${boardname}_surface"/>
     <child link="${boardname}_part6_small_pulley"/>
-    <origin rpy="0.0 0.0 ${pi*0.5}" xyz="0.06 0.07 0.0085"/>
+    <origin rpy="0.0 0.0 ${pi*0.0}" xyz="0.06 0.34 0.0085"/>
   </joint>
   <link name="${boardname}_part6_small_pulley">
@@ -125,5 +125,5 @@
     <parent link="${boardname}_surface"/>
     <child link="${boardname}_part7_1"/>
-    <origin rpy="0.0 0.0 ${pi*0.0}" xyz="0.351 0.056 0.0505"/>
+    <origin rpy="0.0 0.0 ${pi*-0.5}" xyz="0.056 0.039 0.0505"/>
   </joint>
   <link name="${boardname}_part7_1"/>
@@ -131,5 +131,5 @@
     <parent link="${boardname}_surface"/>
     <child link="${boardname}_part8"/>
-    <origin rpy="0.0 0.0 ${pi*0.5}" xyz="0.32 0.24 0.012"/>
+    <origin rpy="0.0 0.0 ${pi*0.5}" xyz="0.25 0.08 0.012"/>
   </joint>
   <link name="${boardname}_part8">
@@ -147,5 +147,5 @@
     <parent link="${boardname}_surface"/>
     <child link="${boardname}_part9"/>
-    <origin rpy="0.0 0.0 ${pi*0.5}" xyz="0.28 0.13 0.009"/>
+    <origin rpy="0.0 0.0 ${pi*0.5}" xyz="0.15 0.14 0.009"/>
   </joint>
   <link name="${boardname}_part9">
@@ -163,5 +163,5 @@
     <parent link="${boardname}_surface"/>
     <child link="${boardname}_part10"/>
-    <origin rpy="0.0 0.0 ${pi*0.5}" xyz="0.19 0.34 0.0515"/>
+    <origin rpy="0.0 0.0 ${pi*0.5}" xyz="0.36 0.24 0.0515"/>
   </joint>
   <link name="${boardname}_part10">
@@ -179,5 +179,5 @@
     <parent link="${boardname}_surface"/>
     <child link="${boardname}_part11"/>
-    <origin rpy="0.0 0.0 ${pi*0.5}" xyz="0.07 0.17 0.0"/>
+    <origin rpy="0.0 0.0 ${pi*0.5}" xyz="0.18 0.34 0.0"/>
   </joint>
   <link name="${boardname}_part11"/>
@@ -185,5 +185,5 @@
     <parent link="${boardname}_surface"/>
     <child link="${boardname}_part12"/>
-    <origin rpy="0.0 0.0 ${pi*0.5}" xyz="0.15 0.15 0.0"/>
+    <origin rpy="0.0 ${pi/2} ${pi*0.5}" xyz="0.14 0.26 0.0"/>
   </joint>
   <link name="${boardname}_part12"/>
@@ -191,5 +191,5 @@
     <parent link="${boardname}_surface"/>
     <child link="${boardname}_part13"/>
-    <origin rpy="0.0 0.0 ${pi*0.5}" xyz="0.05 0.25 0.078"/>
+    <origin rpy="0.0 0.0 ${pi*0.5}" xyz="0.26 0.33 0.078"/>
   </joint>
   <link name="${boardname}_part13"/>
@@ -197,5 +197,5 @@
     <parent link="${boardname}_surface"/>
     <child link="${boardname}_part14"/>
-    <origin rpy="0.0 0.0 ${pi*0.5}" xyz="0.22 0.22 0.0515"/>
+    <origin rpy="0.0 ${pi/2} ${pi*0.5}" xyz="0.23 0.17 0.0515"/>
   </joint>
   <link name="${boardname}_part14">

Commit message: Fix taskboard frame rotations

File: o2as_scene_description/urdf/task_board.xacro (robot description, xacro)
@@ -191,5 +191,5 @@
     <parent link="${boardname}_surface"/>
     <child link="${boardname}_part13"/>
-    <origin rpy="0.0 0.0 ${pi*0.5}" xyz="0.26 0.33 0.078"/>
+    <origin rpy="0.0 ${pi/2} ${pi*0.5}" xyz="0.26 0.33 0.078"/>
   </joint>
   <link name="${boardname}_part13"/>
@@ -197,5 +197,5 @@
     <parent link="${boardname}_surface"/>
     <child link="${boardname}_part14"/>
-    <origin rpy="0.0 ${pi/2} ${pi*0.5}" xyz="0.23 0.17 0.0515"/>
+    <origin rpy="0.0 0.0 ${pi*0.5}" xyz="0.23 0.17 0.0515"/>
   </joint>
   <link name="${boardname}_part14">

Commit message: Change taskboard orientation, fix frames

File: o2as_scene_description/urdf/task_board.xacro (robot description, xacro)
@@ -63,5 +63,5 @@
     <parent link="${boardname}_surface"/>
     <child link="${boardname}_part1"/>
-    <origin rpy="0.0 0.0 ${pi*0.5}" xyz="0.33 0.33 0.0"/>
+    <origin rpy="0.0 0.0 ${pi*0.5}" xyz="0.06 0.34 0.0"/>
   </joint>
   <link name="${boardname}_part1"/>
@@ -69,5 +69,5 @@
     <parent link="${boardname}_surface"/>
     <child link="${boardname}_part2"/>
-    <origin rpy="0.0 0.0 ${pi*0.5}" xyz="0.06 0.36 0.0"/>
+    <origin rpy="0.0 0.0 ${pi*0.5}" xyz="0.05 0.05 0.0"/>
   </joint>
   <link name="${boardname}_part2"/>
@@ -75,5 +75,5 @@
     <parent link="${boardname}_surface"/>
     <child link="${boardname}_part3"/>
-    <origin rpy="0.0 0.0 ${pi*0.5}" xyz="0.09 0.3 0.0"/>
+    <origin rpy="0.0 0.0 ${pi*0.5}" xyz="0.09 0.08 0.0"/>
   </joint>
   <link name="${boardname}_part3"/>
@@ -81,5 +81,5 @@
     <parent link="${boardname}_surface"/>
     <child link="${boardname}_part4"/>
-    <origin rpy="0.0 0.0 ${pi*0.5}" xyz="0.16 0.27 0.0"/>
+    <origin rpy="0.0 0.0 ${pi*0.5}" xyz="0.12 0.15 0.0"/>
   </joint>
   <link name="${boardname}_part4"/>
@@ -87,5 +87,5 @@
     <parent link="${boardname}_surface"/>
     <child link="${boardname}_part5"/>
-    <origin rpy="0.0 0.0 ${pi*0.5}" xyz="0.05 0.25 0.002"/>
+    <origin rpy="0.0 0.0 ${pi*0.5}" xyz="0.14 0.07 0.002"/>
   </joint>
   <link name="${boardname}_part5">
@@ -103,5 +103,5 @@
     <parent link="${boardname}_surface"/>
     <child link="${boardname}_part15"/>
-    <origin rpy="0.0 0.0 ${pi*0.5}" xyz="0.05 0.25 0.0772"/>
+    <origin rpy="0.0 0.0 ${pi*0.5}" xyz="0.14 0.07 0.0772"/>
   </joint>
   <link name="${boardname}_part15"/>
@@ -109,5 +109,5 @@
     <parent link="${boardname}_surface"/>
     <child link="${boardname}_part6_small_pulley"/>
-    <origin rpy="0.0 0.0 ${pi*0.5}" xyz="0.06 0.07 0.0085"/>
+    <origin rpy="0.0 0.0 ${pi*1.0}" xyz="0.34 0.06 0.0085"/>
   </joint>
   <link name="${boardname}_part6_small_pulley">
@@ -125,5 +125,5 @@
     <parent link="${boardname}_surface"/>
     <child link="${boardname}_part7_1"/>
-    <origin rpy="0.0 0.0 ${pi*0.0}" xyz="0.351 0.056 0.0505"/>
+    <origin rpy="0.0 0.0 ${pi*0.5}" xyz="0.344 0.361 0.0505"/>
   </joint>
   <link name="${boardname}_part7_1"/>
@@ -131,5 +131,5 @@
     <parent link="${boardname}_surface"/>
     <child link="${boardname}_part8"/>
-    <origin rpy="0.0 0.0 ${pi*0.5}" xyz="0.32 0.24 0.012"/>
+    <origin rpy="0.0 0.0 ${pi*0.5}" xyz="0.15 0.32 0.012"/>
   </joint>
   <link name="${boardname}_part8">
@@ -147,5 +147,5 @@
     <parent link="${boardname}_surface"/>
     <child link="${boardname}_part9"/>
-    <origin rpy="0.0 0.0 ${pi*0.5}" xyz="0.28 0.13 0.009"/>
+    <origin rpy="0.0 0.0 ${pi*0.5}" xyz="0.25 0.26 0.009"/>
   </joint>
   <link name="${boardname}_part9">
@@ -163,5 +163,5 @@
     <parent link="${boardname}_surface"/>
     <child link="${boardname}_part10"/>
-    <origin rpy="0.0 0.0 ${pi*0.5}" xyz="0.19 0.34 0.0515"/>
+    <origin rpy="0.0 0.0 ${pi*0.5}" xyz="0.04 0.16 0.0515"/>
   </joint>
   <link name="${boardname}_part10">
@@ -179,5 +179,5 @@
     <parent link="${boardname}_surface"/>
     <child link="${boardname}_part11"/>
-    <origin rpy="0.0 0.0 ${pi*0.5}" xyz="0.07 0.17 0.0"/>
+    <origin rpy="0.0 0.0 ${pi*0.5}" xyz="0.22 0.06 0.0"/>
   </joint>
   <link name="${boardname}_part11"/>
@@ -185,5 +185,5 @@
     <parent link="${boardname}_surface"/>
     <child link="${boardname}_part12"/>
-    <origin rpy="0.0 0.0 ${pi*0.5}" xyz="0.15 0.15 0.0"/>
+    <origin rpy="${pi*-0.5} ${pi*0.5} ${pi*0.}" xyz="0.26 0.14 0.0"/>
   </joint>
   <link name="${boardname}_part12"/>
@@ -191,5 +191,5 @@
     <parent link="${boardname}_surface"/>
     <child link="${boardname}_part13"/>
-    <origin rpy="0.0 0.0 ${pi*0.5}" xyz="0.05 0.25 0.078"/>
+    <origin rpy="${pi*-0.5} ${pi*0.5} ${pi*0.}" xyz="0.14 0.07 0.078"/>
   </joint>
   <link name="${boardname}_part13"/>
@@ -197,5 +197,5 @@
     <parent link="${boardname}_surface"/>
     <child link="${boardname}_part14"/>
-    <origin rpy="0.0 0.0 ${pi*0.5}" xyz="0.22 0.22 0.0515"/>
+    <origin rpy="0.0 0.0 ${pi*0.5}" xyz="0.17 0.23 0.0515"/>
   </joint>
   <link name="${boardname}_part14">
