Commit message: Add taskboard belt task test

File: o2as_scene_description/urdf/taskboard_scene.xacro (robot description, xacro)
@@ -18,5 +18,5 @@
     <parent link="taskboard"/>
     <child link="belt_placement_tool"/>
-    <origin rpy="0.0 0.0 ${pi/2}" xyz="-0.07 0.0 0.0"/>
+    <origin rpy="0.0 0.0 0" xyz="-0.06 0.06 0"/>
   </joint>
   <link name="belt_placement_tool"/>

Commit message: add seq and calibrate the precision gripper

File: o2as_scene_description/urdf/taskboard_scene.xacro (robot description, xacro)
@@ -21,3 +21,15 @@
   </joint>
   <link name="belt_placement_tool"/>
+  <joint name="M10nut_tool" type="fixed">
+    <parent link="taskboard"/>
+    <child link="M10nut_tool"/>
+    <origin rpy="0.0 0.0 0" xyz="-0.06 0.46 0"/>
+  </joint>
+  <link name="M10nut_tool"/>
+  <joint name="Peg_tool" type="fixed">
+    <parent link="taskboard"/>
+    <child link="Peg_tool"/>
+    <origin rpy="0.0 0.0 0" xyz="-0.06 0.56 0"/>
+  </joint>
+  <link name="Peg_tool"/>
 </robot>

Commit message: WIP: Add taskboard part 6 (peg)
The tool broke while testing this. The last step (screwing the peg in) is not tested.

File: o2as_scene_description/urdf/taskboard_scene.xacro (robot description, xacro)
@@ -27,9 +27,9 @@
   </joint>
   <link name="M10nut_tool"/>
-  <joint name="Peg_tool" type="fixed">
+  <joint name="peg_tool" type="fixed">
     <parent link="taskboard"/>
-    <child link="Peg_tool"/>
+    <child link="peg_tool"/>
     <origin rpy="0.0 0.0 0" xyz="-0.06 0.56 0"/>
   </joint>
-  <link name="Peg_tool"/>
+  <link name="peg_tool"/>
 </robot>

Commit message: Add new tools, taskboard calibration

File: o2as_scene_description/urdf/taskboard_scene.xacro (robot description, xacro)
@@ -16,9 +16,15 @@
   </xacro:o2as_mat>
   <joint name="belt_placement_tool" type="fixed">
-    <parent link="taskboard"/>
+    <parent link="workspace_center"/>
     <child link="belt_placement_tool"/>
-    <origin rpy="0.0 0.0 0" xyz="-0.06 0.06 0"/>
+    <origin rpy="0.0 0.0 0" xyz="-.15 0.3 0"/>
   </joint>
   <link name="belt_placement_tool"/>
+  <joint name="retainer_pin_insertion_tool" type="fixed">
+    <parent link="workspace_center"/>
+    <child link="retainer_pin_insertion_tool"/>
+    <origin rpy="0.0 0.0 0" xyz="-0.1 0.3 0"/>
+  </joint>
+  <link name="retainer_pin_insertion_tool"/>
   <joint name="M10nut_tool" type="fixed">
     <parent link="taskboard"/>

Commit message: Move placement mat forward to avoid collisions

File: o2as_scene_description/urdf/taskboard_scene.xacro (robot description, xacro)
@@ -13,5 +13,5 @@
   <xacro:property name="p_l" value="0.4"/>
   <xacro:o2as_mat matname="mat" mat_w="${p_w}" mat_l="${p_l}" mat_h=".0001" parent="taskboard">
-    <origin xyz="0.0 0.41 0.0" rpy="0 0 0" />
+    <origin xyz="0.0 0.45 0.0" rpy="0 0 0" />
   </xacro:o2as_mat>
   <joint name="belt_placement_tool" type="fixed">

Commit message: WIP: Part 7, but with moved taskboard

File: o2as_scene_description/urdf/taskboard_scene.xacro (robot description, xacro)
@@ -5,5 +5,5 @@
   <xacro:include filename="$(find o2as_scene_description)/urdf/task_board.xacro" />
   <xacro:task_board boardname="taskboard" parent="workspace_center">
-    <origin xyz="-0.35 0.2 0.0" rpy="0 0 ${-pi/2}" />
+    <origin xyz="-0.3 0.26 0.0" rpy="0 0 ${-pi/2}" />
     <!-- <origin xyz="-0.35 0.1 0.0" rpy="0 0 ${-pi/2}" />  -->
   </xacro:task_board>
@@ -12,6 +12,6 @@
   <xacro:property name="p_w" value="0.4"/>
   <xacro:property name="p_l" value="0.4"/>
-  <xacro:o2as_mat matname="mat" mat_w="${p_w}" mat_l="${p_l}" mat_h=".0001" parent="taskboard">
-    <origin xyz="0.0 0.45 0.0" rpy="0 0 0" />
+  <xacro:o2as_mat matname="mat" mat_w="${p_w}" mat_l="${p_l}" mat_h=".0001" parent="workspace_center">
+    <origin xyz="0.14 0.2 0.0" rpy="0 0 ${-pi/2}" />
   </xacro:o2as_mat>
   <joint name="belt_placement_tool" type="fixed">
