Commit message: Add end tip frame for m6 nut tool for c_bot

File: o2as_scene_description/urdf/robotiq_c_bot_gripper.urdf.xacro (robot description, xacro)
@@ -32,4 +32,10 @@
     </joint>
     <link name="${prefix}screw_tool_m3_tip_link"/>
+    <joint name="${prefix}robotiq_85_nut_tool_m6_tip_joint" type="fixed">
+      <parent link="${prefix}robotiq_85_tip_rotation_helper_link"/>
+      <child link="${prefix}nut_tool_m6_tip_link"/>
+      <origin rpy="0 0 0" xyz="0.052 0.0 .006 "/>
+    </joint>
+    <link name="${prefix}nut_tool_m6_tip_link"/>
   </xacro:macro>
 </robot>

Commit message: Enable nut tool m6 for c_bot

File: o2as_scene_description/urdf/robotiq_c_bot_gripper.urdf.xacro (robot description, xacro)
@@ -6,14 +6,21 @@
     <xacro:include filename="$(find o2as_scene_description)/urdf/robotiq_85_gripper_with_ft300.urdf.xacro" />
     <xacro:robotiq_85_gripper_with_ft300 prefix="${prefix}" parent="${parent}"/>
-    <!-- This helper frame is oriented like the screw tool tip frame -->
-    <joint name="${prefix}robotiq_85_tip_rotation_helper_joint" type="fixed">
+    <!-- This helper frame is oriented like the screw tool tip frames -->
+    <joint name="${prefix}robotiq_85_tip_45deg_helper_joint" type="fixed">
       <parent link="${prefix}robotiq_85_tip_link"/>
-      <child link="${prefix}robotiq_85_tip_rotation_helper_link"/>
+      <child link="${prefix}robotiq_85_tip_45deg_helper_link"/>
       <origin rpy="0.0 ${-pi/4} 0.0" xyz="-.03 0 0"/>
     </joint>
-    <link name="${prefix}robotiq_85_tip_rotation_helper_link"/>
+    <link name="${prefix}robotiq_85_tip_45deg_helper_link"/>
+    <!-- This helper frame is oriented like the nut tool tip frame -->
+    <joint name="${prefix}robotiq_85_tip_30deg_helper_joint" type="fixed">
+      <parent link="${prefix}robotiq_85_tip_link"/>
+      <child link="${prefix}robotiq_85_tip_30deg_helper_link"/>
+      <origin rpy="0.0 ${-pi/6} 0.0" xyz="-.03 0 0"/>
+    </joint>
+    <link name="${prefix}robotiq_85_tip_30deg_helper_link"/>
     <!-- Screw tool tips. X-axis points along the screw into the hole. -->
     <joint name="${prefix}robotiq_85_m6_screw_tool_tip_joint" type="fixed">
-      <parent link="${prefix}robotiq_85_tip_rotation_helper_link"/>
+      <parent link="${prefix}robotiq_85_tip_45deg_helper_link"/>
       <child link="${prefix}screw_tool_m6_tip_link"/>
       <origin rpy="0.0 0 0" xyz="0.12 0 .006"/>
@@ -21,5 +28,5 @@
     <link name="${prefix}screw_tool_m6_tip_link"/>
     <joint name="${prefix}robotiq_85_m4_screw_tool_tip_joint" type="fixed">
-      <parent link="${prefix}robotiq_85_tip_rotation_helper_link"/>
+      <parent link="${prefix}robotiq_85_tip_45deg_helper_link"/>
       <child link="${prefix}screw_tool_m4_tip_link"/>
       <origin rpy="0.0 0 0" xyz="0.151 0 .006"/>
@@ -27,5 +34,5 @@
     <link name="${prefix}screw_tool_m4_tip_link"/>
     <joint name="${prefix}robotiq_85_m3_screw_tool_tip_joint" type="fixed">
-      <parent link="${prefix}robotiq_85_tip_rotation_helper_link"/>
+      <parent link="${prefix}robotiq_85_tip_45deg_helper_link"/>
       <child link="${prefix}screw_tool_m3_tip_link"/>
       <origin rpy="0.0 0 0" xyz="0.132 0 .006"/>
@@ -33,7 +40,7 @@
     <link name="${prefix}screw_tool_m3_tip_link"/>
     <joint name="${prefix}robotiq_85_nut_tool_m6_tip_joint" type="fixed">
-      <parent link="${prefix}robotiq_85_tip_rotation_helper_link"/>
+      <parent link="${prefix}robotiq_85_tip_30deg_helper_link"/>
       <child link="${prefix}nut_tool_m6_tip_link"/>
-      <origin rpy="0 0 0" xyz="0.052 0.0 .006 "/>
+      <origin rpy="0 0 0" xyz="0.057 0.0 -.014 "/>
     </joint>
     <link name="${prefix}nut_tool_m6_tip_link"/>

File: o2as_scene_description/urdf/screw_tools.xacro (robot description, xacro)
@@ -99,5 +99,5 @@
     <parent link="screw_tool_holder" />
     <child link="nut_tool_m6_link" />
-    <origin xyz="-0.05 ${tool_offset} 0.004" rpy="0.0 0.0 0.0" />
+    <origin xyz="-0.35 ${tool_offset} 0.004" rpy="0.0 0.0 0.0" />
   </joint>
   <link name="suction_tool_link">

Commit message: Increase c_bot nut tool grasp angle

File: o2as_scene_description/urdf/robotiq_c_bot_gripper.urdf.xacro (robot description, xacro)
@@ -14,10 +14,10 @@
     <link name="${prefix}robotiq_85_tip_45deg_helper_link"/>
     <!-- This helper frame is oriented like the nut tool tip frame -->
-    <joint name="${prefix}robotiq_85_tip_30deg_helper_joint" type="fixed">
+    <joint name="${prefix}robotiq_85_tip_40deg_helper_joint" type="fixed">
       <parent link="${prefix}robotiq_85_tip_link"/>
-      <child link="${prefix}robotiq_85_tip_30deg_helper_link"/>
-      <origin rpy="0.0 ${-pi/6} 0.0" xyz="-.03 0 0"/>
+      <child link="${prefix}robotiq_85_tip_40deg_helper_link"/>
+      <origin rpy="0.0 ${-pi*40/180} 0.0" xyz="-.03 0 0"/>
     </joint>
-    <link name="${prefix}robotiq_85_tip_30deg_helper_link"/>
+    <link name="${prefix}robotiq_85_tip_40deg_helper_link"/>
     <!-- Screw tool tips. X-axis points along the screw into the hole. -->
     <joint name="${prefix}robotiq_85_m6_screw_tool_tip_joint" type="fixed">
@@ -40,5 +40,5 @@
     <link name="${prefix}screw_tool_m3_tip_link"/>
     <joint name="${prefix}robotiq_85_nut_tool_m6_tip_joint" type="fixed">
-      <parent link="${prefix}robotiq_85_tip_30deg_helper_link"/>
+      <parent link="${prefix}robotiq_85_tip_40deg_helper_link"/>
       <child link="${prefix}nut_tool_m6_tip_link"/>
       <origin rpy="0 0 0" xyz="0.057 0.0 -.014 "/>
