Commit message: Add placement_mat urdf generator. Clean-up

File: o2as_scene_description/urdf/o2as_mat.xacro (robot description, xacro)
@@ -36,4 +36,94 @@
       <xacro:insert_block name="origin"/>
     </joint>
+    <joint name="${matname}_part1" type="fixed">
+      <parent link="${matname}"/>
+      <child link="${matname}_part1"/>
+      <origin rpy="0.0 0.0 ${pi/2}" xyz="0.0025 0.003 0.01"/>
+    </joint>
+    <link name="${matname}_part1"/>
+    <joint name="${matname}_part2" type="fixed">
+      <parent link="${matname}"/>
+      <child link="${matname}_part2"/>
+      <origin rpy="0.0 0.0 ${pi/2}" xyz="0.003 0.004 0.01"/>
+    </joint>
+    <link name="${matname}_part2"/>
+    <joint name="${matname}_part3" type="fixed">
+      <parent link="${matname}"/>
+      <child link="${matname}_part3"/>
+      <origin rpy="0.0 0.0 ${pi/2}" xyz="0.005 0.005 0.01"/>
+    </joint>
+    <link name="${matname}_part3"/>
+    <joint name="${matname}_part4" type="fixed">
+      <parent link="${matname}"/>
+      <child link="${matname}_part4"/>
+      <origin rpy="0.0 0.0 ${pi/2}" xyz="0.0072 0.006 0.01"/>
+    </joint>
+    <link name="${matname}_part4"/>
+    <joint name="${matname}_part5" type="fixed">
+      <parent link="${matname}"/>
+      <child link="${matname}_part5"/>
+      <origin rpy="0.0 0.0 ${pi/2}" xyz="0.003 0.006 0.01"/>
+    </joint>
+    <link name="${matname}_part5"/>
+    <joint name="${matname}_part6" type="fixed">
+      <parent link="${matname}"/>
+      <child link="${matname}_part6"/>
+      <origin rpy="0.0 0.0 ${pi/2}" xyz="0.00822 0.007 0.01"/>
+    </joint>
+    <link name="${matname}_part6"/>
+    <joint name="${matname}_part7" type="fixed">
+      <parent link="${matname}"/>
+      <child link="${matname}_part7"/>
+      <origin rpy="0.0 0.0 ${pi/2}" xyz="0.073 0.008 0.01"/>
+    </joint>
+    <link name="${matname}_part7"/>
+    <joint name="${matname}_part8" type="fixed">
+      <parent link="${matname}"/>
+      <child link="${matname}_part8"/>
+      <origin rpy="0.0 0.0 ${pi/2}" xyz="0.006 0.008 0.01"/>
+    </joint>
+    <link name="${matname}_part8"/>
+    <joint name="${matname}_part9" type="fixed">
+      <parent link="${matname}"/>
+      <child link="${matname}_part9"/>
+      <origin rpy="0.0 0.0 ${pi/2}" xyz="0.054 0.004 0.01"/>
+    </joint>
+    <link name="${matname}_part9"/>
+    <joint name="${matname}_part10" type="fixed">
+      <parent link="${matname}"/>
+      <child link="${matname}_part10"/>
+      <origin rpy="0.0 0.0 ${pi/2}" xyz="0.034 0.034 0.01"/>
+    </joint>
+    <link name="${matname}_part10"/>
+    <joint name="${matname}_part11" type="fixed">
+      <parent link="${matname}"/>
+      <child link="${matname}_part11"/>
+      <origin rpy="0.0 0.0 ${pi/2}" xyz="0.436 0.043 0.01"/>
+    </joint>
+    <link name="${matname}_part11"/>
+    <joint name="${matname}_part12" type="fixed">
+      <parent link="${matname}"/>
+      <child link="${matname}_part12"/>
+      <origin rpy="0.0 0.0 ${pi/2}" xyz="2.624 0.254 0.01"/>
+    </joint>
+    <link name="${matname}_part12"/>
+    <joint name="${matname}_part13" type="fixed">
+      <parent link="${matname}"/>
+      <child link="${matname}_part13"/>
+      <origin rpy="0.0 0.0 ${pi/2}" xyz="0.024 0.046 0.01"/>
+    </joint>
+    <link name="${matname}_part13"/>
+    <joint name="${matname}_part14" type="fixed">
+      <parent link="${matname}"/>
+      <child link="${matname}_part14"/>
+      <origin rpy="0.0 0.0 ${pi/2}" xyz="0.234 0.345 0.01"/>
+    </joint>
+    <link name="${matname}_part14"/>
+    <joint name="${matname}_part15" type="fixed">
+      <parent link="${matname}"/>
+      <child link="${matname}_part15"/>
+      <origin rpy="0.0 0.0 ${pi/2}" xyz="0.046 7.687 0.01"/>
+    </joint>
+    <link name="${matname}_part15"/>
   </xacro:macro>
 </robot>

File: o2as_scene_description/urdf/task_board.xacro (robot description, xacro)
@@ -35,5 +35,5 @@
     <parent link="${boardname}"/>
     <child link="${boardname}_part1"/>
-    <origin rpy="0.0 0.0 0.0" xyz="0.34 0.34 0.01"/>
+    <origin rpy="0.0 0.0 ${pi/2}" xyz="0.34 0.34 0.01"/>
   </joint>
   <link name="${boardname}_part1"/>
@@ -41,5 +41,5 @@
     <parent link="${boardname}"/>
     <child link="${boardname}_part2"/>
-    <origin rpy="0.0 0.0 0.0" xyz="0.05 0.35 0.01"/>
+    <origin rpy="0.0 0.0 ${pi/2}" xyz="0.05 0.35 0.01"/>
   </joint>
   <link name="${boardname}_part2"/>
@@ -47,5 +47,5 @@
     <parent link="${boardname}"/>
     <child link="${boardname}_part3"/>
-    <origin rpy="0.0 0.0 0.0" xyz="0.08 0.31 0.01"/>
+    <origin rpy="0.0 0.0 ${pi/2}" xyz="0.08 0.31 0.01"/>
   </joint>
   <link name="${boardname}_part3"/>
@@ -53,5 +53,5 @@
     <parent link="${boardname}"/>
     <child link="${boardname}_part4"/>
-    <origin rpy="0.0 0.0 0.0" xyz="0.15 0.28 0.01"/>
+    <origin rpy="0.0 0.0 ${pi/2}" xyz="0.15 0.28 0.01"/>
   </joint>
   <link name="${boardname}_part4"/>
@@ -59,5 +59,5 @@
     <parent link="${boardname}"/>
     <child link="${boardname}_part5"/>
-    <origin rpy="0.0 0.0 0.0" xyz="0.07 0.26 0.01"/>
+    <origin rpy="0.0 0.0 ${pi/2}" xyz="0.07 0.26 0.01"/>
   </joint>
   <link name="${boardname}_part5"/>
@@ -65,5 +65,5 @@
     <parent link="${boardname}"/>
     <child link="${boardname}_part6"/>
-    <origin rpy="0.0 0.0 0.0" xyz="0.2 0.2 0.01"/>
+    <origin rpy="0.0 0.0 ${pi/2}" xyz="0.2 0.2 0.01"/>
   </joint>
   <link name="${boardname}_part6"/>
@@ -71,5 +71,5 @@
     <parent link="${boardname}"/>
     <child link="${boardname}_part8"/>
-    <origin rpy="0.0 0.0 0.0" xyz="0.32 0.25 0.01"/>
+    <origin rpy="0.0 0.0 ${pi/2}" xyz="0.32 0.25 0.01"/>
   </joint>
   <link name="${boardname}_part8"/>
@@ -77,5 +77,5 @@
     <parent link="${boardname}"/>
     <child link="${boardname}_part9"/>
-    <origin rpy="0.0 0.0 0.0" xyz="0.26 0.15 0.01"/>
+    <origin rpy="0.0 0.0 ${pi/2}" xyz="0.26 0.15 0.01"/>
   </joint>
   <link name="${boardname}_part9"/>
@@ -83,5 +83,5 @@
     <parent link="${boardname}"/>
     <child link="${boardname}_part10"/>
-    <origin rpy="0.0 0.0 0.0" xyz="0.16 0.36 0.01"/>
+    <origin rpy="0.0 0.0 ${pi/2}" xyz="0.16 0.36 0.01"/>
   </joint>
   <link name="${boardname}_part10"/>
@@ -89,5 +89,5 @@
     <parent link="${boardname}"/>
     <child link="${boardname}_part11"/>
-    <origin rpy="0.0 0.0 0.0" xyz="0.06 0.18 0.01"/>
+    <origin rpy="0.0 0.0 ${pi/2}" xyz="0.06 0.18 0.01"/>
   </joint>
   <link name="${boardname}_part11"/>
@@ -95,5 +95,5 @@
     <parent link="${boardname}"/>
     <child link="${boardname}_part12"/>
-    <origin rpy="0.0 0.0 0.0" xyz="0.14 0.14 0.01"/>
+    <origin rpy="0.0 0.0 ${pi/2}" xyz="0.14 0.14 0.01"/>
   </joint>
   <link name="${boardname}_part12"/>
@@ -101,5 +101,5 @@
     <parent link="${boardname}"/>
     <child link="${boardname}_part13"/>
-    <origin rpy="0.0 0.0 0.0" xyz="0.35 0.12 0.01"/>
+    <origin rpy="0.0 0.0 ${pi/2}" xyz="0.35 0.12 0.01"/>
   </joint>
   <link name="${boardname}_part13"/>
@@ -107,5 +107,5 @@
     <parent link="${boardname}"/>
     <child link="${boardname}_part14"/>
-    <origin rpy="0.0 0.0 0.0" xyz="0.23 0.23 0.01"/>
+    <origin rpy="0.0 0.0 ${pi/2}" xyz="0.23 0.23 0.01"/>
   </joint>
   <link name="${boardname}_part14"/>
@@ -113,5 +113,5 @@
     <parent link="${boardname}"/>
     <child link="${boardname}_part15"/>
-    <origin rpy="0.0 0.0 0.0" xyz="0.16 0.36 0.06"/>
+    <origin rpy="0.0 0.0 ${pi/2}" xyz="0.16 0.36 0.06"/>
   </joint>
   <link name="${boardname}_part15"/>

Commit message: Clean-up

File: o2as_scene_description/urdf/o2as_mat.xacro (robot description, xacro)
@@ -39,5 +39,5 @@
       <parent link="${matname}"/>
       <child link="${matname}_part1"/>
-      <origin rpy="0.0 0.0 ${pi/2}" xyz="0.0025 0.003 0.01"/>
+      <origin rpy="0.0 0.0 ${pi/2}" xyz="0.05 0.01 0.01"/>
     </joint>
     <link name="${matname}_part1"/>
@@ -45,5 +45,5 @@
       <parent link="${matname}"/>
       <child link="${matname}_part2"/>
-      <origin rpy="0.0 0.0 ${pi/2}" xyz="0.003 0.004 0.01"/>
+      <origin rpy="0.0 0.0 ${pi/2}" xyz="0.3 0.023 0.01"/>
     </joint>
     <link name="${matname}_part2"/>
@@ -51,5 +51,5 @@
       <parent link="${matname}"/>
       <child link="${matname}_part3"/>
-      <origin rpy="0.0 0.0 ${pi/2}" xyz="0.005 0.005 0.01"/>
+      <origin rpy="0.0 0.0 ${pi/2}" xyz="0.29 0.355 0.01"/>
     </joint>
     <link name="${matname}_part3"/>
@@ -57,5 +57,5 @@
       <parent link="${matname}"/>
       <child link="${matname}_part4"/>
-      <origin rpy="0.0 0.0 ${pi/2}" xyz="0.0072 0.006 0.01"/>
+      <origin rpy="0.0 0.0 ${pi/2}" xyz="0.279 0.066 0.01"/>
     </joint>
     <link name="${matname}_part4"/>
@@ -63,5 +63,5 @@
       <parent link="${matname}"/>
       <child link="${matname}_part5"/>
-      <origin rpy="0.0 0.0 ${pi/2}" xyz="0.003 0.006 0.01"/>
+      <origin rpy="0.0 0.0 ${pi/2}" xyz="0.024 0.255 0.01"/>
     </joint>
     <link name="${matname}_part5"/>
@@ -69,5 +69,5 @@
       <parent link="${matname}"/>
       <child link="${matname}_part6"/>
-      <origin rpy="0.0 0.0 ${pi/2}" xyz="0.00822 0.007 0.01"/>
+      <origin rpy="0.0 0.0 ${pi/2}" xyz="0.345 0.115 0.01"/>
     </joint>
     <link name="${matname}_part6"/>
@@ -75,5 +75,5 @@
       <parent link="${matname}"/>
       <child link="${matname}_part7"/>
-      <origin rpy="0.0 0.0 ${pi/2}" xyz="0.073 0.008 0.01"/>
+      <origin rpy="0.0 0.0 ${pi/2}" xyz="0.065 0.223 0.01"/>
     </joint>
     <link name="${matname}_part7"/>
@@ -81,5 +81,5 @@
       <parent link="${matname}"/>
       <child link="${matname}_part8"/>
-      <origin rpy="0.0 0.0 ${pi/2}" xyz="0.006 0.008 0.01"/>
+      <origin rpy="0.0 0.0 ${pi/2}" xyz="0.354 0.052 0.01"/>
     </joint>
     <link name="${matname}_part8"/>
@@ -87,5 +87,5 @@
       <parent link="${matname}"/>
       <child link="${matname}_part9"/>
-      <origin rpy="0.0 0.0 ${pi/2}" xyz="0.054 0.004 0.01"/>
+      <origin rpy="0.0 0.0 ${pi/2}" xyz="0.043 0.045 0.01"/>
     </joint>
     <link name="${matname}_part9"/>
@@ -93,5 +93,5 @@
       <parent link="${matname}"/>
       <child link="${matname}_part10"/>
-      <origin rpy="0.0 0.0 ${pi/2}" xyz="0.034 0.034 0.01"/>
+      <origin rpy="0.0 0.0 ${pi/2}" xyz="0.055 0.245 0.01"/>
     </joint>
     <link name="${matname}_part10"/>
@@ -99,5 +99,5 @@
       <parent link="${matname}"/>
       <child link="${matname}_part11"/>
-      <origin rpy="0.0 0.0 ${pi/2}" xyz="0.436 0.043 0.01"/>
+      <origin rpy="0.0 0.0 ${pi/2}" xyz="0.259 0.011 0.01"/>
     </joint>
     <link name="${matname}_part11"/>
@@ -105,5 +105,5 @@
       <parent link="${matname}"/>
       <child link="${matname}_part12"/>
-      <origin rpy="0.0 0.0 ${pi/2}" xyz="2.624 0.254 0.01"/>
+      <origin rpy="0.0 0.0 ${pi/2}" xyz="0.05 0.234 0.01"/>
     </joint>
     <link name="${matname}_part12"/>
@@ -111,5 +111,5 @@
       <parent link="${matname}"/>
       <child link="${matname}_part13"/>
-      <origin rpy="0.0 0.0 ${pi/2}" xyz="0.024 0.046 0.01"/>
+      <origin rpy="0.0 0.0 ${pi/2}" xyz="0.024 0.345 0.01"/>
     </joint>
     <link name="${matname}_part13"/>
@@ -123,5 +123,5 @@
       <parent link="${matname}"/>
       <child link="${matname}_part15"/>
-      <origin rpy="0.0 0.0 ${pi/2}" xyz="0.046 7.687 0.01"/>
+      <origin rpy="0.0 0.0 ${pi/2}" xyz="0.046 0.151 0.01"/>
     </joint>
     <link name="${matname}_part15"/>

Commit message: Set up full robot system, clean up

File: o2as_scene_description/urdf/o2as_mat.xacro (robot description, xacro)
@@ -57,5 +57,5 @@
       <parent link="${matname}"/>
       <child link="${matname}_part4"/>
-      <origin rpy="0.0 0.0 ${pi/2}" xyz="0.279 0.066 0.01"/>
+      <origin rpy="0.0 0.0 ${pi/2}" xyz="0.328 0.163 0.01"/>
     </joint>
     <link name="${matname}_part4"/>

File: o2as_scene_description/urdf/precision_gripper.xacro (robot description, xacro)
@@ -9,5 +9,5 @@
     </inertial>
     <visual>
-      <origin rpy="0 0 ${-pi/2}" xyz="0.02 0 0"/>
+      <origin rpy="0 ${pi/2} ${-pi/2}" xyz="0.02 0 0"/>
       <geometry>
         <mesh filename="${mesh_file}" scale="1 1 1"/>
@@ -18,5 +18,5 @@
     </visual>
     <collision>
-      <origin rpy="0 0 0" xyz="-0.11 0 0"/>
+      <origin rpy="0 ${pi/2} 0" xyz="-0.11 0 0"/>
       <geometry>
         <box size="0.22 0.15 0.1"/>

File: o2as_scene_description/urdf/task_board.xacro (robot description, xacro)
@@ -116,4 +116,28 @@
   </joint>
   <link name="${boardname}_part15"/>
+  <joint name="${boardname}_corner1" type="fixed">
+    <parent link="${boardname}"/>
+    <child link="${boardname}_corner1"/>
+    <origin rpy="0.0 0.0 ${pi/2}" xyz="0.01 0.39 0.06"/>
+  </joint>
+  <link name="${boardname}_corner1"/>
+  <joint name="${boardname}_corner2" type="fixed">
+    <parent link="${boardname}"/>
+    <child link="${boardname}_corner2"/>
+    <origin rpy="0.0 0.0 ${pi/2}" xyz="0.39 0.39 0.06"/>
+  </joint>
+  <link name="${boardname}_corner2"/>
+  <joint name="${boardname}_corner3" type="fixed">
+    <parent link="${boardname}"/>
+    <child link="${boardname}_corner3"/>
+    <origin rpy="0.0 0.0 ${pi/2}" xyz="0.39 0.01 0.06"/>
+  </joint>
+  <link name="${boardname}_corner3"/>
+  <joint name="${boardname}_corner4" type="fixed">
+    <parent link="${boardname}"/>
+    <child link="${boardname}_corner4"/>
+    <origin rpy="0.0 0.0 ${pi/2}" xyz="0.01 0.01 0.06"/>
+  </joint>
+  <link name="${boardname}_corner4"/>
   </xacro:macro>
   <!-- Add additional links for us to plan with.-->

Commit message: Add taskboard task sequence draft

File: o2as_scene_description/urdf/o2as_mat.xacro (robot description, xacro)
@@ -51,5 +51,5 @@
       <parent link="${matname}"/>
       <child link="${matname}_part3"/>
-      <origin rpy="0.0 0.0 ${pi/2}" xyz="0.29 0.355 0.01"/>
+      <origin rpy="0.0 0.0 ${pi/2}" xyz="0.257 0.107 0.01"/>
     </joint>
     <link name="${matname}_part3"/>

Commit message: Change taskboard mat to black border

File: o2as_scene_description/urdf/o2as_mat.xacro (robot description, xacro)
@@ -126,4 +126,28 @@
     </joint>
     <link name="${matname}_part15"/>
+    <joint name="${matname}_corner1" type="fixed">
+      <parent link="${matname}"/>
+      <child link="${matname}_corner1"/>
+      <origin rpy="0.0 0.0 ${pi/2}" xyz="0.00 0.00 0.06"/>
+    </joint>
+    <link name="${matname}_corner1"/>
+    <joint name="${matname}_corner2" type="fixed">
+      <parent link="${matname}"/>
+      <child link="${matname}_corner2"/>
+      <origin rpy="0.0 0.0 ${pi/2}" xyz="0.38 0.00 0.06"/>
+    </joint>
+    <link name="${matname}_corner2"/>
+    <joint name="${matname}_corner3" type="fixed">
+      <parent link="${matname}"/>
+      <child link="${matname}_corner3"/>
+      <origin rpy="0.0 0.0 ${pi/2}" xyz="0.38 0.38 0.06"/>
+    </joint>
+    <link name="${matname}_corner3"/>
+    <joint name="${matname}_corner4" type="fixed">
+      <parent link="${matname}"/>
+      <child link="${matname}_corner4"/>
+      <origin rpy="0.0 0.0 ${pi/2}" xyz="0.00 0.38 0.06"/>
+    </joint>
+    <link name="${matname}_corner4"/>
   </xacro:macro>
 </robot>

File: o2as_scene_description/urdf/taskboard_scene.xacro (robot description, xacro)
@@ -9,8 +9,8 @@
   <!-- Placement mat -->
   <xacro:include filename="$(find o2as_scene_description)/urdf/o2as_mat.xacro" />
-  <xacro:property name="p_w" value="0.4"/>   <!--0.84 -->
-  <xacro:property name="p_l" value="0.4"/>   <!--0.62 -->
+  <xacro:property name="p_w" value="0.38"/>   <!--0.84 -->
+  <xacro:property name="p_l" value="0.38"/>   <!--0.62 -->
   <xacro:o2as_mat matname="mat" mat_w="${p_w}" mat_l="${p_l}" mat_h=".001" parent="taskboard">
-    <origin xyz="0 0.41 -0.029" rpy="0 0 0" />
+    <origin xyz="0.01 0.42 -0.029" rpy="0 0 0" />
   </xacro:o2as_mat>
 </robot>

Commit message: Sorry, the black line was not a good choice.

File: o2as_scene_description/urdf/o2as_mat.xacro (robot description, xacro)
@@ -129,5 +129,5 @@
       <parent link="${matname}"/>
       <child link="${matname}_corner1"/>
-      <origin rpy="0.0 0.0 ${pi/2}" xyz="0.00 0.00 0.06"/>
+      <origin rpy="0.0 0.0 ${pi/2}" xyz="0.01 0.01 0.06"/>
     </joint>
     <link name="${matname}_corner1"/>
@@ -135,5 +135,5 @@
       <parent link="${matname}"/>
       <child link="${matname}_corner2"/>
-      <origin rpy="0.0 0.0 ${pi/2}" xyz="0.38 0.00 0.06"/>
+      <origin rpy="0.0 0.0 ${pi/2}" xyz="0.39 0.01 0.06"/>
     </joint>
     <link name="${matname}_corner2"/>
@@ -141,5 +141,5 @@
       <parent link="${matname}"/>
       <child link="${matname}_corner3"/>
-      <origin rpy="0.0 0.0 ${pi/2}" xyz="0.38 0.38 0.06"/>
+      <origin rpy="0.0 0.0 ${pi/2}" xyz="0.39 0.39 0.06"/>
     </joint>
     <link name="${matname}_corner3"/>
@@ -147,5 +147,5 @@
       <parent link="${matname}"/>
       <child link="${matname}_corner4"/>
-      <origin rpy="0.0 0.0 ${pi/2}" xyz="0.00 0.38 0.06"/>
+      <origin rpy="0.0 0.0 ${pi/2}" xyz="0.01 0.39 0.06"/>
     </joint>
     <link name="${matname}_corner4"/>

File: o2as_scene_description/urdf/taskboard_scene.xacro (robot description, xacro)
@@ -9,8 +9,8 @@
   <!-- Placement mat -->
   <xacro:include filename="$(find o2as_scene_description)/urdf/o2as_mat.xacro" />
-  <xacro:property name="p_w" value="0.38"/>   <!--0.84 -->
-  <xacro:property name="p_l" value="0.38"/>   <!--0.62 -->
+  <xacro:property name="p_w" value="0.4"/>
+  <xacro:property name="p_l" value="0.4"/>
   <xacro:o2as_mat matname="mat" mat_w="${p_w}" mat_l="${p_l}" mat_h=".001" parent="taskboard">
-    <origin xyz="0.01 0.42 -0.029" rpy="0 0 0" />
+    <origin xyz="0.0 0.41 -0.029" rpy="0 0 0" />
   </xacro:o2as_mat>
 </robot>

Commit message: Measured placement mat for test run

File: o2as_scene_description/urdf/o2as_mat.xacro (robot description, xacro)
@@ -39,5 +39,5 @@
       <parent link="${matname}"/>
       <child link="${matname}_part1"/>
-      <origin rpy="0.0 0.0 ${pi/2}" xyz="0.05 0.01 0.01"/>
+      <origin rpy="0.0 0.0 ${pi/2}" xyz="0.073 0.285 0.01"/>
     </joint>
     <link name="${matname}_part1"/>
@@ -45,5 +45,5 @@
       <parent link="${matname}"/>
       <child link="${matname}_part2"/>
-      <origin rpy="0.0 0.0 ${pi/2}" xyz="0.3 0.023 0.01"/>
+      <origin rpy="0.0 0.0 ${pi/2}" xyz="0.0525 0.207 0.01"/>
     </joint>
     <link name="${matname}_part2"/>
@@ -51,5 +51,5 @@
       <parent link="${matname}"/>
       <child link="${matname}_part3"/>
-      <origin rpy="0.0 0.0 ${pi/2}" xyz="0.257 0.107 0.01"/>
+      <origin rpy="0.0 0.0 ${pi/2}" xyz="0.261 0.323 0.01"/>
     </joint>
     <link name="${matname}_part3"/>
@@ -57,5 +57,5 @@
       <parent link="${matname}"/>
       <child link="${matname}_part4"/>
-      <origin rpy="0.0 0.0 ${pi/2}" xyz="0.328 0.163 0.01"/>
+      <origin rpy="0.0 0.0 ${pi/2}" xyz="0.343 0.3235 0.01"/>
     </joint>
     <link name="${matname}_part4"/>
@@ -63,5 +63,5 @@
       <parent link="${matname}"/>
       <child link="${matname}_part5"/>
-      <origin rpy="0.0 0.0 ${pi/2}" xyz="0.024 0.255 0.01"/>
+      <origin rpy="0.0 0.0 ${pi/2}" xyz="0.328 0.163 0.01"/>
     </joint>
     <link name="${matname}_part5"/>
@@ -69,5 +69,5 @@
       <parent link="${matname}"/>
       <child link="${matname}_part6"/>
-      <origin rpy="0.0 0.0 ${pi/2}" xyz="0.345 0.115 0.01"/>
+      <origin rpy="0.0 0.0 ${pi/2}" xyz="0.2 0.2 0.01"/>
     </joint>
     <link name="${matname}_part6"/>
@@ -75,5 +75,5 @@
       <parent link="${matname}"/>
       <child link="${matname}_part7"/>
-      <origin rpy="0.0 0.0 ${pi/2}" xyz="0.065 0.223 0.01"/>
+      <origin rpy="0.0 0.0 ${pi/2}" xyz="0.011 0.011 0.01"/>
     </joint>
     <link name="${matname}_part7"/>
@@ -81,5 +81,5 @@
       <parent link="${matname}"/>
       <child link="${matname}_part8"/>
-      <origin rpy="0.0 0.0 ${pi/2}" xyz="0.354 0.052 0.01"/>
+      <origin rpy="0.0 0.0 ${pi/2}" xyz="0.011 0.013 0.01"/>
     </joint>
     <link name="${matname}_part8"/>
@@ -87,5 +87,5 @@
       <parent link="${matname}"/>
       <child link="${matname}_part9"/>
-      <origin rpy="0.0 0.0 ${pi/2}" xyz="0.043 0.045 0.01"/>
+      <origin rpy="0.0 0.0 ${pi/2}" xyz="0.155 0.094 0.01"/>
     </joint>
     <link name="${matname}_part9"/>
@@ -93,5 +93,5 @@
       <parent link="${matname}"/>
       <child link="${matname}_part10"/>
-      <origin rpy="0.0 0.0 ${pi/2}" xyz="0.055 0.245 0.01"/>
+      <origin rpy="0.0 0.0 ${pi/2}" xyz="0.252 0.106 0.01"/>
     </joint>
     <link name="${matname}_part10"/>
@@ -99,5 +99,5 @@
       <parent link="${matname}"/>
       <child link="${matname}_part11"/>
-      <origin rpy="0.0 0.0 ${pi/2}" xyz="0.259 0.011 0.01"/>
+      <origin rpy="0.0 0.0 ${pi/2}" xyz="0.0 0.001 0.01"/>
     </joint>
     <link name="${matname}_part11"/>
@@ -105,5 +105,5 @@
       <parent link="${matname}"/>
       <child link="${matname}_part12"/>
-      <origin rpy="0.0 0.0 ${pi/2}" xyz="0.05 0.234 0.01"/>
+      <origin rpy="0.0 0.0 ${pi/2}" xyz="0.002 0.003 0.01"/>
     </joint>
     <link name="${matname}_part12"/>
@@ -111,5 +111,5 @@
       <parent link="${matname}"/>
       <child link="${matname}_part13"/>
-      <origin rpy="0.0 0.0 ${pi/2}" xyz="0.024 0.345 0.01"/>
+      <origin rpy="0.0 0.0 ${pi/2}" xyz="0.003 0.003 0.01"/>
     </joint>
     <link name="${matname}_part13"/>
@@ -117,5 +117,5 @@
       <parent link="${matname}"/>
       <child link="${matname}_part14"/>
-      <origin rpy="0.0 0.0 ${pi/2}" xyz="0.234 0.345 0.01"/>
+      <origin rpy="0.0 0.0 ${pi/2}" xyz="0.249 0.0445 0.01"/>
     </joint>
     <link name="${matname}_part14"/>
@@ -123,5 +123,5 @@
       <parent link="${matname}"/>
       <child link="${matname}_part15"/>
-      <origin rpy="0.0 0.0 ${pi/2}" xyz="0.046 0.151 0.01"/>
+      <origin rpy="0.0 0.0 ${pi/2}" xyz="0.3465 0.051 0.01"/>
     </joint>
     <link name="${matname}_part15"/>
