Commit message: Fix taskboard & placement mat scene
The height of the placement mat was 1 cm too high.

File: o2as_scene_description/urdf/o2as_mat.xacro (robot description, xacro)
@@ -7,4 +7,13 @@
       <visual>
         <origin xyz="${mat_w/2} ${mat_l/2} ${mat_h/2}" rpy="0 0 0"/>
+        <geometry>
+          <box size="${mat_w} ${mat_l} ${mat_h}"/>
+        </geometry>
+        <material name="white">
+          <color rgba="1 1 1 1"/>
+        </material>
+      </visual>
+      <visual>
+        <origin xyz="${mat_w/2} ${mat_l/2} ${mat_h/2}+.0001" rpy="0 0 0"/>
         <geometry>
           <box size="${mat_w} ${mat_l} ${mat_h}"/>
@@ -39,5 +48,5 @@
       <parent link="${matname}"/>
       <child link="${matname}_part1"/>
-      <origin rpy="0.0 0.0 ${pi/2}" xyz="0.073 0.285 0.01"/>
+      <origin rpy="0.0 0.0 ${pi/2}" xyz="0.073 0.285 0.0"/>
     </joint>
     <link name="${matname}_part1"/>
@@ -45,5 +54,5 @@
       <parent link="${matname}"/>
       <child link="${matname}_part2"/>
-      <origin rpy="0.0 0.0 ${pi/2}" xyz="0.0525 0.207 0.01"/>
+      <origin rpy="0.0 0.0 ${pi/2}" xyz="0.0525 0.207 0.0"/>
     </joint>
     <link name="${matname}_part2"/>
@@ -51,5 +60,5 @@
       <parent link="${matname}"/>
       <child link="${matname}_part3"/>
-      <origin rpy="0.0 0.0 ${pi/2}" xyz="0.261 0.323 0.01"/>
+      <origin rpy="0.0 0.0 ${pi/2}" xyz="0.261 0.323 0.0"/>
     </joint>
     <link name="${matname}_part3"/>
@@ -57,5 +66,5 @@
       <parent link="${matname}"/>
       <child link="${matname}_part4"/>
-      <origin rpy="0.0 0.0 ${pi/2}" xyz="0.343 0.3235 0.01"/>
+      <origin rpy="0.0 0.0 ${pi/2}" xyz="0.343 0.3235 0.0"/>
     </joint>
     <link name="${matname}_part4"/>
@@ -63,5 +72,5 @@
       <parent link="${matname}"/>
       <child link="${matname}_part5"/>
-      <origin rpy="0.0 0.0 ${pi/2}" xyz="0.328 0.163 0.01"/>
+      <origin rpy="0.0 0.0 ${pi/2}" xyz="0.328 0.163 0.0"/>
     </joint>
     <link name="${matname}_part5"/>
@@ -69,5 +78,5 @@
       <parent link="${matname}"/>
       <child link="${matname}_part6"/>
-      <origin rpy="0.0 0.0 ${pi/2}" xyz="0.2 0.2 0.01"/>
+      <origin rpy="0.0 0.0 ${pi/2}" xyz="0.2 0.2 0.0"/>
     </joint>
     <link name="${matname}_part6"/>
@@ -75,5 +84,5 @@
       <parent link="${matname}"/>
       <child link="${matname}_part7"/>
-      <origin rpy="0.0 0.0 ${pi/2}" xyz="0.011 0.011 0.01"/>
+      <origin rpy="0.0 0.0 ${pi/2}" xyz="0.011 0.011 0.0"/>
     </joint>
     <link name="${matname}_part7"/>
@@ -81,5 +90,5 @@
       <parent link="${matname}"/>
       <child link="${matname}_part8"/>
-      <origin rpy="0.0 0.0 ${pi/2}" xyz="0.011 0.013 0.01"/>
+      <origin rpy="0.0 0.0 ${pi/2}" xyz="0.011 0.013 0.0"/>
     </joint>
     <link name="${matname}_part8"/>
@@ -87,5 +96,5 @@
       <parent link="${matname}"/>
       <child link="${matname}_part9"/>
-      <origin rpy="0.0 0.0 ${pi/2}" xyz="0.155 0.094 0.01"/>
+      <origin rpy="0.0 0.0 ${pi/2}" xyz="0.155 0.094 0.0"/>
     </joint>
     <link name="${matname}_part9"/>
@@ -93,5 +102,5 @@
       <parent link="${matname}"/>
       <child link="${matname}_part10"/>
-      <origin rpy="0.0 0.0 ${pi/2}" xyz="0.252 0.106 0.01"/>
+      <origin rpy="0.0 0.0 ${pi/2}" xyz="0.252 0.106 0.0"/>
     </joint>
     <link name="${matname}_part10"/>
@@ -99,5 +108,5 @@
       <parent link="${matname}"/>
       <child link="${matname}_part11"/>
-      <origin rpy="0.0 0.0 ${pi/2}" xyz="0.0 0.001 0.01"/>
+      <origin rpy="0.0 0.0 ${pi/2}" xyz="0.0 0.001 0.0"/>
     </joint>
     <link name="${matname}_part11"/>
@@ -105,5 +114,5 @@
       <parent link="${matname}"/>
       <child link="${matname}_part12"/>
-      <origin rpy="0.0 0.0 ${pi/2}" xyz="0.002 0.003 0.01"/>
+      <origin rpy="0.0 0.0 ${pi/2}" xyz="0.002 0.003 0.0"/>
     </joint>
     <link name="${matname}_part12"/>
@@ -111,5 +120,5 @@
       <parent link="${matname}"/>
       <child link="${matname}_part13"/>
-      <origin rpy="0.0 0.0 ${pi/2}" xyz="0.003 0.003 0.01"/>
+      <origin rpy="0.0 0.0 ${pi/2}" xyz="0.003 0.003 0.0"/>
     </joint>
     <link name="${matname}_part13"/>
@@ -117,5 +126,5 @@
       <parent link="${matname}"/>
       <child link="${matname}_part14"/>
-      <origin rpy="0.0 0.0 ${pi/2}" xyz="0.249 0.0445 0.01"/>
+      <origin rpy="0.0 0.0 ${pi/2}" xyz="0.249 0.0445 0.0"/>
     </joint>
     <link name="${matname}_part14"/>
@@ -123,5 +132,5 @@
       <parent link="${matname}"/>
       <child link="${matname}_part15"/>
-      <origin rpy="0.0 0.0 ${pi/2}" xyz="0.3465 0.051 0.01"/>
+      <origin rpy="0.0 0.0 ${pi/2}" xyz="0.3465 0.051 0.0"/>
     </joint>
     <link name="${matname}_part15"/>
@@ -129,5 +138,5 @@
       <parent link="${matname}"/>
       <child link="${matname}_corner1"/>
-      <origin rpy="0.0 0.0 ${pi/2}" xyz="0.01 0.01 0.06"/>
+      <origin rpy="0.0 0.0 ${pi/2}" xyz="0.01 0.01 0.0"/>
     </joint>
     <link name="${matname}_corner1"/>
@@ -135,5 +144,5 @@
       <parent link="${matname}"/>
       <child link="${matname}_corner2"/>
-      <origin rpy="0.0 0.0 ${pi/2}" xyz="0.39 0.01 0.06"/>
+      <origin rpy="0.0 0.0 ${pi/2}" xyz="0.39 0.01 0.0"/>
     </joint>
     <link name="${matname}_corner2"/>
@@ -141,5 +150,5 @@
       <parent link="${matname}"/>
       <child link="${matname}_corner3"/>
-      <origin rpy="0.0 0.0 ${pi/2}" xyz="0.39 0.39 0.06"/>
+      <origin rpy="0.0 0.0 ${pi/2}" xyz="0.39 0.39 0.0"/>
     </joint>
     <link name="${matname}_corner3"/>
@@ -147,5 +156,5 @@
       <parent link="${matname}"/>
       <child link="${matname}_corner4"/>
-      <origin rpy="0.0 0.0 ${pi/2}" xyz="0.01 0.39 0.06"/>
+      <origin rpy="0.0 0.0 ${pi/2}" xyz="0.01 0.39 0.0"/>
     </joint>
     <link name="${matname}_corner4"/>

File: o2as_scene_description/urdf/task_board.xacro (robot description, xacro)
@@ -1,17 +1,15 @@
 <robot xmlns:xacro="http://www.ros.org/wiki/xacro" name="task_board">
   <xacro:macro name="task_board" params="boardname parent *origin">
-  <!-- The lines above don't work, the lines below do. Why?? This seems like a bug. -->
   <xacro:property name="mesh_file" value="package://o2as_scene_description/meshes/taskBoard.STL" />
   <link name="${boardname}">
     <inertial>
-      <origin rpy="0 0 0" xyz="0 0 0"/>
+      <origin rpy="0 0 0" xyz="0 0 0.03"/>
       <mass value="1.0"/>
       <inertia ixx="1.0" ixy="0" ixz="0" iyy="1.0" iyz="0" izz="1.0"/>
     </inertial>
     <visual>
-      <origin rpy="0 0 0" xyz="0 0 0"/>
+      <origin rpy="0 0 0" xyz="0 0 0.03"/>
       <geometry>
         <mesh filename="${mesh_file}" scale="1 1 1"/>
-        <!-- <mesh filename="package://ur_description/meshes/ur5/visual/shoulder.dae"/> -->
       </geometry>
       <material name="white">
@@ -20,8 +18,7 @@
     </visual>
     <collision>
-      <origin rpy="0 0 0" xyz="0 0 0"/>
+      <origin rpy="0 0 0" xyz="0 0 0.03"/>
       <geometry>
         <mesh filename="${mesh_file}" scale="1 1 1"/>
-        <!-- <mesh filename="package://ur_description/meshes/ur5/collision/shoulder.stl"/> -->
       </geometry>
     </collision>
@@ -32,37 +29,43 @@
     <xacro:insert_block name="origin"/>
   </joint>
+  <joint name="${boardname}_surface" type="fixed">
+    <parent link="${boardname}" />
+    <child link = "${boardname}_surface"/>
+    <origin rpy="0.0 0.0 0.0" xyz="0.0 0.0 0.04"/>
+  </joint>
+  <link name="${boardname}_surface"/>
   <joint name="${boardname}_part1" type="fixed">
-    <parent link="${boardname}"/>
+    <parent link="${boardname}_surface"/>
     <child link="${boardname}_part1"/>
-    <origin rpy="0.0 0.0 ${pi/2}" xyz="0.34 0.34 0.01"/>
+    <origin rpy="0.0 0.0 ${pi/2}" xyz="0.34 0.34 0.0"/>
   </joint>
   <link name="${boardname}_part1"/>
   <joint name="${boardname}_part2" type="fixed">
-    <parent link="${boardname}"/>
+    <parent link="${boardname}_surface"/>
     <child link="${boardname}_part2"/>
-    <origin rpy="0.0 0.0 ${pi/2}" xyz="0.05 0.35 0.01"/>
+    <origin rpy="0.0 0.0 ${pi/2}" xyz="0.05 0.35 0.0"/>
   </joint>
   <link name="${boardname}_part2"/>
   <joint name="${boardname}_part3" type="fixed">
-    <parent link="${boardname}"/>
+    <parent link="${boardname}_surface"/>
     <child link="${boardname}_part3"/>
-    <origin rpy="0.0 0.0 ${pi/2}" xyz="0.08 0.31 0.01"/>
+    <origin rpy="0.0 0.0 ${pi/2}" xyz="0.08 0.31 0.0"/>
   </joint>
   <link name="${boardname}_part3"/>
   <joint name="${boardname}_part4" type="fixed">
-    <parent link="${boardname}"/>
+    <parent link="${boardname}_surface"/>
     <child link="${boardname}_part4"/>
-    <origin rpy="0.0 0.0 ${pi/2}" xyz="0.15 0.28 0.01"/>
+    <origin rpy="0.0 0.0 ${pi/2}" xyz="0.15 0.28 0.0"/>
   </joint>
   <link name="${boardname}_part4"/>
   <joint name="${boardname}_part5" type="fixed">
-    <parent link="${boardname}"/>
+    <parent link="${boardname}_surface"/>
     <child link="${boardname}_part5"/>
-    <origin rpy="0.0 0.0 ${pi/2}" xyz="0.07 0.26 0.0145"/>
+    <origin rpy="0.0 0.0 ${pi/2}" xyz="0.07 0.26 0.0045"/>
   </joint>
   <link name="${boardname}_part5"/>
   <!--  -->
   <joint name="${boardname}_part6_small_pulley" type="fixed">
-    <parent link="${boardname}"/>
+    <parent link="${boardname}_surface"/>
     <child link="${boardname}_part6_small_pulley"/>
     <origin rpy="0.0 0.0 ${pi/2}" xyz="0.06 0.06 0.0085"/>
@@ -70,5 +73,5 @@
   <link name="${boardname}_part6_small_pulley"/>
   <joint name="${boardname}_part6_large_pulley" type="fixed">
-    <parent link="${boardname}"/>
+    <parent link="${boardname}_surface"/>
     <child link="${boardname}_part6_large_pulley"/>
     <origin rpy="0.0 0.0 ${pi/2}" xyz="0.188 0.06 0.0085"/>
@@ -78,5 +81,5 @@
   <!--  -->
   <joint name="${boardname}_part7a" type="fixed">
-    <parent link="${boardname}"/>
+    <parent link="${boardname}_surface"/>
     <child link="${boardname}_part7a"/>
     <origin rpy="0.0 0.0 ${pi/2}" xyz="0.335 0.056 0.05"/>
@@ -84,5 +87,5 @@
   <link name="${boardname}_part7a"/>
   <joint name="${boardname}_part7b" type="fixed">
-    <parent link="${boardname}"/>
+    <parent link="${boardname}_surface"/>
     <child link="${boardname}_part7b"/>
     <origin rpy="0.0 0.0 ${pi/2}" xyz="0.338 0.056 0.05"/>
@@ -91,73 +94,73 @@
   <!--  -->
   <joint name="${boardname}_part8" type="fixed">
-    <parent link="${boardname}"/>
+    <parent link="${boardname}_surface"/>
     <child link="${boardname}_part8"/>
-    <origin rpy="0.0 0.0 ${pi/2}" xyz="0.32 0.25 0.022"/>
+    <origin rpy="0.0 0.0 ${pi/2}" xyz="0.32 0.25 0.012"/>
   </joint>
   <link name="${boardname}_part8"/>
   <joint name="${boardname}_part9" type="fixed">
-    <parent link="${boardname}"/>
+    <parent link="${boardname}_surface"/>
     <child link="${boardname}_part9"/>
-    <origin rpy="0.0 0.0 ${pi/2}" xyz="0.26 0.15 0.019"/>
+    <origin rpy="0.0 0.0 ${pi/2}" xyz="0.26 0.15 0.009"/>
   </joint>
   <link name="${boardname}_part9"/>
   <joint name="${boardname}_part10" type="fixed">
-    <parent link="${boardname}"/>
+    <parent link="${boardname}_surface"/>
     <child link="${boardname}_part10"/>
-    <origin rpy="0.0 0.0 ${pi/2}" xyz="0.16 0.36 0.06"/>
+    <origin rpy="0.0 0.0 ${pi/2}" xyz="0.16 0.36 0.05"/>
   </joint>
   <link name="${boardname}_part10"/>
   <joint name="${boardname}_part11" type="fixed">
-    <parent link="${boardname}"/>
+    <parent link="${boardname}_surface"/>
     <child link="${boardname}_part11"/>
-    <origin rpy="0.0 0.0 ${pi/2}" xyz="0.06 0.18 0.01"/>
+    <origin rpy="0.0 0.0 ${pi/2}" xyz="0.06 0.18 0.0"/>
   </joint>
   <link name="${boardname}_part11"/>
   <joint name="${boardname}_part12" type="fixed">
-    <parent link="${boardname}"/>
+    <parent link="${boardname}_surface"/>
     <child link="${boardname}_part12"/>
-    <origin rpy="0.0 0.0 ${pi/2}" xyz="0.14 0.14 0.01"/>
+    <origin rpy="0.0 0.0 ${pi/2}" xyz="0.14 0.14 0.0"/>
   </joint>
   <link name="${boardname}_part12"/>
   <joint name="${boardname}_part13" type="fixed">
-    <parent link="${boardname}"/>
+    <parent link="${boardname}_surface"/>
     <child link="${boardname}_part13"/>
-    <origin rpy="0.0 0.0 ${pi/2}" xyz="0.35 0.12 0.01"/>
+    <origin rpy="0.0 0.0 ${pi/2}" xyz="0.35 0.12 0.0"/>
   </joint>
   <link name="${boardname}_part13"/>
   <joint name="${boardname}_part14" type="fixed">
-    <parent link="${boardname}"/>
+    <parent link="${boardname}_surface"/>
     <child link="${boardname}_part14"/>
-    <origin rpy="0.0 0.0 ${pi/2}" xyz="0.23 0.23 0.06"/>
+    <origin rpy="0.0 0.0 ${pi/2}" xyz="0.23 0.23 0.05"/>
   </joint>
   <link name="${boardname}_part14"/>
   <joint name="${boardname}_part15" type="fixed">
-    <parent link="${boardname}"/>
+    <parent link="${boardname}_surface"/>
     <child link="${boardname}_part15"/>
-    <origin rpy="0.0 0.0 ${pi/2}" xyz="0.16 0.36 0.06"/>
+    <origin rpy="0.0 0.0 ${pi/2}" xyz="0.16 0.36 0.05"/>
   </joint>
   <link name="${boardname}_part15"/>
   <joint name="${boardname}_corner1" type="fixed">
-    <parent link="${boardname}"/>
+    <parent link="${boardname}_surface"/>
     <child link="${boardname}_corner1"/>
-    <origin rpy="0.0 0.0 ${pi/2}" xyz="0.01 0.39 0.06"/>
+    <origin rpy="0.0 0.0 ${pi/2}" xyz="0.01 0.39 0.0"/>
   </joint>
   <link name="${boardname}_corner1"/>
   <joint name="${boardname}_corner2" type="fixed">
-    <parent link="${boardname}"/>
+    <parent link="${boardname}_surface"/>
     <child link="${boardname}_corner2"/>
-    <origin rpy="0.0 0.0 ${pi/2}" xyz="0.39 0.39 0.06"/>
+    <origin rpy="0.0 0.0 ${pi/2}" xyz="0.39 0.39 0.0"/>
   </joint>
   <link name="${boardname}_corner2"/>
   <joint name="${boardname}_corner3" type="fixed">
-    <parent link="${boardname}"/>
+    <parent link="${boardname}_surface"/>
     <child link="${boardname}_corner3"/>
-    <origin rpy="0.0 0.0 ${pi/2}" xyz="0.39 0.01 0.06"/>
+    <origin rpy="0.0 0.0 ${pi/2}" xyz="0.39 0.01 0.0"/>
   </joint>
   <link name="${boardname}_corner3"/>
   <joint name="${boardname}_corner4" type="fixed">
-    <parent link="${boardname}"/>
+    <parent link="${boardname}_surface"/>
     <child link="${boardname}_corner4"/>
-    <origin rpy="0.0 0.0 ${pi/2}" xyz="0.01 0.01 0.06"/>
+    <origin rpy="0.0 0.0 ${pi/2}" xyz="0.01 0.01 0.0"/>
   </joint>
   <link name="${boardname}_corner4"/>

File: o2as_scene_description/urdf/taskboard_scene.xacro (robot description, xacro)
@@ -5,5 +5,5 @@
   <xacro:include filename="$(find o2as_scene_description)/urdf/task_board.xacro" />
   <xacro:task_board boardname="taskboard" parent="workspace_center">
-    <origin xyz="-0.35 0.2 0.030" rpy="0 0 ${-pi/2}" />
+    <origin xyz="-0.35 0.2 0.0" rpy="0 0 ${-pi/2}" />
   </xacro:task_board>
   <!-- Placement mat -->
@@ -11,6 +11,6 @@
   <xacro:property name="p_w" value="0.4"/>
   <xacro:property name="p_l" value="0.4"/>
-  <xacro:o2as_mat matname="mat" mat_w="${p_w}" mat_l="${p_l}" mat_h=".001" parent="taskboard">
-    <origin xyz="0.0 0.41 -0.029" rpy="0 0 0" />
+  <xacro:o2as_mat matname="mat" mat_w="${p_w}" mat_l="${p_l}" mat_h=".0001" parent="taskboard">
+    <origin xyz="0.0 0.41 0.0" rpy="0 0 0" />
   </xacro:o2as_mat>
 </robot>

Commit message: Remeasured mat to reattempt pick

File: o2as_scene_description/urdf/o2as_mat.xacro (robot description, xacro)
@@ -88,5 +88,5 @@
       <parent link="${matname}"/>
       <child link="${matname}_part3"/>
-      <origin rpy="0.0 0.0 ${pi/2}" xyz="0.261 0.323 0.0"/>
+      <origin rpy="0.0 0.0 ${pi/2}" xyz="0.262 0.323 0.0"/>
     </joint>
     <link name="${matname}_part3"/>
@@ -130,5 +130,5 @@
       <parent link="${matname}"/>
       <child link="${matname}_part10"/>
-      <origin rpy="0.0 0.0 ${pi/2}" xyz="0.252 0.106 0.0"/>
+      <origin rpy="0.0 0.0 ${pi/2}" xyz="0.2565 0.1065 0.0"/>
     </joint>
     <link name="${matname}_part10"/>
@@ -160,5 +160,5 @@
       <parent link="${matname}"/>
       <child link="${matname}_part15"/>
-      <origin rpy="0.0 0.0 ${pi/2}" xyz="0.3465 0.051 0.0"/>
+      <origin rpy="0.0 0.0 ${pi/2}" xyz="0.346 0.0515 0.0"/>
     </joint>
     <link name="${matname}_part15"/>

Commit message: Add part7 locations to mat URDF manually

File: o2as_scene_description/urdf/o2as_mat.xacro (robot description, xacro)
@@ -109,10 +109,16 @@
     </joint>
     <link name="${matname}_part6"/>
-    <joint name="${matname}_part7" type="fixed">
+    <joint name="${matname}_part7a" type="fixed">
       <parent link="${matname}"/>
-      <child link="${matname}_part7"/>
-      <origin rpy="0.0 0.0 ${pi/2}" xyz="0.011 0.011 0.0"/>
+      <child link="${matname}_part7a"/>
+      <origin rpy="0.0 0.0 ${pi/2}" xyz="0.0785 0.116 0.0"/>
     </joint>
-    <link name="${matname}_part7"/>
+    <link name="${matname}_part7a"/>
+    <joint name="${matname}_part7b" type="fixed">
+      <parent link="${matname}"/>
+      <child link="${matname}_part7b"/>
+      <origin rpy="0.0 0.0 ${pi/2}" xyz="0.0785 0.116 0.0"/>
+    </joint>
+    <link name="${matname}_part7b"/>
     <joint name="${matname}_part8" type="fixed">
       <parent link="${matname}"/>

Commit message: add osaka test environment

File: o2as_scene_description/urdf/o2as_mat.xacro (robot description, xacro)
@@ -73,5 +73,5 @@
       <xacro:insert_block name="origin"/>
     </joint>
-    <joint name="${matname}_part1" type="fixed">
+        <joint name="${matname}_part1" type="fixed">
       <parent link="${matname}"/>
       <child link="${matname}_part1"/>
@@ -88,5 +88,5 @@
       <parent link="${matname}"/>
       <child link="${matname}_part3"/>
-      <origin rpy="0.0 0.0 ${pi/2}" xyz="0.262 0.323 0.0"/>
+      <origin rpy="0.0 0.0 ${pi/2}" xyz="0.261 0.323 0.0"/>
     </joint>
     <link name="${matname}_part3"/>
@@ -109,16 +109,10 @@
     </joint>
     <link name="${matname}_part6"/>
-    <joint name="${matname}_part7a" type="fixed">
+    <joint name="${matname}_part7" type="fixed">
       <parent link="${matname}"/>
-      <child link="${matname}_part7a"/>
-      <origin rpy="0.0 0.0 ${pi/2}" xyz="0.0785 0.116 0.0"/>
+      <child link="${matname}_part7"/>
+      <origin rpy="0.0 0.0 ${pi/2}" xyz="0.011 0.011 0.0"/>
     </joint>
-    <link name="${matname}_part7a"/>
-    <joint name="${matname}_part7b" type="fixed">
-      <parent link="${matname}"/>
-      <child link="${matname}_part7b"/>
-      <origin rpy="0.0 0.0 ${pi/2}" xyz="0.0785 0.116 0.0"/>
-    </joint>
-    <link name="${matname}_part7b"/>
+    <link name="${matname}_part7"/>
     <joint name="${matname}_part8" type="fixed">
       <parent link="${matname}"/>
@@ -136,5 +130,5 @@
       <parent link="${matname}"/>
       <child link="${matname}_part10"/>
-      <origin rpy="0.0 0.0 ${pi/2}" xyz="0.2565 0.1065 0.0"/>
+      <origin rpy="0.0 0.0 ${pi/2}" xyz="0.252 0.106 0.0"/>
     </joint>
     <link name="${matname}_part10"/>
@@ -166,5 +160,5 @@
       <parent link="${matname}"/>
       <child link="${matname}_part15"/>
-      <origin rpy="0.0 0.0 ${pi/2}" xyz="0.346 0.0515 0.0"/>
+      <origin rpy="0.0 0.0 ${pi/2}" xyz="0.3465 0.051 0.0"/>
     </joint>
     <link name="${matname}_part15"/>
@@ -172,5 +166,5 @@
       <parent link="${matname}"/>
       <child link="${matname}_corner1"/>
-      <origin rpy="0.0 0.0 ${pi/2}" xyz="0.01 0.01 0.0"/>
+      <origin rpy="0.0 0.0 ${pi/2}" xyz="0.01 0.01 0.06"/>
     </joint>
     <link name="${matname}_corner1"/>
@@ -178,5 +172,5 @@
       <parent link="${matname}"/>
       <child link="${matname}_corner2"/>
-      <origin rpy="0.0 0.0 ${pi/2}" xyz="0.39 0.01 0.0"/>
+      <origin rpy="0.0 0.0 ${pi/2}" xyz="0.39 0.01 0.06"/>
     </joint>
     <link name="${matname}_corner2"/>
@@ -184,5 +178,5 @@
       <parent link="${matname}"/>
       <child link="${matname}_corner3"/>
-      <origin rpy="0.0 0.0 ${pi/2}" xyz="0.39 0.39 0.0"/>
+      <origin rpy="0.0 0.0 ${pi/2}" xyz="0.39 0.39 0.06"/>
     </joint>
     <link name="${matname}_corner3"/>
@@ -190,5 +184,5 @@
       <parent link="${matname}"/>
       <child link="${matname}_corner4"/>
-      <origin rpy="0.0 0.0 ${pi/2}" xyz="0.01 0.39 0.0"/>
+      <origin rpy="0.0 0.0 ${pi/2}" xyz="0.01 0.39 0.06"/>
     </joint>
     <link name="${matname}_corner4"/>

File: o2as_scene_description/urdf/o2as_osakabase_scene.urdf.xacro (robot description, xacro)
@@ -54,5 +54,5 @@
   <xacro:include filename="$(find o2as_scene_description)/urdf/screw_tools.xacro" />
   <!-- Feeders -->
-  <xacro:include filename="$(find o2as_scene_description)/urdf/screw_feeder.xacro" />
+  <!-- <xacro:include filename="$(find o2as_scene_description)/urdf/screw_feeder.xacro" />
   <xacro:screw_feeder feedername="m3_feeder" parent="a_bot_base_smfl">
     <origin xyz=".1 .4 .05" rpy="0 0 ${pi/2}" />
@@ -60,5 +60,5 @@
   <xacro:screw_feeder feedername="m4_feeder" parent="c_bot_base_smfl">
     <origin xyz=".45 .05 .05" rpy="0 0 0" />
-  </xacro:screw_feeder>
+  </xacro:screw_feeder> -->
   <!-- <xacro:screw_feeder feedername="m5_feeder" parent="c_bot_base_smfl">
     <origin xyz=".45 .2 .05" rpy="0 0 0" />

File: o2as_scene_description/urdf/taskboard_scene.xacro (robot description, xacro)
@@ -5,5 +5,6 @@
   <xacro:include filename="$(find o2as_scene_description)/urdf/task_board.xacro" />
   <xacro:task_board boardname="taskboard" parent="workspace_center">
-    <origin xyz="-0.35 0.2 0.0" rpy="0 0 ${-pi/2}" />
+    <!-- <origin xyz="-0.35 0.2 0.0" rpy="0 0 ${-pi/2}" />    -->
+    <origin xyz="-0.35 0.1 0.0" rpy="0 0 ${-pi/2}" />
   </xacro:task_board>
   <!-- Placement mat -->
