Commit message: Add nut tool adjustments etc.
This contains a lot of other bugfixes as well

File: o2as_scene_description/urdf/o2as_mat.xacro (robot description, xacro)
@@ -118,5 +118,5 @@
       <parent link="${matname}"/>
       <child link="${matname}_part7_2"/>
-      <origin rpy="0.0 0.0 ${pi/2}" xyz="0.1 0.1 0.0"/>
+      <origin rpy="0.0 0.0 ${pi/2}" xyz="0.319 0.154 0.0"/>
     </joint>
     <link name="${matname}_part7_2"/>
@@ -124,5 +124,5 @@
       <parent link="${matname}"/>
       <child link="${matname}_part8"/>
-      <origin rpy="0.0 0.0 ${pi/2}" xyz="0.1 0.1 0.0"/>
+      <origin rpy="0.0 0.0 ${pi/2}" xyz="0.068 0.108 0.0"/>
     </joint>
     <link name="${matname}_part8"/>
@@ -142,5 +142,5 @@
       <parent link="${matname}"/>
       <child link="${matname}_part11"/>
-      <origin rpy="0.0 0.0 ${pi/2}" xyz="0.1 0.1 0.0"/>
+      <origin rpy="0.0 0.0 ${pi/2}" xyz="0.321 0.091 0.0"/>
     </joint>
     <link name="${matname}_part11"/>
@@ -148,5 +148,5 @@
       <parent link="${matname}"/>
       <child link="${matname}_part12"/>
-      <origin rpy="0.0 0.0 ${pi/2}" xyz="0.1 0.1 0.0"/>
+      <origin rpy="0.0 0.0 ${pi/2}" xyz="0.051 0.038 0.0"/>
     </joint>
     <link name="${matname}_part12"/>
@@ -154,5 +154,5 @@
       <parent link="${matname}"/>
       <child link="${matname}_part13"/>
-      <origin rpy="0.0 0.0 ${pi/2}" xyz="0.1 0.1 0.0"/>
+      <origin rpy="0.0 0.0 ${pi/2}" xyz="0.135 0.032 0.0"/>
     </joint>
     <link name="${matname}_part13"/>

File: o2as_scene_description/urdf/robotiq_b_bot_gripper.urdf.xacro (robot description, xacro)
@@ -9,5 +9,5 @@
     <xacro:property name="dx" value="-.03"/>
     <!-- Screw tool tips. X-axis points along the screw into the hole. -->
-    <joint name="${prefix}robotiq_85_m6_screw_tool_tip_joint" type="fixed">
+    <joint name="${prefix}robotiq_85_screw_tool_m6_tip_joint" type="fixed">
       <parent link="${prefix}robotiq_85_tip_link"/>
       <child link="${prefix}screw_tool_m6_tip_link"/>
@@ -15,5 +15,11 @@
     </joint>
     <link name="${prefix}screw_tool_m6_tip_link"/>
-    <joint name="${prefix}robotiq_85_m4_screw_tool_tip_joint" type="fixed">
+    <joint name="${prefix}robotiq_85_nut_tool_m6_tip_joint" type="fixed">
+      <parent link="${prefix}robotiq_85_tip_link"/>
+      <child link="${prefix}nut_tool_m6_tip_link"/>
+      <origin rpy="0.0 ${pi/4} 0.0" xyz="${dx} 0.0 -0.12 "/>
+    </joint>
+    <link name="${prefix}nut_tool_m6_tip_link"/>
+    <joint name="${prefix}robotiq_85_screw_tool_m4_tip_joint" type="fixed">
       <parent link="${prefix}robotiq_85_tip_link"/>
       <child link="${prefix}screw_tool_m4_tip_link"/>
@@ -21,5 +27,5 @@
     </joint>
     <link name="${prefix}screw_tool_m4_tip_link"/>
-    <joint name="${prefix}robotiq_85_m3_screw_tool_tip_joint" type="fixed">
+    <joint name="${prefix}robotiq_85_screw_tool_m3_tip_joint" type="fixed">
       <parent link="${prefix}robotiq_85_tip_link"/>
       <child link="${prefix}screw_tool_m3_tip_link"/>
@@ -27,4 +33,10 @@
     </joint>
     <link name="${prefix}screw_tool_m3_tip_link"/>
+    <joint name="${prefix}robotiq_85_set_screw_tool_tip_joint" type="fixed">
+      <parent link="${prefix}robotiq_85_tip_link"/>
+      <child link="${prefix}set_screw_tool_tip_link"/>
+      <origin rpy="0.0 ${pi/2} 0.0" xyz="${dx+.01} 0.0 -0.085 "/>
+    </joint>
+    <link name="${prefix}set_screw_tool_tip_link"/>
   </xacro:macro>
 </robot>

File: o2as_scene_description/urdf/screw_tools.xacro (robot description, xacro)
@@ -74,4 +74,31 @@
     <origin xyz="-0.05 ${tool_offset} 0.004" rpy="0.0 0.0 0.0" />
   </joint>
+  <link name="nut_tool_m6_link">
+    <inertial>
+      <origin rpy="0 0 0" xyz="0 0 0"/>
+      <mass value="1.0"/>
+      <inertia ixx="1" ixy="0" ixz="0" iyy="1" iyz="0" izz="1"/>
+    </inertial>
+    <!-- <visual>
+      <origin rpy="0 0 0" xyz="0 0 0"/>
+      <geometry>
+        <mesh filename="package://o2as_scene_description/meshes/nut_tool_m6_BC5-XL320-LG20-R_v2.stl" scale="0.001 0.001 0.001"/>
+      </geometry>
+      <material name="white">
+        <color rgba=".9 .9 .9 1"/>
+      </material>
+    </visual>
+    <collision>
+      <origin rpy="0 0 0" xyz="0 ${bit_cushion_to_axis - .02} .0275"/>
+      <geometry>
+        <box size=".026 .04 .055"/>
+      </geometry>
+    </collision> -->
+  </link>
+  <joint name="nut_tool_m6_to_holder" type="fixed">
+    <parent link="screw_tool_holder" />
+    <child link="nut_tool_m6_link" />
+    <origin xyz="-0.05 ${tool_offset} 0.004" rpy="0.0 0.0 0.0" />
+  </joint>
   <link name="screw_tool_m4_link">
     <inertial>
@@ -147,3 +174,9 @@
     <origin xyz="0.0 0.0 0.0" rpy="0.0 0.0 ${-pi/2}" />
   </joint>
+  <link name="nut_tool_m6_helper_link"/>
+  <joint name="nut_tool_m6_helper_joint" type="fixed">
+    <parent link="nut_tool_m6_link" />
+    <child link="nut_tool_m6_helper_link" />
+    <origin xyz="0.0 0.0 0.0" rpy="0.0 0.0 ${-pi/2}" />
+  </joint>
 </robot>

File: o2as_scene_description/urdf/taskboard_scene.xacro (robot description, xacro)
@@ -33,3 +33,9 @@
   </joint>
   <link name="peg_tool"/>
+  <joint name="taskboard_set_screw_tool_joint" type="fixed">
+    <parent link="taskboard"/>
+    <child link="taskboard_set_screw_tool_link"/>
+    <origin rpy="0.0 ${pi/2} ${pi/2}" xyz="-0.08 0.3 0"/>
+  </joint>
+  <link name="taskboard_set_screw_tool_link"/>
 </robot>

Commit message: WIP: Dump commit, end of Monday (Day 1)

File: o2as_scene_description/urdf/o2as_mat.xacro (robot description, xacro)
@@ -76,5 +76,5 @@
       <parent link="${matname}"/>
       <child link="${matname}_part1"/>
-      <origin rpy="0.0 0.0 ${pi/2}" xyz="0.074 0.2835 0.0"/>
+      <origin rpy="0.0 0.0 ${pi/2}" xyz="0.088 0.285 0.0"/>
     </joint>
     <link name="${matname}_part1"/>
@@ -82,5 +82,5 @@
       <parent link="${matname}"/>
       <child link="${matname}_part2"/>
-      <origin rpy="0.0 0.0 ${pi/2}" xyz="0.0525 0.207 0.0"/>
+      <origin rpy="0.0 0.0 ${pi/2}" xyz="0.0835 0.342 0.0"/>
     </joint>
     <link name="${matname}_part2"/>
@@ -88,5 +88,5 @@
       <parent link="${matname}"/>
       <child link="${matname}_part3"/>
-      <origin rpy="0.0 0.0 ${pi/2}" xyz="0.259 0.322 0.0"/>
+      <origin rpy="0.0 0.0 ${pi/2}" xyz="0.256 0.1075 0.0"/>
     </joint>
     <link name="${matname}_part3"/>
@@ -94,5 +94,5 @@
       <parent link="${matname}"/>
       <child link="${matname}_part4"/>
-      <origin rpy="0.0 0.0 ${pi/2}" xyz="0.342 0.3215 0.0"/>
+      <origin rpy="0.0 0.0 ${pi/2}" xyz="0.1535 0.0955 0.0"/>
     </joint>
     <link name="${matname}_part4"/>
@@ -100,5 +100,5 @@
       <parent link="${matname}"/>
       <child link="${matname}_part5"/>
-      <origin rpy="0.0 0.0 ${pi/2}" xyz="0.328 0.163 0.0"/>
+      <origin rpy="0.0 0.0 ${pi/2}" xyz="0.2 0.206 0.0"/>
     </joint>
     <link name="${matname}_part5"/>
@@ -106,5 +106,5 @@
       <parent link="${matname}"/>
       <child link="${matname}_part6"/>
-      <origin rpy="0.0 0.0 ${pi/2}" xyz="0.2 0.2 0.0"/>
+      <origin rpy="0.0 0.0 ${pi/2}" xyz="0.2 0.206 0.0"/>
     </joint>
     <link name="${matname}_part6"/>
@@ -112,5 +112,5 @@
       <parent link="${matname}"/>
       <child link="${matname}_part7_1"/>
-      <origin rpy="0.0 0.0 ${pi/2}" xyz="0.0795 0.116 0.0"/>
+      <origin rpy="0.0 0.0 ${pi/2}" xyz="0.3275 0.165 0.0"/>
     </joint>
     <link name="${matname}_part7_1"/>
@@ -118,5 +118,5 @@
       <parent link="${matname}"/>
       <child link="${matname}_part7_2"/>
-      <origin rpy="0.0 0.0 ${pi/2}" xyz="0.319 0.154 0.0"/>
+      <origin rpy="0.0 0.0 ${pi/2}" xyz="0.3275 0.236 0.0"/>
     </joint>
     <link name="${matname}_part7_2"/>
@@ -124,5 +124,5 @@
       <parent link="${matname}"/>
       <child link="${matname}_part8"/>
-      <origin rpy="0.0 0.0 ${pi/2}" xyz="0.068 0.108 0.0"/>
+      <origin rpy="0.0 0.0 ${pi/2}" xyz="0.1175 0.0775 0.0"/>
     </joint>
     <link name="${matname}_part8"/>
@@ -130,5 +130,5 @@
       <parent link="${matname}"/>
       <child link="${matname}_part9"/>
-      <origin rpy="0.0 0.0 ${pi/2}" xyz="0.153 0.093 0.0"/>
+      <origin rpy="0.0 0.0 ${pi/2}" xyz="0.156 0.095 0.0"/>
     </joint>
     <link name="${matname}_part9"/>
@@ -136,5 +136,5 @@
       <parent link="${matname}"/>
       <child link="${matname}_part10"/>
-      <origin rpy="0.0 0.0 ${pi/2}" xyz="0.2555 0.105 0.0"/>
+      <origin rpy="0.0 0.0 ${pi/2}" xyz="0.256 0.107 0.0"/>
     </joint>
     <link name="${matname}_part10"/>
@@ -142,5 +142,5 @@
       <parent link="${matname}"/>
       <child link="${matname}_part11"/>
-      <origin rpy="0.0 0.0 ${pi/2}" xyz="0.321 0.091 0.0"/>
+      <origin rpy="0.0 0.0 ${pi/2}" xyz="0.0 0.0 0.0"/>
     </joint>
     <link name="${matname}_part11"/>
@@ -148,5 +148,5 @@
       <parent link="${matname}"/>
       <child link="${matname}_part12"/>
-      <origin rpy="0.0 0.0 ${pi/2}" xyz="0.051 0.038 0.0"/>
+      <origin rpy="0.0 0.0 ${pi/2}" xyz="0.0585 0.048 0.0"/>
     </joint>
     <link name="${matname}_part12"/>
@@ -154,5 +154,5 @@
       <parent link="${matname}"/>
       <child link="${matname}_part13"/>
-      <origin rpy="0.0 0.0 ${pi/2}" xyz="0.135 0.032 0.0"/>
+      <origin rpy="0.0 0.0 ${pi/2}" xyz="0.144 0.042 0.0"/>
     </joint>
     <link name="${matname}_part13"/>
@@ -160,5 +160,5 @@
       <parent link="${matname}"/>
       <child link="${matname}_part14"/>
-      <origin rpy="0.0 0.0 ${pi/2}" xyz="0.248 0.0445 0.0"/>
+      <origin rpy="0.0 0.0 ${pi/2}" xyz="0.248 0.047 0.0"/>
     </joint>
     <link name="${matname}_part14"/>
@@ -166,5 +166,5 @@
       <parent link="${matname}"/>
       <child link="${matname}_part15"/>
-      <origin rpy="0.0 0.0 ${pi/2}" xyz="0.344 0.0505 0.0"/>
+      <origin rpy="0.0 0.0 ${pi/2}" xyz="0.3475 0.0525 0.0"/>
     </joint>
     <link name="${matname}_part15"/>

Commit message: Update taskboard and mat positions

File: o2as_scene_description/urdf/o2as_mat.xacro (robot description, xacro)
@@ -76,5 +76,5 @@
       <parent link="${matname}"/>
       <child link="${matname}_part1"/>
-      <origin rpy="0.0 0.0 ${pi/2}" xyz="0.088 0.285 0.0"/>
+      <origin rpy="0.0 0.0 ${pi/2}" xyz="0.074 0.2865 0.0"/>
     </joint>
     <link name="${matname}_part1"/>
@@ -82,5 +82,5 @@
       <parent link="${matname}"/>
       <child link="${matname}_part2"/>
-      <origin rpy="0.0 0.0 ${pi/2}" xyz="0.0835 0.342 0.0"/>
+      <origin rpy="0.0 0.0 ${pi/2}" xyz="0.175 0.3325 0.0"/>
     </joint>
     <link name="${matname}_part2"/>
@@ -88,5 +88,5 @@
       <parent link="${matname}"/>
       <child link="${matname}_part3"/>
-      <origin rpy="0.0 0.0 ${pi/2}" xyz="0.256 0.1075 0.0"/>
+      <origin rpy="0.0 0.0 ${pi/2}" xyz="0.2625 0.324 0.0"/>
     </joint>
     <link name="${matname}_part3"/>
@@ -94,5 +94,5 @@
       <parent link="${matname}"/>
       <child link="${matname}_part4"/>
-      <origin rpy="0.0 0.0 ${pi/2}" xyz="0.1535 0.0955 0.0"/>
+      <origin rpy="0.0 0.0 ${pi/2}" xyz="0.3445 0.324 0.0"/>
     </joint>
     <link name="${matname}_part4"/>
@@ -100,5 +100,5 @@
       <parent link="${matname}"/>
       <child link="${matname}_part5"/>
-      <origin rpy="0.0 0.0 ${pi/2}" xyz="0.2 0.206 0.0"/>
+      <origin rpy="0.0 0.0 ${pi/2}" xyz="0.0 0.0 0.0"/>
     </joint>
     <link name="${matname}_part5"/>
@@ -106,5 +106,5 @@
       <parent link="${matname}"/>
       <child link="${matname}_part6"/>
-      <origin rpy="0.0 0.0 ${pi/2}" xyz="0.2 0.206 0.0"/>
+      <origin rpy="0.0 0.0 ${pi/2}" xyz="0.205 0.205 0.0"/>
     </joint>
     <link name="${matname}_part6"/>
@@ -112,5 +112,5 @@
       <parent link="${matname}"/>
       <child link="${matname}_part7_1"/>
-      <origin rpy="0.0 0.0 ${pi/2}" xyz="0.3275 0.165 0.0"/>
+      <origin rpy="0.0 0.0 ${pi/2}" xyz="0.327 0.164 0.0"/>
     </joint>
     <link name="${matname}_part7_1"/>
@@ -118,5 +118,5 @@
       <parent link="${matname}"/>
       <child link="${matname}_part7_2"/>
-      <origin rpy="0.0 0.0 ${pi/2}" xyz="0.3275 0.236 0.0"/>
+      <origin rpy="0.0 0.0 ${pi/2}" xyz="0.328 0.236 0.0"/>
     </joint>
     <link name="${matname}_part7_2"/>
@@ -124,5 +124,5 @@
       <parent link="${matname}"/>
       <child link="${matname}_part8"/>
-      <origin rpy="0.0 0.0 ${pi/2}" xyz="0.1175 0.0775 0.0"/>
+      <origin rpy="0.0 0.0 ${pi/2}" xyz="0.079 0.117 0.0"/>
     </joint>
     <link name="${matname}_part8"/>
@@ -130,5 +130,5 @@
       <parent link="${matname}"/>
       <child link="${matname}_part9"/>
-      <origin rpy="0.0 0.0 ${pi/2}" xyz="0.156 0.095 0.0"/>
+      <origin rpy="0.0 0.0 ${pi/2}" xyz="0.1555 0.0955 0.0"/>
     </joint>
     <link name="${matname}_part9"/>
@@ -136,5 +136,5 @@
       <parent link="${matname}"/>
       <child link="${matname}_part10"/>
-      <origin rpy="0.0 0.0 ${pi/2}" xyz="0.256 0.107 0.0"/>
+      <origin rpy="0.0 0.0 ${pi/2}" xyz="0.257 0.1075 0.0"/>
     </joint>
     <link name="${matname}_part10"/>
@@ -148,5 +148,5 @@
       <parent link="${matname}"/>
       <child link="${matname}_part12"/>
-      <origin rpy="0.0 0.0 ${pi/2}" xyz="0.0585 0.048 0.0"/>
+      <origin rpy="0.0 0.0 ${pi/2}" xyz="0.06 0.048 0.0"/>
     </joint>
     <link name="${matname}_part12"/>
@@ -154,5 +154,5 @@
       <parent link="${matname}"/>
       <child link="${matname}_part13"/>
-      <origin rpy="0.0 0.0 ${pi/2}" xyz="0.144 0.042 0.0"/>
+      <origin rpy="0.0 0.0 ${pi/2}" xyz="0.145 0.042 0.0"/>
     </joint>
     <link name="${matname}_part13"/>
@@ -160,5 +160,5 @@
       <parent link="${matname}"/>
       <child link="${matname}_part14"/>
-      <origin rpy="0.0 0.0 ${pi/2}" xyz="0.248 0.047 0.0"/>
+      <origin rpy="0.0 0.0 ${pi/2}" xyz="0.25 0.0465 0.0"/>
     </joint>
     <link name="${matname}_part14"/>

File: o2as_scene_description/urdf/task_board.xacro (robot description, xacro)
@@ -63,5 +63,5 @@
     <parent link="${boardname}_surface"/>
     <child link="${boardname}_part1"/>
-    <origin rpy="0.0 0.0 ${pi*0.5}" xyz="0.06 0.34 0.0"/>
+    <origin rpy="0.0 0.0 ${pi*0.5}" xyz="0.34 0.06 0.0"/>
   </joint>
   <link name="${boardname}_part1"/>
@@ -69,5 +69,5 @@
     <parent link="${boardname}_surface"/>
     <child link="${boardname}_part2"/>
-    <origin rpy="0.0 0.0 ${pi*0.5}" xyz="0.05 0.05 0.0"/>
+    <origin rpy="0.0 0.0 ${pi*0.5}" xyz="0.35 0.35 0.0"/>
   </joint>
   <link name="${boardname}_part2"/>
@@ -75,5 +75,5 @@
     <parent link="${boardname}_surface"/>
     <child link="${boardname}_part3"/>
-    <origin rpy="0.0 0.0 ${pi*0.5}" xyz="0.09 0.08 0.0"/>
+    <origin rpy="0.0 0.0 ${pi*0.5}" xyz="0.31 0.32 0.0"/>
   </joint>
   <link name="${boardname}_part3"/>
@@ -81,5 +81,5 @@
     <parent link="${boardname}_surface"/>
     <child link="${boardname}_part4"/>
-    <origin rpy="0.0 0.0 ${pi*0.5}" xyz="0.12 0.15 0.0"/>
+    <origin rpy="0.0 0.0 ${pi*0.5}" xyz="0.28 0.25 0.0"/>
   </joint>
   <link name="${boardname}_part4"/>
@@ -87,5 +87,5 @@
     <parent link="${boardname}_surface"/>
     <child link="${boardname}_part5"/>
-    <origin rpy="0.0 0.0 ${pi*0.5}" xyz="0.14 0.07 0.002"/>
+    <origin rpy="0.0 0.0 ${pi*0.5}" xyz="0.26 0.33 0.002"/>
   </joint>
   <link name="${boardname}_part5">
@@ -103,5 +103,5 @@
     <parent link="${boardname}_surface"/>
     <child link="${boardname}_part15"/>
-    <origin rpy="0.0 0.0 ${pi*0.5}" xyz="0.14 0.07 0.0772"/>
+    <origin rpy="0.0 0.0 ${pi*0.5}" xyz="0.26 0.33 0.0772"/>
   </joint>
   <link name="${boardname}_part15"/>
@@ -109,5 +109,5 @@
     <parent link="${boardname}_surface"/>
     <child link="${boardname}_part6_small_pulley"/>
-    <origin rpy="0.0 0.0 ${pi*1.0}" xyz="0.34 0.06 0.0085"/>
+    <origin rpy="0.0 0.0 ${pi*0.0}" xyz="0.06 0.34 0.0085"/>
   </joint>
   <link name="${boardname}_part6_small_pulley">
@@ -125,5 +125,5 @@
     <parent link="${boardname}_surface"/>
     <child link="${boardname}_part7_1"/>
-    <origin rpy="0.0 0.0 ${pi*0.5}" xyz="0.344 0.361 0.0505"/>
+    <origin rpy="0.0 0.0 ${pi*1.5}" xyz="0.056 0.039 0.0505"/>
   </joint>
   <link name="${boardname}_part7_1"/>
@@ -131,5 +131,5 @@
     <parent link="${boardname}_surface"/>
     <child link="${boardname}_part8"/>
-    <origin rpy="0.0 0.0 ${pi*0.5}" xyz="0.15 0.32 0.012"/>
+    <origin rpy="0.0 0.0 ${pi*0.5}" xyz="0.25 0.08 0.012"/>
   </joint>
   <link name="${boardname}_part8">
@@ -147,5 +147,5 @@
     <parent link="${boardname}_surface"/>
     <child link="${boardname}_part9"/>
-    <origin rpy="0.0 0.0 ${pi*0.5}" xyz="0.25 0.26 0.009"/>
+    <origin rpy="0.0 0.0 ${pi*0.5}" xyz="0.15 0.14 0.009"/>
   </joint>
   <link name="${boardname}_part9">
@@ -163,5 +163,5 @@
     <parent link="${boardname}_surface"/>
     <child link="${boardname}_part10"/>
-    <origin rpy="0.0 0.0 ${pi*0.5}" xyz="0.04 0.16 0.0515"/>
+    <origin rpy="0.0 0.0 ${pi*0.5}" xyz="0.36 0.24 0.0515"/>
   </joint>
   <link name="${boardname}_part10">
@@ -179,5 +179,5 @@
     <parent link="${boardname}_surface"/>
     <child link="${boardname}_part11"/>
-    <origin rpy="0.0 0.0 ${pi*0.5}" xyz="0.22 0.06 0.0"/>
+    <origin rpy="0.0 0.0 ${pi*0.5}" xyz="0.18 0.34 0.0"/>
   </joint>
   <link name="${boardname}_part11"/>
@@ -185,5 +185,5 @@
     <parent link="${boardname}_surface"/>
     <child link="${boardname}_part12"/>
-    <origin rpy="${pi*-0.5} ${pi*0.5} ${pi*0.}" xyz="0.26 0.14 0.0"/>
+    <origin rpy="${pi*-0.5} ${pi*0.5} ${pi*0.}" xyz="0.14 0.26 0.0"/>
   </joint>
   <link name="${boardname}_part12"/>
@@ -191,5 +191,5 @@
     <parent link="${boardname}_surface"/>
     <child link="${boardname}_part13"/>
-    <origin rpy="${pi*-0.5} ${pi*0.5} ${pi*0.}" xyz="0.14 0.07 0.078"/>
+    <origin rpy="${pi*-0.5} ${pi*0.5} ${pi*0.}" xyz="0.26 0.33 0.078"/>
   </joint>
   <link name="${boardname}_part13"/>
@@ -197,5 +197,5 @@
     <parent link="${boardname}_surface"/>
     <child link="${boardname}_part14"/>
-    <origin rpy="0.0 0.0 ${pi*0.5}" xyz="0.17 0.23 0.0515"/>
+    <origin rpy="0.0 0.0 ${pi*0.5}" xyz="0.23 0.17 0.0515"/>
   </joint>
   <link name="${boardname}_part14">

File: o2as_scene_description/urdf/taskboard_scene.xacro (robot description, xacro)
@@ -18,5 +18,5 @@
     <parent link="workspace_center"/>
     <child link="belt_placement_tool"/>
-    <origin rpy="0.0 0.0 0" xyz="-.2 0.3 0"/>
+    <origin rpy="0.0 0.0 0" xyz="-.2 0.37 0"/>
   </joint>
   <link name="belt_placement_tool"/>
@@ -24,5 +24,5 @@
     <parent link="workspace_center"/>
     <child link="retainer_pin_insertion_tool"/>
-    <origin rpy="0.0 0.0 0" xyz="-0.1 0.3 0"/>
+    <origin rpy="0.0 0.0 0" xyz="-0.1 0.36 0"/>
   </joint>
   <link name="retainer_pin_insertion_tool"/>

Commit message: Dump commit of taskboard retrial 1

File: o2as_scene_description/urdf/o2as_mat.xacro (robot description, xacro)
@@ -76,5 +76,5 @@
       <parent link="${matname}"/>
       <child link="${matname}_part1"/>
-      <origin rpy="0.0 0.0 ${pi/2}" xyz="0.193 0.22 0.0"/>
+      <origin rpy="0.0 0.0 ${pi/2}" xyz="0.08 0.2325 0.0"/>
     </joint>
     <link name="${matname}_part1"/>
@@ -82,5 +82,5 @@
       <parent link="${matname}"/>
       <child link="${matname}_part2"/>
-      <origin rpy="0.0 0.0 ${pi/2}" xyz="0.351 0.213 0.0"/>
+      <origin rpy="0.0 0.0 ${pi/2}" xyz="0.345 0.353 0.0"/>
     </joint>
     <link name="${matname}_part2"/>
@@ -88,5 +88,5 @@
       <parent link="${matname}"/>
       <child link="${matname}_part3"/>
-      <origin rpy="0.0 0.0 ${pi/2}" xyz="0.14 0.135 0.0"/>
+      <origin rpy="0.0 0.0 ${pi/2}" xyz="0.324 0.056 0.0"/>
     </joint>
     <link name="${matname}_part3"/>
@@ -94,5 +94,5 @@
       <parent link="${matname}"/>
       <child link="${matname}_part4"/>
-      <origin rpy="0.0 0.0 ${pi/2}" xyz="0.052 0.306 0.0"/>
+      <origin rpy="0.0 0.0 ${pi/2}" xyz="0.18 0.2015 0.0"/>
     </joint>
     <link name="${matname}_part4"/>
@@ -106,5 +106,5 @@
       <parent link="${matname}"/>
       <child link="${matname}_part6"/>
-      <origin rpy="0.0 0.0 ${pi/2}" xyz="0.275 0.1 0.0"/>
+      <origin rpy="0.0 0.0 ${pi/2}" xyz="0.301 0.176 0.0"/>
     </joint>
     <link name="${matname}_part6"/>
@@ -112,5 +112,5 @@
       <parent link="${matname}"/>
       <child link="${matname}_part7_1"/>
-      <origin rpy="0.0 0.0 ${pi/2}" xyz="0.276 0.324 0.0"/>
+      <origin rpy="0.0 0.0 ${pi/2}" xyz="0.0 0.0 0.0"/>
     </joint>
     <link name="${matname}_part7_1"/>
@@ -118,5 +118,5 @@
       <parent link="${matname}"/>
       <child link="${matname}_part7_2"/>
-      <origin rpy="0.0 0.0 ${pi/2}" xyz="0.347 0.323 0.0"/>
+      <origin rpy="0.0 0.0 ${pi/2}" xyz="0.0 0.0 0.0"/>
     </joint>
     <link name="${matname}_part7_2"/>
@@ -124,5 +124,5 @@
       <parent link="${matname}"/>
       <child link="${matname}_part8"/>
-      <origin rpy="0.0 0.0 ${pi/2}" xyz="0.126 0.0525 0.0"/>
+      <origin rpy="0.0 0.0 ${pi/2}" xyz="0.231 0.3505 0.0"/>
     </joint>
     <link name="${matname}_part8"/>
@@ -130,5 +130,5 @@
       <parent link="${matname}"/>
       <child link="${matname}_part9"/>
-      <origin rpy="0.0 0.0 ${pi/2}" xyz="0.077 0.231 0.0"/>
+      <origin rpy="0.0 0.0 ${pi/2}" xyz="0.099 0.048 0.0"/>
     </joint>
     <link name="${matname}_part9"/>
@@ -136,5 +136,5 @@
       <parent link="${matname}"/>
       <child link="${matname}_part10"/>
-      <origin rpy="0.0 0.0 ${pi/2}" xyz="0.293 0.248 0.0"/>
+      <origin rpy="0.0 0.0 ${pi/2}" xyz="0.1755 0.2875 0.0"/>
     </joint>
     <link name="${matname}_part10"/>
@@ -148,5 +148,5 @@
       <parent link="${matname}"/>
       <child link="${matname}_part12"/>
-      <origin rpy="0.0 0.0 ${pi/2}" xyz="0.214 0.348 0.0"/>
+      <origin rpy="0.0 0.0 ${pi/2}" xyz="0.3015 0.2975 0.0"/>
     </joint>
     <link name="${matname}_part12"/>
@@ -154,5 +154,5 @@
       <parent link="${matname}"/>
       <child link="${matname}_part13"/>
-      <origin rpy="0.0 0.0 ${pi/2}" xyz="0.164 0.049 0.0"/>
+      <origin rpy="0.0 0.0 ${pi/2}" xyz="0.0655 0.3105 0.0"/>
     </joint>
     <link name="${matname}_part13"/>
@@ -160,5 +160,5 @@
       <parent link="${matname}"/>
       <child link="${matname}_part14"/>
-      <origin rpy="0.0 0.0 ${pi/2}" xyz="0.345 0.106 0.0"/>
+      <origin rpy="0.0 0.0 ${pi/2}" xyz="0.218 0.056 0.0"/>
     </joint>
     <link name="${matname}_part14"/>
@@ -166,5 +166,5 @@
       <parent link="${matname}"/>
       <child link="${matname}_part15"/>
-      <origin rpy="0.0 0.0 ${pi/2}" xyz="0.0495 0.069 0.0"/>
+      <origin rpy="0.0 0.0 ${pi/2}" xyz="0.046 0.107 0.0"/>
     </joint>
     <link name="${matname}_part15"/>
