Commit message: Modify xacro files to use .dae files instead of .obj

File: o2as_scene_description/urdf/kitting_bins.xacro (robot description, xacro)
@@ -3,5 +3,5 @@
   <xacro:macro name="kitting_bin_internal" params="binname parent filename *origin">
     <xacro:property name="mesh_file" value="package://o2as_scene_description/meshes/${filename}.stl" />
-    <xacro:property name="mesh_file_col" value="package://o2as_scene_description/meshes/${filename}.vhacd.obj" />
+    <xacro:property name="mesh_file_col" value="package://o2as_scene_description/meshes/${filename}.vhacd.dae" />
     <link name="${binname}">
       <inertial>

File: o2as_scene_description/urdf/kitting_tray.xacro (robot description, xacro)
@@ -4,8 +4,8 @@
   <!-- This creates a box with the origin in the bottom corner, connected to the world link. -->
   <!-- <xacro:property name="mesh_file" value="$(find o2as_scene_description)/meshes/bin1_EA661CA-11.stl" />
-  <xacro:property name="mesh_file_col" value="$(find o2as_scene_description)/meshes/bin1_EA661CA-11.vhacd.obj" /> -->
+  <xacro:property name="mesh_file_col" value="$(find o2as_scene_description)/meshes/bin1_EA661CA-11.vhacd.dae" /> -->
   <!-- The lines above don't work, the lines below do. Why?? This seems like a bug. -->
   <xacro:property name="mesh_file" value="package://o2as_scene_description/meshes/tray_PZ-0006-B.stl" />
-  <xacro:property name="mesh_file_col" value="package://o2as_scene_description/meshes/tray_PZ-0006-B.vhacd.obj" />
+  <xacro:property name="mesh_file_col" value="package://o2as_scene_description/meshes/tray_PZ-0006-B.vhacd.dae" />
   <link name="${binname}">
     <inertial>

Commit message: Adjust height of container coordinate frames

File: o2as_scene_description/urdf/kitting_bins.xacro (robot description, xacro)
@@ -1,15 +1,16 @@
 <?xml version="1.0" ?>
 <robot xmlns:xacro="http://ros.org/wiki/xacro" name="kitting_bin">
-  <xacro:macro name="kitting_bin_internal" params="binname parent filename *origin">
+  <!-- z-origin-offset should be set such that the frame is on the surface of the bin -->
+  <xacro:macro name="kitting_bin_internal" params="binname parent filename z_origin_offset *origin">
     <xacro:property name="mesh_file" value="package://o2as_scene_description/meshes/${filename}.stl" />
     <xacro:property name="mesh_file_col" value="package://o2as_scene_description/meshes/${filename}.vhacd.dae" />
     <link name="${binname}">
       <inertial>
-        <origin rpy="0 0 0" xyz="0 0 0"/>
+        <origin rpy="0 0 0" xyz="0 0 ${z_origin_offset}"/>
         <mass value="1.0"/>
         <inertia ixx="1.0" ixy="0" ixz="0" iyy="1.0" iyz="0" izz="1.0"/>
       </inertial>
       <visual>
-        <origin rpy="${pi/2} 0 ${pi/2}" xyz="0 0 0"/>
+        <origin rpy="${pi/2} 0 ${pi/2}" xyz="0 0 ${z_origin_offset}"/>
         <geometry>
           <mesh filename="${mesh_file}" scale="0.001 0.001 0.001"/>
@@ -21,5 +22,5 @@
       </visual>
       <collision>
-        <origin rpy="${pi/2} 0 ${pi/2}" xyz="0 0 0"/>
+        <origin rpy="${pi/2} 0 ${pi/2}" xyz="0 0 ${z_origin_offset}"/>
         <geometry>
           <mesh filename="${mesh_file_col}" scale="0.001 0.001 0.001"/>
@@ -37,16 +38,16 @@
     </joint>
   </xacro:macro>
-  <xacro:macro name="kitting_bin_1" params="binname parent *origin">
-    <xacro:kitting_bin_internal binname="${binname}" parent="${parent}" filename="bin1_EA661CA-11">
+  <xacro:macro name="kitting_bin_1" params="binname parent z_origin_offset *origin">
+    <xacro:kitting_bin_internal binname="${binname}" parent="${parent}" filename="bin1_EA661CA-11" z_origin_offset="${z_origin_offset}">
       <xacro:insert_block name="origin"/>
     </xacro:kitting_bin_internal>
   </xacro:macro>
-  <xacro:macro name="kitting_bin_2" params="binname parent *origin">
-    <xacro:kitting_bin_internal binname="${binname}" parent="${parent}" filename="bin2_SK-HL1-BL">
+  <xacro:macro name="kitting_bin_2" params="binname parent z_origin_offset *origin">
+    <xacro:kitting_bin_internal binname="${binname}" parent="${parent}" filename="bin2_SK-HL1-BL" z_origin_offset="${z_origin_offset}">
       <xacro:insert_block name="origin"/>
     </xacro:kitting_bin_internal>
   </xacro:macro>
-  <xacro:macro name="kitting_bin_3" params="binname parent *origin">
-    <xacro:kitting_bin_internal binname="${binname}" parent="${parent}" filename="bin3_T3-YG">
+  <xacro:macro name="kitting_bin_3" params="binname parent z_origin_offset *origin">
+    <xacro:kitting_bin_internal binname="${binname}" parent="${parent}" filename="bin3_T3-YG" z_origin_offset="${z_origin_offset}">
       <xacro:insert_block name="origin"/>
     </xacro:kitting_bin_internal>

File: o2as_scene_description/urdf/kitting_scene.xacro (robot description, xacro)
@@ -15,24 +15,25 @@
   <xacro:property name="set1_x" value=".00"/>
   <xacro:property name="set1_y" value="${.32-bin1_width/2}"/>
-  <xacro:property name="set1_z" value=".00" />
+  <xacro:property name="set1_z" value=".01" />
+  <xacro:property name="z_origin_offset_1" value="-.008" />
   <!-- set1_bin1_1 -->
-  <xacro:kitting_bin_1 binname="set1_bin1_1" parent="workspace_center">
-    <origin xyz="${set1_x} ${set1_y} ${set1_z}" rpy="0 0 0" />
+  <xacro:kitting_bin_1 binname="set1_bin1_1" parent="workspace_center" z_origin_offset="${z_origin_offset_1}">
+    <origin xyz="${set1_x} ${set1_y} ${set1_z - z_origin_offset_1}" rpy="0 0 0" />
   </xacro:kitting_bin_1>
   <!-- set1_bin1_2 -->
-  <xacro:kitting_bin_1 binname="set1_bin1_2" parent="workspace_center">
-    <origin xyz="${set1_x} ${set1_y - bin1_width*1} ${set1_z}" rpy="0 0 0" />
+  <xacro:kitting_bin_1 binname="set1_bin1_2" parent="workspace_center" z_origin_offset="${z_origin_offset_1}">
+    <origin xyz="${set1_x} ${set1_y - bin1_width*1} ${set1_z - z_origin_offset_1}" rpy="0 0 0" />
   </xacro:kitting_bin_1>
   <!-- set1_bin1_3 -->
-  <xacro:kitting_bin_1 binname="set1_bin1_3" parent="workspace_center">
-    <origin xyz="${set1_x} ${set1_y - bin1_width*2} ${set1_z}" rpy="0 0 0" />
+  <xacro:kitting_bin_1 binname="set1_bin1_3" parent="workspace_center" z_origin_offset="${z_origin_offset_1}">
+    <origin xyz="${set1_x} ${set1_y - bin1_width*2} ${set1_z - z_origin_offset_1}" rpy="0 0 0" />
   </xacro:kitting_bin_1>
   <!-- set1_bin1_4 -->
-  <xacro:kitting_bin_1 binname="set1_bin1_4" parent="workspace_center">
-    <origin xyz="${set1_x} ${set1_y - bin1_width*3} ${set1_z}" rpy="0 0 0" />
+  <xacro:kitting_bin_1 binname="set1_bin1_4" parent="workspace_center" z_origin_offset="${z_origin_offset_1}">
+    <origin xyz="${set1_x} ${set1_y - bin1_width*3} ${set1_z - z_origin_offset_1}" rpy="0 0 0" />
   </xacro:kitting_bin_1>
   <!-- set1_bin1_5 -->
-  <xacro:kitting_bin_1 binname="set1_bin1_5" parent="workspace_center">
-    <origin xyz="${set1_x} ${set1_y - bin1_width*4} ${set1_z}" rpy="0 0 0" />
+  <xacro:kitting_bin_1 binname="set1_bin1_5" parent="workspace_center" z_origin_offset="${z_origin_offset_1}">
+    <origin xyz="${set1_x} ${set1_y - bin1_width*4} ${set1_z - z_origin_offset_1}" rpy="0 0 0" />
   </xacro:kitting_bin_1>
   <!-- A row of bin2 and bin3 -->
@@ -41,34 +42,36 @@
   <xacro:property name="set2_y" value="${.32-bin3_width/2}" />
   <xacro:property name="set2_z" value=".00" />
+  <xacro:property name="z_origin_offset_2" value="-.009" />
+  <xacro:property name="z_origin_offset_3" value="-.004" />
   <!-- set2_bin3 -->
-  <xacro:kitting_bin_3 binname="set2_bin3" parent="workspace_center">
-    <origin xyz="${set2_x_bin3} ${set2_y} ${set2_z}" rpy="0 0 0" />
+  <xacro:kitting_bin_3 binname="set2_bin3" parent="workspace_center" z_origin_offset="${z_origin_offset_3}">
+    <origin xyz="${set2_x_bin3} ${set2_y} ${set2_z - z_origin_offset_3}" rpy="0 0 0" />
   </xacro:kitting_bin_3>
   <!-- set2_bin2_1 -->
-  <xacro:kitting_bin_2 binname="set2_bin2_1" parent="workspace_center">
-    <origin xyz="${set2_x_bin2} ${set2_y-bin3_width/2-bin2_width/2*1} ${set2_z}" rpy="0 0 0" />
+  <xacro:kitting_bin_2 binname="set2_bin2_1" parent="workspace_center" z_origin_offset="${z_origin_offset_2}">
+    <origin xyz="${set2_x_bin2} ${set2_y-bin3_width/2-bin2_width/2*1} ${set2_z - z_origin_offset_2}" rpy="0 0 0" />
   </xacro:kitting_bin_2>
   <!-- set2_bin2_2 -->
-  <xacro:kitting_bin_2 binname="set2_bin2_2" parent="workspace_center">
-    <origin xyz="${set2_x_bin2} ${set2_y-bin3_width/2-bin2_width*3/2} ${set2_z}" rpy="0 0 0" />
+  <xacro:kitting_bin_2 binname="set2_bin2_2" parent="workspace_center" z_origin_offset="${z_origin_offset_2}">
+    <origin xyz="${set2_x_bin2} ${set2_y-bin3_width/2-bin2_width*3/2} ${set2_z - z_origin_offset_2}" rpy="0 0 0" />
   </xacro:kitting_bin_2>
   <!-- set2_bin2_3 -->
-  <xacro:kitting_bin_2 binname="set2_bin2_3" parent="workspace_center">
-    <origin xyz="${set2_x_bin2} ${set2_y-bin3_width/2-bin2_width*5/2} ${set2_z}" rpy="0 0 0" />
+  <xacro:kitting_bin_2 binname="set2_bin2_3" parent="workspace_center" z_origin_offset="${z_origin_offset_2}">
+    <origin xyz="${set2_x_bin2} ${set2_y-bin3_width/2-bin2_width*5/2} ${set2_z - z_origin_offset_2}" rpy="0 0 0" />
   </xacro:kitting_bin_2>
   <!-- set2_bin2_4 -->
-  <xacro:kitting_bin_2 binname="set2_bin2_4" parent="workspace_center">
-    <origin xyz="${set2_x_bin2} ${set2_y-bin3_width/2-bin2_width*7/2} ${set2_z}" rpy="0 0 0" />
+  <xacro:kitting_bin_2 binname="set2_bin2_4" parent="workspace_center" z_origin_offset="${z_origin_offset_2}">
+    <origin xyz="${set2_x_bin2} ${set2_y-bin3_width/2-bin2_width*7/2} ${set2_z - z_origin_offset_2}" rpy="0 0 0" />
   </xacro:kitting_bin_2>
   <!-- A row of tray -->
   <xacro:property name="set3_x" value="${-(bin1_length/2+tray_length/2)}" />
   <xacro:property name="set3_y" value="${.32-tray_width/2}" />
-  <xacro:property name="set3_z" value=".00" />
+  <xacro:property name="set3_z" value=".007" />
   <!-- set3_tray_1 -->
-  <xacro:kitting_tray binname="set3_tray_1" parent="workspace_center">
+  <xacro:kitting_tray trayname="set3_tray_1" parent="workspace_center">
     <origin xyz="${set3_x} ${set3_y} ${set3_z}" rpy="0 0 0" />
   </xacro:kitting_tray>
   <!-- set3_tray_2 -->
-  <xacro:kitting_tray binname="set3_tray_2" parent="workspace_center">
+  <xacro:kitting_tray trayname="set3_tray_2" parent="workspace_center">
     <origin xyz="${set3_x} ${set3_y-tray_width} ${set3_z}" rpy="0 0 0" />
   </xacro:kitting_tray>

File: o2as_scene_description/urdf/kitting_tray.xacro (robot description, xacro)
@@ -1,5 +1,5 @@
 <?xml version="1.0" ?>
 <robot xmlns:xacro="http://ros.org/wiki/xacro" name="kitting_bin">
-  <xacro:macro name="kitting_tray" params="binname parent *origin">
+  <xacro:macro name="kitting_tray" params="trayname parent *origin">
   <!-- This creates a box with the origin in the bottom corner, connected to the world link. -->
   <!-- <xacro:property name="mesh_file" value="$(find o2as_scene_description)/meshes/bin1_EA661CA-11.stl" />
@@ -8,12 +8,13 @@
   <xacro:property name="mesh_file" value="package://o2as_scene_description/meshes/tray_PZ-0006-B.stl" />
   <xacro:property name="mesh_file_col" value="package://o2as_scene_description/meshes/tray_PZ-0006-B.vhacd.dae" />
-  <link name="${binname}">
+  <xacro:property name="z_origin_offset" value="-.007" />
+  <link name="${trayname}">
     <inertial>
-      <origin rpy="0 0 0" xyz="0 0 0"/>
+      <origin rpy="0 0 0" xyz="0 0 ${z_origin_offset}"/>
       <mass value="1.0"/>
       <inertia ixx="1.0" ixy="0" ixz="0" iyy="1.0" iyz="0" izz="1.0"/>
     </inertial>
     <visual>
-      <origin rpy="${pi/2} 0 ${pi/2}" xyz="0 0 0"/>
+      <origin rpy="${pi/2} 0 ${pi/2}" xyz="0 0 ${z_origin_offset}"/>
       <geometry>
         <mesh filename="${mesh_file}" scale="0.001 0.001 0.001"/>
@@ -25,5 +26,5 @@
     </visual>
     <collision>
-      <origin rpy="${pi/2} 0 ${pi/2}" xyz="0 0 0"/>
+      <origin rpy="${pi/2} 0 ${pi/2}" xyz="0 0 ${z_origin_offset}"/>
       <geometry>
         <mesh filename="${mesh_file_col}" scale="0.001 0.001 0.001"/>
@@ -32,7 +33,7 @@
     </collision>
   </link>
-  <joint name="${binname}" type="fixed">
+  <joint name="${trayname}" type="fixed">
       <parent link="${parent}" />
-      <child link = "${binname}" />
+      <child link = "${trayname}" />
       <xacro:insert_block name="origin"/>
     </joint>

Commit message: Clean-up

File: o2as_scene_description/urdf/kitting_bins.xacro (robot description, xacro)
@@ -1,4 +1,5 @@
 <?xml version="1.0" ?>
 <robot xmlns:xacro="http://ros.org/wiki/xacro" name="kitting_bin">
+  <!-- These macros define the three bins from which items are picked in the kitting -->
   <!-- z-origin-offset should be set such that the frame is on the surface of the bin -->
   <xacro:macro name="kitting_bin_internal" params="binname parent filename z_origin_offset *origin">

File: o2as_scene_description/urdf/kitting_tray.xacro (robot description, xacro)
@@ -1,9 +1,6 @@
 <?xml version="1.0" ?>
 <robot xmlns:xacro="http://ros.org/wiki/xacro" name="kitting_bin">
+  <!-- This file defines a tray that could be used for temporarily placing items for regrasping during the kitting tray -->
   <xacro:macro name="kitting_tray" params="trayname parent *origin">
-  <!-- This creates a box with the origin in the bottom corner, connected to the world link. -->
-  <!-- <xacro:property name="mesh_file" value="$(find o2as_scene_description)/meshes/bin1_EA661CA-11.stl" />
-  <xacro:property name="mesh_file_col" value="$(find o2as_scene_description)/meshes/bin1_EA661CA-11.vhacd.dae" /> -->
-  <!-- The lines above don't work, the lines below do. Why?? This seems like a bug. -->
   <xacro:property name="mesh_file" value="package://o2as_scene_description/meshes/tray_PZ-0006-B.stl" />
   <xacro:property name="mesh_file_col" value="package://o2as_scene_description/meshes/tray_PZ-0006-B.vhacd.dae" />
