Commit message: Import dual_suction_gripper

File: o2as_scene_description/urdf/kitting_bins.xacro (robot description, xacro)
@@ -1,5 +1,4 @@
 <?xml version="1.0" ?>
 <robot xmlns:xacro="http://ros.org/wiki/xacro" name="kitting_bin">
-  <!-- These macros define the three bins from which items are picked in the kitting -->
   <!-- z-origin-offset should be set such that the frame is on the surface of the bin -->
   <xacro:macro name="kitting_bin_internal" params="binname parent filename z_origin_offset *origin">

File: o2as_scene_description/urdf/kitting_tray.xacro (robot description, xacro)
@@ -1,6 +1,9 @@
 <?xml version="1.0" ?>
 <robot xmlns:xacro="http://ros.org/wiki/xacro" name="kitting_bin">
-  <!-- This file defines a tray that could be used for temporarily placing items for regrasping during the kitting tray -->
   <xacro:macro name="kitting_tray" params="trayname parent *origin">
+  <!-- This creates a box with the origin in the bottom corner, connected to the world link. -->
+  <!-- <xacro:property name="mesh_file" value="$(find o2as_scene_description)/meshes/bin1_EA661CA-11.stl" />
+  <xacro:property name="mesh_file_col" value="$(find o2as_scene_description)/meshes/bin1_EA661CA-11.vhacd.dae" /> -->
+  <!-- The lines above don't work, the lines below do. Why?? This seems like a bug. -->
   <xacro:property name="mesh_file" value="package://o2as_scene_description/meshes/tray_PZ-0006-B.stl" />
   <xacro:property name="mesh_file_col" value="package://o2as_scene_description/meshes/tray_PZ-0006-B.vhacd.dae" />
@@ -16,4 +19,5 @@
       <geometry>
         <mesh filename="${mesh_file}" scale="0.001 0.001 0.001"/>
+        <!-- <mesh filename="package://ur_description/meshes/ur5/visual/shoulder.dae"/> -->
       </geometry>
       <material name="white">
@@ -25,4 +29,5 @@
       <geometry>
         <mesh filename="${mesh_file_col}" scale="0.001 0.001 0.001"/>
+        <!-- <mesh filename="package://ur_description/meshes/ur5/collision/shoulder.stl"/> -->
       </geometry>
     </collision>

File: o2as_scene_description/urdf/o2as_base.xacro (robot description, xacro)
@@ -14,9 +14,8 @@
         </geometry>
         <material name="DarkGrey">
-          <color rgba="0.4 0.4 0.4 1.0"/>
+          <color rgba="0.2 0.2 0.2 1.0"/>
         </material>
       </visual>
       <collision>
-        <origin xyz="${box_w/2} ${box_l/2} ${box_h/2}" rpy="0 0 0"/>
         <geometry>
           <box size="${box_w} ${box_l} ${box_h}"/>

File: o2as_scene_description/urdf/o2as_base_scene.urdf.xacro (robot description, xacro)
@@ -2,13 +2,12 @@
 <robot xmlns:xacro="http://ros.org/wiki/xacro"
        name="o2as_base_scene" >
-  <!-- This is the main file defining our robot arrangement and physical environment. -->
-  <!-- These values are still not fixed -->
   <xacro:property name="a_bot_x" value="0.0"/>
-  <xacro:property name="a_bot_y" value="-0.65"/>
+  <xacro:property name="a_bot_y" value="-0.6"/>
   <xacro:property name="b_bot_x" value="0.0"/>
-  <xacro:property name="b_bot_y" value="0.65"/>
+  <xacro:property name="b_bot_y" value="0.6"/>
   <xacro:property name="c_bot_x" value="-0.5"/>
   <xacro:property name="c_bot_y" value="0.0"/>
   <xacro:property name="bots_z" value="0.75"/>
+  <!-- This is the main file defining our robot arrangement and physical environment. -->
   <!-- common stuff -->
   <xacro:include filename="$(find ur_description)/urdf/common.gazebo.xacro" />
@@ -21,5 +20,5 @@
   <!-- Scene items (trays, bins...) -->
   <xacro:include filename="$(find o2as_scene_description)/urdf/walls.xacro" />
-  <xacro:include filename="$(find o2as_scene_description)/urdf/taskboard_scene.xacro" />
+  <xacro:include filename="$(find o2as_scene_description)/urdf/kitting_scene.xacro" />
   <!-- Robot bases -->
   <!-- Putting these at height 0.0 makes them intersect with the ground, so they are elevated. -->
@@ -27,19 +26,19 @@
   <xacro:include filename="$(find o2as_scene_description)/urdf/o2as_base.xacro" />
   <xacro:o2as_base boxname="a_bot_base_smfl" parent="o2as_ground">
-    <origin xyz="${a_bot_x-.65/2} ${a_bot_y-.65/2} ${bots_z-.06}" rpy="0 0 0" />
+    <origin xyz="${a_bot_x-.65/2} ${a_bot_y-.65/2} 0.65" rpy="0 0 0" />
   </xacro:o2as_base>
   <xacro:o2as_base boxname="b_bot_base_smfl" parent="o2as_ground">
-    <origin xyz="${b_bot_x-.65/2} ${b_bot_y-.65/2} ${bots_z-.06}" rpy="0 0 0" />
+    <origin xyz="${b_bot_x-.65/2} ${b_bot_y-.65/2} 0.65" rpy="0 0 0" />
   </xacro:o2as_base>
   <xacro:o2as_base boxname="c_bot_base_smfl" parent="o2as_ground">
-    <origin xyz="${c_bot_x-.65/2-.16} ${c_bot_y-.65/2-.1} ${bots_z-.06}" rpy="0 0 0" />
+    <origin xyz="${c_bot_x-.65/2-.22} ${c_bot_y-.65/2-.22} 0.65" rpy="0 0 0" />
   </xacro:o2as_base>
   <!-- Main workspace -->
   <!-- The surface is 0.01 m below the robot bases and the "workspace_center" frame. -->
   <xacro:include filename="$(find o2as_scene_description)/urdf/o2as_box.xacro" />
-  <xacro:property name="plate_w" value="0.9"/>
-  <xacro:property name="plate_l" value="0.75"/>
+  <xacro:property name="plate_w" value="0.84"/>
+  <xacro:property name="plate_l" value="0.62"/>
   <xacro:o2as_box boxname="workbox" box_w="${plate_w}" box_l="${plate_l}" box_h=".01" parent="o2as_ground">
-    <origin xyz="${-plate_w/2+.1} ${-plate_l/2} ${bots_z}" rpy="0 0 0" />
+    <origin xyz="${-plate_w/2} ${-plate_l/2} ${bots_z+.09}" rpy="0 0 0" />
   </xacro:o2as_box>
   <link name="workspace_center" />
@@ -47,39 +46,26 @@
     <parent link="o2as_ground" />
     <child link="workspace_center" />
-    <origin xyz="0.0 0.0 ${bots_z+.01}" rpy="0.0 0.0 0.0" />
+    <origin xyz="0.0 0.0 ${bots_z+.1}" rpy="0.0 0.0 0.0" />
   </joint>
-  <!-- Screw holder & screw tool visual -->
-  <xacro:include filename="$(find o2as_scene_description)/urdf/screw_tools.xacro" />
-  <!-- Feeders -->
-  <xacro:include filename="$(find o2as_scene_description)/urdf/screw_feeder.xacro" />
-  <xacro:screw_feeder feedername="m3_feeder" parent="a_bot_base_smfl">
-    <origin xyz=".1 .4 .05" rpy="0 0 ${pi/2}" />
-  </xacro:screw_feeder>
-  <xacro:screw_feeder feedername="m4_feeder" parent="c_bot_base_smfl">
-    <origin xyz=".45 .05 .05" rpy="0 0 0" />
-  </xacro:screw_feeder>
-  <!-- <xacro:screw_feeder feedername="m5_feeder" parent="c_bot_base_smfl">
-    <origin xyz=".45 .2 .05" rpy="0 0 0" />
-  </xacro:screw_feeder> -->
   <!-- robot arms -->
-  <xacro:ur5_robot prefix="a_bot_" joint_limited="false"
-    shoulder_pan_lower_limit="0.0" shoulder_pan_upper_limit="${pi}"
-    shoulder_lift_lower_limit="${-pi}" shoulder_lift_upper_limit="0.0"
+  <xacro:ur5_robot prefix="a_bot_" joint_limited="true"
+    shoulder_pan_lower_limit="${-pi}" shoulder_pan_upper_limit="${pi}"
+    shoulder_lift_lower_limit="${-pi}" shoulder_lift_upper_limit="${pi}"
     elbow_joint_lower_limit="0.0" elbow_joint_upper_limit="${pi}"
-    wrist_1_lower_limit="${-pi}" wrist_1_upper_limit="0.3"
+    wrist_1_lower_limit="${-pi}" wrist_1_upper_limit="${pi}"
     wrist_2_lower_limit="${-pi}" wrist_2_upper_limit="${pi}"
     wrist_3_lower_limit="${-pi}" wrist_3_upper_limit="${pi}"/>
   <xacro:ur5_robot prefix="b_bot_" joint_limited="true"
     shoulder_pan_lower_limit="${-pi}" shoulder_pan_upper_limit="${pi}"
-    shoulder_lift_lower_limit="${-pi}" shoulder_lift_upper_limit="0.0"
+    shoulder_lift_lower_limit="${-pi}" shoulder_lift_upper_limit="${pi}"
     elbow_joint_lower_limit="0.0" elbow_joint_upper_limit="${pi}"
-    wrist_1_lower_limit="${-pi}" wrist_1_upper_limit="0.3"
+    wrist_1_lower_limit="${-pi}" wrist_1_upper_limit="${pi}"
     wrist_2_lower_limit="${-pi}" wrist_2_upper_limit="${pi}"
     wrist_3_lower_limit="${-pi}" wrist_3_upper_limit="${pi}"/>
   <xacro:ur3_robot prefix="c_bot_" joint_limited="true"
-    shoulder_pan_lower_limit="0.0" shoulder_pan_upper_limit="${pi}"
-    shoulder_lift_lower_limit="${-pi}" shoulder_lift_upper_limit="0.0"
+    shoulder_pan_lower_limit="${-pi}" shoulder_pan_upper_limit="${pi}"
+    shoulder_lift_lower_limit="${-pi}" shoulder_lift_upper_limit="${pi}"
     elbow_joint_lower_limit="0.0" elbow_joint_upper_limit="${pi}"
-    wrist_1_lower_limit="${-pi}" wrist_1_upper_limit="0.3"
+    wrist_1_lower_limit="${-pi}" wrist_1_upper_limit="${pi}"
     wrist_2_lower_limit="${-pi}" wrist_2_upper_limit="${pi}"
     wrist_3_lower_limit="${-pi}" wrist_3_upper_limit="${pi}"/>
@@ -101,11 +87,19 @@
   </joint>
   <!-- spawn and attach grippers -->
-  <xacro:include filename="$(find o2as_scene_description)/urdf/precision_gripper.xacro" />
-  <xacro:precision_gripper prefix="a_bot_"  grippername = "gripper" parent = "a_bot_tool0">
-    <origin xyz="0.0 0 0.04" rpy="0 ${pi/2} 0"/>
-  </xacro:precision_gripper>
-  <xacro:include filename="$(find o2as_scene_description)/urdf/robotiq_85_gripper_with_ft300.urdf.xacro" />
-  <xacro:robotiq_85_gripper_o2as prefix="b_bot_" parent = "b_bot_ee_link" />
-  <xacro:robotiq_85_gripper_o2as prefix="c_bot_" parent = "c_bot_ee_link"/>
+  <xacro:include filename="$(find o2as_scene_description)/urdf/robotiq_85_gripper.urdf.xacro" />
+  <xacro:robotiq_85_gripper_o2as prefix="a_bot_" parent = "a_bot_ee_link">
+    <origin xyz="0.0 0 0.0" rpy="0 0 0"/>
+  </xacro:robotiq_85_gripper_o2as>
+  <!-- <xacro:robotiq_85_gripper_o2as prefix="b_bot_" parent = "b_bot_ee_link"> -->
+  <!--   <origin xyz="0.0 0 0.0" rpy="0 0 0"/> -->
+  <!-- </xacro:robotiq_85_gripper_o2as> -->
+  <xacro:robotiq_85_gripper_o2as prefix="c_bot_" parent = "c_bot_ee_link">
+    <origin xyz="0.0 0 0.0" rpy="0 0 0"/>
+  </xacro:robotiq_85_gripper_o2as>
+  <!-- spawn and attach diual suction grippers -->
+  <xacro:include filename="$(find o2as_scene_description)/urdf/dual_suction_gripper.urdf.xacro" />
+  <xacro:dual_suction_gripper_o2as prefix="b_bot_" parent = "b_bot_ee_link">
+    <origin xyz="0 0 0" rpy="0 0 0"/>
+  </xacro:dual_suction_gripper_o2as>
   <!-- Add cameras -->
   <link name="b_bot_cam_holder_link" />
@@ -118,5 +112,5 @@
     <origin xyz="0 0 0" rpy="0 0 0"/>
   </xacro:sensor_d435>
-  <!-- I would like to remove the "world" link definition, but apparently it is necessary for Gazebo -->
+  <!-- I meant to remove the "world" link definition, but apparently it is necessary for Gazebo -->
   <link name="world" />
   <joint name="world_o2as_joint" type="fixed">

File: o2as_scene_description/urdf/o2as_box.xacro (robot description, xacro)
@@ -15,5 +15,4 @@
       </visual>
       <collision>
-        <origin xyz="${box_w/2} ${box_l/2} ${box_h/2}" rpy="0 0 0"/>
         <geometry>
           <box size="${box_w} ${box_l} ${box_h}"/>

File: o2as_scene_description/urdf/walls.xacro (robot description, xacro)
@@ -21,5 +21,15 @@
         </geometry>
       </collision>
+      <!-- Tall objects seem to be instable in Gazebo, so we ignore the walls for the physical simulation. -->
+      <!-- <inertial>
+        <mass value="1.0" />
+        <inertia ixx="1.0" ixy="0.0" ixz="0.0"
+          iyy="1.0" iyz="0.0"
+          izz="1.0" />
+      </inertial> -->
     </link>
+    <!-- <gazebo reference="${wall_name}">
+      <material>Gazebo/Brick</material>
+    </gazebo> -->
     <joint name="${wall_name}" type="fixed">
       <parent link="world" />
@@ -29,6 +39,6 @@
   </xacro:macro>
   <!-- ############################# -->
-  <xacro:o2as_wall wall_name="wall_a" wall_w="${wall_width}" wall_l="${wall_thickness}" wall_h="${wall_height}">
-    <origin xyz="0.0 -1.2 0.0" rpy="0.0 0.0 0.0" />
+  <xacro:o2as_wall wall_name="wall_b" wall_w="${wall_width}" wall_l="${wall_thickness}" wall_h="${wall_height}">
+    <origin xyz="0.0 -1.0 0.0" rpy="0.0 0.0 0.0" />
   </xacro:o2as_wall>
   <xacro:o2as_wall wall_name="wall_c" wall_w="${wall_width}" wall_l="${wall_thickness}" wall_h="${wall_height}">

Commit message: Fixed tabletop camera position.

File: o2as_scene_description/urdf/kitting_bins.xacro (robot description, xacro)
@@ -44,23 +44,23 @@
       <origin xyz=".0 -0.2325 0.018" rpy="0 0 0" />
   </xacro:kitting_bin_1>
+  <!--set2_bin3_1_-->
+  <xacro:kitting_bin_3 binname="set2_bin3_1" parent="workspace_center" z_origin_offset="-.004">
+      <origin xyz=".20 0.234 0.004" rpy="0 0 0" />
+  </xacro:kitting_bin_3>
   <!--set2_bin2_1_-->
   <xacro:kitting_bin_2 binname="set2_bin2_1" parent="workspace_center" z_origin_offset="-.009">
-      <origin xyz=".20 0.274 0.009" rpy="0 0 0" />
+      <origin xyz=".20 0.082 0.009" rpy="0 0 0" />
   </xacro:kitting_bin_2>
   <!--set2_bin2_2_-->
   <xacro:kitting_bin_2 binname="set2_bin2_2" parent="workspace_center" z_origin_offset="-.009">
-      <origin xyz=".20 0.162 0.009" rpy="0 0 0" />
+      <origin xyz=".20 -0.03 0.009" rpy="0 0 0" />
   </xacro:kitting_bin_2>
   <!--set2_bin2_3_-->
   <xacro:kitting_bin_2 binname="set2_bin2_3" parent="workspace_center" z_origin_offset="-.009">
-      <origin xyz=".20 0.05 0.009" rpy="0 0 0" />
+      <origin xyz=".20 -0.142 0.009" rpy="0 0 0" />
   </xacro:kitting_bin_2>
   <!--set2_bin2_4_-->
   <xacro:kitting_bin_2 binname="set2_bin2_4" parent="workspace_center" z_origin_offset="-.009">
-      <origin xyz=".20 -0.062 0.009" rpy="0 0 0" />
+      <origin xyz=".20 -0.254 0.009" rpy="0 0 0" />
   </xacro:kitting_bin_2>
-  <!--set2_bin3_1_-->
-  <xacro:kitting_bin_3 binname="set2_bin3_1" parent="workspace_center" z_origin_offset="-.004">
-      <origin xyz=".20 -0.214 0.004" rpy="0 0 0" />
-  </xacro:kitting_bin_3>
 </robot>

File: o2as_scene_description/urdf/kitting_scene.xacro (robot description, xacro)
@@ -1,6 +1,6 @@
 <?xml version="1.0"?>
 <robot xmlns:xacro="http://www.ros.org/wiki/xacro" name="kitting_scene">
-  <xacro:include filename="$(find o2as_scene_description)/urdf/kitting_bins.xacro" />
-  <xacro:include filename="$(find o2as_scene_description)/urdf/kitting_tray_with_partitions.xacro" />
+  <!-- <xacro:include filename="$(find o2as_scene_description)/urdf/kitting_bins.xacro" /> -->
+  <!-- <xacro:include filename="$(find o2as_scene_description)/urdf/kitting_tray_with_partitions.xacro" /> -->
   <xacro:include filename="$(find realsense2_camera)/urdf/_d435.urdf.xacro" />
   <!-- spawn and attach dual suction grippers -->
@@ -16,5 +16,5 @@
     <parent link="workspace_center" />
     <child  link="workspace_cam_holder_link" />
-    <origin xyz="-0.05 0 0.0" rpy="0.0 -${pi/2} 0.0" />
+    <origin xyz="0 0 0" rpy="0.0 -${pi/2} 0.0" />
   </joint>
   <xacro:sensor_d435 prefix="workspace_" parent="workspace_cam_holder_link">
@@ -23,5 +23,5 @@
   <!-- TODO: Deal with this camera? -->
   <!-- A row of tray -->
-  <xacro:property name="set3_x" value="${-.3}" />
+  <!-- <xacro:property name="set3_x" value="${-.3}" />
   <xacro:property name="set3_y" value="${0}" />
   <xacro:property name="set3_z" value=".00" />
@@ -31,4 +31,4 @@
   <xacro:kitting_tray2 trayname="set3_tray_2" parent="workspace_center">
     <origin xyz="${set3_x} ${set3_y-tray_width} ${set3_z}" rpy="0 0 0" />
-  </xacro:kitting_tray2>
+  </xacro:kitting_tray2> -->
 </robot>

Commit message: Modified kitting bins origins and trays positions.

File: o2as_scene_description/urdf/kitting_bins.xacro (robot description, xacro)
@@ -18,49 +18,49 @@
  <!-- A row of bin1 -->
  <xacro:property name="set1_x" value=".1675"/>
- <xacro:property name="set1_y" value="0.33"/>
- <xacro:property name="set1_z" value=".0"/>
+ <xacro:property name="set1_y" value="0.31"/>
+ <xacro:property name="set1_z" value="0"/>
  <!-- A row of bin2 -->
  <xacro:property name="set2_x" value=".376"/>
- <xacro:property name="set2_y" value="0.33"/>
- <xacro:property name="set2_z" value=".0"/>
+ <xacro:property name="set2_y" value="0.31"/>
+ <xacro:property name="set2_z" value="0"/>
  <!--set1_bin3_1_-->
   <xacro:kitting_bin_3 binname="set1_bin3_1" parent="workspace_center" z_origin_offset="-.004">
-      <origin xyz=".1675 0.234 0.004" rpy="0 0 0" />
+      <origin xyz=".1675 0.214 0.004" rpy="0 0 0" />
   </xacro:kitting_bin_3>
   <!--set1_bin2_1_-->
   <xacro:kitting_bin_2 binname="set1_bin2_1" parent="workspace_center" z_origin_offset="-.009">
-      <origin xyz=".1675 0.082 0.009" rpy="0 0 0" />
+      <origin xyz=".1675 0.062 0.009" rpy="0 0 0" />
   </xacro:kitting_bin_2>
   <!--set1_bin2_2_-->
   <xacro:kitting_bin_2 binname="set1_bin2_2" parent="workspace_center" z_origin_offset="-.009">
-      <origin xyz=".1675 -0.03 0.009" rpy="0 0 0" />
+      <origin xyz=".1675 -0.05 0.009" rpy="0 0 0" />
   </xacro:kitting_bin_2>
   <!--set1_bin2_3_-->
   <xacro:kitting_bin_2 binname="set1_bin2_3" parent="workspace_center" z_origin_offset="-.009">
-      <origin xyz=".1675 -0.142 0.009" rpy="0 0 0" />
+      <origin xyz=".1675 -0.162 0.009" rpy="0 0 0" />
   </xacro:kitting_bin_2>
   <!--set1_bin2_4_-->
   <xacro:kitting_bin_2 binname="set1_bin2_4" parent="workspace_center" z_origin_offset="-.009">
-      <origin xyz=".1675 -0.254 0.009" rpy="0 0 0" />
+      <origin xyz=".1675 -0.274 0.009" rpy="0 0 0" />
   </xacro:kitting_bin_2>
   <!--set2_bin1_1_-->
   <xacro:kitting_bin_1 binname="set2_bin1_1" parent="workspace_center" z_origin_offset="-.008">
-      <origin xyz=".376 0.2675 0.008" rpy="0 0 0" />
+      <origin xyz=".376 0.2475 0.008" rpy="0 0 0" />
   </xacro:kitting_bin_1>
   <!--set2_bin1_2_-->
   <xacro:kitting_bin_1 binname="set2_bin1_2" parent="workspace_center" z_origin_offset="-.008">
-      <origin xyz=".376 0.1425 0.008" rpy="0 0 0" />
+      <origin xyz=".376 0.1225 0.008" rpy="0 0 0" />
   </xacro:kitting_bin_1>
   <!--set2_bin1_3_-->
   <xacro:kitting_bin_1 binname="set2_bin1_3" parent="workspace_center" z_origin_offset="-.008">
-      <origin xyz=".376 0.0175 0.008" rpy="0 0 0" />
+      <origin xyz=".376 -0.0025 0.008" rpy="0 0 0" />
   </xacro:kitting_bin_1>
   <!--set2_bin1_4_-->
   <xacro:kitting_bin_1 binname="set2_bin1_4" parent="workspace_center" z_origin_offset="-.008">
-      <origin xyz=".376 -0.1075 0.008" rpy="0 0 0" />
+      <origin xyz=".376 -0.1275 0.008" rpy="0 0 0" />
   </xacro:kitting_bin_1>
   <!--set2_bin1_5_-->
   <xacro:kitting_bin_1 binname="set2_bin1_5" parent="workspace_center" z_origin_offset="-.008">
-      <origin xyz=".376 -0.2325 0.008" rpy="0 0 0" />
+      <origin xyz=".376 -0.2525 0.008" rpy="0 0 0" />
   </xacro:kitting_bin_1>
 </robot>

File: o2as_scene_description/urdf/kitting_scene.xacro (robot description, xacro)
@@ -5,8 +5,8 @@
   <xacro:include filename="$(find realsense2_camera)/urdf/_d435.urdf.xacro" />
   <!-- spawn and attach dual suction grippers -->
-  <!-- <xacro:include filename="$(find o2as_scene_description)/urdf/dual_suction_gripper.urdf.xacro" /> -->
-  <!-- <xacro:dual_suction_gripper_o2as prefix="b_bot_" parent = "b_bot_ee_link">
+  <xacro:include filename="$(find o2as_scene_description)/urdf/dual_suction_gripper.urdf.xacro" />
+  <xacro:dual_suction_gripper_o2as prefix="b_bot_" parent = "b_bot_ee_link">
     <origin xyz="0 0 0" rpy="0 0 0"/>
-  </xacro:dual_suction_gripper_o2as> -->
+  </xacro:dual_suction_gripper_o2as>
   <xacro:property name="tray_width" value=".300" />
   <xacro:property name="tray_length" value=".210" />
@@ -23,7 +23,7 @@
   <!-- TODO: Deal with this camera? -->
   <!-- A row of tray -->
-  <xacro:property name="set3_x" value="${-.3}" />
-  <xacro:property name="set3_y" value="${0}" />
-  <xacro:property name="set3_z" value=".00" />
+  <xacro:property name="set3_x" value="${-tray_length-.05}" />
+  <xacro:property name="set3_y" value="0" />
+  <xacro:property name="set3_z" value="0" />
   <xacro:kitting_tray1 trayname="set3_tray_1" parent="workspace_center">
     <origin xyz="${set3_x} ${set3_y} ${set3_z}" rpy="0 0 0" />

File: o2as_scene_description/urdf/o2as_base_scene.urdf.xacro (robot description, xacro)
@@ -105,5 +105,6 @@
   <!-- spawn and attach dual robotiq 85 grippers -->
   <xacro:include filename="$(find o2as_scene_description)/urdf/robotiq_85_gripper_with_ft300.urdf.xacro" />
-  <xacro:robotiq_85_gripper_o2as prefix="b_bot_" parent = "b_bot_ee_link" />
+  <!-- b_bot uses dual suction gripper for kitting task. -->
+  <!-- <xacro:robotiq_85_gripper_o2as prefix="b_bot_" parent = "b_bot_ee_link" /> -->
   <xacro:robotiq_85_gripper_o2as prefix="c_bot_" parent = "c_bot_ee_link"/>
   <!-- Add cameras -->

Commit message: Updated kitting layout for aist setting.

File: o2as_scene_description/urdf/kitting_bins.xacro (robot description, xacro)
@@ -24,24 +24,24 @@
  <xacro:property name="set2_y" value="0.31"/>
  <xacro:property name="set2_z" value="0"/>
- <!--set1_bin3_1_-->
-  <xacro:kitting_bin_3 binname="set1_bin3_1" parent="workspace_center" z_origin_offset="-.004">
-      <origin xyz=".1675 0.214 0.004" rpy="0 0 0" />
-  </xacro:kitting_bin_3>
-  <!--set1_bin2_1_-->
+ <!--set1_bin2_1_-->
   <xacro:kitting_bin_2 binname="set1_bin2_1" parent="workspace_center" z_origin_offset="-.009">
-      <origin xyz=".1675 0.062 0.009" rpy="0 0 0" />
+      <origin xyz=".1675 0.254 0.009" rpy="0 0 0" />
   </xacro:kitting_bin_2>
   <!--set1_bin2_2_-->
   <xacro:kitting_bin_2 binname="set1_bin2_2" parent="workspace_center" z_origin_offset="-.009">
-      <origin xyz=".1675 -0.05 0.009" rpy="0 0 0" />
+      <origin xyz=".1675 0.142 0.009" rpy="0 0 0" />
   </xacro:kitting_bin_2>
   <!--set1_bin2_3_-->
   <xacro:kitting_bin_2 binname="set1_bin2_3" parent="workspace_center" z_origin_offset="-.009">
-      <origin xyz=".1675 -0.162 0.009" rpy="0 0 0" />
+      <origin xyz=".1675 0.03 0.009" rpy="0 0 0" />
   </xacro:kitting_bin_2>
   <!--set1_bin2_4_-->
   <xacro:kitting_bin_2 binname="set1_bin2_4" parent="workspace_center" z_origin_offset="-.009">
-      <origin xyz=".1675 -0.274 0.009" rpy="0 0 0" />
+      <origin xyz=".1675 -0.082 0.009" rpy="0 0 0" />
   </xacro:kitting_bin_2>
+  <!--set1_bin3_1_-->
+  <xacro:kitting_bin_3 binname="set1_bin3_1" parent="workspace_center" z_origin_offset="-.004">
+      <origin xyz=".1675 -0.234 0.004" rpy="0 0 0" />
+  </xacro:kitting_bin_3>
   <!--set2_bin1_1_-->
   <xacro:kitting_bin_1 binname="set2_bin1_1" parent="workspace_center" z_origin_offset="-.008">
