Commit message: Add racks (to carry bins and trays) in kitting scene.
With fixed bin layout generator.

File: o2as_scene_description/urdf/kitting_bins.xacro (robot description, xacro)
@@ -2,5 +2,14 @@
 <robot xmlns:xacro="http://www.ros.org/wiki/xacro" name="kitting_scene">
   <xacro:include filename="$(find o2as_scene_description)/urdf/kitting_bin_macros.xacro" />
-  <xacro:property name="rack_width" value=".640" />
+  <xacro:include filename="$(find o2as_scene_description)/urdf/o2as_box.xacro"/>
+  <!-- add rack -->
+  <xacro:o2as_box boxname="rack_bins" box_w="0.42" box_l="0.680" box_h=".015" parent="workspace_center">
+    <origin xyz="0 -.32 0" rpy="0 0 0" />
+  </xacro:o2as_box>
+  <link name="rack_bins_center" />
+  <joint name="rack_bins_joint" type="fixed">
+    <parent link="workspace_center" />
+    <child link="rack_bins_center"/>
+  </joint>
  <!-- space for bin -->
  <!-- bin1_definition -->
@@ -18,49 +27,49 @@
  <!-- A row of bin1 -->
  <xacro:property name="set1_x" value=".1675"/>
- <xacro:property name="set1_y" value="0.31"/>
- <xacro:property name="set1_z" value="0"/>
+ <xacro:property name="set1_y" value="0.32"/>
+ <xacro:property name="set1_z" value="0.015"/>
  <!-- A row of bin2 -->
  <xacro:property name="set2_x" value=".376"/>
- <xacro:property name="set2_y" value="0.31"/>
- <xacro:property name="set2_z" value="0"/>
+ <xacro:property name="set2_y" value="0.32"/>
+ <xacro:property name="set2_z" value="0.015"/>
  <!--set1_bin2_1_-->
-  <xacro:kitting_bin_2 binname="set1_bin2_1" parent="workspace_center" z_origin_offset="-.009">
-      <origin xyz=".1675 0.254 0.009" rpy="0 0 0" />
+  <xacro:kitting_bin_2 binname="set1_bin2_1" parent="rack_bins_center" z_origin_offset="-.009">
+      <origin xyz=".1675 0.264 0.024" rpy="0 0 0" />
   </xacro:kitting_bin_2>
   <!--set1_bin2_2_-->
-  <xacro:kitting_bin_2 binname="set1_bin2_2" parent="workspace_center" z_origin_offset="-.009">
-      <origin xyz=".1675 0.142 0.009" rpy="0 0 0" />
+  <xacro:kitting_bin_2 binname="set1_bin2_2" parent="rack_bins_center" z_origin_offset="-.009">
+      <origin xyz=".1675 0.152 0.024" rpy="0 0 0" />
   </xacro:kitting_bin_2>
   <!--set1_bin2_3_-->
-  <xacro:kitting_bin_2 binname="set1_bin2_3" parent="workspace_center" z_origin_offset="-.009">
-      <origin xyz=".1675 0.03 0.009" rpy="0 0 0" />
+  <xacro:kitting_bin_2 binname="set1_bin2_3" parent="rack_bins_center" z_origin_offset="-.009">
+      <origin xyz=".1675 0.04 0.024" rpy="0 0 0" />
   </xacro:kitting_bin_2>
   <!--set1_bin2_4_-->
-  <xacro:kitting_bin_2 binname="set1_bin2_4" parent="workspace_center" z_origin_offset="-.009">
-      <origin xyz=".1675 -0.082 0.009" rpy="0 0 0" />
+  <xacro:kitting_bin_2 binname="set1_bin2_4" parent="rack_bins_center" z_origin_offset="-.009">
+      <origin xyz=".1675 -0.072 0.024" rpy="0 0 0" />
   </xacro:kitting_bin_2>
   <!--set1_bin3_1_-->
-  <xacro:kitting_bin_3 binname="set1_bin3_1" parent="workspace_center" z_origin_offset="-.004">
-      <origin xyz=".1675 -0.234 0.004" rpy="0 0 0" />
+  <xacro:kitting_bin_3 binname="set1_bin3_1" parent="rack_bins_center" z_origin_offset="-.004">
+      <origin xyz=".1675 -0.224 0.019" rpy="0 0 0" />
   </xacro:kitting_bin_3>
   <!--set2_bin1_1_-->
-  <xacro:kitting_bin_1 binname="set2_bin1_1" parent="workspace_center" z_origin_offset="-.008">
-      <origin xyz=".376 0.2475 0.008" rpy="0 0 0" />
+  <xacro:kitting_bin_1 binname="set2_bin1_1" parent="rack_bins_center" z_origin_offset="-.008">
+      <origin xyz=".376 0.2575 0.023" rpy="0 0 0" />
   </xacro:kitting_bin_1>
   <!--set2_bin1_2_-->
-  <xacro:kitting_bin_1 binname="set2_bin1_2" parent="workspace_center" z_origin_offset="-.008">
-      <origin xyz=".376 0.1225 0.008" rpy="0 0 0" />
+  <xacro:kitting_bin_1 binname="set2_bin1_2" parent="rack_bins_center" z_origin_offset="-.008">
+      <origin xyz=".376 0.1325 0.023" rpy="0 0 0" />
   </xacro:kitting_bin_1>
   <!--set2_bin1_3_-->
-  <xacro:kitting_bin_1 binname="set2_bin1_3" parent="workspace_center" z_origin_offset="-.008">
-      <origin xyz=".376 -0.0025 0.008" rpy="0 0 0" />
+  <xacro:kitting_bin_1 binname="set2_bin1_3" parent="rack_bins_center" z_origin_offset="-.008">
+      <origin xyz=".376 0.0075 0.023" rpy="0 0 0" />
   </xacro:kitting_bin_1>
   <!--set2_bin1_4_-->
-  <xacro:kitting_bin_1 binname="set2_bin1_4" parent="workspace_center" z_origin_offset="-.008">
-      <origin xyz=".376 -0.1275 0.008" rpy="0 0 0" />
+  <xacro:kitting_bin_1 binname="set2_bin1_4" parent="rack_bins_center" z_origin_offset="-.008">
+      <origin xyz=".376 -0.1175 0.023" rpy="0 0 0" />
   </xacro:kitting_bin_1>
   <!--set2_bin1_5_-->
-  <xacro:kitting_bin_1 binname="set2_bin1_5" parent="workspace_center" z_origin_offset="-.008">
-      <origin xyz=".376 -0.2525 0.008" rpy="0 0 0" />
+  <xacro:kitting_bin_1 binname="set2_bin1_5" parent="rack_bins_center" z_origin_offset="-.008">
+      <origin xyz=".376 -0.2425 0.023" rpy="0 0 0" />
   </xacro:kitting_bin_1>
 </robot>

File: o2as_scene_description/urdf/kitting_scene.xacro (robot description, xacro)
@@ -4,4 +4,5 @@
   <xacro:include filename="$(find o2as_scene_description)/urdf/kitting_tray_with_partitions.xacro" />
   <xacro:include filename="$(find realsense2_camera)/urdf/_d435.urdf.xacro" />
+  <xacro:include filename="$(find o2as_scene_description)/urdf/o2as_box.xacro"/>
   <!-- spawn and attach dual suction grippers -->
   <xacro:include filename="$(find o2as_scene_description)/urdf/dual_suction_gripper.urdf.xacro" />
@@ -22,12 +23,21 @@
   </xacro:sensor_d435>
   <!-- TODO: Deal with this camera? -->
-  <!-- A row of tray -->
+  <!-- add tray rack -->
+  <xacro:o2as_box boxname="rack_trays" box_w="0.21" box_l="0.60" box_h=".015" parent="workspace_center">
+    <origin xyz="-.26 -0.3 0" rpy="0 0 0" />
+  </xacro:o2as_box>
+  <link name="rack_trays_center" />
+  <joint name="rack_trays_joint" type="fixed">
+    <parent link="workspace_center" />
+    <child link="rack_trays_center"/>
+  </joint>
+  <!-- add trays -->
   <xacro:property name="set3_x" value="${-tray_length-.05}" />
   <xacro:property name="set3_y" value="0" />
-  <xacro:property name="set3_z" value="0" />
-  <xacro:kitting_tray1 trayname="set3_tray_1" parent="workspace_center">
+  <xacro:property name="set3_z" value="0.015" />
+  <xacro:kitting_tray1 trayname="set3_tray_1" parent="rack_trays_center">
     <origin xyz="${set3_x} ${set3_y} ${set3_z}" rpy="0 0 0" />
   </xacro:kitting_tray1>
-  <xacro:kitting_tray2 trayname="set3_tray_2" parent="workspace_center">
+  <xacro:kitting_tray2 trayname="set3_tray_2" parent="rack_trays_center">
     <origin xyz="${set3_x} ${set3_y-tray_width} ${set3_z}" rpy="0 0 0" />
   </xacro:kitting_tray2>

File: o2as_scene_description/urdf/templates/o2as_bin_template_front.xacro (robot description, xacro)
@@ -2,3 +2,12 @@
 <robot xmlns:xacro="http://www.ros.org/wiki/xacro" name="kitting_scene">
   <xacro:include filename="$(find o2as_scene_description)/urdf/kitting_bin_macros.xacro" />
-  <xacro:property name="rack_width" value=".640" />
+  <xacro:include filename="$(find o2as_scene_description)/urdf/o2as_box.xacro"/>
+  <!-- add rack -->
+  <xacro:o2as_box boxname="rack_bins" box_w="0.42" box_l="0.680" box_h=".015" parent="workspace_center">
+    <origin xyz="0 -.32 0" rpy="0 0 0" />
+  </xacro:o2as_box>
+  <link name="rack_bins_center" />
+  <joint name="rack_bins_joint" type="fixed">
+    <parent link="workspace_center" />
+    <child link="rack_bins_center"/>
+  </joint>

Commit message: WIP: add auxiliary frame to partition.

File: o2as_scene_description/urdf/kitting_bins.xacro (robot description, xacro)
@@ -2,5 +2,14 @@
 <robot xmlns:xacro="http://www.ros.org/wiki/xacro" name="kitting_scene">
   <xacro:include filename="$(find o2as_scene_description)/urdf/kitting_bin_macros.xacro" />
-  <xacro:property name="rack_width" value=".640" />
+  <xacro:include filename="$(find o2as_scene_description)/urdf/o2as_box.xacro"/>
+  <!-- add rack -->
+  <xacro:o2as_box boxname="rack_bins" box_w="0.42" box_l="0.680" box_h=".015" parent="workspace_center">
+    <origin xyz="0 -.32 0" rpy="0 0 0" />
+  </xacro:o2as_box>
+  <link name="rack_bins_center" />
+  <joint name="rack_bins_joint" type="fixed">
+    <parent link="workspace_center" />
+    <child link="rack_bins_center"/>
+  </joint>
  <!-- space for bin -->
  <!-- bin1_definition -->
@@ -17,50 +26,50 @@
  <xacro:property name="z_origin_offset_3" value="-.004" />
  <!-- A row of bin1 -->
- <xacro:property name="set1_x" value=".0"/>
- <xacro:property name="set1_y" value="0.33"/>
- <xacro:property name="set1_z" value=".01"/>
+ <xacro:property name="set1_x" value=".1675"/>
+ <xacro:property name="set1_y" value="0.32"/>
+ <xacro:property name="set1_z" value="0.015"/>
  <!-- A row of bin2 -->
- <xacro:property name="set2_x" value=".20"/>
- <xacro:property name="set2_y" value="0.33"/>
- <xacro:property name="set2_z" value=".00"/>
- <!--set1_bin1_1_-->
-  <xacro:kitting_bin_1 binname="set1_bin1_1" parent="workspace_center" z_origin_offset="-.008">
-      <origin xyz=".0 0.2675 0.018" rpy="0 0 0" />
+ <xacro:property name="set2_x" value=".376"/>
+ <xacro:property name="set2_y" value="0.32"/>
+ <xacro:property name="set2_z" value="0.015"/>
+ <!--set1_bin2_1_-->
+  <xacro:kitting_bin_2 binname="set1_bin2_1" parent="rack_bins_center" z_origin_offset="-.009">
+      <origin xyz=".1675 0.264 0.024" rpy="0 0 0" />
+  </xacro:kitting_bin_2>
+  <!--set1_bin2_2_-->
+  <xacro:kitting_bin_2 binname="set1_bin2_2" parent="rack_bins_center" z_origin_offset="-.009">
+      <origin xyz=".1675 0.152 0.024" rpy="0 0 0" />
+  </xacro:kitting_bin_2>
+  <!--set1_bin2_3_-->
+  <xacro:kitting_bin_2 binname="set1_bin2_3" parent="rack_bins_center" z_origin_offset="-.009">
+      <origin xyz=".1675 0.04 0.024" rpy="0 0 0" />
+  </xacro:kitting_bin_2>
+  <!--set1_bin2_4_-->
+  <xacro:kitting_bin_2 binname="set1_bin2_4" parent="rack_bins_center" z_origin_offset="-.009">
+      <origin xyz=".1675 -0.072 0.024" rpy="0 0 0" />
+  </xacro:kitting_bin_2>
+  <!--set1_bin3_1_-->
+  <xacro:kitting_bin_3 binname="set1_bin3_1" parent="rack_bins_center" z_origin_offset="-.004">
+      <origin xyz=".1675 -0.224 0.019" rpy="0 0 0" />
+  </xacro:kitting_bin_3>
+  <!--set2_bin1_1_-->
+  <xacro:kitting_bin_1 binname="set2_bin1_1" parent="rack_bins_center" z_origin_offset="-.008">
+      <origin xyz=".376 0.2575 0.023" rpy="0 0 0" />
   </xacro:kitting_bin_1>
-  <!--set1_bin1_2_-->
-  <xacro:kitting_bin_1 binname="set1_bin1_2" parent="workspace_center" z_origin_offset="-.008">
-      <origin xyz=".0 0.1425 0.018" rpy="0 0 0" />
+  <!--set2_bin1_2_-->
+  <xacro:kitting_bin_1 binname="set2_bin1_2" parent="rack_bins_center" z_origin_offset="-.008">
+      <origin xyz=".376 0.1325 0.023" rpy="0 0 0" />
   </xacro:kitting_bin_1>
-  <!--set1_bin1_3_-->
-  <xacro:kitting_bin_1 binname="set1_bin1_3" parent="workspace_center" z_origin_offset="-.008">
-      <origin xyz=".0 0.0175 0.018" rpy="0 0 0" />
+  <!--set2_bin1_3_-->
+  <xacro:kitting_bin_1 binname="set2_bin1_3" parent="rack_bins_center" z_origin_offset="-.008">
+      <origin xyz=".376 0.0075 0.023" rpy="0 0 0" />
   </xacro:kitting_bin_1>
-  <!--set1_bin1_4_-->
-  <xacro:kitting_bin_1 binname="set1_bin1_4" parent="workspace_center" z_origin_offset="-.008">
-      <origin xyz=".0 -0.1075 0.018" rpy="0 0 0" />
+  <!--set2_bin1_4_-->
+  <xacro:kitting_bin_1 binname="set2_bin1_4" parent="rack_bins_center" z_origin_offset="-.008">
+      <origin xyz=".376 -0.1175 0.023" rpy="0 0 0" />
   </xacro:kitting_bin_1>
-  <!--set1_bin1_5_-->
-  <xacro:kitting_bin_1 binname="set1_bin1_5" parent="workspace_center" z_origin_offset="-.008">
-      <origin xyz=".0 -0.2325 0.018" rpy="0 0 0" />
+  <!--set2_bin1_5_-->
+  <xacro:kitting_bin_1 binname="set2_bin1_5" parent="rack_bins_center" z_origin_offset="-.008">
+      <origin xyz=".376 -0.2425 0.023" rpy="0 0 0" />
   </xacro:kitting_bin_1>
-  <!--set2_bin2_1_-->
-  <xacro:kitting_bin_2 binname="set2_bin2_1" parent="workspace_center" z_origin_offset="-.009">
-      <origin xyz=".20 0.274 0.009" rpy="0 0 0" />
-  </xacro:kitting_bin_2>
-  <!--set2_bin2_2_-->
-  <xacro:kitting_bin_2 binname="set2_bin2_2" parent="workspace_center" z_origin_offset="-.009">
-      <origin xyz=".20 0.162 0.009" rpy="0 0 0" />
-  </xacro:kitting_bin_2>
-  <!--set2_bin2_3_-->
-  <xacro:kitting_bin_2 binname="set2_bin2_3" parent="workspace_center" z_origin_offset="-.009">
-      <origin xyz=".20 0.05 0.009" rpy="0 0 0" />
-  </xacro:kitting_bin_2>
-  <!--set2_bin2_4_-->
-  <xacro:kitting_bin_2 binname="set2_bin2_4" parent="workspace_center" z_origin_offset="-.009">
-      <origin xyz=".20 -0.062 0.009" rpy="0 0 0" />
-  </xacro:kitting_bin_2>
-  <!--set2_bin3_1_-->
-  <xacro:kitting_bin_3 binname="set2_bin3_1" parent="workspace_center" z_origin_offset="-.004">
-      <origin xyz=".20 -0.214 0.004" rpy="0 0 0" />
-  </xacro:kitting_bin_3>
 </robot>

File: o2as_scene_description/urdf/kitting_scene.xacro (robot description, xacro)
@@ -4,9 +4,10 @@
   <xacro:include filename="$(find o2as_scene_description)/urdf/kitting_tray_with_partitions.xacro" />
   <xacro:include filename="$(find realsense2_camera)/urdf/_d435.urdf.xacro" />
+  <xacro:include filename="$(find o2as_scene_description)/urdf/o2as_box.xacro"/>
   <!-- spawn and attach dual suction grippers -->
-  <!-- <xacro:include filename="$(find o2as_scene_description)/urdf/dual_suction_gripper.urdf.xacro" /> -->
-  <!-- <xacro:dual_suction_gripper_o2as prefix="b_bot_" parent = "b_bot_ee_link">
+  <xacro:include filename="$(find o2as_scene_description)/urdf/dual_suction_gripper.urdf.xacro" />
+  <xacro:dual_suction_gripper_o2as prefix="b_bot_" parent = "b_bot_ee_link">
     <origin xyz="0 0 0" rpy="0 0 0"/>
-  </xacro:dual_suction_gripper_o2as> -->
+  </xacro:dual_suction_gripper_o2as>
   <xacro:property name="tray_width" value=".300" />
   <xacro:property name="tray_length" value=".210" />
@@ -16,5 +17,5 @@
     <parent link="workspace_center" />
     <child  link="workspace_cam_holder_link" />
-    <origin xyz="-0.05 0 0.0" rpy="0.0 -${pi/2} 0.0" />
+    <origin xyz="0 0 0" rpy="0.0 -${pi/2} 0.0" />
   </joint>
   <xacro:sensor_d435 prefix="workspace_" parent="workspace_cam_holder_link">
@@ -22,12 +23,21 @@
   </xacro:sensor_d435>
   <!-- TODO: Deal with this camera? -->
-  <!-- A row of tray -->
-  <xacro:property name="set3_x" value="${-.3}" />
-  <xacro:property name="set3_y" value="${0}" />
-  <xacro:property name="set3_z" value=".00" />
-  <xacro:kitting_tray1 trayname="set3_tray_1" parent="workspace_center">
+  <!-- add tray rack -->
+  <xacro:o2as_box boxname="rack_trays" box_w="0.21" box_l="0.60" box_h=".015" parent="workspace_center">
+    <origin xyz="-.26 -0.3 0" rpy="0 0 0" />
+  </xacro:o2as_box>
+  <link name="rack_trays_center" />
+  <joint name="rack_trays_joint" type="fixed">
+    <parent link="workspace_center" />
+    <child link="rack_trays_center"/>
+  </joint>
+  <!-- add trays -->
+  <xacro:property name="set3_x" value="${-tray_length-.05}" />
+  <xacro:property name="set3_y" value="0" />
+  <xacro:property name="set3_z" value="0.015" />
+  <xacro:kitting_tray1 trayname="set3_tray_1" parent="rack_trays_center">
     <origin xyz="${set3_x} ${set3_y} ${set3_z}" rpy="0 0 0" />
   </xacro:kitting_tray1>
-  <xacro:kitting_tray2 trayname="set3_tray_2" parent="workspace_center">
+  <xacro:kitting_tray2 trayname="set3_tray_2" parent="rack_trays_center">
     <origin xyz="${set3_x} ${set3_y-tray_width} ${set3_z}" rpy="0 0 0" />
   </xacro:kitting_tray2>

File: o2as_scene_description/urdf/kitting_tray_with_partitions.xacro (robot description, xacro)
@@ -133,28 +133,28 @@
     </xacro:tray_contents>
     <!-- ========== The extra frames to place and pick items are defined below -->
-    <!-- <xacro:auxiliary_frame parent="${trayname}" framename="partition_1">
-      <origin rpy="0.0 0.0 0.0" xyz="0.04 0.16 0.02"/>
+    <xacro:auxiliary_frame parent="${trayname}" framename="partition_1">
+      <origin rpy="0.0 0.0 0.0" xyz="0.17 0.1375 0.02"/>
     </xacro:auxiliary_frame>
     <xacro:auxiliary_frame parent="${trayname}" framename="partition_2">
-      <origin rpy="0.0 0.0 0.0" xyz="0.11 0.13 0.02"/>
+      <origin rpy="0.0 0.0 0.0" xyz="0.105 0.1725 0.02"/>
     </xacro:auxiliary_frame>
     <xacro:auxiliary_frame parent="${trayname}" framename="partition_3">
-      <origin rpy="0.0 0.0 0.0" xyz="0.17 0.13 0.02"/>
+      <origin rpy="0.0 0.0 0.0" xyz="0.04 0.1725 0.02"/>
     </xacro:auxiliary_frame>
     <xacro:auxiliary_frame parent="${trayname}" framename="partition_4">
-      <origin rpy="0.0 0.0 0.0" xyz="0.11 0.19 0.02"/>
+      <origin rpy="0.0 0.0 0.0" xyz="0.105 0.1125 0.02"/>
     </xacro:auxiliary_frame>
     <xacro:auxiliary_frame parent="${trayname}" framename="partition_5">
-      <origin rpy="0.0 0.0 0.0" xyz="0.17 0.19 0.02"/>
+      <origin rpy="0.0 0.0 0.0" xyz="0.04 0.1125 0.02"/>
     </xacro:auxiliary_frame>
     <xacro:auxiliary_frame parent="${trayname}" framename="partition_6">
-      <origin rpy="0.0 0.0 0.0" xyz="0.04 0.25 0.02"/>
+      <origin rpy="0.0 0.0 0.0" xyz="0.17 0.0525 0.02"/>
     </xacro:auxiliary_frame>
     <xacro:auxiliary_frame parent="${trayname}" framename="partition_7">
-      <origin rpy="0.0 0.0 0.0" xyz="0.11 0.25 0.02"/>
+      <origin rpy="0.0 0.0 0.0" xyz="0.105 0.0525 0.02"/>
     </xacro:auxiliary_frame>
     <xacro:auxiliary_frame parent="${trayname}" framename="partition_8">
-      <origin rpy="0.0 0.0 0.0" xyz="0.17 0.25 0.02"/>
-    </xacro:auxiliary_frame> -->
+      <origin rpy="0.0 0.0 0.0" xyz="0.04 0.0525 0.02"/>
+    </xacro:auxiliary_frame>
     <!-- TODO: Insert the rest and fine tune -->
     <!-- <xacro:property name="m4_x_0" value="0.18"/>

Commit message: Add check point for pick-and-place.

File: o2as_scene_description/urdf/kitting_bins.xacro (robot description, xacro)
@@ -11,4 +11,5 @@
     <parent link="workspace_center" />
     <child link="rack_bins_center"/>
+    <origin xyz=".21 0 0.015" rpy="0 0 0"/>
   </joint>
  <!-- space for bin -->
@@ -34,41 +35,41 @@
  <xacro:property name="set2_z" value="0.015"/>
  <!--set1_bin2_1_-->
-  <xacro:kitting_bin_2 binname="set1_bin2_1" parent="rack_bins_center" z_origin_offset="-.009">
+  <xacro:kitting_bin_2 binname="set1_bin2_1" parent="workspace_center" z_origin_offset="-.009">
       <origin xyz=".1675 0.264 0.024" rpy="0 0 0" />
   </xacro:kitting_bin_2>
   <!--set1_bin2_2_-->
-  <xacro:kitting_bin_2 binname="set1_bin2_2" parent="rack_bins_center" z_origin_offset="-.009">
+  <xacro:kitting_bin_2 binname="set1_bin2_2" parent="workspace_center" z_origin_offset="-.009">
       <origin xyz=".1675 0.152 0.024" rpy="0 0 0" />
   </xacro:kitting_bin_2>
   <!--set1_bin2_3_-->
-  <xacro:kitting_bin_2 binname="set1_bin2_3" parent="rack_bins_center" z_origin_offset="-.009">
+  <xacro:kitting_bin_2 binname="set1_bin2_3" parent="workspace_center" z_origin_offset="-.009">
       <origin xyz=".1675 0.04 0.024" rpy="0 0 0" />
   </xacro:kitting_bin_2>
   <!--set1_bin2_4_-->
-  <xacro:kitting_bin_2 binname="set1_bin2_4" parent="rack_bins_center" z_origin_offset="-.009">
+  <xacro:kitting_bin_2 binname="set1_bin2_4" parent="workspace_center" z_origin_offset="-.009">
       <origin xyz=".1675 -0.072 0.024" rpy="0 0 0" />
   </xacro:kitting_bin_2>
   <!--set1_bin3_1_-->
-  <xacro:kitting_bin_3 binname="set1_bin3_1" parent="rack_bins_center" z_origin_offset="-.004">
+  <xacro:kitting_bin_3 binname="set1_bin3_1" parent="workspace_center" z_origin_offset="-.004">
       <origin xyz=".1675 -0.224 0.019" rpy="0 0 0" />
   </xacro:kitting_bin_3>
   <!--set2_bin1_1_-->
-  <xacro:kitting_bin_1 binname="set2_bin1_1" parent="rack_bins_center" z_origin_offset="-.008">
+  <xacro:kitting_bin_1 binname="set2_bin1_1" parent="workspace_center" z_origin_offset="-.008">
       <origin xyz=".376 0.2575 0.023" rpy="0 0 0" />
   </xacro:kitting_bin_1>
   <!--set2_bin1_2_-->
-  <xacro:kitting_bin_1 binname="set2_bin1_2" parent="rack_bins_center" z_origin_offset="-.008">
+  <xacro:kitting_bin_1 binname="set2_bin1_2" parent="workspace_center" z_origin_offset="-.008">
       <origin xyz=".376 0.1325 0.023" rpy="0 0 0" />
   </xacro:kitting_bin_1>
   <!--set2_bin1_3_-->
-  <xacro:kitting_bin_1 binname="set2_bin1_3" parent="rack_bins_center" z_origin_offset="-.008">
+  <xacro:kitting_bin_1 binname="set2_bin1_3" parent="workspace_center" z_origin_offset="-.008">
       <origin xyz=".376 0.0075 0.023" rpy="0 0 0" />
   </xacro:kitting_bin_1>
   <!--set2_bin1_4_-->
-  <xacro:kitting_bin_1 binname="set2_bin1_4" parent="rack_bins_center" z_origin_offset="-.008">
+  <xacro:kitting_bin_1 binname="set2_bin1_4" parent="workspace_center" z_origin_offset="-.008">
       <origin xyz=".376 -0.1175 0.023" rpy="0 0 0" />
   </xacro:kitting_bin_1>
   <!--set2_bin1_5_-->
-  <xacro:kitting_bin_1 binname="set2_bin1_5" parent="rack_bins_center" z_origin_offset="-.008">
+  <xacro:kitting_bin_1 binname="set2_bin1_5" parent="workspace_center" z_origin_offset="-.008">
       <origin xyz=".376 -0.2425 0.023" rpy="0 0 0" />
   </xacro:kitting_bin_1>

File: o2as_scene_description/urdf/kitting_scene.xacro (robot description, xacro)
@@ -31,4 +31,5 @@
     <parent link="workspace_center" />
     <child link="rack_trays_center"/>
+    <origin xyz="-.13 0 0.015" rpy="0 0 0"/>
   </joint>
   <!-- add trays -->
@@ -36,8 +37,8 @@
   <xacro:property name="set3_y" value="0" />
   <xacro:property name="set3_z" value="0.015" />
-  <xacro:kitting_tray1 trayname="set3_tray_1" parent="rack_trays_center">
+  <xacro:kitting_tray1 trayname="set3_tray_1" parent="workspace_center">
     <origin xyz="${set3_x} ${set3_y} ${set3_z}" rpy="0 0 0" />
   </xacro:kitting_tray1>
-  <xacro:kitting_tray2 trayname="set3_tray_2" parent="rack_trays_center">
+  <xacro:kitting_tray2 trayname="set3_tray_2" parent="workspace_center">
     <origin xyz="${set3_x} ${set3_y-tray_width} ${set3_z}" rpy="0 0 0" />
   </xacro:kitting_tray2>

File: o2as_scene_description/urdf/templates/o2as_bin_template_front.xacro (robot description, xacro)
@@ -11,3 +11,4 @@
     <parent link="workspace_center" />
     <child link="rack_bins_center"/>
+    <origin xyz=".21 0 0.015" rpy="0 0 0"/>
   </joint>
