Commit message: WIP: various fixed
For picking using suction and graspability estimation.

File: o2as_scene_description/urdf/kitting_bins.xacro (robot description, xacro)
@@ -27,50 +27,50 @@
  <xacro:property name="z_origin_offset_3" value="-.004" />
  <!-- A row of bin1 -->
- <xacro:property name="set1_x" value=".1675"/>
- <xacro:property name="set1_y" value="0.32"/>
+ <xacro:property name="set1_x" value=".135"/>
+ <xacro:property name="set1_y" value="0.285"/>
  <xacro:property name="set1_z" value="0.015"/>
  <!-- A row of bin2 -->
- <xacro:property name="set2_x" value=".376"/>
- <xacro:property name="set2_y" value="0.32"/>
+ <xacro:property name="set2_x" value=".35"/>
+ <xacro:property name="set2_y" value="0.285"/>
  <xacro:property name="set2_z" value="0.015"/>
  <!--set1_bin2_1_-->
   <xacro:kitting_bin_2 binname="set1_bin2_1" parent="workspace_center" z_origin_offset="-.009">
-      <origin xyz=".1675 0.264 0.024" rpy="0 0 0" />
+      <origin xyz=".135 0.229 0.024" rpy="0 0 0" />
   </xacro:kitting_bin_2>
   <!--set1_bin2_2_-->
   <xacro:kitting_bin_2 binname="set1_bin2_2" parent="workspace_center" z_origin_offset="-.009">
-      <origin xyz=".1675 0.152 0.024" rpy="0 0 0" />
+      <origin xyz=".135 0.117 0.024" rpy="0 0 0" />
   </xacro:kitting_bin_2>
   <!--set1_bin2_3_-->
   <xacro:kitting_bin_2 binname="set1_bin2_3" parent="workspace_center" z_origin_offset="-.009">
-      <origin xyz=".1675 0.04 0.024" rpy="0 0 0" />
+      <origin xyz=".135 0.005 0.024" rpy="0 0 0" />
   </xacro:kitting_bin_2>
   <!--set1_bin2_4_-->
   <xacro:kitting_bin_2 binname="set1_bin2_4" parent="workspace_center" z_origin_offset="-.009">
-      <origin xyz=".1675 -0.072 0.024" rpy="0 0 0" />
+      <origin xyz=".135 -0.107 0.024" rpy="0 0 0" />
   </xacro:kitting_bin_2>
   <!--set1_bin3_1_-->
   <xacro:kitting_bin_3 binname="set1_bin3_1" parent="workspace_center" z_origin_offset="-.004">
-      <origin xyz=".1675 -0.224 0.019" rpy="0 0 0" />
+      <origin xyz=".135 -0.259 0.019" rpy="0 0 0" />
   </xacro:kitting_bin_3>
   <!--set2_bin1_1_-->
   <xacro:kitting_bin_1 binname="set2_bin1_1" parent="workspace_center" z_origin_offset="-.008">
-      <origin xyz=".376 0.2575 0.023" rpy="0 0 0" />
+      <origin xyz=".35 0.2225 0.023" rpy="0 0 0" />
   </xacro:kitting_bin_1>
   <!--set2_bin1_2_-->
   <xacro:kitting_bin_1 binname="set2_bin1_2" parent="workspace_center" z_origin_offset="-.008">
-      <origin xyz=".376 0.1325 0.023" rpy="0 0 0" />
+      <origin xyz=".35 0.0975 0.023" rpy="0 0 0" />
   </xacro:kitting_bin_1>
   <!--set2_bin1_3_-->
   <xacro:kitting_bin_1 binname="set2_bin1_3" parent="workspace_center" z_origin_offset="-.008">
-      <origin xyz=".376 0.0075 0.023" rpy="0 0 0" />
+      <origin xyz=".35 -0.0275 0.023" rpy="0 0 0" />
   </xacro:kitting_bin_1>
   <!--set2_bin1_4_-->
   <xacro:kitting_bin_1 binname="set2_bin1_4" parent="workspace_center" z_origin_offset="-.008">
-      <origin xyz=".376 -0.1175 0.023" rpy="0 0 0" />
+      <origin xyz=".35 -0.1525 0.023" rpy="0 0 0" />
   </xacro:kitting_bin_1>
   <!--set2_bin1_5_-->
   <xacro:kitting_bin_1 binname="set2_bin1_5" parent="workspace_center" z_origin_offset="-.008">
-      <origin xyz=".376 -0.2425 0.023" rpy="0 0 0" />
+      <origin xyz=".35 -0.2775 0.023" rpy="0 0 0" />
   </xacro:kitting_bin_1>
 </robot>

File: o2as_scene_description/urdf/o2as_base_scene.urdf.xacro (robot description, xacro)
@@ -1,12 +1,14 @@
 <?xml version="1.0"?>
-<robot xmlns:xacro="http://ros.org/wiki/xacro"
+<robot xmlns:xacro="http://www.ros.org/wiki/xacro"
        name="o2as_base_scene" >
   <!-- Calibration from 20 August 2018 -->
   <!-- Calibration help: If the robot is not moving far enough to the calibration point, increase these distances -->
-  <xacro:property name="a_bot_x" value="-0.00"/>
-  <xacro:property name="a_bot_y" value="-0.45"/>
-  <xacro:property name="b_bot_x" value="0.00"/>
-  <xacro:property name="b_bot_y" value="0.55"/>
-  <xacro:property name="c_bot_x" value="-0.5"/>
+  <xacro:property name="a_bot_x" value="-0.01"/>
+  <xacro:property name="a_bot_y" value="-0.5"/>
+  <xacro:property name="b_bot_x" value="-0.009"/>
+  <xacro:property name="b_bot_y" value="0.503"/>
+  <xacro:property name="b_bot_theta" value="-3.12832815"/>
+  <!-- The above is 0.76 degrees away from pi (Sep 17; not perfect) -->
+  <xacro:property name="c_bot_x" value="-0.499"/>
   <xacro:property name="c_bot_y" value="0.0"/>
   <xacro:property name="bots_z" value="0.75"/>
@@ -28,19 +30,24 @@
   <xacro:include filename="$(find o2as_scene_description)/urdf/o2as_base.xacro" />
   <xacro:o2as_base boxname="a_bot_base_smfl" parent="o2as_ground">
-    <origin xyz="${a_bot_x-.65/2} ${a_bot_y-.65/2} 0.65" rpy="0 0 0" />
+    <origin xyz="${a_bot_x-.65/2} ${a_bot_y-.65/2} 0.69" rpy="0 0 0" />
   </xacro:o2as_base>
   <xacro:o2as_base boxname="b_bot_base_smfl" parent="o2as_ground">
-    <origin xyz="${b_bot_x-.65/2} ${b_bot_y-.65/2} 0.65" rpy="0 0 0" />
+    <origin xyz="${b_bot_x-.65/2} ${b_bot_y-.65/2} 0.69" rpy="0 0 0" />
   </xacro:o2as_base>
   <xacro:o2as_base boxname="c_bot_base_smfl" parent="o2as_ground">
-    <origin xyz="${c_bot_x-.65/2-.22} ${c_bot_y-.65/2-.22} 0.65" rpy="0 0 0" />
+    <origin xyz="${c_bot_x-.65/2-.165} ${c_bot_y-.65/2-.095} 0.69" rpy="0 0 0" />
   </xacro:o2as_base>
   <!-- Main workspace -->
   <!-- The surface is 0.01 m below the robot bases and the "workspace_center" frame. -->
   <xacro:include filename="$(find o2as_scene_description)/urdf/o2as_box.xacro" />
-  <xacro:property name="plate_w" value="0.84"/>
-  <xacro:property name="plate_l" value="0.62"/>
-  <xacro:o2as_box boxname="workbox" box_w="${plate_w}" box_l="${plate_l}" box_h=".01" parent="o2as_ground">
-    <origin xyz="${-plate_w/2} ${-plate_l/2} ${bots_z}" rpy="0 0 0" />
+  <xacro:property name="plate_w" value="0.9"/>
+  <xacro:property name="plate_l" value="0.75"/>
+  <xacro:property name="plate_cut_w" value="0.03"/>
+  <xacro:property name="plate_cut_l" value="0.14"/>
+  <xacro:o2as_box boxname="workbox1" box_w="${plate_w}" box_l="${plate_l-plate_cut_l}" box_h=".01" parent="o2as_ground">
+    <origin xyz="${-plate_w/2 +.08} ${-(plate_l/2)} ${bots_z}" rpy="0 0 0" />
+  </xacro:o2as_box>
+  <xacro:o2as_box boxname="workbox2" box_w="${plate_w-plate_cut_w}" box_l="${plate_cut_l}" box_h=".01" parent="o2as_ground">
+    <origin xyz="${-plate_w/2 +.08+0.03} ${-plate_l/2+plate_l-plate_cut_l} ${bots_z}" rpy="0 0 0" />
   </xacro:o2as_box>
   <link name="workspace_center" />
@@ -68,5 +75,5 @@
     wrist_2_lower_limit="${-pi}" wrist_2_upper_limit="${pi}"
     wrist_3_lower_limit="${-pi}" wrist_3_upper_limit="${pi}"/>
-  <xacro:ur5_robot prefix="b_bot_" joint_limited="true"
+  <xacro:ur5_robot prefix="b_bot_" joint_limited="false"
     shoulder_pan_lower_limit="${-pi}" shoulder_pan_upper_limit="${pi}"
     shoulder_lift_lower_limit="${-pi}" shoulder_lift_upper_limit="${pi}"
@@ -91,5 +98,5 @@
     <parent link="o2as_ground" />
     <child link = "b_bot_base_link" />
-    <origin xyz="${b_bot_x} ${b_bot_y} ${bots_z}" rpy="0.0 0.0 ${-pi}" />
+    <origin xyz="${b_bot_x} ${b_bot_y} ${bots_z}" rpy="0.0 0.0 ${b_bot_theta}" />
   </joint>
   <joint name="world_c_bot_joint" type="fixed">
@@ -105,16 +112,15 @@
   <!-- spawn and attach dual robotiq 85 grippers -->
   <xacro:include filename="$(find o2as_scene_description)/urdf/robotiq_85_gripper_with_ft300.urdf.xacro" />
-  <!-- b_bot uses dual suction gripper for kitting task. -->
   <!-- <xacro:robotiq_85_gripper_o2as prefix="b_bot_" parent = "b_bot_ee_link" /> -->
   <xacro:robotiq_85_gripper_o2as prefix="c_bot_" parent = "c_bot_ee_link"/>
   <!-- Add cameras -->
   <xacro:include filename="$(find o2as_realsense2_camera)/urdf/_d435.urdf.xacro" />
-  <link name="b_bot_cam_holder_link" />
-  <joint name="b_bot_cam_holder_joint" type="fixed">
-    <parent link="b_bot_wrist_2_link" />
-    <child  link="b_bot_cam_holder_link" />
-    <origin xyz="0.0 -0.06 0.16" rpy="0.0 0.0 ${pi/2}" />
+  <link name="c_bot_cam_holder_link" />
+  <joint name="c_bot_cam_holder_joint" type="fixed">
+    <parent link="c_bot_wrist_2_link" />
+    <child  link="c_bot_cam_holder_link" />
+    <origin xyz="0.0 -0.06 ${0.09465 + .13}" rpy="0.0 0.0 ${pi/2}" />
   </joint>
-  <xacro:sensor_d435 prefix="b_bot_" parent="b_bot_cam_holder_link">
+  <xacro:sensor_d435 prefix="c_bot_" parent="c_bot_cam_holder_link">
     <origin xyz="0 0 0" rpy="0 0 0"/>
   </xacro:sensor_d435>
@@ -123,5 +129,5 @@
   </xacro:sensor_d435> -->
   <!-- spawn and attach AR markers -->
-  <xacro:include filename="$(find o2as_gazebo)/urdf/o2as_ar_marker.urdf.xacro"/>
+  <!-- <xacro:include filename="$(find o2as_gazebo)/urdf/o2as_ar_marker.urdf.xacro"/>
   <xacro:o2as_ar_marker prefix="a_bot_" parent="a_bot_wrist_3_link"
    marker_id="17">
@@ -135,9 +141,12 @@
    marker_id="256">
     <origin xyz="0.0 0.12 0.05" rpy="0 0 ${pi/2}"/>
-  </xacro:o2as_ar_marker>
+  </xacro:o2as_ar_marker> -->
   <!-- Add PhoXi 3D scanners -->
   <xacro:include filename="$(find o2as_scene_description)/urdf/phoxi_m_camera.urdf.xacro" />
   <xacro:phoxi_m_camera prefix="a_" parent="o2as_ground">
-    <origin xyz="0.61696890577  0.17103542533 1.42309125675" rpy="-2.626594398897875 0.2001733992896885 1.5970042364211503"/>
+    <!-- osx phoxi setting (maybe) -->
+    <!-- <origin xyz="0.46 0 ${bots_z + .1 + .8}" rpy="${-160*pi/180} 0 ${pi/2}"/> -->
+    <!-- aist phoxi setting  -->
+    <origin xyz="0.616968905765895 0.171035425329841 1.423091256751067" rpy="-2.626594398897875 0.2001733992896885 1.5970042364211503"/>
   </xacro:phoxi_m_camera>
   <!-- I would like to remove the "world" link definition, but apparently it is necessary for Gazebo -->

Commit message: WIP: integrate graspability estimation for test.

File: o2as_scene_description/urdf/kitting_bins.xacro (robot description, xacro)
@@ -31,5 +31,5 @@
  <xacro:property name="set1_z" value="0.015"/>
  <!-- A row of bin2 -->
- <xacro:property name="set2_x" value=".35"/>
+ <xacro:property name="set2_x" value=".345"/>
  <xacro:property name="set2_y" value="0.285"/>
  <xacro:property name="set2_z" value="0.015"/>
@@ -56,21 +56,21 @@
   <!--set2_bin1_1_-->
   <xacro:kitting_bin_1 binname="set2_bin1_1" parent="workspace_center" z_origin_offset="-.008">
-      <origin xyz=".35 0.2225 0.023" rpy="0 0 0" />
+      <origin xyz=".345 0.2225 0.023" rpy="0 0 0" />
   </xacro:kitting_bin_1>
   <!--set2_bin1_2_-->
   <xacro:kitting_bin_1 binname="set2_bin1_2" parent="workspace_center" z_origin_offset="-.008">
-      <origin xyz=".35 0.0975 0.023" rpy="0 0 0" />
+      <origin xyz=".345 0.0975 0.023" rpy="0 0 0" />
   </xacro:kitting_bin_1>
   <!--set2_bin1_3_-->
   <xacro:kitting_bin_1 binname="set2_bin1_3" parent="workspace_center" z_origin_offset="-.008">
-      <origin xyz=".35 -0.0275 0.023" rpy="0 0 0" />
+      <origin xyz=".345 -0.0275 0.023" rpy="0 0 0" />
   </xacro:kitting_bin_1>
   <!--set2_bin1_4_-->
   <xacro:kitting_bin_1 binname="set2_bin1_4" parent="workspace_center" z_origin_offset="-.008">
-      <origin xyz=".35 -0.1525 0.023" rpy="0 0 0" />
+      <origin xyz=".345 -0.1525 0.023" rpy="0 0 0" />
   </xacro:kitting_bin_1>
   <!--set2_bin1_5_-->
   <xacro:kitting_bin_1 binname="set2_bin1_5" parent="workspace_center" z_origin_offset="-.008">
-      <origin xyz=".35 -0.2775 0.023" rpy="0 0 0" />
+      <origin xyz=".345 -0.2775 0.023" rpy="0 0 0" />
   </xacro:kitting_bin_1>
 </robot>

File: o2as_scene_description/urdf/o2as_osaka_scene.urdf.xacro (robot description, xacro)
@@ -103,8 +103,8 @@
   </joint>
   <!-- spawn and attach grippers -->
-  <xacro:include filename="$(find o2as_scene_description)/urdf/precision_gripper.xacro" />
+  <!-- <xacro:include filename="$(find o2as_scene_description)/urdf/precision_gripper.xacro" />
   <xacro:precision_gripper prefix="a_bot_"  grippername = "gripper" parent = "a_bot_tool0">
     <origin xyz="0.0 0 0.04" rpy="0 ${pi/2} 0"/>
-  </xacro:precision_gripper>
+  </xacro:precision_gripper> -->
   <xacro:include filename="$(find o2as_scene_description)/urdf/robotiq_85_gripper_with_ft300.urdf.xacro" />
   <xacro:robotiq_85_gripper_o2as prefix="b_bot_" parent = "b_bot_ee_link" />

Commit message: Add debug real robot and real scene for aist.

File: o2as_scene_description/urdf/kitting_bins.xacro (robot description, xacro)
@@ -28,49 +28,49 @@
  <!-- A row of bin1 -->
  <xacro:property name="set1_x" value=".135"/>
- <xacro:property name="set1_y" value="0.285"/>
+ <xacro:property name="set1_y" value="0.28"/>
  <xacro:property name="set1_z" value="0.015"/>
  <!-- A row of bin2 -->
  <xacro:property name="set2_x" value=".345"/>
- <xacro:property name="set2_y" value="0.285"/>
+ <xacro:property name="set2_y" value="0.28"/>
  <xacro:property name="set2_z" value="0.015"/>
  <!--set1_bin2_1_-->
   <xacro:kitting_bin_2 binname="set1_bin2_1" parent="workspace_center" z_origin_offset="-.009">
-      <origin xyz=".135 0.229 0.024" rpy="0 0 0" />
+      <origin xyz=".135 0.224 0.024" rpy="0 0 0" />
   </xacro:kitting_bin_2>
   <!--set1_bin2_2_-->
   <xacro:kitting_bin_2 binname="set1_bin2_2" parent="workspace_center" z_origin_offset="-.009">
-      <origin xyz=".135 0.117 0.024" rpy="0 0 0" />
+      <origin xyz=".135 0.112 0.024" rpy="0 0 0" />
   </xacro:kitting_bin_2>
   <!--set1_bin2_3_-->
   <xacro:kitting_bin_2 binname="set1_bin2_3" parent="workspace_center" z_origin_offset="-.009">
-      <origin xyz=".135 0.005 0.024" rpy="0 0 0" />
+      <origin xyz=".135 4.16333634234e-17 0.024" rpy="0 0 0" />
   </xacro:kitting_bin_2>
   <!--set1_bin2_4_-->
   <xacro:kitting_bin_2 binname="set1_bin2_4" parent="workspace_center" z_origin_offset="-.009">
-      <origin xyz=".135 -0.107 0.024" rpy="0 0 0" />
+      <origin xyz=".135 -0.112 0.024" rpy="0 0 0" />
   </xacro:kitting_bin_2>
   <!--set1_bin3_1_-->
   <xacro:kitting_bin_3 binname="set1_bin3_1" parent="workspace_center" z_origin_offset="-.004">
-      <origin xyz=".135 -0.259 0.019" rpy="0 0 0" />
+      <origin xyz=".135 -0.264 0.019" rpy="0 0 0" />
   </xacro:kitting_bin_3>
   <!--set2_bin1_1_-->
   <xacro:kitting_bin_1 binname="set2_bin1_1" parent="workspace_center" z_origin_offset="-.008">
-      <origin xyz=".345 0.2225 0.023" rpy="0 0 0" />
+      <origin xyz=".345 0.2175 0.023" rpy="0 0 0" />
   </xacro:kitting_bin_1>
   <!--set2_bin1_2_-->
   <xacro:kitting_bin_1 binname="set2_bin1_2" parent="workspace_center" z_origin_offset="-.008">
-      <origin xyz=".345 0.0975 0.023" rpy="0 0 0" />
+      <origin xyz=".345 0.0925 0.023" rpy="0 0 0" />
   </xacro:kitting_bin_1>
   <!--set2_bin1_3_-->
   <xacro:kitting_bin_1 binname="set2_bin1_3" parent="workspace_center" z_origin_offset="-.008">
-      <origin xyz=".345 -0.0275 0.023" rpy="0 0 0" />
+      <origin xyz=".345 -0.0325 0.023" rpy="0 0 0" />
   </xacro:kitting_bin_1>
   <!--set2_bin1_4_-->
   <xacro:kitting_bin_1 binname="set2_bin1_4" parent="workspace_center" z_origin_offset="-.008">
-      <origin xyz=".345 -0.1525 0.023" rpy="0 0 0" />
+      <origin xyz=".345 -0.1575 0.023" rpy="0 0 0" />
   </xacro:kitting_bin_1>
   <!--set2_bin1_5_-->
   <xacro:kitting_bin_1 binname="set2_bin1_5" parent="workspace_center" z_origin_offset="-.008">
-      <origin xyz=".345 -0.2775 0.023" rpy="0 0 0" />
+      <origin xyz=".345 -0.2825 0.023" rpy="0 0 0" />
   </xacro:kitting_bin_1>
 </robot>

File: o2as_scene_description/urdf/o2as_base_scene.urdf.xacro (robot description, xacro)
@@ -23,6 +23,6 @@
   <!-- Scene items (trays, bins...) -->
   <!-- <xacro:include filename="$(find o2as_scene_description)/urdf/taskboard_scene.xacro" /> -->
-  <!-- <xacro:include filename="$(find o2as_scene_description)/urdf/kitting_scene.xacro" /> -->
-  <xacro:include filename="$(find o2as_scene_description)/urdf/assembly_scene.xacro" />
+  <xacro:include filename="$(find o2as_scene_description)/urdf/kitting_scene.xacro" />
+  <!-- <xacro:include filename="$(find o2as_scene_description)/urdf/assembly_scene.xacro" /> -->
   <!-- Robot bases -->
   <!-- Putting these at height 0.0 makes them intersect with the ground, so they are elevated. -->
@@ -149,5 +149,5 @@
     <!-- <origin xyz="0.46 0 ${bots_z + .1 + .8}" rpy="${-160*pi/180} 0 ${pi/2}"/> -->
     <!-- aist phoxi setting  -->
-    <origin xyz="0.616968905765895 0.171035425329841 1.423091256751067" rpy="-2.626594398897875 0.2001733992896885 1.5970042364211503"/>
+    <origin xyz="0.616968905765895 0.121035425329841 1.423091256751067" rpy="-2.626594398897875 0.2001733992896885 1.5970042364211503"/>
   </xacro:phoxi_m_camera>
   <!-- I would like to remove the "world" link definition, but apparently it is necessary for Gazebo -->

Commit message: WIP: fix picking point error.

File: o2as_scene_description/urdf/kitting_bins.xacro (robot description, xacro)
@@ -27,50 +27,50 @@
  <xacro:property name="z_origin_offset_3" value="-.004" />
  <!-- A row of bin1 -->
- <xacro:property name="set1_x" value=".135"/>
- <xacro:property name="set1_y" value="0.28"/>
+ <xacro:property name="set1_x" value=".1425"/>
+ <xacro:property name="set1_y" value="0.245"/>
  <xacro:property name="set1_z" value="0.015"/>
  <!-- A row of bin2 -->
- <xacro:property name="set2_x" value=".345"/>
- <xacro:property name="set2_y" value="0.28"/>
+ <xacro:property name="set2_x" value=".349"/>
+ <xacro:property name="set2_y" value="0.245"/>
  <xacro:property name="set2_z" value="0.015"/>
  <!--set1_bin2_1_-->
   <xacro:kitting_bin_2 binname="set1_bin2_1" parent="workspace_center" z_origin_offset="-.009">
-      <origin xyz=".135 0.224 0.024" rpy="0 0 0" />
+      <origin xyz=".1425 0.189 0.024" rpy="0 0 0" />
   </xacro:kitting_bin_2>
   <!--set1_bin2_2_-->
   <xacro:kitting_bin_2 binname="set1_bin2_2" parent="workspace_center" z_origin_offset="-.009">
-      <origin xyz=".135 0.112 0.024" rpy="0 0 0" />
+      <origin xyz=".1425 0.077 0.024" rpy="0 0 0" />
   </xacro:kitting_bin_2>
   <!--set1_bin2_3_-->
   <xacro:kitting_bin_2 binname="set1_bin2_3" parent="workspace_center" z_origin_offset="-.009">
-      <origin xyz=".135 4.16333634234e-17 0.024" rpy="0 0 0" />
+      <origin xyz=".1425 -0.035 0.024" rpy="0 0 0" />
   </xacro:kitting_bin_2>
   <!--set1_bin2_4_-->
   <xacro:kitting_bin_2 binname="set1_bin2_4" parent="workspace_center" z_origin_offset="-.009">
-      <origin xyz=".135 -0.112 0.024" rpy="0 0 0" />
+      <origin xyz=".1425 -0.147 0.024" rpy="0 0 0" />
   </xacro:kitting_bin_2>
   <!--set1_bin3_1_-->
   <xacro:kitting_bin_3 binname="set1_bin3_1" parent="workspace_center" z_origin_offset="-.004">
-      <origin xyz=".135 -0.264 0.019" rpy="0 0 0" />
+      <origin xyz=".1425 -0.299 0.019" rpy="0 0 0" />
   </xacro:kitting_bin_3>
   <!--set2_bin1_1_-->
   <xacro:kitting_bin_1 binname="set2_bin1_1" parent="workspace_center" z_origin_offset="-.008">
-      <origin xyz=".345 0.2175 0.023" rpy="0 0 0" />
+      <origin xyz=".349 0.1825 0.023" rpy="0 0 0" />
   </xacro:kitting_bin_1>
   <!--set2_bin1_2_-->
   <xacro:kitting_bin_1 binname="set2_bin1_2" parent="workspace_center" z_origin_offset="-.008">
-      <origin xyz=".345 0.0925 0.023" rpy="0 0 0" />
+      <origin xyz=".349 0.0575 0.023" rpy="0 0 0" />
   </xacro:kitting_bin_1>
   <!--set2_bin1_3_-->
   <xacro:kitting_bin_1 binname="set2_bin1_3" parent="workspace_center" z_origin_offset="-.008">
-      <origin xyz=".345 -0.0325 0.023" rpy="0 0 0" />
+      <origin xyz=".349 -0.0675 0.023" rpy="0 0 0" />
   </xacro:kitting_bin_1>
   <!--set2_bin1_4_-->
   <xacro:kitting_bin_1 binname="set2_bin1_4" parent="workspace_center" z_origin_offset="-.008">
-      <origin xyz=".345 -0.1575 0.023" rpy="0 0 0" />
+      <origin xyz=".349 -0.1925 0.023" rpy="0 0 0" />
   </xacro:kitting_bin_1>
   <!--set2_bin1_5_-->
   <xacro:kitting_bin_1 binname="set2_bin1_5" parent="workspace_center" z_origin_offset="-.008">
-      <origin xyz=".345 -0.2825 0.023" rpy="0 0 0" />
+      <origin xyz=".349 -0.3175 0.023" rpy="0 0 0" />
   </xacro:kitting_bin_1>
 </robot>

File: o2as_scene_description/urdf/o2as_base_scene.urdf.xacro (robot description, xacro)
@@ -149,5 +149,5 @@
     <!-- <origin xyz="0.46 0 ${bots_z + .1 + .8}" rpy="${-160*pi/180} 0 ${pi/2}"/> -->
     <!-- aist phoxi setting  -->
-    <origin xyz="0.616968905765895 0.121035425329841 1.423091256751067" rpy="-2.626594398897875 0.2001733992896885 1.5970042364211503"/>
+    <origin xyz="0.594404677631629 0.128504467275411 1.427249342095321" rpy="-2.6268341423102637 0.1979289843311739 1.6062811061489097"/>
   </xacro:phoxi_m_camera>
   <!-- I would like to remove the "world" link definition, but apparently it is necessary for Gazebo -->
