Commit message: Add all 6 trays to kitting scene, clean up

File: o2as_scene_description/urdf/kitting_bins.xacro (robot description, xacro)
@@ -3,14 +3,4 @@
   <xacro:include filename="$(find o2as_scene_description)/urdf/kitting_bin_macros.xacro" />
   <xacro:include filename="$(find o2as_scene_description)/urdf/o2as_box.xacro"/>
-  <!-- add rack -->
-  <xacro:o2as_box boxname="rack_bins" box_w="0.42" box_l="0.680" box_h=".015" parent="workspace_center">
-    <origin xyz="0 -.32 0" rpy="0 0 0" />
-  </xacro:o2as_box>
-  <link name="rack_bins_center" />
-  <joint name="rack_bins_joint" type="fixed">
-    <parent link="workspace_center" />
-    <child link="rack_bins_center"/>
-    <origin xyz=".26 0 0.015" rpy="0 0 0"/>
-  </joint>
  <!-- space for bin -->
  <!-- bin1_definition -->
@@ -29,48 +19,48 @@
  <xacro:property name="set1_x" value=".2425"/>
  <xacro:property name="set1_y" value="0.245"/>
- <xacro:property name="set1_z" value="0.015"/>
+ <xacro:property name="set1_z" value="0"/>
  <!-- A row of bin2 -->
  <xacro:property name="set2_x" value=".449"/>
  <xacro:property name="set2_y" value="0.245"/>
- <xacro:property name="set2_z" value="0.015"/>
+ <xacro:property name="set2_z" value="0"/>
  <!--set1_bin2_1_-->
   <xacro:kitting_bin_2 binname="set1_bin2_1" parent="workspace_center" z_origin_offset="-.009">
-      <origin xyz=".2425 0.189 0.024" rpy="0 0 0" />
+      <origin xyz=".2425 0.189 0.009" rpy="0 0 0" />
   </xacro:kitting_bin_2>
   <!--set1_bin2_2_-->
   <xacro:kitting_bin_2 binname="set1_bin2_2" parent="workspace_center" z_origin_offset="-.009">
-      <origin xyz=".2425 0.077 0.024" rpy="0 0 0" />
+      <origin xyz=".2425 0.077 0.009" rpy="0 0 0" />
   </xacro:kitting_bin_2>
   <!--set1_bin2_3_-->
   <xacro:kitting_bin_2 binname="set1_bin2_3" parent="workspace_center" z_origin_offset="-.009">
-      <origin xyz=".2425 -0.035 0.024" rpy="0 0 0" />
+      <origin xyz=".2425 -0.035 0.009" rpy="0 0 0" />
   </xacro:kitting_bin_2>
   <!--set1_bin2_4_-->
   <xacro:kitting_bin_2 binname="set1_bin2_4" parent="workspace_center" z_origin_offset="-.009">
-      <origin xyz=".2425 -0.147 0.024" rpy="0 0 0" />
+      <origin xyz=".2425 -0.147 0.009" rpy="0 0 0" />
   </xacro:kitting_bin_2>
   <!--set1_bin3_1_-->
   <xacro:kitting_bin_3 binname="set1_bin3_1" parent="workspace_center" z_origin_offset="-.004">
-      <origin xyz=".2425 -0.299 0.019" rpy="0 0 0" />
+      <origin xyz=".2425 -0.299 0.004" rpy="0 0 0" />
   </xacro:kitting_bin_3>
   <!--set2_bin1_1_-->
   <xacro:kitting_bin_1 binname="set2_bin1_1" parent="workspace_center" z_origin_offset="-.008">
-      <origin xyz=".449 0.1825 0.023" rpy="0 0 0" />
+      <origin xyz=".449 0.1825 0.008" rpy="0 0 0" />
   </xacro:kitting_bin_1>
   <!--set2_bin1_2_-->
   <xacro:kitting_bin_1 binname="set2_bin1_2" parent="workspace_center" z_origin_offset="-.008">
-      <origin xyz=".449 0.0575 0.023" rpy="0 0 0" />
+      <origin xyz=".449 0.0575 0.008" rpy="0 0 0" />
   </xacro:kitting_bin_1>
   <!--set2_bin1_3_-->
   <xacro:kitting_bin_1 binname="set2_bin1_3" parent="workspace_center" z_origin_offset="-.008">
-      <origin xyz=".449 -0.0675 0.023" rpy="0 0 0" />
+      <origin xyz=".449 -0.0675 0.008" rpy="0 0 0" />
   </xacro:kitting_bin_1>
   <!--set2_bin1_4_-->
   <xacro:kitting_bin_1 binname="set2_bin1_4" parent="workspace_center" z_origin_offset="-.008">
-      <origin xyz=".449 -0.1925 0.023" rpy="0 0 0" />
+      <origin xyz=".449 -0.1925 0.008" rpy="0 0 0" />
   </xacro:kitting_bin_1>
   <!--set2_bin1_5_-->
   <xacro:kitting_bin_1 binname="set2_bin1_5" parent="workspace_center" z_origin_offset="-.008">
-      <origin xyz=".449 -0.3175 0.023" rpy="0 0 0" />
+      <origin xyz=".449 -0.3175 0.008" rpy="0 0 0" />
   </xacro:kitting_bin_1>
 </robot>

File: o2as_scene_description/urdf/kitting_scene.xacro (robot description, xacro)
@@ -23,5 +23,24 @@
   </joint>
   <!-- add trays -->
-  <xacro:property name="tray_x" value="${-tray_length+.01}" />
+  <!-- Tray type 2 carries the screws -->
+  <xacro:kitting_tray2 trayname="set_1_tray_2" parent="rack_trays_center">
+    <origin xyz="+.01 0 0" rpy="0 0 ${pi}" />
+  </xacro:kitting_tray2>
+  <xacro:kitting_tray2 trayname="set_2_tray_2" parent="rack_trays_center">
+    <origin xyz="${tray_length+.01} 0 -.01" rpy="0 0 ${pi}" />
+  </xacro:kitting_tray2>
+  <xacro:kitting_tray2 trayname="set_3_tray_2" parent="rack_trays_center">
+    <origin xyz="+.01 ${tray_width} 0" rpy="0 0 ${pi}" />
+  </xacro:kitting_tray2>
+  <xacro:kitting_tray1 trayname="set_1_tray_1" parent="rack_trays_center">
+    <origin xyz="+.01 0 -.01" rpy="0 0 0" />
+  </xacro:kitting_tray1>
+  <xacro:kitting_tray1 trayname="set_2_tray_1" parent="b_bot_base">
+    <origin xyz=".55 ${tray_length-.1} 0.01" rpy="0 0 ${pi/2}" />
+  </xacro:kitting_tray1>
+  <xacro:kitting_tray1 trayname="set_3_tray_1" parent="b_bot_base">
+    <origin xyz=".55 -.1 0.01" rpy="0 0 ${pi/2}" />
+  </xacro:kitting_tray1>
+  <!-- <xacro:property name="tray_x" value="${-tray_length+.01}" />
   <xacro:property name="tray_y" value="0" />
   <xacro:kitting_tray1 trayname="tray_1" parent="rack_trays_center">
@@ -30,4 +49,4 @@
   <xacro:kitting_tray2 trayname="tray_2" parent="rack_trays_center">
     <origin xyz="+.01 0 0" rpy="0 0 ${pi}" />
-  </xacro:kitting_tray2>
+  </xacro:kitting_tray2> -->
 </robot>

File: o2as_scene_description/urdf/templates/o2as_bin_template_front.xacro (robot description, xacro)
@@ -3,12 +3,2 @@
   <xacro:include filename="$(find o2as_scene_description)/urdf/kitting_bin_macros.xacro" />
   <xacro:include filename="$(find o2as_scene_description)/urdf/o2as_box.xacro"/>
-  <!-- add rack -->
-  <xacro:o2as_box boxname="rack_bins" box_w="0.42" box_l="0.680" box_h=".015" parent="workspace_center">
-    <origin xyz="0 -.32 0" rpy="0 0 0" />
-  </xacro:o2as_box>
-  <link name="rack_bins_center" />
-  <joint name="rack_bins_joint" type="fixed">
-    <parent link="workspace_center" />
-    <child link="rack_bins_center"/>
-    <origin xyz=".26 0 0.015" rpy="0 0 0"/>
-  </joint>

Commit message: Bug fixed.

File: o2as_scene_description/urdf/kitting_bins.xacro (robot description, xacro)
@@ -24,42 +24,42 @@
  <xacro:property name="set2_y" value="0.245"/>
  <xacro:property name="set2_z" value="0"/>
- <!--set1_bin2_1_-->
-  <xacro:kitting_bin_2 binname="set1_bin2_1" parent="workspace_center" z_origin_offset="-.009">
-      <origin xyz=".2425 0.189 0.009" rpy="0 0 0" />
+ <!--bin3_1_-->
+  <xacro:kitting_bin_3 binname="bin3_1" parent="workspace_center" z_origin_offset="-.004">
+      <origin xyz=".2425 0.149 0.004" rpy="0 0 0" />
+  </xacro:kitting_bin_3>
+  <!--bin2_1_-->
+  <xacro:kitting_bin_2 binname="bin2_1" parent="workspace_center" z_origin_offset="-.009">
+      <origin xyz=".2425 -0.003 0.009" rpy="0 0 0" />
   </xacro:kitting_bin_2>
-  <!--set1_bin2_2_-->
-  <xacro:kitting_bin_2 binname="set1_bin2_2" parent="workspace_center" z_origin_offset="-.009">
-      <origin xyz=".2425 0.077 0.009" rpy="0 0 0" />
+  <!--bin2_2_-->
+  <xacro:kitting_bin_2 binname="bin2_2" parent="workspace_center" z_origin_offset="-.009">
+      <origin xyz=".2425 -0.115 0.009" rpy="0 0 0" />
   </xacro:kitting_bin_2>
-  <!--set1_bin2_3_-->
-  <xacro:kitting_bin_2 binname="set1_bin2_3" parent="workspace_center" z_origin_offset="-.009">
-      <origin xyz=".2425 -0.035 0.009" rpy="0 0 0" />
+  <!--bin2_3_-->
+  <xacro:kitting_bin_2 binname="bin2_3" parent="workspace_center" z_origin_offset="-.009">
+      <origin xyz=".2425 -0.227 0.009" rpy="0 0 0" />
   </xacro:kitting_bin_2>
-  <!--set1_bin2_4_-->
-  <xacro:kitting_bin_2 binname="set1_bin2_4" parent="workspace_center" z_origin_offset="-.009">
-      <origin xyz=".2425 -0.147 0.009" rpy="0 0 0" />
+  <!--bin2_4_-->
+  <xacro:kitting_bin_2 binname="bin2_4" parent="workspace_center" z_origin_offset="-.009">
+      <origin xyz=".2425 -0.339 0.009" rpy="0 0 0" />
   </xacro:kitting_bin_2>
-  <!--set1_bin3_1_-->
-  <xacro:kitting_bin_3 binname="set1_bin3_1" parent="workspace_center" z_origin_offset="-.004">
-      <origin xyz=".2425 -0.299 0.004" rpy="0 0 0" />
-  </xacro:kitting_bin_3>
-  <!--set2_bin1_1_-->
-  <xacro:kitting_bin_1 binname="set2_bin1_1" parent="workspace_center" z_origin_offset="-.008">
+  <!--bin1_1_-->
+  <xacro:kitting_bin_1 binname="bin1_1" parent="workspace_center" z_origin_offset="-.008">
       <origin xyz=".449 0.1825 0.008" rpy="0 0 0" />
   </xacro:kitting_bin_1>
-  <!--set2_bin1_2_-->
-  <xacro:kitting_bin_1 binname="set2_bin1_2" parent="workspace_center" z_origin_offset="-.008">
+  <!--bin1_2_-->
+  <xacro:kitting_bin_1 binname="bin1_2" parent="workspace_center" z_origin_offset="-.008">
       <origin xyz=".449 0.0575 0.008" rpy="0 0 0" />
   </xacro:kitting_bin_1>
-  <!--set2_bin1_3_-->
-  <xacro:kitting_bin_1 binname="set2_bin1_3" parent="workspace_center" z_origin_offset="-.008">
+  <!--bin1_3_-->
+  <xacro:kitting_bin_1 binname="bin1_3" parent="workspace_center" z_origin_offset="-.008">
       <origin xyz=".449 -0.0675 0.008" rpy="0 0 0" />
   </xacro:kitting_bin_1>
-  <!--set2_bin1_4_-->
-  <xacro:kitting_bin_1 binname="set2_bin1_4" parent="workspace_center" z_origin_offset="-.008">
+  <!--bin1_4_-->
+  <xacro:kitting_bin_1 binname="bin1_4" parent="workspace_center" z_origin_offset="-.008">
       <origin xyz=".449 -0.1925 0.008" rpy="0 0 0" />
   </xacro:kitting_bin_1>
-  <!--set2_bin1_5_-->
-  <xacro:kitting_bin_1 binname="set2_bin1_5" parent="workspace_center" z_origin_offset="-.008">
+  <!--bin1_5_-->
+  <xacro:kitting_bin_1 binname="bin1_5" parent="workspace_center" z_origin_offset="-.008">
       <origin xyz=".449 -0.3175 0.008" rpy="0 0 0" />
   </xacro:kitting_bin_1>

Commit message: Cleaning up.

File: o2as_scene_description/urdf/kitting_bins.xacro (robot description, xacro)
@@ -3,64 +3,64 @@
   <xacro:include filename="$(find o2as_scene_description)/urdf/kitting_bin_macros.xacro" />
   <xacro:include filename="$(find o2as_scene_description)/urdf/o2as_box.xacro"/>
- <!-- space for bin -->
- <!-- bin1_definition -->
- <xacro:property name="bin1_width" value="0.125"/>
- <xacro:property name="bin1_length" value="0.128"/>
- <xacro:property name="z_origin_offset_1" value="-.008" />
- <!-- bin2_definition -->
- <xacro:property name="bin2_width" value="0.112"/>
- <xacro:property name="bin2_length" value="0.201"/>
- <xacro:property name="z_origin_offset_2" value="-.009" />
- <!-- bin3_definition -->
- <xacro:property name="bin3_width" value="0.192"/>
- <xacro:property name="bin3_length" value="0.285"/>
- <xacro:property name="z_origin_offset_3" value="-.004" />
- <!-- A row of bin1 -->
- <xacro:property name="set1_x" value=".2425"/>
- <xacro:property name="set1_y" value="0.245"/>
- <xacro:property name="set1_z" value="0"/>
- <!-- A row of bin2 -->
- <xacro:property name="set2_x" value=".449"/>
- <xacro:property name="set2_y" value="0.245"/>
- <xacro:property name="set2_z" value="0"/>
- <!--set1_bin2_1_-->
+  <!-- space for bin -->
+  <!-- bin1_definition -->
+  <xacro:property name="bin1_width" value="0.125"/>
+  <xacro:property name="bin1_length" value="0.128"/>
+  <xacro:property name="z_origin_offset_1" value="-.008" />
+  <!-- bin2_definition -->
+  <xacro:property name="bin2_width" value="0.112"/>
+  <xacro:property name="bin2_length" value="0.201"/>
+  <xacro:property name="z_origin_offset_2" value="-.009" />
+  <!-- bin3_definition -->
+  <xacro:property name="bin3_width" value="0.192"/>
+  <xacro:property name="bin3_length" value="0.285"/>
+  <xacro:property name="z_origin_offset_3" value="-.004" />
+  <!-- A row of bin1 -->
+  <xacro:property name="set1_x" value=".2425"/>
+  <xacro:property name="set1_y" value="0.245"/>
+  <xacro:property name="set1_z" value="0"/>
+  <!-- A row of bin2 -->
+  <xacro:property name="set2_x" value=".449"/>
+  <xacro:property name="set2_y" value="0.245"/>
+  <xacro:property name="set2_z" value="0"/>
+  <!--set1_bin2_1_-->
   <xacro:kitting_bin_2 binname="set1_bin2_1" parent="workspace_center" z_origin_offset="-.009">
-      <origin xyz=".2425 0.189 0.009" rpy="0 0 0" />
+    <origin xyz=".2425 0.189 0.009" rpy="0 0 0" />
   </xacro:kitting_bin_2>
   <!--set1_bin2_2_-->
   <xacro:kitting_bin_2 binname="set1_bin2_2" parent="workspace_center" z_origin_offset="-.009">
-      <origin xyz=".2425 0.077 0.009" rpy="0 0 0" />
+    <origin xyz=".2425 0.077 0.009" rpy="0 0 0" />
   </xacro:kitting_bin_2>
   <!--set1_bin2_3_-->
   <xacro:kitting_bin_2 binname="set1_bin2_3" parent="workspace_center" z_origin_offset="-.009">
-      <origin xyz=".2425 -0.035 0.009" rpy="0 0 0" />
+    <origin xyz=".2425 -0.035 0.009" rpy="0 0 0" />
   </xacro:kitting_bin_2>
   <!--set1_bin2_4_-->
   <xacro:kitting_bin_2 binname="set1_bin2_4" parent="workspace_center" z_origin_offset="-.009">
-      <origin xyz=".2425 -0.147 0.009" rpy="0 0 0" />
+    <origin xyz=".2425 -0.147 0.009" rpy="0 0 0" />
   </xacro:kitting_bin_2>
   <!--set1_bin3_1_-->
   <xacro:kitting_bin_3 binname="set1_bin3_1" parent="workspace_center" z_origin_offset="-.004">
-      <origin xyz=".2425 -0.299 0.004" rpy="0 0 0" />
+    <origin xyz=".2425 -0.299 0.004" rpy="0 0 0" />
   </xacro:kitting_bin_3>
   <!--set2_bin1_1_-->
   <xacro:kitting_bin_1 binname="set2_bin1_1" parent="workspace_center" z_origin_offset="-.008">
-      <origin xyz=".449 0.1825 0.008" rpy="0 0 0" />
+    <origin xyz=".449 0.1825 0.008" rpy="0 0 0" />
   </xacro:kitting_bin_1>
   <!--set2_bin1_2_-->
   <xacro:kitting_bin_1 binname="set2_bin1_2" parent="workspace_center" z_origin_offset="-.008">
-      <origin xyz=".449 0.0575 0.008" rpy="0 0 0" />
+    <origin xyz=".449 0.0575 0.008" rpy="0 0 0" />
   </xacro:kitting_bin_1>
   <!--set2_bin1_3_-->
   <xacro:kitting_bin_1 binname="set2_bin1_3" parent="workspace_center" z_origin_offset="-.008">
-      <origin xyz=".449 -0.0675 0.008" rpy="0 0 0" />
+    <origin xyz=".449 -0.0675 0.008" rpy="0 0 0" />
   </xacro:kitting_bin_1>
   <!--set2_bin1_4_-->
   <xacro:kitting_bin_1 binname="set2_bin1_4" parent="workspace_center" z_origin_offset="-.008">
-      <origin xyz=".449 -0.1925 0.008" rpy="0 0 0" />
+    <origin xyz=".449 -0.1925 0.008" rpy="0 0 0" />
   </xacro:kitting_bin_1>
   <!--set2_bin1_5_-->
   <xacro:kitting_bin_1 binname="set2_bin1_5" parent="workspace_center" z_origin_offset="-.008">
-      <origin xyz=".449 -0.3175 0.008" rpy="0 0 0" />
+    <origin xyz=".449 -0.3175 0.008" rpy="0 0 0" />
   </xacro:kitting_bin_1>
 </robot>

File: o2as_scene_description/urdf/o2as_base_scene.urdf.xacro (robot description, xacro)
@@ -23,5 +23,5 @@
   <!-- Scene items (trays, bins...) -->
   <!-- <xacro:include filename="$(find o2as_scene_description)/urdf/taskboard_scene.xacro" /> -->
-  <!-- <xacro:include filename="$(find o2as_scene_description)/urdf/kitting_scene.xa -->cro" />
+  <!-- <xacro:include filename="$(find o2as_scene_description)/urdf/kitting_scene.xacro" /> -->
   <!-- <xacro:include filename="$(find o2as_scene_description)/urdf/assembly_scene.xacro" /> -->
   <!-- Robot bases -->
@@ -150,9 +150,9 @@
   <!-- spawn and attach AR markers -->
   <xacro:include filename="$(find o2as_gazebo)/urdf/o2as_ar_marker.urdf.xacro"/>
-  <xacro:o2as_ar_marker prefix="a_bot_"
-  			parent="a_bot_ee_link"
-  			marker_id="26">
-    <origin xyz="0.08 0.0 0.065" rpy="0 0 0"/>
-  </xacro:o2as_ar_marker>
+  <!-- <xacro:o2as_ar_marker prefix="a_bot_" -->
+  <!-- 			parent="a_bot_ee_link" -->
+  <!-- 			marker_id="26"> -->
+  <!--   <origin xyz="0.08 0.00 0.065" rpy="0 0 0"/> -->
+  <!-- </xacro:o2as_ar_marker> -->
   <!-- <xacro:o2as_ar_marker prefix="b_bot_" -->
   <!-- 			parent="b_bot_dual_suction_gripper_base_link" -->
@@ -178,5 +178,5 @@
 			parent="workspace_center"
 			marker_id="256">
-    <origin xyz="0.0 0.0 0.0" rpy="0 0 0"/>
+    <origin xyz="0.0 0.0 0.0005" rpy="0 0 0"/>
   </xacro:o2as_ar_marker>
   <!-- Add PhoXi 3D scanners -->

Commit message: Rename package graspability estimation.

File: o2as_scene_description/urdf/kitting_bins.xacro (robot description, xacro)
@@ -18,49 +18,49 @@
  <!-- A row of bin1 -->
  <xacro:property name="set1_x" value=".2425"/>
- <xacro:property name="set1_y" value="0.245"/>
+ <xacro:property name="set1_y" value="0.295"/>
  <xacro:property name="set1_z" value="0"/>
  <!-- A row of bin2 -->
  <xacro:property name="set2_x" value=".449"/>
- <xacro:property name="set2_y" value="0.245"/>
+ <xacro:property name="set2_y" value="0.295"/>
  <xacro:property name="set2_z" value="0"/>
- <!--bin3_1_-->
-  <xacro:kitting_bin_3 binname="bin3_1" parent="workspace_center" z_origin_offset="-.004">
-      <origin xyz=".2425 0.149 0.004" rpy="0 0 0" />
+ <!--set1_bin2_1_-->
+  <xacro:kitting_bin_2 binname="set1_bin2_1" parent="workspace_center" z_origin_offset="-.009">
+      <origin xyz=".2425 0.239 0.009" rpy="0 0 0" />
+  </xacro:kitting_bin_2>
+  <!--set1_bin2_2_-->
+  <xacro:kitting_bin_2 binname="set1_bin2_2" parent="workspace_center" z_origin_offset="-.009">
+      <origin xyz=".2425 0.127 0.009" rpy="0 0 0" />
+  </xacro:kitting_bin_2>
+  <!--set1_bin2_3_-->
+  <xacro:kitting_bin_2 binname="set1_bin2_3" parent="workspace_center" z_origin_offset="-.009">
+      <origin xyz=".2425 0.015 0.009" rpy="0 0 0" />
+  </xacro:kitting_bin_2>
+  <!--set1_bin2_4_-->
+  <xacro:kitting_bin_2 binname="set1_bin2_4" parent="workspace_center" z_origin_offset="-.009">
+      <origin xyz=".2425 -0.097 0.009" rpy="0 0 0" />
+  </xacro:kitting_bin_2>
+  <!--set1_bin3_1_-->
+  <xacro:kitting_bin_3 binname="set1_bin3_1" parent="workspace_center" z_origin_offset="-.004">
+      <origin xyz=".2425 -0.249 0.004" rpy="0 0 0" />
   </xacro:kitting_bin_3>
-  <!--bin2_1_-->
-  <xacro:kitting_bin_2 binname="bin2_1" parent="workspace_center" z_origin_offset="-.009">
-      <origin xyz=".2425 -0.003 0.009" rpy="0 0 0" />
-  </xacro:kitting_bin_2>
-  <!--bin2_2_-->
-  <xacro:kitting_bin_2 binname="bin2_2" parent="workspace_center" z_origin_offset="-.009">
-      <origin xyz=".2425 -0.115 0.009" rpy="0 0 0" />
-  </xacro:kitting_bin_2>
-  <!--bin2_3_-->
-  <xacro:kitting_bin_2 binname="bin2_3" parent="workspace_center" z_origin_offset="-.009">
-      <origin xyz=".2425 -0.227 0.009" rpy="0 0 0" />
-  </xacro:kitting_bin_2>
-  <!--bin2_4_-->
-  <xacro:kitting_bin_2 binname="bin2_4" parent="workspace_center" z_origin_offset="-.009">
-      <origin xyz=".2425 -0.339 0.009" rpy="0 0 0" />
-  </xacro:kitting_bin_2>
-  <!--bin1_1_-->
-  <xacro:kitting_bin_1 binname="bin1_1" parent="workspace_center" z_origin_offset="-.008">
-      <origin xyz=".449 0.1825 0.008" rpy="0 0 0" />
+  <!--set2_bin1_1_-->
+  <xacro:kitting_bin_1 binname="set2_bin1_1" parent="workspace_center" z_origin_offset="-.008">
+      <origin xyz=".449 0.2325 0.008" rpy="0 0 0" />
   </xacro:kitting_bin_1>
-  <!--bin1_2_-->
-  <xacro:kitting_bin_1 binname="bin1_2" parent="workspace_center" z_origin_offset="-.008">
-      <origin xyz=".449 0.0575 0.008" rpy="0 0 0" />
+  <!--set2_bin1_2_-->
+  <xacro:kitting_bin_1 binname="set2_bin1_2" parent="workspace_center" z_origin_offset="-.008">
+      <origin xyz=".449 0.1075 0.008" rpy="0 0 0" />
   </xacro:kitting_bin_1>
-  <!--bin1_3_-->
-  <xacro:kitting_bin_1 binname="bin1_3" parent="workspace_center" z_origin_offset="-.008">
-      <origin xyz=".449 -0.0675 0.008" rpy="0 0 0" />
+  <!--set2_bin1_3_-->
+  <xacro:kitting_bin_1 binname="set2_bin1_3" parent="workspace_center" z_origin_offset="-.008">
+      <origin xyz=".449 -0.0175 0.008" rpy="0 0 0" />
   </xacro:kitting_bin_1>
-  <!--bin1_4_-->
-  <xacro:kitting_bin_1 binname="bin1_4" parent="workspace_center" z_origin_offset="-.008">
-      <origin xyz=".449 -0.1925 0.008" rpy="0 0 0" />
+  <!--set2_bin1_4_-->
+  <xacro:kitting_bin_1 binname="set2_bin1_4" parent="workspace_center" z_origin_offset="-.008">
+      <origin xyz=".449 -0.1425 0.008" rpy="0 0 0" />
   </xacro:kitting_bin_1>
-  <!--bin1_5_-->
-  <xacro:kitting_bin_1 binname="bin1_5" parent="workspace_center" z_origin_offset="-.008">
-      <origin xyz=".449 -0.3175 0.008" rpy="0 0 0" />
+  <!--set2_bin1_5_-->
+  <xacro:kitting_bin_1 binname="set2_bin1_5" parent="workspace_center" z_origin_offset="-.008">
+      <origin xyz=".449 -0.2675 0.008" rpy="0 0 0" />
   </xacro:kitting_bin_1>
 </robot>
