Commit message: First real test

File: o2as_scene_description/urdf/kitting_bins.xacro (robot description, xacro)
@@ -18,49 +18,49 @@
  <!-- A row of bin1 -->
  <xacro:property name="set1_x" value=".2425"/>
- <xacro:property name="set1_y" value="0.245"/>
+ <xacro:property name="set1_y" value="0.295"/>
  <xacro:property name="set1_z" value="0"/>
  <!-- A row of bin2 -->
  <xacro:property name="set2_x" value=".449"/>
- <xacro:property name="set2_y" value="0.245"/>
+ <xacro:property name="set2_y" value="0.295"/>
  <xacro:property name="set2_z" value="0"/>
  <!--bin3_1_-->
   <xacro:kitting_bin_3 binname="bin3_1" parent="workspace_center" z_origin_offset="-.004">
-      <origin xyz=".2425 0.149 0.004" rpy="0 0 0" />
+      <origin xyz=".2425 0.199 0.004" rpy="0 0 0" />
   </xacro:kitting_bin_3>
   <!--bin2_1_-->
   <xacro:kitting_bin_2 binname="bin2_1" parent="workspace_center" z_origin_offset="-.009">
-      <origin xyz=".2425 -0.003 0.009" rpy="0 0 0" />
+      <origin xyz=".2425 0.047 0.009" rpy="0 0 0" />
   </xacro:kitting_bin_2>
   <!--bin2_2_-->
   <xacro:kitting_bin_2 binname="bin2_2" parent="workspace_center" z_origin_offset="-.009">
-      <origin xyz=".2425 -0.115 0.009" rpy="0 0 0" />
+      <origin xyz=".2425 -0.065 0.009" rpy="0 0 0" />
   </xacro:kitting_bin_2>
   <!--bin2_3_-->
   <xacro:kitting_bin_2 binname="bin2_3" parent="workspace_center" z_origin_offset="-.009">
-      <origin xyz=".2425 -0.227 0.009" rpy="0 0 0" />
+      <origin xyz=".2425 -0.177 0.009" rpy="0 0 0" />
   </xacro:kitting_bin_2>
   <!--bin2_4_-->
   <xacro:kitting_bin_2 binname="bin2_4" parent="workspace_center" z_origin_offset="-.009">
-      <origin xyz=".2425 -0.339 0.009" rpy="0 0 0" />
+      <origin xyz=".2425 -0.289 0.009" rpy="0 0 0" />
   </xacro:kitting_bin_2>
   <!--bin1_1_-->
   <xacro:kitting_bin_1 binname="bin1_1" parent="workspace_center" z_origin_offset="-.008">
-      <origin xyz=".449 0.1825 0.008" rpy="0 0 0" />
+      <origin xyz=".449 0.2325 0.008" rpy="0 0 0" />
   </xacro:kitting_bin_1>
   <!--bin1_2_-->
   <xacro:kitting_bin_1 binname="bin1_2" parent="workspace_center" z_origin_offset="-.008">
-      <origin xyz=".449 0.0575 0.008" rpy="0 0 0" />
+      <origin xyz=".449 0.1075 0.008" rpy="0 0 0" />
+  </xacro:kitting_bin_1>
+  <!--bin1_4_-->
+  <xacro:kitting_bin_1 binname="bin1_4" parent="workspace_center" z_origin_offset="-.008">
+      <origin xyz=".449 -0.0175 0.008" rpy="0 0 0" />
+  </xacro:kitting_bin_1>
+  <!--bin1_5_-->
+  <xacro:kitting_bin_1 binname="bin1_5" parent="workspace_center" z_origin_offset="-.008">
+      <origin xyz=".449 -0.1425 0.008" rpy="0 0 0" />
   </xacro:kitting_bin_1>
   <!--bin1_3_-->
   <xacro:kitting_bin_1 binname="bin1_3" parent="workspace_center" z_origin_offset="-.008">
-      <origin xyz=".449 -0.0675 0.008" rpy="0 0 0" />
-  </xacro:kitting_bin_1>
-  <!--bin1_4_-->
-  <xacro:kitting_bin_1 binname="bin1_4" parent="workspace_center" z_origin_offset="-.008">
-      <origin xyz=".449 -0.1925 0.008" rpy="0 0 0" />
-  </xacro:kitting_bin_1>
-  <!--bin1_5_-->
-  <xacro:kitting_bin_1 binname="bin1_5" parent="workspace_center" z_origin_offset="-.008">
-      <origin xyz=".449 -0.3175 0.008" rpy="0 0 0" />
+      <origin xyz=".449 -0.2675 0.008" rpy="0 0 0" />
   </xacro:kitting_bin_1>
 </robot>

Commit message: Calibration & Cleanup

File: o2as_scene_description/urdf/kitting_bins.xacro (robot description, xacro)
@@ -7,9 +7,9 @@
  <xacro:property name="bin1_width" value="0.125"/>
  <xacro:property name="bin1_length" value="0.128"/>
- <xacro:property name="z_origin_offset_1" value="-.008" />
+ <xacro:property name="z_origin_offset_1" value="-.005" />
  <!-- bin2_definition -->
  <xacro:property name="bin2_width" value="0.112"/>
  <xacro:property name="bin2_length" value="0.201"/>
- <xacro:property name="z_origin_offset_2" value="-.009" />
+ <xacro:property name="z_origin_offset_2" value="-.008" />
  <!-- bin3_definition -->
  <xacro:property name="bin3_width" value="0.192"/>
@@ -22,5 +22,5 @@
  <!-- A row of bin2 -->
  <xacro:property name="set2_x" value=".449"/>
- <xacro:property name="set2_y" value="0.295"/>
+ <xacro:property name="set2_y" value="0.245"/>
  <xacro:property name="set2_z" value="0"/>
  <!--bin3_1_-->
@@ -29,38 +29,38 @@
   </xacro:kitting_bin_3>
   <!--bin2_1_-->
-  <xacro:kitting_bin_2 binname="bin2_1" parent="workspace_center" z_origin_offset="-.009">
-      <origin xyz=".2425 0.047 0.009" rpy="0 0 0" />
+  <xacro:kitting_bin_2 binname="bin2_1" parent="workspace_center" z_origin_offset="-.008">
+      <origin xyz=".2425 0.047 0.008" rpy="0 0 0" />
   </xacro:kitting_bin_2>
   <!--bin2_2_-->
-  <xacro:kitting_bin_2 binname="bin2_2" parent="workspace_center" z_origin_offset="-.009">
-      <origin xyz=".2425 -0.065 0.009" rpy="0 0 0" />
+  <xacro:kitting_bin_2 binname="bin2_2" parent="workspace_center" z_origin_offset="-.008">
+      <origin xyz=".2425 -0.065 0.008" rpy="0 0 0" />
   </xacro:kitting_bin_2>
   <!--bin2_3_-->
-  <xacro:kitting_bin_2 binname="bin2_3" parent="workspace_center" z_origin_offset="-.009">
-      <origin xyz=".2425 -0.177 0.009" rpy="0 0 0" />
+  <xacro:kitting_bin_2 binname="bin2_3" parent="workspace_center" z_origin_offset="-.008">
+      <origin xyz=".2425 -0.177 0.008" rpy="0 0 0" />
   </xacro:kitting_bin_2>
   <!--bin2_4_-->
-  <xacro:kitting_bin_2 binname="bin2_4" parent="workspace_center" z_origin_offset="-.009">
-      <origin xyz=".2425 -0.289 0.009" rpy="0 0 0" />
+  <xacro:kitting_bin_2 binname="bin2_4" parent="workspace_center" z_origin_offset="-.008">
+      <origin xyz=".2425 -0.289 0.008" rpy="0 0 0" />
   </xacro:kitting_bin_2>
   <!--bin1_1_-->
-  <xacro:kitting_bin_1 binname="bin1_1" parent="workspace_center" z_origin_offset="-.008">
-      <origin xyz=".449 0.2325 0.008" rpy="0 0 0" />
+  <xacro:kitting_bin_1 binname="bin1_1" parent="workspace_center" z_origin_offset="-.005">
+      <origin xyz=".449 0.1825 0.005" rpy="0 0 0" />
   </xacro:kitting_bin_1>
   <!--bin1_2_-->
-  <xacro:kitting_bin_1 binname="bin1_2" parent="workspace_center" z_origin_offset="-.008">
-      <origin xyz=".449 0.1075 0.008" rpy="0 0 0" />
+  <xacro:kitting_bin_1 binname="bin1_2" parent="workspace_center" z_origin_offset="-.005">
+      <origin xyz=".449 0.0575 0.005" rpy="0 0 0" />
   </xacro:kitting_bin_1>
   <!--bin1_4_-->
-  <xacro:kitting_bin_1 binname="bin1_4" parent="workspace_center" z_origin_offset="-.008">
-      <origin xyz=".449 -0.0175 0.008" rpy="0 0 0" />
+  <xacro:kitting_bin_1 binname="bin1_4" parent="workspace_center" z_origin_offset="-.005">
+      <origin xyz=".449 -0.0675 0.005" rpy="0 0 0" />
   </xacro:kitting_bin_1>
   <!--bin1_5_-->
-  <xacro:kitting_bin_1 binname="bin1_5" parent="workspace_center" z_origin_offset="-.008">
-      <origin xyz=".449 -0.1425 0.008" rpy="0 0 0" />
+  <xacro:kitting_bin_1 binname="bin1_5" parent="workspace_center" z_origin_offset="-.005">
+      <origin xyz=".449 -0.1925 0.005" rpy="0 0 0" />
   </xacro:kitting_bin_1>
   <!--bin1_3_-->
-  <xacro:kitting_bin_1 binname="bin1_3" parent="workspace_center" z_origin_offset="-.008">
-      <origin xyz=".449 -0.2675 0.008" rpy="0 0 0" />
+  <xacro:kitting_bin_1 binname="bin1_3" parent="workspace_center" z_origin_offset="-.005">
+      <origin xyz=".449 -0.3175 0.005" rpy="0 0 0" />
   </xacro:kitting_bin_1>
 </robot>

File: o2as_scene_description/urdf/robotiq_b_bot_gripper.urdf.xacro (robot description, xacro)
@@ -42,5 +42,5 @@
       <parent link="${prefix}robotiq_85_tip_link"/>
       <child link="${prefix}suction_tool_tip_link"/>
-      <origin rpy="0.0 ${pi/2} 0.0" xyz="${dx+.008} 0.0 -0.126 "/>
+      <origin rpy="0.0 ${pi/2} 0.0" xyz="${dx+.013} 0.0 -0.131 "/>
     </joint>
     <link name="${prefix}suction_tool_tip_link"/>

Commit message: Dump commit @ evening kitting test

File: o2as_scene_description/urdf/kitting_bins.xacro (robot description, xacro)
@@ -12,8 +12,8 @@
  <xacro:property name="bin2_length" value="0.201"/>
  <xacro:property name="z_origin_offset_2" value="-.008" />
-  <!-- bin3_definition -->
-  <xacro:property name="bin3_width" value="0.192"/>
-  <xacro:property name="bin3_length" value="0.285"/>
-  <xacro:property name="z_origin_offset_3" value="-.004" />
+ <!-- bin3_definition -->
+ <xacro:property name="bin3_width" value="0.192"/>
+ <xacro:property name="bin3_length" value="0.285"/>
+ <xacro:property name="z_origin_offset_3" value="-.004" />
  <!-- A row of bin1 -->
  <xacro:property name="set1_x" value=".2425"/>
@@ -24,42 +24,42 @@
  <xacro:property name="set2_y" value="0.245"/>
  <xacro:property name="set2_z" value="0"/>
- <!--bin3_1_-->
-  <xacro:kitting_bin_3 binname="bin3_1" parent="workspace_center" z_origin_offset="-.004">
-      <origin xyz=".2425 0.199 0.004" rpy="0 0 0" />
-  </xacro:kitting_bin_3>
-  <!--bin2_1_-->
+ <!--bin2_1_-->
   <xacro:kitting_bin_2 binname="bin2_1" parent="workspace_center" z_origin_offset="-.008">
-      <origin xyz=".2425 0.047 0.008" rpy="0 0 0" />
+      <origin xyz=".2425 0.239 0.008" rpy="0 0 0" />
   </xacro:kitting_bin_2>
   <!--bin2_2_-->
   <xacro:kitting_bin_2 binname="bin2_2" parent="workspace_center" z_origin_offset="-.008">
-      <origin xyz=".2425 -0.065 0.008" rpy="0 0 0" />
+      <origin xyz=".2425 0.127 0.008" rpy="0 0 0" />
   </xacro:kitting_bin_2>
-  <!--bin2_3_-->
-  <xacro:kitting_bin_2 binname="bin2_3" parent="workspace_center" z_origin_offset="-.008">
-      <origin xyz=".2425 -0.177 0.008" rpy="0 0 0" />
-  </xacro:kitting_bin_2>
-  <!--bin2_4_-->
-  <xacro:kitting_bin_2 binname="bin2_4" parent="workspace_center" z_origin_offset="-.008">
-      <origin xyz=".2425 -0.289 0.008" rpy="0 0 0" />
-  </xacro:kitting_bin_2>
-  <!--bin1_1_-->
-  <xacro:kitting_bin_1 binname="bin1_1" parent="workspace_center" z_origin_offset="-.005">
-      <origin xyz=".449 0.1825 0.005" rpy="0 0 0" />
+  <!--bin1_3_-->
+  <xacro:kitting_bin_1 binname="bin1_3" parent="workspace_center" z_origin_offset="-.005">
+      <origin xyz=".2425 0.0085 0.005" rpy="0 0 0" />
   </xacro:kitting_bin_1>
   <!--bin1_2_-->
   <xacro:kitting_bin_1 binname="bin1_2" parent="workspace_center" z_origin_offset="-.005">
-      <origin xyz=".449 0.0575 0.005" rpy="0 0 0" />
+      <origin xyz=".2425 -0.1165 0.005" rpy="0 0 0" />
+  </xacro:kitting_bin_1>
+  <!--bin1_1_-->
+  <xacro:kitting_bin_1 binname="bin1_1" parent="workspace_center" z_origin_offset="-.005">
+      <origin xyz=".2425 -0.2415 0.005" rpy="0 0 0" />
   </xacro:kitting_bin_1>
   <!--bin1_4_-->
   <xacro:kitting_bin_1 binname="bin1_4" parent="workspace_center" z_origin_offset="-.005">
-      <origin xyz=".449 -0.0675 0.005" rpy="0 0 0" />
+      <origin xyz=".449 0.1825 0.005" rpy="0 0 0" />
   </xacro:kitting_bin_1>
   <!--bin1_5_-->
   <xacro:kitting_bin_1 binname="bin1_5" parent="workspace_center" z_origin_offset="-.005">
+      <origin xyz=".449 0.0575 0.005" rpy="0 0 0" />
+  </xacro:kitting_bin_1>
+  <!--bin1_7_-->
+  <xacro:kitting_bin_1 binname="bin1_7" parent="workspace_center" z_origin_offset="-.005">
+      <origin xyz=".449 -0.0675 0.005" rpy="0 0 0" />
+  </xacro:kitting_bin_1>
+  <!--bin1_8_-->
+  <xacro:kitting_bin_1 binname="bin1_8" parent="workspace_center" z_origin_offset="-.005">
       <origin xyz=".449 -0.1925 0.005" rpy="0 0 0" />
   </xacro:kitting_bin_1>
-  <!--bin1_3_-->
-  <xacro:kitting_bin_1 binname="bin1_3" parent="workspace_center" z_origin_offset="-.005">
+  <!--bin1_6_-->
+  <xacro:kitting_bin_1 binname="bin1_6" parent="workspace_center" z_origin_offset="-.005">
       <origin xyz=".449 -0.3175 0.005" rpy="0 0 0" />
   </xacro:kitting_bin_1>

File: o2as_scene_description/urdf/o2as_base_scene.urdf.xacro (robot description, xacro)
@@ -21,6 +21,6 @@
   <xacro:include filename="$(find o2as_scene_description)/urdf/ur3.urdf.xacro" />
   <!-- Scene items (trays, bins...) -->
-  <xacro:include filename="$(find o2as_scene_description)/urdf/taskboard_scene.xacro" />
-  <!-- <xacro:include filename="$(find o2as_scene_description)/urdf/kitting_scene.xacro" /> -->
+  <!-- <xacro:include filename="$(find o2as_scene_description)/urdf/taskboard_scene.xacro" /> -->
+  <xacro:include filename="$(find o2as_scene_description)/urdf/kitting_scene.xacro" />
   <!-- <xacro:include filename="$(find o2as_scene_description)/urdf/assembly_scene.xacro" /> -->
   <!-- <xacro:include filename="$(find o2as_scene_description)/urdf/calibration_scene.xacro" /> -->
@@ -148,6 +148,5 @@
   <xacro:include filename="$(find o2as_scene_description)/urdf/phoxi_m_camera.urdf.xacro" />
   <xacro:phoxi_m_camera prefix="a_" parent="o2as_ground">
-  <origin xyz="0.656427245186 -0.0191234201169 1.50626196172"
-          rpy="${-161.285833025*pi/180} ${0.547979734685*pi/180} ${91.027298919*pi/180}"/>
+  <origin xyz="0.652663578768 -0.0142895785849 1.50687788672" rpy="${-161.381811856*pi/180} ${2.99567722105*pi/180} ${90.8962573459*pi/180}"/>
   </xacro:phoxi_m_camera>
   <!-- I would like to remove the "world" link definition, but apparently it is necessary for Gazebo -->

Commit message: Kitting trial 1

File: o2as_scene_description/urdf/kitting_bins.xacro (robot description, xacro)
@@ -24,42 +24,42 @@
  <xacro:property name="set2_y" value="0.245"/>
  <xacro:property name="set2_z" value="0"/>
- <!--bin2_1_-->
-  <xacro:kitting_bin_2 binname="bin2_1" parent="workspace_center" z_origin_offset="-.008">
-      <origin xyz=".2425 0.239 0.008" rpy="0 0 0" />
+ <!--bin3_1_-->
+  <xacro:kitting_bin_3 binname="bin3_1" parent="workspace_center" z_origin_offset="-.004">
+      <origin xyz=".2425 0.199 0.004" rpy="0 0 0" />
+  </xacro:kitting_bin_3>
+  <!--bin2_4_-->
+  <xacro:kitting_bin_2 binname="bin2_4" parent="workspace_center" z_origin_offset="-.008">
+      <origin xyz=".2425 0.047 0.008" rpy="0 0 0" />
+  </xacro:kitting_bin_2>
+  <!--bin2_3_-->
+  <xacro:kitting_bin_2 binname="bin2_3" parent="workspace_center" z_origin_offset="-.008">
+      <origin xyz=".2425 -0.065 0.008" rpy="0 0 0" />
   </xacro:kitting_bin_2>
   <!--bin2_2_-->
   <xacro:kitting_bin_2 binname="bin2_2" parent="workspace_center" z_origin_offset="-.008">
-      <origin xyz=".2425 0.127 0.008" rpy="0 0 0" />
+      <origin xyz=".2425 -0.177 0.008" rpy="0 0 0" />
   </xacro:kitting_bin_2>
-  <!--bin1_3_-->
-  <xacro:kitting_bin_1 binname="bin1_3" parent="workspace_center" z_origin_offset="-.005">
-      <origin xyz=".2425 0.0085 0.005" rpy="0 0 0" />
-  </xacro:kitting_bin_1>
+  <!--bin2_1_-->
+  <xacro:kitting_bin_2 binname="bin2_1" parent="workspace_center" z_origin_offset="-.008">
+      <origin xyz=".2425 -0.289 0.008" rpy="0 0 0" />
+  </xacro:kitting_bin_2>
   <!--bin1_2_-->
   <xacro:kitting_bin_1 binname="bin1_2" parent="workspace_center" z_origin_offset="-.005">
-      <origin xyz=".2425 -0.1165 0.005" rpy="0 0 0" />
+      <origin xyz=".449 0.1825 0.005" rpy="0 0 0" />
   </xacro:kitting_bin_1>
   <!--bin1_1_-->
   <xacro:kitting_bin_1 binname="bin1_1" parent="workspace_center" z_origin_offset="-.005">
-      <origin xyz=".2425 -0.2415 0.005" rpy="0 0 0" />
+      <origin xyz=".449 0.0575 0.005" rpy="0 0 0" />
   </xacro:kitting_bin_1>
   <!--bin1_4_-->
   <xacro:kitting_bin_1 binname="bin1_4" parent="workspace_center" z_origin_offset="-.005">
-      <origin xyz=".449 0.1825 0.005" rpy="0 0 0" />
+      <origin xyz=".449 -0.0675 0.005" rpy="0 0 0" />
   </xacro:kitting_bin_1>
   <!--bin1_5_-->
   <xacro:kitting_bin_1 binname="bin1_5" parent="workspace_center" z_origin_offset="-.005">
-      <origin xyz=".449 0.0575 0.005" rpy="0 0 0" />
-  </xacro:kitting_bin_1>
-  <!--bin1_7_-->
-  <xacro:kitting_bin_1 binname="bin1_7" parent="workspace_center" z_origin_offset="-.005">
-      <origin xyz=".449 -0.0675 0.005" rpy="0 0 0" />
-  </xacro:kitting_bin_1>
-  <!--bin1_8_-->
-  <xacro:kitting_bin_1 binname="bin1_8" parent="workspace_center" z_origin_offset="-.005">
       <origin xyz=".449 -0.1925 0.005" rpy="0 0 0" />
   </xacro:kitting_bin_1>
-  <!--bin1_6_-->
-  <xacro:kitting_bin_1 binname="bin1_6" parent="workspace_center" z_origin_offset="-.005">
+  <!--bin1_3_-->
+  <xacro:kitting_bin_1 binname="bin1_3" parent="workspace_center" z_origin_offset="-.005">
       <origin xyz=".449 -0.3175 0.005" rpy="0 0 0" />
   </xacro:kitting_bin_1>

Commit message: Kitting trial 2
We went in blind and the order file did not include the washers (a_bot locks up)

File: o2as_scene_description/urdf/kitting_bins.xacro (robot description, xacro)
@@ -24,42 +24,42 @@
  <xacro:property name="set2_y" value="0.245"/>
  <xacro:property name="set2_z" value="0"/>
- <!--bin3_1_-->
-  <xacro:kitting_bin_3 binname="bin3_1" parent="workspace_center" z_origin_offset="-.004">
-      <origin xyz=".2425 0.199 0.004" rpy="0 0 0" />
-  </xacro:kitting_bin_3>
+ <!--bin2_5_-->
+  <xacro:kitting_bin_2 binname="bin2_5" parent="workspace_center" z_origin_offset="-.008">
+      <origin xyz=".2425 0.239 0.008" rpy="0 0 0" />
+  </xacro:kitting_bin_2>
   <!--bin2_4_-->
   <xacro:kitting_bin_2 binname="bin2_4" parent="workspace_center" z_origin_offset="-.008">
-      <origin xyz=".2425 0.047 0.008" rpy="0 0 0" />
+      <origin xyz=".2425 0.127 0.008" rpy="0 0 0" />
+  </xacro:kitting_bin_2>
+  <!--bin2_1_-->
+  <xacro:kitting_bin_2 binname="bin2_1" parent="workspace_center" z_origin_offset="-.008">
+      <origin xyz=".2425 0.015 0.008" rpy="0 0 0" />
   </xacro:kitting_bin_2>
   <!--bin2_3_-->
   <xacro:kitting_bin_2 binname="bin2_3" parent="workspace_center" z_origin_offset="-.008">
-      <origin xyz=".2425 -0.065 0.008" rpy="0 0 0" />
+      <origin xyz=".2425 -0.097 0.008" rpy="0 0 0" />
   </xacro:kitting_bin_2>
   <!--bin2_2_-->
   <xacro:kitting_bin_2 binname="bin2_2" parent="workspace_center" z_origin_offset="-.008">
-      <origin xyz=".2425 -0.177 0.008" rpy="0 0 0" />
+      <origin xyz=".2425 -0.209 0.008" rpy="0 0 0" />
   </xacro:kitting_bin_2>
-  <!--bin2_1_-->
-  <xacro:kitting_bin_2 binname="bin2_1" parent="workspace_center" z_origin_offset="-.008">
-      <origin xyz=".2425 -0.289 0.008" rpy="0 0 0" />
-  </xacro:kitting_bin_2>
+  <!--bin1_3_-->
+  <xacro:kitting_bin_1 binname="bin1_3" parent="workspace_center" z_origin_offset="-.005">
+      <origin xyz=".449 0.1825 0.005" rpy="0 0 0" />
+  </xacro:kitting_bin_1>
+  <!--bin1_4_-->
+  <xacro:kitting_bin_1 binname="bin1_4" parent="workspace_center" z_origin_offset="-.005">
+      <origin xyz=".449 0.0575 0.005" rpy="0 0 0" />
+  </xacro:kitting_bin_1>
+  <!--bin1_5_-->
+  <xacro:kitting_bin_1 binname="bin1_5" parent="workspace_center" z_origin_offset="-.005">
+      <origin xyz=".449 -0.0675 0.005" rpy="0 0 0" />
+  </xacro:kitting_bin_1>
   <!--bin1_2_-->
   <xacro:kitting_bin_1 binname="bin1_2" parent="workspace_center" z_origin_offset="-.005">
-      <origin xyz=".449 0.1825 0.005" rpy="0 0 0" />
+      <origin xyz=".449 -0.1925 0.005" rpy="0 0 0" />
   </xacro:kitting_bin_1>
   <!--bin1_1_-->
   <xacro:kitting_bin_1 binname="bin1_1" parent="workspace_center" z_origin_offset="-.005">
-      <origin xyz=".449 0.0575 0.005" rpy="0 0 0" />
-  </xacro:kitting_bin_1>
-  <!--bin1_4_-->
-  <xacro:kitting_bin_1 binname="bin1_4" parent="workspace_center" z_origin_offset="-.005">
-      <origin xyz=".449 -0.0675 0.005" rpy="0 0 0" />
-  </xacro:kitting_bin_1>
-  <!--bin1_5_-->
-  <xacro:kitting_bin_1 binname="bin1_5" parent="workspace_center" z_origin_offset="-.005">
-      <origin xyz=".449 -0.1925 0.005" rpy="0 0 0" />
-  </xacro:kitting_bin_1>
-  <!--bin1_3_-->
-  <xacro:kitting_bin_1 binname="bin1_3" parent="workspace_center" z_origin_offset="-.005">
       <origin xyz=".449 -0.3175 0.005" rpy="0 0 0" />
   </xacro:kitting_bin_1>
