Commit message: Add relay, calibration, various fixes

File: o2as_scene_description/urdf/robotiq_b_bot_gripper.urdf.xacro (robot description, xacro)
@@ -30,5 +30,5 @@
       <parent link="${prefix}robotiq_85_tip_link"/>
       <child link="${prefix}screw_tool_m3_tip_link"/>
-      <origin rpy="0.0 ${pi/2} 0.0" xyz="${dx} 0.0 -0.112 "/>
+      <origin rpy="0.0 ${pi/2} 0.0" xyz="${dx} 0.0 -0.132 "/>
     </joint>
     <link name="${prefix}screw_tool_m3_tip_link"/>
@@ -42,5 +42,5 @@
       <parent link="${prefix}robotiq_85_tip_link"/>
       <child link="${prefix}suction_tool_tip_link"/>
-      <origin rpy="0.0 ${pi/2} 0.0" xyz="${dx+.008} 0.0 -0.131 "/>
+      <origin rpy="0.0 ${pi/2} 0.0" xyz="${dx+.02} 0.0 -0.131 "/>
     </joint>
     <link name="${prefix}suction_tool_tip_link"/>

File: o2as_scene_description/urdf/robotiq_c_bot_gripper.urdf.xacro (robot description, xacro)
@@ -29,5 +29,5 @@
       <parent link="${prefix}robotiq_85_tip_rotation_helper_link"/>
       <child link="${prefix}screw_tool_m3_tip_link"/>
-      <origin rpy="0.0 0 0" xyz="0.112 0 .006"/>
+      <origin rpy="0.0 0 0" xyz="0.132 0 .006"/>
     </joint>
     <link name="${prefix}screw_tool_m3_tip_link"/>

File: o2as_scene_description/urdf/screw_tools.xacro (robot description, xacro)
@@ -126,5 +126,5 @@
     <parent link="screw_tool_holder" />
     <child link="suction_tool_link" />
-    <origin xyz="-0.355 ${tool_offset} 0.004" rpy="0.0 0.0 0.0" />
+    <origin xyz="-0.355 ${tool_offset - .025} 0.004" rpy="0.0 0.0 0.0" />
   </joint>
   <link name="screw_tool_m4_link">

Commit message: Add calibration methods, m3 tool update

File: o2as_scene_description/urdf/robotiq_b_bot_gripper.urdf.xacro (robot description, xacro)
@@ -30,5 +30,5 @@
       <parent link="${prefix}robotiq_85_tip_link"/>
       <child link="${prefix}screw_tool_m3_tip_link"/>
-      <origin rpy="0.0 ${pi/2} 0.0" xyz="${dx} 0.0 -0.132 "/>
+      <origin rpy="0.0 ${pi/2} 0.0" xyz="${dx-.004} 0.0 -0.125 "/>
     </joint>
     <link name="${prefix}screw_tool_m3_tip_link"/>

Commit message: WIP: Taskboard tests and part 7
Everything except 7 works

File: o2as_scene_description/urdf/robotiq_b_bot_gripper.urdf.xacro (robot description, xacro)
@@ -12,5 +12,5 @@
       <parent link="${prefix}robotiq_85_tip_link"/>
       <child link="${prefix}screw_tool_m6_tip_link"/>
-      <origin rpy="0.0 ${pi/2} 0.0" xyz="${dx} 0.0 -0.12 "/>
+      <origin rpy="0.0 ${pi/2} 0.0" xyz="${dx} 0.0 -0.135 "/>
     </joint>
     <link name="${prefix}screw_tool_m6_tip_link"/>

File: o2as_scene_description/urdf/robotiq_c_bot_gripper.urdf.xacro (robot description, xacro)
@@ -24,5 +24,5 @@
       <parent link="${prefix}robotiq_85_tip_45deg_helper_link"/>
       <child link="${prefix}screw_tool_m6_tip_link"/>
-      <origin rpy="0.0 0 0" xyz="0.12 0 .006"/>
+      <origin rpy="0.0 0 0" xyz="0.135 0 .006"/>
     </joint>
     <link name="${prefix}screw_tool_m6_tip_link"/>

Commit message: Dirty offset fix for strange behavior of m4 tool

File: o2as_scene_description/urdf/robotiq_b_bot_gripper.urdf.xacro (robot description, xacro)
@@ -24,5 +24,5 @@
       <parent link="${prefix}robotiq_85_tip_link"/>
       <child link="${prefix}screw_tool_m4_tip_link"/>
-      <origin rpy="0.0 ${pi/2} 0.0" xyz="${dx} 0.0 -0.146 "/>
+      <origin rpy="0.0 ${pi/2} 0.0" xyz="${dx-.002} 0.0 -0.146 "/>
     </joint>
     <link name="${prefix}screw_tool_m4_tip_link"/>
