Commit message: Add auxiliary frames in kitting tray.

File: o2as_scene_description/urdf/kitting_tray_with_partitions.xacro (robot description, xacro)
@@ -93,5 +93,5 @@
       <parent link="${trayname}" />
       <child link = "${trayname}_partition_1"/>
-      <origin rpy="0.0 0.0 0.0" xyz="0.05 0.05 0.02"/>
+      <origin rpy="0.0 0.0 0.0" xyz="0.06 0.05 0.02"/>
     </joint>
     <link name="${trayname}_partition_1"/>
@@ -99,5 +99,5 @@
       <parent link="${trayname}" />
       <child link = "${trayname}_partition_2"/>
-      <origin rpy="0.0 0.0 0.0" xyz="0.15 0.05 0.02"/>
+      <origin rpy="0.0 0.0 0.0" xyz="0.16 0.05 0.02"/>
     </joint>
     <link name="${trayname}_partition_2"/>
@@ -105,7 +105,19 @@
       <parent link="${trayname}" />
       <child link = "${trayname}_partition_3"/>
-      <origin rpy="0.0 0.0 0.0" xyz="0.105 0.15 0.02"/>
+      <origin rpy="0.0 0.0 0.0" xyz="0.11 0.16 0.02"/>
     </joint>
     <link name="${trayname}_partition_3"/>
+    <joint name="${trayname}_partition_4" type="fixed">
+      <parent link="${trayname}" />
+      <child link = "${trayname}_partition_4"/>
+      <origin rpy="0.0 0.0 0.0" xyz="0.07 0.26 0.02"/>
+    </joint>
+    <link name="${trayname}_partition_4"/>
+    <joint name="${trayname}_partition_5" type="fixed">
+      <parent link="${trayname}" />
+      <child link = "${trayname}_partition_5"/>
+      <origin rpy="0.0 0.0 0.0" xyz="0.16 0.26 0.02"/>
+    </joint>
+    <link name="${trayname}_partition_5"/>
   </xacro:macro>
   <!-- ========== The tray with the screws and small parts -->
@@ -122,5 +134,26 @@
     <!-- ========== The extra frames to place and pick items are defined below -->
     <xacro:auxiliary_frame parent="${trayname}" framename="partition_1">
-      <origin rpy="0.0 0.0 0.0" xyz="0.05 0.15 0.02"/>
+      <origin rpy="0.0 0.0 0.0" xyz="0.04 0.16 0.02"/>
+    </xacro:auxiliary_frame>
+    <xacro:auxiliary_frame parent="${trayname}" framename="partition_2">
+      <origin rpy="0.0 0.0 0.0" xyz="0.11 0.13 0.02"/>
+    </xacro:auxiliary_frame>
+    <xacro:auxiliary_frame parent="${trayname}" framename="partition_3">
+      <origin rpy="0.0 0.0 0.0" xyz="0.17 0.13 0.02"/>
+    </xacro:auxiliary_frame>
+    <xacro:auxiliary_frame parent="${trayname}" framename="partition_4">
+      <origin rpy="0.0 0.0 0.0" xyz="0.11 0.19 0.02"/>
+    </xacro:auxiliary_frame>
+    <xacro:auxiliary_frame parent="${trayname}" framename="partition_5">
+      <origin rpy="0.0 0.0 0.0" xyz="0.17 0.19 0.02"/>
+    </xacro:auxiliary_frame>
+    <xacro:auxiliary_frame parent="${trayname}" framename="partition_6">
+      <origin rpy="0.0 0.0 0.0" xyz="0.04 0.25 0.02"/>
+    </xacro:auxiliary_frame>
+    <xacro:auxiliary_frame parent="${trayname}" framename="partition_7">
+      <origin rpy="0.0 0.0 0.0" xyz="0.11 0.25 0.02"/>
+    </xacro:auxiliary_frame>
+    <xacro:auxiliary_frame parent="${trayname}" framename="partition_8">
+      <origin rpy="0.0 0.0 0.0" xyz="0.17 0.25 0.02"/>
     </xacro:auxiliary_frame>
     <!-- TODO: Insert the rest and fine tune -->

Commit message: Fixed kitting tray (includes screw holders) without auxiliary frames.

File: o2as_scene_description/urdf/kitting_tray_with_partitions.xacro (robot description, xacro)
@@ -93,5 +93,5 @@
       <parent link="${trayname}" />
       <child link = "${trayname}_partition_1"/>
-      <origin rpy="0.0 0.0 0.0" xyz="0.05 0.05 0.02"/>
+      <origin rpy="0.0 0.0 0.0" xyz="0.06 0.05 0.02"/>
     </joint>
     <link name="${trayname}_partition_1"/>
@@ -99,5 +99,5 @@
       <parent link="${trayname}" />
       <child link = "${trayname}_partition_2"/>
-      <origin rpy="0.0 0.0 0.0" xyz="0.15 0.05 0.02"/>
+      <origin rpy="0.0 0.0 0.0" xyz="0.16 0.05 0.02"/>
     </joint>
     <link name="${trayname}_partition_2"/>
@@ -105,7 +105,19 @@
       <parent link="${trayname}" />
       <child link = "${trayname}_partition_3"/>
-      <origin rpy="0.0 0.0 0.0" xyz="0.105 0.15 0.02"/>
+      <origin rpy="0.0 0.0 0.0" xyz="0.11 0.16 0.02"/>
     </joint>
     <link name="${trayname}_partition_3"/>
+    <joint name="${trayname}_partition_4" type="fixed">
+      <parent link="${trayname}" />
+      <child link = "${trayname}_partition_4"/>
+      <origin rpy="0.0 0.0 0.0" xyz="0.07 0.26 0.02"/>
+    </joint>
+    <link name="${trayname}_partition_4"/>
+    <joint name="${trayname}_partition_5" type="fixed">
+      <parent link="${trayname}" />
+      <child link = "${trayname}_partition_5"/>
+      <origin rpy="0.0 0.0 0.0" xyz="0.16 0.26 0.02"/>
+    </joint>
+    <link name="${trayname}_partition_5"/>
   </xacro:macro>
   <!-- ========== The tray with the screws and small parts -->
@@ -115,15 +127,36 @@
     </xacro:kitting_tray>
     <xacro:tray_contents trayname="${trayname}" contents="divider2">
-      <origin xyz="${tray_width/2 + mesh_offset_x - 0.095} ${tray_length/2 + mesh_offset_y +0.14} ${dividers_z_offset}" rpy="0 0 ${-pi/2}"/>
+      <origin xyz="${tray_width/2 + mesh_offset_x + 0.095} ${tray_length/2 + mesh_offset_y -0.14} ${dividers_z_offset}" rpy="${pi} ${pi} ${-pi/2}"/>
     </xacro:tray_contents>
     <xacro:tray_contents trayname="${trayname}" contents="screw_holder">
-      <origin xyz="${tray_width/2 + mesh_offset_x - 0.095} ${tray_length/2 + mesh_offset_y -0.05} ${dividers_z_offset}" rpy="0 0 ${-pi/2}"/>
+      <origin xyz="${tray_width/2 + mesh_offset_x + 0.095} ${tray_length/2 + mesh_offset_y +0.05} ${dividers_z_offset}" rpy="${pi} ${pi} ${-pi/2}"/>
     </xacro:tray_contents>
     <!-- ========== The extra frames to place and pick items are defined below -->
-    <xacro:auxiliary_frame parent="${trayname}" framename="partition_1">
-      <origin rpy="0.0 0.0 0.0" xyz="0.05 0.15 0.02"/>
-    </xacro:auxiliary_frame>
+    <!-- <xacro:auxiliary_frame parent="${trayname}" framename="partition_1">
+      <origin rpy="0.0 0.0 0.0" xyz="0.04 0.16 0.02"/>
+    </xacro:auxiliary_frame>
+    <xacro:auxiliary_frame parent="${trayname}" framename="partition_2">
+      <origin rpy="0.0 0.0 0.0" xyz="0.11 0.13 0.02"/>
+    </xacro:auxiliary_frame>
+    <xacro:auxiliary_frame parent="${trayname}" framename="partition_3">
+      <origin rpy="0.0 0.0 0.0" xyz="0.17 0.13 0.02"/>
+    </xacro:auxiliary_frame>
+    <xacro:auxiliary_frame parent="${trayname}" framename="partition_4">
+      <origin rpy="0.0 0.0 0.0" xyz="0.11 0.19 0.02"/>
+    </xacro:auxiliary_frame>
+    <xacro:auxiliary_frame parent="${trayname}" framename="partition_5">
+      <origin rpy="0.0 0.0 0.0" xyz="0.17 0.19 0.02"/>
+    </xacro:auxiliary_frame>
+    <xacro:auxiliary_frame parent="${trayname}" framename="partition_6">
+      <origin rpy="0.0 0.0 0.0" xyz="0.04 0.25 0.02"/>
+    </xacro:auxiliary_frame>
+    <xacro:auxiliary_frame parent="${trayname}" framename="partition_7">
+      <origin rpy="0.0 0.0 0.0" xyz="0.11 0.25 0.02"/>
+    </xacro:auxiliary_frame>
+    <xacro:auxiliary_frame parent="${trayname}" framename="partition_8">
+      <origin rpy="0.0 0.0 0.0" xyz="0.17 0.25 0.02"/>
+    </xacro:auxiliary_frame> -->
     <!-- TODO: Insert the rest and fine tune -->
-    <xacro:property name="m4_x_0" value="0.18"/>
+    <!-- <xacro:property name="m4_x_0" value="0.18"/>
     <xacro:property name="m4_x_delta" value="-0.03"/>
     <xacro:property name="m4_y_0" value="0.03"/>
@@ -179,5 +212,5 @@
     <xacro:auxiliary_frame parent="${trayname}" framename="screw_m3_6">
       <origin xyz="${m3_x_0 + m3_x_delta*1} ${m3_y_0 + m3_y_delta*2} ${m3_z_0}" rpy="0 ${pi/2} 0" />
-    </xacro:auxiliary_frame>
+    </xacro:auxiliary_frame> -->
   </xacro:macro>
 </robot>

Commit message: Add auxiliary frames in screw holder.

File: o2as_scene_description/urdf/kitting_tray_with_partitions.xacro (robot description, xacro)
@@ -158,8 +158,8 @@
     </xacro:auxiliary_frame>
     <!-- TODO: Insert the rest and fine tune -->
-    <!-- <xacro:property name="m4_x_0" value="0.18"/>
-    <xacro:property name="m4_x_delta" value="-0.03"/>
-    <xacro:property name="m4_y_0" value="0.03"/>
-    <xacro:property name="m4_y_delta" value="0.03"/>
+    <xacro:property name="m4_x_0" value="0.04"/>
+    <xacro:property name="m4_x_delta" value="0.03"/>
+    <xacro:property name="m4_y_0" value="0.275"/>
+    <xacro:property name="m4_y_delta" value="-0.03"/>
     <xacro:property name="m4_z_0" value="0.05"/>
     <xacro:auxiliary_frame parent="${trayname}" framename="screw_m4_1">
@@ -190,8 +190,8 @@
       <origin xyz="${m4_x_0 + m4_x_delta*2} ${m4_y_0 + m4_y_delta*2} ${m4_z_0}" rpy="0 ${pi/2} 0" />
     </xacro:auxiliary_frame>
-    <xacro:property name="m3_x_0" value="0.08"/>
-    <xacro:property name="m3_x_delta" value="-0.03"/>
-    <xacro:property name="m3_y_0" value="0.03"/>
-    <xacro:property name="m3_y_delta" value="0.03"/>
+    <xacro:property name="m3_x_0" value="0.14"/>
+    <xacro:property name="m3_x_delta" value="0.03"/>
+    <xacro:property name="m3_y_0" value="0.275"/>
+    <xacro:property name="m3_y_delta" value="-0.03"/>
     <xacro:property name="m3_z_0" value="0.05"/>
     <xacro:auxiliary_frame parent="${trayname}" framename="screw_m3_1">
@@ -212,5 +212,5 @@
     <xacro:auxiliary_frame parent="${trayname}" framename="screw_m3_6">
       <origin xyz="${m3_x_0 + m3_x_delta*1} ${m3_y_0 + m3_y_delta*2} ${m3_z_0}" rpy="0 ${pi/2} 0" />
-    </xacro:auxiliary_frame> -->
+    </xacro:auxiliary_frame>
   </xacro:macro>
 </robot>

Commit message: Improve screw/changeTool actions

File: o2as_scene_description/urdf/kitting_tray_with_partitions.xacro (robot description, xacro)
@@ -160,5 +160,5 @@
     <xacro:property name="m4_y_0" value="0.275"/>
     <xacro:property name="m4_y_delta" value="-0.03"/>
-    <xacro:property name="m4_z_0" value="0.05"/>
+    <xacro:property name="m4_z_0" value="0.025"/>
     <xacro:auxiliary_frame parent="${trayname}" framename="screw_m4_1">
       <origin xyz="${m4_x_0 + m4_x_delta*0} ${m4_y_0 + m4_y_delta*0} ${m4_z_0}" rpy="0 ${pi/2} 0" />
@@ -192,5 +192,5 @@
     <xacro:property name="m3_y_0" value="0.275"/>
     <xacro:property name="m3_y_delta" value="-0.03"/>
-    <xacro:property name="m3_z_0" value="0.05"/>
+    <xacro:property name="m3_z_0" value="0.025"/>
     <xacro:auxiliary_frame parent="${trayname}" framename="screw_m3_1">
       <origin xyz="${m3_x_0 + m3_x_delta*0} ${m3_y_0 + m3_y_delta*0} ${m3_z_0}" rpy="0 ${pi/2} 0" />

Commit message: Update scene

File: o2as_scene_description/urdf/kitting_tray_with_partitions.xacro (robot description, xacro)
@@ -160,5 +160,5 @@
     <xacro:property name="m4_y_0" value="0.275"/>
     <xacro:property name="m4_y_delta" value="-0.03"/>
-    <xacro:property name="m4_z_0" value="0.025"/>
+    <xacro:property name="m4_z_0" value="0.035"/>
     <xacro:auxiliary_frame parent="${trayname}" framename="screw_m4_1">
       <origin xyz="${m4_x_0 + m4_x_delta*0} ${m4_y_0 + m4_y_delta*0} ${m4_z_0}" rpy="0 ${pi/2} 0" />
@@ -192,5 +192,5 @@
     <xacro:property name="m3_y_0" value="0.275"/>
     <xacro:property name="m3_y_delta" value="-0.03"/>
-    <xacro:property name="m3_z_0" value="0.025"/>
+    <xacro:property name="m3_z_0" value="0.035"/>
     <xacro:auxiliary_frame parent="${trayname}" framename="screw_m3_1">
       <origin xyz="${m3_x_0 + m3_x_delta*0} ${m3_y_0 + m3_y_delta*0} ${m3_z_0}" rpy="0 ${pi/2} 0" />

File: o2as_scene_description/urdf/robotiq_b_bot_gripper.urdf.xacro (robot description, xacro)
@@ -18,5 +18,5 @@
       <parent link="${prefix}robotiq_85_tip_link"/>
       <child link="${prefix}screw_tool_m4_tip_link"/>
-      <origin rpy="0.0 ${pi/2} 0.0" xyz="${dx} 0.0 -0.13 "/>
+      <origin rpy="0.0 ${pi/2} 0.0" xyz="${dx} 0.0 -0.146 "/>
     </joint>
     <link name="${prefix}screw_tool_m4_tip_link"/>

File: o2as_scene_description/urdf/robotiq_c_bot_gripper.urdf.xacro (robot description, xacro)
@@ -23,5 +23,5 @@
       <parent link="${prefix}robotiq_85_tip_rotation_helper_link"/>
       <child link="${prefix}screw_tool_m4_tip_link"/>
-      <origin rpy="0.0 0 0" xyz="0.13 0 .006"/>
+      <origin rpy="0.0 0 0" xyz="0.151 0 .006"/>
     </joint>
     <link name="${prefix}screw_tool_m4_tip_link"/>

Commit message: Add placeScrew function for the kitting task

File: o2as_scene_description/urdf/kitting_tray_with_partitions.xacro (robot description, xacro)
@@ -160,5 +160,5 @@
     <xacro:property name="m4_y_0" value="0.275"/>
     <xacro:property name="m4_y_delta" value="-0.03"/>
-    <xacro:property name="m4_z_0" value="0.035"/>
+    <xacro:property name="m4_z_0" value="0.025"/>
     <xacro:auxiliary_frame parent="${trayname}" framename="screw_m4_1">
       <origin xyz="${m4_x_0 + m4_x_delta*0} ${m4_y_0 + m4_y_delta*0} ${m4_z_0}" rpy="0 ${pi/2} 0" />
@@ -192,5 +192,5 @@
     <xacro:property name="m3_y_0" value="0.275"/>
     <xacro:property name="m3_y_delta" value="-0.03"/>
-    <xacro:property name="m3_z_0" value="0.035"/>
+    <xacro:property name="m3_z_0" value="0.025"/>
     <xacro:auxiliary_frame parent="${trayname}" framename="screw_m3_1">
       <origin xyz="${m3_x_0 + m3_x_delta*0} ${m3_y_0 + m3_y_delta*0} ${m3_z_0}" rpy="0 ${pi/2} 0" />

File: o2as_scene_description/urdf/screw_feeder.xacro (robot description, xacro)
@@ -74,5 +74,5 @@
     <!-- <origin rpy="0.0 0 0.0" xyz="${length-.01} ${width/2} ${height/2 + .02}"/> -->
     <!-- <origin rpy="0.0 ${pi/2} 0.0" xyz="${-height/2 - .02} ${width/2} ${length-.01}"/> -->
-    <origin rpy="0.0 ${pi/2} 0.0" xyz="${length-.01} ${width/2} ${height/2 + .02}"/>
+    <origin rpy="0.0 ${pi/2} 0.0" xyz="${length-.01} ${width/2} ${height/2}"/>
   </joint>
   <link name="${feedername}_outlet_link"/>

Commit message: Move pin to corner, reset screw count

File: o2as_scene_description/urdf/kitting_tray_with_partitions.xacro (robot description, xacro)
@@ -162,5 +162,5 @@
     </xacro:auxiliary_frame>
     <xacro:auxiliary_frame parent="${trayname}_partition_2" framename="pickup">
-      <origin rpy="0.0 0.0 0.0" xyz="0 0 0.02"/>
+      <origin rpy="0.0 0.0 0.0" xyz="${-partition_length/2 + .0015} ${-partition_width/2 + .0015} 0"/>
     </xacro:auxiliary_frame>
     <xacro:auxiliary_frame parent="${trayname}_partition_3" framename="pickup">

Commit message: Assembly trial 2

File: o2as_scene_description/urdf/kitting_tray_with_partitions.xacro (robot description, xacro)
@@ -189,5 +189,5 @@
     <xacro:property name="m4_y_0" value="0.275"/>
     <xacro:property name="m4_y_delta" value="-0.03"/>
-    <xacro:property name="m4_z_0" value="0.025"/>
+    <xacro:property name="m4_z_0" value="0.021"/>
     <xacro:auxiliary_frame parent="${trayname}" framename="screw_m4_1">
       <origin xyz="${m4_x_0 + m4_x_delta*0} ${m4_y_0 + m4_y_delta*0} ${m4_z_0}" rpy="0 ${pi/2} 0" />
@@ -221,5 +221,5 @@
     <xacro:property name="m3_y_0" value="0.275"/>
     <xacro:property name="m3_y_delta" value="-0.03"/>
-    <xacro:property name="m3_z_0" value="0.025"/>
+    <xacro:property name="m3_z_0" value="0.021"/>
     <xacro:auxiliary_frame parent="${trayname}" framename="screw_m3_1">
       <origin xyz="${m3_x_0 + m3_x_delta*0} ${m3_y_0 + m3_y_delta*0} ${m3_z_0}" rpy="0 ${pi/2} 0" />
