Commit message: Improved INFO message of o2as_phoxi_camera.

File: o2as_scene_description/urdf/calibration_scene.xacro (robot description, xacro)
@@ -8,9 +8,9 @@
   <!--   <origin xyz="0.08 0.00 0.065" rpy="0 0 0"/> -->
   <!-- </xacro:o2as_ar_marker> -->
-  <!-- <xacro:o2as_ar_marker prefix="b_bot_" -->
-  <!-- 			parent="b_bot_dual_suction_gripper_base_link" -->
-  <!-- 			marker_id="26"> -->
-  <!--   <origin xyz="0.063 0.0 0.0215" rpy="0 0 0"/> -->
-  <!-- </xacro:o2as_ar_marker> -->
+  <xacro:o2as_ar_marker prefix="b_bot_"
+  			parent="b_bot_dual_suction_gripper_base_link"
+  			marker_id="26">
+    <origin xyz="0.063 0.0 0.0215" rpy="0 0 0"/>
+  </xacro:o2as_ar_marker>
   <!-- <xacro:o2as_ar_marker prefix="b_bot_" -->
   <!-- 			parent="b_bot_single_suction_gripper_base_link" -->
@@ -18,9 +18,9 @@
   <!--   <origin xyz="0.063 0.0 0.0215" rpy="0 0 0"/> -->
   <!-- </xacro:o2as_ar_marker> -->
-  <xacro:o2as_ar_marker prefix="b_bot_"
-			parent="b_bot_robotiq_85_tip_link"
-			marker_id="26">
-    <origin xyz="0.0 0.0 0.0185" rpy="0 0 0"/>
-  </xacro:o2as_ar_marker>
+  <!-- <xacro:o2as_ar_marker prefix="b_bot_" -->
+  <!-- 			parent="b_bot_robotiq_85_tip_link" -->
+  <!-- 			marker_id="26"> -->
+  <!--   <origin xyz="0.0 0.0 0.0185" rpy="0 0 0"/> -->
+  <!-- </xacro:o2as_ar_marker> -->
   <xacro:o2as_ar_marker prefix="c_bot_"
 			parent="c_bot_robotiq_85_tip_link"

File: o2as_scene_description/urdf/o2as_base_scene.urdf.xacro (robot description, xacro)
@@ -115,11 +115,11 @@
   </xacro:InnerOnlyGripper>
   <!-- spawn and attach dual suction grippers -->
-  <xacro:include filename="$(find o2as_scene_description)/urdf/dual_suction_gripper.urdf.xacro" />
-  <xacro:dual_suction_gripper_o2as prefix="b_bot_" parent = "b_bot_ee_link">
-    <origin xyz="0 0 0" rpy="0 0 0"/>
-  </xacro:dual_suction_gripper_o2as>
+  <!-- <xacro:include filename="$(find o2as_scene_description)/urdf/dual_suction_gripper.urdf.xacro" /> -->
+  <!-- <xacro:dual_suction_gripper_o2as prefix="b_bot_" parent = "b_bot_ee_link"> -->
+  <!--   <origin xyz="0 0 0" rpy="0 0 0"/> -->
+  <!-- </xacro:dual_suction_gripper_o2as> -->
   <!-- spawn and attach dual robotiq 85 grippers -->
-  <!-- <xacro:include filename="$(find o2as_scene_description)/urdf/robotiq_b_bot_gripper.urdf.xacro" /> -->
-  <!-- <xacro:o2as_b_bot_gripper prefix="b_bot_" parent = "b_bot_ee_link" /> -->
+  <xacro:include filename="$(find o2as_scene_description)/urdf/robotiq_b_bot_gripper.urdf.xacro" />
+  <xacro:o2as_b_bot_gripper prefix="b_bot_" parent = "b_bot_ee_link" />
   <xacro:include filename="$(find o2as_scene_description)/urdf/robotiq_c_bot_gripper.urdf.xacro" />
   <xacro:o2as_c_bot_gripper prefix="c_bot_" parent = "c_bot_ee_link"/>
@@ -155,9 +155,9 @@
   <!--   <origin xyz="0.08 0.00 0.065" rpy="0 0 0"/> -->
   <!-- </xacro:o2as_ar_marker> -->
-  <xacro:o2as_ar_marker prefix="b_bot_"
-  			parent="b_bot_dual_suction_gripper_base_link"
-  			marker_id="26">
-    <origin xyz="0.063 0.0 0.0215" rpy="0 0 0"/>
-  </xacro:o2as_ar_marker>
+  <!-- <xacro:o2as_ar_marker prefix="b_bot_" -->
+  <!-- 			parent="b_bot_dual_suction_gripper_base_link" -->
+  <!-- 			marker_id="26"> -->
+  <!--   <origin xyz="0.063 0.0 0.0215" rpy="0 0 0"/> -->
+  <!-- </xacro:o2as_ar_marker> -->
   <!-- <xacro:o2as_ar_marker prefix="b_bot_" -->
   <!-- 			parent="b_bot_single_suction_gripper_base_link" -->
@@ -165,9 +165,9 @@
   <!--   <origin xyz="0.063 0.0 0.0215" rpy="0 0 0"/> -->
   <!-- </xacro:o2as_ar_marker> -->
-  <!-- <xacro:o2as_ar_marker prefix="b_bot_" -->
-  <!-- 			parent="b_bot_robotiq_85_tip_link" -->
-  <!-- 			marker_id="26"> -->
-  <!--   <origin xyz="0.0 0.0 0.0185" rpy="0 0 0"/> -->
-  <!-- </xacro:o2as_ar_marker> -->
+  <xacro:o2as_ar_marker prefix="b_bot_"
+  			parent="b_bot_robotiq_85_tip_link"
+  			marker_id="26">
+    <origin xyz="0.0 0.0 0.0185" rpy="0 0 0"/>
+  </xacro:o2as_ar_marker>
   <xacro:o2as_ar_marker prefix="c_bot_"
 			parent="c_bot_robotiq_85_tip_link"

Commit message: Improved error messages.

File: o2as_scene_description/urdf/calibration_scene.xacro (robot description, xacro)
@@ -1,4 +1,4 @@
 <?xml version="1.0"?>
-<robot xmlns:xacro="http://www.ros.org/wiki/xacro" name="kitting_scene">
+<robot xmlns:xacro="http://www.ros.org/wiki/xacro" name="calibration_scene">
   <!-- spawn and attach AR markers -->
   <xacro:include filename="$(find o2as_gazebo)/urdf/o2as_ar_marker.urdf.xacro"/>

File: o2as_scene_description/urdf/o2as_base_scene.urdf.xacro (robot description, xacro)
@@ -2,12 +2,11 @@
 <robot xmlns:xacro="http://www.ros.org/wiki/xacro"
        name="o2as_base_scene" >
-  <!-- Calibration from 20 August 2018 -->
+  <!-- Calibration from 12 October 2018 -->
   <!-- Calibration help: If the robot is not moving far enough to the calibration point, increase these distances -->
   <xacro:property name="a_bot_x" value="-0.01"/>
   <xacro:property name="a_bot_y" value="-0.5"/>
-  <xacro:property name="b_bot_x" value="-0.009"/>
-  <xacro:property name="b_bot_y" value="0.503"/>
-  <xacro:property name="b_bot_theta" value="-3.12832815"/>
-  <!-- The above is 0.76 degrees away from pi (Sep 17; not perfect) -->
+  <xacro:property name="b_bot_x" value="-0.008"/>
+  <xacro:property name="b_bot_y" value="0.50"/>
+  <xacro:property name="b_bot_theta" value="-3.14"/>
   <xacro:property name="c_bot_x" value="-0.499"/>
   <xacro:property name="c_bot_y" value="0.0"/>
@@ -25,4 +24,6 @@
   <!-- <xacro:include filename="$(find o2as_scene_description)/urdf/kitting_scene.xacro" /> -->
   <!-- <xacro:include filename="$(find o2as_scene_description)/urdf/assembly_scene.xacro" /> -->
+  <!-- <xacro:include filename="$(find o2as_scene_description)/urdf/calibration_scene.xacro" /> -->
+  <!-- <xacro:include filename="$(find o2as_scene_description)/urdf/assembly_new_parts_scene.xacro" /> -->
   <!-- Robot bases -->
   <!-- Putting these at height 0.0 makes them intersect with the ground, so they are elevated. -->
@@ -59,12 +60,4 @@
   <!-- Screw holder & screw tool visual -->
   <xacro:include filename="$(find o2as_scene_description)/urdf/screw_tools.xacro" />
-  <!-- Feeders -->
-  <xacro:include filename="$(find o2as_scene_description)/urdf/screw_feeder.xacro" />
-  <xacro:screw_feeder feedername="m3_feeder" parent="c_bot_base_smfl">
-    <origin xyz=".66 -0.25 .065" rpy="0 0 ${pi/2}" />
-  </xacro:screw_feeder>
-  <xacro:screw_feeder feedername="m4_feeder" parent="c_bot_base_smfl">
-    <origin xyz=".52 -0.25 .065" rpy="0 0 ${pi/2}" />
-  </xacro:screw_feeder>
   <!-- robot arms -->
   <xacro:ur5_robot prefix="a_bot_" joint_limited="false"
@@ -106,26 +99,21 @@
   </joint>
   <!-- spawn and attach grippers -->
-  <!-- <xacro:include filename="$(find o2as_scene_description)/urdf/precision_gripper.xacro" />
-  <xacro:precision_gripper prefix="a_bot_"  grippername = "gripper" parent = "a_bot_tool0">
-    <origin xyz="0.0 0 0.04" rpy="0 ${pi/2} 0"/>
-  </xacro:precision_gripper> -->
   <xacro:include filename="$(find o2as_scene_description)/urdf/InnerOnlyGripper.xacro" />
   <xacro:InnerOnlyGripper prefix="a_bot_"  grippername = "gripper" parent = "a_bot_tool0">
     <origin xyz="0.0 0 0.0" rpy="0 0 0"/>
   </xacro:InnerOnlyGripper>
-  <!-- spawn and attach dual suction grippers -->
-  <!-- <xacro:include filename="$(find o2as_scene_description)/urdf/dual_suction_gripper.urdf.xacro" /> -->
-  <!-- <xacro:dual_suction_gripper_o2as prefix="b_bot_" parent = "b_bot_ee_link"> -->
-  <!--   <origin xyz="0 0 0" rpy="0 0 0"/> -->
-  <!-- </xacro:dual_suction_gripper_o2as> -->
-  <xacro:include filename="$(find o2as_scene_description)/urdf/single_suction_gripper.urdf.xacro" />
-  <xacro:single_suction_gripper_o2as prefix="b_bot_" parent = "b_bot_ee_link">
-    <origin xyz="0 0 0" rpy="0 0 0"/>
-  </xacro:single_suction_gripper_o2as>
   <!-- spawn and attach dual robotiq 85 grippers -->
-  <!-- <xacro:include filename="$(find o2as_scene_description)/urdf/robotiq_b_bot_gripper.urdf.xacro" /> -->
-  <!-- <xacro:o2as_b_bot_gripper prefix="b_bot_" parent = "b_bot_ee_link" /> -->
+  <xacro:include filename="$(find o2as_scene_description)/urdf/robotiq_b_bot_gripper.urdf.xacro" />
+  <xacro:o2as_b_bot_gripper prefix="b_bot_" parent = "b_bot_ee_link" />
   <xacro:include filename="$(find o2as_scene_description)/urdf/robotiq_c_bot_gripper.urdf.xacro" />
   <xacro:o2as_c_bot_gripper prefix="c_bot_" parent = "c_bot_ee_link"/>
+  <!-- Feeders -->
+  <xacro:include filename="$(find o2as_scene_description)/urdf/screw_feeder.xacro" />
+  <xacro:screw_feeder feedername="m3_feeder" parent="c_bot_base_smfl">
+    <origin xyz=".64 -0.25 .035" rpy="0 0 ${pi/2}" />
+  </xacro:screw_feeder>
+  <xacro:screw_feeder feedername="m4_feeder" parent="c_bot_base_smfl">
+    <origin xyz=".50 -0.25 .035" rpy="0 0 ${pi/2}" />
+  </xacro:screw_feeder>
   <!-- Add cameras -->
   <xacro:include filename="$(find o2as_realsense2_camera)/urdf/_d435.urdf.xacro" />
@@ -144,13 +132,24 @@
     <parent link="a_bot_wrist_2_link" />
     <child  link="a_bot_cam_holder_link" />
-    <origin xyz="0.0 -0.06 ${0.09465 + .13}" rpy="0.0 0.0 ${pi/2}" />
+    <origin xyz="0.04 -0.06 0.20" rpy="${12*pi/180} 0.0 ${pi/2}" />
   </joint>
   <xacro:sensor_d435 prefix="a_bot_" parent="a_bot_cam_holder_link">
     <origin xyz="0 0 0" rpy="0 0 0"/>
   </xacro:sensor_d435>
+  <link name="a_bot_camera_calibrated_frame_link" />
+  <joint name="a_bot_camera_calibrated_frame_joint" type="fixed">
+    <parent link="a_bot_wrist_2_link" />
+    <child  link="a_bot_camera_calibrated_frame_link" />
+    <origin xyz="-0.00584875065097 -0.0601140904909 0.190359410313" rpy="-1.631 -0.020 -0.016" />
+  </joint>
   <!-- <xacro:sensor_d435 prefix="d_bot_" parent="o2as_ground">
     <origin xyz="0 0 ${bots_z + 0.9}" rpy="0 ${pi/2} 0"/>
   </xacro:sensor_d435> -->
-  <!-- spawn and attach AR markers -->
+  <!-- Add PhoXi 3D scanners -->
+  <xacro:include filename="$(find o2as_scene_description)/urdf/phoxi_m_camera.urdf.xacro" />
+  <xacro:phoxi_m_camera prefix="a_" parent="o2as_ground">
+  <origin xyz="0.652663578768 -0.0142895785849 1.50687788672" rpy="${-161.381811856*pi/180} ${2.99567722105*pi/180} ${90.8962573459*pi/180}"/>
+  </xacro:phoxi_m_camera>
+  <!-- Add AR markers -->
   <xacro:include filename="$(find o2as_gazebo)/urdf/o2as_ar_marker.urdf.xacro"/>
   <xacro:o2as_ar_marker prefix="a_bot_"
@@ -164,17 +163,17 @@
   <!--   <origin xyz="0.063 0.0 0.0215" rpy="0 0 0"/> -->
   <!-- </xacro:o2as_ar_marker> -->
+  <!-- <xacro:o2as_ar_marker prefix="b_bot_" -->
+  <!-- 			parent="b_bot_single_suction_gripper_base_link" -->
+  <!-- 			marker_id="26"> -->
+  <!--   <origin xyz="0.063 0.0 0.0215" rpy="0 0 0"/> -->
+  <!-- </xacro:o2as_ar_marker> -->
   <xacro:o2as_ar_marker prefix="b_bot_"
-  			parent="b_bot_ee_link"
+  			parent="b_bot_robotiq_85_tip_link"
   			marker_id="26">
-    <origin xyz="0.063 0.0 0.0215" rpy="0 0 0"/>
+    <origin xyz="0.0 0.0 0.0185" rpy="0 0 0"/>
   </xacro:o2as_ar_marker>
-  <!-- <xacro:o2as_ar_marker prefix="b_bot_" -->
-  <!-- 			parent="b_bot_robotiq_85_tip_link" -->
-  <!-- 			marker_id="26"> -->
-  <!--   <origin xyz="0.0 0.0 0.0185" rpy="0 0 0"/> -->
-  <!-- </xacro:o2as_ar_marker> -->
   <xacro:o2as_ar_marker prefix="c_bot_"
-  			parent="c_bot_robotiq_85_tip_link"
-  			marker_id="26">
+			parent="c_bot_robotiq_85_tip_link"
+			marker_id="26">
     <origin xyz="0.0 0.0 0.0185" rpy="0 0 0"/>
   </xacro:o2as_ar_marker>
@@ -184,26 +183,4 @@
     <origin xyz="0.0 0.0 0.0005" rpy="0 0 0"/>
   </xacro:o2as_ar_marker_16cm>
-  <!-- Add PhoXi 3D scanners -->
-  <xacro:include filename="$(find o2as_scene_description)/urdf/phoxi_m_camera.urdf.xacro" />
-  <xacro:phoxi_m_camera prefix="a_" parent="o2as_ground">
-    <!-- <origin xyz="0.56 0 ${bots_z + .1 + .8}"
-	 rpy="${-160*pi/180} 0 ${pi/2}"/> -->
-    <!-- 181005@OSX -->
-    <!-- <origin xyz="0.65526 -0.018791 1.4169" -->
-    <!-- 	    rpy="${-149.595*pi/180} ${0.473*pi/180} ${91.976*pi/180}"/> -->
-    <!-- 181007@OSX -->
-    <!-- <origin xyz="0.6554 -0.020392 1.413" -->
-    <!-- 	    rpy="${-149.604*pi/180} ${0.34821*pi/180} ${91.866*pi/180}"/> -->
-    <!-- 181008@OSX -->
-    <!-- <origin xyz="0.674391 -0.0223742 ${bots_z + 0.696023}" -->
-    <!-- 	    rpy="${-149.801*pi/180} ${0.156861*pi/180} ${91.2544*pi/180}"/> -->
-    <!-- 181013@AIST -->
-    <!-- <origin xyz="0.620344080768 -0.0393922568732 1.44658358063" -->
-    <!-- 	    rpy="${-151.339295995*pi/180} ${1.39136148158*pi/180} -->
-    <!-- 		 ${86.8890568086*pi/180}"/> -->
-    <origin xyz="0.656427245186 -0.0191234201169 1.50626196172"
-	    rpy="${-161.285833025*pi/180} ${0.547979734685*pi/180}
-		 ${91.027298919*pi/180}"/>
-  </xacro:phoxi_m_camera>
   <!-- I would like to remove the "world" link definition, but apparently it is necessary for Gazebo -->
   <link name="world" />
