Commit message: check_calibration.py now displays positions of arrival.

File: o2as_scene_description/urdf/single_suction_gripper.urdf.xacro (robot description, xacro)
@@ -41,6 +41,7 @@
       <child  link="${prefix}single_suction_gripper_pad_link"/>
       <!-- <origin xyz="0.187 0 0" rpy="0 0 0"/> -->
-      <origin xyz="0.186976645492 -0.000326336140176 -0.00293726833731"
-	      rpy="${0.0*pi/180} ${0.9*pi/180} ${-0.1*pi/180}"/>
+      <origin xyz="0.186933357299 -0.000978789714711
+		   -0.00489508933357"
+	      rpy="${0.0*pi/180} ${1.5*pi/180} ${-0.3*pi/180}"/>>
     </joint>
   </xacro:macro>
