Commit message: Calibrate new gripper and taskboard

File: o2as_scene_description/urdf/InnerOnlyGripper.xacro (robot description, xacro)
@@ -24,10 +24,10 @@
       </geometry>
     </collision>
-    <visual>
+    <!-- <visual>
       <origin rpy="0 0 0" xyz="0.0 -0.01 0.062"/>
       <geometry>
         <box size="0.07 0.09 0.18"/>
       </geometry>
-    </visual>
+    </visual> -->
   </link>
   <joint name="${prefix}${grippername}" type="fixed">
@@ -40,5 +40,5 @@
     <parent link="${parent}"/>
     <child link="${prefix}${grippername}_tip_link"/>
-    <origin rpy="0.0 ${-pi/2} 0.0" xyz="0.0 -0.015 .158"/>
+    <origin rpy="0.0 ${-pi/2} 0.0" xyz="-0.002 -0.017 .163"/>
   </joint>
   <link name="${prefix}${grippername}_tip_link"/>

File: o2as_scene_description/urdf/o2as_base_scene.urdf.xacro (robot description, xacro)
@@ -22,7 +22,7 @@
   <xacro:include filename="$(find o2as_scene_description)/urdf/ur3.urdf.xacro" />
   <!-- Scene items (trays, bins...) -->
-  <!-- <xacro:include filename="$(find o2as_scene_description)/urdf/taskboard_scene.xacro" /> -->
+  <xacro:include filename="$(find o2as_scene_description)/urdf/taskboard_scene.xacro" />
   <!-- <xacro:include filename="$(find o2as_scene_description)/urdf/kitting_scene.xacro" /> -->
-  <xacro:include filename="$(find o2as_scene_description)/urdf/assembly_scene.xacro" />
+  <!-- <xacro:include filename="$(find o2as_scene_description)/urdf/assembly_scene.xacro" /> -->
   <!-- Robot bases -->
   <!-- Putting these at height 0.0 makes them intersect with the ground, so they are elevated. -->
@@ -68,5 +68,5 @@
   </xacro:screw_feeder>
   <!-- robot arms -->
-  <xacro:ur5_robot prefix="a_bot_" joint_limited="false"
+  <xacro:ur5_robot prefix="a_bot_" joint_limited="true"
     shoulder_pan_lower_limit="${-pi}" shoulder_pan_upper_limit="${pi}"
     shoulder_lift_lower_limit="${-pi}" shoulder_lift_upper_limit="${pi}"
@@ -106,8 +106,12 @@
   </joint>
   <!-- spawn and attach grippers -->
-  <xacro:include filename="$(find o2as_scene_description)/urdf/precision_gripper.xacro" />
+  <!-- <xacro:include filename="$(find o2as_scene_description)/urdf/precision_gripper.xacro" />
   <xacro:precision_gripper prefix="a_bot_"  grippername = "gripper" parent = "a_bot_tool0">
     <origin xyz="0.0 0 0.04" rpy="0 ${pi/2} 0"/>
-  </xacro:precision_gripper>
+  </xacro:precision_gripper> -->
+  <xacro:include filename="$(find o2as_scene_description)/urdf/InnerOnlyGripper.xacro" />
+  <xacro:InnerOnlyGripper prefix="a_bot_"  grippername = "gripper" parent = "a_bot_tool0">
+    <origin xyz="0.0 0 0.0" rpy="0 0 0"/>
+  </xacro:InnerOnlyGripper>
   <!-- spawn and attach dual robotiq 85 grippers -->
   <xacro:include filename="$(find o2as_scene_description)/urdf/robotiq_b_bot_gripper.urdf.xacro" />

File: o2as_scene_description/urdf/o2as_mat.xacro (robot description, xacro)
@@ -52,5 +52,4 @@
       <!-- Done with boundary drawing -->
       <collision>
-        <origin xyz="${mat_w/2} .01 ${mat_h}" rpy="0 0 0"/>
         <geometry>
           <box size="${mat_w} ${mat_l} ${mat_h}"/>
@@ -110,10 +109,16 @@
     </joint>
     <link name="${matname}_part6"/>
-    <joint name="${matname}_part7" type="fixed">
+    <joint name="${matname}_part7_1" type="fixed">
       <parent link="${matname}"/>
-      <child link="${matname}_part7"/>
+      <child link="${matname}_part7_1"/>
+      <origin rpy="0.0 0.0 ${pi/2}" xyz="0.0785 0.116 0.0"/>
+    </joint>
+    <link name="${matname}_part7_1"/>
+    <joint name="${matname}_part7_2" type="fixed">
+      <parent link="${matname}"/>
+      <child link="${matname}_part7_2"/>
       <origin rpy="0.0 0.0 ${pi/2}" xyz="0.011 0.011 0.0"/>
     </joint>
-    <link name="${matname}_part7"/>
+    <link name="${matname}_part7_2"/>
     <joint name="${matname}_part8" type="fixed">
       <parent link="${matname}"/>

File: o2as_scene_description/urdf/task_board.xacro (robot description, xacro)
@@ -110,16 +110,16 @@
   <!-- ======== -->
   <!-- The nut and bolt on the metal sheet -->
-  <joint name="${boardname}_part7a" type="fixed">
-    <parent link="${boardname}_surface"/>
-    <child link="${boardname}_part7a"/>
+  <joint name="${boardname}_part7_1" type="fixed">
+    <parent link="${boardname}_surface"/>
+    <child link="${boardname}_part7_1"/>
     <origin rpy="0.0 0.0 ${pi/2}" xyz="0.335 0.056 0.05"/>
   </joint>
-  <link name="${boardname}_part7a"/>
-  <joint name="${boardname}_part7b" type="fixed">
-    <parent link="${boardname}_surface"/>
-    <child link="${boardname}_part7b"/>
+  <link name="${boardname}_part7_1"/>
+  <joint name="${boardname}_part7_2" type="fixed">
+    <parent link="${boardname}_surface"/>
+    <child link="${boardname}_part7_2"/>
     <origin rpy="0.0 0.0 ${pi/2}" xyz="0.338 0.056 0.05"/>
   </joint>
-  <link name="${boardname}_part7b">
+  <link name="${boardname}_part7_2">
     <visual>
       <origin xyz="0 0.0015 -.015" rpy="0 0 0"/>

Commit message: Fix taskboard bugs, calibration
This picks parts 3,4,9,10 without issues.

File: o2as_scene_description/urdf/InnerOnlyGripper.xacro (robot description, xacro)
@@ -40,5 +40,5 @@
     <parent link="${parent}"/>
     <child link="${prefix}${grippername}_tip_link"/>
-    <origin rpy="0.0 ${-pi/2} 0.0" xyz="-0.002 -0.017 .163"/>
+    <origin rpy="0.0 ${-pi/2} 0.0" xyz="-0.002 -0.014 .163"/>
   </joint>
   <link name="${prefix}${grippername}_tip_link"/>

File: o2as_scene_description/urdf/o2as_mat.xacro (robot description, xacro)
@@ -76,5 +76,5 @@
       <parent link="${matname}"/>
       <child link="${matname}_part1"/>
-      <origin rpy="0.0 0.0 ${pi/2}" xyz="0.073 0.285 0.0"/>
+      <origin rpy="0.0 0.0 ${pi/2}" xyz="0.074 0.2835 0.0"/>
     </joint>
     <link name="${matname}_part1"/>
@@ -88,5 +88,5 @@
       <parent link="${matname}"/>
       <child link="${matname}_part3"/>
-      <origin rpy="0.0 0.0 ${pi/2}" xyz="0.261 0.323 0.0"/>
+      <origin rpy="0.0 0.0 ${pi/2}" xyz="0.259 0.322 0.0"/>
     </joint>
     <link name="${matname}_part3"/>
@@ -94,5 +94,5 @@
       <parent link="${matname}"/>
       <child link="${matname}_part4"/>
-      <origin rpy="0.0 0.0 ${pi/2}" xyz="0.343 0.3235 0.0"/>
+      <origin rpy="0.0 0.0 ${pi/2}" xyz="0.342 0.3215 0.0"/>
     </joint>
     <link name="${matname}_part4"/>
@@ -112,5 +112,5 @@
       <parent link="${matname}"/>
       <child link="${matname}_part7_1"/>
-      <origin rpy="0.0 0.0 ${pi/2}" xyz="0.0785 0.116 0.0"/>
+      <origin rpy="0.0 0.0 ${pi/2}" xyz="0.0795 0.116 0.0"/>
     </joint>
     <link name="${matname}_part7_1"/>
@@ -118,5 +118,5 @@
       <parent link="${matname}"/>
       <child link="${matname}_part7_2"/>
-      <origin rpy="0.0 0.0 ${pi/2}" xyz="0.011 0.011 0.0"/>
+      <origin rpy="0.0 0.0 ${pi/2}" xyz="0.1 0.1 0.0"/>
     </joint>
     <link name="${matname}_part7_2"/>
@@ -124,5 +124,5 @@
       <parent link="${matname}"/>
       <child link="${matname}_part8"/>
-      <origin rpy="0.0 0.0 ${pi/2}" xyz="0.011 0.013 0.0"/>
+      <origin rpy="0.0 0.0 ${pi/2}" xyz="0.1 0.1 0.0"/>
     </joint>
     <link name="${matname}_part8"/>
@@ -130,5 +130,5 @@
       <parent link="${matname}"/>
       <child link="${matname}_part9"/>
-      <origin rpy="0.0 0.0 ${pi/2}" xyz="0.155 0.094 0.0"/>
+      <origin rpy="0.0 0.0 ${pi/2}" xyz="0.153 0.093 0.0"/>
     </joint>
     <link name="${matname}_part9"/>
@@ -136,5 +136,5 @@
       <parent link="${matname}"/>
       <child link="${matname}_part10"/>
-      <origin rpy="0.0 0.0 ${pi/2}" xyz="0.252 0.106 0.0"/>
+      <origin rpy="0.0 0.0 ${pi/2}" xyz="0.2555 0.105 0.0"/>
     </joint>
     <link name="${matname}_part10"/>
@@ -142,5 +142,5 @@
       <parent link="${matname}"/>
       <child link="${matname}_part11"/>
-      <origin rpy="0.0 0.0 ${pi/2}" xyz="0.0 0.001 0.0"/>
+      <origin rpy="0.0 0.0 ${pi/2}" xyz="0.1 0.1 0.0"/>
     </joint>
     <link name="${matname}_part11"/>
@@ -148,5 +148,5 @@
       <parent link="${matname}"/>
       <child link="${matname}_part12"/>
-      <origin rpy="0.0 0.0 ${pi/2}" xyz="0.002 0.003 0.0"/>
+      <origin rpy="0.0 0.0 ${pi/2}" xyz="0.1 0.1 0.0"/>
     </joint>
     <link name="${matname}_part12"/>
@@ -154,5 +154,5 @@
       <parent link="${matname}"/>
       <child link="${matname}_part13"/>
-      <origin rpy="0.0 0.0 ${pi/2}" xyz="0.003 0.003 0.0"/>
+      <origin rpy="0.0 0.0 ${pi/2}" xyz="0.1 0.1 0.0"/>
     </joint>
     <link name="${matname}_part13"/>
@@ -160,5 +160,5 @@
       <parent link="${matname}"/>
       <child link="${matname}_part14"/>
-      <origin rpy="0.0 0.0 ${pi/2}" xyz="0.249 0.0445 0.0"/>
+      <origin rpy="0.0 0.0 ${pi/2}" xyz="0.248 0.0445 0.0"/>
     </joint>
     <link name="${matname}_part14"/>
@@ -166,5 +166,5 @@
       <parent link="${matname}"/>
       <child link="${matname}_part15"/>
-      <origin rpy="0.0 0.0 ${pi/2}" xyz="0.3465 0.051 0.0"/>
+      <origin rpy="0.0 0.0 ${pi/2}" xyz="0.344 0.0505 0.0"/>
     </joint>
     <link name="${matname}_part15"/>

Commit message: WIP: Add screw handover from a_bot

File: o2as_scene_description/urdf/InnerOnlyGripper.xacro (robot description, xacro)
@@ -43,4 +43,10 @@
   </joint>
   <link name="${prefix}${grippername}_tip_link"/>
+  <joint name="${prefix}${grippername}_screw_pickup_joint" type="fixed">
+    <parent link="${prefix}${grippername}_tip_link"/>
+    <child link="${prefix}${grippername}_screw_pickup"/>
+    <origin rpy="0.0 ${pi/2} 0.0" xyz="-.032 0 -0.003"/>
+  </joint>
+  <link name="${prefix}${grippername}_screw_pickup"/>
   </xacro:macro>
 </robot>

Commit message: clean up

File: o2as_scene_description/urdf/InnerOnlyGripper.xacro (robot description, xacro)
@@ -24,9 +24,27 @@
       </geometry>
     </collision>
+    <collision>
+      <origin rpy="0 0 0" xyz="0 -0.015 0.116"/>
+      <geometry>
+        <box size=".04 .05 .08"/>
+      </geometry>
+    </collision>
     <!-- <visual>
-      <origin rpy="0 0 0" xyz="0.0 -0.01 0.062"/>
+      <origin rpy="0 0 0" xyz="0.0 -0.015 0.062"/>
       <geometry>
-        <box size="0.07 0.09 0.18"/>
+        <box size="0.07 0.09 0.1"/>
       </geometry>
+      <material name="green2">
+        <color rgba="0.1 0.8 0.1 0.3"/>
+      </material>
+    </visual>
+    <visual>
+      <origin rpy="0 0 0" xyz="0 -0.015 0.116"/>
+      <geometry>
+        <box size=".04 .05 .08"/>
+      </geometry>
+      <material name="cyan2">
+        <color rgba="0.3 0.5 0.5 0.3"/>
+      </material>
     </visual> -->
   </link>

File: o2as_scene_description/urdf/precision_gripper.xacro (robot description, xacro)
@@ -17,5 +17,5 @@
         </material>
     </visual>
-    <!-- <visual>
+    <visual>
       <origin rpy="0 ${pi/2} 0" xyz="-0.05 0 0"/>
       <geometry>
@@ -34,5 +34,5 @@
         <color rgba="0.3 0.5 0.5 0.3"/>
       </material>
-    </visual> -->
+    </visual>
     <!-- TODO: Do this properly and check the offset above. -->
     <!-- Back part -->

File: o2as_scene_description/urdf/task_board.xacro (robot description, xacro)
@@ -219,5 +219,5 @@
     <parent link="${boardname}_surface"/>
     <child link="${boardname}_part15"/>
-    <origin rpy="0.0 0.0 ${pi/2}" xyz="0.16 0.36 0.0515"/>
+    <origin rpy="0.0 0.0 ${pi/2}" xyz="0.08 0.31 0.076"/>
   </joint>
   <link name="${boardname}_part15"/>

Commit message: Gripper fixes & recalibration

File: o2as_scene_description/urdf/InnerOnlyGripper.xacro (robot description, xacro)
@@ -58,5 +58,6 @@
     <parent link="${parent}"/>
     <child link="${prefix}${grippername}_tip_link"/>
-    <origin rpy="0.0 ${-pi/2} 0.0" xyz="-0.002 -0.014 .163"/>
+    <origin rpy="0.0 ${-pi/2} 0.0" xyz="0.002 -0.01 .162"/>
+    <!-- +y is the same, +x in the new frame is +z in the parent, +z is -x in the parent? -->
   </joint>
   <link name="${prefix}${grippername}_tip_link"/>

File: o2as_scene_description/urdf/taskboard_scene.xacro (robot description, xacro)
@@ -18,5 +18,5 @@
     <parent link="workspace_center"/>
     <child link="belt_placement_tool"/>
-    <origin rpy="0.0 0.0 0" xyz="-.15 0.3 0"/>
+    <origin rpy="0.0 0.0 0" xyz="-.2 0.3 0"/>
   </joint>
   <link name="belt_placement_tool"/>
@@ -33,10 +33,4 @@
   </joint>
   <link name="M10nut_tool"/>
-  <joint name="peg_tool" type="fixed">
-    <parent link="taskboard"/>
-    <child link="peg_tool"/>
-    <origin rpy="0.0 0.0 0" xyz="-0.06 0.56 0"/>
-  </joint>
-  <link name="peg_tool"/>
   <joint name="taskboard_set_screw_tool_joint" type="fixed">
     <parent link="taskboard"/>

Commit message: Squash commit of 2019 changes
- Bugfixes
- Robotiq gripper driver update
- xela sensor integration
- Assembly task demo in April 2019

File: o2as_scene_description/urdf/InnerOnlyGripper.xacro (robot description, xacro)
@@ -58,5 +58,5 @@
     <parent link="${parent}"/>
     <child link="${prefix}${grippername}_tip_link"/>
-    <origin rpy="0.0 ${-pi/2} 0.0" xyz="0.002 -0.01 .162"/>
+    <origin rpy="0.0 ${-pi/2} 0.0" xyz="0.001 -0.008 .162"/>
     <!-- +y is the same, +x in the new frame is +z in the parent, +z is -x in the parent? -->
   </joint>

File: o2as_scene_description/urdf/assembly_scene.xacro (robot description, xacro)
@@ -28,5 +28,5 @@
   <xacro:include filename="$(find o2as_parts_description)/urdf/assembly_parts_macros.urdf.xacro"/>
   <!-- <xacro:include filename="$(find o2as_parts_description)/urdf/display_all_parts.urdf.xacro"/> -->
-  <xacro:property name="assy_dx" value="-.01" />
+  <xacro:property name="assy_dx" value="-.008" />
   <!-- <xacro:include filename="$(find o2as_parts_description)/urdf/generated/full_assembly.urdf.xacro"/>
   <xacro:full_assembly prefix="assembled_" parent="workspace_center">

File: o2as_scene_description/urdf/o2as_mat.xacro (robot description, xacro)
@@ -76,5 +76,5 @@
       <parent link="${matname}"/>
       <child link="${matname}_part1"/>
-      <origin rpy="0.0 0.0 ${pi/2}" xyz="0.3355 0.163 0.0"/>
+      <origin rpy="0.0 0.0 ${pi/2}" xyz="0.074 0.2865 0.0"/>
     </joint>
     <link name="${matname}_part1"/>
@@ -82,5 +82,5 @@
       <parent link="${matname}"/>
       <child link="${matname}_part2"/>
-      <origin rpy="0.0 0.0 ${pi/2}" xyz="0.2305 0.038 0.0"/>
+      <origin rpy="0.0 0.0 ${pi/2}" xyz="0.175 0.3325 0.0"/>
     </joint>
     <link name="${matname}_part2"/>
@@ -88,5 +88,5 @@
       <parent link="${matname}"/>
       <child link="${matname}_part3"/>
-      <origin rpy="0.0 0.0 ${pi/2}" xyz="0.3075 0.252 0.0"/>
+      <origin rpy="0.0 0.0 ${pi/2}" xyz="0.2625 0.324 0.0"/>
     </joint>
     <link name="${matname}_part3"/>
@@ -94,5 +94,5 @@
       <parent link="${matname}"/>
       <child link="${matname}_part4"/>
-      <origin rpy="0.0 0.0 ${pi/2}" xyz="0.1625 0.075 0.0"/>
+      <origin rpy="0.0 0.0 ${pi/2}" xyz="0.3445 0.324 0.0"/>
     </joint>
     <link name="${matname}_part4"/>
@@ -106,5 +106,5 @@
       <parent link="${matname}"/>
       <child link="${matname}_part6"/>
-      <origin rpy="0.0 0.0 ${pi/2}" xyz="0.098 0.263 0.0"/>
+      <origin rpy="0.0 0.0 ${pi/2}" xyz="0.205 0.205 0.0"/>
     </joint>
     <link name="${matname}_part6"/>
@@ -112,5 +112,5 @@
       <parent link="${matname}"/>
       <child link="${matname}_part7_1"/>
-      <origin rpy="0.0 0.0 ${pi/2}" xyz="0.0 0.0 0.0"/>
+      <origin rpy="0.0 0.0 ${pi/2}" xyz="0.327 0.164 0.0"/>
     </joint>
     <link name="${matname}_part7_1"/>
@@ -118,5 +118,5 @@
       <parent link="${matname}"/>
       <child link="${matname}_part7_2"/>
-      <origin rpy="0.0 0.0 ${pi/2}" xyz="0.0 0.0 0.0"/>
+      <origin rpy="0.0 0.0 ${pi/2}" xyz="0.328 0.236 0.0"/>
     </joint>
     <link name="${matname}_part7_2"/>
@@ -124,5 +124,5 @@
       <parent link="${matname}"/>
       <child link="${matname}_part8"/>
-      <origin rpy="0.0 0.0 ${pi/2}" xyz="0.22 0.256 0.0"/>
+      <origin rpy="0.0 0.0 ${pi/2}" xyz="0.079 0.117 0.0"/>
     </joint>
     <link name="${matname}_part8"/>
@@ -130,5 +130,5 @@
       <parent link="${matname}"/>
       <child link="${matname}_part9"/>
-      <origin rpy="0.0 0.0 ${pi/2}" xyz="0.233 0.157 0.0"/>
+      <origin rpy="0.0 0.0 ${pi/2}" xyz="0.1555 0.0955 0.0"/>
     </joint>
     <link name="${matname}_part9"/>
@@ -136,5 +136,5 @@
       <parent link="${matname}"/>
       <child link="${matname}_part10"/>
-      <origin rpy="0.0 0.0 ${pi/2}" xyz="0.22 0.351 0.0"/>
+      <origin rpy="0.0 0.0 ${pi/2}" xyz="0.257 0.1075 0.0"/>
     </joint>
     <link name="${matname}_part10"/>
@@ -148,5 +148,5 @@
       <parent link="${matname}"/>
       <child link="${matname}_part12"/>
-      <origin rpy="0.0 0.0 ${pi/2}" xyz="0.338 0.047 0.0"/>
+      <origin rpy="0.0 0.0 ${pi/2}" xyz="0.06 0.048 0.0"/>
     </joint>
     <link name="${matname}_part12"/>
@@ -154,5 +154,5 @@
       <parent link="${matname}"/>
       <child link="${matname}_part13"/>
-      <origin rpy="0.0 0.0 ${pi/2}" xyz="0.332 0.327 0.0"/>
+      <origin rpy="0.0 0.0 ${pi/2}" xyz="0.145 0.042 0.0"/>
     </joint>
     <link name="${matname}_part13"/>
@@ -160,5 +160,5 @@
       <parent link="${matname}"/>
       <child link="${matname}_part14"/>
-      <origin rpy="0.0 0.0 ${pi/2}" xyz="0.078 0.0475 0.0"/>
+      <origin rpy="0.0 0.0 ${pi/2}" xyz="0.25 0.0465 0.0"/>
     </joint>
     <link name="${matname}_part14"/>
@@ -166,5 +166,5 @@
       <parent link="${matname}"/>
       <child link="${matname}_part15"/>
-      <origin rpy="0.0 0.0 ${pi/2}" xyz="0.282 0.0875 0.0"/>
+      <origin rpy="0.0 0.0 ${pi/2}" xyz="0.3475 0.0525 0.0"/>
     </joint>
     <link name="${matname}_part15"/>

File: o2as_scene_description/urdf/task_board.xacro (robot description, xacro)
@@ -125,5 +125,5 @@
     <parent link="${boardname}_surface"/>
     <child link="${boardname}_part7_1"/>
-    <origin rpy="0.0 0.0 ${pi*-0.5}" xyz="0.056 0.049 0.0505"/>
+    <origin rpy="0.0 0.0 ${pi*-0.5}" xyz="0.058 0.049 0.054"/>
   </joint>
   <link name="${boardname}_part7_1"/>
@@ -147,5 +147,5 @@
     <parent link="${boardname}_surface"/>
     <child link="${boardname}_part9"/>
-    <origin rpy="0.0 0.0 ${pi*0.5}" xyz="0.13 0.12 0.007"/>
+    <origin rpy="0.0 0.0 ${pi*0.5}" xyz="0.129 0.121 0.007"/>
   </joint>
   <link name="${boardname}_part9">
