Commit message: WIP: Connect all parts in URDF
The parameters in frames_to_mate.csv are not read in yet.

File: o2as_scene_description/urdf/assembly_scene.xacro (robot description, xacro)
@@ -16,5 +16,5 @@
   <link name="pulley_front_end"/>
   <xacro:include filename="$(find o2as_parts_description)/urdf/assembly_parts_macros.urdf"/>
-  <xacro:assy_part_01 prefix="" parent="workspace_center">
+  <!-- <xacro:assy_part_01 prefix="" parent="workspace_center">
     <origin xyz="0.05 0.08 0.07" rpy="0 0 ${-pi/2}" />
   </xacro:assy_part_01>
@@ -27,5 +27,9 @@
   <xacro:assy_part_13 prefix="" parent="workspace_center">
     <origin xyz="0.0 0.0 0.13" rpy="0 0 0" />
-  </xacro:assy_part_13>
-  <xacro:include filename="$(find o2as_parts_description)/urdf/display_all_parts.urdf"/>
+  </xacro:assy_part_13> -->
+  <!-- <xacro:include filename="$(find o2as_parts_description)/urdf/display_all_parts.urdf"/> -->
+  <xacro:include filename="$(find o2as_parts_description)/urdf/full_assembly.urdf"/>
+  <xacro:full_assembly prefix="assembled_" parent="workspace_center">
+    <origin xyz="0 0 .4" rpy="0 0 0" />
+  </xacro:full_assembly>
 </robot>

Commit message: Add "naked" (frame-only) assembly URDF
The file is almost correct, except for some CAD models and fine tuning. The underlying method is still off, though.

File: o2as_scene_description/urdf/assembly_scene.xacro (robot description, xacro)
@@ -28,8 +28,12 @@
     <origin xyz="0.0 0.0 0.13" rpy="0 0 0" />
   </xacro:assy_part_13> -->
-  <!-- <xacro:include filename="$(find o2as_parts_description)/urdf/display_all_parts.urdf"/> -->
+  <xacro:include filename="$(find o2as_parts_description)/urdf/display_all_parts.urdf"/>
   <xacro:include filename="$(find o2as_parts_description)/urdf/generated/full_assembly.urdf"/>
   <xacro:full_assembly prefix="assembled_" parent="workspace_center">
     <origin xyz="0 0 .4" rpy="0 0 0" />
   </xacro:full_assembly>
+    <xacro:include filename="$(find o2as_parts_description)/urdf/generated/full_assembly_frames_only.urdf"/>
+  <xacro:full_assembly_frames_only prefix="assembled_frames_only_" parent="workspace_center">
+    <origin xyz="0 .15 .4" rpy="0 0 0" />
+  </xacro:full_assembly_frames_only>
 </robot>

Commit message: Add assembly to scene, fix some bugs

File: o2as_scene_description/urdf/assembly_scene.xacro (robot description, xacro)
@@ -16,24 +16,12 @@
   <link name="pulley_front_end"/>
   <xacro:include filename="$(find o2as_parts_description)/urdf/assembly_parts_macros.urdf"/>
-  <!-- <xacro:assy_part_01 prefix="" parent="workspace_center">
-    <origin xyz="0.05 0.08 0.07" rpy="0 0 ${-pi/2}" />
-  </xacro:assy_part_01>
-  <xacro:assy_part_02 prefix="" parent="workspace_center">
-    <origin xyz="0.0 -0.3 0.0" rpy="0 0 ${pi/2}" />
-  </xacro:assy_part_02>
-  <xacro:assy_part_03 prefix="" parent="workspace_center">
-    <origin xyz="0.0 0.22 0.0" rpy="0 0 ${pi/2}" />
-  </xacro:assy_part_03>
-  <xacro:assy_part_13 prefix="" parent="workspace_center">
-    <origin xyz="0.0 0.0 0.13" rpy="0 0 0" />
-  </xacro:assy_part_13> -->
-  <xacro:include filename="$(find o2as_parts_description)/urdf/display_all_parts.urdf"/>
+  <!-- <xacro:include filename="$(find o2as_parts_description)/urdf/display_all_parts.urdf"/> -->
   <xacro:include filename="$(find o2as_parts_description)/urdf/generated/full_assembly.urdf"/>
   <xacro:full_assembly prefix="assembled_" parent="workspace_center">
-    <origin xyz="0 0 .4" rpy="0 0 0" />
+    <origin xyz="0 0.1 .065" rpy="0 0 ${-pi/2}" />
   </xacro:full_assembly>
-    <xacro:include filename="$(find o2as_parts_description)/urdf/generated/full_assembly_frames_only.urdf"/>
+    <!-- <xacro:include filename="$(find o2as_parts_description)/urdf/generated/full_assembly_frames_only.urdf"/>
   <xacro:full_assembly_frames_only prefix="assembled_frames_only_" parent="workspace_center">
-    <origin xyz="0 .15 .4" rpy="0 0 0" />
-  </xacro:full_assembly_frames_only>
+    <origin xyz="0 0.1 .065" rpy="0 0 ${-pi/2}" />
+  </xacro:full_assembly_frames_only> -->
 </robot>

Commit message: Add trays to assembly scene

File: o2as_scene_description/urdf/assembly_scene.xacro (robot description, xacro)
@@ -4,15 +4,11 @@
   <xacro:include filename="$(find o2as_scene_description)/urdf/kitting_tray.xacro" />
   <!-- Insert: -->
-  <!-- Tray 1 -->
-  <!-- Tray 2 -->
+  <xacro:kitting_tray1 trayname="tray_1" parent="workspace_center">
+    <origin xyz="-.2 -.27 0" rpy="0 0 ${pi/2}" />
+  </xacro:kitting_tray1>
+  <xacro:kitting_tray2 trayname="tray_2" parent="workspace_center">
+    <origin xyz="-.2 .27 0" rpy="0 0 ${-pi/2}" />
+  </xacro:kitting_tray2>
   <!-- The base plate -->
-  <!-- All the other parts need to be added somehow so that their frames can be updated, I guess. Hmmmmmmm. -->
-  <!-- Manually defined pulley frame for the small test on 21 August. -->
-  <joint name="test_joint" type="fixed">
-    <parent link="workspace_center"/>
-    <child link="pulley_front_end"/>
-    <origin rpy="0.0 0.0 ${pi}" xyz="0.0 0.0 0.07 "/>
-  </joint>
-  <link name="pulley_front_end"/>
   <xacro:include filename="$(find o2as_parts_description)/urdf/assembly_parts_macros.urdf"/>
   <!-- <xacro:include filename="$(find o2as_parts_description)/urdf/display_all_parts.urdf"/> -->

File: o2as_scene_description/urdf/kitting_tray.xacro (robot description, xacro)
@@ -1,4 +1,4 @@
 <?xml version="1.0" ?>
-<robot xmlns:xacro="http://ros.org/wiki/xacro" name="kitting_bin">
+<robot xmlns:xacro="http://ros.org/wiki/xacro" name="kitting_tray">
   <!-- This file defines a tray that could be used for temporarily placing items for regrasping during the kitting tray -->
   <xacro:macro name="kitting_tray" params="trayname parent *origin">

File: o2as_scene_description/urdf/o2as_base_scene.urdf.xacro (robot description, xacro)
@@ -21,6 +21,8 @@
   <xacro:include filename="$(find o2as_scene_description)/urdf/ur3.urdf.xacro" />
   <!-- Scene items (trays, bins...) -->
+  <xacro:include filename="$(find o2as_scene_description)/urdf/kitting_tray_with_partitions.xacro" />
   <!-- <xacro:include filename="$(find o2as_scene_description)/urdf/taskboard_scene.xacro" /> -->
-  <xacro:include filename="$(find o2as_scene_description)/urdf/kitting_scene.xacro" />
+  <!-- <xacro:include filename="$(find o2as_scene_description)/urdf/kitting_scene.xacro" /> -->
+  <xacro:include filename="$(find o2as_scene_description)/urdf/assembly_scene.xacro" />
   <!-- Robot bases -->
   <!-- Putting these at height 0.0 makes them intersect with the ground, so they are elevated. -->

Commit message: Scene clean-up

File: o2as_scene_description/urdf/assembly_scene.xacro (robot description, xacro)
@@ -1,6 +1,5 @@
 <?xml version="1.0"?>
 <robot xmlns:xacro="http://www.ros.org/wiki/xacro" name="kitting_scene">
-  <xacro:include filename="$(find o2as_scene_description)/urdf/kitting_bins.xacro" />
-  <xacro:include filename="$(find o2as_scene_description)/urdf/kitting_tray.xacro" />
+  <xacro:include filename="$(find o2as_scene_description)/urdf/kitting_tray_with_partitions.xacro" />
   <!-- Insert: -->
   <xacro:kitting_tray1 trayname="tray_1" parent="workspace_center">

File: o2as_scene_description/urdf/kitting_bins.xacro (robot description, xacro)
@@ -1,55 +1,66 @@
-<?xml version="1.0" ?>
-<robot xmlns:xacro="http://ros.org/wiki/xacro" name="kitting_bin">
-  <!-- z-origin-offset should be set such that the frame is on the surface of the bin -->
-  <xacro:macro name="kitting_bin_internal" params="binname parent filename z_origin_offset *origin">
-    <xacro:property name="mesh_file" value="package://o2as_scene_description/meshes/${filename}.stl" />
-    <xacro:property name="mesh_file_col" value="package://o2as_scene_description/meshes/${filename}.vhacd.dae" />
-    <link name="${binname}">
-      <inertial>
-        <origin rpy="0 0 0" xyz="0 0 ${z_origin_offset}"/>
-        <mass value="1.0"/>
-        <inertia ixx="1.0" ixy="0" ixz="0" iyy="1.0" iyz="0" izz="1.0"/>
-      </inertial>
-      <visual>
-        <origin rpy="${pi/2} 0 ${pi/2}" xyz="0 0 ${z_origin_offset}"/>
-        <geometry>
-          <mesh filename="${mesh_file}" scale="0.001 0.001 0.001"/>
-          <!-- <mesh filename="package://ur_description/meshes/ur5/visual/shoulder.dae"/> -->
-        </geometry>
-        <material name="orange">
-          <color rgba="1 0.5088 0.0468 1"/>
-        </material>
-      </visual>
-      <collision>
-        <origin rpy="${pi/2} 0 ${pi/2}" xyz="0 0 ${z_origin_offset}"/>
-        <geometry>
-          <mesh filename="${mesh_file_col}" scale="0.001 0.001 0.001"/>
-          <!-- <mesh filename="package://ur_description/meshes/ur5/collision/shoulder.stl"/> -->
-        </geometry>
-      </collision>
-    </link>
-    <gazebo reference="${binname}">
-      <material>Gazebo/Orange</material>
-    </gazebo>
-    <joint name="${binname}" type="fixed">
-      <parent link="${parent}" />
-      <child link = "${binname}" />
-      <xacro:insert_block name="origin"/>
-    </joint>
-  </xacro:macro>
-  <xacro:macro name="kitting_bin_1" params="binname parent z_origin_offset *origin">
-    <xacro:kitting_bin_internal binname="${binname}" parent="${parent}" filename="bin1_EA661CA-11" z_origin_offset="${z_origin_offset}">
-      <xacro:insert_block name="origin"/>
-    </xacro:kitting_bin_internal>
-  </xacro:macro>
-  <xacro:macro name="kitting_bin_2" params="binname parent z_origin_offset *origin">
-    <xacro:kitting_bin_internal binname="${binname}" parent="${parent}" filename="bin2_SK-HL1-BL" z_origin_offset="${z_origin_offset}">
-      <xacro:insert_block name="origin"/>
-    </xacro:kitting_bin_internal>
-  </xacro:macro>
-  <xacro:macro name="kitting_bin_3" params="binname parent z_origin_offset *origin">
-    <xacro:kitting_bin_internal binname="${binname}" parent="${parent}" filename="bin3_T3-YG" z_origin_offset="${z_origin_offset}">
-      <xacro:insert_block name="origin"/>
-    </xacro:kitting_bin_internal>
-  </xacro:macro>
+<?xml version="1.0"?>
+<robot xmlns:xacro="http://www.ros.org/wiki/xacro" name="kitting_scene">
+  <xacro:include filename="$(find o2as_scene_description)/urdf/kitting_bin_macros.xacro" />
+  <xacro:property name="rack_width" value=".640" />
+ <!-- space for bin -->
+ <!-- bin1_definition -->
+ <xacro:property name="bin1_width" value="0.125"/>
+ <xacro:property name="bin1_length" value="0.128"/>
+ <xacro:property name="z_origin_offset_1" value="-.008" />
+ <!-- bin2_definition -->
+ <xacro:property name="bin2_width" value="0.112"/>
+ <xacro:property name="bin2_length" value="0.201"/>
+ <xacro:property name="z_origin_offset_2" value="-.009" />
+ <!-- bin3_definition -->
+ <xacro:property name="bin3_width" value="0.192"/>
+ <xacro:property name="bin3_length" value="0.285"/>
+ <xacro:property name="z_origin_offset_3" value="-.004" />
+ <!-- A row of bin1 -->
+ <xacro:property name="set1_x" value=".0"/>
+ <xacro:property name="set1_y" value="0.33"/>
+ <xacro:property name="set1_z" value=".01"/>
+ <!-- A row of bin2 -->
+ <xacro:property name="set2_x" value=".20"/>
+ <xacro:property name="set2_y" value="0.33"/>
+ <xacro:property name="set2_z" value=".00"/>
+ <!--set1_bin1_1_-->
+  <xacro:kitting_bin_1 binname="set1_bin1_1" parent="workspace_center" z_origin_offset="-.008">
+      <origin xyz=".0 0.2675 0.018" rpy="0 0 0" />
+  </xacro:kitting_bin_1>
+  <!--set1_bin1_2_-->
+  <xacro:kitting_bin_1 binname="set1_bin1_2" parent="workspace_center" z_origin_offset="-.008">
+      <origin xyz=".0 0.1425 0.018" rpy="0 0 0" />
+  </xacro:kitting_bin_1>
+  <!--set1_bin1_3_-->
+  <xacro:kitting_bin_1 binname="set1_bin1_3" parent="workspace_center" z_origin_offset="-.008">
+      <origin xyz=".0 0.0175 0.018" rpy="0 0 0" />
+  </xacro:kitting_bin_1>
+  <!--set1_bin1_4_-->
+  <xacro:kitting_bin_1 binname="set1_bin1_4" parent="workspace_center" z_origin_offset="-.008">
+      <origin xyz=".0 -0.1075 0.018" rpy="0 0 0" />
+  </xacro:kitting_bin_1>
+  <!--set1_bin1_5_-->
+  <xacro:kitting_bin_1 binname="set1_bin1_5" parent="workspace_center" z_origin_offset="-.008">
+      <origin xyz=".0 -0.2325 0.018" rpy="0 0 0" />
+  </xacro:kitting_bin_1>
+  <!--set2_bin2_1_-->
+  <xacro:kitting_bin_2 binname="set2_bin2_1" parent="workspace_center" z_origin_offset="-.009">
+      <origin xyz=".20 0.274 0.009" rpy="0 0 0" />
+  </xacro:kitting_bin_2>
+  <!--set2_bin2_2_-->
+  <xacro:kitting_bin_2 binname="set2_bin2_2" parent="workspace_center" z_origin_offset="-.009">
+      <origin xyz=".20 0.162 0.009" rpy="0 0 0" />
+  </xacro:kitting_bin_2>
+  <!--set2_bin2_3_-->
+  <xacro:kitting_bin_2 binname="set2_bin2_3" parent="workspace_center" z_origin_offset="-.009">
+      <origin xyz=".20 0.05 0.009" rpy="0 0 0" />
+  </xacro:kitting_bin_2>
+  <!--set2_bin2_4_-->
+  <xacro:kitting_bin_2 binname="set2_bin2_4" parent="workspace_center" z_origin_offset="-.009">
+      <origin xyz=".20 -0.062 0.009" rpy="0 0 0" />
+  </xacro:kitting_bin_2>
+  <!--set2_bin3_1_-->
+  <xacro:kitting_bin_3 binname="set2_bin3_1" parent="workspace_center" z_origin_offset="-.004">
+      <origin xyz=".20 -0.214 0.004" rpy="0 0 0" />
+  </xacro:kitting_bin_3>
 </robot>

File: o2as_scene_description/urdf/kitting_scene.xacro (robot description, xacro)
@@ -2,95 +2,13 @@
 <robot xmlns:xacro="http://www.ros.org/wiki/xacro" name="kitting_scene">
   <xacro:include filename="$(find o2as_scene_description)/urdf/kitting_bins.xacro" />
-  <!-- <xacro:include filename="$(find o2as_scene_description)/urdf/kitting_tray.xacro" /> -->
   <xacro:include filename="$(find o2as_scene_description)/urdf/kitting_tray_with_partitions.xacro" />
   <xacro:include filename="$(find realsense2_camera)/urdf/_d435.urdf.xacro" />
-  <xacro:property name="bin1_width" value=".125"/>
-  <xacro:property name="bin1_length" value=".128" />
-  <xacro:property name="bin2_width" value=".112" />
-  <xacro:property name="bin2_length" value=".201" />
-  <xacro:property name="bin3_width" value=".192" />
-  <xacro:property name="bin3_length" value=".285" />
+  <!-- spawn and attach dual suction grippers -->
+  <!-- <xacro:include filename="$(find o2as_scene_description)/urdf/dual_suction_gripper.urdf.xacro" /> -->
+  <!-- <xacro:dual_suction_gripper_o2as prefix="b_bot_" parent = "b_bot_ee_link">
+    <origin xyz="0 0 0" rpy="0 0 0"/>
+  </xacro:dual_suction_gripper_o2as> -->
   <xacro:property name="tray_width" value=".300" />
   <xacro:property name="tray_length" value=".210" />
-  <xacro:property name="z_origin_offset_1" value="-.008" />
-  <xacro:property name="z_origin_offset_2" value="-.009" />
-  <xacro:property name="z_origin_offset_3" value="-.004" />
-  <xacro:property name="set1_x" value="${bin3_length/2}" />
-  <xacro:property name="set1_y" value="${-.33 + bin3_width / 2}" />
-  <!-- <xacro:property name="set1_z" value="0.01" /> -->
-  <xacro:property name="set1_z" value="0.0" />
-  <xacro:kitting_bin_3 binname="part_6" parent="workspace_center" z_origin_offset="${z_origin_offset_3}">
-    <origin xyz="${set1_x} ${set1_y} ${set1_z - z_origin_offset_3}" rpy="0 0 ${pi}" />
-  </xacro:kitting_bin_3>
-  <xacro:kitting_bin_2 binname="part_4" parent="workspace_center" z_origin_offset="${z_origin_offset_2}">
-    <origin xyz="${set1_x} ${set1_y + bin3_width / 2 + bin2_width / 2} ${set1_z - z_origin_offset_2}" rpy="0 0 ${pi}" />
-  </xacro:kitting_bin_2>
-  <xacro:kitting_bin_2 binname="part_8" parent="workspace_center" z_origin_offset="${z_origin_offset_2}">
-    <origin xyz="${set1_x} ${set1_y + bin3_width / 2 + 3 * bin2_width / 2} ${set1_z - z_origin_offset_2}" rpy="0 0 ${pi}" />
-  </xacro:kitting_bin_2>
-  <xacro:kitting_bin_2 binname="part_11" parent="workspace_center" z_origin_offset="${z_origin_offset_2}">
-    <origin xyz="${set1_x} ${set1_y + bin3_width / 2 + 5 * bin2_width / 2} ${set1_z - z_origin_offset_2}" rpy="0 0 ${pi}" />
-  </xacro:kitting_bin_2>
-  <xacro:kitting_bin_2 binname="part_13" parent="workspace_center" z_origin_offset="${z_origin_offset_2}">
-    <origin xyz="${set1_x} ${set1_y + bin3_width / 2 + 7 * bin2_width / 2} ${set1_z - z_origin_offset_2}" rpy="0 0 ${pi}" />
-  </xacro:kitting_bin_2>
-  <xacro:property name="set2_x" value="${.42-bin1_length/2}" />
-  <xacro:property name="set2_y" value="0" />
-  <!-- <xacro:property name="set2_z" value="0.01" /> -->
-  <xacro:property name="set2_z" value="0.0" />
-  <xacro:kitting_bin_1 binname="part_9" parent="workspace_center" z_origin_offset="${z_origin_offset_1}">
-    <origin xyz="${set2_x} ${set2_y} ${set2_z - z_origin_offset_1}" rpy="0 0 ${pi}" />
-  </xacro:kitting_bin_1>
-  <xacro:kitting_bin_1 binname="part_12" parent="workspace_center" z_origin_offset="${z_origin_offset_1}">
-    <origin xyz="${set2_x} ${set2_y - bin1_width} ${set2_z - z_origin_offset_1}" rpy="0 0 ${pi}" />
-  </xacro:kitting_bin_1>
-  <xacro:kitting_bin_1 binname="part_16" parent="workspace_center" z_origin_offset="${z_origin_offset_1}">
-    <origin xyz="${set2_x} ${set2_y + bin1_width} ${set2_z - z_origin_offset_1}" rpy="0 0 ${pi}" />
-  </xacro:kitting_bin_1>
-  <xacro:kitting_bin_1 binname="part_17" parent="workspace_center" z_origin_offset="${z_origin_offset_1}">
-    <origin xyz="${set2_x} ${set2_y - 2 * bin1_width} ${set2_z - z_origin_offset_1}" rpy="0 0 ${pi}" />
-  </xacro:kitting_bin_1>
-  <xacro:kitting_bin_1 binname="part_18" parent="workspace_center" z_origin_offset="${z_origin_offset_1}">
-    <origin xyz="${set2_x} ${set2_y + 2 * bin1_width} ${set2_z - z_origin_offset_1}" rpy="0 0 ${pi}" />
-  </xacro:kitting_bin_1>
-  <!-- <xacro:property name="set1_x" value="+0.05"/>
-  <xacro:property name="set1_y" value="${.32-bin1_width/2}"/>
-  <xacro:property name="set1_z" value=".01" />
-  <xacro:kitting_bin_1 binname="set1_bin1_1" parent="workspace_center" z_origin_offset="${z_origin_offset_1}">
-    <origin xyz="${set1_x} ${set1_y} ${set1_z - z_origin_offset_1}" rpy="0 0 0" />
-  </xacro:kitting_bin_1>
-  <xacro:kitting_bin_1 binname="set1_bin1_2" parent="workspace_center" z_origin_offset="${z_origin_offset_1}">
-    <origin xyz="${set1_x} ${set1_y - bin1_width*1} ${set1_z - z_origin_offset_1}" rpy="0 0 0" />
-  </xacro:kitting_bin_1>
-  <xacro:kitting_bin_1 binname="set1_bin1_3" parent="workspace_center" z_origin_offset="${z_origin_offset_1}">
-    <origin xyz="${set1_x} ${set1_y - bin1_width*2} ${set1_z - z_origin_offset_1}" rpy="0 0 0" />
-  </xacro:kitting_bin_1>
-  <xacro:kitting_bin_1 binname="set1_bin1_4" parent="workspace_center" z_origin_offset="${z_origin_offset_1}">
-    <origin xyz="${set1_x} ${set1_y - bin1_width*3} ${set1_z - z_origin_offset_1}" rpy="0 0 0" />
-  </xacro:kitting_bin_1>
-  <xacro:kitting_bin_1 binname="set1_bin1_5" parent="workspace_center" z_origin_offset="${z_origin_offset_1}">
-    <origin xyz="${set1_x} ${set1_y - bin1_width*4} ${set1_z - z_origin_offset_1}" rpy="0 0 0" />
-  </xacro:kitting_bin_1> -->
-  <!-- A row of bin2 and bin3 -->
-  <!-- <xacro:property name="set2_x_bin3" value="${bin1_length/2+bin3_length/2+0.05}" />
-  <xacro:property name="set2_x_bin2" value="${bin1_length/2+bin2_length/2+0.05}" />
-  <xacro:property name="set2_y" value="${.32-bin3_width/2}" />
-  <xacro:property name="set2_z" value=".00" />
-   -->
-  <!-- <xacro:kitting_bin_3 binname="set2_bin3" parent="workspace_center" z_origin_offset="${z_origin_offset_3}">
-    <origin xyz="${set2_x_bin3} ${set2_y} ${set2_z - z_origin_offset_3}" rpy="0 0 0" />
-  </xacro:kitting_bin_3>
-  <xacro:kitting_bin_2 binname="set2_bin2_1" parent="workspace_center" z_origin_offset="${z_origin_offset_2}">
-    <origin xyz="${set2_x_bin2} ${set2_y-bin3_width/2-bin2_width/2*1} ${set2_z - z_origin_offset_2}" rpy="0 0 0" />
-  </xacro:kitting_bin_2>
-  <xacro:kitting_bin_2 binname="set2_bin2_2" parent="workspace_center" z_origin_offset="${z_origin_offset_2}">
-    <origin xyz="${set2_x_bin2} ${set2_y-bin3_width/2-bin2_width*3/2} ${set2_z - z_origin_offset_2}" rpy="0 0 0" />
-  </xacro:kitting_bin_2>
-  <xacro:kitting_bin_2 binname="set2_bin2_3" parent="workspace_center" z_origin_offset="${z_origin_offset_2}">
-    <origin xyz="${set2_x_bin2} ${set2_y-bin3_width/2-bin2_width*5/2} ${set2_z - z_origin_offset_2}" rpy="0 0 0" />
-  </xacro:kitting_bin_2>
-  <xacro:kitting_bin_2 binname="set2_bin2_4" parent="workspace_center" z_origin_offset="${z_origin_offset_2}">
-    <origin xyz="${set2_x_bin2} ${set2_y-bin3_width/2-bin2_width*7/2} ${set2_z - z_origin_offset_2}" rpy="0 0 0" />
-  </xacro:kitting_bin_2> -->
   <!-- add camera for pose matching on the table -->
   <link name="workspace_cam_holder_link" />
@@ -103,19 +21,12 @@
     <origin xyz="0 0 0" rpy="0 0 0"/>
   </xacro:sensor_d435>
+  <!-- TODO: Deal with this camera? -->
   <!-- A row of tray -->
-  <xacro:property name="set3_x" value="${-(bin1_length/2+tray_length/2)-0.05}" />
-  <xacro:property name="set3_y" value="${.32-tray_width/2}" />
+  <xacro:property name="set3_x" value="${-.3}" />
+  <xacro:property name="set3_y" value="${0}" />
   <xacro:property name="set3_z" value=".00" />
-  <!-- set3_tray_1 -->
-  <!-- <xacro:kitting_tray trayname="set3_tray_1" parent="workspace_center"> -->
-  <!--   <origin xyz="${set3_x} ${set3_y} ${set3_z}" rpy="0 0 0" /> -->
-  <!-- </xacro:kitting_tray> -->
   <xacro:kitting_tray1 trayname="set3_tray_1" parent="workspace_center">
     <origin xyz="${set3_x} ${set3_y} ${set3_z}" rpy="0 0 0" />
   </xacro:kitting_tray1>
-  <!-- set3_tray_2 -->
-  <!-- <xacro:kitting_tray trayname="set3_tray_2" parent="workspace_center"> -->
-  <!--   <origin xyz="${set3_x} ${set3_y-tray_width} ${set3_z}" rpy="0 0 0" /> -->
-  <!-- </xacro:kitting_tray> -->
   <xacro:kitting_tray2 trayname="set3_tray_2" parent="workspace_center">
     <origin xyz="${set3_x} ${set3_y-tray_width} ${set3_z}" rpy="0 0 0" />
