Commit message: Scene clean-up

File: o2as_scene_description/urdf/kitting_tray_with_partitions.xacro (robot description, xacro)
@@ -2,5 +2,47 @@
 <robot xmlns:xacro="http://ros.org/wiki/xacro"
        name="kitting_tray2_o2as">
-  <xacro:include filename="$(find o2as_scene_description)/urdf/kitting_tray.xacro" />
+  <!-- ========== This file defines the trays for the assembly and kitting task -->
+  <xacro:property name="tray_width" value=".300" />
+  <xacro:property name="tray_length" value=".210" />
+  <!-- TODO: Please adjust the width and length so that the origin is at the corner of the tray (this is easier to calibrate later) -->
+  <xacro:property name="mesh_offset_x" value="-.045" />
+  <xacro:property name="mesh_offset_y" value=".045" />
+  <!-- TODO: Is this mesh centered? Where is the coordinate origin? Check the dividers too. -->
+  <!-- ========== The basic tray, without partitions -->
+  <xacro:macro name="kitting_tray" params="trayname parent *origin">
+    <xacro:property name="mesh_file" value="package://o2as_scene_description/meshes/tray_PZ-0006-B.stl" />
+    <xacro:property name="mesh_file_col" value="package://o2as_scene_description/meshes/tray_PZ-0006-B.vhacd.dae" />
+    <link name="${trayname}">
+      <inertial>
+        <origin rpy="0 0 0" xyz="${tray_width/2} ${tray_length/2} 0"/>
+        <mass value="1.0"/>
+        <inertia ixx="1.0" ixy="0" ixz="0" iyy="1.0" iyz="0" izz="1.0"/>
+      </inertial>
+      <visual>
+        <origin rpy="${pi/2} 0 ${pi/2}" xyz="${tray_width/2 +mesh_offset_x} ${tray_length/2 + mesh_offset_y} 0"/>
+        <geometry>
+          <mesh filename="${mesh_file}" scale="0.001 0.001 0.001"/>
+          <!-- <mesh filename="package://ur_description/meshes/ur5/visual/shoulder.dae"/> -->
+        </geometry>
+        <material name="white">
+          <color rgba="1 1 1 1"/>
+        </material>
+      </visual>
+      <collision>
+        <origin rpy="${pi/2} 0 ${pi/2}" xyz="${tray_width/2 +mesh_offset_x} ${tray_length/2 + mesh_offset_y} 0"/>
+        <geometry>
+          <mesh filename="${mesh_file_col}" scale="0.001 0.001 0.001"/>
+          <!-- <mesh filename="package://ur_description/meshes/ur5/collision/shoulder.stl"/> -->
+        </geometry>
+      </collision>
+    </link>
+    <joint name="${trayname}" type="fixed">
+      <parent link="${parent}" />
+      <child link = "${trayname}" />
+      <xacro:insert_block name="origin"/>
+    </joint>
+  </xacro:macro>
+  <!-- ========== -->
+  <!-- ========== The partitions as separate macros -->
   <xacro:macro name="tray_contents" params="trayname contents *origin">
     <link name="${trayname}_${contents}">
@@ -26,25 +68,116 @@
     </joint>
   </xacro:macro>
+  <!-- ========== A helper macro for readability in the screw holder definition -->
+  <xacro:macro name="auxiliary_frame" params="parent framename *origin">
+    <joint name="${parent}_${framename}" type="fixed">
+      <parent link="${parent}" />
+      <child link = "${parent}_${framename}"/>
+      <xacro:insert_block name="origin"/>
+    </joint>
+    <link name="${parent}_${framename}"/>
+  </xacro:macro>
+  <xacro:property name="dividers_z_offset" value="0.0" />
+  <!-- ========== The tray with the belt and motor -->
   <xacro:macro name="kitting_tray1" params="trayname parent *origin">
     <xacro:kitting_tray trayname="${trayname}" parent="${parent}">
       <xacro:insert_block name="origin"/>
     </xacro:kitting_tray>
-    <xacro:tray_contents trayname="${trayname}" contents="partition1_1">
-      <origin xyz="-0.095 0.14 0" rpy="0 0 ${-pi/2}"/>
+    <xacro:tray_contents trayname="${trayname}" contents="divider1_1">
+      <origin xyz="${tray_width/2 + mesh_offset_x - 0.095} ${tray_length/2 + mesh_offset_y + 0.14} ${dividers_z_offset}" rpy="0 0 ${-pi/2}"/>
     </xacro:tray_contents>
-    <xacro:tray_contents trayname="${trayname}" contents="partition1_2">
-      <origin xyz="-0.095 -0.062 0" rpy="0 0 ${-pi/2}"/>
+    <xacro:tray_contents trayname="${trayname}" contents="divider1_2">
+      <origin xyz="${tray_width/2 + mesh_offset_x - 0.095} ${tray_length/2 + mesh_offset_y -0.062} ${dividers_z_offset}" rpy="0 0 ${-pi/2}"/>
     </xacro:tray_contents>
+    <!-- ========== The extra frames to place and pick items are defined below -->
+    <joint name="${trayname}_partition_1" type="fixed">
+      <parent link="${trayname}" />
+      <child link = "${trayname}_partition_1"/>
+      <origin rpy="0.0 0.0 0.0" xyz="0.05 0.05 0.02"/>
+    </joint>
+    <link name="${trayname}_partition_1"/>
+    <joint name="${trayname}_partition_2" type="fixed">
+      <parent link="${trayname}" />
+      <child link = "${trayname}_partition_2"/>
+      <origin rpy="0.0 0.0 0.0" xyz="0.15 0.05 0.02"/>
+    </joint>
+    <link name="${trayname}_partition_2"/>
+    <joint name="${trayname}_partition_3" type="fixed">
+      <parent link="${trayname}" />
+      <child link = "${trayname}_partition_3"/>
+      <origin rpy="0.0 0.0 0.0" xyz="0.105 0.15 0.02"/>
+    </joint>
+    <link name="${trayname}_partition_3"/>
   </xacro:macro>
+  <!-- ========== The tray with the screws and small parts -->
   <xacro:macro name="kitting_tray2" params="trayname parent *origin">
     <xacro:kitting_tray trayname="${trayname}" parent="${parent}">
       <xacro:insert_block name="origin"/>
     </xacro:kitting_tray>
-    <xacro:tray_contents trayname="${trayname}" contents="partition2">
-      <origin xyz="-0.095 0.14 0" rpy="0 0 ${-pi/2}"/>
+    <xacro:tray_contents trayname="${trayname}" contents="divider2">
+      <origin xyz="${tray_width/2 + mesh_offset_x - 0.095} ${tray_length/2 + mesh_offset_y +0.14} ${dividers_z_offset}" rpy="0 0 ${-pi/2}"/>
     </xacro:tray_contents>
     <xacro:tray_contents trayname="${trayname}" contents="screw_holder">
-      <origin xyz="-0.095 -0.05 0" rpy="0 0 ${-pi/2}"/>
+      <origin xyz="${tray_width/2 + mesh_offset_x - 0.095} ${tray_length/2 + mesh_offset_y -0.05} ${dividers_z_offset}" rpy="0 0 ${-pi/2}"/>
     </xacro:tray_contents>
+    <!-- ========== The extra frames to place and pick items are defined below -->
+    <xacro:auxiliary_frame parent="${trayname}" framename="partition_1">
+      <origin rpy="0.0 0.0 0.0" xyz="0.05 0.15 0.02"/>
+    </xacro:auxiliary_frame>
+    <!-- TODO: Insert the rest and fine tune -->
+    <xacro:property name="m4_x_0" value="0.18"/>
+    <xacro:property name="m4_x_delta" value="-0.03"/>
+    <xacro:property name="m4_y_0" value="0.03"/>
+    <xacro:property name="m4_y_delta" value="0.03"/>
+    <xacro:property name="m4_z_0" value="0.05"/>
+    <xacro:auxiliary_frame parent="${trayname}" framename="screw_m4_1">
+      <origin xyz="${m4_x_0 + m4_x_delta*0} ${m4_y_0 + m4_y_delta*0} ${m4_z_0}" rpy="0 ${pi/2} 0" />
+    </xacro:auxiliary_frame>
+    <xacro:auxiliary_frame parent="${trayname}" framename="screw_m4_2">
+      <origin xyz="${m4_x_0 + m4_x_delta*0} ${m4_y_0 + m4_y_delta*1} ${m4_z_0}" rpy="0 ${pi/2} 0" />
+    </xacro:auxiliary_frame>
+    <xacro:auxiliary_frame parent="${trayname}" framename="screw_m4_3">
+      <origin xyz="${m4_x_0 + m4_x_delta*0} ${m4_y_0 + m4_y_delta*2} ${m4_z_0}" rpy="0 ${pi/2} 0" />
+    </xacro:auxiliary_frame>
+    <xacro:auxiliary_frame parent="${trayname}" framename="screw_m4_4">
+      <origin xyz="${m4_x_0 + m4_x_delta*1} ${m4_y_0 + m4_y_delta*0} ${m4_z_0}" rpy="0 ${pi/2} 0" />
+    </xacro:auxiliary_frame>
+    <xacro:auxiliary_frame parent="${trayname}" framename="screw_m4_5">
+      <origin xyz="${m4_x_0 + m4_x_delta*1} ${m4_y_0 + m4_y_delta*1} ${m4_z_0}" rpy="0 ${pi/2} 0" />
+    </xacro:auxiliary_frame>
+    <xacro:auxiliary_frame parent="${trayname}" framename="screw_m4_6">
+      <origin xyz="${m4_x_0 + m4_x_delta*1} ${m4_y_0 + m4_y_delta*2} ${m4_z_0}" rpy="0 ${pi/2} 0" />
+    </xacro:auxiliary_frame>
+    <xacro:auxiliary_frame parent="${trayname}" framename="screw_m4_7">
+      <origin xyz="${m4_x_0 + m4_x_delta*2} ${m4_y_0 + m4_y_delta*0} ${m4_z_0}" rpy="0 ${pi/2} 0" />
+    </xacro:auxiliary_frame>
+    <xacro:auxiliary_frame parent="${trayname}" framename="screw_m4_8">
+      <origin xyz="${m4_x_0 + m4_x_delta*2} ${m4_y_0 + m4_y_delta*1} ${m4_z_0}" rpy="0 ${pi/2} 0" />
+    </xacro:auxiliary_frame>
+    <xacro:auxiliary_frame parent="${trayname}" framename="screw_m4_9">
+      <origin xyz="${m4_x_0 + m4_x_delta*2} ${m4_y_0 + m4_y_delta*2} ${m4_z_0}" rpy="0 ${pi/2} 0" />
+    </xacro:auxiliary_frame>
+    <xacro:property name="m3_x_0" value="0.08"/>
+    <xacro:property name="m3_x_delta" value="-0.03"/>
+    <xacro:property name="m3_y_0" value="0.03"/>
+    <xacro:property name="m3_y_delta" value="0.03"/>
+    <xacro:property name="m3_z_0" value="0.05"/>
+    <xacro:auxiliary_frame parent="${trayname}" framename="screw_m3_1">
+      <origin xyz="${m3_x_0 + m3_x_delta*0} ${m3_y_0 + m3_y_delta*0} ${m3_z_0}" rpy="0 ${pi/2} 0" />
+    </xacro:auxiliary_frame>
+    <xacro:auxiliary_frame parent="${trayname}" framename="screw_m3_2">
+      <origin xyz="${m3_x_0 + m3_x_delta*0} ${m3_y_0 + m3_y_delta*1} ${m3_z_0}" rpy="0 ${pi/2} 0" />
+    </xacro:auxiliary_frame>
+    <xacro:auxiliary_frame parent="${trayname}" framename="screw_m3_3">
+      <origin xyz="${m3_x_0 + m3_x_delta*0} ${m3_y_0 + m3_y_delta*2} ${m3_z_0}" rpy="0 ${pi/2} 0" />
+    </xacro:auxiliary_frame>
+    <xacro:auxiliary_frame parent="${trayname}" framename="screw_m3_4">
+      <origin xyz="${m3_x_0 + m3_x_delta*1} ${m3_y_0 + m3_y_delta*0} ${m3_z_0}" rpy="0 ${pi/2} 0" />
+    </xacro:auxiliary_frame>
+    <xacro:auxiliary_frame parent="${trayname}" framename="screw_m3_5">
+      <origin xyz="${m3_x_0 + m3_x_delta*1} ${m3_y_0 + m3_y_delta*1} ${m3_z_0}" rpy="0 ${pi/2} 0" />
+    </xacro:auxiliary_frame>
+    <xacro:auxiliary_frame parent="${trayname}" framename="screw_m3_6">
+      <origin xyz="${m3_x_0 + m3_x_delta*1} ${m3_y_0 + m3_y_delta*2} ${m3_z_0}" rpy="0 ${pi/2} 0" />
+    </xacro:auxiliary_frame>
   </xacro:macro>
 </robot>

File: o2as_scene_description/urdf/o2as_base_scene.urdf.xacro (robot description, xacro)
@@ -20,7 +20,6 @@
   <xacro:include filename="$(find o2as_scene_description)/urdf/ur3.urdf.xacro" />
   <!-- Scene items (trays, bins...) -->
-  <!-- <xacro:include filename="$(find o2as_scene_description)/urdf/kitting_tray_with_partitions.xacro" /> -->
-  <xacro:include filename="$(find o2as_scene_description)/urdf/taskboard_scene.xacro" />
-  <!-- <xacro:include filename="$(find o2as_scene_description)/urdf/kitting_scene.xacro" /> -->
+  <!-- <xacro:include filename="$(find o2as_scene_description)/urdf/taskboard_scene.xacro" /> -->
+  <xacro:include filename="$(find o2as_scene_description)/urdf/kitting_scene.xacro" />
   <!-- <xacro:include filename="$(find o2as_scene_description)/urdf/assembly_scene.xacro" /> -->
   <!-- Robot bases -->
@@ -60,7 +59,4 @@
   <xacro:screw_feeder feedername="m4_feeder" parent="c_bot_base_smfl">
     <origin xyz=".45 .05 .05" rpy="0 0 0" />
-  </xacro:screw_feeder> -->
-  <!-- <xacro:screw_feeder feedername="m5_feeder" parent="c_bot_base_smfl">
-    <origin xyz=".45 .2 .05" rpy="0 0 0" />
   </xacro:screw_feeder> -->
   <!-- robot arms -->
@@ -106,19 +102,9 @@
   <xacro:precision_gripper prefix="a_bot_"  grippername = "gripper" parent = "a_bot_tool0">
     <origin xyz="0.0 0 0.04" rpy="0 ${pi/2} 0"/>
-  </xacro:precision_gripper> -->
-  <!-- spawn and attach dual suction grippers -->
-  <!-- <xacro:include filename="$(find o2as_scene_description)/urdf/dual_suction_gripper.urdf.xacro" /> -->
-  <!-- <xacro:dual_suction_gripper_o2as prefix="b_bot_" parent = "b_bot_ee_link"> -->
-  <!--   <origin xyz="0 0 0" rpy="0 0 0"/> -->
-  <!-- </xacro:dual_suction_gripper_o2as> -->
+  </xacro:precision_gripper>
   <!-- spawn and attach dual robotiq 85 grippers -->
   <xacro:include filename="$(find o2as_scene_description)/urdf/robotiq_85_gripper_with_ft300.urdf.xacro" />
   <xacro:robotiq_85_gripper_o2as prefix="b_bot_" parent = "b_bot_ee_link" />
   <xacro:robotiq_85_gripper_o2as prefix="c_bot_" parent = "c_bot_ee_link"/>
-  <!-- spawn and attach dual suction grippers -->
-  <!-- <xacro:include filename="$(find o2as_scene_description)/urdf/dual_suction_gripper.urdf.xacro" /> -->
-  <!-- <xacro:dual_suction_gripper_o2as prefix="b_bot_" parent = "b_bot_ee_link">
-    <origin xyz="0 0 0" rpy="0 0 0"/>
-  </xacro:dual_suction_gripper_o2as> -->
   <!-- Add cameras -->
   <xacro:include filename="$(find o2as_realsense2_camera)/urdf/_d435.urdf.xacro" />
@@ -152,5 +138,4 @@
   <xacro:include filename="$(find o2as_scene_description)/urdf/phoxi_m_camera.urdf.xacro" />
   <xacro:phoxi_m_camera prefix="a_" parent="o2as_ground">
-    <!-- <origin xyz="0.56 0 ${bots_z + .1 + .8}" rpy="${-160*pi/180} 0 ${pi/2}"/> -->
     <origin xyz="0.46 0 ${bots_z + .1 + .8}" rpy="${-160*pi/180} 0 ${pi/2}"/>
   </xacro:phoxi_m_camera>

File: o2as_scene_description/urdf/templates/o2as_bin_template_front.xacro (robot description, xacro)
@@ -1,7 +1,4 @@
 <?xml version="1.0"?>
 <robot xmlns:xacro="http://www.ros.org/wiki/xacro" name="kitting_scene">
-  <xacro:include filename="$(find o2as_scene_description)/urdf/kitting_bin.xacro" />
-  <xacro:include filename="$(find o2as_scene_description)/urdf/kitting_tray.xacro" />
+  <xacro:include filename="$(find o2as_scene_description)/urdf/kitting_bin_macros.xacro" />
   <xacro:property name="rack_width" value=".640" />
-  <xacro:property name="tray_width" value=".300" />
-  <xacro:property name="tray_length" value=".210" />

File: o2as_scene_description/urdf/templates/o2as_bin_template_tail.xacro (robot description, xacro)
@@ -1,13 +1 @@
-  <!-- A row of tray -->
-  <xacro:property name="set3_x" value="${-(bin1_length/2+tray_length/2)}" />
-  <xacro:property name="set3_y" value="${.32-tray_width/2}" />
-  <xacro:property name="set3_z" value=".007" />
-  <!-- set3_tray_1 -->
-  <xacro:kitting_tray trayname="set3_tray_1" parent="workspace_center">
-    <origin xyz="${set3_x} ${set3_y} ${set3_z}" rpy="0 0 0" />
-  </xacro:kitting_tray>
-  <!-- set3_tray_2 -->
-  <xacro:kitting_tray trayname="set3_tray_2" parent="workspace_center">
-    <origin xyz="${set3_x} ${set3_y-tray_width} ${set3_z}" rpy="0 0 0" />
-  </xacro:kitting_tray>
 </robot>

Commit message: Update scene, calibrate robots

File: o2as_scene_description/urdf/assembly_scene.xacro (robot description, xacro)
@@ -4,8 +4,8 @@
   <!-- Insert: -->
   <xacro:kitting_tray1 trayname="tray_1" parent="workspace_center">
-    <origin xyz="-.2 -.27 0" rpy="0 0 ${pi/2}" />
+    <origin xyz="-.3 -.1 0" rpy="0 0 ${-pi/2}" />
   </xacro:kitting_tray1>
   <xacro:kitting_tray2 trayname="tray_2" parent="workspace_center">
-    <origin xyz="-.2 .27 0" rpy="0 0 ${-pi/2}" />
+    <origin xyz="-.3 .3 0" rpy="0 0 ${-pi/2}" />
   </xacro:kitting_tray2>
   <!-- The base plate -->

File: o2as_scene_description/urdf/o2as_base_scene.urdf.xacro (robot description, xacro)
@@ -21,5 +21,5 @@
   <!-- Scene items (trays, bins...) -->
   <!-- <xacro:include filename="$(find o2as_scene_description)/urdf/taskboard_scene.xacro" /> -->
-  <xacro:include filename="$(find o2as_scene_description)/urdf/kitting_scene.xacro" />
+  <!-- <xacro:include filename="$(find o2as_scene_description)/urdf/kitting_scene.xacro" /> -->
   <!-- <xacro:include filename="$(find o2as_scene_description)/urdf/assembly_scene.xacro" /> -->
   <!-- Robot bases -->
@@ -28,19 +28,19 @@
   <xacro:include filename="$(find o2as_scene_description)/urdf/o2as_base.xacro" />
   <xacro:o2as_base boxname="a_bot_base_smfl" parent="o2as_ground">
-    <origin xyz="${a_bot_x-.65/2} ${a_bot_y-.65/2} 0.65" rpy="0 0 0" />
+    <origin xyz="${a_bot_x-.65/2} ${a_bot_y-.65/2} 0.69" rpy="0 0 0" />
   </xacro:o2as_base>
   <xacro:o2as_base boxname="b_bot_base_smfl" parent="o2as_ground">
-    <origin xyz="${b_bot_x-.65/2} ${b_bot_y-.65/2} 0.65" rpy="0 0 0" />
+    <origin xyz="${b_bot_x-.65/2} ${b_bot_y-.65/2} 0.69" rpy="0 0 0" />
   </xacro:o2as_base>
   <xacro:o2as_base boxname="c_bot_base_smfl" parent="o2as_ground">
-    <origin xyz="${c_bot_x-.65/2-.22} ${c_bot_y-.65/2-.22} 0.65" rpy="0 0 0" />
+    <origin xyz="${c_bot_x-.65/2-.165} ${c_bot_y-.65/2-.095} 0.69" rpy="0 0 0" />
   </xacro:o2as_base>
   <!-- Main workspace -->
   <!-- The surface is 0.01 m below the robot bases and the "workspace_center" frame. -->
   <xacro:include filename="$(find o2as_scene_description)/urdf/o2as_box.xacro" />
-  <xacro:property name="plate_w" value="0.84"/>
-  <xacro:property name="plate_l" value="0.62"/>
+  <xacro:property name="plate_w" value="0.9"/>
+  <xacro:property name="plate_l" value="0.75"/>
   <xacro:o2as_box boxname="workbox" box_w="${plate_w}" box_l="${plate_l}" box_h=".01" parent="o2as_ground">
-    <origin xyz="${-plate_w/2} ${-plate_l/2} ${bots_z}" rpy="0 0 0" />
+    <origin xyz="${-plate_w/2 +.08} ${-plate_l/2} ${bots_z}" rpy="0 0 0" />
   </xacro:o2as_box>
   <link name="workspace_center" />
@@ -113,5 +113,5 @@
     <parent link="b_bot_wrist_2_link" />
     <child  link="b_bot_cam_holder_link" />
-    <origin xyz="0.0 -0.06 0.16" rpy="0.0 0.0 ${pi/2}" />
+    <origin xyz="0.0 -0.06 ${0.09465 + .13}" rpy="0.0 0.0 ${pi/2}" />
   </joint>
   <xacro:sensor_d435 prefix="b_bot_" parent="b_bot_cam_holder_link">

File: o2as_scene_description/urdf/robotiq_85_gripper_with_ft300.urdf.xacro (robot description, xacro)
@@ -5,5 +5,5 @@
   <!-- This seems too long when measuring the sensor,
        but works out when calibrating the tip_link to the world. -->
-  <xacro:property name="ft300_length" value="0.0555"/>
+  <xacro:property name="ft300_length" value="0.0525"/>
   <xacro:macro name="robotiq_85_gripper_o2as" params="prefix parent">
     <!-- Add the force sensor in front of the gripper. -->

Commit message: Fixes to changeTool, Screw actions
Also adds named frames to the screw tools

File: o2as_scene_description/urdf/assembly_scene.xacro (robot description, xacro)
@@ -4,8 +4,8 @@
   <!-- Insert: -->
   <xacro:kitting_tray1 trayname="tray_1" parent="workspace_center">
-    <origin xyz="-.3 -.1 0" rpy="0 0 ${-pi/2}" />
+    <origin xyz="-.15 0 0" rpy="0 0 ${-pi}" />
   </xacro:kitting_tray1>
   <xacro:kitting_tray2 trayname="tray_2" parent="workspace_center">
-    <origin xyz="-.3 .3 0" rpy="0 0 ${-pi/2}" />
+    <origin xyz="-.36 0 0" rpy="0 0 0" />
   </xacro:kitting_tray2>
   <!-- The base plate -->
@@ -16,7 +16,10 @@
     <origin xyz="0 0.1 .065" rpy="0 0 ${-pi/2}" />
   </xacro:full_assembly> -->
-    <xacro:include filename="$(find o2as_parts_description)/urdf/generated/full_assembly_frames_only.urdf.xacro"/>
+  <xacro:include filename="$(find o2as_parts_description)/urdf/generated/full_assembly_frames_only.urdf.xacro"/>
   <xacro:full_assembly_frames_only prefix="assembled_frames_only_" parent="workspace_center">
     <origin xyz="0 0.1 .065" rpy="0 0 ${-pi/2}" />
   </xacro:full_assembly_frames_only>
+  <xacro:assy_part_01 prefix="dummy" parent="assembled_frames_only_assy_part_01" spawn_attached="true">
+    <origin xyz="0 0 0" rpy="0 0 0" />
+  </xacro:assy_part_01>
 </robot>
