Commit message: Update scene, add assembly calibration

File: o2as_scene_description/urdf/assembly_scene.xacro (robot description, xacro)
@@ -2,10 +2,10 @@
 <robot xmlns:xacro="http://www.ros.org/wiki/xacro" name="kitting_scene">
   <xacro:include filename="$(find o2as_scene_description)/urdf/kitting_tray_with_partitions.xacro" />
-  <!-- Insert: -->
+  <!-- Trays: 30 cm x 21 cm -->
   <xacro:kitting_tray1 trayname="tray_1" parent="workspace_center">
-    <origin xyz="-.15 0 0" rpy="0 0 ${-pi}" />
+    <origin xyz="-.12 0 0" rpy="0 0 ${-pi}" />
   </xacro:kitting_tray1>
   <xacro:kitting_tray2 trayname="tray_2" parent="workspace_center">
-    <origin xyz="-.36 0 0" rpy="0 0 0" />
+    <origin xyz="-.12 .3 0" rpy="0 0 ${-pi}" />
   </xacro:kitting_tray2>
   <!-- The base plate -->
@@ -14,12 +14,19 @@
   <!-- <xacro:include filename="$(find o2as_parts_description)/urdf/generated/full_assembly.urdf.xacro"/>
   <xacro:full_assembly prefix="assembled_" parent="workspace_center">
-    <origin xyz="0 0.1 .065" rpy="0 0 ${-pi/2}" />
+    <origin xyz="-.04 0.1 .065" rpy="0 0 ${-pi/2}" />
   </xacro:full_assembly> -->
+  <xacro:property name="assy_dx" value="-.01" />
   <xacro:include filename="$(find o2as_parts_description)/urdf/generated/full_assembly_frames_only.urdf.xacro"/>
-  <xacro:full_assembly_frames_only prefix="assembled_frames_only_" parent="workspace_center">
-    <origin xyz="0 0.1 .065" rpy="0 0 ${-pi/2}" />
+  <xacro:full_assembly_frames_only prefix="assembled_" parent="workspace_center">
+    <origin xyz="${assy_dx} 0.1 .08" rpy="0 0 ${-pi/2}" />
   </xacro:full_assembly_frames_only>
-  <xacro:assy_part_01 prefix="dummy" parent="assembled_frames_only_assy_part_01" spawn_attached="true">
+  <xacro:assy_part_01 prefix="dummy" parent="assembled_assy_part_01" spawn_attached="true">
     <origin xyz="0 0 0" rpy="0 0 0" />
   </xacro:assy_part_01>
+  <xacro:assy_part_02 prefix="initial_" parent="workspace_center" spawn_attached="true">
+    <origin xyz="${assy_dx} 0.21 0" rpy="0 0 ${pi}" />
+  </xacro:assy_part_02>
+  <xacro:assy_part_03 prefix="initial_" parent="workspace_center" spawn_attached="true">
+    <origin xyz="${assy_dx} -0.2 0" rpy="0 0 ${pi}" />
+  </xacro:assy_part_03>
 </robot>

File: o2as_scene_description/urdf/kitting_tray_with_partitions.xacro (robot description, xacro)
@@ -5,8 +5,6 @@
   <xacro:property name="tray_width" value=".300" />
   <xacro:property name="tray_length" value=".210" />
-  <!-- TODO: Please adjust the width and length so that the origin is at the corner of the tray (this is easier to calibrate later) -->
   <xacro:property name="mesh_offset_x" value="-.045" />
   <xacro:property name="mesh_offset_y" value=".045" />
-  <!-- TODO: Is this mesh centered? Where is the coordinate origin? Check the dividers too. -->
   <!-- ========== The basic tray, without partitions -->
   <xacro:macro name="kitting_tray" params="trayname parent *origin">

File: o2as_scene_description/urdf/o2as_base_scene.urdf.xacro (robot description, xacro)
@@ -68,5 +68,5 @@
     wrist_2_lower_limit="${-pi}" wrist_2_upper_limit="${pi}"
     wrist_3_lower_limit="${-pi}" wrist_3_upper_limit="${pi}"/>
-  <xacro:ur5_robot prefix="b_bot_" joint_limited="true"
+  <xacro:ur5_robot prefix="b_bot_" joint_limited="false"
     shoulder_pan_lower_limit="${-pi}" shoulder_pan_upper_limit="${pi}"
     shoulder_lift_lower_limit="${-pi}" shoulder_lift_upper_limit="${pi}"
@@ -109,11 +109,11 @@
   <!-- Add cameras -->
   <xacro:include filename="$(find o2as_realsense2_camera)/urdf/_d435.urdf.xacro" />
-  <link name="b_bot_cam_holder_link" />
-  <joint name="b_bot_cam_holder_joint" type="fixed">
-    <parent link="b_bot_wrist_2_link" />
-    <child  link="b_bot_cam_holder_link" />
+  <link name="c_bot_cam_holder_link" />
+  <joint name="c_bot_cam_holder_joint" type="fixed">
+    <parent link="c_bot_wrist_2_link" />
+    <child  link="c_bot_cam_holder_link" />
     <origin xyz="0.0 -0.06 ${0.09465 + .13}" rpy="0.0 0.0 ${pi/2}" />
   </joint>
-  <xacro:sensor_d435 prefix="b_bot_" parent="b_bot_cam_holder_link">
+  <xacro:sensor_d435 prefix="c_bot_" parent="c_bot_cam_holder_link">
     <origin xyz="0 0 0" rpy="0 0 0"/>
   </xacro:sensor_d435>
@@ -122,5 +122,5 @@
   </xacro:sensor_d435> -->
   <!-- spawn and attach AR markers -->
-  <xacro:include filename="$(find o2as_gazebo)/urdf/o2as_ar_marker.urdf.xacro"/>
+  <!-- <xacro:include filename="$(find o2as_gazebo)/urdf/o2as_ar_marker.urdf.xacro"/>
   <xacro:o2as_ar_marker prefix="a_bot_" parent="a_bot_wrist_3_link"
    marker_id="17">
@@ -134,5 +134,5 @@
    marker_id="256">
     <origin xyz="0.0 0.12 0.05" rpy="0 0 ${pi/2}"/>
-  </xacro:o2as_ar_marker>
+  </xacro:o2as_ar_marker> -->
   <!-- Add PhoXi 3D scanners -->
   <xacro:include filename="$(find o2as_scene_description)/urdf/phoxi_m_camera.urdf.xacro" />

Commit message: Update assembly scene

File: o2as_scene_description/urdf/assembly_scene.xacro (robot description, xacro)
@@ -1,11 +1,11 @@
 <?xml version="1.0"?>
-<robot xmlns:xacro="http://www.ros.org/wiki/xacro" name="kitting_scene">
+<robot xmlns:xacro="http://www.ros.org/wiki/xacro" name="assembly_scene">
   <xacro:include filename="$(find o2as_scene_description)/urdf/kitting_tray_with_partitions.xacro" />
   <!-- Trays: 30 cm x 21 cm -->
   <xacro:kitting_tray1 trayname="tray_1" parent="workspace_center">
-    <origin xyz="-.12 0 0" rpy="0 0 ${-pi}" />
+    <origin xyz="0.1 -0.315 0" rpy="0 0 ${pi/2}" />
   </xacro:kitting_tray1>
   <xacro:kitting_tray2 trayname="tray_2" parent="workspace_center">
-    <origin xyz="-.12 .3 0" rpy="0 0 ${-pi}" />
+    <origin xyz="-0.2 0.315 0" rpy="0 0 ${-pi/2}" />
   </xacro:kitting_tray2>
   <!-- The base plate -->
@@ -25,8 +25,8 @@
   </xacro:assy_part_01>
   <xacro:assy_part_02 prefix="initial_" parent="workspace_center" spawn_attached="true">
-    <origin xyz="${assy_dx} 0.21 0" rpy="0 0 ${pi}" />
+    <origin xyz="-.2 0.06 0" rpy="0 0 ${pi}" />
   </xacro:assy_part_02>
   <xacro:assy_part_03 prefix="initial_" parent="workspace_center" spawn_attached="true">
-    <origin xyz="${assy_dx} -0.2 0" rpy="0 0 ${pi}" />
+    <origin xyz="-.2 -0.05 0" rpy="0 0 ${pi}" />
   </xacro:assy_part_03>
 </robot>

Commit message: Update scene, add calibration tests

File: o2as_scene_description/urdf/assembly_scene.xacro (robot description, xacro)
@@ -4,8 +4,8 @@
   <!-- Trays: 30 cm x 21 cm -->
   <xacro:kitting_tray1 trayname="tray_1" parent="workspace_center">
-    <origin xyz="0.1 -0.315 0" rpy="0 0 ${pi/2}" />
+    <origin xyz="0.05 0. 0" rpy="0 0 ${-pi/2}" />
   </xacro:kitting_tray1>
   <xacro:kitting_tray2 trayname="tray_2" parent="workspace_center">
-    <origin xyz="-0.2 0.315 0" rpy="0 0 ${-pi/2}" />
+    <origin xyz="0.35 0. 0" rpy="0 0 ${pi/2}" />
   </xacro:kitting_tray2>
   <!-- The base plate -->
@@ -24,9 +24,9 @@
     <origin xyz="0 0 0" rpy="0 0 0" />
   </xacro:assy_part_01>
-  <xacro:assy_part_02 prefix="initial_" parent="workspace_center" spawn_attached="true">
-    <origin xyz="-.2 0.06 0" rpy="0 0 ${pi}" />
-  </xacro:assy_part_02>
-  <xacro:assy_part_03 prefix="initial_" parent="workspace_center" spawn_attached="true">
-    <origin xyz="-.2 -0.05 0" rpy="0 0 ${pi}" />
-  </xacro:assy_part_03>
+  <xacro:assy_part_frames_only_02 prefix="initial_" parent="workspace_center" spawn_attached="true">
+    <origin xyz="-.18 -0.1 0" rpy="0 0 ${pi}" />
+  </xacro:assy_part_frames_only_02>
+  <xacro:assy_part_frames_only_03 prefix="initial_" parent="workspace_center" spawn_attached="true">
+    <origin xyz="-.18 0.095 0" rpy="0 0 ${pi}" />
+  </xacro:assy_part_frames_only_03>
 </robot>

Commit message: WIP: Add routine for idler assembly

File: o2as_scene_description/urdf/assembly_scene.xacro (robot description, xacro)
@@ -30,3 +30,6 @@
     <origin xyz="-.18 0.095 0" rpy="0 0 ${pi}" />
   </xacro:assy_part_frames_only_03>
+  <xacro:assy_part_frames_only_14 prefix="intermediate_" parent="workspace_center" spawn_attached="true">
+    <origin xyz=".25 -0.15 .40" rpy="${pi/2} ${-pi/2} 0" />
+  </xacro:assy_part_frames_only_14>
 </robot>

Commit message: Update assembly calibration and scene

File: o2as_scene_description/urdf/assembly_scene.xacro (robot description, xacro)
@@ -9,4 +9,21 @@
     <origin xyz="0.35 0. 0" rpy="0 0 ${pi/2}" />
   </xacro:kitting_tray2>
+  <!-- Retainer pin jig -->
+  <joint name="idler_pin_jig_joint" type="fixed">
+    <parent link="workspace_center"/>
+    <child link="idler_pin_jig_link"/>
+    <origin rpy="0.0 0.0 ${pi/2}" xyz="0.1 -0.3 0.032"/>
+  </joint>
+  <link name="idler_pin_jig_link">
+    <visual>
+      <origin xyz="0 0 ${-.032+.025/2}" rpy="0 0 0"/>
+      <geometry>
+        <cylinder length=".025" radius="0.01"/>
+      </geometry>
+      <material name="Brown">
+        <color rgba="0.7 0.4 0.2 1.0"/>
+      </material>
+    </visual>
+  </link>
   <xacro:include filename="$(find o2as_parts_description)/urdf/assembly_parts_macros.urdf.xacro"/>
   <!-- <xacro:include filename="$(find o2as_parts_description)/urdf/display_all_parts.urdf.xacro"/> -->
@@ -25,8 +42,8 @@
   </xacro:assy_part_01>
   <xacro:assy_part_frames_only_02 prefix="initial_" parent="workspace_center" spawn_attached="true">
-    <origin xyz="-.18 -0.1 0" rpy="0 0 ${pi}" />
+    <origin xyz="-.18 -0.05 0" rpy="0 0 ${pi}" />
   </xacro:assy_part_frames_only_02>
   <xacro:assy_part_frames_only_03 prefix="initial_" parent="workspace_center" spawn_attached="true">
-    <origin xyz="-.18 0.095 0" rpy="0 0 ${pi}" />
+    <origin xyz="-.18 0.045 0" rpy="0 0 ${pi}" />
   </xacro:assy_part_frames_only_03>
   <xacro:assy_part_frames_only_14 prefix="intermediate_" parent="workspace_center" spawn_attached="true">

Commit message: Fix pickup poses from tray

File: o2as_scene_description/urdf/assembly_scene.xacro (robot description, xacro)
@@ -10,10 +10,10 @@
   </xacro:kitting_tray2>
   <!-- Retainer pin jig -->
-  <joint name="idler_pin_jig_joint" type="fixed">
+  <joint name="retainer_pin_holder_joint" type="fixed">
     <parent link="workspace_center"/>
-    <child link="idler_pin_jig_link"/>
+    <child link="retainer_pin_holder_link"/>
     <origin rpy="0.0 0.0 ${pi/2}" xyz="0.1 -0.3 0.032"/>
   </joint>
-  <link name="idler_pin_jig_link">
+  <link name="retainer_pin_holder_link">
     <visual>
       <origin xyz="0 0 ${-.032+.025/2}" rpy="0 0 0"/>

File: o2as_scene_description/urdf/kitting_tray_with_partitions.xacro (robot description, xacro)
@@ -88,34 +88,34 @@
     </xacro:tray_contents>
     <!-- ========== The extra frames to place and pick items are defined below -->
-    <joint name="${trayname}_partition_1" type="fixed">
-      <parent link="${trayname}" />
-      <child link = "${trayname}_partition_1"/>
+    <xacro:auxiliary_frame parent="${trayname}" framename="_partition_1">
       <origin rpy="0.0 0.0 0.0" xyz="0.06 0.05 0.02"/>
-    </joint>
-    <link name="${trayname}_partition_1"/>
-    <joint name="${trayname}_partition_2" type="fixed">
-      <parent link="${trayname}" />
-      <child link = "${trayname}_partition_2"/>
+    </xacro:auxiliary_frame>
+    <xacro:auxiliary_frame parent="${trayname}" framename="_partition_2">
       <origin rpy="0.0 0.0 0.0" xyz="0.16 0.05 0.02"/>
-    </joint>
-    <link name="${trayname}_partition_2"/>
-    <joint name="${trayname}_partition_3" type="fixed">
-      <parent link="${trayname}" />
-      <child link = "${trayname}_partition_3"/>
+    </xacro:auxiliary_frame>
+    <xacro:auxiliary_frame parent="${trayname}" framename="_partition_3">
       <origin rpy="0.0 0.0 0.0" xyz="0.11 0.16 0.02"/>
-    </joint>
-    <link name="${trayname}_partition_3"/>
-    <joint name="${trayname}_partition_4" type="fixed">
-      <parent link="${trayname}" />
-      <child link = "${trayname}_partition_4"/>
+    </xacro:auxiliary_frame>
+    <xacro:auxiliary_frame parent="${trayname}" framename="_partition_4">
       <origin rpy="0.0 0.0 0.0" xyz="0.07 0.26 0.02"/>
-    </joint>
-    <link name="${trayname}_partition_4"/>
-    <joint name="${trayname}_partition_5" type="fixed">
-      <parent link="${trayname}" />
-      <child link = "${trayname}_partition_5"/>
+    </xacro:auxiliary_frame>
+    <xacro:auxiliary_frame parent="${trayname}" framename="_partition_5">
       <origin rpy="0.0 0.0 0.0" xyz="0.16 0.26 0.02"/>
-    </joint>
-    <link name="${trayname}_partition_5"/>
+    </xacro:auxiliary_frame>
+    <xacro:auxiliary_frame parent="${trayname}_partition_1" framename="pickup">
+      <origin rpy="0.0 0 0" xyz="0 0 0"/>
+    </xacro:auxiliary_frame>
+    <xacro:auxiliary_frame parent="${trayname}_partition_2" framename="pickup">
+      <origin rpy="0.0 0.0 0.0" xyz="0 0 0"/>
+    </xacro:auxiliary_frame>
+    <xacro:auxiliary_frame parent="${trayname}_partition_3" framename="pickup">
+      <origin rpy="0.0 0.0 0" xyz="-.05 0 0"/>
+    </xacro:auxiliary_frame>
+    <xacro:auxiliary_frame parent="${trayname}_partition_4" framename="pickup">
+      <origin rpy="0.0 ${pi*80/180} ${pi*20/180}" xyz="0 0 0.02"/>
+    </xacro:auxiliary_frame>
+    <xacro:auxiliary_frame parent="${trayname}_partition_5" framename="pickup">
+      <origin rpy="0.0 0.0 0" xyz="0 0 0"/>
+    </xacro:auxiliary_frame>
   </xacro:macro>
   <!-- ========== The tray with the screws and small parts -->
@@ -155,5 +155,34 @@
       <origin rpy="0.0 0.0 0.0" xyz="0.04 0.0525 0.02"/>
     </xacro:auxiliary_frame>
-    <!-- TODO: Insert the rest and fine tune -->
+    <!-- Frames used for picking up parts during assembly -->
+    <xacro:property name="partition_width" value="0.055"/>
+    <xacro:property name="partition_length" value="0.06"/>
+    <xacro:auxiliary_frame parent="${trayname}_partition_1" framename="pickup">
+      <origin rpy="0.0 0.0 ${-pi/4}" xyz="-.007 -.024 0"/>
+    </xacro:auxiliary_frame>
+    <xacro:auxiliary_frame parent="${trayname}_partition_2" framename="pickup">
+      <origin rpy="0.0 0.0 0.0" xyz="0 0 0.02"/>
+    </xacro:auxiliary_frame>
+    <xacro:auxiliary_frame parent="${trayname}_partition_3" framename="pickup">
+      <origin rpy="0.0 0.0 0.0" xyz="${partition_length/2 - .0045} ${-partition_width/2 + .0045} 0"/>
+    </xacro:auxiliary_frame>
+    <xacro:auxiliary_frame parent="${trayname}_partition_4" framename="pickup">
+      <origin rpy="0.0 0.0 0.0" xyz="${-partition_length/2 + .007} ${partition_width/2 - .007} 0"/>
+    </xacro:auxiliary_frame>
+    <xacro:auxiliary_frame parent="${trayname}_partition_5" framename="pickup">
+      <origin rpy="0.0 0.0 0.0" xyz="${partition_length/2 - .00475} ${partition_width/2 - .0055} 0"/>
+    </xacro:auxiliary_frame>
+    <xacro:auxiliary_frame parent="${trayname}_partition_6" framename="pickup">
+      <origin rpy="0.0 0.0 0.0" xyz="${-partition_length/2 + .015} ${partition_width/2 - .015} 0"/>
+    </xacro:auxiliary_frame>
+    <xacro:auxiliary_frame parent="${trayname}_partition_7" framename="pickup">
+      <origin rpy="0.0 0.0 0.0" xyz="${-partition_length/2 + .0085} ${partition_width/2 - .0085} 0"/>
+    </xacro:auxiliary_frame>
+    <xacro:auxiliary_frame parent="${trayname}_partition_8" framename="pickup_1">
+      <origin rpy="0.0 0.0 0.0" xyz="${partition_length/2 - .006} ${partition_width/2 - .006} 0"/>
+    </xacro:auxiliary_frame>
+    <xacro:auxiliary_frame parent="${trayname}_partition_8" framename="pickup_2">
+      <origin rpy="0.0 0.0 0.0" xyz="${-partition_length/2 + .006} ${partition_width/2 - .006} 0"/>
+    </xacro:auxiliary_frame>
     <xacro:property name="m4_x_0" value="0.04"/>
     <xacro:property name="m4_x_delta" value="0.03"/>

Commit message: WIP: Idler pin subtask

File: o2as_scene_description/urdf/assembly_scene.xacro (robot description, xacro)
@@ -48,5 +48,5 @@
   </xacro:assy_part_frames_only_03>
   <xacro:assy_part_frames_only_14 prefix="intermediate_" parent="workspace_center" spawn_attached="true">
-    <origin xyz=".25 -0.15 .40" rpy="${pi/2} ${-pi/2} 0" />
+    <origin xyz=".25 -0.15 .50" rpy="${pi/2} ${-pi/2} 0" />
   </xacro:assy_part_frames_only_14>
 </robot>

File: o2as_scene_description/urdf/kitting_tray_with_partitions.xacro (robot description, xacro)
@@ -88,17 +88,17 @@
     </xacro:tray_contents>
     <!-- ========== The extra frames to place and pick items are defined below -->
-    <xacro:auxiliary_frame parent="${trayname}" framename="_partition_1">
+    <xacro:auxiliary_frame parent="${trayname}" framename="partition_1">
       <origin rpy="0.0 0.0 0.0" xyz="0.06 0.05 0.02"/>
     </xacro:auxiliary_frame>
-    <xacro:auxiliary_frame parent="${trayname}" framename="_partition_2">
+    <xacro:auxiliary_frame parent="${trayname}" framename="partition_2">
       <origin rpy="0.0 0.0 0.0" xyz="0.16 0.05 0.02"/>
     </xacro:auxiliary_frame>
-    <xacro:auxiliary_frame parent="${trayname}" framename="_partition_3">
+    <xacro:auxiliary_frame parent="${trayname}" framename="partition_3">
       <origin rpy="0.0 0.0 0.0" xyz="0.11 0.16 0.02"/>
     </xacro:auxiliary_frame>
-    <xacro:auxiliary_frame parent="${trayname}" framename="_partition_4">
+    <xacro:auxiliary_frame parent="${trayname}" framename="partition_4">
       <origin rpy="0.0 0.0 0.0" xyz="0.07 0.26 0.02"/>
     </xacro:auxiliary_frame>
-    <xacro:auxiliary_frame parent="${trayname}" framename="_partition_5">
+    <xacro:auxiliary_frame parent="${trayname}" framename="partition_5">
       <origin rpy="0.0 0.0 0.0" xyz="0.16 0.26 0.02"/>
     </xacro:auxiliary_frame>

Commit message: Fixes for assembly idler pin
Still needs to push down on the bearing

File: o2as_scene_description/urdf/assembly_scene.xacro (robot description, xacro)
@@ -4,8 +4,8 @@
   <!-- Trays -->
   <xacro:kitting_tray1 trayname="tray_1" parent="workspace_center">
-    <origin xyz="0.05 0. 0" rpy="0 0 ${-pi/2}" />
+    <origin xyz="0.05 -.03 0" rpy="0 0 ${-pi/2}" />
   </xacro:kitting_tray1>
   <xacro:kitting_tray2 trayname="tray_2" parent="workspace_center">
-    <origin xyz="0.35 0. 0" rpy="0 0 ${pi/2}" />
+    <origin xyz="0.35 0 0" rpy="0 0 ${pi/2}" />
   </xacro:kitting_tray2>
   <!-- Retainer pin jig -->

File: o2as_scene_description/urdf/kitting_tray_with_partitions.xacro (robot description, xacro)
@@ -113,8 +113,8 @@
     </xacro:auxiliary_frame>
     <xacro:auxiliary_frame parent="${trayname}_partition_4" framename="pickup">
-      <origin rpy="0.0 ${pi*80/180} ${pi*20/180}" xyz="0 0 0.02"/>
+      <origin rpy="0.0 ${pi*80/180} ${pi*20/180}" xyz="0.03 -.01 0.02"/>
     </xacro:auxiliary_frame>
     <xacro:auxiliary_frame parent="${trayname}_partition_5" framename="pickup">
-      <origin rpy="0.0 0.0 0" xyz="0 0 0"/>
+      <origin rpy="0.0 0.0 0" xyz="-.02 -.01 0"/>
     </xacro:auxiliary_frame>
   </xacro:macro>

File: o2as_scene_description/urdf/o2as_base_scene.urdf.xacro (robot description, xacro)
@@ -22,6 +22,6 @@
   <!-- Scene items (trays, bins...) -->
   <!-- <xacro:include filename="$(find o2as_scene_description)/urdf/taskboard_scene.xacro" /> -->
-  <xacro:include filename="$(find o2as_scene_description)/urdf/kitting_scene.xacro" />
-  <!-- <xacro:include filename="$(find o2as_scene_description)/urdf/assembly_scene.xacro" /> -->
+  <!-- <xacro:include filename="$(find o2as_scene_description)/urdf/kitting_scene.xacro" /> -->
+  <xacro:include filename="$(find o2as_scene_description)/urdf/assembly_scene.xacro" />
   <!-- <xacro:include filename="$(find o2as_scene_description)/urdf/calibration_scene.xacro" /> -->
   <!-- Robot bases -->

File: o2as_scene_description/urdf/robotiq_c_bot_gripper.urdf.xacro (robot description, xacro)
@@ -42,5 +42,5 @@
       <parent link="${prefix}robotiq_85_tip_40deg_helper_link"/>
       <child link="${prefix}nut_tool_m6_tip_link"/>
-      <origin rpy="0 0 0" xyz="0.057 0.0 -.014 "/>
+      <origin rpy="0 0 0" xyz="0.05 0.0 -.018 "/>
     </joint>
     <link name="${prefix}nut_tool_m6_tip_link"/>

Commit message: WIP: Pulley fixes

File: o2as_scene_description/urdf/assembly_scene.xacro (robot description, xacro)
@@ -27,14 +27,14 @@
   </link>
   <xacro:include filename="$(find o2as_parts_description)/urdf/assembly_parts_macros.urdf.xacro"/>
-  <xacro:include filename="$(find o2as_parts_description)/urdf/display_all_parts.urdf.xacro"/>
-  <xacro:include filename="$(find o2as_parts_description)/urdf/generated/full_assembly.urdf.xacro"/>
+  <!-- <xacro:include filename="$(find o2as_parts_description)/urdf/display_all_parts.urdf.xacro"/> -->
+  <xacro:property name="assy_dx" value="-.01" />
+  <!-- <xacro:include filename="$(find o2as_parts_description)/urdf/generated/full_assembly.urdf.xacro"/>
   <xacro:full_assembly prefix="assembled_" parent="workspace_center">
-    <origin xyz="-.04 0.1 .065" rpy="0 0 ${-pi/2}" />
-  </xacro:full_assembly>
-  <xacro:property name="assy_dx" value="-.01" />
+    <origin xyz="${assy_dx} 0.1 .08" rpy="0 0 ${-pi/2}" />
+  </xacro:full_assembly> -->
   <xacro:include filename="$(find o2as_parts_description)/urdf/generated/full_assembly_frames_only.urdf.xacro"/>
-  <!-- <xacro:full_assembly_frames_only prefix="assembled_" parent="workspace_center">
+  <xacro:full_assembly_frames_only prefix="assembled_" parent="workspace_center">
     <origin xyz="${assy_dx} 0.1 .08" rpy="0 0 ${-pi/2}" />
-  </xacro:full_assembly_frames_only> -->
+  </xacro:full_assembly_frames_only>
   <!-- The base plate -->
   <xacro:assy_part_01 prefix="dummy" parent="assembled_assy_part_01" spawn_attached="true">
