Commit message: Clean code, set up scene, add some comments

File: o2as_scene_description/urdf/assembly_scene.xacro (robot description, xacro)
@@ -9,5 +9,5 @@
     <origin xyz="0.35 0 0" rpy="0 0 ${pi/2}" />
   </xacro:kitting_tray2>
-  <!-- Retainer pin jig -->
+  <!-- Retainer pin jig (used to hold the retainer pin for resetting during the task) -->
   <joint name="retainer_pin_holder_joint" type="fixed">
     <parent link="workspace_center"/>

File: o2as_scene_description/urdf/kitting_scene.xacro (robot description, xacro)
@@ -13,5 +13,5 @@
     <origin xyz=".52 -0.25 .065" rpy="0 0 ${pi/2}" />
   </xacro:screw_feeder> -->
-  <!-- spawn and attach dual suction grippers -->
+  <!-- spawn and attach dual suction grippers (used for testing at AIST) -->
   <!-- <xacro:include filename="$(find o2as_scene_description)/urdf/dual_suction_gripper.urdf.xacro" />
   <xacro:dual_suction_gripper_o2as prefix="b_bot_" parent = "b_bot_ee_link">
@@ -50,11 +50,3 @@
     <origin xyz=".55 ${tray_length-.1} 0.01" rpy="0 0 ${pi/2}" />
   </xacro:kitting_tray1>
-  <!-- <xacro:property name="tray_x" value="${-tray_length+.01}" />
-  <xacro:property name="tray_y" value="0" />
-  <xacro:kitting_tray1 trayname="tray_1" parent="rack_trays_center">
-    <origin xyz="${tray_x} ${tray_y} 0" rpy="0 0 0" />
-  </xacro:kitting_tray1>
-  <xacro:kitting_tray2 trayname="tray_2" parent="rack_trays_center">
-    <origin xyz="+.01 0 0" rpy="0 0 ${pi}" />
-  </xacro:kitting_tray2> -->
 </robot>

File: o2as_scene_description/urdf/o2as_base_scene.urdf.xacro (robot description, xacro)
@@ -23,7 +23,7 @@
   <!-- <xacro:include filename="$(find o2as_scene_description)/urdf/taskboard_scene.xacro" /> -->
   <!-- <xacro:include filename="$(find o2as_scene_description)/urdf/kitting_scene.xacro" /> -->
-  <!-- <xacro:include filename="$(find o2as_scene_description)/urdf/assembly_scene.xacro" /> -->
+  <xacro:include filename="$(find o2as_scene_description)/urdf/assembly_scene.xacro" />
   <!-- <xacro:include filename="$(find o2as_scene_description)/urdf/calibration_scene.xacro" /> -->
-  <xacro:include filename="$(find o2as_scene_description)/urdf/assembly_new_parts_scene.xacro" />
+  <!-- <xacro:include filename="$(find o2as_scene_description)/urdf/assembly_new_parts_scene.xacro" /> -->
   <!-- Robot bases -->
   <!-- Putting these at height 0.0 makes them intersect with the ground, so they are elevated. -->
@@ -103,14 +103,16 @@
     <origin xyz="0.0 0 0.0" rpy="0 0 0"/>
   </xacro:InnerOnlyGripper>
-  <xacro:include filename="$(find o2as_scene_description)/urdf/dual_suction_gripper.urdf.xacro"/>
+  <!-- spawn and attach dual robotiq 85 grippers (two different macros are used because different tool frames are defined inside) -->
+  <xacro:include filename="$(find o2as_scene_description)/urdf/robotiq_b_bot_gripper.urdf.xacro" />
+  <xacro:o2as_b_bot_gripper prefix="b_bot_" parent = "b_bot_ee_link" />
+  <xacro:include filename="$(find o2as_scene_description)/urdf/robotiq_c_bot_gripper.urdf.xacro" />
+  <xacro:o2as_c_bot_gripper prefix="c_bot_" parent = "c_bot_ee_link"/>
+  <!-- Alternative suction-only grippers used to test at AIST -->
+  <!-- <xacro:include filename="$(find o2as_scene_description)/urdf/dual_suction_gripper.urdf.xacro"/>
   <xacro:dual_suction_gripper_o2as prefix="b_bot_" parent="b_bot_ee_link">
     <origin xyz="0 0 0" rpy="0 0 0" />
-  </xacro:dual_suction_gripper_o2as>
-  <!-- spawn and attach dual robotiq 85 grippers -->
-  <!-- <xacro:o2as_b_bot_gripper prefix="b_bot_" parent = "b_bot_ee_link" /> -->
-  <xacro:include filename="$(find o2as_scene_description)/urdf/robotiq_c_bot_gripper.urdf.xacro" />
-  <xacro:o2as_c_bot_gripper prefix="c_bot_" parent = "c_bot_ee_link"/>
-  <!-- Feeders -->
-  <xacro:include filename="$(find o2as_scene_description)/urdf/screw_feeder.xacro" />
+  </xacro:dual_suction_gripper_o2as> -->
+  <!-- Feeders (used only during kitting and taskboard task) -->
+  <!-- <xacro:include filename="$(find o2as_scene_description)/urdf/screw_feeder.xacro" />
   <xacro:screw_feeder feedername="m3_feeder" parent="c_bot_base_smfl">
     <origin xyz=".64 -0.25 .035" rpy="0 0 ${pi/2}" />
@@ -118,5 +120,5 @@
   <xacro:screw_feeder feedername="m4_feeder" parent="c_bot_base_smfl">
     <origin xyz=".50 -0.25 .035" rpy="0 0 ${pi/2}" />
-  </xacro:screw_feeder>
+  </xacro:screw_feeder> -->
   <!-- Add cameras -->
   <xacro:include filename="$(find o2as_realsense2_camera)/urdf/_d435.urdf.xacro" />
@@ -130,5 +132,4 @@
     <origin xyz="0 0 0" rpy="0 0 0"/>
   </xacro:sensor_d435>
-  <xacro:include filename="$(find o2as_realsense2_camera)/urdf/_d435.urdf.xacro" />
   <link name="a_bot_cam_holder_link" />
   <joint name="a_bot_cam_holder_joint" type="fixed">
@@ -140,41 +141,9 @@
     <origin xyz="0 0 0" rpy="0 0 0"/>
   </xacro:sensor_d435>
-  <!-- Add PhoXi 3D scanners -->
+  <!-- Add PhoXi 3D scanner -->
   <xacro:include filename="$(find o2as_scene_description)/urdf/phoxi_m_camera.urdf.xacro" />
   <xacro:phoxi_m_camera prefix="a_" parent="o2as_ground">
   <origin xyz="0.652663578768 -0.0142895785849 1.50687788672" rpy="${-161.381811856*pi/180} ${2.99567722105*pi/180} ${90.8962573459*pi/180}"/>
   </xacro:phoxi_m_camera>
-  <!-- Add AR markers -->
-  <xacro:include filename="$(find o2as_gazebo)/urdf/o2as_ar_marker.urdf.xacro"/>
-  <xacro:o2as_ar_marker prefix="a_bot_"
-  			parent="a_bot_ee_link"
-  			marker_id="26">
-    <origin xyz="0.08 0.00 0.065" rpy="0 0 0"/>
-  </xacro:o2as_ar_marker>
-  <xacro:o2as_ar_marker prefix="b_bot_"
-  			parent="b_bot_dual_suction_gripper_base_link"
-  			marker_id="26">
-    <origin xyz="0.063 0.0 0.0215" rpy="0 0 0"/>
-  </xacro:o2as_ar_marker>
-  <!-- <xacro:o2as_ar_marker prefix="b_bot_" -->
-  <!-- 			parent="b_bot_single_suction_gripper_base_link" -->
-  <!-- 			marker_id="26"> -->
-  <!--   <origin xyz="0.063 0.0 0.0215" rpy="0 0 0"/> -->
-  <!-- </xacro:o2as_ar_marker> -->
-  <!-- <xacro:o2as_ar_marker prefix="b_bot_" -->
-  <!-- 			parent="b_bot_robotiq_85_tip_link" -->
-  <!-- 			marker_id="26"> -->
-  <!--   <origin xyz="0.0 0.0 0.0185" rpy="0 0 0"/> -->
-  <!-- </xacro:o2as_ar_marker> -->
-  <xacro:o2as_ar_marker prefix="c_bot_"
-			parent="c_bot_robotiq_85_tip_link"
-			marker_id="26">
-    <origin xyz="0.0 0.0 0.0185" rpy="0 0 0"/>
-  </xacro:o2as_ar_marker>
-  <xacro:o2as_ar_marker_16cm prefix="workspace_"
-  			     parent="workspace_center"
-  			     marker_id="32">
-    <origin xyz="0.0 0.0 0.0005" rpy="0 0 0"/>
-  </xacro:o2as_ar_marker_16cm>
   <!-- I would like to remove the "world" link definition, but apparently it is necessary for Gazebo -->
   <link name="world" />
