Commit message: WIP: Works with all robots, but without wall collision

File: o2as_scene_description/urdf/o2as_base_scene.urdf.xacro (robot description, xacro)
@@ -3,7 +3,7 @@
        name="o2as_base_scene" >
   <xacro:property name="a_bot_x" value="0.0"/>
-  <xacro:property name="a_bot_y" value="-0.5"/>
+  <xacro:property name="a_bot_y" value="-0.6"/>
   <xacro:property name="b_bot_x" value="0.0"/>
-  <xacro:property name="b_bot_y" value="0.5"/>
+  <xacro:property name="b_bot_y" value="0.6"/>
   <xacro:property name="c_bot_x" value="-0.5"/>
   <xacro:property name="c_bot_y" value="0.0"/>
@@ -17,5 +17,5 @@
   <xacro:include filename="$(find o2as_scene_description)/urdf/ur3.urdf.xacro" />
   <!-- Scene items (trays, bins...) -->
-  <xacro:include filename="$(find o2as_scene_description)/urdf/walls.xacro" />
+  <!-- <xacro:include filename="$(find o2as_scene_description)/urdf/walls.xacro" /> -->
   <xacro:include filename="$(find o2as_scene_description)/urdf/kitting_scene.xacro" />
   <!-- Robot bases -->
@@ -47,4 +47,8 @@
   </joint>
   <!-- robot arms -->
+    <xacro:ur5_robot prefix="a_bot_" joint_limited="false"/>
+  <xacro:ur5_robot prefix="b_bot_" joint_limited="false"/>
+  <xacro:ur3_robot prefix="c_bot_" joint_limited="false"/>
+<!--
   <xacro:ur5_robot prefix="a_bot_" joint_limited="true"
     shoulder_pan_lower_limit="${-pi}" shoulder_pan_upper_limit="${pi}"
@@ -67,5 +71,5 @@
     wrist_1_lower_limit="${-pi}" wrist_1_upper_limit="${pi}"
     wrist_2_lower_limit="${-pi}" wrist_2_upper_limit="${pi}"
-    wrist_3_lower_limit="${-pi}" wrist_3_upper_limit="${pi}"/>
+    wrist_3_lower_limit="${-pi}" wrist_3_upper_limit="${pi}"/> -->
   <link name="o2as_ground" />
   <joint name="world_a_bot_joint" type="fixed">

File: o2as_scene_description/urdf/walls.xacro (robot description, xacro)
@@ -39,5 +39,5 @@
   <!-- ############################# -->
   <xacro:o2as_wall wall_name="wall_b" wall_w="${wall_width}" wall_l="${wall_thickness}" wall_h="${wall_height}">
-    <origin xyz="0.0 -0.9 0.0" rpy="0.0 0.0 0.0" />
+    <origin xyz="0.0 -1.0 0.0" rpy="0.0 0.0 0.0" />
   </xacro:o2as_wall>
   <xacro:o2as_wall wall_name="wall_c" wall_w="${wall_width}" wall_l="${wall_thickness}" wall_h="${wall_height}">

Commit message: Add walls, readme
Also moved the launch file out of the definition package

File: o2as_scene_description/urdf/o2as_base_scene.urdf.xacro (robot description, xacro)
@@ -17,5 +17,5 @@
   <xacro:include filename="$(find o2as_scene_description)/urdf/ur3.urdf.xacro" />
   <!-- Scene items (trays, bins...) -->
-  <!-- <xacro:include filename="$(find o2as_scene_description)/urdf/walls.xacro" /> -->
+  <xacro:include filename="$(find o2as_scene_description)/urdf/walls.xacro" />
   <xacro:include filename="$(find o2as_scene_description)/urdf/kitting_scene.xacro" />
   <!-- Robot bases -->
@@ -47,8 +47,4 @@
   </joint>
   <!-- robot arms -->
-    <xacro:ur5_robot prefix="a_bot_" joint_limited="false"/>
-  <xacro:ur5_robot prefix="b_bot_" joint_limited="false"/>
-  <xacro:ur3_robot prefix="c_bot_" joint_limited="false"/>
-<!--
   <xacro:ur5_robot prefix="a_bot_" joint_limited="true"
     shoulder_pan_lower_limit="${-pi}" shoulder_pan_upper_limit="${pi}"
@@ -71,5 +67,5 @@
     wrist_1_lower_limit="${-pi}" wrist_1_upper_limit="${pi}"
     wrist_2_lower_limit="${-pi}" wrist_2_upper_limit="${pi}"
-    wrist_3_lower_limit="${-pi}" wrist_3_upper_limit="${pi}"/> -->
+    wrist_3_lower_limit="${-pi}" wrist_3_upper_limit="${pi}"/>
   <link name="o2as_ground" />
   <joint name="world_a_bot_joint" type="fixed">

File: o2as_scene_description/urdf/walls.xacro (robot description, xacro)
@@ -16,4 +16,5 @@
       </visual>
       <collision>
+      <origin xyz="0 ${wall_l/2} ${wall_h/2}" rpy="0 0 0"/>
         <geometry>
           <box size="${wall_w} ${wall_l} ${wall_h}"/>
@@ -42,5 +43,5 @@
   </xacro:o2as_wall>
   <xacro:o2as_wall wall_name="wall_c" wall_w="${wall_width}" wall_l="${wall_thickness}" wall_h="${wall_height}">
-    <origin xyz="-1.3 0.0 0.0" rpy="0.0 0.0 ${pi/2}" />
+    <origin xyz="-1.0 0.0 0.0" rpy="0.0 0.0 ${pi/2}" />
   </xacro:o2as_wall>
 </robot>

Commit message: Attach camera to correct wrist link

File: o2as_scene_description/urdf/o2as_base_scene.urdf.xacro (robot description, xacro)
@@ -100,7 +100,7 @@
   <link name="b_bot_cam_holder_link" />
   <joint name="b_bot_cam_holder_joint" type="fixed">
-    <parent link="b_bot_wrist_3_link" />
+    <parent link="b_bot_wrist_2_link" />
     <child link = "b_bot_cam_holder_link" />
-    <origin xyz="0.0 -0.06 0.06" rpy="0.0 0.0 ${pi/2}" />
+    <origin xyz="0.0 -0.06 0.16" rpy="0.0 0.0 ${pi/2}" />
   </joint>
   <xacro:sensor_r410 prefix="b_bot_" parent = "b_bot_cam_holder_link">

Commit message: Add d435 camera, fix dependency error

File: o2as_scene_description/urdf/o2as_base_scene.urdf.xacro (robot description, xacro)
@@ -13,5 +13,5 @@
   <xacro:include filename="$(find ur_description)/urdf/common.gazebo.xacro" />
   <xacro:include filename="$(find o2as_scene_description)/urdf/o2as_base_scene.gazebo" />
-  <xacro:include filename="$(find realsense2_camera)/urdf/_r410.urdf.xacro" />
+  <xacro:include filename="$(find realsense2_camera)/urdf/_d435.urdf.xacro" />
   <!-- robots -->
   <!-- <xacro:include filename="$(find o2as_scene_description)/urdf/ur10.urdf.xacro" /> -->
@@ -104,7 +104,8 @@
     <origin xyz="0.0 -0.06 0.16" rpy="0.0 0.0 ${pi/2}" />
   </joint>
-  <xacro:sensor_r410 prefix="b_bot_" parent = "b_bot_cam_holder_link">
-    <origin xyz="0 0.05 0" rpy="0 0 0"/>
-  </xacro:sensor_r410>
+  <!-- prefix="b_bot_"  -->
+  <xacro:sensor_d435 parent = "b_bot_cam_holder_link">
+    <origin xyz="0 0 0" rpy="0 0 0"/>
+  </xacro:sensor_d435>
   <!-- I meant to remove the "world" link definition, but apparently it is necessary for Gazebo -->
   <link name="world" />

Commit message: Move camera

File: o2as_scene_description/urdf/o2as_base_scene.urdf.xacro (robot description, xacro)
@@ -100,7 +100,9 @@
   <link name="b_bot_cam_holder_link" />
   <joint name="b_bot_cam_holder_joint" type="fixed">
-    <parent link="b_bot_wrist_2_link" />
+    <!-- <parent link="b_bot_wrist_2_link" /> -->
+    <parent link="workspace_center" />
     <child link = "b_bot_cam_holder_link" />
-    <origin xyz="0.0 -0.06 0.16" rpy="0.0 0.0 ${pi/2}" />
+    <!-- <origin xyz="0.0 -0.06 0.16" rpy="0.0 0.0 ${pi/2}" /> -->
+    <origin xyz="0.0 0.0 0.7" rpy="0.0 ${pi/2} 0.0" />
   </joint>
   <xacro:sensor_d435 prefix="b_bot_" parent="b_bot_cam_holder_link">

Commit message: Revert camera changes

File: o2as_scene_description/urdf/o2as_base_scene.urdf.xacro (robot description, xacro)
@@ -12,5 +12,5 @@
   <!-- common stuff -->
   <xacro:include filename="$(find ur_description)/urdf/common.gazebo.xacro" />
-  <xacro:include filename="$(find o2as_gazebo)/launch/o2as_base_scene.gazebo" />
+  <xacro:include filename="$(find o2as_gazebo)/urdf/o2as_base_scene.gazebo" />
   <xacro:include filename="$(find realsense2_camera)/urdf/_d435.urdf.xacro" />
   <!-- robots -->
@@ -100,9 +100,7 @@
   <link name="b_bot_cam_holder_link" />
   <joint name="b_bot_cam_holder_joint" type="fixed">
-    <!-- <parent link="b_bot_wrist_2_link" /> -->
-    <parent link="workspace_center" />
+    <parent link="b_bot_wrist_2_link" />
     <child link = "b_bot_cam_holder_link" />
-    <!-- <origin xyz="0.0 -0.06 0.16" rpy="0.0 0.0 ${pi/2}" /> -->
-    <origin xyz="0.0 0.0 0.7" rpy="0.0 ${pi/2} 0.0" />
+    <origin xyz="0.0 -0.06 0.16" rpy="0.0 0.0 ${pi/2}" />
   </joint>
   <xacro:sensor_d435 prefix="b_bot_" parent="b_bot_cam_holder_link">

Commit message: Add screw tools to scene & screw skill stubs

File: o2as_scene_description/urdf/o2as_base_scene.urdf.xacro (robot description, xacro)
@@ -2,12 +2,13 @@
 <robot xmlns:xacro="http://ros.org/wiki/xacro"
        name="o2as_base_scene" >
+  <!-- This is the main file defining our robot arrangement and physical environment. -->
+  <!-- These values are still not fixed -->
   <xacro:property name="a_bot_x" value="0.0"/>
-  <xacro:property name="a_bot_y" value="-0.6"/>
+  <xacro:property name="a_bot_y" value="-0.65"/>
   <xacro:property name="b_bot_x" value="0.0"/>
-  <xacro:property name="b_bot_y" value="0.6"/>
+  <xacro:property name="b_bot_y" value="0.65"/>
   <xacro:property name="c_bot_x" value="-0.5"/>
   <xacro:property name="c_bot_y" value="0.0"/>
   <xacro:property name="bots_z" value="0.75"/>
-  <!-- This is the main file defining our robot arrangement and physical environment. -->
   <!-- common stuff -->
   <xacro:include filename="$(find ur_description)/urdf/common.gazebo.xacro" />
@@ -26,19 +27,19 @@
   <xacro:include filename="$(find o2as_scene_description)/urdf/o2as_base.xacro" />
   <xacro:o2as_base boxname="a_bot_base_smfl" parent="o2as_ground">
-    <origin xyz="${a_bot_x-.65/2} ${a_bot_y-.65/2} 0.65" rpy="0 0 0" />
+    <origin xyz="${a_bot_x-.65/2} ${a_bot_y-.65/2} ${bots_z-.06}" rpy="0 0 0" />
   </xacro:o2as_base>
   <xacro:o2as_base boxname="b_bot_base_smfl" parent="o2as_ground">
-    <origin xyz="${b_bot_x-.65/2} ${b_bot_y-.65/2} 0.65" rpy="0 0 0" />
+    <origin xyz="${b_bot_x-.65/2} ${b_bot_y-.65/2} ${bots_z-.06}" rpy="0 0 0" />
   </xacro:o2as_base>
   <xacro:o2as_base boxname="c_bot_base_smfl" parent="o2as_ground">
-    <origin xyz="${c_bot_x-.65/2-.22} ${c_bot_y-.65/2-.22} 0.65" rpy="0 0 0" />
+    <origin xyz="${c_bot_x-.65/2-.16} ${c_bot_y-.65/2-.1} ${bots_z-.06}" rpy="0 0 0" />
   </xacro:o2as_base>
   <!-- Main workspace -->
   <!-- The surface is 0.01 m below the robot bases and the "workspace_center" frame. -->
   <xacro:include filename="$(find o2as_scene_description)/urdf/o2as_box.xacro" />
-  <xacro:property name="plate_w" value="0.84"/>
-  <xacro:property name="plate_l" value="0.62"/>
+  <xacro:property name="plate_w" value="0.9"/>
+  <xacro:property name="plate_l" value="0.75"/>
   <xacro:o2as_box boxname="workbox" box_w="${plate_w}" box_l="${plate_l}" box_h=".01" parent="o2as_ground">
-    <origin xyz="${-plate_w/2} ${-plate_l/2} ${bots_z+.09}" rpy="0 0 0" />
+    <origin xyz="${-plate_w/2+.1} ${-plate_l/2} ${bots_z}" rpy="0 0 0" />
   </xacro:o2as_box>
   <link name="workspace_center" />
@@ -46,6 +47,19 @@
     <parent link="o2as_ground" />
     <child link="workspace_center" />
-    <origin xyz="0.0 0.0 ${bots_z+.1}" rpy="0.0 0.0 0.0" />
+    <origin xyz="0.0 0.0 ${bots_z+.01}" rpy="0.0 0.0 0.0" />
   </joint>
+  <!-- Screw holder & screw tool visual -->
+  <xacro:include filename="$(find o2as_scene_description)/urdf/screw_tools.xacro" />
+  <!-- Feeders -->
+  <xacro:include filename="$(find o2as_scene_description)/urdf/screw_feeder.xacro" />
+  <xacro:screw_feeder feedername="m3_feeder" parent="a_bot_base_smfl">
+    <origin xyz=".1 .4 .05" rpy="0 0 ${pi/2}" />
+  </xacro:screw_feeder>
+  <xacro:screw_feeder feedername="m4_feeder" parent="c_bot_base_smfl">
+    <origin xyz=".45 .05 .05" rpy="0 0 0" />
+  </xacro:screw_feeder>
+  <xacro:screw_feeder feedername="m5_feeder" parent="c_bot_base_smfl">
+    <origin xyz=".45 .2 .05" rpy="0 0 0" />
+  </xacro:screw_feeder>
   <!-- robot arms -->
   <xacro:ur5_robot prefix="a_bot_" joint_limited="true"
@@ -107,5 +121,5 @@
     <origin xyz="0 0 0" rpy="0 0 0"/>
   </xacro:sensor_d435>
-  <!-- I meant to remove the "world" link definition, but apparently it is necessary for Gazebo -->
+  <!-- I would like to remove the "world" link definition, but apparently it is necessary for Gazebo -->
   <link name="world" />
   <joint name="world_o2as_joint" type="fixed">

Commit message: Attach AR marker on b_bot

File: o2as_scene_description/urdf/o2as_base_scene.urdf.xacro (robot description, xacro)
@@ -107,4 +107,9 @@
     <origin xyz="0 0 0" rpy="0 0 0"/>
   </xacro:sensor_d435>
+  <!-- spawn and attach AR marker -->
+  <xacro:include filename="$(find o2as_gazebo)/urdf/o2as_ar_marker.urdf.xacro"/>
+  <xacro:o2as_ar_marker prefix="b_bot_" parent="b_bot_wrist_3_link">
+    <origin xyz="0.0 0.0 0.05" rpy="0 0 0"/>
+  </xacro:o2as_ar_marker>
   <!-- I meant to remove the "world" link definition, but apparently it is necessary for Gazebo -->
   <link name="world" />

Commit message: Hacky fix for UR ee_link bug
The ee_link transform should be fixed to the wrist_3_link, but it seems to be published in the robot base frame when connected to the real robot, which results in a different orientation than during simulation. This adds another frame that is untouched by the bug, but it doesn't solve the underlying problem. To be investigated.

File: o2as_scene_description/urdf/o2as_base_scene.urdf.xacro (robot description, xacro)
@@ -102,11 +102,11 @@
   <!-- spawn and attach grippers -->
   <xacro:include filename="$(find o2as_scene_description)/urdf/robotiq_85_gripper.urdf.xacro" />
-  <xacro:robotiq_85_gripper_o2as prefix="a_bot_" parent = "a_bot_ee_link">
+  <xacro:robotiq_85_gripper_o2as prefix="a_bot_" parent = "a_bot_ee_duplicate_link">
     <origin xyz="0.0 0 0.0" rpy="0 0 0"/>
   </xacro:robotiq_85_gripper_o2as>
-  <xacro:robotiq_85_gripper_o2as prefix="b_bot_" parent = "b_bot_ee_link">
+  <xacro:robotiq_85_gripper_o2as prefix="b_bot_" parent = "b_bot_ee_duplicate_link">
     <origin xyz="0.0 0 0.0" rpy="0 0 0"/>
   </xacro:robotiq_85_gripper_o2as>
-  <xacro:robotiq_85_gripper_o2as prefix="c_bot_" parent = "c_bot_ee_link">
+  <xacro:robotiq_85_gripper_o2as prefix="c_bot_" parent = "c_bot_ee_duplicate_link">
     <origin xyz="0.0 0 0.0" rpy="0 0 0"/>
   </xacro:robotiq_85_gripper_o2as>

File: o2as_scene_description/urdf/ur3.urdf.xacro (robot description, xacro)
@@ -275,4 +275,17 @@
       </collision>
     </link>
+    <joint name="${prefix}ee_duplicate_fixed_joint" type="fixed">
+      <parent link="${prefix}wrist_3_link" />
+      <child link = "${prefix}ee_duplicate_link" />
+      <origin xyz="0.0 ${ur5_wrist_3_length} 0.0" rpy="0.0 0.0 ${pi/2.0}" />
+    </joint>
+    <link name="${prefix}ee_duplicate_link">
+      <collision>
+        <geometry>
+          <box size="0.01 0.01 0.01"/>
+        </geometry>
+        <origin rpy="0 0 0" xyz="-0.01 0 0"/>
+      </collision>
+    </link>
     <xacro:ur_arm_transmission prefix="${prefix}" />
     <xacro:ur_arm_gazebo prefix="${prefix}" />

File: o2as_scene_description/urdf/ur5.urdf.xacro (robot description, xacro)
@@ -291,4 +291,17 @@
       </collision>
     </link>
+    <joint name="${prefix}ee_duplicate_fixed_joint" type="fixed">
+      <parent link="${prefix}wrist_3_link" />
+      <child link = "${prefix}ee_duplicate_link" />
+      <origin xyz="0.0 ${ur5_wrist_3_length} 0.0" rpy="0.0 0.0 ${pi/2.0}" />
+    </joint>
+    <link name="${prefix}ee_duplicate_link">
+      <collision>
+        <geometry>
+          <box size="0.01 0.01 0.01"/>
+        </geometry>
+        <origin rpy="0 0 0" xyz="-0.01 0 0"/>
+      </collision>
+    </link>
     <xacro:ur_arm_transmission prefix="${prefix}" />
     <xacro:ur_arm_gazebo prefix="${prefix}" />

Commit message: Fix ee_link bug
https://github.com/Zagitta/ur_modern_driver/issues/26

File: o2as_scene_description/urdf/o2as_base_scene.urdf.xacro (robot description, xacro)
@@ -102,11 +102,11 @@
   <!-- spawn and attach grippers -->
   <xacro:include filename="$(find o2as_scene_description)/urdf/robotiq_85_gripper.urdf.xacro" />
-  <xacro:robotiq_85_gripper_o2as prefix="a_bot_" parent = "a_bot_ee_duplicate_link">
+  <xacro:robotiq_85_gripper_o2as prefix="a_bot_" parent = "a_bot_ee_link">
     <origin xyz="0.0 0 0.0" rpy="0 0 0"/>
   </xacro:robotiq_85_gripper_o2as>
-  <xacro:robotiq_85_gripper_o2as prefix="b_bot_" parent = "b_bot_ee_duplicate_link">
+  <xacro:robotiq_85_gripper_o2as prefix="b_bot_" parent = "b_bot_ee_link">
     <origin xyz="0.0 0 0.0" rpy="0 0 0"/>
   </xacro:robotiq_85_gripper_o2as>
-  <xacro:robotiq_85_gripper_o2as prefix="c_bot_" parent = "c_bot_ee_duplicate_link">
+  <xacro:robotiq_85_gripper_o2as prefix="c_bot_" parent = "c_bot_ee_link">
     <origin xyz="0.0 0 0.0" rpy="0 0 0"/>
   </xacro:robotiq_85_gripper_o2as>

File: o2as_scene_description/urdf/ur3.urdf.xacro (robot description, xacro)
@@ -275,17 +275,4 @@
       </collision>
     </link>
-    <joint name="${prefix}ee_duplicate_fixed_joint" type="fixed">
-      <parent link="${prefix}wrist_3_link" />
-      <child link = "${prefix}ee_duplicate_link" />
-      <origin xyz="0.0 ${ur5_wrist_3_length} 0.0" rpy="0.0 0.0 ${pi/2.0}" />
-    </joint>
-    <link name="${prefix}ee_duplicate_link">
-      <collision>
-        <geometry>
-          <box size="0.01 0.01 0.01"/>
-        </geometry>
-        <origin rpy="0 0 0" xyz="-0.01 0 0"/>
-      </collision>
-    </link>
     <xacro:ur_arm_transmission prefix="${prefix}" />
     <xacro:ur_arm_gazebo prefix="${prefix}" />

File: o2as_scene_description/urdf/ur5.urdf.xacro (robot description, xacro)
@@ -291,17 +291,4 @@
       </collision>
     </link>
-    <joint name="${prefix}ee_duplicate_fixed_joint" type="fixed">
-      <parent link="${prefix}wrist_3_link" />
-      <child link = "${prefix}ee_duplicate_link" />
-      <origin xyz="0.0 ${ur5_wrist_3_length} 0.0" rpy="0.0 0.0 ${pi/2.0}" />
-    </joint>
-    <link name="${prefix}ee_duplicate_link">
-      <collision>
-        <geometry>
-          <box size="0.01 0.01 0.01"/>
-        </geometry>
-        <origin rpy="0 0 0" xyz="-0.01 0 0"/>
-      </collision>
-    </link>
     <xacro:ur_arm_transmission prefix="${prefix}" />
     <xacro:ur_arm_gazebo prefix="${prefix}" />

Commit message: WIP: Add gripper URDF
Collisions are not working correctly

File: o2as_scene_description/urdf/o2as_base_scene.urdf.xacro (robot description, xacro)
@@ -101,8 +101,9 @@
   </joint>
   <!-- spawn and attach grippers -->
+  <xacro:include filename="$(find o2as_scene_description)/urdf/combined_gripper.xacro" />
+  <xacro:combined_gripper prefix="a_bot_"  grippername = "gripper" parent = "a_bot_tool0">
+    <origin xyz="0.0 0 0.04" rpy="0 ${pi/2} 0"/>
+  </xacro:combined_gripper>
   <xacro:include filename="$(find o2as_scene_description)/urdf/robotiq_85_gripper.urdf.xacro" />
-  <xacro:robotiq_85_gripper_o2as prefix="a_bot_" parent = "a_bot_ee_link">
-    <origin xyz="0.0 0 0.0" rpy="0 0 0"/>
-  </xacro:robotiq_85_gripper_o2as>
   <xacro:robotiq_85_gripper_o2as prefix="b_bot_" parent = "b_bot_ee_link">
     <origin xyz="0.0 0 0.0" rpy="0 0 0"/>

Commit message: Add the taskboard scene

File: o2as_scene_description/urdf/o2as_base_scene.urdf.xacro (robot description, xacro)
@@ -21,5 +21,5 @@
   <!-- Scene items (trays, bins...) -->
   <xacro:include filename="$(find o2as_scene_description)/urdf/walls.xacro" />
-  <xacro:include filename="$(find o2as_scene_description)/urdf/kitting_scene.xacro" />
+  <xacro:include filename="$(find o2as_scene_description)/urdf/taskboard_scene.xacro" />
   <!-- Robot bases -->
   <!-- Putting these at height 0.0 makes them intersect with the ground, so they are elevated. -->

File: o2as_scene_description/urdf/precision_gripper.xacro (robot description, xacro)
@@ -14,14 +14,5 @@
       </geometry>
         <material name="darkgrey">
-          <color rgba="0.5 0.1 0.1 1"/>
-        </material>
-    </visual>
-    <visual>
-    <origin rpy="0 0 0" xyz="-0.11 0 0"/>
-      <geometry>
-        <box size="0.22 0.15 0.1"/>
-      </geometry>
-      <material name="darkgrey2">
-          <color rgba="0.1 0.1 0.1 0.3"/>
+          <color rgba="0.1 0.1 0.1 1"/>
         </material>
     </visual>

Commit message: Add camera_info topic to o2as_phoxi_camera.

File: o2as_scene_description/urdf/o2as_base_scene.urdf.xacro (robot description, xacro)
@@ -91,15 +91,15 @@
     <origin xyz="0.0 0 0.0" rpy="0 0 0"/>
   </xacro:robotiq_85_gripper_o2as>
-  <!-- <xacro:robotiq_85_gripper_o2as prefix="b_bot_" parent = "b_bot_ee_link"> -->
-  <!--   <origin xyz="0.0 0 0.0" rpy="0 0 0"/> -->
-  <!-- </xacro:robotiq_85_gripper_o2as> -->
+  <xacro:robotiq_85_gripper_o2as prefix="b_bot_" parent = "b_bot_ee_link">
+    <origin xyz="0.0 0 0.0" rpy="0 0 0"/>
+  </xacro:robotiq_85_gripper_o2as>
   <xacro:robotiq_85_gripper_o2as prefix="c_bot_" parent = "c_bot_ee_link">
     <origin xyz="0.0 0 0.0" rpy="0 0 0"/>
   </xacro:robotiq_85_gripper_o2as>
   <!-- spawn and attach diual suction grippers -->
-  <xacro:include filename="$(find o2as_scene_description)/urdf/dual_suction_gripper.urdf.xacro" />
-  <xacro:dual_suction_gripper_o2as prefix="b_bot_" parent = "b_bot_ee_link">
-    <origin xyz="0 0 0" rpy="0 0 0"/>
-  </xacro:dual_suction_gripper_o2as>
+  <!-- <xacro:include filename="$(find o2as_scene_description)/urdf/dual_suction_gripper.urdf.xacro" /> -->
+  <!-- <xacro:dual_suction_gripper_o2as prefix="b_bot_" parent = "b_bot_ee_link"> -->
+  <!--   <origin xyz="0 0 0" rpy="0 0 0"/> -->
+  <!-- </xacro:dual_suction_gripper_o2as> -->
   <!-- Add cameras -->
   <link name="b_bot_cam_holder_link" />
@@ -112,4 +112,9 @@
     <origin xyz="0 0 0" rpy="0 0 0"/>
   </xacro:sensor_d435>
+  <!-- Add PhoXi 3D scanners -->
+  <xacro:include filename="$(find o2as_scene_description)/urdf/phoxi_m_camera.urdf.xacro" />
+  <xacro:phoxi_m_camera_o2as prefix="a_" parent="o2as_ground">
+    <origin xyz="0.56 0 ${bots_z + .1 + .8}" rpy="${170*pi/180} 0 ${-pi/2}"/>
+  </xacro:phoxi_m_camera_o2as>
   <!-- I meant to remove the "world" link definition, but apparently it is necessary for Gazebo -->
   <link name="world" />
