Commit message: Add FT300 sensor

File: o2as_scene_description/urdf/o2as_base_scene.urdf.xacro (robot description, xacro)
@@ -105,11 +105,7 @@
     <origin xyz="0.0 0 0.04" rpy="0 ${pi/2} 0"/>
   </xacro:precision_gripper>
-  <xacro:include filename="$(find o2as_scene_description)/urdf/robotiq_85_gripper.urdf.xacro" />
-  <xacro:robotiq_85_gripper_o2as prefix="b_bot_" parent = "b_bot_ee_link">
-    <origin xyz="0.0 0 0.0" rpy="0 0 0"/>
-  </xacro:robotiq_85_gripper_o2as>
-  <xacro:robotiq_85_gripper_o2as prefix="c_bot_" parent = "c_bot_ee_link">
-    <origin xyz="0.0 0 0.0" rpy="0 0 0"/>
-  </xacro:robotiq_85_gripper_o2as>
+  <xacro:include filename="$(find o2as_scene_description)/urdf/robotiq_85_gripper_with_ft300.urdf.xacro" />
+  <xacro:robotiq_85_gripper_o2as prefix="b_bot_" parent = "b_bot_ee_link" />
+  <xacro:robotiq_85_gripper_o2as prefix="c_bot_" parent = "c_bot_ee_link"/>
   <!-- Add cameras -->
   <link name="b_bot_cam_holder_link" />

File: o2as_scene_description/urdf/robotiq_85_gripper_with_ft300.urdf.xacro (robot description, xacro)
@@ -3,8 +3,26 @@
 <!-- The position of the TF frame has not been measured at all and needs to be calibrated. -->
 <robot name="robotiq_85_gripper_o2as" xmlns:xacro="http://www.ros.org/wiki/xacro">
-  <xacro:macro name="robotiq_85_gripper_o2as" params="prefix parent *origin">
+  <xacro:property name="ft300_length" value="0.034"/>
+  <xacro:macro name="robotiq_85_gripper_o2as" params="prefix parent">
+    <!-- Add the force sensor in front of the gripper. -->
+    <joint name="${prefix}ft300_joint" type="fixed">
+      <parent link="${parent}"/>
+      <child link="${prefix}ft300_link"/>
+      <origin rpy="0.0 ${pi/2} 0.0" xyz="${ft300_length/2} 0.0 0.0"/>
+    </joint>
+    <link name="${prefix}ft300_link">
+      <visual>
+        <origin xyz="0 0 0" rpy="0 0 0"/>
+        <geometry>
+          <cylinder length="${ft300_length}" radius="0.0375"/>
+        </geometry>
+        <material name="Black">
+          <color rgba="0.2 0.2 0.2 1.0"/>
+        </material>
+      </visual>
+    </link>
     <xacro:include filename="$(find robotiq_description)/urdf/robotiq_85_gripper.urdf.xacro" />
     <xacro:robotiq_85_gripper prefix="${prefix}" parent="${parent}">
-        <xacro:insert_block name="origin"/>
+        <origin rpy="0.0 0.0 0.0" xyz="${ft300_length} 0.0 0.0"/>
     </xacro:robotiq_85_gripper>
     <!-- Add additional links for us to plan with. Oriented like the UR frame. -->

Commit message: Run taskboard calibration

File: o2as_scene_description/urdf/o2as_base_scene.urdf.xacro (robot description, xacro)
@@ -59,7 +59,7 @@
     <origin xyz=".45 .05 .05" rpy="0 0 0" />
   </xacro:screw_feeder>
-  <xacro:screw_feeder feedername="m5_feeder" parent="c_bot_base_smfl">
+  <!-- <xacro:screw_feeder feedername="m5_feeder" parent="c_bot_base_smfl">
     <origin xyz=".45 .2 .05" rpy="0 0 0" />
-  </xacro:screw_feeder>
+  </xacro:screw_feeder> -->
   <!-- robot arms -->
   <xacro:ur5_robot prefix="a_bot_" joint_limited="true"

File: o2as_scene_description/urdf/precision_gripper.xacro (robot description, xacro)
@@ -17,8 +17,35 @@
         </material>
     </visual>
+    <!-- <visual>
+      <origin rpy="0 ${pi/2} 0" xyz="-0.16 0 0"/>
+      <geometry>
+        <box size=".1 .08 .07"/>
+      </geometry>
+      <material name="cyan2">
+        <color rgba="0.3 0.5 0.5 0.3"/>
+      </material>
+    </visual>
+    <visual>
+      <origin rpy="0 ${pi/2} 0" xyz="-0.05 0 0"/>
+      <geometry>
+        <box size="0.18 0.09 0.13"/>
+      </geometry>
+      <material name="green2">
+        <color rgba="0.1 0.8 0.1 0.3"/>
+      </material>
+    </visual> -->
+    <!-- TODO: Do this properly and check the offset above. -->
+    <!-- Back part -->
     <collision>
-      <origin rpy="0 ${pi/2} 0" xyz="-0.11 0 0"/>
+      <origin rpy="0 ${pi/2} 0" xyz="-0.05 0 0"/>
       <geometry>
-        <box size="0.22 0.15 0.1"/>
+        <box size="0.18 0.09 0.13"/>
+      </geometry>
+    </collision>
+    <!-- Front part -->
+    <collision>
+      <origin rpy="0 ${pi/2} 0" xyz="-0.16 0 0"/>
+      <geometry>
+        <box size=".1 .08 .07"/>
       </geometry>
     </collision>

Commit message: Attach a robotiq gripper but a suction gripper to b_bot.

File: o2as_scene_description/urdf/o2as_base_scene.urdf.xacro (robot description, xacro)
@@ -91,15 +91,15 @@
     <origin xyz="0.0 0 0.0" rpy="0 0 0"/>
   </xacro:robotiq_85_gripper_o2as>
-  <!-- <xacro:robotiq_85_gripper_o2as prefix="b_bot_" parent = "b_bot_ee_link"> -->
-  <!--   <origin xyz="0.0 0 0.0" rpy="0 0 0"/> -->
-  <!-- </xacro:robotiq_85_gripper_o2as> -->
+  <xacro:robotiq_85_gripper_o2as prefix="b_bot_" parent = "b_bot_ee_link">
+    <origin xyz="0.0 0 0.0" rpy="0 0 0"/>
+  </xacro:robotiq_85_gripper_o2as>
   <xacro:robotiq_85_gripper_o2as prefix="c_bot_" parent = "c_bot_ee_link">
     <origin xyz="0.0 0 0.0" rpy="0 0 0"/>
   </xacro:robotiq_85_gripper_o2as>
-  <!-- spawn and attach diual suction grippers -->
-  <xacro:include filename="$(find o2as_scene_description)/urdf/dual_suction_gripper.urdf.xacro" />
-  <xacro:dual_suction_gripper_o2as prefix="b_bot_" parent = "b_bot_ee_link">
-    <origin xyz="0 0 0" rpy="0 0 0"/>
-  </xacro:dual_suction_gripper_o2as>
+  <!-- spawn and attach dual suction grippers -->
+  <!-- <xacro:include filename="$(find o2as_scene_description)/urdf/dual_suction_gripper.urdf.xacro" /> -->
+  <!-- <xacro:dual_suction_gripper_o2as prefix="b_bot_" parent = "b_bot_ee_link"> -->
+  <!--   <origin xyz="0 0 0" rpy="0 0 0"/> -->
+  <!-- </xacro:dual_suction_gripper_o2as> -->
   <!-- Add cameras -->
   <link name="b_bot_cam_holder_link" />

Commit message: Improve calibration function, add calibrated values

File: o2as_scene_description/urdf/o2as_base_scene.urdf.xacro (robot description, xacro)
@@ -3,9 +3,10 @@
        name="o2as_base_scene" >
   <!-- This is the main file defining our robot arrangement and physical environment. -->
-  <!-- These values are still not fixed -->
-  <xacro:property name="a_bot_x" value="0.0"/>
-  <xacro:property name="a_bot_y" value="-0.65"/>
-  <xacro:property name="b_bot_x" value="0.0"/>
-  <xacro:property name="b_bot_y" value="0.65"/>
+  <!-- Calibration from 20 August 2018 -->
+  <!-- Calibration help: If the robot is not moving far enough to the calibration point, increase these distances -->
+  <xacro:property name="a_bot_x" value="-0.005"/>
+  <xacro:property name="a_bot_y" value="-0.543"/>
+  <xacro:property name="b_bot_x" value="0.001"/>
+  <xacro:property name="b_bot_y" value="0.529"/>
   <xacro:property name="c_bot_x" value="-0.5"/>
   <xacro:property name="c_bot_y" value="0.0"/>
@@ -20,6 +21,7 @@
   <xacro:include filename="$(find o2as_scene_description)/urdf/ur3.urdf.xacro" />
   <!-- Scene items (trays, bins...) -->
-  <xacro:include filename="$(find o2as_scene_description)/urdf/walls.xacro" />
-  <xacro:include filename="$(find o2as_scene_description)/urdf/taskboard_scene.xacro" />
+  <!-- <xacro:include filename="$(find o2as_scene_description)/urdf/taskboard_scene.xacro" /> -->
+  <!-- <xacro:include filename="$(find o2as_scene_description)/urdf/kitting_scene.xacro" /> -->
+  <!-- <xacro:include filename="$(find o2as_scene_description)/urdf/assembly_scene.xacro" /> -->
   <!-- Robot bases -->
   <!-- Putting these at height 0.0 makes them intersect with the ground, so they are elevated. -->

File: o2as_scene_description/urdf/robotiq_85_gripper_with_ft300.urdf.xacro (robot description, xacro)
@@ -3,5 +3,7 @@
 <!-- The position of the TF frame has not been measured at all and needs to be calibrated. -->
 <robot name="robotiq_85_gripper_o2as" xmlns:xacro="http://www.ros.org/wiki/xacro">
-  <xacro:property name="ft300_length" value="0.034"/>
+  <!-- This seems too long when measuring the sensor,
+       but works out when calibrating the tip_link to the world. -->
+  <xacro:property name="ft300_length" value="0.056"/>
   <xacro:macro name="robotiq_85_gripper_o2as" params="prefix parent">
     <!-- Add the force sensor in front of the gripper. -->

Commit message: Attach suction gripper to a_bot.

File: o2as_scene_description/urdf/o2as_base_scene.urdf.xacro (robot description, xacro)
@@ -88,16 +88,16 @@
   </joint>
   <!-- spawn and attach grippers -->
-  <xacro:include filename="$(find o2as_scene_description)/urdf/precision_gripper.xacro" />
+  <!-- <xacro:include filename="$(find o2as_scene_description)/urdf/precision_gripper.xacro" />
   <xacro:precision_gripper prefix="a_bot_"  grippername = "gripper" parent = "a_bot_tool0">
     <origin xyz="0.0 0 0.04" rpy="0 ${pi/2} 0"/>
-  </xacro:precision_gripper>
+  </xacro:precision_gripper> -->
   <xacro:include filename="$(find o2as_scene_description)/urdf/robotiq_85_gripper_with_ft300.urdf.xacro" />
   <xacro:robotiq_85_gripper_o2as prefix="b_bot_" parent = "b_bot_ee_link" />
   <xacro:robotiq_85_gripper_o2as prefix="c_bot_" parent = "c_bot_ee_link"/>
   <!-- spawn and attach dual suction grippers -->
-  <!-- <xacro:include filename="$(find o2as_scene_description)/urdf/dual_suction_gripper.urdf.xacro" /> -->
-  <!-- <xacro:dual_suction_gripper_o2as prefix="b_bot_" parent = "b_bot_ee_link"> -->
-  <!--   <origin xyz="0 0 0" rpy="0 0 0"/> -->
-  <!-- </xacro:dual_suction_gripper_o2as> -->
+  <xacro:include filename="$(find o2as_scene_description)/urdf/dual_suction_gripper.urdf.xacro" />
+  <xacro:dual_suction_gripper_o2as prefix="a_bot_" parent = "a_bot_ee_link">
+    <origin xyz="0 0 0" rpy="0 0 0"/>
+  </xacro:dual_suction_gripper_o2as>
   <!-- Add cameras -->
   <link name="b_bot_cam_holder_link" />

Commit message: Add picking and moving robot to named pose.

File: o2as_scene_description/urdf/o2as_base_scene.urdf.xacro (robot description, xacro)
@@ -41,5 +41,5 @@
   <xacro:property name="plate_l" value="0.62"/>
   <xacro:o2as_box boxname="workbox" box_w="${plate_w}" box_l="${plate_l}" box_h=".01" parent="o2as_ground">
-    <origin xyz="${-plate_w/2} ${-plate_l/2} ${bots_z+.09}" rpy="0 0 0" />
+    <origin xyz="${-plate_w/2} ${-plate_l/2} ${bots_z}" rpy="0 0 0" />
   </xacro:o2as_box>
   <link name="workspace_center" />
@@ -47,5 +47,5 @@
     <parent link="o2as_ground" />
     <child link="workspace_center" />
-    <origin xyz="0.0 0.0 ${bots_z+.1}" rpy="0.0 0.0 0.0" />
+    <origin xyz="0.0 0.0 ${bots_z+.01}" rpy="0.0 0.0 0.0" />
   </joint>
   <!-- robot arms -->
@@ -94,5 +94,5 @@
   <xacro:include filename="$(find o2as_scene_description)/urdf/robotiq_85_gripper_with_ft300.urdf.xacro" />
   <xacro:robotiq_85_gripper_o2as prefix="b_bot_" parent = "b_bot_ee_link" />
-  <xacro:robotiq_85_gripper_o2as prefix="c_bot_" parent = "c_bot_ee_link"/>
+  <!-- <xacro:robotiq_85_gripper_o2as prefix="c_bot_" parent = "c_bot_ee_link"/> -->
   <!-- spawn and attach dual suction grippers -->
   <xacro:include filename="$(find o2as_scene_description)/urdf/dual_suction_gripper.urdf.xacro" />

Commit message: Fixed conflicts.

File: o2as_scene_description/urdf/o2as_base_scene.urdf.xacro (robot description, xacro)
@@ -2,10 +2,4 @@
 <robot xmlns:xacro="http://ros.org/wiki/xacro"
        name="o2as_base_scene" >
-<<<<<<< HEAD
-  <xacro:property name="a_bot_x" value="0.0"/>
-  <xacro:property name="a_bot_y" value="-0.6"/>
-  <xacro:property name="b_bot_x" value="0.0"/>
-  <xacro:property name="b_bot_y" value="0.6"/>
-=======
   <!-- Calibration from 20 August 2018 -->
   <!-- Calibration help: If the robot is not moving far enough to the calibration point, increase these distances -->
@@ -14,5 +8,4 @@
   <xacro:property name="b_bot_x" value="0.001"/>
   <xacro:property name="b_bot_y" value="0.529"/>
->>>>>>> 156be353b0da943b90a267d6d15847b35054a9a3
   <xacro:property name="c_bot_x" value="-0.5"/>
   <xacro:property name="c_bot_y" value="0.0"/>

Commit message: Update b_bot gripper for kitting.
change to suction gripper.

File: o2as_scene_description/urdf/o2as_base_scene.urdf.xacro (robot description, xacro)
@@ -107,11 +107,11 @@
   </xacro:precision_gripper>
   <xacro:include filename="$(find o2as_scene_description)/urdf/robotiq_85_gripper_with_ft300.urdf.xacro" />
-  <xacro:robotiq_85_gripper_o2as prefix="b_bot_" parent = "b_bot_ee_link" />
+  <!-- <xacro:robotiq_85_gripper_o2as prefix="b_bot_" parent = "b_bot_ee_link" /> -->
   <xacro:robotiq_85_gripper_o2as prefix="c_bot_" parent = "c_bot_ee_link"/>
   <!-- spawn and attach dual suction grippers -->
-  <!-- <xacro:include filename="$(find o2as_scene_description)/urdf/dual_suction_gripper.urdf.xacro" /> -->
-  <!-- <xacro:dual_suction_gripper_o2as prefix="b_bot_" parent = "b_bot_ee_link"> -->
-  <!--   <origin xyz="0 0 0" rpy="0 0 0"/> -->
-  <!-- </xacro:dual_suction_gripper_o2as> -->
+  <xacro:include filename="$(find o2as_scene_description)/urdf/dual_suction_gripper.urdf.xacro" />
+  <xacro:dual_suction_gripper_o2as prefix="b_bot_" parent = "b_bot_ee_link">
+    <origin xyz="0 0 0" rpy="0 0 0"/>
+  </xacro:dual_suction_gripper_o2as>
   <!-- Add cameras -->
   <link name="b_bot_cam_holder_link" />
@@ -124,13 +124,13 @@
     <origin xyz="0 0 0" rpy="0 0 0"/>
   </xacro:sensor_d435>
-  <!-- <link name="d_bot_cam_holder_link" /> -->
-  <!-- <joint name="d_bot_cam_holder_joint" type="fixed"> -->
-  <!--   <parent link="o2as_ground" /> -->
-  <!--   <child  link="d_bot_cam_holder_link" /> -->
-  <!--   <origin xyz="0.0 0.0 2.0" rpy="0.0 ${pi/2} 0.0" /> -->
-  <!-- </joint> -->
-  <!-- <xacro:sensor_d435 prefix="d_bot_" parent="d_bot_cam_holder_link"> -->
-  <!--   <origin xyz="0 0 0" rpy="0 0 0"/> -->
-  <!-- </xacro:sensor_d435> -->
+  <!-- <link name="d_bot_cam_holder_link" />
+  <joint name="d_bot_cam_holder_joint" type="fixed">
+    <parent link="o2as_ground" />
+    <child  link="d_bot_cam_holder_link" />
+    <origin xyz="0.0 0.0 2.0" rpy="0.0 ${pi/2} 0.0" />
+  </joint>
+  <xacro:sensor_d435 prefix="d_bot_" parent="d_bot_cam_holder_link">
+    <origin xyz="0 0 0" rpy="0 0 0"/>
+  </xacro:sensor_d435> -->
   <!-- spawn and attach AR marker -->
   <xacro:include filename="$(find o2as_gazebo)/urdf/o2as_ar_marker.urdf.xacro"/>

Commit message: Change textures of AR markers for a_bot and c_bot

File: o2as_scene_description/urdf/o2as_base_scene.urdf.xacro (robot description, xacro)
@@ -133,9 +133,17 @@
   <!--   <origin xyz="0 0 0" rpy="0 0 0"/> -->
   <!-- </xacro:sensor_d435> -->
-  <!-- spawn and attach AR marker -->
+  <!-- spawn and attach AR markers -->
   <xacro:include filename="$(find o2as_gazebo)/urdf/o2as_ar_marker.urdf.xacro"/>
+  <xacro:o2as_ar_marker prefix="a_bot_" parent="a_bot_wrist_3_link"
+   marker_id="17">
+    <origin xyz="0.0 -0.06 0.0" rpy="${pi/2} 0 0"/>
+  </xacro:o2as_ar_marker>
   <xacro:o2as_ar_marker prefix="b_bot_" parent="b_bot_wrist_3_link"
    marker_id="26">
-    <origin xyz="0.0 -0.07 0.0" rpy="${pi/2} 0 0"/>
+    <origin xyz="0.0 -0.06 0.0" rpy="${pi/2} 0 0"/>
+  </xacro:o2as_ar_marker>
+    <xacro:o2as_ar_marker prefix="c_bot_" parent="c_bot_wrist_3_link"
+   marker_id="256">
+    <origin xyz="0.0 -0.05 0.0" rpy="${pi/2} 0 0"/>
   </xacro:o2as_ar_marker>
   <!-- Add PhoXi 3D scanners -->

Commit message: Fix position of AR marker in simulator

File: o2as_scene_description/urdf/o2as_base_scene.urdf.xacro (robot description, xacro)
@@ -137,13 +137,13 @@
   <xacro:o2as_ar_marker prefix="a_bot_" parent="a_bot_wrist_3_link"
    marker_id="17">
-    <origin xyz="0.0 -0.06 0.0" rpy="${pi/2} 0 0"/>
+    <origin xyz="0.0 -0.07 0.0" rpy="${pi/2} 0 0"/>
   </xacro:o2as_ar_marker>
   <xacro:o2as_ar_marker prefix="b_bot_" parent="b_bot_wrist_3_link"
    marker_id="26">
-    <origin xyz="0.0 -0.06 0.0" rpy="${pi/2} 0 0"/>
+    <origin xyz="0.0 -0.07 0.0" rpy="${pi/2} 0 0"/>
   </xacro:o2as_ar_marker>
     <xacro:o2as_ar_marker prefix="c_bot_" parent="c_bot_wrist_3_link"
    marker_id="256">
-    <origin xyz="0.0 -0.05 0.0" rpy="${pi/2} 0 0"/>
+    <origin xyz="0.0 -0.06 0.0" rpy="${pi/2} 0 0"/>
   </xacro:o2as_ar_marker>
   <!-- Add PhoXi 3D scanners -->

Commit message: Remove modification of manufacturer camera macro

File: o2as_scene_description/urdf/o2as_base_scene.urdf.xacro (robot description, xacro)
@@ -15,5 +15,5 @@
   <xacro:include filename="$(find ur_description)/urdf/common.gazebo.xacro" />
   <xacro:include filename="$(find o2as_gazebo)/urdf/o2as_base_scene.gazebo" />
-  <xacro:include filename="$(find realsense2_camera)/urdf/_d435.urdf.xacro" />
+  <xacro:include filename="$(find o2as_scene_description)/urdf/_d435.urdf.xacro" />
   <!-- robots -->
   <!-- <xacro:include filename="$(find o2as_scene_description)/urdf/ur10.urdf.xacro" /> -->
@@ -117,7 +117,7 @@
     <origin xyz="0.0 -0.06 0.16" rpy="0.0 0.0 ${pi/2}" />
   </joint>
-  <xacro:sensor_d435 prefix="b_bot_" parent="b_bot_cam_holder_link">
+  <xacro:o2as_sensor_d435 prefix="b_bot_" parent="b_bot_cam_holder_link">
     <origin xyz="0 0 0" rpy="0 0 0"/>
-  </xacro:sensor_d435>
+  </xacro:o2as_sensor_d435>
   <!-- I would like to remove the "world" link definition, but apparently it is necessary for Gazebo -->
   <link name="world" />

File: realsense/realsense2_camera/urdf/_d435.urdf.xacro (robot description, xacro)
@@ -64,10 +64,4 @@
     </joint>
     <link name="${prefix}camera_depth_frame"/>
-    <joint name="camera_depth_image_joint" type="fixed">
-      <origin xyz="0 0 0" rpy="${M_PI/2} ${M_PI} ${M_PI/2}"/>
-      <parent link="${prefix}camera_depth_frame"/>
-      <child link="${prefix}camera_depth_image_frame" />
-    </joint>
-    <link name="${prefix}camera_depth_image_frame"/>
     <joint name="camera_depth_optical_joint" type="fixed">
       <origin xyz="0 0 0" rpy="${-M_PI/2} 0 ${-M_PI/2}" />

Commit message: Update robot calibration & procedure

File: o2as_scene_description/urdf/o2as_base_scene.urdf.xacro (robot description, xacro)
@@ -5,8 +5,8 @@
   <!-- Calibration from 20 August 2018 -->
   <!-- Calibration help: If the robot is not moving far enough to the calibration point, increase these distances -->
-  <xacro:property name="a_bot_x" value="-0.005"/>
-  <xacro:property name="a_bot_y" value="-0.543"/>
-  <xacro:property name="b_bot_x" value="0.001"/>
-  <xacro:property name="b_bot_y" value="0.529"/>
+  <xacro:property name="a_bot_x" value="-0.011"/>
+  <xacro:property name="a_bot_y" value="-0.5"/>
+  <xacro:property name="b_bot_x" value="-0.004"/>
+  <xacro:property name="b_bot_y" value="0.5"/>
   <xacro:property name="c_bot_x" value="-0.5"/>
   <xacro:property name="c_bot_y" value="0.0"/>

Commit message: Added support for calibration of PhoXi scanners.

File: o2as_scene_description/urdf/o2as_base_scene.urdf.xacro (robot description, xacro)
@@ -126,5 +126,6 @@
   </xacro:sensor_d435>
   <xacro:sensor_d435 prefix="d_bot_" parent="o2as_ground">
-    <origin xyz="0 0 ${bots_z + 0.9}" rpy="0 ${pi/2} 0"/>
+    <!-- <origin xyz="0 0 ${bots_z + 0.9}" rpy="0 ${pi/2} ${pi}"/> -->
+    <origin xyz="0 0 2" rpy="0 ${pi/2} ${pi}"/>
   </xacro:sensor_d435>
   <!-- spawn and attach AR markers -->

File: o2as_scene_description/urdf/phoxi_m_camera.urdf.xacro (robot description, xacro)
@@ -12,9 +12,9 @@
       <xacro:PhoXi3DscannerM_meshes />
     </xacro:PhoXi3Dscanner>
-    <link name="${prefix}phoxi_m_tip"/>
-    <joint name="${prefix}phoxi_m_sensor_to_${prefix}phoxi_m_tip"
+    <link name="${prefix}phoxi_m_camera_link"/>
+    <joint name="${prefix}phoxi_m_sensor_to_${prefix}phoxi_m_camera_link"
     	   type="fixed">
       <parent link="${prefix}phoxi_m_sensor"/>
-      <child  link="${prefix}phoxi_m_tip"/>
+      <child  link="${prefix}phoxi_m_camera_link"/>
       <origin xyz="0 0 0" rpy="${pi/2} ${-pi/2} 0"/>
     </joint>

Commit message: Remove d_bot_camera and change the pose of the AR marker on c_bot

File: o2as_scene_description/urdf/o2as_base_scene.urdf.xacro (robot description, xacro)
@@ -125,7 +125,7 @@
     <origin xyz="0 0 0" rpy="0 0 0"/>
   </xacro:sensor_d435>
-  <xacro:sensor_d435 prefix="d_bot_" parent="o2as_ground">
+  <!-- <xacro:sensor_d435 prefix="d_bot_" parent="o2as_ground">
     <origin xyz="0 0 ${bots_z + 0.9}" rpy="0 ${pi/2} 0"/>
-  </xacro:sensor_d435>
+  </xacro:sensor_d435> -->
   <!-- spawn and attach AR markers -->
   <xacro:include filename="$(find o2as_gazebo)/urdf/o2as_ar_marker.urdf.xacro"/>
@@ -140,5 +140,5 @@
     <xacro:o2as_ar_marker prefix="c_bot_" parent="c_bot_wrist_3_link"
    marker_id="256">
-    <origin xyz="0.0 -0.06 0.0" rpy="${pi/2} 0 0"/>
+    <origin xyz="0.0 0.12 0.05" rpy="0 0 ${pi/2}"/>
   </xacro:o2as_ar_marker>
   <!-- Add PhoXi 3D scanners -->

Commit message: Add move_to_goal_pose in aist_kitting.
Includes update base_scene for kitting in aist.

File: o2as_scene_description/urdf/o2as_base_scene.urdf.xacro (robot description, xacro)
@@ -7,5 +7,7 @@
   <xacro:property name="a_bot_y" value="-0.543"/>
   <xacro:property name="b_bot_x" value="0.001"/>
-  <xacro:property name="b_bot_y" value="0.529"/>
+  <!-- <xacro:property name="b_bot_y" value="0.529"/> -->
+  <!-- forkitting -->
+  <xacro:property name="b_bot_y" value="0.6"/>
   <xacro:property name="c_bot_x" value="-0.5"/>
   <xacro:property name="c_bot_y" value="0.0"/>

Commit message: Switched from assemply to kitting scene.

File: o2as_scene_description/urdf/o2as_base_scene.urdf.xacro (robot description, xacro)
@@ -23,6 +23,6 @@
   <xacro:include filename="$(find o2as_scene_description)/urdf/kitting_tray_with_partitions.xacro" />
   <!-- <xacro:include filename="$(find o2as_scene_description)/urdf/taskboard_scene.xacro" /> -->
-  <!-- <xacro:include filename="$(find o2as_scene_description)/urdf/kitting_scene.xacro" /> -->
-  <xacro:include filename="$(find o2as_scene_description)/urdf/assembly_scene.xacro" />
+  <xacro:include filename="$(find o2as_scene_description)/urdf/kitting_scene.xacro" />
+  <!-- <xacro:include filename="$(find o2as_scene_description)/urdf/assembly_scene.xacro" /> -->
   <!-- Robot bases -->
   <!-- Putting these at height 0.0 makes them intersect with the ground, so they are elevated. -->
@@ -123,8 +123,8 @@
     <origin xyz="0.0 -0.06 0.16" rpy="0.0 0.0 ${pi/2}" />
   </joint>
-  <xacro:o2as_sensor_d435 prefix="b_bot_" parent="b_bot_cam_holder_link">
+  <xacro:sensor_d435 prefix="b_bot_" parent="b_bot_cam_holder_link">
     <origin xyz="0 0 0" rpy="0 0 0"/>
-  </xacro:o2as_sensor_d435>
-  <!-- <link name="d_bot_cam_holder_link" />
+  </xacro:sensor_d435>
+  <link name="d_bot_cam_holder_link" />
   <joint name="d_bot_cam_holder_joint" type="fixed">
     <parent link="o2as_ground" />
@@ -134,5 +134,5 @@
   <xacro:sensor_d435 prefix="d_bot_" parent="d_bot_cam_holder_link">
     <origin xyz="0 0 0" rpy="0 0 0"/>
-  </xacro:sensor_d435> -->
+  </xacro:sensor_d435>
   <!-- spawn and attach AR marker -->
   <xacro:include filename="$(find o2as_gazebo)/urdf/o2as_ar_marker.urdf.xacro"/>
