Commit message: Calibrate robots to new workplate

File: o2as_scene_description/urdf/o2as_base_scene.urdf.xacro (robot description, xacro)
@@ -4,8 +4,8 @@
   <!-- Calibration from 20 August 2018 -->
   <!-- Calibration help: If the robot is not moving far enough to the calibration point, increase these distances -->
-  <xacro:property name="a_bot_x" value="-0.005"/>
-  <xacro:property name="a_bot_y" value="-0.543"/>
-  <xacro:property name="b_bot_x" value="0.001"/>
-  <xacro:property name="b_bot_y" value="0.529"/>
+  <xacro:property name="a_bot_x" value="-0.01"/>
+  <xacro:property name="a_bot_y" value="-0.5"/>
+  <xacro:property name="b_bot_x" value="-0.005"/>
+  <xacro:property name="b_bot_y" value="0.5"/>
   <xacro:property name="c_bot_x" value="-0.5"/>
   <xacro:property name="c_bot_y" value="0.0"/>

File: o2as_scene_description/urdf/robotiq_85_gripper_with_ft300.urdf.xacro (robot description, xacro)
@@ -5,5 +5,5 @@
   <!-- This seems too long when measuring the sensor,
        but works out when calibrating the tip_link to the world. -->
-  <xacro:property name="ft300_length" value="0.056"/>
+  <xacro:property name="ft300_length" value="0.0555"/>
   <xacro:macro name="robotiq_85_gripper_o2as" params="prefix parent">
     <!-- Add the force sensor in front of the gripper. -->
@@ -32,5 +32,5 @@
       <parent link="${prefix}robotiq_85_base_link"/>
       <child link="${prefix}robotiq_85_tip_link"/>
-      <origin rpy="0.0 0.0 0.0" xyz=".16 0.0 0.0"/>
+      <origin rpy="0.0 0.0 0.0" xyz=".163 0.0 0.0"/>
     </joint>
     <link name="${prefix}robotiq_85_tip_link"/>

Commit message: o2as_calibrate.launch now supports real robots and cameras.

File: o2as_scene_description/urdf/o2as_base_scene.urdf.xacro (robot description, xacro)
@@ -138,13 +138,13 @@
   <xacro:o2as_ar_marker prefix="a_bot_" parent="a_bot_ee_link"
 			marker_id="17">
-    <origin xyz="0.25 0.0 0.055" rpy="0 0 ${pi}"/>
+    <origin xyz="0.25 0.0 -0.045" rpy="${pi} 0 ${pi}"/>
   </xacro:o2as_ar_marker>
   <xacro:o2as_ar_marker prefix="b_bot_" parent="b_bot_ee_link"
 			marker_id="26">
-    <origin xyz="0.064 0.0 0.019" rpy="0 0 ${pi}"/>
+    <origin xyz="0.064 0.0 -0.020" rpy="${pi} 0 ${pi}"/>
   </xacro:o2as_ar_marker>
     <xacro:o2as_ar_marker prefix="c_bot_" parent="c_bot_ee_link"
 			  marker_id="256">
-    <origin xyz="0.22 0.0 0.016" rpy="0 0 ${pi}"/>
+    <origin xyz="0.22 0.0 -0.016" rpy="${pi} 0 ${pi}"/>
   </xacro:o2as_ar_marker>
   <!-- Add PhoXi 3D scanners -->

Commit message: Calibration script is modified to be applied to real robots.

File: o2as_scene_description/urdf/o2as_base_scene.urdf.xacro (robot description, xacro)
@@ -136,15 +136,18 @@
   <!-- spawn and attach AR markers -->
   <xacro:include filename="$(find o2as_gazebo)/urdf/o2as_ar_marker.urdf.xacro"/>
-  <xacro:o2as_ar_marker prefix="a_bot_" parent="a_bot_ee_link"
+  <xacro:o2as_ar_marker prefix="a_bot_"
+			parent="a_bot_ee_link"
 			marker_id="17">
     <origin xyz="0.25 0.0 0.047" rpy="0 0 0"/>
   </xacro:o2as_ar_marker>
-  <xacro:o2as_ar_marker prefix="b_bot_" parent="b_bot_dual_suction_gripper_base_link"
+  <xacro:o2as_ar_marker prefix="b_bot_"
+			parent="b_bot_dual_suction_gripper_base_link"
 			marker_id="26">
     <origin xyz="0.063 0.0 0.0215" rpy="0 0 0"/>
   </xacro:o2as_ar_marker>
-    <xacro:o2as_ar_marker prefix="c_bot_" parent="c_bot_ee_link"
-			  marker_id="256">
-    <origin xyz="0.22 0.0 0.0185" rpy="0 0 0"/>
+  <xacro:o2as_ar_marker prefix="c_bot_"
+			parent="c_bot_robotiq_85_tip_link"
+			marker_id="256">
+    <origin xyz="0.0 0.0 0.0185" rpy="0 0 0"/>
   </xacro:o2as_ar_marker>
   <!-- Add PhoXi 3D scanners -->

Commit message: Modifiled base scene.
It allows b_bot reach bins and trays without collision
in the scene which workspace width (y-axis in world coordinates)
is 1000mm.

File: o2as_scene_description/urdf/o2as_base_scene.urdf.xacro (robot description, xacro)
@@ -4,8 +4,8 @@
   <!-- Calibration from 20 August 2018 -->
   <!-- Calibration help: If the robot is not moving far enough to the calibration point, increase these distances -->
-  <xacro:property name="a_bot_x" value="-0.005"/>
-  <xacro:property name="a_bot_y" value="-0.543"/>
-  <xacro:property name="b_bot_x" value="0.001"/>
-  <xacro:property name="b_bot_y" value="0.529"/>
+  <xacro:property name="a_bot_x" value="-0.00"/>
+  <xacro:property name="a_bot_y" value="-0.45"/>
+  <xacro:property name="b_bot_x" value="0.00"/>
+  <xacro:property name="b_bot_y" value="0.55"/>
   <xacro:property name="c_bot_x" value="-0.5"/>
   <xacro:property name="c_bot_y" value="0.0"/>

Commit message: Add cut to worktable in simulator

File: o2as_scene_description/urdf/o2as_base_scene.urdf.xacro (robot description, xacro)
@@ -41,6 +41,11 @@
   <xacro:property name="plate_w" value="0.9"/>
   <xacro:property name="plate_l" value="0.75"/>
-  <xacro:o2as_box boxname="workbox" box_w="${plate_w}" box_l="${plate_l}" box_h=".01" parent="o2as_ground">
-    <origin xyz="${-plate_w/2 +.08} ${-plate_l/2} ${bots_z}" rpy="0 0 0" />
+  <xacro:property name="plate_cut_w" value="0.03"/>
+  <xacro:property name="plate_cut_l" value="0.14"/>
+  <xacro:o2as_box boxname="workbox1" box_w="${plate_w}" box_l="${plate_l-plate_cut_l}" box_h=".01" parent="o2as_ground">
+    <origin xyz="${-plate_w/2 +.08} ${-(plate_l/2)} ${bots_z}" rpy="0 0 0" />
+  </xacro:o2as_box>
+  <xacro:o2as_box boxname="workbox2" box_w="${plate_w-plate_cut_w}" box_l="${plate_cut_l}" box_h=".01" parent="o2as_ground">
+    <origin xyz="${-plate_w/2 +.08+0.03} ${-plate_l/2+plate_l-plate_cut_l} ${bots_z}" rpy="0 0 0" />
   </xacro:o2as_box>
   <link name="workspace_center" />

Commit message: Calibration updates

File: o2as_scene_description/urdf/o2as_base_scene.urdf.xacro (robot description, xacro)
@@ -6,7 +6,9 @@
   <xacro:property name="a_bot_x" value="-0.01"/>
   <xacro:property name="a_bot_y" value="-0.5"/>
-  <xacro:property name="b_bot_x" value="-0.005"/>
-  <xacro:property name="b_bot_y" value="0.5"/>
-  <xacro:property name="c_bot_x" value="-0.5"/>
+  <xacro:property name="b_bot_x" value="-0.009"/>
+  <xacro:property name="b_bot_y" value="0.503"/>
+  <xacro:property name="b_bot_theta" value="-3.12832815"/>
+  <!-- The above is 0.76 degrees away from pi (Sep 17; not perfect) -->
+  <xacro:property name="c_bot_x" value="-0.499"/>
   <xacro:property name="c_bot_y" value="0.0"/>
   <xacro:property name="bots_z" value="0.75"/>
@@ -91,5 +93,5 @@
     <parent link="o2as_ground" />
     <child link = "b_bot_base_link" />
-    <origin xyz="${b_bot_x} ${b_bot_y} ${bots_z}" rpy="0.0 0.0 ${-pi}" />
+    <origin xyz="${b_bot_x} ${b_bot_y} ${bots_z}" rpy="0.0 0.0 ${b_bot_theta}" />
   </joint>
   <joint name="world_c_bot_joint" type="fixed">

File: o2as_scene_description/urdf/screw_tools.xacro (robot description, xacro)
@@ -40,5 +40,6 @@
     <parent link="c_bot_base_smfl" />
     <child link="screw_tool_holder" />
-    <origin xyz="${0.65-0.045} ${0.65+.004} 0.06" rpy="0.0 0.0 0.0" />
+    <origin xyz="${0.65-0.045 +.005} ${0.65+.004} 0.06" rpy="0.0 0.0 0.0" />
+    <!-- +.005 is a MAGIC NUMBER added on Sep 17 to put the tool roughly between c_bot and b_bot's physical position. -->
   </joint>
   <!-- ++++++++++++++++++++++++++++ -->

Commit message: Add separate TCPs for c_bot gripper

File: o2as_scene_description/urdf/o2as_base_scene.urdf.xacro (robot description, xacro)
@@ -111,7 +111,8 @@
   </xacro:precision_gripper>
   <!-- spawn and attach dual robotiq 85 grippers -->
-  <xacro:include filename="$(find o2as_scene_description)/urdf/robotiq_85_gripper_with_ft300.urdf.xacro" />
-  <xacro:robotiq_85_gripper_o2as prefix="b_bot_" parent = "b_bot_ee_link" />
-  <xacro:robotiq_85_gripper_o2as prefix="c_bot_" parent = "c_bot_ee_link"/>
+  <xacro:include filename="$(find o2as_scene_description)/urdf/robotiq_b_bot_gripper.urdf.xacro" />
+  <xacro:include filename="$(find o2as_scene_description)/urdf/robotiq_c_bot_gripper.urdf.xacro" />
+  <xacro:o2as_b_bot_gripper prefix="b_bot_" parent = "b_bot_ee_link" />
+  <xacro:o2as_c_bot_gripper prefix="c_bot_" parent = "c_bot_ee_link"/>
   <!-- Add cameras -->
   <xacro:include filename="$(find o2as_realsense2_camera)/urdf/_d435.urdf.xacro" />

File: o2as_scene_description/urdf/robotiq_85_gripper_with_ft300.urdf.xacro (robot description, xacro)
@@ -6,5 +6,5 @@
        but works out when calibrating the tip_link to the world. -->
   <xacro:property name="ft300_length" value="0.0525"/>
-  <xacro:macro name="robotiq_85_gripper_o2as" params="prefix parent">
+  <xacro:macro name="robotiq_85_gripper_with_ft300" params="prefix parent">
     <!-- Add the force sensor in front of the gripper. -->
     <joint name="${prefix}ft300_joint" type="fixed">
@@ -35,23 +35,4 @@
     </joint>
     <link name="${prefix}robotiq_85_tip_link"/>
-    <!-- Screw tool tips. X-axis points along the screw into the hole. -->
-    <joint name="${prefix}robotiq_85_m6_screw_tool_tip_joint" type="fixed">
-      <parent link="${prefix}robotiq_85_tip_link"/>
-      <child link="${prefix}screw_tool_m6_tip_link"/>
-      <origin rpy="0.0 ${pi/2} 0.0" xyz="-0.03 0.0 -0.12 "/>
-    </joint>
-    <link name="${prefix}screw_tool_m6_tip_link"/>
-    <joint name="${prefix}robotiq_85_m4_screw_tool_tip_joint" type="fixed">
-      <parent link="${prefix}robotiq_85_tip_link"/>
-      <child link="${prefix}screw_tool_m4_tip_link"/>
-      <origin rpy="0.0 ${pi/2} 0.0" xyz="-0.03 0.0 -0.13 "/>
-    </joint>
-    <link name="${prefix}screw_tool_m4_tip_link"/>
-    <joint name="${prefix}robotiq_85_m3_screw_tool_tip_joint" type="fixed">
-      <parent link="${prefix}robotiq_85_tip_link"/>
-      <child link="${prefix}screw_tool_m3_tip_link"/>
-      <origin rpy="0.0 ${pi/2} 0.0" xyz="-0.03 0.0 -0.112 "/>
-    </joint>
-    <link name="${prefix}screw_tool_m3_tip_link"/>
   </xacro:macro>
 </robot>

Commit message: grasp and calibrate screw tool

File: o2as_scene_description/urdf/o2as_base_scene.urdf.xacro (robot description, xacro)
@@ -88,5 +88,5 @@
     wrist_1_lower_limit="${-pi}" wrist_1_upper_limit="${pi}"
     wrist_2_lower_limit="${-pi}" wrist_2_upper_limit="${pi}"
-    wrist_3_lower_limit="${-pi}" wrist_3_upper_limit="${pi}"/>
+    wrist_3_lower_limit="${-pi*5/4}" wrist_3_upper_limit="${pi*5/4}"/>
   <link name="o2as_ground" />
   <joint name="world_a_bot_joint" type="fixed">

File: o2as_scene_description/urdf/robotiq_c_bot_gripper.urdf.xacro (robot description, xacro)
@@ -10,5 +10,5 @@
       <parent link="${prefix}robotiq_85_tip_link"/>
       <child link="${prefix}robotiq_85_tip_rotation_helper_link"/>
-      <origin rpy="0.0 ${pi*3/4} 0.0" xyz="-.03 0 0"/>
+      <origin rpy="0.0 ${-pi/4} 0.0" xyz="-.03 0 0"/>
     </joint>
     <link name="${prefix}robotiq_85_tip_rotation_helper_link"/>
@@ -17,5 +17,5 @@
       <parent link="${prefix}robotiq_85_tip_rotation_helper_link"/>
       <child link="${prefix}screw_tool_m6_tip_link"/>
-      <origin rpy="0.0 0 0" xyz="-0.12 0 0 "/>
+      <origin rpy="0.0 0 0" xyz="0.12 0 .006"/>
     </joint>
     <link name="${prefix}screw_tool_m6_tip_link"/>
@@ -23,5 +23,5 @@
       <parent link="${prefix}robotiq_85_tip_rotation_helper_link"/>
       <child link="${prefix}screw_tool_m4_tip_link"/>
-      <origin rpy="0.0 0 0" xyz="-0.13 0 0 "/>
+      <origin rpy="0.0 0 0" xyz="0.13 0 .006"/>
     </joint>
     <link name="${prefix}screw_tool_m4_tip_link"/>
@@ -29,5 +29,5 @@
       <parent link="${prefix}robotiq_85_tip_rotation_helper_link"/>
       <child link="${prefix}screw_tool_m3_tip_link"/>
-      <origin rpy="0.0 0 0" xyz="-0.112 0 0 "/>
+      <origin rpy="0.0 0 0" xyz="0.112 0 .006"/>
     </joint>
     <link name="${prefix}screw_tool_m3_tip_link"/>

Commit message: Add screw feeders and calibration test

File: o2as_scene_description/urdf/o2as_base_scene.urdf.xacro (robot description, xacro)
@@ -60,11 +60,11 @@
   <xacro:include filename="$(find o2as_scene_description)/urdf/screw_tools.xacro" />
   <!-- Feeders -->
-  <!-- <xacro:include filename="$(find o2as_scene_description)/urdf/screw_feeder.xacro" />
-  <xacro:screw_feeder feedername="m3_feeder" parent="a_bot_base_smfl">
-    <origin xyz=".3 .4 .05" rpy="0 0 ${pi/2}" />
+  <xacro:include filename="$(find o2as_scene_description)/urdf/screw_feeder.xacro" />
+  <xacro:screw_feeder feedername="m3_feeder" parent="c_bot_base_smfl">
+    <origin xyz=".66 -0.25 .065" rpy="0 0 ${pi/2}" />
   </xacro:screw_feeder>
   <xacro:screw_feeder feedername="m4_feeder" parent="c_bot_base_smfl">
-    <origin xyz=".45 .05 .05" rpy="0 0 0" />
-  </xacro:screw_feeder> -->
+    <origin xyz=".54 -0.25 .065" rpy="0 0 ${pi/2}" />
+  </xacro:screw_feeder>
   <!-- robot arms -->
   <xacro:ur5_robot prefix="a_bot_" joint_limited="true"

File: o2as_scene_description/urdf/screw_feeder.xacro (robot description, xacro)
@@ -72,5 +72,7 @@
     <parent link="${feedername}_link"/>
     <child link="${feedername}_outlet_link"/>
-    <origin rpy="0.0 0.0 0.0" xyz="${length-.01} ${width/2} ${height/2 + .02}"/>
+    <!-- <origin rpy="0.0 0 0.0" xyz="${length-.01} ${width/2} ${height/2 + .02}"/> -->
+    <!-- <origin rpy="0.0 ${pi/2} 0.0" xyz="${-height/2 - .02} ${width/2} ${length-.01}"/> -->
+    <origin rpy="0.0 ${pi/2} 0.0" xyz="${length-.01} ${width/2} ${height/2 + .02}"/>
   </joint>
   <link name="${feedername}_outlet_link"/>

Commit message: WIP add camera on a_bot improve view_bin

File: o2as_scene_description/urdf/o2as_base_scene.urdf.xacro (robot description, xacro)
@@ -130,4 +130,14 @@
     <origin xyz="0 0 0" rpy="0 0 0"/>
   </xacro:sensor_d435>
+  <xacro:include filename="$(find o2as_realsense2_camera)/urdf/_d435.urdf.xacro" />
+  <link name="a_bot_cam_holder_link" />
+  <joint name="a_bot_cam_holder_joint" type="fixed">
+    <parent link="a_bot_wrist_2_link" />
+    <child  link="a_bot_cam_holder_link" />
+    <origin xyz="0.0 -0.06 ${0.09465 + .13}" rpy="0.0 0.0 ${pi/2}" />
+  </joint>
+  <xacro:sensor_d435 prefix="a_bot_" parent="a_bot_cam_holder_link">
+    <origin xyz="0 0 0" rpy="0 0 0"/>
+  </xacro:sensor_d435>
   <!-- <xacro:sensor_d435 prefix="d_bot_" parent="o2as_ground">
     <origin xyz="0 0 ${bots_z + 0.9}" rpy="0 ${pi/2} 0"/>

Commit message: Created a calibration point sequence for b_bot.

File: o2as_scene_description/urdf/o2as_base_scene.urdf.xacro (robot description, xacro)
@@ -135,9 +135,9 @@
   <!-- spawn and attach AR markers -->
   <xacro:include filename="$(find o2as_gazebo)/urdf/o2as_ar_marker.urdf.xacro"/>
-  <!-- <xacro:o2as_ar_marker prefix="a_bot_"
-			parent="a_bot_ee_link"
-			marker_id="17">
-    <origin xyz="0.25 0.0 0.047" rpy="0 0 0"/>
-  </xacro:o2as_ar_marker> -->
+  <!-- <xacro:o2as_ar_marker prefix="a_bot_" -->
+  <!-- 			parent="a_bot_ee_link" -->
+  <!-- 			marker_id="17"> -->
+  <!--   <origin xyz="0.17 0.0 0.047" rpy="0 0 0"/> -->
+  <!-- </xacro:o2as_ar_marker> -->
   <!-- <xacro:o2as_ar_marker prefix="b_bot_"
 			parent="b_bot_dual_suction_gripper_base_link"
@@ -150,9 +150,14 @@
   <!--   <origin xyz="0.063 0.0 0.0215" rpy="0 0 0"/> -->
   <!-- </xacro:o2as_ar_marker> -->
-  <!-- <xacro:o2as_ar_marker prefix="c_bot_"
+  <xacro:o2as_ar_marker prefix="b_bot_"
+			parent="b_bot_robotiq_85_tip_link"
+			marker_id="26">
+    <origin xyz="0.0 0.0 0.0185" rpy="0 0 0"/>
+  </xacro:o2as_ar_marker>
+  <xacro:o2as_ar_marker prefix="c_bot_"
 			parent="c_bot_robotiq_85_tip_link"
 			marker_id="256">
     <origin xyz="0.0 0.0 0.0185" rpy="0 0 0"/>
-  </xacro:o2as_ar_marker> -->
+  </xacro:o2as_ar_marker>
   <!-- Add PhoXi 3D scanners -->
   <xacro:include filename="$(find o2as_scene_description)/urdf/phoxi_m_camera.urdf.xacro" />

Commit message: Modified hand-eye calibration points.

File: o2as_scene_description/urdf/o2as_base_scene.urdf.xacro (robot description, xacro)
@@ -135,14 +135,14 @@
   <!-- spawn and attach AR markers -->
   <xacro:include filename="$(find o2as_gazebo)/urdf/o2as_ar_marker.urdf.xacro"/>
-  <!-- <xacro:o2as_ar_marker prefix="a_bot_" -->
-  <!-- 			parent="a_bot_ee_link" -->
-  <!-- 			marker_id="17"> -->
-  <!--   <origin xyz="0.17 0.0 0.047" rpy="0 0 0"/> -->
+  <xacro:o2as_ar_marker prefix="a_bot_"
+  			parent="a_bot_ee_link"
+  			marker_id="17">
+    <origin xyz="0.08 0.0 0.065" rpy="0 0 0"/>
+  </xacro:o2as_ar_marker>
+  <!-- <xacro:o2as_ar_marker prefix="b_bot_" -->
+  <!-- 			parent="b_bot_dual_suction_gripper_base_link" -->
+  <!-- 			marker_id="26"> -->
+  <!--   <origin xyz="0.063 0.0 0.0215" rpy="0 0 0"/> -->
   <!-- </xacro:o2as_ar_marker> -->
-  <!-- <xacro:o2as_ar_marker prefix="b_bot_"
-			parent="b_bot_dual_suction_gripper_base_link"
-			marker_id="26">
-    <origin xyz="0.063 0.0 0.0215" rpy="0 0 0"/>
-  </xacro:o2as_ar_marker> -->
   <!-- <xacro:o2as_ar_marker prefix="b_bot_" -->
   <!-- 			parent="b_bot_single_suction_gripper_base_link" -->

Commit message: Remove outer gripper motor

File: o2as_scene_description/urdf/o2as_base_scene.urdf.xacro (robot description, xacro)
@@ -65,5 +65,5 @@
   </xacro:screw_feeder>
   <xacro:screw_feeder feedername="m4_feeder" parent="c_bot_base_smfl">
-    <origin xyz=".54 -0.25 .065" rpy="0 0 ${pi/2}" />
+    <origin xyz=".52 -0.25 .065" rpy="0 0 ${pi/2}" />
   </xacro:screw_feeder>
   <!-- robot arms -->

Commit message: Imported handeye_server from easy_handeye.

File: o2as_scene_description/urdf/o2as_base_scene.urdf.xacro (robot description, xacro)
@@ -114,8 +114,13 @@
     <origin xyz="0.0 0 0.0" rpy="0 0 0"/>
   </xacro:InnerOnlyGripper>
+  <!-- spawn and attach dual suction grippers -->
+  <!-- <xacro:include filename="$(find o2as_scene_description)/urdf/dual_suction_gripper.urdf.xacro" />
+  <xacro:dual_suction_gripper_o2as prefix="b_bot_" parent = "b_bot_ee_link">
+    <origin xyz="0 0 0" rpy="0 0 0"/>
+  </xacro:dual_suction_gripper_o2as> -->
   <!-- spawn and attach dual robotiq 85 grippers -->
   <xacro:include filename="$(find o2as_scene_description)/urdf/robotiq_b_bot_gripper.urdf.xacro" />
+  <xacro:o2as_b_bot_gripper prefix="b_bot_" parent = "b_bot_ee_link" />
   <xacro:include filename="$(find o2as_scene_description)/urdf/robotiq_c_bot_gripper.urdf.xacro" />
-  <xacro:o2as_b_bot_gripper prefix="b_bot_" parent = "b_bot_ee_link" />
   <xacro:o2as_c_bot_gripper prefix="c_bot_" parent = "c_bot_ee_link"/>
   <!-- Add cameras -->
@@ -147,12 +152,12 @@
   <xacro:o2as_ar_marker prefix="a_bot_"
   			parent="a_bot_ee_link"
-  			marker_id="17">
+  			marker_id="26">
     <origin xyz="0.08 0.0 0.065" rpy="0 0 0"/>
   </xacro:o2as_ar_marker>
-  <xacro:o2as_ar_marker prefix="b_bot_"
-  			parent="b_bot_dual_suction_gripper_base_link"
-  			marker_id="26">
-    <origin xyz="0.063 0.0 0.0215" rpy="0 0 0"/>
-  </xacro:o2as_ar_marker>
+  <!-- <xacro:o2as_ar_marker prefix="b_bot_" -->
+  <!-- 			parent="b_bot_dual_suction_gripper_base_link" -->
+  <!-- 			marker_id="26"> -->
+  <!--   <origin xyz="0.063 0.0 0.0215" rpy="0 0 0"/> -->
+  <!-- </xacro:o2as_ar_marker> -->
   <!-- <xacro:o2as_ar_marker prefix="b_bot_" -->
   <!-- 			parent="b_bot_single_suction_gripper_base_link" -->
@@ -160,12 +165,12 @@
   <!--   <origin xyz="0.063 0.0 0.0215" rpy="0 0 0"/> -->
   <!-- </xacro:o2as_ar_marker> -->
-  <!-- <xacro:o2as_ar_marker prefix="b_bot_" -->
-  <!-- 			parent="b_bot_robotiq_85_tip_link" -->
-  <!-- 			marker_id="26"> -->
-  <!--   <origin xyz="0.0 0.0 0.0185" rpy="0 0 0"/> -->
-  <!-- </xacro:o2as_ar_marker> -->
+  <xacro:o2as_ar_marker prefix="b_bot_"
+			parent="b_bot_robotiq_85_tip_link"
+			marker_id="26">
+    <origin xyz="0.0 0.0 0.0185" rpy="0 0 0"/>
+  </xacro:o2as_ar_marker>
   <xacro:o2as_ar_marker prefix="c_bot_"
 			parent="c_bot_robotiq_85_tip_link"
-			marker_id="256">
+			marker_id="26">
     <origin xyz="0.0 0.0 0.0185" rpy="0 0 0"/>
   </xacro:o2as_ar_marker>

Commit message: Cleaning up.

File: o2as_scene_description/urdf/o2as_base_scene.urdf.xacro (robot description, xacro)
@@ -23,5 +23,5 @@
   <!-- Scene items (trays, bins...) -->
   <!-- <xacro:include filename="$(find o2as_scene_description)/urdf/taskboard_scene.xacro" /> -->
-  <xacro:include filename="$(find o2as_scene_description)/urdf/kitting_scene.xacro" />
+  <!-- <xacro:include filename="$(find o2as_scene_description)/urdf/kitting_scene.xa -->cro" />
   <!-- <xacro:include filename="$(find o2as_scene_description)/urdf/assembly_scene.xacro" /> -->
   <!-- Robot bases -->
@@ -175,9 +175,15 @@
     <origin xyz="0.0 0.0 0.0185" rpy="0 0 0"/>
   </xacro:o2as_ar_marker>
+  <xacro:o2as_ar_marker prefix="workspace_"
+			parent="workspace_center"
+			marker_id="256">
+    <origin xyz="0.0 0.0 0.0" rpy="0 0 0"/>
+  </xacro:o2as_ar_marker>
   <!-- Add PhoXi 3D scanners -->
   <xacro:include filename="$(find o2as_scene_description)/urdf/phoxi_m_camera.urdf.xacro" />
   <xacro:phoxi_m_camera prefix="a_" parent="o2as_ground">
     <!-- <origin xyz="0.56 0 ${bots_z + .1 + .8}" rpy="${-160*pi/180} 0 ${pi/2}"/> -->
-    <origin xyz="0.46 0 ${bots_z + .1 + .8}" rpy="${-160*pi/180} 0 ${pi/2}"/>
+    <origin xyz="0.56824 -0.0047217 1.3994"
+	    rpy="${-154.926*pi/180} ${-0.221*pi/180} ${89.704*pi/180}"/>
   </xacro:phoxi_m_camera>
   <!-- I would like to remove the "world" link definition, but apparently it is necessary for Gazebo -->

Commit message: Changed b_bot's path for calibration.

File: o2as_scene_description/urdf/o2as_base_scene.urdf.xacro (robot description, xacro)
@@ -184,6 +184,6 @@
   <xacro:phoxi_m_camera prefix="a_" parent="o2as_ground">
     <!-- <origin xyz="0.56 0 ${bots_z + .1 + .8}" rpy="${-160*pi/180} 0 ${pi/2}"/> -->
-    <origin xyz="0.56824 -0.0047217 1.3994"
-	    rpy="${-154.926*pi/180} ${-0.221*pi/180} ${89.704*pi/180}"/>
+    <origin xyz="0.66765 -0.01114 1.4583"
+	    rpy="${-149.516*pi/180} ${0.274*pi/180} ${92.033*pi/180}"/>
   </xacro:phoxi_m_camera>
   <!-- I would like to remove the "world" link definition, but apparently it is necessary for Gazebo -->

Commit message: Calibration at OSX updated.

File: o2as_scene_description/urdf/o2as_base_scene.urdf.xacro (robot description, xacro)
@@ -184,6 +184,6 @@
   <xacro:phoxi_m_camera prefix="a_" parent="o2as_ground">
     <!-- <origin xyz="0.56 0 ${bots_z + .1 + .8}" rpy="${-160*pi/180} 0 ${pi/2}"/> -->
-    <origin xyz="0.66765 -0.01114 1.4583"
-	    rpy="${-149.516*pi/180} ${0.274*pi/180} ${92.033*pi/180}"/>
+    <origin xyz="0.65526 -0.018791 1.4169"
+	    rpy="${-149.595*pi/180} ${0.473*pi/180} ${91.976*pi/180}"/>
   </xacro:phoxi_m_camera>
   <!-- I would like to remove the "world" link definition, but apparently it is necessary for Gazebo -->

Commit message: WIP: update phoxi pose.

File: o2as_scene_description/urdf/o2as_base_scene.urdf.xacro (robot description, xacro)
@@ -161,5 +161,6 @@
   <xacro:phoxi_m_camera prefix="a_" parent="o2as_ground">
     <!-- <origin xyz="0.56 0 ${bots_z + .1 + .8}" rpy="${-160*pi/180} 0 ${pi/2}"/> -->
-    <origin xyz="0.46 0 ${bots_z + .1 + .8}" rpy="${-160*pi/180} 0 ${pi/2}"/>
+    <!-- <origin xyz="0.46 0 ${bots_z + .1 + .8}" rpy="${-160*pi/180} 0 ${pi/2}"/> -->
+    <origin xyz="0.65526 -0.018791 1.4169" rpy="${-149.595*pi/180} ${0.473*pi/180} ${91.976*pi/180}" />
   </xacro:phoxi_m_camera>
   <!-- I would like to remove the "world" link definition, but apparently it is necessary for Gazebo -->
