Commit message: Missing files are added.

File: o2as_scene_description/urdf/o2as_base_scene.urdf.xacro (robot description, xacro)
@@ -175,9 +175,15 @@
     <origin xyz="0.0 0.0 0.0185" rpy="0 0 0"/>
   </xacro:o2as_ar_marker>
-  <xacro:o2as_ar_marker prefix="workspace_"
-			parent="workspace_center"
-			marker_id="256">
+  <!-- <xacro:o2as_ar_marker prefix="workspace_" -->
+  <!-- 			parent="workspace_center" -->
+  <!-- 			marker_id="256"> -->
+  <!--   <origin xyz="0.0 0.0 0.0005" rpy="0 0 0"/> -->
+  <!-- </xacro:o2as_ar_marker> -->
+  <xacro:include filename="$(find o2as_gazebo)/urdf/o2as_ar_marker_16cm.urdf.xacro"/>
+  <xacro:o2as_ar_marker_16cm prefix="workspace_"
+  			parent="workspace_center"
+  			marker_id="32">
     <origin xyz="0.0 0.0 0.0005" rpy="0 0 0"/>
-  </xacro:o2as_ar_marker>
+  </xacro:o2as_ar_marker_16cm>
   <!-- Add PhoXi 3D scanners -->
   <xacro:include filename="$(find o2as_scene_description)/urdf/phoxi_m_camera.urdf.xacro" />

Commit message: State of the test on Sunday 18h

File: o2as_scene_description/urdf/o2as_base_scene.urdf.xacro (robot description, xacro)
@@ -136,20 +136,5 @@
   </xacro:sensor_d435> -->
   <!-- spawn and attach AR markers -->
-  <xacro:include filename="$(find o2as_gazebo)/urdf/o2as_ar_marker.urdf.xacro"/>
-  <!-- <xacro:o2as_ar_marker prefix="a_bot_" -->
-  <!-- 			parent="a_bot_ee_link" -->
-  <!-- 			marker_id="26"> -->
-  <!--   <origin xyz="0.08 0.00 0.065" rpy="0 0 0"/> -->
-  <!-- </xacro:o2as_ar_marker> -->
-  <!-- <xacro:o2as_ar_marker prefix="b_bot_" -->
-  <!-- 			parent="b_bot_dual_suction_gripper_base_link" -->
-  <!-- 			marker_id="26"> -->
-  <!--   <origin xyz="0.063 0.0 0.0215" rpy="0 0 0"/> -->
-  <!-- </xacro:o2as_ar_marker> -->
-  <!-- <xacro:o2as_ar_marker prefix="b_bot_" -->
-  <!-- 			parent="b_bot_single_suction_gripper_base_link" -->
-  <!-- 			marker_id="26"> -->
-  <!--   <origin xyz="0.063 0.0 0.0215" rpy="0 0 0"/> -->
-  <!-- </xacro:o2as_ar_marker> -->
+  <!-- <xacro:include filename="$(find o2as_gazebo)/urdf/o2as_ar_marker.urdf.xacro"/>
   <xacro:o2as_ar_marker prefix="b_bot_"
 			parent="b_bot_robotiq_85_tip_link"
@@ -162,14 +147,9 @@
     <origin xyz="0.0 0.0 0.0185" rpy="0 0 0"/>
   </xacro:o2as_ar_marker>
-  <!-- <xacro:o2as_ar_marker prefix="workspace_" -->
-  <!-- 			parent="workspace_center" -->
-  <!-- 			marker_id="256"> -->
-  <!--   <origin xyz="0.0 0.0 0.0005" rpy="0 0 0"/> -->
-  <!-- </xacro:o2as_ar_marker> -->
   <xacro:o2as_ar_marker_16cm prefix="workspace_"
   			parent="workspace_center"
   			marker_id="32">
     <origin xyz="0.0 0.0 0.0005" rpy="0 0 0"/>
-  </xacro:o2as_ar_marker_16cm>
+  </xacro:o2as_ar_marker_16cm> -->
   <!-- Add PhoXi 3D scanners -->
   <xacro:include filename="$(find o2as_scene_description)/urdf/phoxi_m_camera.urdf.xacro" />

Commit message: update a_bot camera pose in urdf

File: o2as_scene_description/urdf/o2as_base_scene.urdf.xacro (robot description, xacro)
@@ -127,5 +127,5 @@
     <parent link="a_bot_wrist_2_link" />
     <child  link="a_bot_cam_holder_link" />
-    <origin xyz="0.0 -0.06 ${0.09465 + .13}" rpy="0.0 0.0 ${pi/2}" />
+    <origin xyz="0.04 -0.06 0.20" rpy="${12*pi/180} 0.0 ${pi/2}" />
   </joint>
   <xacro:sensor_d435 prefix="a_bot_" parent="a_bot_cam_holder_link">

Commit message: Cleaning up.

File: o2as_scene_description/urdf/o2as_base_scene.urdf.xacro (robot description, xacro)
@@ -175,9 +175,9 @@
     <origin xyz="0.0 0.0 0.0185" rpy="0 0 0"/>
   </xacro:o2as_ar_marker>
-  <xacro:o2as_ar_marker prefix="workspace_"
-  			parent="workspace_center"
-  			marker_id="256">
+  <xacro:o2as_ar_marker_16cm prefix="workspace_"
+  			     parent="workspace_center"
+  			     marker_id="32">
     <origin xyz="0.0 0.0 0.0005" rpy="0 0 0"/>
-  </xacro:o2as_ar_marker>
+  </xacro:o2as_ar_marker_16cm>
   <!-- <xacro:o2as_ar_marker prefix="workspace_" -->
   <!-- 			parent="workspace_center" -->
@@ -188,7 +188,15 @@
   <xacro:include filename="$(find o2as_scene_description)/urdf/phoxi_m_camera.urdf.xacro" />
   <xacro:phoxi_m_camera prefix="a_" parent="o2as_ground">
-    <!-- <origin xyz="0.56 0 ${bots_z + .1 + .8}" rpy="${-160*pi/180} 0 ${pi/2}"/> -->
-    <origin xyz="0.65526 -0.018791 1.4169"
-	    rpy="${-149.595*pi/180} ${0.473*pi/180} ${91.976*pi/180}"/>
+    <!-- <origin xyz="0.56 0 ${bots_z + .1 + .8}"
+	 rpy="${-160*pi/180} 0 ${pi/2}"/> -->
+    <!-- 181005@OSX -->
+    <!-- <origin xyz="0.65526 -0.018791 1.4169" -->
+    <!-- 	    rpy="${-149.595*pi/180} ${0.473*pi/180} ${91.976*pi/180}"/> -->
+    <!-- 181007@OSX -->
+    <!-- <origin xyz="0.6554 -0.020392 1.413" -->
+    <!-- 	    rpy="${-149.604*pi/180} ${0.34821*pi/180} ${91.866*pi/180}"/> -->
+    <!-- 181008@OSX -->
+    <origin xyz="0.674391 -0.0223742 ${bots_z + 0.696023}"
+	    rpy="${-149.801*pi/180} ${0.156861*pi/180} ${91.2544*pi/180}"/>
   </xacro:phoxi_m_camera>
   <!-- I would like to remove the "world" link definition, but apparently it is necessary for Gazebo -->

Commit message: Add simple handeye routine

File: o2as_scene_description/urdf/o2as_base_scene.urdf.xacro (robot description, xacro)
@@ -145,4 +145,10 @@
     <origin xyz="0 0 0" rpy="0 0 0"/>
   </xacro:sensor_d435>
+  <link name="a_bot_camera_calibrated_frame_link" />
+  <joint name="a_bot_camera_calibrated_frame_joint" type="fixed">
+    <parent link="a_bot_wrist_2_link" />
+    <child  link="a_bot_camera_calibrated_frame_link" />
+    <origin xyz="-0.00742849565969 -0.055347079996 0.196043734813" rpy="-1.517 -0.015 -0.014" />
+  </joint>
   <!-- <xacro:sensor_d435 prefix="d_bot_" parent="o2as_ground">
     <origin xyz="0 0 ${bots_z + 0.9}" rpy="0 ${pi/2} 0"/>

Commit message: Add realsense calibration result

File: o2as_scene_description/urdf/o2as_base_scene.urdf.xacro (robot description, xacro)
@@ -132,4 +132,10 @@
     <origin xyz="0 0 0" rpy="0 0 0"/>
   </xacro:sensor_d435>
+  <link name="a_bot_camera_calibrated_frame_link" />
+  <joint name="a_bot_camera_calibrated_frame_joint" type="fixed">
+    <parent link="a_bot_wrist_2_link" />
+    <child  link="a_bot_camera_calibrated_frame_link" />
+    <origin xyz="-0.00742849565969 -0.055347079996 0.196043734813" rpy="-1.517 -0.015 -0.014" />
+  </joint>
   <!-- <xacro:sensor_d435 prefix="d_bot_" parent="o2as_ground">
     <origin xyz="0 0 ${bots_z + 0.9}" rpy="0 ${pi/2} 0"/>

Commit message: Merge fix-kitting into check-handeye-calibration-realsense

File: o2as_scene_description/urdf/o2as_base_scene.urdf.xacro (robot description, xacro)
@@ -140,5 +140,5 @@
     <parent link="a_bot_wrist_2_link" />
     <child  link="a_bot_cam_holder_link" />
-    <origin xyz="0.0 -0.06 ${0.09465 + .13}" rpy="0.0 0.0 ${pi/2}" />
+    <origin xyz="0.04 -0.06 0.20" rpy="${12*pi/180} 0.0 ${pi/2}" />
   </joint>
   <xacro:sensor_d435 prefix="a_bot_" parent="a_bot_cam_holder_link">

File: o2as_scene_description/urdf/robotiq_b_bot_gripper.urdf.xacro (robot description, xacro)
@@ -30,5 +30,5 @@
       <parent link="${prefix}robotiq_85_tip_link"/>
       <child link="${prefix}screw_tool_m3_tip_link"/>
-      <origin rpy="0.0 ${pi/2} 0.0" xyz="${dx} 0.0 -0.112 "/>
+      <origin rpy="0.0 ${pi/2} 0.0" xyz="${dx} 0.0 -0.132 "/>
     </joint>
     <link name="${prefix}screw_tool_m3_tip_link"/>
@@ -42,5 +42,5 @@
       <parent link="${prefix}robotiq_85_tip_link"/>
       <child link="${prefix}suction_tool_tip_link"/>
-      <origin rpy="0.0 ${pi/2} 0.0" xyz="${dx+.013} 0.0 -0.131 "/>
+      <origin rpy="0.0 ${pi/2} 0.0" xyz="${dx+.02} 0.0 -0.131 "/>
     </joint>
     <link name="${prefix}suction_tool_tip_link"/>

File: o2as_scene_description/urdf/screw_tools.xacro (robot description, xacro)
@@ -126,5 +126,5 @@
     <parent link="screw_tool_holder" />
     <child link="suction_tool_link" />
-    <origin xyz="-0.05 ${tool_offset} 0.004" rpy="0.0 0.0 0.0" />
+    <origin xyz="-0.355 ${tool_offset - .025} 0.004" rpy="0.0 0.0 0.0" />
   </joint>
   <link name="screw_tool_m4_link">

Commit message: Improve realsense calibration

File: o2as_scene_description/urdf/o2as_base_scene.urdf.xacro (robot description, xacro)
@@ -149,5 +149,5 @@
     <parent link="a_bot_wrist_2_link" />
     <child  link="a_bot_camera_calibrated_frame_link" />
-    <origin xyz="-0.00742849565969 -0.055347079996 0.196043734813" rpy="-1.517 -0.015 -0.014" />
+    <origin xyz="-0.00584875065097 -0.0601140904909 0.190359410313" rpy="-1.631 -0.020 -0.016" />
   </joint>
   <!-- <xacro:sensor_d435 prefix="d_bot_" parent="o2as_ground">

Commit message: Add calibration scene

File: o2as_scene_description/urdf/o2as_base_scene.urdf.xacro (robot description, xacro)
@@ -23,6 +23,7 @@
   <!-- Scene items (trays, bins...) -->
   <!-- <xacro:include filename="$(find o2as_scene_description)/urdf/taskboard_scene.xacro" /> -->
-  <!-- <xacro:include filename="$(find o2as_scene_description)/urdf/kitting_scene.xacro" /> -->
+  <xacro:include filename="$(find o2as_scene_description)/urdf/kitting_scene.xacro" />
   <!-- <xacro:include filename="$(find o2as_scene_description)/urdf/assembly_scene.xacro" /> -->
+  <!-- <xacro:include filename="$(find o2as_scene_description)/urdf/calibration_scene.xacro" /> -->
   <!-- Robot bases -->
   <!-- Putting these at height 0.0 makes them intersect with the ground, so they are elevated. -->
@@ -59,12 +60,4 @@
   <!-- Screw holder & screw tool visual -->
   <xacro:include filename="$(find o2as_scene_description)/urdf/screw_tools.xacro" />
-  <!-- Feeders -->
-  <xacro:include filename="$(find o2as_scene_description)/urdf/screw_feeder.xacro" />
-  <xacro:screw_feeder feedername="m3_feeder" parent="c_bot_base_smfl">
-    <origin xyz=".66 -0.25 .065" rpy="0 0 ${pi/2}" />
-  </xacro:screw_feeder>
-  <xacro:screw_feeder feedername="m4_feeder" parent="c_bot_base_smfl">
-    <origin xyz=".52 -0.25 .065" rpy="0 0 ${pi/2}" />
-  </xacro:screw_feeder>
   <!-- robot arms -->
   <xacro:ur5_robot prefix="a_bot_" joint_limited="false"
@@ -106,17 +99,8 @@
   </joint>
   <!-- spawn and attach grippers -->
-  <!-- <xacro:include filename="$(find o2as_scene_description)/urdf/precision_gripper.xacro" />
-  <xacro:precision_gripper prefix="a_bot_"  grippername = "gripper" parent = "a_bot_tool0">
-    <origin xyz="0.0 0 0.04" rpy="0 ${pi/2} 0"/>
-  </xacro:precision_gripper> -->
   <xacro:include filename="$(find o2as_scene_description)/urdf/InnerOnlyGripper.xacro" />
   <xacro:InnerOnlyGripper prefix="a_bot_"  grippername = "gripper" parent = "a_bot_tool0">
     <origin xyz="0.0 0 0.0" rpy="0 0 0"/>
   </xacro:InnerOnlyGripper>
-  <!-- spawn and attach dual suction grippers -->
-  <!-- <xacro:include filename="$(find o2as_scene_description)/urdf/dual_suction_gripper.urdf.xacro" />
-  <xacro:dual_suction_gripper_o2as prefix="b_bot_" parent = "b_bot_ee_link">
-    <origin xyz="0 0 0" rpy="0 0 0"/>
-  </xacro:dual_suction_gripper_o2as> -->
   <!-- spawn and attach dual robotiq 85 grippers -->
   <xacro:include filename="$(find o2as_scene_description)/urdf/robotiq_b_bot_gripper.urdf.xacro" />
@@ -154,53 +138,7 @@
     <origin xyz="0 0 ${bots_z + 0.9}" rpy="0 ${pi/2} 0"/>
   </xacro:sensor_d435> -->
-  <!-- spawn and attach AR markers -->
-  <xacro:include filename="$(find o2as_gazebo)/urdf/o2as_ar_marker.urdf.xacro"/>
-  <!-- <xacro:o2as_ar_marker prefix="a_bot_" -->
-  <!-- 			parent="a_bot_ee_link" -->
-  <!-- 			marker_id="26"> -->
-  <!--   <origin xyz="0.08 0.00 0.065" rpy="0 0 0"/> -->
-  <!-- </xacro:o2as_ar_marker> -->
-  <!-- <xacro:o2as_ar_marker prefix="b_bot_" -->
-  <!-- 			parent="b_bot_dual_suction_gripper_base_link" -->
-  <!-- 			marker_id="26"> -->
-  <!--   <origin xyz="0.063 0.0 0.0215" rpy="0 0 0"/> -->
-  <!-- </xacro:o2as_ar_marker> -->
-  <!-- <xacro:o2as_ar_marker prefix="b_bot_" -->
-  <!-- 			parent="b_bot_single_suction_gripper_base_link" -->
-  <!-- 			marker_id="26"> -->
-  <!--   <origin xyz="0.063 0.0 0.0215" rpy="0 0 0"/> -->
-  <!-- </xacro:o2as_ar_marker> -->
-  <xacro:o2as_ar_marker prefix="b_bot_"
-			parent="b_bot_robotiq_85_tip_link"
-			marker_id="26">
-    <origin xyz="0.0 0.0 0.0185" rpy="0 0 0"/>
-  </xacro:o2as_ar_marker>
-  <xacro:o2as_ar_marker prefix="c_bot_"
-			parent="c_bot_robotiq_85_tip_link"
-			marker_id="26">
-    <origin xyz="0.0 0.0 0.0185" rpy="0 0 0"/>
-  </xacro:o2as_ar_marker>
-  <xacro:o2as_ar_marker_16cm prefix="workspace_"
-  			     parent="workspace_center"
-  			     marker_id="32">
-    <origin xyz="0.0 0.0 0.0005" rpy="0 0 0"/>
-  </xacro:o2as_ar_marker_16cm>
-  <!-- <xacro:o2as_ar_marker prefix="workspace_" -->
-  <!-- 			parent="workspace_center" -->
-  <!-- 			marker_id="26"> -->
-  <!--   <origin xyz="0.0 0.0 0.0005" rpy="0 0 0"/> -->
-  <!-- </xacro:o2as_ar_marker> -->
   <!-- Add PhoXi 3D scanners -->
   <xacro:include filename="$(find o2as_scene_description)/urdf/phoxi_m_camera.urdf.xacro" />
   <xacro:phoxi_m_camera prefix="a_" parent="o2as_ground">
-    <!-- <origin xyz="0.56 0 ${bots_z + .1 + .8}"
-	 rpy="${-160*pi/180} 0 ${pi/2}"/> -->
-    <!-- 181005@OSX -->
-    <!-- <origin xyz="0.65526 -0.018791 1.4169" -->
-    <!-- 	    rpy="${-149.595*pi/180} ${0.473*pi/180} ${91.976*pi/180}"/> -->
-    <!-- 181007@OSX -->
-    <!-- <origin xyz="0.6554 -0.020392 1.413" -->
-    <!-- 	    rpy="${-149.604*pi/180} ${0.34821*pi/180} ${91.866*pi/180}"/> -->
-    <!-- 181008@OSX -->
     <origin xyz="0.674391 -0.0223742 ${bots_z + 0.696023}"
 	    rpy="${-149.801*pi/180} ${0.156861*pi/180} ${91.2544*pi/180}"/>

Commit message: Update calibration
Still not perfect, especially with the screw tool and rotations, but hopefully good enough

File: o2as_scene_description/urdf/o2as_base_scene.urdf.xacro (robot description, xacro)
@@ -2,12 +2,11 @@
 <robot xmlns:xacro="http://www.ros.org/wiki/xacro"
        name="o2as_base_scene" >
-  <!-- Calibration from 20 August 2018 -->
+  <!-- Calibration from 12 October 2018 -->
   <!-- Calibration help: If the robot is not moving far enough to the calibration point, increase these distances -->
   <xacro:property name="a_bot_x" value="-0.01"/>
   <xacro:property name="a_bot_y" value="-0.5"/>
-  <xacro:property name="b_bot_x" value="-0.009"/>
-  <xacro:property name="b_bot_y" value="0.503"/>
-  <xacro:property name="b_bot_theta" value="-3.12832815"/>
-  <!-- The above is 0.76 degrees away from pi (Sep 17; not perfect) -->
+  <xacro:property name="b_bot_x" value="-0.008"/>
+  <xacro:property name="b_bot_y" value="0.50"/>
+  <xacro:property name="b_bot_theta" value="-3.14"/>
   <xacro:property name="c_bot_x" value="-0.499"/>
   <xacro:property name="c_bot_y" value="0.0"/>

Commit message: Update the taskboard urdf (for part7 and part5)

File: o2as_scene_description/urdf/o2as_base_scene.urdf.xacro (robot description, xacro)
@@ -21,5 +21,5 @@
   <xacro:include filename="$(find o2as_scene_description)/urdf/ur3.urdf.xacro" />
   <!-- Scene items (trays, bins...) -->
-  <!-- <xacro:include filename="$(find o2as_scene_description)/urdf/taskboard_scene.xacro" /> -->
+  <xacro:include filename="$(find o2as_scene_description)/urdf/taskboard_scene.xacro" />
   <!-- <xacro:include filename="$(find o2as_scene_description)/urdf/kitting_scene.xacro" /> -->
   <xacro:include filename="$(find o2as_scene_description)/urdf/assembly_scene.xacro" />

File: o2as_scene_description/urdf/task_board.xacro (robot description, xacro)
@@ -62,11 +62,12 @@
     <parent link="${boardname}_surface"/>
     <child link="${boardname}_part5"/>
-    <origin rpy="0.0 0.0 ${pi/2}" xyz="0.07 0.26 0.0045"/>
+    <origin rpy="0.0 0.0 ${pi/2}" xyz="0.07 0.26 0.002"/>
   </joint>
   <link name="${boardname}_part5">
     <visual>
-      <origin xyz="0 0 -.00275" rpy="0 0 0"/>
-      <geometry>
-        <cylinder length=".0045" radius=".002"/>
+      <origin xyz="0 0 .0375" rpy="0 0 0"/>
+      <geometry>
+        <!-- <cylinder length=".0045" radius=".002"/>  -->
+        <cylinder length=".075" radius=".005"/>
       </geometry>
       <material name="grey">
@@ -113,5 +114,5 @@
     <parent link="${boardname}_surface"/>
     <child link="${boardname}_part7_1"/>
-    <origin rpy="0.0 0.0 ${pi/2}" xyz="0.335 0.056 0.05"/>
+    <origin rpy="0.0 0.0 ${pi/2}" xyz="0.362 0.056 0.05"/>
   </joint>
   <link name="${boardname}_part7_1"/>
@@ -119,5 +120,5 @@
     <parent link="${boardname}_surface"/>
     <child link="${boardname}_part7_2"/>
-    <origin rpy="0.0 0.0 ${pi/2}" xyz="0.338 0.056 0.05"/>
+    <origin rpy="0.0 0.0 ${pi/2}" xyz="0.365 0.056 0.05"/>
   </joint>
   <link name="${boardname}_part7_2">

Commit message: Add taskboard seq

File: o2as_scene_description/urdf/o2as_base_scene.urdf.xacro (robot description, xacro)
@@ -23,5 +23,5 @@
   <xacro:include filename="$(find o2as_scene_description)/urdf/taskboard_scene.xacro" />
   <!-- <xacro:include filename="$(find o2as_scene_description)/urdf/kitting_scene.xacro" /> -->
-  <xacro:include filename="$(find o2as_scene_description)/urdf/assembly_scene.xacro" />
+  <!-- <xacro:include filename="$(find o2as_scene_description)/urdf/assembly_scene.xacro" /> -->
   <!-- <xacro:include filename="$(find o2as_scene_description)/urdf/calibration_scene.xacro" /> -->
   <!-- Robot bases -->
@@ -107,4 +107,12 @@
   <xacro:include filename="$(find o2as_scene_description)/urdf/robotiq_c_bot_gripper.urdf.xacro" />
   <xacro:o2as_c_bot_gripper prefix="c_bot_" parent = "c_bot_ee_link"/>
+  <!-- Feeders -->
+  <xacro:include filename="$(find o2as_scene_description)/urdf/screw_feeder.xacro" />
+  <xacro:screw_feeder feedername="m3_feeder" parent="c_bot_base_smfl">
+    <origin xyz=".66 -0.25 .065" rpy="0 0 ${pi/2}" />
+  </xacro:screw_feeder>
+  <xacro:screw_feeder feedername="m4_feeder" parent="c_bot_base_smfl">
+    <origin xyz=".52 -0.25 .065" rpy="0 0 ${pi/2}" />
+  </xacro:screw_feeder>
   <!-- Add cameras -->
   <xacro:include filename="$(find o2as_realsense2_camera)/urdf/_d435.urdf.xacro" />

File: o2as_scene_description/urdf/task_board.xacro (robot description, xacro)
@@ -197,5 +197,5 @@
     <parent link="${boardname}_surface"/>
     <child link="${boardname}_part13"/>
-    <origin rpy="0.0 0.0 ${pi/2}" xyz="0.35 0.12 0.0"/>
+    <origin rpy="0.0 0.0 ${pi/2}" xyz="0.07 0.26 0.078"/>
   </joint>
   <link name="${boardname}_part13"/>
@@ -219,5 +219,5 @@
     <parent link="${boardname}_surface"/>
     <child link="${boardname}_part15"/>
-    <origin rpy="0.0 0.0 ${pi/2}" xyz="0.08 0.31 0.076"/>
+    <origin rpy="0.0 0.0 ${pi/2}" xyz="0.07 0.26 0.0772"/>
   </joint>
   <link name="${boardname}_part15"/>

Commit message: Fix small things, calibration

File: o2as_scene_description/urdf/o2as_base_scene.urdf.xacro (robot description, xacro)
@@ -22,6 +22,6 @@
   <!-- Scene items (trays, bins...) -->
   <!-- <xacro:include filename="$(find o2as_scene_description)/urdf/taskboard_scene.xacro" /> -->
-  <!-- <xacro:include filename="$(find o2as_scene_description)/urdf/kitting_scene.xacro" /> -->
-  <xacro:include filename="$(find o2as_scene_description)/urdf/assembly_scene.xacro" />
+  <xacro:include filename="$(find o2as_scene_description)/urdf/kitting_scene.xacro" />
+  <!-- <xacro:include filename="$(find o2as_scene_description)/urdf/assembly_scene.xacro" /> -->
   <!-- <xacro:include filename="$(find o2as_scene_description)/urdf/calibration_scene.xacro" /> -->
   <!-- Robot bases -->

File: o2as_scene_description/urdf/screw_tools.xacro (robot description, xacro)
@@ -126,5 +126,5 @@
     <parent link="screw_tool_holder" />
     <child link="suction_tool_link" />
-    <origin xyz="-0.355 ${tool_offset - .025} 0.004" rpy="0.0 0.0 0.0" />
+    <origin xyz="-0.355 ${tool_offset - .015} 0.004" rpy="0.0 0.0 0.0" />
   </joint>
   <link name="screw_tool_m4_link">

Commit message: Added plane_detector node.

File: o2as_scene_description/urdf/o2as_base_scene.urdf.xacro (robot description, xacro)
@@ -115,11 +115,11 @@
   </xacro:InnerOnlyGripper>
   <!-- spawn and attach dual suction grippers -->
-  <!-- <xacro:include filename="$(find o2as_scene_description)/urdf/dual_suction_gripper.urdf.xacro" />
+  <xacro:include filename="$(find o2as_scene_description)/urdf/dual_suction_gripper.urdf.xacro" />
   <xacro:dual_suction_gripper_o2as prefix="b_bot_" parent = "b_bot_ee_link">
     <origin xyz="0 0 0" rpy="0 0 0"/>
-  </xacro:dual_suction_gripper_o2as> -->
+  </xacro:dual_suction_gripper_o2as>
   <!-- spawn and attach dual robotiq 85 grippers -->
-  <xacro:include filename="$(find o2as_scene_description)/urdf/robotiq_b_bot_gripper.urdf.xacro" />
-  <xacro:o2as_b_bot_gripper prefix="b_bot_" parent = "b_bot_ee_link" />
+  <!-- <xacro:include filename="$(find o2as_scene_description)/urdf/robotiq_b_bot_gripper.urdf.xacro" /> -->
+  <!-- <xacro:o2as_b_bot_gripper prefix="b_bot_" parent = "b_bot_ee_link" /> -->
   <xacro:include filename="$(find o2as_scene_description)/urdf/robotiq_c_bot_gripper.urdf.xacro" />
   <xacro:o2as_c_bot_gripper prefix="c_bot_" parent = "c_bot_ee_link"/>
@@ -155,9 +155,9 @@
   <!--   <origin xyz="0.08 0.00 0.065" rpy="0 0 0"/> -->
   <!-- </xacro:o2as_ar_marker> -->
-  <!-- <xacro:o2as_ar_marker prefix="b_bot_" -->
-  <!-- 			parent="b_bot_dual_suction_gripper_base_link" -->
-  <!-- 			marker_id="26"> -->
-  <!--   <origin xyz="0.063 0.0 0.0215" rpy="0 0 0"/> -->
-  <!-- </xacro:o2as_ar_marker> -->
+  <xacro:o2as_ar_marker prefix="b_bot_"
+  			parent="b_bot_dual_suction_gripper_base_link"
+  			marker_id="26">
+    <origin xyz="0.063 0.0 0.0215" rpy="0 0 0"/>
+  </xacro:o2as_ar_marker>
   <!-- <xacro:o2as_ar_marker prefix="b_bot_" -->
   <!-- 			parent="b_bot_single_suction_gripper_base_link" -->
@@ -165,9 +165,9 @@
   <!--   <origin xyz="0.063 0.0 0.0215" rpy="0 0 0"/> -->
   <!-- </xacro:o2as_ar_marker> -->
-  <xacro:o2as_ar_marker prefix="b_bot_"
-			parent="b_bot_robotiq_85_tip_link"
-			marker_id="26">
-    <origin xyz="0.0 0.0 0.0185" rpy="0 0 0"/>
-  </xacro:o2as_ar_marker>
+  <!-- <xacro:o2as_ar_marker prefix="b_bot_" -->
+  <!-- 			parent="b_bot_robotiq_85_tip_link" -->
+  <!-- 			marker_id="26"> -->
+  <!--   <origin xyz="0.0 0.0 0.0185" rpy="0 0 0"/> -->
+  <!-- </xacro:o2as_ar_marker> -->
   <xacro:o2as_ar_marker prefix="c_bot_"
 			parent="c_bot_robotiq_85_tip_link"

Commit message: publish.py in o2as_easy_handeye now produces the <origin> entry for o2as_base_scene.urdf.xacro.

File: o2as_scene_description/urdf/o2as_base_scene.urdf.xacro (robot description, xacro)
@@ -197,6 +197,10 @@
     <!-- 	    rpy="${-149.604*pi/180} ${0.34821*pi/180} ${91.866*pi/180}"/> -->
     <!-- 181008@OSX -->
-    <origin xyz="0.674391 -0.0223742 ${bots_z + 0.696023}"
-	    rpy="${-149.801*pi/180} ${0.156861*pi/180} ${91.2544*pi/180}"/>
+    <!-- <origin xyz="0.674391 -0.0223742 ${bots_z + 0.696023}" -->
+    <!-- 	    rpy="${-149.801*pi/180} ${0.156861*pi/180} ${91.2544*pi/180}"/> -->
+    <!-- 181013@AIST -->
+    <origin xyz="0.620344080768 -0.0393922568732 1.44658358063"
+	    rpy="${-151.339295995*pi/180} ${1.39136148158*pi/180}
+		 ${86.8890568086*pi/180}"/>
   </xacro:phoxi_m_camera>
   <!-- I would like to remove the "world" link definition, but apparently it is necessary for Gazebo -->
