Commit message: Cleaning up.

File: o2as_scene_description/urdf/o2as_base_scene.urdf.xacro (robot description, xacro)
@@ -165,9 +165,9 @@
   <!--   <origin xyz="0.063 0.0 0.0215" rpy="0 0 0"/> -->
   <!-- </xacro:o2as_ar_marker> -->
-  <xacro:o2as_ar_marker prefix="b_bot_"
-  			parent="b_bot_robotiq_85_tip_link"
-  			marker_id="26">
-    <origin xyz="0.0 0.0 0.0185" rpy="0 0 0"/>
-  </xacro:o2as_ar_marker>
+  <!-- <xacro:o2as_ar_marker prefix="b_bot_" -->
+  <!-- 			parent="b_bot_robotiq_85_tip_link" -->
+  <!-- 			marker_id="26"> -->
+  <!--   <origin xyz="0.0 0.0 0.0185" rpy="0 0 0"/> -->
+  <!-- </xacro:o2as_ar_marker> -->
   <xacro:o2as_ar_marker prefix="c_bot_"
 			parent="c_bot_robotiq_85_tip_link"

Commit message: Fixed paramters by calibration.

File: o2as_scene_description/urdf/o2as_base_scene.urdf.xacro (robot description, xacro)
@@ -148,6 +148,6 @@
   <xacro:include filename="$(find o2as_scene_description)/urdf/phoxi_m_camera.urdf.xacro" />
   <xacro:phoxi_m_camera prefix="a_" parent="o2as_ground">
-    <origin xyz="0.674391 -0.0223742 ${bots_z + 0.696023}"
-	    rpy="${-149.801*pi/180} ${0.156861*pi/180} ${91.2544*pi/180}"/>
+  <origin xyz="0.656427245186 -0.0191234201169 1.50626196172"
+          rpy="${-161.285833025*pi/180} ${0.547979734685*pi/180} ${91.027298919*pi/180}"/>
   </xacro:phoxi_m_camera>
   <!-- I would like to remove the "world" link definition, but apparently it is necessary for Gazebo -->

Commit message: Fix feeder location

File: o2as_scene_description/urdf/o2as_base_scene.urdf.xacro (robot description, xacro)
@@ -110,8 +110,8 @@
   <xacro:include filename="$(find o2as_scene_description)/urdf/screw_feeder.xacro" />
   <xacro:screw_feeder feedername="m3_feeder" parent="c_bot_base_smfl">
-    <origin xyz=".66 -0.25 .065" rpy="0 0 ${pi/2}" />
+    <origin xyz=".64 -0.25 .035" rpy="0 0 ${pi/2}" />
   </xacro:screw_feeder>
   <xacro:screw_feeder feedername="m4_feeder" parent="c_bot_base_smfl">
-    <origin xyz=".52 -0.25 .065" rpy="0 0 ${pi/2}" />
+    <origin xyz=".50 -0.25 .035" rpy="0 0 ${pi/2}" />
   </xacro:screw_feeder>
   <!-- Add cameras -->

Commit message: Cleaning up.

File: o2as_scene_description/urdf/o2as_base_scene.urdf.xacro (robot description, xacro)
@@ -150,9 +150,9 @@
   <!-- spawn and attach AR markers -->
   <xacro:include filename="$(find o2as_gazebo)/urdf/o2as_ar_marker.urdf.xacro"/>
-  <!-- <xacro:o2as_ar_marker prefix="a_bot_" -->
-  <!-- 			parent="a_bot_ee_link" -->
-  <!-- 			marker_id="26"> -->
-  <!--   <origin xyz="0.08 0.00 0.065" rpy="0 0 0"/> -->
-  <!-- </xacro:o2as_ar_marker> -->
+  <xacro:o2as_ar_marker prefix="a_bot_"
+  			parent="a_bot_ee_link"
+  			marker_id="26">
+    <origin xyz="0.08 0.00 0.065" rpy="0 0 0"/>
+  </xacro:o2as_ar_marker>
   <!-- <xacro:o2as_ar_marker prefix="b_bot_" -->
   <!-- 			parent="b_bot_dual_suction_gripper_base_link" -->
@@ -170,17 +170,17 @@
   <!--   <origin xyz="0.0 0.0 0.0185" rpy="0 0 0"/> -->
   <!-- </xacro:o2as_ar_marker> -->
-  <xacro:o2as_ar_marker prefix="c_bot_"
-			parent="c_bot_robotiq_85_tip_link"
-			marker_id="26">
-    <origin xyz="0.0 0.0 0.0185" rpy="0 0 0"/>
-  </xacro:o2as_ar_marker>
-  <xacro:o2as_ar_marker_16cm prefix="workspace_"
-  			     parent="workspace_center"
-  			     marker_id="32">
-    <origin xyz="0.0 0.0 0.0005" rpy="0 0 0"/>
-  </xacro:o2as_ar_marker_16cm>
+  <!-- <xacro:o2as_ar_marker prefix="c_bot_" -->
+  <!-- 			parent="c_bot_robotiq_85_tip_link" -->
+  <!-- 			marker_id="26"> -->
+  <!--   <origin xyz="0.0 0.0 0.0185" rpy="0 0 0"/> -->
+  <!-- </xacro:o2as_ar_marker> -->
+  <!-- <xacro:o2as_ar_marker_16cm prefix="workspace_" -->
+  <!-- 			     parent="workspace_center" -->
+  <!-- 			     marker_id="32"> -->
+  <!--   <origin xyz="0.0 0.0 0.0005" rpy="0 0 0"/> -->
+  <!-- </xacro:o2as_ar_marker_16cm> -->
   <!-- <xacro:o2as_ar_marker prefix="workspace_" -->
   <!-- 			parent="workspace_center" -->
-  <!-- 			marker_id="26"> -->
+  <!-- 			marker_id="32"> -->
   <!--   <origin xyz="0.0 0.0 0.0005" rpy="0 0 0"/> -->
   <!-- </xacro:o2as_ar_marker> -->
@@ -200,7 +200,10 @@
     <!-- 	    rpy="${-149.801*pi/180} ${0.156861*pi/180} ${91.2544*pi/180}"/> -->
     <!-- 181013@AIST -->
-    <origin xyz="0.620344080768 -0.0393922568732 1.44658358063"
-	    rpy="${-151.339295995*pi/180} ${1.39136148158*pi/180}
-		 ${86.8890568086*pi/180}"/>
+    <!-- <origin xyz="0.620344080768 -0.0393922568732 1.44658358063" -->
+    <!-- 	    rpy="${-151.339295995*pi/180} ${1.39136148158*pi/180} -->
+    <!-- 		 ${86.8890568086*pi/180}"/> -->
+    <origin xyz="0.656427245186 -0.0191234201169 1.50626196172"
+	    rpy="${-161.285833025*pi/180} ${0.547979734685*pi/180}
+		 ${91.027298919*pi/180}"/>
   </xacro:phoxi_m_camera>
   <!-- I would like to remove the "world" link definition, but apparently it is necessary for Gazebo -->

Commit message: Dump commit before taskboard round 1
Not working: Part 7

File: o2as_scene_description/urdf/o2as_base_scene.urdf.xacro (robot description, xacro)
@@ -21,5 +21,5 @@
   <xacro:include filename="$(find o2as_scene_description)/urdf/ur3.urdf.xacro" />
   <!-- Scene items (trays, bins...) -->
-  <xacro:include filename="$(find o2as_scene_description)/urdf/taskboard_scene.xacro" />
+  <xacro:include filename="$(find o2as_scene_description)/urdf/taskboar d_scene.xacro" />
   <!-- <xacro:include filename="$(find o2as_scene_description)/urdf/kitting_scene.xacro" /> -->
   <!-- <xacro:include filename="$(find o2as_scene_description)/urdf/assembly_scene.xacro" /> -->

File: o2as_scene_description/urdf/taskboard_scene.xacro (robot description, xacro)
@@ -18,5 +18,5 @@
     <parent link="workspace_center"/>
     <child link="belt_placement_tool"/>
-    <origin rpy="0.0 0.0 0" xyz="-.2 0.37 0"/>
+    <origin rpy="0.0 0.0 0" xyz="-.23 0.34 0"/>
   </joint>
   <link name="belt_placement_tool"/>

Commit message: State of taskboard trial 1

File: o2as_scene_description/urdf/o2as_base_scene.urdf.xacro (robot description, xacro)
@@ -21,5 +21,5 @@
   <xacro:include filename="$(find o2as_scene_description)/urdf/ur3.urdf.xacro" />
   <!-- Scene items (trays, bins...) -->
-  <xacro:include filename="$(find o2as_scene_description)/urdf/taskboar d_scene.xacro" />
+  <xacro:include filename="$(find o2as_scene_description)/urdf/taskboard_scene.xacro" />
   <!-- <xacro:include filename="$(find o2as_scene_description)/urdf/kitting_scene.xacro" /> -->
   <!-- <xacro:include filename="$(find o2as_scene_description)/urdf/assembly_scene.xacro" /> -->

File: o2as_scene_description/urdf/o2as_mat.xacro (robot description, xacro)
@@ -76,5 +76,5 @@
       <parent link="${matname}"/>
       <child link="${matname}_part1"/>
-      <origin rpy="0.0 0.0 ${pi/2}" xyz="0.074 0.2865 0.0"/>
+      <origin rpy="0.0 0.0 ${pi/2}" xyz="0.193 0.22 0.0"/>
     </joint>
     <link name="${matname}_part1"/>
@@ -82,5 +82,5 @@
       <parent link="${matname}"/>
       <child link="${matname}_part2"/>
-      <origin rpy="0.0 0.0 ${pi/2}" xyz="0.175 0.3325 0.0"/>
+      <origin rpy="0.0 0.0 ${pi/2}" xyz="0.351 0.213 0.0"/>
     </joint>
     <link name="${matname}_part2"/>
@@ -88,5 +88,5 @@
       <parent link="${matname}"/>
       <child link="${matname}_part3"/>
-      <origin rpy="0.0 0.0 ${pi/2}" xyz="0.2625 0.324 0.0"/>
+      <origin rpy="0.0 0.0 ${pi/2}" xyz="0.14 0.135 0.0"/>
     </joint>
     <link name="${matname}_part3"/>
@@ -94,5 +94,5 @@
       <parent link="${matname}"/>
       <child link="${matname}_part4"/>
-      <origin rpy="0.0 0.0 ${pi/2}" xyz="0.3445 0.324 0.0"/>
+      <origin rpy="0.0 0.0 ${pi/2}" xyz="0.052 0.306 0.0"/>
     </joint>
     <link name="${matname}_part4"/>
@@ -106,5 +106,5 @@
       <parent link="${matname}"/>
       <child link="${matname}_part6"/>
-      <origin rpy="0.0 0.0 ${pi/2}" xyz="0.205 0.205 0.0"/>
+      <origin rpy="0.0 0.0 ${pi/2}" xyz="0.275 0.1 0.0"/>
     </joint>
     <link name="${matname}_part6"/>
@@ -112,5 +112,5 @@
       <parent link="${matname}"/>
       <child link="${matname}_part7_1"/>
-      <origin rpy="0.0 0.0 ${pi/2}" xyz="0.327 0.164 0.0"/>
+      <origin rpy="0.0 0.0 ${pi/2}" xyz="0.276 0.324 0.0"/>
     </joint>
     <link name="${matname}_part7_1"/>
@@ -118,5 +118,5 @@
       <parent link="${matname}"/>
       <child link="${matname}_part7_2"/>
-      <origin rpy="0.0 0.0 ${pi/2}" xyz="0.328 0.236 0.0"/>
+      <origin rpy="0.0 0.0 ${pi/2}" xyz="0.347 0.323 0.0"/>
     </joint>
     <link name="${matname}_part7_2"/>
@@ -124,5 +124,5 @@
       <parent link="${matname}"/>
       <child link="${matname}_part8"/>
-      <origin rpy="0.0 0.0 ${pi/2}" xyz="0.079 0.117 0.0"/>
+      <origin rpy="0.0 0.0 ${pi/2}" xyz="0.126 0.0525 0.0"/>
     </joint>
     <link name="${matname}_part8"/>
@@ -130,5 +130,5 @@
       <parent link="${matname}"/>
       <child link="${matname}_part9"/>
-      <origin rpy="0.0 0.0 ${pi/2}" xyz="0.1555 0.0955 0.0"/>
+      <origin rpy="0.0 0.0 ${pi/2}" xyz="0.077 0.231 0.0"/>
     </joint>
     <link name="${matname}_part9"/>
@@ -136,5 +136,5 @@
       <parent link="${matname}"/>
       <child link="${matname}_part10"/>
-      <origin rpy="0.0 0.0 ${pi/2}" xyz="0.257 0.1075 0.0"/>
+      <origin rpy="0.0 0.0 ${pi/2}" xyz="0.293 0.248 0.0"/>
     </joint>
     <link name="${matname}_part10"/>
@@ -148,5 +148,5 @@
       <parent link="${matname}"/>
       <child link="${matname}_part12"/>
-      <origin rpy="0.0 0.0 ${pi/2}" xyz="0.06 0.048 0.0"/>
+      <origin rpy="0.0 0.0 ${pi/2}" xyz="0.214 0.348 0.0"/>
     </joint>
     <link name="${matname}_part12"/>
@@ -154,5 +154,5 @@
       <parent link="${matname}"/>
       <child link="${matname}_part13"/>
-      <origin rpy="0.0 0.0 ${pi/2}" xyz="0.145 0.042 0.0"/>
+      <origin rpy="0.0 0.0 ${pi/2}" xyz="0.164 0.049 0.0"/>
     </joint>
     <link name="${matname}_part13"/>
@@ -160,5 +160,5 @@
       <parent link="${matname}"/>
       <child link="${matname}_part14"/>
-      <origin rpy="0.0 0.0 ${pi/2}" xyz="0.25 0.0465 0.0"/>
+      <origin rpy="0.0 0.0 ${pi/2}" xyz="0.345 0.106 0.0"/>
     </joint>
     <link name="${matname}_part14"/>
@@ -166,5 +166,5 @@
       <parent link="${matname}"/>
       <child link="${matname}_part15"/>
-      <origin rpy="0.0 0.0 ${pi/2}" xyz="0.3475 0.0525 0.0"/>
+      <origin rpy="0.0 0.0 ${pi/2}" xyz="0.0495 0.069 0.0"/>
     </joint>
     <link name="${matname}_part15"/>

File: o2as_scene_description/urdf/task_board.xacro (robot description, xacro)
@@ -63,5 +63,5 @@
     <parent link="${boardname}_surface"/>
     <child link="${boardname}_part1"/>
-    <origin rpy="0.0 0.0 ${pi*0.5}" xyz="0.34 0.06 0.0"/>
+    <origin rpy="0.0 0.0 ${pi*0.5}" xyz="0.33 0.07 0.0"/>
   </joint>
   <link name="${boardname}_part1"/>
@@ -69,5 +69,5 @@
     <parent link="${boardname}_surface"/>
     <child link="${boardname}_part2"/>
-    <origin rpy="0.0 0.0 ${pi*0.5}" xyz="0.35 0.35 0.0"/>
+    <origin rpy="0.0 0.0 ${pi*0.5}" xyz="0.36 0.34 0.0"/>
   </joint>
   <link name="${boardname}_part2"/>
@@ -75,5 +75,5 @@
     <parent link="${boardname}_surface"/>
     <child link="${boardname}_part3"/>
-    <origin rpy="0.0 0.0 ${pi*0.5}" xyz="0.31 0.32 0.0"/>
+    <origin rpy="0.0 0.0 ${pi*0.5}" xyz="0.3 0.31 0.0"/>
   </joint>
   <link name="${boardname}_part3"/>
@@ -81,5 +81,5 @@
     <parent link="${boardname}_surface"/>
     <child link="${boardname}_part4"/>
-    <origin rpy="0.0 0.0 ${pi*0.5}" xyz="0.28 0.25 0.0"/>
+    <origin rpy="0.0 0.0 ${pi*0.5}" xyz="0.27 0.24 0.0"/>
   </joint>
   <link name="${boardname}_part4"/>
@@ -87,5 +87,5 @@
     <parent link="${boardname}_surface"/>
     <child link="${boardname}_part5"/>
-    <origin rpy="0.0 0.0 ${pi*0.5}" xyz="0.26 0.33 0.002"/>
+    <origin rpy="0.0 0.0 ${pi*0.5}" xyz="0.25 0.35 0.002"/>
   </joint>
   <link name="${boardname}_part5">
@@ -103,5 +103,5 @@
     <parent link="${boardname}_surface"/>
     <child link="${boardname}_part15"/>
-    <origin rpy="0.0 0.0 ${pi*0.5}" xyz="0.26 0.33 0.0772"/>
+    <origin rpy="0.0 0.0 ${pi*0.5}" xyz="0.25 0.35 0.0772"/>
   </joint>
   <link name="${boardname}_part15"/>
@@ -109,5 +109,5 @@
     <parent link="${boardname}_surface"/>
     <child link="${boardname}_part6_small_pulley"/>
-    <origin rpy="0.0 0.0 ${pi*0.0}" xyz="0.06 0.34 0.0085"/>
+    <origin rpy="0.0 0.0 ${pi*0.0}" xyz="0.07 0.34 0.0085"/>
   </joint>
   <link name="${boardname}_part6_small_pulley">
@@ -125,5 +125,5 @@
     <parent link="${boardname}_surface"/>
     <child link="${boardname}_part7_1"/>
-    <origin rpy="0.0 0.0 ${pi*1.5}" xyz="0.056 0.039 0.0505"/>
+    <origin rpy="0.0 0.0 ${pi*-0.5}" xyz="0.056 0.049 0.0505"/>
   </joint>
   <link name="${boardname}_part7_1"/>
@@ -131,5 +131,5 @@
     <parent link="${boardname}_surface"/>
     <child link="${boardname}_part8"/>
-    <origin rpy="0.0 0.0 ${pi*0.5}" xyz="0.25 0.08 0.012"/>
+    <origin rpy="0.0 0.0 ${pi*0.5}" xyz="0.24 0.08 0.012"/>
   </joint>
   <link name="${boardname}_part8">
@@ -147,5 +147,5 @@
     <parent link="${boardname}_surface"/>
     <child link="${boardname}_part9"/>
-    <origin rpy="0.0 0.0 ${pi*0.5}" xyz="0.15 0.14 0.009"/>
+    <origin rpy="0.0 0.0 ${pi*0.5}" xyz="0.13 0.12 0.009"/>
   </joint>
   <link name="${boardname}_part9">
@@ -163,5 +163,5 @@
     <parent link="${boardname}_surface"/>
     <child link="${boardname}_part10"/>
-    <origin rpy="0.0 0.0 ${pi*0.5}" xyz="0.36 0.24 0.0515"/>
+    <origin rpy="0.0 0.0 ${pi*0.5}" xyz="0.34 0.21 0.0515"/>
   </joint>
   <link name="${boardname}_part10">
@@ -179,5 +179,5 @@
     <parent link="${boardname}_surface"/>
     <child link="${boardname}_part11"/>
-    <origin rpy="0.0 0.0 ${pi*0.5}" xyz="0.18 0.34 0.0"/>
+    <origin rpy="0.0 0.0 ${pi*0.5}" xyz="0.17 0.33 0.0"/>
   </joint>
   <link name="${boardname}_part11"/>
@@ -185,5 +185,5 @@
     <parent link="${boardname}_surface"/>
     <child link="${boardname}_part12"/>
-    <origin rpy="${pi*-0.5} ${pi*0.5} ${pi*0.}" xyz="0.14 0.26 0.0"/>
+    <origin rpy="${pi*-0.5} ${pi*0.5} ${pi*0.}" xyz="0.15 0.25 0.0"/>
   </joint>
   <link name="${boardname}_part12"/>
@@ -191,5 +191,5 @@
     <parent link="${boardname}_surface"/>
     <child link="${boardname}_part13"/>
-    <origin rpy="${pi*-0.5} ${pi*0.5} ${pi*0.}" xyz="0.26 0.33 0.078"/>
+    <origin rpy="${pi*-0.5} ${pi*0.5} ${pi*0.}" xyz="0.25 0.35 0.078"/>
   </joint>
   <link name="${boardname}_part13"/>
@@ -197,5 +197,5 @@
     <parent link="${boardname}_surface"/>
     <child link="${boardname}_part14"/>
-    <origin rpy="0.0 0.0 ${pi*0.5}" xyz="0.23 0.17 0.0515"/>
+    <origin rpy="0.0 0.0 ${pi*0.5}" xyz="0.22 0.18 0.0515"/>
   </joint>
   <link name="${boardname}_part14">

Commit message: Cleaning up.

File: o2as_scene_description/urdf/o2as_base_scene.urdf.xacro (robot description, xacro)
@@ -165,19 +165,19 @@
   <!--   <origin xyz="0.063 0.0 0.0215" rpy="0 0 0"/> -->
   <!-- </xacro:o2as_ar_marker> -->
-  <!-- <xacro:o2as_ar_marker prefix="b_bot_" -->
-  <!-- 			parent="b_bot_robotiq_85_tip_link" -->
-  <!-- 			marker_id="26"> -->
-  <!--   <origin xyz="0.0 0.0 0.0185" rpy="0 0 0"/> -->
-  <!-- </xacro:o2as_ar_marker> -->
-  <!-- <xacro:o2as_ar_marker prefix="c_bot_" -->
-  <!-- 			parent="c_bot_robotiq_85_tip_link" -->
-  <!-- 			marker_id="26"> -->
-  <!--   <origin xyz="0.0 0.0 0.0185" rpy="0 0 0"/> -->
-  <!-- </xacro:o2as_ar_marker> -->
-  <!-- <xacro:o2as_ar_marker_16cm prefix="workspace_" -->
-  <!-- 			     parent="workspace_center" -->
-  <!-- 			     marker_id="32"> -->
-  <!--   <origin xyz="0.0 0.0 0.0005" rpy="0 0 0"/> -->
-  <!-- </xacro:o2as_ar_marker_16cm> -->
+  <xacro:o2as_ar_marker prefix="b_bot_"
+  			parent="b_bot_robotiq_85_tip_link"
+  			marker_id="26">
+    <origin xyz="0.0 0.0 0.0185" rpy="0 0 0"/>
+  </xacro:o2as_ar_marker>
+  <xacro:o2as_ar_marker prefix="c_bot_"
+  			parent="c_bot_robotiq_85_tip_link"
+  			marker_id="26">
+    <origin xyz="0.0 0.0 0.0185" rpy="0 0 0"/>
+  </xacro:o2as_ar_marker>
+  <xacro:o2as_ar_marker_16cm prefix="workspace_"
+  			     parent="workspace_center"
+  			     marker_id="32">
+    <origin xyz="0.0 0.0 0.0005" rpy="0 0 0"/>
+  </xacro:o2as_ar_marker_16cm>
   <!-- <xacro:o2as_ar_marker prefix="workspace_" -->
   <!-- 			parent="workspace_center" -->

Commit message: Improved calibration script.

File: o2as_scene_description/urdf/o2as_base_scene.urdf.xacro (robot description, xacro)
@@ -119,7 +119,11 @@
   <!--   <origin xyz="0 0 0" rpy="0 0 0"/> -->
   <!-- </xacro:dual_suction_gripper_o2as> -->
+  <xacro:include filename="$(find o2as_scene_description)/urdf/single_suction_gripper.urdf.xacro" />
+  <xacro:single_suction_gripper_o2as prefix="b_bot_" parent = "b_bot_ee_link">
+    <origin xyz="0 0 0" rpy="0 0 0"/>
+  </xacro:single_suction_gripper_o2as>
   <!-- spawn and attach dual robotiq 85 grippers -->
-  <xacro:include filename="$(find o2as_scene_description)/urdf/robotiq_b_bot_gripper.urdf.xacro" />
-  <xacro:o2as_b_bot_gripper prefix="b_bot_" parent = "b_bot_ee_link" />
+  <!-- <xacro:include filename="$(find o2as_scene_description)/urdf/robotiq_b_bot_gripper.urdf.xacro" /> -->
+  <!-- <xacro:o2as_b_bot_gripper prefix="b_bot_" parent = "b_bot_ee_link" /> -->
   <xacro:include filename="$(find o2as_scene_description)/urdf/robotiq_c_bot_gripper.urdf.xacro" />
   <xacro:o2as_c_bot_gripper prefix="c_bot_" parent = "c_bot_ee_link"/>
@@ -160,9 +164,9 @@
   <!--   <origin xyz="0.063 0.0 0.0215" rpy="0 0 0"/> -->
   <!-- </xacro:o2as_ar_marker> -->
-  <!-- <xacro:o2as_ar_marker prefix="b_bot_" -->
-  <!-- 			parent="b_bot_single_suction_gripper_base_link" -->
-  <!-- 			marker_id="26"> -->
-  <!--   <origin xyz="0.063 0.0 0.0215" rpy="0 0 0"/> -->
-  <!-- </xacro:o2as_ar_marker> -->
+  <xacro:o2as_ar_marker prefix="b_bot_"
+  			parent="b_bot_ee_link"
+  			marker_id="26">
+    <origin xyz="0.063 0.0 0.0215" rpy="0 0 0"/>
+  </xacro:o2as_ar_marker>
   <!-- <xacro:o2as_ar_marker prefix="b_bot_" -->
   <!-- 			parent="b_bot_robotiq_85_tip_link" -->
@@ -170,19 +174,14 @@
   <!--   <origin xyz="0.0 0.0 0.0185" rpy="0 0 0"/> -->
   <!-- </xacro:o2as_ar_marker> -->
-  <!-- <xacro:o2as_ar_marker prefix="c_bot_" -->
-  <!-- 			parent="c_bot_robotiq_85_tip_link" -->
-  <!-- 			marker_id="26"> -->
-  <!--   <origin xyz="0.0 0.0 0.0185" rpy="0 0 0"/> -->
-  <!-- </xacro:o2as_ar_marker> -->
-  <!-- <xacro:o2as_ar_marker_16cm prefix="workspace_" -->
-  <!-- 			     parent="workspace_center" -->
-  <!-- 			     marker_id="32"> -->
-  <!--   <origin xyz="0.0 0.0 0.0005" rpy="0 0 0"/> -->
-  <!-- </xacro:o2as_ar_marker_16cm> -->
-  <!-- <xacro:o2as_ar_marker prefix="workspace_" -->
-  <!-- 			parent="workspace_center" -->
-  <!-- 			marker_id="32"> -->
-  <!--   <origin xyz="0.0 0.0 0.0005" rpy="0 0 0"/> -->
-  <!-- </xacro:o2as_ar_marker> -->
+  <xacro:o2as_ar_marker prefix="c_bot_"
+  			parent="c_bot_robotiq_85_tip_link"
+  			marker_id="26">
+    <origin xyz="0.0 0.0 0.0185" rpy="0 0 0"/>
+  </xacro:o2as_ar_marker>
+  <xacro:o2as_ar_marker_16cm prefix="workspace_"
+  			     parent="workspace_center"
+  			     marker_id="32">
+    <origin xyz="0.0 0.0 0.0005" rpy="0 0 0"/>
+  </xacro:o2as_ar_marker_16cm>
   <!-- Add PhoXi 3D scanners -->
   <xacro:include filename="$(find o2as_scene_description)/urdf/phoxi_m_camera.urdf.xacro" />

Commit message: Redesign robot trajectory for calibration.

File: o2as_scene_description/urdf/o2as_base_scene.urdf.xacro (robot description, xacro)
@@ -137,13 +137,4 @@
     <origin xyz="0 0 0" rpy="0 0 0"/>
   </xacro:sensor_d435>
-  <link name="a_bot_camera_calibrated_frame_link" />
-  <joint name="a_bot_camera_calibrated_frame_joint" type="fixed">
-    <parent link="a_bot_wrist_2_link" />
-    <child  link="a_bot_camera_calibrated_frame_link" />
-    <origin xyz="-0.00584875065097 -0.0601140904909 0.190359410313" rpy="-1.631 -0.020 -0.016" />
-  </joint>
-  <!-- <xacro:sensor_d435 prefix="d_bot_" parent="o2as_ground">
-    <origin xyz="0 0 ${bots_z + 0.9}" rpy="0 ${pi/2} 0"/>
-  </xacro:sensor_d435> -->
   <!-- Add PhoXi 3D scanners -->
   <xacro:include filename="$(find o2as_scene_description)/urdf/phoxi_m_camera.urdf.xacro" />

Commit message: Display quantitative planarity in plane_deteoctor.

File: o2as_scene_description/urdf/o2as_base_scene.urdf.xacro (robot description, xacro)
@@ -103,7 +103,10 @@
     <origin xyz="0.0 0 0.0" rpy="0 0 0"/>
   </xacro:InnerOnlyGripper>
+  <xacro:include filename="$(find o2as_scene_description)/urdf/dual_suction_gripper.urdf.xacro"/>
+  <xacro:dual_suction_gripper_o2as prefix="b_bot_" parent="b_bot_ee_link">
+    <origin xyz="0 0 0" rpy="0 0 0" />
+  </xacro:dual_suction_gripper_o2as>
   <!-- spawn and attach dual robotiq 85 grippers -->
-  <xacro:include filename="$(find o2as_scene_description)/urdf/robotiq_b_bot_gripper.urdf.xacro" />
-  <xacro:o2as_b_bot_gripper prefix="b_bot_" parent = "b_bot_ee_link" />
+  <!-- <xacro:o2as_b_bot_gripper prefix="b_bot_" parent = "b_bot_ee_link" /> -->
   <xacro:include filename="$(find o2as_scene_description)/urdf/robotiq_c_bot_gripper.urdf.xacro" />
   <xacro:o2as_c_bot_gripper prefix="c_bot_" parent = "c_bot_ee_link"/>
@@ -149,9 +152,9 @@
     <origin xyz="0.08 0.00 0.065" rpy="0 0 0"/>
   </xacro:o2as_ar_marker>
-  <!-- <xacro:o2as_ar_marker prefix="b_bot_" -->
-  <!-- 			parent="b_bot_dual_suction_gripper_base_link" -->
-  <!-- 			marker_id="26"> -->
-  <!--   <origin xyz="0.063 0.0 0.0215" rpy="0 0 0"/> -->
-  <!-- </xacro:o2as_ar_marker> -->
+  <xacro:o2as_ar_marker prefix="b_bot_"
+  			parent="b_bot_dual_suction_gripper_base_link"
+  			marker_id="26">
+    <origin xyz="0.063 0.0 0.0215" rpy="0 0 0"/>
+  </xacro:o2as_ar_marker>
   <!-- <xacro:o2as_ar_marker prefix="b_bot_" -->
   <!-- 			parent="b_bot_single_suction_gripper_base_link" -->
@@ -159,9 +162,9 @@
   <!--   <origin xyz="0.063 0.0 0.0215" rpy="0 0 0"/> -->
   <!-- </xacro:o2as_ar_marker> -->
-  <xacro:o2as_ar_marker prefix="b_bot_"
-  			parent="b_bot_robotiq_85_tip_link"
-  			marker_id="26">
-    <origin xyz="0.0 0.0 0.0185" rpy="0 0 0"/>
-  </xacro:o2as_ar_marker>
+  <!-- <xacro:o2as_ar_marker prefix="b_bot_" -->
+  <!-- 			parent="b_bot_robotiq_85_tip_link" -->
+  <!-- 			marker_id="26"> -->
+  <!--   <origin xyz="0.0 0.0 0.0185" rpy="0 0 0"/> -->
+  <!-- </xacro:o2as_ar_marker> -->
   <xacro:o2as_ar_marker prefix="c_bot_"
 			parent="c_bot_robotiq_85_tip_link"
