Commit message: Confirmed that aist_ftsensor works on UR5e.

File: o2as_scene_description/urdf/ur5e.urdf.xacro (robot description, xacro)
@@ -311,4 +311,10 @@
       <child link="${prefix}tool0"/>
     </joint>
+    <link name="${prefix}wrench_link"/>
+    <joint name="${prefix}wrench_joint" type="fixed">
+      <parent link="${prefix}ee_link"/>
+      <child  link="${prefix}wrench_link"/>
+      <origin xyz="0 0 0" rpy="${-pi/2} 0 ${pi/2}"/>
+    </joint>
   </xacro:macro>
 </robot>
