Commit message: o2as_usb_relay now supports IWT303 USB relay module.

File: o2as_scene_description/urdf/dual_suction_gripper.urdf.xacro (robot description, xacro)
@@ -19,6 +19,5 @@
       <parent link="${parent}"/>
       <child  link="${prefix}dual_suction_gripper_base_link"/>
-      <child  link="base_link"/>
-      <xacro:insert_block name="origin"/>
+       <xacro:insert_block name="origin"/>
     </joint>
   </xacro:macro>

Commit message: Add collision information to dual_suction_gripper and kitting trays with partitions.

File: o2as_scene_description/urdf/dual_suction_gripper.urdf.xacro (robot description, xacro)
@@ -7,4 +7,5 @@
       <color rgba="0.8 0.8 0.8 1"/>
     </material>
+    <!-- A link representing the gripper and a joint attaching it to parnet -->
     <link name="${prefix}dual_suction_gripper_base_link">
       <visual>
@@ -15,4 +16,15 @@
 	<material name="light_grey"/>
       </visual>
+      <collision>
+	<geometry>
+	  <mesh
+	      filename="package://o2as_scene_description/meshes/dual_suction_gripper.vhacd.dae"/>
+	</geometry>
+      </collision>
+      <inertial>
+	  <mass value="0.3"/>
+	  <inertia ixx="0.4" ixy="0.0" ixz="0.0" iyy="0.4"
+		   iyz="0.0" izz ="0.2"/>
+      </inertial>
     </link>
     <joint name="${prefix}dual_suction_gripper_joint" type="fixed">
@@ -21,4 +33,20 @@
        <xacro:insert_block name="origin"/>
     </joint>
+    <!-- A link representing the tip of the pad and a joint attaching
+	 it to the gripper -->
+    <link name="${prefix}dual_suction_gripper_pad_link"/>
+    <joint name="${prefix}dual_suction_gripper_pad_joint" type="fixed">
+      <parent link="${prefix}dual_suction_gripper_base_link"/>
+      <child  link="${prefix}dual_suction_gripper_pad_link"/>
+      <origin xyz="0.187 0 0" rpy="0 0 0"/>
+    </joint>
+    <!-- A link representing the tip of the coander gripper
+	 and a joint attaching it to the gripper -->
+    <link name="${prefix}dual_suction_gripper_coanda_link"/>
+    <joint name="${prefix}dual_suction_gripper_coanda_joint" type="fixed">
+      <parent link="${prefix}dual_suction_gripper_base_link"/>
+      <child  link="${prefix}dual_suction_gripper_coanda_link"/>
+      <origin xyz="0.0505 0.145 0" rpy="0 0 ${pi/2}"/>
+    </joint>
   </xacro:macro>
 </robot>

File: o2as_scene_description/urdf/kitting_scene.xacro (robot description, xacro)
@@ -3,6 +3,5 @@
   <xacro:include filename="$(find o2as_scene_description)/urdf/kitting_bins.xacro" />
   <!-- <xacro:include filename="$(find o2as_scene_description)/urdf/kitting_tray.xacro" /> -->
-  <xacro:include filename="$(find o2as_scene_description)/urdf/kitting_tray1.xacro" />
-  <xacro:include filename="$(find o2as_scene_description)/urdf/kitting_tray2.xacro" />
+  <xacro:include filename="$(find o2as_scene_description)/urdf/kitting_tray_with_partitions.xacro" />
   <xacro:property name="bin1_width" value=".125"/>
   <xacro:property name="bin1_length" value=".128" />

File: o2as_scene_description/urdf/o2as_base_scene.urdf.xacro (robot description, xacro)
@@ -118,5 +118,5 @@
   <joint name="b_bot_cam_holder_joint" type="fixed">
     <parent link="b_bot_wrist_2_link" />
-    <child link = "b_bot_cam_holder_link" />
+    <child  link="b_bot_cam_holder_link" />
     <origin xyz="0.0 -0.06 0.16" rpy="0.0 0.0 ${pi/2}" />
   </joint>
@@ -124,4 +124,13 @@
     <origin xyz="0 0 0" rpy="0 0 0"/>
   </xacro:sensor_d435>
+  <!-- <link name="d_bot_cam_holder_link" /> -->
+  <!-- <joint name="d_bot_cam_holder_joint" type="fixed"> -->
+  <!--   <parent link="o2as_ground" /> -->
+  <!--   <child  link="d_bot_cam_holder_link" /> -->
+  <!--   <origin xyz="0.0 0.0 2.0" rpy="0.0 ${pi/2} 0.0" /> -->
+  <!-- </joint> -->
+  <!-- <xacro:sensor_d435 prefix="d_bot_" parent="d_bot_cam_holder_link"> -->
+  <!--   <origin xyz="0 0 0" rpy="0 0 0"/> -->
+  <!-- </xacro:sensor_d435> -->
   <!-- spawn and attach AR marker -->
   <xacro:include filename="$(find o2as_gazebo)/urdf/o2as_ar_marker.urdf.xacro"/>

File: o2as_scene_description/urdf/phoxi_m_camera.urdf.xacro (robot description, xacro)
@@ -2,8 +2,4 @@
 <robot name="phoxi_m_camera_o2as" xmlns:xacro="http://ros.org/wiki/xacro">
   <xacro:macro name="phoxi_m_camera_o2as" params="prefix parent *origin">
-    <!-- <gazebo> -->
-    <!--   <static>true</static> -->
-    <!-- </gazebo> -->
-    <!-- <xacro:include filename="$(find o2as_gazebo)/urdf/phoxi_m_camera.gazebo"/> -->
     <xacro:include filename="$(find o2as_phoxi_camera)/urdf/PhoXi3Dscanner_values.xacro"/>
     <xacro:include filename="$(find o2as_phoxi_camera)/urdf/PhoXi3Dscanner_macro.xacro"/>
@@ -16,4 +12,8 @@
       <xacro:PhoXi3DscannerM_meshes />
     </xacro:PhoXi3Dscanner>
+    <!-- <gazebo> -->
+    <!--   <static>true</static> -->
+    <!-- </gazebo> -->
+    <!-- <xacro:include filename="$(find o2as_gazebo)/urdf/${prefix}phoxi_m_camera.gazebo"/> -->
   </xacro:macro>
 </robot>

Commit message: Improve xacro descriptions of dual_suction_gripper for supporting multiple instances.

File: o2as_scene_description/urdf/dual_suction_gripper.urdf.xacro (robot description, xacro)
@@ -4,7 +4,4 @@
   <xacro:macro name="dual_suction_gripper_o2as"
 	       params="prefix parent *origin">
-    <material name="light_grey">
-      <color rgba="0.8 0.8 0.8 1"/>
-    </material>
     <!-- A link representing the gripper and a joint attaching it to parnet -->
     <link name="${prefix}dual_suction_gripper_base_link">
@@ -14,5 +11,7 @@
           <mesh filename="package://o2as_scene_description/meshes/dual_suction_gripper.stl"/>
 	</geometry>
-	<material name="light_grey"/>
+	<material name="light_grey">
+	  <color rgba="0.8 0.8 0.8 1"/>
+	</material>
       </visual>
       <collision>

File: o2as_scene_description/urdf/o2as_base_scene.urdf.xacro (robot description, xacro)
@@ -107,21 +107,25 @@
   </xacro:precision_gripper>
   <xacro:include filename="$(find o2as_scene_description)/urdf/robotiq_85_gripper_with_ft300.urdf.xacro" />
-  <xacro:robotiq_85_gripper_o2as prefix="b_bot_" parent = "b_bot_ee_link" />
+  <!-- <xacro:robotiq_85_gripper_o2as prefix="b_bot_" parent = "b_bot_ee_link" /> -->
   <xacro:robotiq_85_gripper_o2as prefix="c_bot_" parent = "c_bot_ee_link"/>
   <!-- spawn and attach dual suction grippers -->
-  <!-- <xacro:include filename="$(find o2as_scene_description)/urdf/dual_suction_gripper.urdf.xacro" /> -->
-  <!-- <xacro:dual_suction_gripper_o2as prefix="b_bot_" parent = "b_bot_ee_link"> -->
+  <xacro:include filename="$(find o2as_scene_description)/urdf/dual_suction_gripper.urdf.xacro" />
+  <xacro:dual_suction_gripper_o2as prefix="b_bot_" parent = "b_bot_ee_link">
+    <origin xyz="0 0 0" rpy="0 0 0"/>
+  </xacro:dual_suction_gripper_o2as>
+  <!-- Add cameras -->
+  <!-- <link name="b_bot_cam_holder_link" /> -->
+  <!-- <joint name="b_bot_cam_holder_joint" type="fixed"> -->
+  <!--   <parent link="b_bot_wrist_2_link" /> -->
+  <!--   <child  link="b_bot_cam_holder_link" /> -->
+  <!--   <origin xyz="0.0 -0.06 0.16" rpy="0.0 0.0 ${pi/2}" /> -->
+  <!-- </joint> -->
+  <!-- <xacro:sensor_d435 prefix="b_bot_" parent="b_bot_cam_holder_link"> -->
   <!--   <origin xyz="0 0 0" rpy="0 0 0"/> -->
-  <!-- </xacro:dual_suction_gripper_o2as> -->
-  <!-- Add cameras -->
-  <link name="b_bot_cam_holder_link" />
-  <joint name="b_bot_cam_holder_joint" type="fixed">
-    <parent link="b_bot_wrist_2_link" />
-    <child  link="b_bot_cam_holder_link" />
-    <origin xyz="0.0 -0.06 0.16" rpy="0.0 0.0 ${pi/2}" />
-  </joint>
-  <xacro:sensor_d435 prefix="b_bot_" parent="b_bot_cam_holder_link">
-    <origin xyz="0 0 0" rpy="0 0 0"/>
-  </xacro:sensor_d435>
+  <!-- </xacro:sensor_d435> -->
+  <xacro:include filename="$(find o2as_scene_description)/urdf/d435_camera.urdf.xacro"/>
+  <xacro:d435_camera prefix="d_bot_" parent="o2as_ground">
+    <origin xyz="0 0 ${bots_z + 0.9}" rpy="0 ${pi/2} 0"/>
+  </xacro:d435_camera>
   <!-- <link name="d_bot_cam_holder_link" /> -->
   <!-- <joint name="d_bot_cam_holder_joint" type="fixed"> -->

File: realsense/realsense2_camera/urdf/_d435.urdf.xacro (robot description, xacro)
@@ -26,9 +26,9 @@
     <xacro:property name="d435_cam_depth_py" value="-0.0075"/>
     <xacro:property name="d435_cam_depth_pz" value="${d435_cam_height/2}"/>
-    <material name="aluminum">
-      <color rgba="0.5 0.5 0.5 1"/>
-    </material>
+    <!-- <material name="aluminum"> -->
+    <!--   <color rgba="0.5 0.5 0.5 1"/> -->
+    <!-- </material> -->
     <!-- camera body, with origin at bottom screw mount -->
-    <joint name="camera_joint" type="fixed">
+    <joint name="${prefix}camera_joint" type="fixed">
       <xacro:insert_block name="origin" />
       <parent link="${parent}"/>
@@ -42,5 +42,8 @@
 	        <mesh filename="package://realsense2_camera/meshes/d435.dae" />
         </geometry>
-        <material name="aluminum"/>
+	<material name="aluminum">
+	  <color rgba="0.5 0.5 0.5 1"/>
+	</material>
+        <!-- <material name="aluminum"/> -->
       </visual>
       <collision>
@@ -58,5 +61,5 @@
     </link>
     <!-- camera depth joints and links -->
-    <joint name="camera_depth_joint" type="fixed">
+    <joint name="${prefix}camera_depth_joint" type="fixed">
       <origin xyz="${d435_cam_depth_px} ${d435_cam_depth_py} ${d435_cam_depth_pz}" rpy="0 0 0"/>
       <parent link="${prefix}camera_link"/>
@@ -64,5 +67,5 @@
     </joint>
     <link name="${prefix}camera_depth_frame"/>
-    <joint name="camera_depth_optical_joint" type="fixed">
+    <joint name="${prefix}camera_depth_optical_joint" type="fixed">
       <origin xyz="0 0 0" rpy="${-M_PI/2} 0 ${-M_PI/2}" />
       <parent link="${prefix}camera_depth_frame" />
@@ -71,5 +74,5 @@
     <link name="${prefix}camera_depth_optical_frame"/>
     <!-- camera left IR joints and links -->
-    <joint name="camera_left_ir_joint" type="fixed">
+    <joint name="${prefix}camera_left_ir_joint" type="fixed">
       <origin xyz="0 ${d435_cam_depth_to_left_ir_offset} 0" rpy="0 0 0" />
       <parent link="${prefix}camera_depth_frame" />
@@ -77,5 +80,5 @@
     </joint>
     <link name="${prefix}camera_left_ir_frame"/>
-    <joint name="camera_left_ir_optical_joint" type="fixed">
+    <joint name="${prefix}camera_left_ir_optical_joint" type="fixed">
       <origin xyz="0 0 0" rpy="${-M_PI/2} 0 ${-M_PI/2}" />
       <parent link="${prefix}camera_left_ir_frame" />
@@ -84,5 +87,5 @@
     <link name="${prefix}camera_left_ir_optical_frame"/>
     <!-- camera right IR joints and links -->
-    <joint name="camera_right_ir_joint" type="fixed">
+    <joint name="${prefix}camera_right_ir_joint" type="fixed">
       <origin xyz="0 ${d435_cam_depth_to_right_ir_offset} 0" rpy="0 0 0" />
       <parent link="${prefix}camera_depth_frame" />
@@ -90,12 +93,12 @@
     </joint>
     <link name="${prefix}camera_right_ir_frame"/>
-    <joint name="camera_right_ir_optical_joint" type="fixed">
+    <joint name="${prefix}camera_right_ir_optical_joint" type="fixed">
       <origin xyz="0 0 0" rpy="${-M_PI/2} 0 ${-M_PI/2}" />
       <parent link="${prefix}camera_right_ir_frame" />
-      <child link="camera_right_ir_optical_frame" />
+      <child link="${prefix}camera_right_ir_optical_frame" />
     </joint>
-    <link name="camera_right_ir_optical_frame"/>
+    <link name="${prefix}camera_right_ir_optical_frame"/>
     <!-- camera fisheye joints and links -->
-    <joint name="camera_fisheye_joint" type="fixed">
+    <joint name="${prefix}camera_fisheye_joint" type="fixed">
       <origin xyz="0 ${d435_cam_depth_to_fisheye_offset} 0" rpy="0 0 0" />
       <parent link="${prefix}camera_depth_frame" />
@@ -103,5 +106,5 @@
     </joint>
     <link name="${prefix}camera_fisheye_frame"/>
-    <joint name="camera_fisheye_optical_joint" type="fixed">
+    <joint name="${prefix}camera_fisheye_optical_joint" type="fixed">
       <origin xyz="0 0 0" rpy="${-M_PI/2} 0 ${-M_PI/2}" />
       <parent link="${prefix}camera_fisheye_frame" />

Commit message: Fixed urdf files of PhoXi and Realasense cameras.

File: o2as_scene_description/urdf/dual_suction_gripper.urdf.xacro (robot description, xacro)
@@ -16,7 +16,7 @@
       </visual>
       <collision>
+	<origin xyz="0.187 -0.035 -0.035" rpy="0 0 ${pi/2}"/>
 	<geometry>
-	  <mesh
-	      filename="package://o2as_scene_description/meshes/dual_suction_gripper.vhacd.dae"/>
+	  <mesh filename="package://o2as_scene_description/meshes/dual_suction_gripper.vhacd.dae"/>
 	</geometry>
       </collision>

File: o2as_scene_description/urdf/o2as_base_scene.urdf.xacro (robot description, xacro)
@@ -15,5 +15,4 @@
   <xacro:include filename="$(find ur_description)/urdf/common.gazebo.xacro" />
   <xacro:include filename="$(find o2as_gazebo)/urdf/o2as_base_scene.gazebo" />
-  <xacro:include filename="$(find realsense2_camera)/urdf/_d435.urdf.xacro" />
   <!-- robots -->
   <!-- <xacro:include filename="$(find o2as_scene_description)/urdf/ur10.urdf.xacro" /> -->
@@ -101,40 +100,32 @@
     <origin xyz="${c_bot_x} ${c_bot_y} ${bots_z}" rpy="0.0 0.0 ${-pi/2}" />
   </joint>
-  <!-- spawn and attach grippers -->
+  <!-- spawn and attach precision grippers -->
   <xacro:include filename="$(find o2as_scene_description)/urdf/precision_gripper.xacro" />
   <xacro:precision_gripper prefix="a_bot_"  grippername = "gripper" parent = "a_bot_tool0">
     <origin xyz="0.0 0 0.04" rpy="0 ${pi/2} 0"/>
   </xacro:precision_gripper>
+  <!-- spawn and attach dual suction grippers -->
+  <!-- <xacro:include filename="$(find o2as_scene_description)/urdf/dual_suction_gripper.urdf.xacro" /> -->
+  <!-- <xacro:dual_suction_gripper_o2as prefix="b_bot_" parent = "b_bot_ee_link"> -->
+  <!--   <origin xyz="0 0 0" rpy="0 0 0"/> -->
+  <!-- </xacro:dual_suction_gripper_o2as> -->
+  <!-- spawn and attach dual robotiq 85 grippers -->
   <xacro:include filename="$(find o2as_scene_description)/urdf/robotiq_85_gripper_with_ft300.urdf.xacro" />
-  <!-- <xacro:robotiq_85_gripper_o2as prefix="b_bot_" parent = "b_bot_ee_link" /> -->
+  <xacro:robotiq_85_gripper_o2as prefix="b_bot_" parent = "b_bot_ee_link" />
   <xacro:robotiq_85_gripper_o2as prefix="c_bot_" parent = "c_bot_ee_link"/>
-  <!-- spawn and attach dual suction grippers -->
-  <xacro:include filename="$(find o2as_scene_description)/urdf/dual_suction_gripper.urdf.xacro" />
-  <xacro:dual_suction_gripper_o2as prefix="b_bot_" parent = "b_bot_ee_link">
+  <!-- Add cameras -->
+  <xacro:include filename="$(find o2as_realsense2_camera)/urdf/_d435.urdf.xacro" />
+  <link name="b_bot_cam_holder_link" />
+  <joint name="b_bot_cam_holder_joint" type="fixed">
+    <parent link="b_bot_wrist_2_link" />
+    <child  link="b_bot_cam_holder_link" />
+    <origin xyz="0.0 -0.06 0.16" rpy="0.0 0.0 ${pi/2}" />
+  </joint>
+  <xacro:sensor_d435 prefix="b_bot_" parent="b_bot_cam_holder_link">
     <origin xyz="0 0 0" rpy="0 0 0"/>
-  </xacro:dual_suction_gripper_o2as>
-  <!-- Add cameras -->
-  <!-- <link name="b_bot_cam_holder_link" /> -->
-  <!-- <joint name="b_bot_cam_holder_joint" type="fixed"> -->
-  <!--   <parent link="b_bot_wrist_2_link" /> -->
-  <!--   <child  link="b_bot_cam_holder_link" /> -->
-  <!--   <origin xyz="0.0 -0.06 0.16" rpy="0.0 0.0 ${pi/2}" /> -->
-  <!-- </joint> -->
-  <!-- <xacro:sensor_d435 prefix="b_bot_" parent="b_bot_cam_holder_link"> -->
-  <!--   <origin xyz="0 0 0" rpy="0 0 0"/> -->
-  <!-- </xacro:sensor_d435> -->
-  <xacro:include filename="$(find o2as_scene_description)/urdf/d435_camera.urdf.xacro"/>
-  <xacro:d435_camera prefix="d_bot_" parent="o2as_ground">
+  </xacro:sensor_d435>
+  <xacro:sensor_d435 prefix="d_bot_" parent="o2as_ground">
     <origin xyz="0 0 ${bots_z + 0.9}" rpy="0 ${pi/2} 0"/>
-  </xacro:d435_camera>
-  <!-- <link name="d_bot_cam_holder_link" /> -->
-  <!-- <joint name="d_bot_cam_holder_joint" type="fixed"> -->
-  <!--   <parent link="o2as_ground" /> -->
-  <!--   <child  link="d_bot_cam_holder_link" /> -->
-  <!--   <origin xyz="0.0 0.0 2.0" rpy="0.0 ${pi/2} 0.0" /> -->
-  <!-- </joint> -->
-  <!-- <xacro:sensor_d435 prefix="d_bot_" parent="d_bot_cam_holder_link"> -->
-  <!--   <origin xyz="0 0 0" rpy="0 0 0"/> -->
-  <!-- </xacro:sensor_d435> -->
+  </xacro:sensor_d435>
   <!-- spawn and attach AR marker -->
   <xacro:include filename="$(find o2as_gazebo)/urdf/o2as_ar_marker.urdf.xacro"/>
@@ -145,7 +136,8 @@
   <!-- Add PhoXi 3D scanners -->
   <xacro:include filename="$(find o2as_scene_description)/urdf/phoxi_m_camera.urdf.xacro" />
-  <xacro:phoxi_m_camera_o2as prefix="a_" parent="o2as_ground">
-    <origin xyz="0.56 0 ${bots_z + .1 + .8}" rpy="${170*pi/180} 0 ${-pi/2}"/>
-  </xacro:phoxi_m_camera_o2as>
+  <xacro:phoxi_m_camera prefix="a_" parent="o2as_ground">
+    <!-- <origin xyz="0.56 0 ${bots_z + .1 + .8}" rpy="${-160*pi/180} 0 ${pi/2}"/> -->
+    <origin xyz="0.46 0 ${bots_z + .1 + .8}" rpy="${-160*pi/180} 0 ${pi/2}"/>
+  </xacro:phoxi_m_camera>
   <!-- I would like to remove the "world" link definition, but apparently it is necessary for Gazebo -->
   <link name="world" />

File: o2as_scene_description/urdf/phoxi_m_camera.urdf.xacro (robot description, xacro)
@@ -1,5 +1,5 @@
 <?xml version="1.0"?>
-<robot name="phoxi_m_camera_o2as" xmlns:xacro="http://ros.org/wiki/xacro">
-  <xacro:macro name="phoxi_m_camera_o2as" params="prefix parent *origin">
+<robot name="phoxi_m_camera" xmlns:xacro="http://ros.org/wiki/xacro">
+  <xacro:macro name="phoxi_m_camera" params="prefix parent *origin">
     <xacro:include filename="$(find o2as_phoxi_camera)/urdf/PhoXi3Dscanner_values.xacro"/>
     <xacro:include filename="$(find o2as_phoxi_camera)/urdf/PhoXi3Dscanner_macro.xacro"/>
@@ -12,8 +12,11 @@
       <xacro:PhoXi3DscannerM_meshes />
     </xacro:PhoXi3Dscanner>
-    <!-- <gazebo> -->
-    <!--   <static>true</static> -->
-    <!-- </gazebo> -->
-    <!-- <xacro:include filename="$(find o2as_gazebo)/urdf/${prefix}phoxi_m_camera.gazebo"/> -->
+    <link name="${prefix}phoxi_m_tip"/>
+    <joint name="${prefix}phoxi_m_sensor_to_${prefix}phoxi_m_tip"
+    	   type="fixed">
+      <parent link="${prefix}phoxi_m_sensor"/>
+      <child  link="${prefix}phoxi_m_tip"/>
+      <origin xyz="0 0 0" rpy="${pi/2} ${-pi/2} 0"/>
+    </joint>
   </xacro:macro>
 </robot>

Commit message: WIP: update various things for kitting in aist.

File: o2as_scene_description/urdf/dual_suction_gripper.urdf.xacro (robot description, xacro)
@@ -10,5 +10,5 @@
     <link name="${prefix}dual_suction_gripper_base_link">
       <visual>
-	<origin xyz="0.187 -0.035 -0.035" rpy="0 0 ${pi/2}"/>
+        <origin xyz="0.187 -0.035 -0.035" rpy="0 0 ${pi/2}"/>
 	<geometry>
           <mesh filename="package://o2as_scene_description/meshes/dual_suction_gripper.stl"/>
@@ -17,7 +17,9 @@
       </visual>
       <collision>
+      <!-- avoid collision -->
+	<origin xyz="0.192 -0.035 -0.035" rpy="0 0 ${pi/2}"/>
+	<!-- <origin xyz="0.187 -0.035 -0.035" rpy="0 0 ${pi/2}"/> -->
 	<geometry>
-	  <mesh
-	      filename="package://o2as_scene_description/meshes/dual_suction_gripper.vhacd.dae"/>
+	  <mesh filename="package://o2as_scene_description/meshes/dual_suction_gripper.vhacd.dae"/>
 	</geometry>
       </collision>

File: o2as_scene_description/urdf/kitting_scene.xacro (robot description, xacro)
@@ -18,5 +18,6 @@
   <xacro:property name="set1_x" value="${bin3_length/2}" />
   <xacro:property name="set1_y" value="${-.33 + bin3_width / 2}" />
-  <xacro:property name="set1_z" value="0.01" />
+  <!-- <xacro:property name="set1_z" value="0.01" /> -->
+  <xacro:property name="set1_z" value="0.0" />
   <xacro:kitting_bin_3 binname="part_6" parent="workspace_center" z_origin_offset="${z_origin_offset_3}">
     <origin xyz="${set1_x} ${set1_y} ${set1_z - z_origin_offset_3}" rpy="0 0 ${pi}" />
@@ -36,5 +37,6 @@
   <xacro:property name="set2_x" value="${.42-bin1_length/2}" />
   <xacro:property name="set2_y" value="0" />
-  <xacro:property name="set2_z" value="0.01" />
+  <!-- <xacro:property name="set2_z" value="0.01" /> -->
+  <xacro:property name="set2_z" value="0.0" />
   <xacro:kitting_bin_1 binname="part_9" parent="workspace_center" z_origin_offset="${z_origin_offset_1}">
     <origin xyz="${set2_x} ${set2_y} ${set2_z - z_origin_offset_1}" rpy="0 0 ${pi}" />
@@ -104,5 +106,5 @@
   <xacro:property name="set3_x" value="${-(bin1_length/2+tray_length/2)-0.05}" />
   <xacro:property name="set3_y" value="${.32-tray_width/2}" />
-  <xacro:property name="set3_z" value=".007" />
+  <xacro:property name="set3_z" value=".00" />
   <!-- set3_tray_1 -->
   <!-- <xacro:kitting_tray trayname="set3_tray_1" parent="workspace_center"> -->

File: o2as_scene_description/urdf/o2as_base_scene.urdf.xacro (robot description, xacro)
@@ -110,4 +110,5 @@
   <xacro:include filename="$(find o2as_scene_description)/urdf/robotiq_85_gripper_with_ft300.urdf.xacro" />
   <!-- <xacro:robotiq_85_gripper_o2as prefix="b_bot_" parent = "b_bot_ee_link" /> -->
+  <!-- <xacro:robotiq_85_gripper_o2as prefix="a_bot_" parent = "a_bot_ee_link"/> -->
   <xacro:robotiq_85_gripper_o2as prefix="c_bot_" parent = "c_bot_ee_link"/>
   <!-- spawn and attach dual suction grippers -->
