Commit message: Added a model of single_suction_gripper. Updated a model of dual_suction_gripper.

File: o2as_scene_description/urdf/dual_suction_gripper.urdf.xacro (robot description, xacro)
@@ -9,5 +9,5 @@
         <origin xyz="0.187 -0.035 -0.035" rpy="0 0 ${pi/2}"/>
 	<geometry>
-          <mesh filename="package://o2as_scene_description/meshes/dual_suction_gripper.stl"/>
+          <mesh filename="package://o2as_scene_description/meshes/dual_suction_gripper.stl" scale="0.001 0.001 0.001"/>
 	</geometry>
 	<material name="light_grey">
@@ -17,8 +17,8 @@
       <collision>
       <!-- avoid collision -->
-	<origin xyz="0.192 -0.035 -0.035" rpy="0 0 ${pi/2}"/>
+	<origin xyz="0.188 -0.035 -0.035" rpy="0 0 ${pi/2}"/>
 	<!-- <origin xyz="0.187 -0.035 -0.035" rpy="0 0 ${pi/2}"/> -->
 	<geometry>
-	  <mesh filename="package://o2as_scene_description/meshes/dual_suction_gripper.vhacd.dae"/>
+	  <mesh filename="package://o2as_scene_description/meshes/dual_suction_gripper.vhacd.dae" scale="0.001 0.001 0.001"/>
 	</geometry>
       </collision>

File: o2as_scene_description/urdf/o2as_base_scene.urdf.xacro (robot description, xacro)
@@ -111,13 +111,13 @@
     <origin xyz="0 0 0" rpy="${pi/2} 0 0"/>
   </xacro:dual_suction_gripper_o2as>
+  <!-- spawn and attach single suction grippers -->
+  <!-- <xacro:include filename="$(find o2as_scene_description)/urdf/single_suction_gripper.urdf.xacro" /> -->
+  <!-- <xacro:single_suction_gripper_o2as prefix="b_bot_" parent = "b_bot_ee_link"> -->
+  <!--   <origin xyz="0 0 0" rpy="${pi/2} 0 0"/> -->
+  <!-- </xacro:single_suction_gripper_o2as> -->
   <!-- spawn and attach dual robotiq 85 grippers -->
   <xacro:include filename="$(find o2as_scene_description)/urdf/robotiq_85_gripper_with_ft300.urdf.xacro" />
   <!-- <xacro:robotiq_85_gripper_o2as prefix="b_bot_" parent = "b_bot_ee_link" /> -->
   <xacro:robotiq_85_gripper_o2as prefix="c_bot_" parent = "c_bot_ee_link"/>
-  <!-- spawn and attach dual suction grippers -->
-  <!-- <xacro:include filename="$(find o2as_scene_description)/urdf/dual_suction_gripper.urdf.xacro" /> -->
-  <!-- <xacro:dual_suction_gripper_o2as prefix="b_bot_" parent = "b_bot_ee_link">
-    <origin xyz="0 0 0" rpy="0 0 0"/>
-  </xacro:dual_suction_gripper_o2as> -->
   <!-- Add cameras -->
   <xacro:include filename="$(find o2as_realsense2_camera)/urdf/_d435.urdf.xacro" />
@@ -146,4 +146,9 @@
     <origin xyz="0.063 0.0 0.0215" rpy="0 0 0"/>
   </xacro:o2as_ar_marker>
+  <!-- <xacro:o2as_ar_marker prefix="b_bot_" -->
+  <!-- 			parent="b_bot_single_suction_gripper_base_link" -->
+  <!-- 			marker_id="26"> -->
+  <!--   <origin xyz="0.063 0.0 0.0215" rpy="0 0 0"/> -->
+  <!-- </xacro:o2as_ar_marker> -->
   <xacro:o2as_ar_marker prefix="c_bot_"
 			parent="c_bot_robotiq_85_tip_link"

Commit message: Add suction tool link to AIST scene
This makes the calibration scripts work the same way in both systems.

File: o2as_scene_description/urdf/dual_suction_gripper.urdf.xacro (robot description, xacro)
@@ -42,4 +42,10 @@
       <origin xyz="0.187 0 0" rpy="0 0 0"/>
     </joint>
+    <joint name="${prefix}robotiq_85_suction_tool_tip_joint" type="fixed">
+      <parent link="${prefix}dual_suction_gripper_pad_link"/>
+      <child link="${prefix}suction_tool_tip_link"/>
+      <origin rpy="0.0 0.0 0.0" xyz="0.0 0.0 0.0 "/>
+    </joint>
+    <link name="${prefix}suction_tool_tip_link"/>
     <!-- A link representing the tip of the coander gripper
 	 and a joint attaching it to the gripper -->

Commit message: Fixed bug in base.paramtuples().

File: o2as_scene_description/urdf/dual_suction_gripper.urdf.xacro (robot description, xacro)
@@ -7,5 +7,5 @@
     <link name="${prefix}dual_suction_gripper_base_link">
       <visual>
-        <origin xyz="0.187 -0.035 -0.035" rpy="0 0 ${pi/2}"/>
+        <origin xyz="0.1855 -0.035 -0.035" rpy="0 0 ${pi/2}"/>
 	<geometry>
           <mesh filename="package://o2as_scene_description/meshes/dual_suction_gripper.stl" scale="0.001 0.001 0.001"/>
@@ -17,5 +17,5 @@
       <collision>
       <!-- avoid collision -->
-	<origin xyz="0.188 -0.035 -0.035" rpy="0 0 ${pi/2}"/>
+	<origin xyz="0.1855 -0.035 -0.035" rpy="0 0 ${pi/2}"/>
 	<!-- <origin xyz="0.187 -0.035 -0.035" rpy="0 0 ${pi/2}"/> -->
 	<geometry>
@@ -40,5 +40,5 @@
       <parent link="${prefix}dual_suction_gripper_base_link"/>
       <child  link="${prefix}dual_suction_gripper_pad_link"/>
-      <origin xyz="0.187 0 0" rpy="0 0 0"/>
+      <origin xyz="0.1855 0 0" rpy="0 0 0"/>
     </joint>
     <joint name="${prefix}robotiq_85_suction_tool_tip_joint" type="fixed">

File: o2as_scene_description/urdf/single_suction_gripper.urdf.xacro (robot description, xacro)
@@ -7,5 +7,5 @@
     <link name="${prefix}single_suction_gripper_base_link">
       <visual>
-        <origin xyz="0.187 -0.035 -0.035" rpy="0 0 ${pi/2}"/>
+        <origin xyz="0.1855 -0.035 -0.035" rpy="0 0 ${pi/2}"/>
 	<geometry>
           <mesh filename="package://o2as_scene_description/meshes/single_suction_gripper.stl" scale="0.001 0.001 0.001"/>
@@ -18,5 +18,5 @@
       <!-- avoid collision -->
         <!-- <origin xyz="0.188 -0.035 -0.035" rpy="0 0 ${pi/2}"/> -->
-	<origin xyz="0.187 -0.035 -0.035" rpy="0 0 ${pi/2}"/>
+	<origin xyz="0.1855 -0.035 -0.035" rpy="0 0 ${pi/2}"/>
 	<geometry>
 	  <mesh filename="package://o2as_scene_description/meshes/single_suction_gripper.vhacd.dae" scale="0.001 0.001 0.001"/>
@@ -40,5 +40,5 @@
       <parent link="${prefix}single_suction_gripper_base_link"/>
       <child  link="${prefix}single_suction_gripper_pad_link"/>
-      <origin xyz="0.187 0 0" rpy="0 0 0"/>
+      <origin xyz="0.1855 0 0" rpy="0 0 0"/>
     </joint>
   </xacro:macro>
