Commit message: Modify camera and marker position for testing easy handeye

File: o2as_gazebo/urdf/d_bot_camera.urdf.xacro (robot description, xacro)
@@ -17,5 +17,5 @@
     <parent link="d_bot_base" />
     <child link="d_bot_link" />
-    <origin xyz="0.0 0.0 0.0" ryp="0.0 0.0 0.0" />
+    <origin xyz="0.0 0.0 2.0" rpy="0.0 ${pi/2} 0.0" />
   </joint>
   <!-- <virtual_joint name="d_bot_joint" type="fixed"
@@ -25,8 +25,8 @@
     <parent link="d_bot_link" />
     <child link="d_bot_cam_holder_link" />
-    <origin xyz="0.0 0.0 0.0" ryp="0 0 0" />
+    <origin xyz="0.0 0.0 0.0" rpy="0 0 0" />
   </joint>
   <xacro:sensor_d435 prefix="d_bot_" parent="d_bot_cam_holder_link">
-    <origin xyz="0.0 0 1.5" rpy="0 ${pi/2} 0"/>
+    <origin xyz="0 0 0" rpy="0 0 0"/>
   </xacro:sensor_d435>
 </robot>

File: o2as_scene_description/urdf/o2as_base_scene.urdf.xacro (robot description, xacro)
@@ -110,5 +110,5 @@
   <xacro:include filename="$(find o2as_gazebo)/urdf/o2as_ar_marker.urdf.xacro"/>
   <xacro:o2as_ar_marker prefix="b_bot_" parent="b_bot_wrist_3_link">
-    <origin xyz="0.0 0.0 0.05" rpy="0 0 0"/>
+    <origin xyz="0.0 -0.07 0.0" rpy="${pi/2} 0 0"/>
   </xacro:o2as_ar_marker>
   <!-- I meant to remove the "world" link definition, but apparently it is necessary for Gazebo -->
