Commit message: Parametrize ID of AR marker

File: o2as_gazebo/urdf/o2as_ar_marker.urdf.xacro (robot description, xacro)
@@ -1,5 +1,5 @@
 <?xml version="1.0" ?>
 <robot name="o2as_ar_marker" xmlns:xacro="http://www.ros.org/wiki/xacro">
-  <xacro:macro name="o2as_ar_marker" params="prefix parent *origin">
+  <xacro:macro name="o2as_ar_marker" params="marker_id prefix parent *origin">
     <joint name="${prefix}ar_marker_joint" type="fixed">
       <parent link="${parent}" />
@@ -24,5 +24,5 @@
          gazebo_media_path in package.xml. -->
     <gazebo reference="${prefix}ar_marker">
-      <material>Aruco/marker26_8cm</material>
+      <material>Aruco/marker${marker_id}</material>
     </gazebo>
   </xacro:macro>

File: o2as_scene_description/urdf/o2as_base_scene.urdf.xacro (robot description, xacro)
@@ -109,5 +109,6 @@
   <!-- spawn and attach AR marker -->
   <xacro:include filename="$(find o2as_gazebo)/urdf/o2as_ar_marker.urdf.xacro"/>
-  <xacro:o2as_ar_marker prefix="b_bot_" parent="b_bot_wrist_3_link">
+  <xacro:o2as_ar_marker prefix="b_bot_" parent="b_bot_wrist_3_link"
+   marker_id="26">
     <origin xyz="0.0 -0.07 0.0" rpy="${pi/2} 0 0"/>
   </xacro:o2as_ar_marker>

Commit message: AR markers are moved from wrist_3_link to ee_link.

File: o2as_gazebo/urdf/o2as_ar_marker.urdf.xacro (robot description, xacro)
@@ -10,5 +10,5 @@
       <visual name="${prefix}ar_marker_visual">
         <geometry>
-          <box size="0.09 0.09 0.001" />
+          <box size="0.08 0.08 0.005" />
         </geometry>
         <!--<material name="orange" />-->
@@ -16,5 +16,5 @@
       <collision name="${prefix}ar_marker_collision">
         <geometry>
-          <box size="0.09 0.09 0.02" />
+          <box size="0.08 0.08 0.005" />
         </geometry>
       </collision>

File: o2as_scene_description/urdf/o2as_base_scene.urdf.xacro (robot description, xacro)
@@ -20,7 +20,6 @@
   <xacro:include filename="$(find o2as_scene_description)/urdf/ur3.urdf.xacro" />
   <!-- Scene items (trays, bins...) -->
-  <!-- <xacro:include filename="$(find o2as_scene_description)/urdf/kitting_tray_with_partitions.xacro" /> -->
-  <xacro:include filename="$(find o2as_scene_description)/urdf/taskboard_scene.xacro" />
-  <!-- <xacro:include filename="$(find o2as_scene_description)/urdf/kitting_scene.xacro" /> -->
+  <!-- <xacro:include filename="$(find o2as_scene_description)/urdf/taskboard_scene.xacro" /> -->
+  <xacro:include filename="$(find o2as_scene_description)/urdf/kitting_scene.xacro" />
   <!-- <xacro:include filename="$(find o2as_scene_description)/urdf/assembly_scene.xacro" /> -->
   <!-- Robot bases -->
@@ -108,11 +107,11 @@
   </xacro:precision_gripper> -->
   <!-- spawn and attach dual suction grippers -->
-  <!-- <xacro:include filename="$(find o2as_scene_description)/urdf/dual_suction_gripper.urdf.xacro" /> -->
-  <!-- <xacro:dual_suction_gripper_o2as prefix="b_bot_" parent = "b_bot_ee_link"> -->
-  <!--   <origin xyz="0 0 0" rpy="0 0 0"/> -->
-  <!-- </xacro:dual_suction_gripper_o2as> -->
+  <xacro:include filename="$(find o2as_scene_description)/urdf/dual_suction_gripper.urdf.xacro" />
+  <xacro:dual_suction_gripper_o2as prefix="b_bot_" parent = "b_bot_ee_link">
+    <origin xyz="0 0 0" rpy="0 0 0"/>
+  </xacro:dual_suction_gripper_o2as>
   <!-- spawn and attach dual robotiq 85 grippers -->
   <xacro:include filename="$(find o2as_scene_description)/urdf/robotiq_85_gripper_with_ft300.urdf.xacro" />
-  <xacro:robotiq_85_gripper_o2as prefix="b_bot_" parent = "b_bot_ee_link" />
+  <!-- <xacro:robotiq_85_gripper_o2as prefix="b_bot_" parent = "b_bot_ee_link" /> -->
   <xacro:robotiq_85_gripper_o2as prefix="c_bot_" parent = "c_bot_ee_link"/>
   <!-- spawn and attach dual suction grippers -->
@@ -137,15 +136,15 @@
   <!-- spawn and attach AR markers -->
   <xacro:include filename="$(find o2as_gazebo)/urdf/o2as_ar_marker.urdf.xacro"/>
-  <xacro:o2as_ar_marker prefix="a_bot_" parent="a_bot_wrist_3_link"
-   marker_id="17">
-    <origin xyz="0.0 -0.07 0.0" rpy="${pi/2} 0 0"/>
+  <xacro:o2as_ar_marker prefix="a_bot_" parent="a_bot_ee_link"
+			marker_id="17">
+    <origin xyz="0.25 0.0 0.055" rpy="0 0 ${pi}"/>
   </xacro:o2as_ar_marker>
-  <xacro:o2as_ar_marker prefix="b_bot_" parent="b_bot_wrist_3_link"
-   marker_id="26">
-    <origin xyz="0.0 -0.07 0.0" rpy="${pi/2} 0 0"/>
+  <xacro:o2as_ar_marker prefix="b_bot_" parent="b_bot_ee_link"
+			marker_id="26">
+    <origin xyz="0.064 0.0 0.019" rpy="0 0 ${pi}"/>
   </xacro:o2as_ar_marker>
-    <xacro:o2as_ar_marker prefix="c_bot_" parent="c_bot_wrist_3_link"
-   marker_id="256">
-    <origin xyz="0.0 0.12 0.05" rpy="0 0 ${pi/2}"/>
+    <xacro:o2as_ar_marker prefix="c_bot_" parent="c_bot_ee_link"
+			  marker_id="256">
+    <origin xyz="0.22 0.0 0.016" rpy="0 0 ${pi}"/>
   </xacro:o2as_ar_marker>
   <!-- Add PhoXi 3D scanners -->

Commit message: Frame of AR marker is rotated by 180 deg. around z-axis.

File: o2as_gazebo/urdf/o2as_ar_marker.urdf.xacro (robot description, xacro)
@@ -9,4 +9,5 @@
     <link name="${prefix}ar_marker">
       <visual name="${prefix}ar_marker_visual">
+	<origin xyz="0 0 0" rpy="0 0 ${pi}"/>
         <geometry>
           <box size="0.08 0.08 0.005" />
@@ -15,4 +16,5 @@
       </visual>
       <collision name="${prefix}ar_marker_collision">
+	<origin xyz="0 0 0" rpy="0 0 ${pi}"/>
         <geometry>
           <box size="0.08 0.08 0.005" />

File: o2as_scene_description/urdf/o2as_base_scene.urdf.xacro (robot description, xacro)
@@ -109,5 +109,5 @@
   <xacro:include filename="$(find o2as_scene_description)/urdf/dual_suction_gripper.urdf.xacro" />
   <xacro:dual_suction_gripper_o2as prefix="b_bot_" parent = "b_bot_ee_link">
-    <origin xyz="0 0 0" rpy="0 0 0"/>
+    <origin xyz="0 0 0" rpy="${pi/2} 0 0"/>
   </xacro:dual_suction_gripper_o2as>
   <!-- spawn and attach dual robotiq 85 grippers -->
@@ -138,13 +138,13 @@
   <xacro:o2as_ar_marker prefix="a_bot_" parent="a_bot_ee_link"
 			marker_id="17">
-    <origin xyz="0.25 0.0 -0.045" rpy="${pi} 0 ${pi}"/>
+    <origin xyz="0.25 0.0 0.045" rpy="0 0 0"/>
   </xacro:o2as_ar_marker>
-  <xacro:o2as_ar_marker prefix="b_bot_" parent="b_bot_ee_link"
+  <xacro:o2as_ar_marker prefix="b_bot_" parent="b_bot_dual_suction_gripper_base_link"
 			marker_id="26">
-    <origin xyz="0.064 0.0 -0.020" rpy="${pi} 0 ${pi}"/>
+    <origin xyz="0.063 0.0 0.019" rpy="0 0 0"/>
   </xacro:o2as_ar_marker>
     <xacro:o2as_ar_marker prefix="c_bot_" parent="c_bot_ee_link"
 			  marker_id="256">
-    <origin xyz="0.22 0.0 -0.016" rpy="${pi} 0 ${pi}"/>
+    <origin xyz="0.22 0.0 0.016" rpy="0 0 0"/>
   </xacro:o2as_ar_marker>
   <!-- Add PhoXi 3D scanners -->

Commit message: Shifted AR marker's frame by 2.5mm along Z-axis.

File: o2as_gazebo/urdf/o2as_ar_marker.urdf.xacro (robot description, xacro)
@@ -9,5 +9,5 @@
     <link name="${prefix}ar_marker">
       <visual name="${prefix}ar_marker_visual">
-	<origin xyz="0 0 0" rpy="0 0 ${pi}"/>
+	<origin xyz="0 0 -0.0025" rpy="0 0 ${pi}"/>
         <geometry>
           <box size="0.08 0.08 0.005" />
@@ -16,5 +16,5 @@
       </visual>
       <collision name="${prefix}ar_marker_collision">
-	<origin xyz="0 0 0" rpy="0 0 ${pi}"/>
+	<origin xyz="0 0 -0.0025" rpy="0 0 ${pi}"/>
         <geometry>
           <box size="0.08 0.08 0.005" />

File: o2as_scene_description/urdf/o2as_base_scene.urdf.xacro (robot description, xacro)
@@ -138,13 +138,13 @@
   <xacro:o2as_ar_marker prefix="a_bot_" parent="a_bot_ee_link"
 			marker_id="17">
-    <origin xyz="0.25 0.0 0.045" rpy="0 0 0"/>
+    <origin xyz="0.25 0.0 0.047" rpy="0 0 0"/>
   </xacro:o2as_ar_marker>
   <xacro:o2as_ar_marker prefix="b_bot_" parent="b_bot_dual_suction_gripper_base_link"
 			marker_id="26">
-    <origin xyz="0.063 0.0 0.019" rpy="0 0 0"/>
+    <origin xyz="0.063 0.0 0.0215" rpy="0 0 0"/>
   </xacro:o2as_ar_marker>
     <xacro:o2as_ar_marker prefix="c_bot_" parent="c_bot_ee_link"
 			  marker_id="256">
-    <origin xyz="0.22 0.0 0.016" rpy="0 0 0"/>
+    <origin xyz="0.22 0.0 0.0185" rpy="0 0 0"/>
   </xacro:o2as_ar_marker>
   <!-- Add PhoXi 3D scanners -->

Commit message: AR marker #32 added.

File: o2as_gazebo/urdf/o2as_ar_marker.urdf.xacro (robot description, xacro)
@@ -29,3 +29,31 @@
     </gazebo>
   </xacro:macro>
+  <xacro:macro name="o2as_ar_marker_18cm" params="marker_id prefix parent *origin">
+    <joint name="${prefix}ar_marker_joint" type="fixed">
+      <parent link="${parent}" />
+      <child link = "${prefix}ar_marker" />
+      <xacro:insert_block name="origin" />
+    </joint>
+    <link name="${prefix}ar_marker">
+      <visual name="${prefix}ar_marker_visual">
+	<origin xyz="0 0 -0.0005" rpy="0 0 ${pi}"/>
+        <geometry>
+          <box size="0.18 0.18 0.001" />
+        </geometry>
+        <!--<material name="orange" />-->
+      </visual>
+      <collision name="${prefix}ar_marker_collision">
+	<origin xyz="0 0 -0.0005" rpy="0 0 ${pi}"/>
+        <geometry>
+          <box size="0.18 0.18 0.001" />
+        </geometry>
+      </collision>
+    </link>
+    <!-- For Gazebo, material of AR marker is defined in
+         o2as_gazebo/media/material. You also need to export
+         gazebo_media_path in package.xml. -->
+    <gazebo reference="${prefix}ar_marker">
+      <material>Aruco/marker${marker_id}-160-10</material>
+    </gazebo>
+  </xacro:macro>
 </robot>

File: o2as_scene_description/urdf/o2as_base_scene.urdf.xacro (robot description, xacro)
@@ -167,9 +167,14 @@
     <origin xyz="0.0 0.0 0.0185" rpy="0 0 0"/>
   </xacro:o2as_ar_marker>
-  <xacro:o2as_ar_marker prefix="workspace_"
+  <!-- <xacro:o2as_ar_marker prefix="workspace_" -->
+  <!-- 			parent="workspace_center" -->
+  <!-- 			marker_id="256"> -->
+  <!--   <origin xyz="0.0 0.0 0.0005" rpy="0 0 0"/> -->
+  <!-- </xacro:o2as_ar_marker> -->
+  <xacro:o2as_ar_marker_18cm prefix="workspace_"
 			parent="workspace_center"
-			marker_id="256">
+			marker_id="32">
     <origin xyz="0.0 0.0 0.0005" rpy="0 0 0"/>
-  </xacro:o2as_ar_marker>
+  </xacro:o2as_ar_marker_18cm>
   <!-- Add PhoXi 3D scanners -->
   <xacro:include filename="$(find o2as_scene_description)/urdf/phoxi_m_camera.urdf.xacro" />

Commit message: Make realsense work again.

File: o2as_gazebo/urdf/o2as_ar_marker.urdf.xacro (robot description, xacro)
@@ -29,5 +29,5 @@
     </gazebo>
   </xacro:macro>
-  <xacro:macro name="o2as_ar_marker_18cm" params="marker_id prefix parent *origin">
+  <xacro:macro name="o2as_ar_marker_16cm" params="marker_id prefix parent *origin">
     <joint name="${prefix}ar_marker_joint" type="fixed">
       <parent link="${parent}" />

File: o2as_scene_description/urdf/o2as_base_scene.urdf.xacro (robot description, xacro)
@@ -180,5 +180,4 @@
   <!--   <origin xyz="0.0 0.0 0.0005" rpy="0 0 0"/> -->
   <!-- </xacro:o2as_ar_marker> -->
-  <xacro:include filename="$(find o2as_gazebo)/urdf/o2as_ar_marker_16cm.urdf.xacro"/>
   <xacro:o2as_ar_marker_16cm prefix="workspace_"
   			parent="workspace_center"
