Commit message: Add assembly scene stub, parts macros

File: o2as_parts_description/urdf/01_BASE.urdf (robot description, URDF)
Before this commit: robot 16_SPWF6, 1 links, 0 joints
Links:
- link baseLink: geometry collision mesh filename=/root/catkin_ws/src/o2as_parts_description/meshes/01-BASE.s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 scale=0.001 0.001 0.001; visual mesh filename=/root/catkin_ws/src/o2as_parts_description/meshes/01-BASE.s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 scale=0.001 0.001 0.001

File: o2as_parts_description/urdf/02_PANEL.urdf (robot description, URDF)
Before this commit: robot 16_SPWF6, 1 links, 0 joints
Links:
- link baseLink: geometry collision mesh filename=/root/catkin_ws/src/o2as_parts_description/meshes/02-PANEL.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 scale=0.001 0.001 0.001; visual mesh filename=/root/catkin_ws/src/o2as_parts_description/meshes/02-PANEL.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 scale=0.001 0.001 0.001

File: o2as_parts_description/urdf/03_PANEL2.urdf (robot description, URDF)
Before this commit: robot 16_SPWF6, 1 links, 0 joints
Links:
- link baseLink: geometry collision mesh filename=/root/catkin_ws/src/o2as_parts_description/meshes/03_PANEL2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 scale=0.001 0.001 0.001; visual mesh filename=/root/catkin_ws/src/o2as_parts_description/meshes/03_PANEL2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 scale=0.001 0.001 0.001

File: o2as_scene_description/urdf/o2as_base_scene.urdf.xacro (robot description, xacro)
@@ -23,5 +23,5 @@
   <!-- <xacro:include filename="$(find o2as_scene_description)/urdf/taskboard_scene.xacro" /> -->
   <!-- <xacro:include filename="$(find o2as_scene_description)/urdf/kitting_scene.xacro" /> -->
-  <!-- <xacro:include filename="$(find o2as_scene_description)/urdf/assembly_scene.xacro" /> -->
+  <xacro:include filename="$(find o2as_scene_description)/urdf/assembly_scene.xacro" />
   <!-- Robot bases -->
   <!-- Putting these at height 0.0 makes them intersect with the ground, so they are elevated. -->
@@ -54,11 +54,11 @@
   <xacro:include filename="$(find o2as_scene_description)/urdf/screw_tools.xacro" />
   <!-- Feeders -->
-  <xacro:include filename="$(find o2as_scene_description)/urdf/screw_feeder.xacro" />
+  <!-- <xacro:include filename="$(find o2as_scene_description)/urdf/screw_feeder.xacro" />
   <xacro:screw_feeder feedername="m3_feeder" parent="a_bot_base_smfl">
-    <origin xyz=".1 .4 .05" rpy="0 0 ${pi/2}" />
+    <origin xyz=".3 .4 .05" rpy="0 0 ${pi/2}" />
   </xacro:screw_feeder>
   <xacro:screw_feeder feedername="m4_feeder" parent="c_bot_base_smfl">
     <origin xyz=".45 .05 .05" rpy="0 0 0" />
-  </xacro:screw_feeder>
+  </xacro:screw_feeder> -->
   <!-- <xacro:screw_feeder feedername="m5_feeder" parent="c_bot_base_smfl">
     <origin xyz=".45 .2 .05" rpy="0 0 0" />
