Commit message: Fixes to previous commit

File: realsense/realsense2_camera/urdf/_d435.urdf.xacro (robot description, xacro)
@@ -40,6 +40,5 @@
         <geometry>
           <!-- <box size="${d435_cam_width} ${d435_cam_height} ${d435_cam_depth}"/> -->
-	  <mesh filename="package://realsense2_camera/meshes/d435.dae" />
-          <!--<mesh filename="package://realsense2_camera/meshes/d435/d435.dae" />-->
+	        <mesh filename="package://realsense2_camera/meshes/d435.dae" />
         </geometry>
         <material name="aluminum"/>

Commit message: Add prefix to d435 macro
This is needed so we can use multiple cameras later

File: realsense/realsense2_camera/urdf/_d435.urdf.xacro (robot description, xacro)
@@ -7,33 +7,33 @@
 -->
 <robot name="sensor_d435" xmlns:xacro="http://ros.org/wiki/xacro">
-  <xacro:property name="M_PI" value="3.1415926535897931" />
-  <!-- The following values are approximate, and the camera node
-   publishing TF values with actual calibrated camera extrinsic values -->
-  <xacro:property name="d435_cam_depth_to_left_ir_offset" value="-0.025"/>
-  <xacro:property name="d435_cam_depth_to_right_ir_offset" value="0.025"/>
-  <xacro:property name="d435_cam_depth_to_fisheye_offset" value="0.040"/>
-  <!-- The following values model the aluminum peripherial case for the
-    D435 camera, with the camera joint represented by the actual
-    peripheral camera tripod mount -->
-  <xacro:property name="d435_cam_width" value="0.090"/>
-  <xacro:property name="d435_cam_height" value="0.025"/>
-  <xacro:property name="d435_cam_depth" value="0.02505"/>
-  <xacro:property name="d435_cam_mount_from_center_offset" value="0.0149"/>
-  <!-- The following offset is relative to the physical D435 camera peripherial
-    camera tripod mount -->
-  <xacro:property name="d435_cam_depth_px" value="${d435_cam_mount_from_center_offset}"/>
-  <xacro:property name="d435_cam_depth_py" value="-0.0075"/>
-  <xacro:property name="d435_cam_depth_pz" value="${d435_cam_height/2}"/>
-  <material name="aluminum">
-    <color rgba="0.5 0.5 0.5 1"/>
-  </material>
-  <xacro:macro name="sensor_d435" params="parent *origin">
+  <xacro:macro name="sensor_d435" params="prefix parent *origin">
+    <xacro:property name="M_PI" value="3.1415926535897931" />
+    <!-- The following values are approximate, and the camera node
+    publishing TF values with actual calibrated camera extrinsic values -->
+    <xacro:property name="d435_cam_depth_to_left_ir_offset" value="-0.025"/>
+    <xacro:property name="d435_cam_depth_to_right_ir_offset" value="0.025"/>
+    <xacro:property name="d435_cam_depth_to_fisheye_offset" value="0.040"/>
+    <!-- The following values model the aluminum peripherial case for the
+      D435 camera, with the camera joint represented by the actual
+      peripheral camera tripod mount -->
+    <xacro:property name="d435_cam_width" value="0.090"/>
+    <xacro:property name="d435_cam_height" value="0.025"/>
+    <xacro:property name="d435_cam_depth" value="0.02505"/>
+    <xacro:property name="d435_cam_mount_from_center_offset" value="0.0149"/>
+    <!-- The following offset is relative to the physical D435 camera peripherial
+      camera tripod mount -->
+    <xacro:property name="d435_cam_depth_px" value="${d435_cam_mount_from_center_offset}"/>
+    <xacro:property name="d435_cam_depth_py" value="-0.0075"/>
+    <xacro:property name="d435_cam_depth_pz" value="${d435_cam_height/2}"/>
+    <material name="aluminum">
+      <color rgba="0.5 0.5 0.5 1"/>
+    </material>
     <!-- camera body, with origin at bottom screw mount -->
     <joint name="camera_joint" type="fixed">
       <xacro:insert_block name="origin" />
       <parent link="${parent}"/>
-      <child link="camera_link" />
+      <child link="${prefix}camera_link" />
     </joint>
-    <link name="camera_link">
+    <link name="${prefix}camera_link">
       <visual>
       <origin xyz="${d435_cam_mount_from_center_offset} 0.0 ${d435_cam_height/2}" rpy="${M_PI/2} 0 ${M_PI/2}"/>
@@ -60,37 +60,37 @@
     <joint name="camera_depth_joint" type="fixed">
       <origin xyz="${d435_cam_depth_px} ${d435_cam_depth_py} ${d435_cam_depth_pz}" rpy="0 0 0"/>
-      <parent link="camera_link"/>
-      <child link="camera_depth_frame" />
+      <parent link="${prefix}camera_link"/>
+      <child link="${prefix}camera_depth_frame" />
     </joint>
-    <link name="camera_depth_frame"/>
+    <link name="${prefix}camera_depth_frame"/>
     <joint name="camera_depth_optical_joint" type="fixed">
       <origin xyz="0 0 0" rpy="${-M_PI/2} 0 ${-M_PI/2}" />
-      <parent link="camera_depth_frame" />
-      <child link="camera_depth_optical_frame" />
+      <parent link="${prefix}camera_depth_frame" />
+      <child link="${prefix}camera_depth_optical_frame" />
     </joint>
-    <link name="camera_depth_optical_frame"/>
+    <link name="${prefix}camera_depth_optical_frame"/>
     <!-- camera left IR joints and links -->
     <joint name="camera_left_ir_joint" type="fixed">
       <origin xyz="0 ${d435_cam_depth_to_left_ir_offset} 0" rpy="0 0 0" />
-      <parent link="camera_depth_frame" />
-      <child link="camera_left_ir_frame" />
+      <parent link="${prefix}camera_depth_frame" />
+      <child link="${prefix}camera_left_ir_frame" />
     </joint>
-    <link name="camera_left_ir_frame"/>
+    <link name="${prefix}camera_left_ir_frame"/>
     <joint name="camera_left_ir_optical_joint" type="fixed">
       <origin xyz="0 0 0" rpy="${-M_PI/2} 0 ${-M_PI/2}" />
-      <parent link="camera_left_ir_frame" />
-      <child link="camera_left_ir_optical_frame" />
+      <parent link="${prefix}camera_left_ir_frame" />
+      <child link="${prefix}camera_left_ir_optical_frame" />
     </joint>
-    <link name="camera_left_ir_optical_frame"/>
+    <link name="${prefix}camera_left_ir_optical_frame"/>
     <!-- camera right IR joints and links -->
     <joint name="camera_right_ir_joint" type="fixed">
       <origin xyz="0 ${d435_cam_depth_to_right_ir_offset} 0" rpy="0 0 0" />
-      <parent link="camera_depth_frame" />
-      <child link="camera_right_ir_frame" />
+      <parent link="${prefix}camera_depth_frame" />
+      <child link="${prefix}camera_right_ir_frame" />
     </joint>
-    <link name="camera_right_ir_frame"/>
+    <link name="${prefix}camera_right_ir_frame"/>
     <joint name="camera_right_ir_optical_joint" type="fixed">
       <origin xyz="0 0 0" rpy="${-M_PI/2} 0 ${-M_PI/2}" />
-      <parent link="camera_right_ir_frame" />
+      <parent link="${prefix}camera_right_ir_frame" />
       <child link="camera_right_ir_optical_frame" />
     </joint>
@@ -99,14 +99,14 @@
     <joint name="camera_fisheye_joint" type="fixed">
       <origin xyz="0 ${d435_cam_depth_to_fisheye_offset} 0" rpy="0 0 0" />
-      <parent link="camera_depth_frame" />
-      <child link="camera_fisheye_frame" />
+      <parent link="${prefix}camera_depth_frame" />
+      <child link="${prefix}camera_fisheye_frame" />
     </joint>
-    <link name="camera_fisheye_frame"/>
+    <link name="${prefix}camera_fisheye_frame"/>
     <joint name="camera_fisheye_optical_joint" type="fixed">
       <origin xyz="0 0 0" rpy="${-M_PI/2} 0 ${-M_PI/2}" />
-      <parent link="camera_fisheye_frame" />
-      <child link="camera_fisheye_optical_frame" />
+      <parent link="${prefix}camera_fisheye_frame" />
+      <child link="${prefix}camera_fisheye_optical_frame" />
     </joint>
-    <link name="camera_fisheye_optical_frame"/>
+    <link name="${prefix}camera_fisheye_optical_frame"/>
   </xacro:macro>
 </robot>

Commit message: Add depth_image_frame to urdf model of realsense2_camera

File: realsense/realsense2_camera/urdf/_d435.urdf.xacro (robot description, xacro)
@@ -64,4 +64,10 @@
     </joint>
     <link name="${prefix}camera_depth_frame"/>
+    <joint name="camera_depth_image_joint" type="fixed">
+      <origin xyz="0 0 0" rpy="${M_PI/2} ${M_PI} ${M_PI/2}"/>
+      <parent link="${prefix}camera_depth_frame"/>
+      <child link="${prefix}camera_depth_image_frame" />
+    </joint>
+    <link name="${prefix}camera_depth_image_frame"/>
     <joint name="camera_depth_optical_joint" type="fixed">
       <origin xyz="0 0 0" rpy="${-M_PI/2} 0 ${-M_PI/2}" />

Commit message: Fix macro to allow multiple realsense cams

File: realsense/realsense2_camera/urdf/_d435.urdf.xacro (robot description, xacro)
@@ -26,9 +26,6 @@
     <xacro:property name="d435_cam_depth_py" value="-0.0075"/>
     <xacro:property name="d435_cam_depth_pz" value="${d435_cam_height/2}"/>
-    <material name="aluminum">
-      <color rgba="0.5 0.5 0.5 1"/>
-    </material>
     <!-- camera body, with origin at bottom screw mount -->
-    <joint name="camera_joint" type="fixed">
+    <joint name="${prefix}camera_joint" type="fixed">
       <xacro:insert_block name="origin" />
       <parent link="${parent}"/>
@@ -42,5 +39,7 @@
 	        <mesh filename="package://realsense2_camera/meshes/d435.dae" />
         </geometry>
-        <material name="aluminum"/>
+        <material name="aluminum">
+          <color rgba="0.5 0.5 0.5 1"/>
+        </material>
       </visual>
       <collision>
@@ -58,5 +57,5 @@
     </link>
     <!-- camera depth joints and links -->
-    <joint name="camera_depth_joint" type="fixed">
+    <joint name="${prefix}camera_depth_joint" type="fixed">
       <origin xyz="${d435_cam_depth_px} ${d435_cam_depth_py} ${d435_cam_depth_pz}" rpy="0 0 0"/>
       <parent link="${prefix}camera_link"/>
@@ -64,5 +63,5 @@
     </joint>
     <link name="${prefix}camera_depth_frame"/>
-    <joint name="camera_depth_optical_joint" type="fixed">
+    <joint name="${prefix}camera_depth_optical_joint" type="fixed">
       <origin xyz="0 0 0" rpy="${-M_PI/2} 0 ${-M_PI/2}" />
       <parent link="${prefix}camera_depth_frame" />
@@ -71,5 +70,5 @@
     <link name="${prefix}camera_depth_optical_frame"/>
     <!-- camera left IR joints and links -->
-    <joint name="camera_left_ir_joint" type="fixed">
+    <joint name="${prefix}camera_left_ir_joint" type="fixed">
       <origin xyz="0 ${d435_cam_depth_to_left_ir_offset} 0" rpy="0 0 0" />
       <parent link="${prefix}camera_depth_frame" />
@@ -77,5 +76,5 @@
     </joint>
     <link name="${prefix}camera_left_ir_frame"/>
-    <joint name="camera_left_ir_optical_joint" type="fixed">
+    <joint name="${prefix}camera_left_ir_optical_joint" type="fixed">
       <origin xyz="0 0 0" rpy="${-M_PI/2} 0 ${-M_PI/2}" />
       <parent link="${prefix}camera_left_ir_frame" />
@@ -84,5 +83,5 @@
     <link name="${prefix}camera_left_ir_optical_frame"/>
     <!-- camera right IR joints and links -->
-    <joint name="camera_right_ir_joint" type="fixed">
+    <joint name="${prefix}camera_right_ir_joint" type="fixed">
       <origin xyz="0 ${d435_cam_depth_to_right_ir_offset} 0" rpy="0 0 0" />
       <parent link="${prefix}camera_depth_frame" />
@@ -90,12 +89,12 @@
     </joint>
     <link name="${prefix}camera_right_ir_frame"/>
-    <joint name="camera_right_ir_optical_joint" type="fixed">
+    <joint name="${prefix}camera_right_ir_optical_joint" type="fixed">
       <origin xyz="0 0 0" rpy="${-M_PI/2} 0 ${-M_PI/2}" />
       <parent link="${prefix}camera_right_ir_frame" />
-      <child link="camera_right_ir_optical_frame" />
+      <child link="${prefix}camera_right_ir_optical_frame" />
     </joint>
-    <link name="camera_right_ir_optical_frame"/>
+    <link name="${prefix}camera_right_ir_optical_frame"/>
     <!-- camera fisheye joints and links -->
-    <joint name="camera_fisheye_joint" type="fixed">
+    <joint name="${prefix}camera_fisheye_joint" type="fixed">
       <origin xyz="0 ${d435_cam_depth_to_fisheye_offset} 0" rpy="0 0 0" />
       <parent link="${prefix}camera_depth_frame" />
@@ -103,5 +102,5 @@
     </joint>
     <link name="${prefix}camera_fisheye_frame"/>
-    <joint name="camera_fisheye_optical_joint" type="fixed">
+    <joint name="${prefix}camera_fisheye_optical_joint" type="fixed">
       <origin xyz="0 0 0" rpy="${-M_PI/2} 0 ${-M_PI/2}" />
       <parent link="${prefix}camera_fisheye_frame" />

File: realsense/realsense2_camera/urdf/_r410.urdf.xacro (robot description, xacro)
@@ -24,7 +24,4 @@
   <xacro:property name="r410_cam_depth_py" value="-0.0425"/>
   <xacro:property name="r410_cam_depth_pz" value="0.026"/>
-  <material name="aluminum">
-    <color rgba="0.5 0.5 0.5 1"/>
-  </material>
   <xacro:macro name="sensor_r410" params="parent prefix *origin">
     <!-- camera body, with origin at bottom screw mount -->
@@ -41,5 +38,7 @@
           <!-- <mesh filename="package://realsense2_camera/meshes/r410/r410.dae" /> -->
         </geometry>
-        <material name="aluminum"/>
+        <material name="aluminum">
+          <color rgba="0.5 0.5 0.5 1"/>
+        </material>
       </visual>
       <collision>
@@ -76,5 +75,5 @@
     </joint>
     <link name="${prefix}camera_left_ir_frame"/>
-    <joint name="camera_left_ir_optical_joint" type="fixed">
+    <joint name="${prefix}camera_left_ir_optical_joint" type="fixed">
       <origin xyz="0 0 0" rpy="${-M_PI/2} 0 ${-M_PI/2}" />
       <parent link="${prefix}camera_left_ir_frame" />
@@ -83,5 +82,5 @@
     <link name="${prefix}camera_left_ir_optical_frame"/>
     <!-- camera right IR joints and links -->
-    <joint name="camera_right_ir_joint" type="fixed">
+    <joint name="${prefix}camera_right_ir_joint" type="fixed">
       <origin xyz="0 ${r410_cam_depth_to_right_ir_offset} 0" rpy="0 0 0" />
       <parent link="${prefix}camera_depth_frame" />
@@ -89,5 +88,5 @@
     </joint>
     <link name="${prefix}camera_right_ir_frame"/>
-    <joint name="camera_right_ir_optical_joint" type="fixed">
+    <joint name="${prefix}camera_right_ir_optical_joint" type="fixed">
       <origin xyz="0 0 0" rpy="${-M_PI/2} 0 ${-M_PI/2}" />
       <parent link="${prefix}camera_right_ir_frame" />

File: realsense/realsense2_camera/urdf/_r430.urdf.xacro (robot description, xacro)
@@ -25,7 +25,4 @@
   <xacro:property name="r430_cam_depth_py" value="-0.035"/>
   <xacro:property name="r430_cam_depth_pz" value="0.028"/>
-  <material name="aluminum">
-    <color rgba="0.5 0.5 0.5 1"/>
-  </material>
   <xacro:macro name="sensor_r430" params="parent prefix *origin">
     <!-- camera body, with origin at bottom screw mount -->
@@ -42,5 +39,7 @@
           <!--<mesh filename="package://realsense2_camera/meshes/r430/r430.dae" />-->
         </geometry>
-        <material name="aluminum"/>
+        <material name="aluminum">
+          <color rgba="0.5 0.5 0.5 1"/>
+        </material>
       </visual>
       <collision>
