Commit message: Fix package name in xacro files

File: o2as_new_parts_description/urdf/templates/assembly_template.urdf.xacro (robot description, xacro)
@@ -1,3 +1,3 @@
 <robot xmlns:xacro="http://www.ros.org/wiki/xacro" name="full_assembly">
-  <xacro:include filename="$(find o2as_parts_description)/urdf/assembly_parts_macros.urdf.xacro"/>
+  <xacro:include filename="$(find o2as_new_parts_description)/urdf/assembly_parts_macros.urdf.xacro"/>
   <xacro:macro name="full_assembly" params="prefix parent *origin">

File: o2as_new_parts_description/urdf/templates/macro_template.urdf.xacro (robot description, xacro)
@@ -5,5 +5,5 @@
         <origin rpy="1.5707 0 0" xyz="0 0 0"/>
         <geometry>
-          <mesh filename="package://o2as_parts_description/meshes/PARTNAME.dae" scale="0.001 0.001 0.001"/>
+          <mesh filename="package://o2as_new_parts_description/meshes/PARTNAME.dae" scale="0.001 0.001 0.001"/>
         </geometry>
         <material name="white">
@@ -14,5 +14,5 @@
         <origin rpy="1.5707 0 0" xyz="0 0 0"/>
         <geometry>
-          <mesh filename="package://o2as_parts_description/meshes/PARTNAME.vhacd.dae" scale="0.001 0.001 0.001"/>
+          <mesh filename="package://o2as_new_parts_description/meshes/PARTNAME.vhacd.dae" scale="0.001 0.001 0.001"/>
         </geometry>
       </collision>

File: o2as_new_parts_description/urdf/templates/non_macro_template.urdf.xacro (robot description, xacro)
@@ -1,4 +1,4 @@
 <robot xmlns:xacro="http://www.ros.org/wiki/xacro" name="MACRONAME_EXTERNAL">
-  <xacro:include filename="$(find o2as_parts_description)/urdf/generated/PARTNAME_macro.urdf.xacro"/>
+  <xacro:include filename="$(find o2as_new_parts_description)/urdf/generated/PARTNAME_macro.urdf.xacro"/>
   <xacro:MACRONAME_EXTERNAL prefix="" parent="world" spawn_attached="false">
     <origin rpy="0 0 0" xyz="0 0 0"/>

File: o2as_new_parts_description/urdf/templates/spawn_template.urdf (robot description, URDF)
Before this commit: robot PARTNAME, 1 links, 0 joints
Links:
- link baseLink: geometry collision mesh filename=/root/catkin_ws/src/o2as_new_parts_description/meshes/PARTN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 scale=0.001 0.001 0.001; visual mesh filename=/root/catkin_ws/src/o2as_new_parts_description/meshes/PARTN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 scale=0.001 0.001 0.001
