Commit message: Add frames of kitting tray corner.

File: aist_scene_description/urdf/kitting_tray_with_partitions.xacro (robot description, xacro)
@@ -5,4 +5,5 @@
   <xacro:property name="tray_width" value=".300" />
   <xacro:property name="tray_length" value=".210" />
+  <xacro:property name="tray_height" value=".023" />
   <xacro:property name="mesh_offset_x" value="-.045" />
   <xacro:property name="mesh_offset_y" value=".045" />
@@ -40,4 +41,28 @@
       <xacro:insert_block name="origin"/>
     </joint>
+    <joint name="${trayname}_top_front_right_corner_joint" type="fixed">
+      <parent link="${trayname}"/>
+      <child link="${trayname}_top_front_right_corner"/>
+      <origin rpy="0.0 0.0 0.0" xyz="${tray_width} ${tray_length} ${tray_height} "/>
+    </joint>
+    <link name="${trayname}_top_front_right_corner"/>
+    <joint name="${trayname}_top_back_right_corner_joint" type="fixed">
+      <parent link="${trayname}"/>
+      <child link="${trayname}_top_back_right_corner"/>
+      <origin rpy="0.0 0.0 0.0" xyz="0 ${tray_length} ${tray_height} "/>
+    </joint>
+    <link name="${trayname}_top_back_right_corner"/>
+    <joint name="${trayname}_top_back_left_corner_joint" type="fixed">
+      <parent link="${trayname}"/>
+      <child link="${trayname}_top_back_left_corner"/>
+      <origin rpy="0.0 0.0 0.0" xyz="0 0 ${tray_height} "/>
+    </joint>
+    <link name="${trayname}_top_back_left_corner"/>
+    <joint name="${trayname}_top_front_left_corner_joint" type="fixed">
+      <parent link="${trayname}"/>
+      <child link="${trayname}_top_front_left_corner"/>
+      <origin rpy="0.0 0.0 0.0" xyz="${tray_width} 0 ${tray_height} "/>
+    </joint>
+    <link name="${trayname}_top_front_left_corner"/>
   </xacro:macro>
   <!-- ========== -->
