Commit message: Add trays in kitting scene.

File: aist_scene_description/urdf/aist_kitting_scene.xacro (robot description, xacro)
@@ -1,5 +1,27 @@
 <?xml version="1.0"?>
-<robot xmlns:xacro="http://www.ros.org/wiki/xacro" name="kitting_scene">
-  <xacro:include filename="$(find o2as_scene_description)/urdf/kitting_tray_with_partitions.xacro" />
+<robot xmlns:xacro="http://www.ros.org/wiki/xacro" name="aist_kitting_scene">
+  <xacro:include filename="$(find aist_scene_description)/urdf/kitting_tray_with_partitions.xacro" />
   <xacro:include filename="$(find o2as_scene_description)/urdf/o2as_box.xacro" />
+  <xacro:property name="tray_width" value=".210" />
+  <xacro:property name="tray_length" value=".300" />
+  <xacro:property name="tray_rack_width" value=".210" />
+  <xacro:property name="tray_rack_length" value=".600" />
+  <xacro:property name="tray_rack_height" value=".015" />
+  <!-- add tray rack -->
+  <xacro:o2as_box boxname="rack_trays" box_w="${tray_rack_width}" box_l="${tray_rack_length}" box_h="${tray_rack_height}" parent="workspace_center">
+    <origin xyz="-.299 ${-tray_rack_length/2}  0" rpy="0 0 0" />
+  </xacro:o2as_box>
+  <link name="tray_rack_center" />
+  <joint name="tray_rack_joint" type="fixed">
+    <parent link="workspace_center" />
+    <child link="tray_rack_center"/>
+    <origin xyz="${-.299+tray_rack_width/2} 0 ${tray_rack_height}" rpy="0 0 0"/>
+  </joint>
+  <!-- add trays -->
+  <xacro:kitting_tray1 trayname="set_1_tray_1" parent="tray_rack_center">
+    <origin xyz="${-tray_rack_width/2} ${-tray_rack_length/2} 0" rpy="0 0 0" />
+  </xacro:kitting_tray1>
+  <xacro:kitting_tray2 trayname="set_1_tray_2" parent="tray_rack_center">
+    <origin xyz="${-tray_rack_width/2} 0 0" rpy="0 0 0" />
+  </xacro:kitting_tray2>
 </robot>

Commit message: Add bins rack in kitting scene.

File: aist_scene_description/urdf/aist_kitting_scene.xacro (robot description, xacro)
@@ -8,6 +8,18 @@
   <xacro:property name="tray_rack_length" value=".600" />
   <xacro:property name="tray_rack_height" value=".015" />
-  <!-- add tray rack -->
-  <xacro:o2as_box boxname="rack_trays" box_w="${tray_rack_width}" box_l="${tray_rack_length}" box_h="${tray_rack_height}" parent="workspace_center">
+  <xacro:property name="bin_rack_width" value=".420" />
+  <xacro:property name="bin_rack_length" value=".680" />
+  <xacro:property name="bin_rack_height" value=".015" />
+  <!-- add racks -->
+  <xacro:o2as_box boxname="bin_rack" box_w="${bin_rack_width}" box_l="${bin_rack_length}" box_h="${bin_rack_height}" parent="workspace_center">
+    <origin xyz="0 ${-bin_rack_length/2}  0" rpy="0 0 0" />
+  </xacro:o2as_box>
+  <link name="bin_rack_center" />
+  <joint name="bin_rack_joint" type="fixed">
+    <parent link="workspace_center" />
+    <child link="bin_rack_center"/>
+    <origin xyz="${bin_rack_width/2} 0 ${bin_rack_height}" rpy="0 0 0"/>
+  </joint>
+  <xacro:o2as_box boxname="tray_rack" box_w="${tray_rack_width}" box_l="${tray_rack_length}" box_h="${tray_rack_height}" parent="workspace_center">
     <origin xyz="-.299 ${-tray_rack_length/2}  0" rpy="0 0 0" />
   </xacro:o2as_box>

Commit message: Add bin rack calibration.

File: aist_scene_description/urdf/aist_kitting_scene.xacro (robot description, xacro)
@@ -1,7 +1,7 @@
 <?xml version="1.0"?>
 <robot xmlns:xacro="http://www.ros.org/wiki/xacro" name="aist_kitting_scene">
-  <xacro:include filename="$(find aist_scene_description)/urdf/kitting_bins.xacro" />
   <xacro:include filename="$(find aist_scene_description)/urdf/kitting_tray_with_partitions.xacro" />
   <xacro:include filename="$(find o2as_scene_description)/urdf/o2as_box.xacro" />
+  <!-- <xacro:include filename="$(find aist_scene_description)/urdf/kitting_bins.xacro" /> -->
   <xacro:property name="tray_width" value=".210" />
   <xacro:property name="tray_length" value=".300" />
@@ -12,5 +12,5 @@
   <xacro:property name="bin_rack_length" value=".680" />
   <xacro:property name="bin_rack_height" value=".015" />
-  <!-- add racks -->
+  <!-- add bin rack -->
   <xacro:o2as_box boxname="bin_rack" box_w="${bin_rack_width}" box_l="${bin_rack_length}" box_h="${bin_rack_height}" parent="workspace_center">
     <origin xyz="0 ${-bin_rack_length/2}  0" rpy="0 0 0" />
@@ -22,4 +22,29 @@
     <origin xyz="${bin_rack_width/2} 0 ${bin_rack_height}" rpy="0 0 0"/>
   </joint>
+  <joint name="bin_rack_top_front_right_corner_joint" type="fixed">
+    <parent link="bin_rack_center"/>
+    <child link="bin_rack_top_front_right_corner"/>
+    <origin rpy="0.0 0.0 0.0" xyz="${bin_rack_width/2} ${bin_rack_length/2} 0 "/>
+  </joint>
+  <link name="bin_rack_top_front_right_corner"/>
+  <joint name="bin_rack_top_back_right_corner_joint" type="fixed">
+    <parent link="bin_rack_center"/>
+    <child link="bin_rack_top_back_right_corner"/>
+    <origin rpy="0.0 0.0 0.0" xyz="${-bin_rack_width/2} ${bin_rack_length/2} 0 "/>
+  </joint>
+  <link name="bin_rack_top_back_right_corner"/>
+  <joint name="bin_rack_top_back_left_corner_joint" type="fixed">
+    <parent link="bin_rack_center"/>
+    <child link="bin_rack_top_back_left_corner"/>
+    <origin rpy="0.0 0.0 0.0" xyz="${-bin_rack_width/2} ${-bin_rack_length/2} 0 "/>
+  </joint>
+  <link name="bin_rack_top_back_left_corner"/>
+  <joint name="bin_rack_top_front_left_corner_joint" type="fixed">
+    <parent link="bin_rack_center"/>
+    <child link="bin_rack_top_front_left_corner"/>
+    <origin rpy="0.0 0.0 0.0" xyz="${bin_rack_width/2} ${-bin_rack_length/2} 0 "/>
+  </joint>
+  <link name="bin_rack_top_front_left_corner"/>
+  <!-- add tray rack -->
   <xacro:o2as_box boxname="tray_rack" box_w="${tray_rack_width}" box_l="${tray_rack_length}" box_h="${tray_rack_height}" parent="workspace_center">
     <origin xyz="-.299 ${-tray_rack_length/2}  0" rpy="0 0 0" />
@@ -31,4 +56,28 @@
     <origin xyz="${-.299+tray_rack_width/2} 0 ${tray_rack_height}" rpy="0 0 0"/>
   </joint>
+  <joint name="tray_rack_top_front_right_corner_joint" type="fixed">
+    <parent link="tray_rack_center"/>
+    <child link="tray_rack_top_front_right_corner"/>
+    <origin rpy="0.0 0.0 0.0" xyz="${tray_rack_width/2} ${tray_rack_length/2} 0 "/>
+  </joint>
+  <link name="tray_rack_top_front_right_corner"/>
+  <joint name="tray_rack_top_back_right_corner_joint" type="fixed">
+    <parent link="tray_rack_center"/>
+    <child link="tray_rack_top_back_right_corner"/>
+    <origin rpy="0.0 0.0 0.0" xyz="${-tray_rack_width/2} ${tray_rack_length/2} 0 "/>
+  </joint>
+  <link name="tray_rack_top_back_right_corner"/>
+  <joint name="tray_rack_top_back_left_corner_joint" type="fixed">
+    <parent link="tray_rack_center"/>
+    <child link="tray_rack_top_back_left_corner"/>
+    <origin rpy="0.0 0.0 0.0" xyz="${-tray_rack_width/2} ${-tray_rack_length/2} 0 "/>
+  </joint>
+  <link name="tray_rack_top_back_left_corner"/>
+  <joint name="tray_rack_top_front_left_corner_joint" type="fixed">
+    <parent link="tray_rack_center"/>
+    <child link="tray_rack_top_front_left_corner"/>
+    <origin rpy="0.0 0.0 0.0" xyz="${tray_rack_width/2} ${-tray_rack_length/2} 0 "/>
+  </joint>
+  <link name="tray_rack_top_front_left_corner"/>
   <!-- add trays -->
   <xacro:kitting_tray1 trayname="set_1_tray_1" parent="tray_rack_center">

Commit message: Calibrated aist kitting scene.

File: aist_scene_description/urdf/aist_kitting_scene.xacro (robot description, xacro)
@@ -3,5 +3,5 @@
   <xacro:include filename="$(find aist_scene_description)/urdf/kitting_tray_with_partitions.xacro" />
   <xacro:include filename="$(find o2as_scene_description)/urdf/o2as_box.xacro" />
-  <!-- <xacro:include filename="$(find aist_scene_description)/urdf/kitting_bins.xacro" /> -->
+  <xacro:include filename="$(find aist_scene_description)/urdf/kitting_bins.xacro" />
   <xacro:property name="tray_width" value=".210" />
   <xacro:property name="tray_length" value=".300" />

File: aist_scene_description/urdf/kitting_bins.xacro (robot description, xacro)
@@ -17,50 +17,50 @@
   <xacro:property name="z_origin_offset_3" value="-.004" />
   <!-- A row of bin1 -->
-  <xacro:property name="set1_x" value="-0.1005"/>
-  <xacro:property name="set1_y" value="0.280"/>
+  <xacro:property name="set1_x" value="-0.1095"/>
+  <xacro:property name="set1_y" value="0.34"/>
   <xacro:property name="set1_z" value="0"/>
   <!-- A row of bin2 -->
-  <xacro:property name="set2_x" value=".064"/>
-  <xacro:property name="set2_y" value="0.3125"/>
+  <xacro:property name="set2_x" value=".055"/>
+  <xacro:property name="set2_y" value="0.34"/>
   <xacro:property name="set2_z" value="0"/>
   <!--bin2_5_-->
   <xacro:kitting_bin_2 binname="bin2_5" parent="bin_rack_center" z_origin_offset="-.008">
-    <origin xyz="-0.1005 0.224 0.008" rpy="0 0 0" />
+    <origin xyz="-0.1095 0.284 0.008" rpy="0 0 0" />
   </xacro:kitting_bin_2>
   <!--bin2_4_-->
   <xacro:kitting_bin_2 binname="bin2_4" parent="bin_rack_center" z_origin_offset="-.008">
-    <origin xyz="-0.1005 0.112 0.008" rpy="0 0 0" />
+    <origin xyz="-0.1095 0.172 0.008" rpy="0 0 0" />
   </xacro:kitting_bin_2>
   <!--bin2_1_-->
   <xacro:kitting_bin_2 binname="bin2_1" parent="bin_rack_center" z_origin_offset="-.008">
-    <origin xyz="-0.1005 4.16333634234e-17 0.008" rpy="0 0 0" />
+    <origin xyz="-0.1095 0.06 0.008" rpy="0 0 0" />
   </xacro:kitting_bin_2>
   <!--bin2_3_-->
   <xacro:kitting_bin_2 binname="bin2_3" parent="bin_rack_center" z_origin_offset="-.008">
-    <origin xyz="-0.1005 -0.112 0.008" rpy="0 0 0" />
+    <origin xyz="-0.1095 -0.052 0.008" rpy="0 0 0" />
   </xacro:kitting_bin_2>
   <!--bin2_2_-->
   <xacro:kitting_bin_2 binname="bin2_2" parent="bin_rack_center" z_origin_offset="-.008">
-    <origin xyz="-0.1005 -0.224 0.008" rpy="0 0 0" />
+    <origin xyz="-0.1095 -0.164 0.008" rpy="0 0 0" />
   </xacro:kitting_bin_2>
   <!--bin1_3_-->
   <xacro:kitting_bin_1 binname="bin1_3" parent="bin_rack_center" z_origin_offset="-.005">
-    <origin xyz=".064 0.25 0.005" rpy="0 0 0" />
+    <origin xyz=".055 0.2775 0.005" rpy="0 0 0" />
   </xacro:kitting_bin_1>
   <!--bin1_4_-->
   <xacro:kitting_bin_1 binname="bin1_4" parent="bin_rack_center" z_origin_offset="-.005">
-    <origin xyz=".064 0.125 0.005" rpy="0 0 0" />
+    <origin xyz=".055 0.1525 0.005" rpy="0 0 0" />
   </xacro:kitting_bin_1>
   <!--bin1_5_-->
   <xacro:kitting_bin_1 binname="bin1_5" parent="bin_rack_center" z_origin_offset="-.005">
-    <origin xyz=".064 0.0 0.005" rpy="0 0 0" />
+    <origin xyz=".055 0.0275 0.005" rpy="0 0 0" />
   </xacro:kitting_bin_1>
   <!--bin1_2_-->
   <xacro:kitting_bin_1 binname="bin1_2" parent="bin_rack_center" z_origin_offset="-.005">
-    <origin xyz=".064 -0.125 0.005" rpy="0 0 0" />
+    <origin xyz=".055 -0.0975 0.005" rpy="0 0 0" />
   </xacro:kitting_bin_1>
   <!--bin1_1_-->
   <xacro:kitting_bin_1 binname="bin1_1" parent="bin_rack_center" z_origin_offset="-.005">
-    <origin xyz=".064 -0.25 0.005" rpy="0 0 0" />
+    <origin xyz=".055 -0.2225 0.005" rpy="0 0 0" />
   </xacro:kitting_bin_1>
 </robot>

Commit message: Add bins to place all items for experiments.

File: aist_scene_description/urdf/aist_kitting_scene.xacro (robot description, xacro)
@@ -4,4 +4,5 @@
   <xacro:include filename="$(find o2as_scene_description)/urdf/o2as_box.xacro" />
   <xacro:include filename="$(find aist_scene_description)/urdf/kitting_bins.xacro" />
+  <xacro:include filename="$(find o2as_scene_description)/urdf/kitting_bin_macros.xacro" />
   <xacro:property name="tray_width" value=".210" />
   <xacro:property name="tray_length" value=".300" />
@@ -81,9 +82,12 @@
   <link name="tray_rack_top_front_left_corner"/>
   <!-- add trays -->
-  <xacro:kitting_tray1 trayname="set_1_tray_1" parent="tray_rack_center">
+  <!-- <xacro:kitting_tray1 trayname="set_1_tray_1" parent="tray_rack_center">
     <origin xyz="${-tray_rack_width/2} ${-tray_rack_length/2} 0" rpy="0 0 0" />
   </xacro:kitting_tray1>
   <xacro:kitting_tray2 trayname="set_1_tray_2" parent="tray_rack_center">
     <origin xyz="${-tray_rack_width/2} 0 0" rpy="0 0 0" />
-  </xacro:kitting_tray2>
+  </xacro:kitting_tray2> -->
+  <xacro:kitting_bin_3 binname="place_bin" parent="tray_rack_center" z_origin_offset="-.004">
+    <origin xyz="0 0 0.004" rpy="0 0 ${pi/2}" />
+  </xacro:kitting_bin_3>
 </robot>

Commit message: Fixed bump bin orientation.

File: aist_scene_description/urdf/aist_kitting_scene.xacro (robot description, xacro)
@@ -89,5 +89,5 @@
   </xacro:kitting_tray2> -->
   <xacro:kitting_bin_3 binname="place_bin" parent="tray_rack_center" z_origin_offset="-.004">
-    <origin xyz="0 0 0.004" rpy="0 0 ${pi/2}" />
+    <origin xyz="0 0 0.004" rpy="0 0 -${pi/2}" />
   </xacro:kitting_bin_3>
 </robot>

Commit message: Fixed small changes

File: aist_scene_description/urdf/aist_kitting_scene.xacro (robot description, xacro)
@@ -14,5 +14,5 @@
   <xacro:property name="bin_rack_height" value=".015" />
   <!-- add bin rack -->
-  <xacro:o2as_box boxname="bin_rack" box_w="${bin_rack_width}" box_l="${bin_rack_length}" box_h="${bin_rack_height}" parent="workspace_center">
+  <!-- <xacro:o2as_box boxname="bin_rack" box_w="${bin_rack_width}" box_l="${bin_rack_length}" box_h="${bin_rack_height}" parent="workspace_center">
     <origin xyz="0 ${-bin_rack_length/2}  0" rpy="0 0 0" />
   </xacro:o2as_box>
@@ -46,7 +46,7 @@
     <origin rpy="0.0 0.0 0.0" xyz="${bin_rack_width/2} ${-bin_rack_length/2} 0 "/>
   </joint>
-  <link name="bin_rack_top_front_left_corner"/>
+  <link name="bin_rack_top_front_left_corner"/> -->
   <!-- add tray rack -->
-  <xacro:o2as_box boxname="tray_rack" box_w="${tray_rack_width}" box_l="${tray_rack_length}" box_h="${tray_rack_height}" parent="workspace_center">
+  <!-- <xacro:o2as_box boxname="tray_rack" box_w="${tray_rack_width}" box_l="${tray_rack_length}" box_h="${tray_rack_height}" parent="workspace_center">
     <origin xyz="-.299 ${-tray_rack_length/2}  0" rpy="0 0 0" />
   </xacro:o2as_box>
@@ -80,5 +80,5 @@
     <origin rpy="0.0 0.0 0.0" xyz="${tray_rack_width/2} ${-tray_rack_length/2} 0 "/>
   </joint>
-  <link name="tray_rack_top_front_left_corner"/>
+  <link name="tray_rack_top_front_left_corner"/> -->
   <!-- add trays -->
   <!-- <xacro:kitting_tray1 trayname="set_1_tray_1" parent="tray_rack_center">
@@ -88,6 +88,6 @@
     <origin xyz="${-tray_rack_width/2} 0 0" rpy="0 0 0" />
   </xacro:kitting_tray2> -->
-  <xacro:kitting_bin_3 binname="place_bin" parent="tray_rack_center" z_origin_offset="-.004">
-    <origin xyz="0 0 0.004" rpy="0 0 -${pi/2}" />
+  <xacro:kitting_bin_3 binname="place_bin" parent="workspace_center" z_origin_offset="-.004">
+    <origin xyz="-.20 0 0.004" rpy="0 0 -${pi/2}" />
   </xacro:kitting_bin_3>
 </robot>

File: aist_scene_description/urdf/kitting_bins.xacro (robot description, xacro)
@@ -21,6 +21,6 @@
   <xacro:property name="set1_z" value="0"/>
   <!--bin_3_part_5_-->
-  <xacro:kitting_bin_3 binname="bin_3_part_5" parent="bin_rack_center" z_origin_offset="-.004">
-    <origin xyz="0 0.0 0.004" rpy="0 0 0" />
+  <xacro:kitting_bin_3 binname="bin_3_part_12" parent="workspace_center" z_origin_offset="-.004">
+    <origin xyz=".15 0.0 0.004" rpy="0 0 0" />
   </xacro:kitting_bin_3>
 </robot>
