Commit message: Fixed bin name definition.

File: aist_scene_description/urdf/kitting_bins.xacro (robot description, xacro)
@@ -5,14 +5,14 @@
   <!-- space for bin -->
   <!-- bin1_definition -->
-  <xacro:property name="bin1_width" value="0.125"/>
-  <xacro:property name="bin1_length" value="0.128"/>
+  <xacro:property name="bin_1_width" value="0.125"/>
+  <xacro:property name="bin_1_length" value="0.128"/>
   <xacro:property name="z_origin_offset_1" value="-.005" />
   <!-- bin2_definition -->
-  <xacro:property name="bin2_width" value="0.112"/>
-  <xacro:property name="bin2_length" value="0.201"/>
+  <xacro:property name="bin_2_width" value="0.112"/>
+  <xacro:property name="bin_2_length" value="0.201"/>
   <xacro:property name="z_origin_offset_2" value="-.008" />
   <!-- bin3_definition -->
-  <xacro:property name="bin3_width" value="0.192"/>
-  <xacro:property name="bin3_length" value="0.285"/>
+  <xacro:property name="bin_3_width" value="0.192"/>
+  <xacro:property name="bin_3_length" value="0.285"/>
   <xacro:property name="z_origin_offset_3" value="-.004" />
   <!-- A row of bin1 -->
@@ -24,42 +24,42 @@
   <xacro:property name="set2_y" value="0.34"/>
   <xacro:property name="set2_z" value="0"/>
-  <!--bin2_5_-->
-  <xacro:kitting_bin_2 binname="bin2_5" parent="bin_rack_center" z_origin_offset="-.008">
+  <!--bin_2_part_11_-->
+  <xacro:kitting_bin_2 binname="bin_2_part_11" parent="bin_rack_center" z_origin_offset="-.008">
     <origin xyz="-0.1095 0.284 0.008" rpy="0 0 0" />
   </xacro:kitting_bin_2>
-  <!--bin2_4_-->
-  <xacro:kitting_bin_2 binname="bin2_4" parent="bin_rack_center" z_origin_offset="-.008">
+  <!--bin_2_part_8_-->
+  <xacro:kitting_bin_2 binname="bin_2_part_8" parent="bin_rack_center" z_origin_offset="-.008">
     <origin xyz="-0.1095 0.172 0.008" rpy="0 0 0" />
   </xacro:kitting_bin_2>
-  <!--bin2_1_-->
-  <xacro:kitting_bin_2 binname="bin2_1" parent="bin_rack_center" z_origin_offset="-.008">
+  <!--bin_2_part_4_-->
+  <xacro:kitting_bin_2 binname="bin_2_part_4" parent="bin_rack_center" z_origin_offset="-.008">
     <origin xyz="-0.1095 0.06 0.008" rpy="0 0 0" />
   </xacro:kitting_bin_2>
-  <!--bin2_3_-->
-  <xacro:kitting_bin_2 binname="bin2_3" parent="bin_rack_center" z_origin_offset="-.008">
+  <!--bin_2_part_7_-->
+  <xacro:kitting_bin_2 binname="bin_2_part_7" parent="bin_rack_center" z_origin_offset="-.008">
     <origin xyz="-0.1095 -0.052 0.008" rpy="0 0 0" />
   </xacro:kitting_bin_2>
-  <!--bin2_2_-->
-  <xacro:kitting_bin_2 binname="bin2_2" parent="bin_rack_center" z_origin_offset="-.008">
+  <!--bin_2_part_5_-->
+  <xacro:kitting_bin_2 binname="bin_2_part_5" parent="bin_rack_center" z_origin_offset="-.008">
     <origin xyz="-0.1095 -0.164 0.008" rpy="0 0 0" />
   </xacro:kitting_bin_2>
-  <!--bin1_3_-->
-  <xacro:kitting_bin_1 binname="bin1_3" parent="bin_rack_center" z_origin_offset="-.005">
+  <!--bin_1_part_16_-->
+  <xacro:kitting_bin_1 binname="bin_1_part_16" parent="bin_rack_center" z_origin_offset="-.005">
     <origin xyz=".055 0.2775 0.005" rpy="0 0 0" />
   </xacro:kitting_bin_1>
-  <!--bin1_4_-->
-  <xacro:kitting_bin_1 binname="bin1_4" parent="bin_rack_center" z_origin_offset="-.005">
+  <!--bin_1_part_17_-->
+  <xacro:kitting_bin_1 binname="bin_1_part_17" parent="bin_rack_center" z_origin_offset="-.005">
     <origin xyz=".055 0.1525 0.005" rpy="0 0 0" />
   </xacro:kitting_bin_1>
-  <!--bin1_5_-->
-  <xacro:kitting_bin_1 binname="bin1_5" parent="bin_rack_center" z_origin_offset="-.005">
+  <!--bin_1_part_18_-->
+  <xacro:kitting_bin_1 binname="bin_1_part_18" parent="bin_rack_center" z_origin_offset="-.005">
     <origin xyz=".055 0.0275 0.005" rpy="0 0 0" />
   </xacro:kitting_bin_1>
-  <!--bin1_2_-->
-  <xacro:kitting_bin_1 binname="bin1_2" parent="bin_rack_center" z_origin_offset="-.005">
+  <!--bin_1_part_15_-->
+  <xacro:kitting_bin_1 binname="bin_1_part_15" parent="bin_rack_center" z_origin_offset="-.005">
     <origin xyz=".055 -0.0975 0.005" rpy="0 0 0" />
   </xacro:kitting_bin_1>
-  <!--bin1_1_-->
-  <xacro:kitting_bin_1 binname="bin1_1" parent="bin_rack_center" z_origin_offset="-.005">
+  <!--bin_1_part_10_-->
+  <xacro:kitting_bin_1 binname="bin_1_part_10" parent="bin_rack_center" z_origin_offset="-.005">
     <origin xyz=".055 -0.2225 0.005" rpy="0 0 0" />
   </xacro:kitting_bin_1>

Commit message: Before experiment.

File: aist_scene_description/urdf/kitting_bins.xacro (robot description, xacro)
@@ -24,42 +24,42 @@
   <xacro:property name="set2_y" value="0.34"/>
   <xacro:property name="set2_z" value="0"/>
-  <!--bin_2_part_11_-->
-  <xacro:kitting_bin_2 binname="bin_2_part_11" parent="bin_rack_center" z_origin_offset="-.008">
+  <!--bin_2_part_a_-->
+  <xacro:kitting_bin_2 binname="bin_2_part_a" parent="bin_rack_center" z_origin_offset="-.008">
     <origin xyz="-0.1095 0.284 0.008" rpy="0 0 0" />
+  </xacro:kitting_bin_2>
+  <!--bin_2_part_4_-->
+  <xacro:kitting_bin_2 binname="bin_2_part_4" parent="bin_rack_center" z_origin_offset="-.008">
+    <origin xyz="-0.1095 0.172 0.008" rpy="0 0 0" />
   </xacro:kitting_bin_2>
   <!--bin_2_part_7_-->
   <xacro:kitting_bin_2 binname="bin_2_part_7" parent="bin_rack_center" z_origin_offset="-.008">
-    <origin xyz="-0.1095 0.172 0.008" rpy="0 0 0" />
-  </xacro:kitting_bin_2>
-  <!--bin_2_part_4_-->
-  <xacro:kitting_bin_2 binname="bin_2_part_4" parent="bin_rack_center" z_origin_offset="-.008">
     <origin xyz="-0.1095 0.06 0.008" rpy="0 0 0" />
   </xacro:kitting_bin_2>
-  <!--bin_2_part_8_-->
-  <xacro:kitting_bin_2 binname="bin_2_part_8" parent="bin_rack_center" z_origin_offset="-.008">
+  <!--bin_2_part_11_-->
+  <xacro:kitting_bin_2 binname="bin_2_part_11" parent="bin_rack_center" z_origin_offset="-.008">
     <origin xyz="-0.1095 -0.052 0.008" rpy="0 0 0" />
   </xacro:kitting_bin_2>
-  <!--bin_2_part_5_-->
-  <xacro:kitting_bin_2 binname="bin_2_part_5" parent="bin_rack_center" z_origin_offset="-.008">
+  <!--bin_2_part_b_-->
+  <xacro:kitting_bin_2 binname="bin_2_part_b" parent="bin_rack_center" z_origin_offset="-.008">
     <origin xyz="-0.1095 -0.164 0.008" rpy="0 0 0" />
   </xacro:kitting_bin_2>
-  <!--bin_1_part_17_-->
-  <xacro:kitting_bin_1 binname="bin_1_part_17" parent="bin_rack_center" z_origin_offset="-.005">
+  <!--bin_1_part_13_-->
+  <xacro:kitting_bin_1 binname="bin_1_part_13" parent="bin_rack_center" z_origin_offset="-.005">
     <origin xyz=".055 0.2775 0.005" rpy="0 0 0" />
   </xacro:kitting_bin_1>
-  <!--bin_1_part_13_-->
-  <xacro:kitting_bin_1 binname="bin_1_part_13" parent="bin_rack_center" z_origin_offset="-.005">
+  <!--bin_1_part_8_-->
+  <xacro:kitting_bin_1 binname="bin_1_part_8" parent="bin_rack_center" z_origin_offset="-.005">
     <origin xyz=".055 0.1525 0.005" rpy="0 0 0" />
   </xacro:kitting_bin_1>
-  <!--bin_1_part_18_-->
-  <xacro:kitting_bin_1 binname="bin_1_part_18" parent="bin_rack_center" z_origin_offset="-.005">
+  <!--bin_1_part_12_-->
+  <xacro:kitting_bin_1 binname="bin_1_part_12" parent="bin_rack_center" z_origin_offset="-.005">
     <origin xyz=".055 0.0275 0.005" rpy="0 0 0" />
   </xacro:kitting_bin_1>
-  <!--bin_1_part_15_-->
-  <xacro:kitting_bin_1 binname="bin_1_part_15" parent="bin_rack_center" z_origin_offset="-.005">
+  <!--bin_1_part_5_-->
+  <xacro:kitting_bin_1 binname="bin_1_part_5" parent="bin_rack_center" z_origin_offset="-.005">
     <origin xyz=".055 -0.0975 0.005" rpy="0 0 0" />
   </xacro:kitting_bin_1>
-  <!--bin_1_part_10_-->
-  <xacro:kitting_bin_1 binname="bin_1_part_10" parent="bin_rack_center" z_origin_offset="-.005">
+  <!--bin_1_part_c_-->
+  <xacro:kitting_bin_1 binname="bin_1_part_c" parent="bin_rack_center" z_origin_offset="-.005">
     <origin xyz=".055 -0.2225 0.005" rpy="0 0 0" />
   </xacro:kitting_bin_1>

Commit message: Revert "Merge branch 'devel-aist' of https://gitlab.com/o2as-aist/ur-o2as into devel-aist"
This reverts commit 44e027a7c2db3c285216a34916cff8fe35f59b8d.

File: aist_scene_description/urdf/kitting_bins.xacro (robot description, xacro)
@@ -24,42 +24,42 @@
   <xacro:property name="set2_y" value="0.34"/>
   <xacro:property name="set2_z" value="0"/>
-  <!--bin_2_part_a_-->
-  <xacro:kitting_bin_2 binname="bin_2_part_a" parent="bin_rack_center" z_origin_offset="-.008">
+  <!--bin_2_part_11_-->
+  <xacro:kitting_bin_2 binname="bin_2_part_11" parent="bin_rack_center" z_origin_offset="-.008">
     <origin xyz="-0.1095 0.284 0.008" rpy="0 0 0" />
+  </xacro:kitting_bin_2>
+  <!--bin_2_part_8_-->
+  <xacro:kitting_bin_2 binname="bin_2_part_8" parent="bin_rack_center" z_origin_offset="-.008">
+    <origin xyz="-0.1095 0.172 0.008" rpy="0 0 0" />
   </xacro:kitting_bin_2>
   <!--bin_2_part_4_-->
   <xacro:kitting_bin_2 binname="bin_2_part_4" parent="bin_rack_center" z_origin_offset="-.008">
-    <origin xyz="-0.1095 0.172 0.008" rpy="0 0 0" />
+    <origin xyz="-0.1095 0.06 0.008" rpy="0 0 0" />
   </xacro:kitting_bin_2>
   <!--bin_2_part_7_-->
   <xacro:kitting_bin_2 binname="bin_2_part_7" parent="bin_rack_center" z_origin_offset="-.008">
-    <origin xyz="-0.1095 0.06 0.008" rpy="0 0 0" />
-  </xacro:kitting_bin_2>
-  <!--bin_2_part_11_-->
-  <xacro:kitting_bin_2 binname="bin_2_part_11" parent="bin_rack_center" z_origin_offset="-.008">
     <origin xyz="-0.1095 -0.052 0.008" rpy="0 0 0" />
   </xacro:kitting_bin_2>
-  <!--bin_2_part_b_-->
-  <xacro:kitting_bin_2 binname="bin_2_part_b" parent="bin_rack_center" z_origin_offset="-.008">
+  <!--bin_2_part_5_-->
+  <xacro:kitting_bin_2 binname="bin_2_part_5" parent="bin_rack_center" z_origin_offset="-.008">
     <origin xyz="-0.1095 -0.164 0.008" rpy="0 0 0" />
   </xacro:kitting_bin_2>
-  <!--bin_1_part_13_-->
-  <xacro:kitting_bin_1 binname="bin_1_part_13" parent="bin_rack_center" z_origin_offset="-.005">
+  <!--bin_1_part_16_-->
+  <xacro:kitting_bin_1 binname="bin_1_part_16" parent="bin_rack_center" z_origin_offset="-.005">
     <origin xyz=".055 0.2775 0.005" rpy="0 0 0" />
   </xacro:kitting_bin_1>
-  <!--bin_1_part_8_-->
-  <xacro:kitting_bin_1 binname="bin_1_part_8" parent="bin_rack_center" z_origin_offset="-.005">
+  <!--bin_1_part_17_-->
+  <xacro:kitting_bin_1 binname="bin_1_part_17" parent="bin_rack_center" z_origin_offset="-.005">
     <origin xyz=".055 0.1525 0.005" rpy="0 0 0" />
   </xacro:kitting_bin_1>
-  <!--bin_1_part_12_-->
-  <xacro:kitting_bin_1 binname="bin_1_part_12" parent="bin_rack_center" z_origin_offset="-.005">
+  <!--bin_1_part_18_-->
+  <xacro:kitting_bin_1 binname="bin_1_part_18" parent="bin_rack_center" z_origin_offset="-.005">
     <origin xyz=".055 0.0275 0.005" rpy="0 0 0" />
   </xacro:kitting_bin_1>
-  <!--bin_1_part_5_-->
-  <xacro:kitting_bin_1 binname="bin_1_part_5" parent="bin_rack_center" z_origin_offset="-.005">
+  <!--bin_1_part_15_-->
+  <xacro:kitting_bin_1 binname="bin_1_part_15" parent="bin_rack_center" z_origin_offset="-.005">
     <origin xyz=".055 -0.0975 0.005" rpy="0 0 0" />
   </xacro:kitting_bin_1>
-  <!--bin_1_part_c_-->
-  <xacro:kitting_bin_1 binname="bin_1_part_c" parent="bin_rack_center" z_origin_offset="-.005">
+  <!--bin_1_part_10_-->
+  <xacro:kitting_bin_1 binname="bin_1_part_10" parent="bin_rack_center" z_origin_offset="-.005">
     <origin xyz=".055 -0.2225 0.005" rpy="0 0 0" />
   </xacro:kitting_bin_1>

Commit message: Prepare to check loading new kitting scene

File: aist_scene_description/urdf/kitting_bins.xacro (robot description, xacro)
@@ -20,7 +20,27 @@
   <xacro:property name="set1_y" value="0.096"/>
   <xacro:property name="set1_z" value="0"/>
-  <!--bin_3_part_8_-->
-  <xacro:kitting_bin_3 binname="bin_3_part_4" parent="workspace_center" z_origin_offset="-.004">
-    <origin xyz=".15 0.1 0.004" rpy="0 0 0" />
+  <!-- A row of bin2 -->
+  <xacro:property name="set2_x" value="0.25"/>
+  <xacro:property name="set2_y" value="0.096"/>
+  <xacro:property name="set2_z" value="0"/>
+  <!--bin_2_part_4_-->
+  <xacro:kitting_bin_2 binname="bin_2_part_4" parent="workspace_center" z_origin_offset="-.008">
+    <origin xyz="0 0.04 0.008" rpy="0 0 0" />
+  </xacro:kitting_bin_2>
+  <!--bin_2_part_7_-->
+  <xacro:kitting_bin_2 binname="bin_2_part_7" parent="workspace_center" z_origin_offset="-.008">
+    <origin xyz="0 -0.072 0.008" rpy="0 0 0" />
+  </xacro:kitting_bin_2>
+  <!--bin_2_part_8_-->
+  <xacro:kitting_bin_2 binname="bin_2_part_8" parent="workspace_center" z_origin_offset="-.008">
+    <origin xyz="0 -0.184 0.008" rpy="0 0 0" />
+  </xacro:kitting_bin_2>
+  <!--bin_3_part_15_-->
+  <xacro:kitting_bin_3 binname="bin_3_part_15" parent="workspace_center" z_origin_offset="-.004">
+    <origin xyz="0.25 0.0 0.004" rpy="0 0 0" />
+  </xacro:kitting_bin_3>
+  <!--bin_3_part_16_-->
+  <xacro:kitting_bin_3 binname="bin_3_part_16" parent="workspace_center" z_origin_offset="-.004">
+    <origin xyz="0.25 -0.192 0.004" rpy="0 0 0" />
   </xacro:kitting_bin_3>
 </robot>
