Commit message: Fixed bug in class PrecisionGripper.

File: aist_scene_description/urdf/InnerOnlyGripper.urdf.xacro (robot description, xacro)
@@ -60,5 +60,6 @@
     <child link="${prefix}${grippername}_tip_link"/>
     <!-- <origin rpy="0.0 ${-pi/2} 0.0" xyz="0.001 -0.008 .162"/> -->
-    <origin rpy="0 0 0" xyz="0.162 -0.008 -0.001"/>
+    <!-- <origin rpy="0 0 0" xyz="0.162 -0.008 -0.001"/> -->
+    <origin rpy="0 0 0" xyz="0.162 -0.015 -0.001"/>
     <!-- +y is the same, +x in the new frame is +z in the parent, +z is -x in the parent? -->
   </joint>

File: aist_scene_description/urdf/pgrp_base_scene.urdf.xacro (robot description, xacro)
@@ -65,5 +65,5 @@
   <xacro:include filename="$(find aist_scene_description)/urdf/InnerOnlyGripper.urdf.xacro" />
   <xacro:InnerOnlyGripper prefix="a_bot_"  grippername = "gripper" parent = "a_bot_ft300_frange_link">
-    <origin xyz="0 0 0" rpy="${-pi/2} 0 0"/>
+    <origin xyz="0 0 0" rpy="${-pi/2} ${-1.3*pi/180} ${0.4*pi/180}"/>
   </xacro:InnerOnlyGripper>
   <xacro:include filename="$(find o2as_scene_description)/urdf/single_suction_gripper.urdf.xacro"/>
@@ -92,5 +92,5 @@
     <parent link="a_bot_wrist_2_link" />
     <child  link="a_bot_cam_holder_link" />
-    <origin xyz="0.04 -0.06 0.20" rpy="${12*pi/180} 0.0 ${pi/2}" />
+    <origin xyz="0.04 -0.06 0.20" rpy="${0*pi/180} 0.0 ${pi/2}" />
   </joint>
   <xacro:sensor_d435 prefix="a_bot_" parent="a_bot_cam_holder_link">
