Commit message: Confirmed linear_push, spiral_motion, insertion and horizontal_insertion UR scripts work.

File: aist_scene_description/urdf/pgrp_kitting.urdf.xacro (robot description, xacro)
@@ -4,6 +4,6 @@
   <!-- base plate -->
   <xacro:include filename="$(find o2as_scene_description)/urdf/o2as_box.xacro"/>
-  <xacro:property name="plate_w" value="0.4"/>
-  <xacro:property name="plate_l" value="0.75"/>
+  <xacro:property name="plate_w" value="0.42"/>
+  <xacro:property name="plate_l" value="0.68"/>
   <xacro:property name="plate_h" value="0.015"/>
   <xacro:o2as_box boxname="plate"

Commit message: Revise kitting scene.

File: aist_scene_description/urdf/pgrp_kitting.urdf.xacro (robot description, xacro)
@@ -2,19 +2,22 @@
 <robot xmlns:xacro="http://www.ros.org/wiki/xacro" name="pgrp_kitting">
   <xacro:include filename="$(find aist_scene_description)/urdf/pgrp_base_scene.urdf.xacro" />
-  <!-- base plate -->
+  <xacro:property name="board_length" value="0.68"/>
+  <xacro:property name="board_width"  value="0.42"/>
+  <xacro:property name="board_height" value="0.015"/>
+  <!-- front board -->
   <xacro:include filename="$(find o2as_scene_description)/urdf/o2as_box.xacro"/>
-  <xacro:property name="plate_w" value="0.42"/>
-  <xacro:property name="plate_l" value="0.68"/>
-  <xacro:property name="plate_h" value="0.015"/>
-  <xacro:o2as_box boxname="plate"
-		  box_w="${plate_w}" box_l="${plate_l}" box_h="${plate_h}"
+  <xacro:o2as_box boxname="board"
+		  box_w="${board_length}"
+		  box_l="${board_width}"
+		  box_h="${board_height}"
 		  parent="workspace_center">
-    <origin xyz="${-plate_w/2} ${-plate_l/2} 0" rpy="0 0 0"/>
+    <origin xyz="${-board_length/2} ${-board_width/2} ${-borad_height/2}"
+	    rpy="0 0 0"/>
   </xacro:o2as_box>
-  <link name="plate_center"/>
-  <joint name="workspace_to_plate" type="fixed">
+  <link name="board_center"/>
+  <joint name="workspace_to_board" type="fixed">
     <parent link="workspace_center"/>
-    <child  link="plate_center"/>
-    <origin xyz="0 0 ${plate_h}" rpy="0 0 0"/>
+    <child  link="board_center"/>
+    <origin xyz="0 0 ${board_height}" rpy="0 0 0"/>
   </joint>
   <!-- bin1_definition -->
@@ -41,40 +44,38 @@
   <!--bin_2_part_4_-->
   <xacro:kitting_bin_2 binname	      ="bin_2_part_4"
-		       parent	      ="plate_center"
+		       parent	      ="board_center"
 		       z_origin_offset="-0.008">
-    <origin xyz="0.285  0 0.004" rpy="0 0 0" />
+    <origin xyz="0.100  0 0.004" rpy="0 0 0" />
   </xacro:kitting_bin_2>
   <!--bin_2_part_7_-->
   <xacro:kitting_bin_2 binname	      ="bin_2_part_7"
-		       parent	      ="plate_center"
+		       parent	      ="board_center"
 		       z_origin_offset="-0.008">
-    <origin xyz="0.285 0.112 0.008" rpy="0 0 0" />
+    <origin xyz="0.100 0.112 0.008" rpy="0 0 0" />
   </xacro:kitting_bin_2>
   <!--bin_2_part_8_-->
   <xacro:kitting_bin_2 binname	      ="bin_2_part_8"
-  		       parent	      ="plate_center"
+  		       parent	      ="board_center"
   		       z_origin_offset="-0.008">
-    <origin xyz="0.285 -0.112 0.008" rpy="0 0 0" />
+    <origin xyz="0.100 -0.112 0.008" rpy="0 0 0" />
   </xacro:kitting_bin_2>
   <!-- bin_3_part_15_ -->
   <xacro:kitting_bin_3 binname	      ="bin_3_part_15"
-  		       parent	      ="plate_center"
+  		       parent	      ="board_center"
   		       z_origin_offset="-0.004">
-    <origin xyz="0 0.096 0.004" rpy="0 0 0" />
+    <origin xyz="-0.143 0.096 0.004" rpy="0 0 0" />
   </xacro:kitting_bin_3>
   <!-- bin_3_part_16_ -->
   <xacro:kitting_bin_3 binname	      ="bin_3_part_16"
-  		       parent	      ="plate_center"
+  		       parent	      ="board_center"
   		       z_origin_offset="-0.004">
-    <origin xyz="0 -0.096 0.004" rpy="0 0 0" />
+    <origin xyz="-0.143 -0.096 0.004" rpy="0 0 0" />
   </xacro:kitting_bin_3>
   <xacro:include filename="$(find aist_scene_description)/urdf/kitting_tray_with_partitions.xacro" />
-  <xacro:property name="tray_width" value=".210" />
-  <xacro:property name="tray_length" value=".300" />
-  <xacro:property name="tray_rack_width" value=".210" />
-  <xacro:property name="tray_rack_length" value=".600" />
-  <xacro:property name="tray_rack_height" value=".015" />
-  <xacro:property name="bin_rack_width" value=".420" />
-  <xacro:property name="bin_rack_length" value=".680" />
-  <xacro:property name="bin_rack_height" value=".015" />
+  <xacro:kitting_tray1 trayname="tray_1" parent="board_center">
+    <origin xyz="0 0 0" rpy="0 0 0" />
+  </xacro:kitting_tray1>
+  <xacro:kitting_tray2 trayname="tray_2" parent="board_center">
+    <origin xyz="0 ${-tray_width - 0.002} 0" rpy="0 0 0" />
+  </xacro:kitting_tray2>
 </robot>

Commit message: Kitting scene revised.

File: aist_scene_description/urdf/pgrp_kitting.urdf.xacro (robot description, xacro)
@@ -2,25 +2,26 @@
 <robot xmlns:xacro="http://www.ros.org/wiki/xacro" name="pgrp_kitting">
   <xacro:include filename="$(find aist_scene_description)/urdf/pgrp_base_scene.urdf.xacro" />
-  <xacro:property name="board_length" value="0.68"/>
-  <xacro:property name="board_width"  value="0.42"/>
-  <xacro:property name="board_height" value="0.015"/>
-  <!-- front board -->
+  <xacro:property name="plate_w" value="0.68"/>
+  <xacro:property name="plate_l" value="0.42"/>
+  <xacro:property name="plate_h" value="0.015"/>
+  <!-- front plate -->
   <xacro:include filename="$(find o2as_scene_description)/urdf/o2as_box.xacro"/>
-  <xacro:o2as_box boxname="board"
-		  box_w="${board_length}"
-		  box_l="${board_width}"
-		  box_h="${board_height}"
+  <xacro:o2as_box boxname="plate"
+		  box_w="${plate_w}"
+		  box_l="${plate_l}"
+		  box_h="${plate_h}"
 		  parent="workspace_center">
-    <origin xyz="${-board_length/2} ${-board_width/2} ${-borad_height/2}"
+    <origin xyz="${table_w/2 - plate_w - 0.08} ${-plate_l/2} 0"
 	    rpy="0 0 0"/>
   </xacro:o2as_box>
-  <link name="board_center"/>
-  <joint name="workspace_to_board" type="fixed">
-    <parent link="workspace_center"/>
-    <child  link="board_center"/>
-    <origin xyz="0 0 ${board_height}" rpy="0 0 0"/>
+  <link name="plate_center"/>
+  <joint name="plate_to_plate_center" type="fixed">
+    <parent link="plate"/>
+    <child  link="plate_center"/>
+    <origin xyz="${plate_w/2} ${plate_l/2} ${plate_h}" rpy="0 0 0"/>
   </joint>
+  <xacro:include filename="$(find o2as_scene_description)/urdf/kitting_bin_macros.xacro" />
+  <xacro:include filename="$(find o2as_scene_description)/urdf/kitting_tray_with_partitions.xacro" />
   <!-- bin1_definition -->
-  <xacro:include filename="$(find o2as_scene_description)/urdf/kitting_bin_macros.xacro" />
   <xacro:property name="bin_1_width"		value="0.125"/>
   <xacro:property name="bin_1_length"		value="0.128"/>
@@ -44,38 +45,52 @@
   <!--bin_2_part_4_-->
   <xacro:kitting_bin_2 binname	      ="bin_2_part_4"
-		       parent	      ="board_center"
-		       z_origin_offset="-0.008">
-    <origin xyz="0.100  0 0.004" rpy="0 0 0" />
+		       parent	      ="plate_center"
+		       z_origin_offset="${z_origin_offset_2}">
+    <origin xyz="${-plate_w/2 + tray_length + bin_3_length + bin_2_length/2}
+		 ${bin_2_width}
+		 ${-z_origin_offset_2}"
+	    rpy="0 0 0" />
   </xacro:kitting_bin_2>
   <!--bin_2_part_7_-->
   <xacro:kitting_bin_2 binname	      ="bin_2_part_7"
-		       parent	      ="board_center"
-		       z_origin_offset="-0.008">
-    <origin xyz="0.100 0.112 0.008" rpy="0 0 0" />
+		       parent	      ="plate_center"
+		       z_origin_offset="${z_origin_offset_2}">
+    <origin xyz="${-plate_w/2 + tray_length + bin_3_length + bin_2_length/2}
+		 0
+		 ${-z_origin_offset_2}"
+	    rpy="0 0 0" />
   </xacro:kitting_bin_2>
   <!--bin_2_part_8_-->
   <xacro:kitting_bin_2 binname	      ="bin_2_part_8"
-  		       parent	      ="board_center"
-  		       z_origin_offset="-0.008">
-    <origin xyz="0.100 -0.112 0.008" rpy="0 0 0" />
+  		       parent	      ="plate_center"
+  		       z_origin_offset="${z_origin_offset_2}">
+    <origin xyz="${-plate_w/2 + tray_length + bin_3_length + bin_2_length/2}
+		 ${-bin_2_width}
+		 ${-z_origin_offset_2}"
+	    rpy="0 0 0" />
   </xacro:kitting_bin_2>
   <!-- bin_3_part_15_ -->
   <xacro:kitting_bin_3 binname	      ="bin_3_part_15"
-  		       parent	      ="board_center"
-  		       z_origin_offset="-0.004">
-    <origin xyz="-0.143 0.096 0.004" rpy="0 0 0" />
+  		       parent	      ="plate_center"
+  		       z_origin_offset="${z_origin_offset_3}">
+    <origin xyz="${-plate_w/2 + tray_length + bin_3_length/2}
+		 ${bin_3_width/2}
+		 ${-z_origin_offset_3}"
+	    rpy="0 0 0" />
   </xacro:kitting_bin_3>
   <!-- bin_3_part_16_ -->
   <xacro:kitting_bin_3 binname	      ="bin_3_part_16"
-  		       parent	      ="board_center"
-  		       z_origin_offset="-0.004">
-    <origin xyz="-0.143 -0.096 0.004" rpy="0 0 0" />
+  		       parent	      ="plate_center"
+  		       z_origin_offset="${z_origin_offset_3}">
+    <origin xyz="${-plate_w/2 + tray_length + bin_3_length/2}
+		 ${-bin_3_width/2}
+		 ${-z_origin_offset_3}"
+	    rpy="0 0 0" />
   </xacro:kitting_bin_3>
-  <xacro:include filename="$(find aist_scene_description)/urdf/kitting_tray_with_partitions.xacro" />
-  <xacro:kitting_tray1 trayname="tray_1" parent="board_center">
-    <origin xyz="0 0 0" rpy="0 0 0" />
+  <xacro:kitting_tray1 trayname="tray_1" parent="plate_center">
+    <origin xyz="${-plate_w/2} 0 0" rpy="0 0 0" />
   </xacro:kitting_tray1>
-  <xacro:kitting_tray2 trayname="tray_2" parent="board_center">
-    <origin xyz="0 ${-tray_width - 0.002} 0" rpy="0 0 0" />
+  <xacro:kitting_tray2 trayname="tray_2" parent="plate_center">
+    <origin xyz="${-plate_w/2} ${-tray_width} 0" rpy="0 0 0" />
   </xacro:kitting_tray2>
 </robot>

Commit message: Kitting scene revised.

File: aist_scene_description/urdf/pgrp_kitting.urdf.xacro (robot description, xacro)
@@ -23,13 +23,13 @@
   <xacro:include filename="$(find o2as_scene_description)/urdf/kitting_bin_macros.xacro" />
   <xacro:include filename="$(find o2as_scene_description)/urdf/kitting_tray_with_partitions.xacro" />
-  <!-- bin1_definition -->
+  <!-- bin_1_definition -->
   <xacro:property name="bin_1_width"		value="0.125"/>
   <xacro:property name="bin_1_length"		value="0.128"/>
   <xacro:property name="z_origin_offset_1"	value="-.005" />
-  <!-- bin2_definition -->
+  <!-- bin_2_definition -->
   <xacro:property name="bin_2_width"		value="0.112"/>
   <xacro:property name="bin_2_length"		value="0.201"/>
   <xacro:property name="z_origin_offset_2"	value="-.008" />
-  <!-- bin3_definition -->
+  <!-- bin_3_definition -->
   <xacro:property name="bin_3_width"		value="0.192"/>
   <xacro:property name="bin_3_length"		value="0.285"/>
@@ -43,9 +43,36 @@
   <xacro:property name="set2_y" value="0.096"/>
   <xacro:property name="set2_z" value="0"/>
-  <!--bin_2_part_4_-->
+  <!--bin_1_part_15_-->
+  <xacro:kitting_bin_1 binname	      ="bin_1_part_15"
+		       parent	      ="plate_center"
+		       z_origin_offset="${z_origin_offset_1}">
+    <origin xyz="${plate_w/2 - bin_1_length/2}
+		 ${bin_1_width}
+		 ${-z_origin_offset_1}"
+	    rpy="0 0 0" />
+  </xacro:kitting_bin_1>
+  <!--bin_1_part_16_-->
+  <xacro:kitting_bin_1 binname	      ="bin_1_part_16"
+		       parent	      ="plate_center"
+		       z_origin_offset="${z_origin_offset_1}">
+    <origin xyz="${plate_w/2 - bin_1_length/2}
+		 0
+		 ${-z_origin_offset_2}"
+	    rpy="0 0 0" />
+  </xacro:kitting_bin_1>
+  <!--bin_1_part_17_-->
+  <xacro:kitting_bin_1 binname	      ="bin_1_part_17"
+  		       parent	      ="plate_center"
+  		       z_origin_offset="${z_origin_offset_1}">
+    <origin xyz="${plate_w/2 - bin_1_length/2}
+		 ${-bin_1_width}
+		 ${-z_origin_offset_1}"
+	    rpy="0 0 0" />
+  </xacro:kitting_bin_1>
+  <!-- bin_2_part_4_ -->
   <xacro:kitting_bin_2 binname	      ="bin_2_part_4"
 		       parent	      ="plate_center"
 		       z_origin_offset="${z_origin_offset_2}">
-    <origin xyz="${-plate_w/2 + tray_length + bin_3_length + bin_2_length/2}
+    <origin xyz="${plate_w/2 - bin_1_length - bin_2_length/2}
 		 ${bin_2_width}
 		 ${-z_origin_offset_2}"
@@ -56,5 +83,5 @@
 		       parent	      ="plate_center"
 		       z_origin_offset="${z_origin_offset_2}">
-    <origin xyz="${-plate_w/2 + tray_length + bin_3_length + bin_2_length/2}
+    <origin xyz="${plate_w/2 - bin_1_length - bin_2_length/2}
 		 0
 		 ${-z_origin_offset_2}"
@@ -65,32 +92,22 @@
   		       parent	      ="plate_center"
   		       z_origin_offset="${z_origin_offset_2}">
-    <origin xyz="${-plate_w/2 + tray_length + bin_3_length + bin_2_length/2}
+    <origin xyz="${plate_w/2 - bin_1_length - bin_2_length/2}
 		 ${-bin_2_width}
 		 ${-z_origin_offset_2}"
 	    rpy="0 0 0" />
   </xacro:kitting_bin_2>
-  <!-- bin_3_part_15_ -->
-  <xacro:kitting_bin_3 binname	      ="bin_3_part_15"
-  		       parent	      ="plate_center"
-  		       z_origin_offset="${z_origin_offset_3}">
-    <origin xyz="${-plate_w/2 + tray_length + bin_3_length/2}
-		 ${bin_3_width/2}
-		 ${-z_origin_offset_3}"
+  <!-- tray_1 -->
+  <xacro:kitting_tray1 trayname="tray_1" parent="plate_center">
+    <origin xyz="${plate_w/2 - bin_1_length - bin_2_length - tray_length}
+		 0
+		 0"
 	    rpy="0 0 0" />
-  </xacro:kitting_bin_3>
-  <!-- bin_3_part_16_ -->
-  <xacro:kitting_bin_3 binname	      ="bin_3_part_16"
-  		       parent	      ="plate_center"
-  		       z_origin_offset="${z_origin_offset_3}">
-    <origin xyz="${-plate_w/2 + tray_length + bin_3_length/2}
-		 ${-bin_3_width/2}
-		 ${-z_origin_offset_3}"
+  </xacro:kitting_tray1>
+  <!-- tray_2 -->
+  <xacro:kitting_tray2 trayname="tray_2" parent="plate_center">
+    <origin xyz="${plate_w/2 - bin_1_length - bin_2_length - tray_length}
+		 ${-tray_width}
+		 0"
 	    rpy="0 0 0" />
-  </xacro:kitting_bin_3>
-  <xacro:kitting_tray1 trayname="tray_1" parent="plate_center">
-    <origin xyz="${-plate_w/2} 0 0" rpy="0 0 0" />
-  </xacro:kitting_tray1>
-  <xacro:kitting_tray2 trayname="tray_2" parent="plate_center">
-    <origin xyz="${-plate_w/2} ${-tray_width} 0" rpy="0 0 0" />
   </xacro:kitting_tray2>
 </robot>
