Commit message: Update phoxi pose.

File: aist_scene_description/urdf/aist_base_scene.urdf.xacro (robot description, xacro)
@@ -58,6 +58,5 @@
   <xacro:include filename="$(find o2as_scene_description)/urdf/phoxi_m_camera.urdf.xacro" />
   <xacro:phoxi_m_camera prefix="a_" parent="o2as_ground">
-  <!-- This is the setting for challenge, so we need to re-calibration before stating experiments in aist. (2018/11/06 Yuma Hijioka) -->
-  <origin xyz="0.652663578768 -0.0142895785849 1.50687788672" rpy="${-161.381811856*pi/180} ${2.99567722105*pi/180} ${90.8962573459*pi/180}"/>
+  <origin xyz="0.63885382925 0.00793354972549 1.45431467674" rpy="${-144.009037015*pi/180} ${0.0354016148982*pi/180} ${85.0410662353*pi/180}"/>
   </xacro:phoxi_m_camera>
   <!-- I would like to remove the "world" link definition, but apparently it is necessary for Gazebo -->

Commit message: Various fixed.

File: aist_scene_description/urdf/aist_base_scene.urdf.xacro (robot description, xacro)
@@ -51,8 +51,6 @@
   </joint>
   <!-- spawn and attach dual suction grippers -->
-  <xacro:include filename="$(find o2as_scene_description)/urdf/dual_suction_gripper.urdf.xacro" />
-  <xacro:dual_suction_gripper_o2as prefix="b_bot_" parent = "b_bot_ee_link">
-    <origin xyz="0 0 0" rpy="0 0 0"/>
-  </xacro:dual_suction_gripper_o2as>
+  <xacro:include filename="$(find aist_scene_description)/urdf/dual_suction_gripper_with_ft300.urdf.xacro" />
+  <xacro:dual_suction_gripper_with_ft300 prefix="b_bot_" parent = "b_bot_ee_link" />
   <!-- Add PhoXi 3D scanners -->
   <xacro:include filename="$(find o2as_scene_description)/urdf/phoxi_m_camera.urdf.xacro" />

Commit message: WIP: Dump commit.

File: aist_scene_description/urdf/aist_base_scene.urdf.xacro (robot description, xacro)
@@ -56,5 +56,5 @@
   <xacro:include filename="$(find o2as_scene_description)/urdf/phoxi_m_camera.urdf.xacro" />
   <xacro:phoxi_m_camera prefix="a_" parent="o2as_ground">
-  <origin xyz="0.63885382925 0.00793354972549 1.45431467674" rpy="${-144.009037015*pi/180} ${0.0354016148982*pi/180} ${85.0410662353*pi/180}"/>
+  <origin xyz="0.64685382925 0.00793354972549 1.47431467674" rpy="${-144.009037015*pi/180} ${0.0354016148982*pi/180} ${85.0410662353*pi/180}"/>
   </xacro:phoxi_m_camera>
   <!-- I would like to remove the "world" link definition, but apparently it is necessary for Gazebo -->

Commit message: Initial version of tool_calibration.py added.

File: aist_scene_description/urdf/aist_base_scene.urdf.xacro (robot description, xacro)
@@ -5,5 +5,5 @@
   <xacro:property name="b_bot_x" value="0"/>
   <xacro:property name="b_bot_y" value="0.50"/>
-  <xacro:property name="b_bot_theta" value="-3.14"/>
+  <xacro:property name="b_bot_theta" value="${pi}"/>
   <xacro:property name="bots_z" value="0.77"/>
   <!-- This is the main file defining our robot arrangement and physical environment. -->
@@ -50,12 +50,13 @@
     <origin xyz="${b_bot_x} ${b_bot_y} ${bots_z}" rpy="0.0 0.0 ${b_bot_theta}" />
   </joint>
-  <!-- spawn and attach single suction grippers -->
+  <!-- Spawn and attach single suction gripper -->
   <xacro:include filename="$(find aist_scene_description)/urdf/single_suction_gripper_with_ft300.urdf.xacro" />
   <xacro:single_suction_gripper_with_ft300 prefix="b_bot_" parent = "b_bot_ee_link" />
-  <!-- Add PhoXi 3D scanners -->
+  <!-- Add PhoXi 3D scanner -->
   <xacro:include filename="$(find o2as_scene_description)/urdf/phoxi_m_camera.urdf.xacro" />
   <xacro:phoxi_m_camera prefix="a_" parent="o2as_ground">
   <origin xyz="0.64685382925 0.00793354972549 1.47431467674" rpy="${-144.009037015*pi/180} ${0.0354016148982*pi/180} ${85.0410662353*pi/180}"/>
   </xacro:phoxi_m_camera>
+  <!-- Add AR markers -->
   <xacro:include filename="$(find aist_gazebo)/urdf/aist_ar_marker.urdf.xacro"/>
   <xacro:aist_ar_marker prefix="b_bot_"

Commit message: Calibrated parameters are reflected in scene description files.

File: aist_scene_description/urdf/aist_base_scene.urdf.xacro (robot description, xacro)
@@ -56,5 +56,6 @@
   <xacro:include filename="$(find o2as_scene_description)/urdf/phoxi_m_camera.urdf.xacro" />
   <xacro:phoxi_m_camera prefix="a_" parent="o2as_ground">
-  <origin xyz="0.64685382925 0.00793354972549 1.47431467674" rpy="${-144.009037015*pi/180} ${0.0354016148982*pi/180} ${85.0410662353*pi/180}"/>
+    <origin xyz="0.645496196414 0.0871790100695 1.47122882444"
+	    rpy="${-143.980928467*pi/180} ${0.224942781411*pi/180} ${85.683086361*pi/180}"/>>
   </xacro:phoxi_m_camera>
   <!-- Add AR markers -->

Commit message: Modified scene

File: aist_scene_description/urdf/aist_base_scene.urdf.xacro (robot description, xacro)
@@ -14,5 +14,5 @@
   <xacro:include filename="$(find o2as_scene_description)/urdf/ur5.urdf.xacro" />
   <!-- Scene items (trays, bins...) -->
-  <!-- <xacro:include filename="$(find aist_scene_description)/urdf/aist_kitting_scene.xacro" /> -->
+  <xacro:include filename="$(find aist_scene_description)/urdf/aist_kitting_scene.xacro" />
   <!-- Robot bases -->
   <!-- Putting these at height 0.0 makes them intersect with the ground, so they are elevated. -->

File: aist_scene_description/urdf/kitting_bins.xacro (robot description, xacro)
@@ -17,50 +17,10 @@
   <xacro:property name="z_origin_offset_3" value="-.004" />
   <!-- A row of bin1 -->
-  <xacro:property name="set1_x" value="-0.1095"/>
-  <xacro:property name="set1_y" value="0.34"/>
+  <xacro:property name="set1_x" value="0"/>
+  <xacro:property name="set1_y" value="0.096"/>
   <xacro:property name="set1_z" value="0"/>
-  <!-- A row of bin2 -->
-  <xacro:property name="set2_x" value=".055"/>
-  <xacro:property name="set2_y" value="0.34"/>
-  <xacro:property name="set2_z" value="0"/>
-  <!--bin_2_part_a_-->
-  <xacro:kitting_bin_2 binname="bin_2_part_a" parent="bin_rack_center" z_origin_offset="-.008">
-    <origin xyz="-0.1095 0.284 0.008" rpy="0 0 0" />
-  </xacro:kitting_bin_2>
-  <!--bin_2_part_4_-->
-  <xacro:kitting_bin_2 binname="bin_2_part_4" parent="bin_rack_center" z_origin_offset="-.008">
-    <origin xyz="-0.1095 0.172 0.008" rpy="0 0 0" />
-  </xacro:kitting_bin_2>
-  <!--bin_2_part_7_-->
-  <xacro:kitting_bin_2 binname="bin_2_part_7" parent="bin_rack_center" z_origin_offset="-.008">
-    <origin xyz="-0.1095 0.06 0.008" rpy="0 0 0" />
-  </xacro:kitting_bin_2>
-  <!--bin_2_part_11_-->
-  <xacro:kitting_bin_2 binname="bin_2_part_11" parent="bin_rack_center" z_origin_offset="-.008">
-    <origin xyz="-0.1095 -0.052 0.008" rpy="0 0 0" />
-  </xacro:kitting_bin_2>
-  <!--bin_2_part_b_-->
-  <xacro:kitting_bin_2 binname="bin_2_part_b" parent="bin_rack_center" z_origin_offset="-.008">
-    <origin xyz="-0.1095 -0.164 0.008" rpy="0 0 0" />
-  </xacro:kitting_bin_2>
-  <!--bin_1_part_13_-->
-  <xacro:kitting_bin_1 binname="bin_1_part_13" parent="bin_rack_center" z_origin_offset="-.005">
-    <origin xyz=".055 0.2775 0.005" rpy="0 0 0" />
-  </xacro:kitting_bin_1>
-  <!--bin_1_part_8_-->
-  <xacro:kitting_bin_1 binname="bin_1_part_8" parent="bin_rack_center" z_origin_offset="-.005">
-    <origin xyz=".055 0.1525 0.005" rpy="0 0 0" />
-  </xacro:kitting_bin_1>
-  <!--bin_1_part_12_-->
-  <xacro:kitting_bin_1 binname="bin_1_part_12" parent="bin_rack_center" z_origin_offset="-.005">
-    <origin xyz=".055 0.0275 0.005" rpy="0 0 0" />
-  </xacro:kitting_bin_1>
-  <!--bin_1_part_5_-->
-  <xacro:kitting_bin_1 binname="bin_1_part_5" parent="bin_rack_center" z_origin_offset="-.005">
-    <origin xyz=".055 -0.0975 0.005" rpy="0 0 0" />
-  </xacro:kitting_bin_1>
-  <!--bin_1_part_c_-->
-  <xacro:kitting_bin_1 binname="bin_1_part_c" parent="bin_rack_center" z_origin_offset="-.005">
-    <origin xyz=".055 -0.2225 0.005" rpy="0 0 0" />
-  </xacro:kitting_bin_1>
+  <!--bin_3_part_5_-->
+  <xacro:kitting_bin_3 binname="bin_3_part_5" parent="bin_rack_center" z_origin_offset="-.004">
+    <origin xyz="0 0.0 0.004" rpy="0 0 0" />
+  </xacro:kitting_bin_3>
 </robot>

Commit message: Cleaning up.

File: aist_scene_description/urdf/aist_base_scene.urdf.xacro (robot description, xacro)
@@ -14,5 +14,5 @@
   <xacro:include filename="$(find o2as_scene_description)/urdf/ur5.urdf.xacro" />
   <!-- Scene items (trays, bins...) -->
-  <xacro:include filename="$(find aist_scene_description)/urdf/aist_kitting_scene.xacro" />
+  <!-- <xacro:include filename="$(find aist_scene_description)/urdf/aist_kitting_scene.xacro" /> -->
   <!-- Robot bases -->
   <!-- Putting these at height 0.0 makes them intersect with the ground, so they are elevated. -->

File: o2as_scene_description/urdf/single_suction_gripper.urdf.xacro (robot description, xacro)
@@ -17,5 +17,5 @@
       <collision>
       <!-- avoid collision -->
-	<origin xyz="0.188 -0.035 -0.035" rpy="0 0 ${pi/2}"/>
+        <origin xyz="0.188 -0.035 -0.035" rpy="0 0 ${pi/2}"/>
 	<!-- <origin xyz="0.187 -0.035 -0.035" rpy="0 0 ${pi/2}"/> -->
 	<geometry>
@@ -40,5 +40,7 @@
       <parent link="${prefix}single_suction_gripper_base_link"/>
       <child  link="${prefix}single_suction_gripper_pad_link"/>
-      <origin xyz="0.187 0 0" rpy="0 0 0"/>
+      <!-- <origin xyz="0.187 0 0" rpy="0 0 0"/> -->
+      <origin xyz="0.186964399692 -0.00163161359769 -0.00326360000377"
+	      rpy="${0.0*pi/180} ${1.0*pi/180} ${-0.5*pi/180}"/>>
     </joint>
   </xacro:macro>

Commit message: Calibrated PhoXi pose in scene
b/c We reset worktable and robot yesterday

File: aist_scene_description/urdf/aist_base_scene.urdf.xacro (robot description, xacro)
@@ -56,6 +56,7 @@
   <xacro:include filename="$(find o2as_scene_description)/urdf/phoxi_m_camera.urdf.xacro" />
   <xacro:phoxi_m_camera prefix="a_" parent="o2as_ground">
-    <origin xyz="0.645496196414 0.0871790100695 1.47122882444"
-	    rpy="${-143.980928467*pi/180} ${0.224942781411*pi/180} ${85.683086361*pi/180}"/>>
+    <origin xyz="0.680222661268 0.0883185826892 1.46923382305"
+	    rpy="${-143.767574699*pi/180} ${0.261166479412*pi/180}
+		 ${85.7064003235*pi/180}"/>
   </xacro:phoxi_m_camera>
   <!-- Add AR markers -->

Commit message: o2as_aruco_ros::o2as_simple now takes lens distortion into account.

File: aist_scene_description/urdf/aist_base_scene.urdf.xacro (robot description, xacro)
@@ -56,6 +56,7 @@
   <xacro:include filename="$(find o2as_scene_description)/urdf/phoxi_m_camera.urdf.xacro" />
   <xacro:phoxi_m_camera prefix="a_" parent="o2as_ground">
-    <origin xyz="0.645496196414 0.0871790100695 1.47122882444"
-	    rpy="${-143.980928467*pi/180} ${0.224942781411*pi/180} ${85.683086361*pi/180}"/>>
+    <origin xyz="0.679378193555 0.0896899509207 1.46884427155"
+	    rpy="${-143.784602932*pi/180}
+		 ${0.342593998659*pi/180} ${85.7589559216*pi/180}"/>>
   </xacro:phoxi_m_camera>
   <!-- Add AR markers -->

File: o2as_scene_description/urdf/single_suction_gripper.urdf.xacro (robot description, xacro)
@@ -41,6 +41,6 @@
       <child  link="${prefix}single_suction_gripper_pad_link"/>
       <!-- <origin xyz="0.187 0 0" rpy="0 0 0"/> -->
-      <origin xyz="0.186964399692 -0.00163161359769 -0.00326360000377"
-	      rpy="${0.0*pi/180} ${1.0*pi/180} ${-0.5*pi/180}"/>>
+      <origin xyz="0.186976645492 -0.000326336140176 -0.00293726833731"
+	      rpy="${0.0*pi/180} ${0.9*pi/180} ${-0.1*pi/180}"/>
     </joint>
   </xacro:macro>

Commit message: Various fixed

File: aist_scene_description/urdf/aist_base_scene.urdf.xacro (robot description, xacro)
@@ -56,7 +56,7 @@
   <xacro:include filename="$(find o2as_scene_description)/urdf/phoxi_m_camera.urdf.xacro" />
   <xacro:phoxi_m_camera prefix="a_" parent="o2as_ground">
-    <origin xyz="0.679378193555 0.0896899509207 1.46884427155"
-	    rpy="${-143.784602932*pi/180}
-		 ${0.342593998659*pi/180} ${85.7589559216*pi/180}"/>>
+    <origin xyz="0.679997723974 0.0866831188148 1.46958049634"
+	    rpy="${-143.76356757*pi/180}
+		 ${0.312453823638*pi/180} ${85.5565266354*pi/180}"/>
   </xacro:phoxi_m_camera>
   <!-- Add AR markers -->

Commit message: Add new robot

File: aist_scene_description/urdf/aist_base_scene.urdf.xacro (robot description, xacro)
@@ -3,4 +3,7 @@
         name="aist_base_scene" >
   <!-- Calibration help: If the robot is not moving far enough to the calibration point, increase these distances -->
+  <xacro:property name="a_bot_x" value="0"/>
+  <xacro:property name="a_bot_y" value="-0.60"/>
+  <!-- <xacro:property name="a_bot_theta" value="${pi}"/> -->
   <xacro:property name="b_bot_x" value="0"/>
   <xacro:property name="b_bot_y" value="0.50"/>
@@ -19,4 +22,7 @@
   <!-- There are some instabilities when the box is big, for some reason. -->
   <xacro:include filename="$(find aist_scene_description)/urdf/aist_base.xacro" />
+  <xacro:aist_base boxname="a_bot_base_smfl" parent="o2as_ground">
+    <origin xyz="${a_bot_x-0.225/2} ${a_bot_y-0.225/2} 0.72" rpy="0 0 0" />
+  </xacro:aist_base>
   <xacro:aist_base boxname="b_bot_base_smfl" parent="o2as_ground">
     <origin xyz="${b_bot_x-0.225/2} ${b_bot_y-0.225/2} 0.72" rpy="0 0 0" />
@@ -37,4 +43,11 @@
   </joint>
   <!-- robot arms -->
+  <xacro:ur5_robot prefix="a_bot_" joint_limited="false"
+    shoulder_pan_lower_limit="${-pi}" shoulder_pan_upper_limit="${pi}"
+    shoulder_lift_lower_limit="${-pi}" shoulder_lift_upper_limit="${pi}"
+    elbow_joint_lower_limit="0.0" elbow_joint_upper_limit="${pi}"
+    wrist_1_lower_limit="${-pi}" wrist_1_upper_limit="${pi}"
+    wrist_2_lower_limit="${-pi}" wrist_2_upper_limit="${pi}"
+    wrist_3_lower_limit="${-pi}" wrist_3_upper_limit="${pi}"/>
   <xacro:ur5_robot prefix="b_bot_" joint_limited="false"
     shoulder_pan_lower_limit="${-pi}" shoulder_pan_upper_limit="${pi}"
@@ -45,4 +58,9 @@
     wrist_3_lower_limit="${-pi}" wrist_3_upper_limit="${pi}"/>
   <link name="o2as_ground" />
+  <joint name="world_a_bot_joint" type="fixed">
+    <parent link="o2as_ground" />
+    <child link = "a_bot_base_link" />
+    <origin xyz="${a_bot_x} ${a_bot_y} ${bots_z}" rpy="0.0 0.0 0.0" />
+  </joint>
   <joint name="world_b_bot_joint" type="fixed">
     <parent link="o2as_ground" />
@@ -50,5 +68,7 @@
     <origin xyz="${b_bot_x} ${b_bot_y} ${bots_z}" rpy="0.0 0.0 ${b_bot_theta}" />
   </joint>
-  <!-- Spawn and attach single suction gripper -->
+  <!-- Spawn and attach gripper -->
+  <xacro:include filename="$(find aist_scene_description)/urdf/robotiq_85_gripper_with_ft300.urdf.xacro" />
+  <xacro:robotiq_85_gripper_with_ft300 prefix="a_bot_" parent="a_bot_ee_link" />
   <xacro:include filename="$(find aist_scene_description)/urdf/single_suction_gripper_with_ft300.urdf.xacro" />
   <xacro:single_suction_gripper_with_ft300 prefix="b_bot_" parent = "b_bot_ee_link" />

Commit message: Calibrate a_bot and small fixed

File: aist_scene_description/urdf/aist_base_scene.urdf.xacro (robot description, xacro)
@@ -3,6 +3,7 @@
         name="aist_base_scene" >
   <!-- Calibration help: If the robot is not moving far enough to the calibration point, increase these distances -->
-  <xacro:property name="a_bot_x" value="0"/>
-  <xacro:property name="a_bot_y" value="-0.60"/>
+  <xacro:property name="a_bot_x" value="-0.006"/>
+  <xacro:property name="a_bot_y" value="-0.625"/>
+  <xacro:property name="a_bot_z" value="0.78" />
   <!-- <xacro:property name="a_bot_theta" value="${pi}"/> -->
   <xacro:property name="b_bot_x" value="0"/>
@@ -17,5 +18,5 @@
   <xacro:include filename="$(find o2as_scene_description)/urdf/ur5.urdf.xacro" />
   <!-- Scene items (trays, bins...) -->
-  <xacro:include filename="$(find aist_scene_description)/urdf/aist_kitting_scene.xacro" />
+  <!-- <xacro:include filename="$(find aist_scene_description)/urdf/aist_kitting_scene.xacro" /> -->
   <!-- Robot bases -->
   <!-- Putting these at height 0.0 makes them intersect with the ground, so they are elevated. -->
@@ -61,5 +62,5 @@
     <parent link="o2as_ground" />
     <child link = "a_bot_base_link" />
-    <origin xyz="${a_bot_x} ${a_bot_y} ${bots_z}" rpy="0.0 0.0 0.0" />
+    <origin xyz="${a_bot_x} ${a_bot_y} ${a_bot_z}" rpy="0.0 0.0 0.0" />
   </joint>
   <joint name="world_b_bot_joint" type="fixed">

Commit message: Modifed kitting routine

File: aist_scene_description/urdf/aist_base_scene.urdf.xacro (robot description, xacro)
@@ -18,5 +18,5 @@
   <xacro:include filename="$(find o2as_scene_description)/urdf/ur5.urdf.xacro" />
   <!-- Scene items (trays, bins...) -->
-  <!-- <xacro:include filename="$(find aist_scene_description)/urdf/aist_kitting_scene.xacro" /> -->
+  <xacro:include filename="$(find aist_scene_description)/urdf/aist_kitting_scene.xacro" />
   <!-- Robot bases -->
   <!-- Putting these at height 0.0 makes them intersect with the ground, so they are elevated. -->

File: aist_scene_description/urdf/kitting_bins.xacro (robot description, xacro)
@@ -21,6 +21,6 @@
   <xacro:property name="set1_z" value="0"/>
   <!--bin_3_part_8_-->
-  <xacro:kitting_bin_3 binname="bin_3_part_7" parent="workspace_center" z_origin_offset="-.004">
-    <origin xyz=".15 0.0 0.004" rpy="0 0 0" />
+  <xacro:kitting_bin_3 binname="bin_3_part_4" parent="workspace_center" z_origin_offset="-.004">
+    <origin xyz=".15 0.1 0.004" rpy="0 0 0" />
   </xacro:kitting_bin_3>
 </robot>

Commit message: Separate ft300 force sensor from griuppers.

File: aist_scene_description/urdf/aist_base_scene.urdf.xacro (robot description, xacro)
@@ -69,9 +69,19 @@
     <origin xyz="${b_bot_x} ${b_bot_y} ${bots_z}" rpy="0.0 0.0 ${b_bot_theta}" />
   </joint>
+  <!-- Spawn and attach force sensor -->
+  <xacro:include filename="$(find o2as_scene_description)/urdf/ft300.urdf.xacro" />
+  <xacro:ft300 prefix="a_bot_" parent="a_bot_ee_link" />
+  <xacro:ft300 prefix="b_bot_" parent="b_bot_ee_link" />
   <!-- Spawn and attach gripper -->
-  <xacro:include filename="$(find aist_scene_description)/urdf/robotiq_85_gripper_with_ft300.urdf.xacro" />
-  <xacro:robotiq_85_gripper_with_ft300 prefix="a_bot_" parent="a_bot_ee_link" />
-  <xacro:include filename="$(find aist_scene_description)/urdf/single_suction_gripper_with_ft300.urdf.xacro" />
-  <xacro:single_suction_gripper_with_ft300 prefix="b_bot_" parent = "b_bot_ee_link" />
+  <xacro:include filename="$(find o2as_scene_description)/urdf/robotiq_85_gripper_with_tip_link.urdf.xacro" />
+  <xacro:robotiq_85_gripper_with_tip_link prefix="a_bot_"
+					  parent="a_bot_ft300_frange_link">
+    <origin xyz="0 0 0" rpy="0 0 0"/>
+  </xacro:robotiq_85_gripper_with_tip_link>
+  <xacro:include filename="$(find o2as_scene_description)/urdf/single_suction_gripper.urdf.xacro" />
+  <xacro:single_suction_gripper_o2as prefix="b_bot_"
+				     parent="b_bot_ft300_frange_link">
+    <origin xyz="0 0 0" rpy="0 0 0"/>
+  </xacro:single_suction_gripper_o2as>
   <!-- Add PhoXi 3D scanner -->
   <xacro:include filename="$(find o2as_scene_description)/urdf/phoxi_m_camera.urdf.xacro" />

File: aist_scene_description/urdf/single_suction_gripper_with_ft300.urdf.xacro (robot description, xacro)
@@ -26,5 +26,7 @@
     <xacro:include filename="$(find o2as_scene_description)/urdf/single_suction_gripper.urdf.xacro" />
     <xacro:single_suction_gripper_o2as prefix="${prefix}" parent="${parent}">
-        <origin rpy="0.0 0.0 0.0" xyz="${ft300_length} 0.0 0.0"/>
+      <origin rpy="0.0 0.0 0.0" xyz="${ft300_length} 0.0 0.0"/>
+      <!-- <oeigin rpy="${0.0*pi/180} ${1.5*pi/180} ${-0.3*pi/180}" -->
+      <!-- 	      xyz="${ft300_length} 0.0 0.0"/> -->
     </xacro:single_suction_gripper_o2as>
   </xacro:macro>

File: o2as_scene_description/urdf/single_suction_gripper.urdf.xacro (robot description, xacro)
@@ -17,6 +17,6 @@
       <collision>
       <!-- avoid collision -->
-        <origin xyz="0.188 -0.035 -0.035" rpy="0 0 ${pi/2}"/>
-	<!-- <origin xyz="0.187 -0.035 -0.035" rpy="0 0 ${pi/2}"/> -->
+        <!-- <origin xyz="0.188 -0.035 -0.035" rpy="0 0 ${pi/2}"/> -->
+	<origin xyz="0.187 -0.035 -0.035" rpy="0 0 ${pi/2}"/>
 	<geometry>
 	  <mesh filename="package://o2as_scene_description/meshes/single_suction_gripper.vhacd.dae" scale="0.001 0.001 0.001"/>
@@ -32,5 +32,5 @@
       <parent link="${parent}"/>
       <child  link="${prefix}single_suction_gripper_base_link"/>
-       <xacro:insert_block name="origin"/>
+      <xacro:insert_block name="origin"/>
     </joint>
     <!-- A link representing the tip of the pad and a joint attaching
@@ -40,8 +40,5 @@
       <parent link="${prefix}single_suction_gripper_base_link"/>
       <child  link="${prefix}single_suction_gripper_pad_link"/>
-      <!-- <origin xyz="0.187 0 0" rpy="0 0 0"/> -->
-      <origin xyz="0.186933357299 -0.000978789714711
-		   -0.00489508933357"
-	      rpy="${0.0*pi/180} ${1.5*pi/180} ${-0.3*pi/180}"/>>
+      <origin xyz="0.187 0 0" rpy="0 0 0"/>
     </joint>
   </xacro:macro>

Commit message: Add AR marker to a_bot.

File: aist_scene_description/urdf/aist_base_scene.urdf.xacro (robot description, xacro)
@@ -18,5 +18,5 @@
   <xacro:include filename="$(find o2as_scene_description)/urdf/ur5.urdf.xacro" />
   <!-- Scene items (trays, bins...) -->
-  <xacro:include filename="$(find aist_scene_description)/urdf/aist_kitting_scene.xacro" />
+  <!-- <xacro:include filename="$(find aist_scene_description)/urdf/aist_kitting_scene.xacro" /> -->
   <!-- Robot bases -->
   <!-- Putting these at height 0.0 makes them intersect with the ground, so they are elevated. -->
@@ -93,4 +93,9 @@
   <!-- Add AR markers -->
   <xacro:include filename="$(find aist_gazebo)/urdf/aist_ar_marker.urdf.xacro"/>
+  <xacro:aist_ar_marker prefix="a_bot_"
+			parent="a_bot_robotiq_85_tip_link"
+			marker_id="26">
+    <origin xyz="0.0 0.0 0.0185" rpy="0 0 0"/>
+  </xacro:aist_ar_marker>
   <xacro:aist_ar_marker prefix="b_bot_"
       parent="b_bot_single_suction_gripper_base_link"

Commit message: Revert rviz config. files.

File: aist_scene_description/urdf/aist_base_scene.urdf.xacro (robot description, xacro)
@@ -81,7 +81,10 @@
   <xacro:include filename="$(find o2as_scene_description)/urdf/single_suction_gripper.urdf.xacro" />
   <xacro:single_suction_gripper_o2as prefix="b_bot_"
-				     parent="b_bot_ft300_frange_link">
-    <origin xyz="0 0 0" rpy="0 0 0"/>
+  				     parent="b_bot_ft300_frange_link">
+    <origin xyz="0 0 0" rpy="0 ${0*pi/180} 0"/>
   </xacro:single_suction_gripper_o2as>
+  <!-- <xacro:include filename="$(find aist_scene_description)/urdf/single_suction_gripper_with_ft300.urdf.xacro" /> -->
+  <!-- <xacro:single_suction_gripper_with_ft300 prefix="b_bot_" -->
+  <!-- 				     parent="b_bot_ee_link"/> -->
   <!-- Add PhoXi 3D scanner -->
   <xacro:include filename="$(find o2as_scene_description)/urdf/phoxi_m_camera.urdf.xacro" />
