Commit message: Fixed bug in printing transforations represented by quaternions.

File: aist_scene_description/urdf/aist_base_scene.urdf.xacro (robot description, xacro)
@@ -84,19 +84,19 @@
     <origin xyz="0 0 0" rpy="0 ${0*pi/180} 0"/>
   </xacro:single_suction_gripper_o2as>
-  <!-- <xacro:include filename="$(find aist_scene_description)/urdf/single_suction_gripper_with_ft300.urdf.xacro" /> -->
-  <!-- <xacro:single_suction_gripper_with_ft300 prefix="b_bot_" -->
-  <!-- 				     parent="b_bot_ee_link"/> -->
   <!-- Add PhoXi 3D scanner -->
   <xacro:include filename="$(find o2as_scene_description)/urdf/phoxi_m_camera.urdf.xacro" />
   <xacro:phoxi_m_camera prefix="a_" parent="o2as_ground">
+    <!-- <origin xyz="0.679997723974 0.0866831188148 1.46958049634" -->
+    <!-- 	    rpy="${-143.76356757*pi/180} -->
+    <!-- 		 ${0.312453823638*pi/180} ${85.5565266354*pi/180}"/> -->
     <origin xyz="0.679997723974 0.0866831188148 1.46958049634"
-	    rpy="${-143.76356757*pi/180}
-		 ${0.312453823638*pi/180} ${85.5565266354*pi/180}"/>
+	    rpy="${-145.0*pi/180}
+		 ${0.0*pi/180} ${90.0*pi/180}"/>
   </xacro:phoxi_m_camera>
   <!-- Add AR markers -->
   <xacro:include filename="$(find aist_gazebo)/urdf/aist_ar_marker.urdf.xacro"/>
   <xacro:aist_ar_marker prefix="a_bot_"
-			parent="a_bot_robotiq_85_tip_link"
-			marker_id="26">
+  			parent="a_bot_robotiq_85_tip_link"
+  			marker_id="26">
     <origin xyz="0.0 0.0 0.0185" rpy="0 0 0"/>
   </xacro:aist_ar_marker>

Commit message: Fix base scene

File: aist_scene_description/urdf/aist_base_scene.urdf.xacro (robot description, xacro)
@@ -3,12 +3,12 @@
         name="aist_base_scene" >
   <!-- Calibration help: If the robot is not moving far enough to the calibration point, increase these distances -->
-  <xacro:property name="a_bot_x" value="-0.006"/>
-  <xacro:property name="a_bot_y" value="-0.625"/>
-  <xacro:property name="a_bot_z" value="0.78" />
+  <xacro:property name="a_bot_x" value="0"/>
+  <xacro:property name="a_bot_y" value="0"/>
+  <xacro:property name="a_bot_z" value="0"/>
   <!-- <xacro:property name="a_bot_theta" value="${pi}"/> -->
   <xacro:property name="b_bot_x" value="0"/>
   <xacro:property name="b_bot_y" value="0.50"/>
   <xacro:property name="b_bot_theta" value="${pi}"/>
-  <xacro:property name="bots_z" value="0.77"/>
+  <xacro:property name="bots_z" value="0"/>
   <!-- This is the main file defining our robot arrangement and physical environment. -->
   <!-- common stuff -->
@@ -22,25 +22,25 @@
   <!-- Putting these at height 0.0 makes them intersect with the ground, so they are elevated. -->
   <!-- There are some instabilities when the box is big, for some reason. -->
-  <xacro:include filename="$(find aist_scene_description)/urdf/aist_base.xacro" />
-  <xacro:aist_base boxname="a_bot_base_smfl" parent="o2as_ground">
-    <origin xyz="${a_bot_x-0.225/2} ${a_bot_y-0.225/2} 0.72" rpy="0 0 0" />
-  </xacro:aist_base>
-  <xacro:aist_base boxname="b_bot_base_smfl" parent="o2as_ground">
-    <origin xyz="${b_bot_x-0.225/2} ${b_bot_y-0.225/2} 0.72" rpy="0 0 0" />
-  </xacro:aist_base>
+  <!-- <xacro:include filename="$(find aist_scene_description)/urdf/aist_base.xacro" /> -->
+  <!-- <xacro:aist_base boxname="a_bot_base_smfl" parent="o2as_ground"> -->
+    <!-- <origin xyz="${a_bot_x-0.225/2} ${a_bot_y-0.225/2} 0.72" rpy="0 0 0" /> -->
+  <!-- </xacro:aist_base> -->
+  <!-- <xacro:aist_base boxname="b_bot_base_smfl" parent="o2as_ground"> -->
+    <!-- <origin xyz="${b_bot_x-0.225/2} ${b_bot_y-0.225/2} 0.72" rpy="0 0 0" /> -->
+  <!-- </xacro:aist_base> -->
   <!-- Main workspace -->
   <!-- The surface is 0.01 m below the robot bases and the "workspace_center" frame. -->
   <xacro:include filename="$(find o2as_scene_description)/urdf/o2as_box.xacro" />
-  <xacro:property name="plate_w" value="0.598"/>
-  <xacro:property name="plate_l" value="0.899"/>
-  <xacro:o2as_box boxname="workbox" box_w="${plate_w}" box_l="${plate_l}" box_h=".01" parent="o2as_ground">
-    <origin xyz="${-plate_w/2} ${-plate_l/2-0.062} ${bots_z}" rpy="0 0 0" />
-  </xacro:o2as_box>
-  <link name="workspace_center" />
-  <joint name="world_to_workspace" type="fixed">
-    <parent link="o2as_ground" />
-    <child link="workspace_center" />
-    <origin xyz="0.0 0.0 ${bots_z+.01}" rpy="0.0 0.0 0.0" />
-  </joint>
+  <!-- <xacro:property name="plate_w" value="0.598"/> -->
+  <!-- <xacro:property name="plate_l" value="0.899"/> -->
+  <!-- <xacro:o2as_box boxname="workbox" box_w="${plate_w}" box_l="${plate_l}" box_h=".01" parent="o2as_ground"> -->
+    <!-- <origin xyz="${-plate_w/2} ${-plate_l/2-0.062} ${bots_z}" rpy="0 0 0" /> -->
+  <!-- </xacro:o2as_box> -->
+  <!-- <link name="workspace_center" /> -->
+  <!-- <joint name="world_to_workspace" type="fixed"> -->
+    <!-- <parent link="o2as_ground" /> -->
+    <!-- <child link="workspace_center" /> -->
+    <!-- <origin xyz="0.0 0.0 ${bots_z+.01}" rpy="0.0 0.0 0.0" /> -->
+  <!-- </joint> -->
   <!-- robot arms -->
   <xacro:ur5_robot prefix="a_bot_" joint_limited="false"
@@ -51,5 +51,5 @@
     wrist_2_lower_limit="${-pi}" wrist_2_upper_limit="${pi}"
     wrist_3_lower_limit="${-pi}" wrist_3_upper_limit="${pi}"/>
-  <xacro:ur5_robot prefix="b_bot_" joint_limited="false"
+  <!-- <xacro:ur5_robot prefix="b_bot_" joint_limited="false"
     shoulder_pan_lower_limit="${-pi}" shoulder_pan_upper_limit="${pi}"
     shoulder_lift_lower_limit="${-pi}" shoulder_lift_upper_limit="${pi}"
@@ -57,5 +57,5 @@
     wrist_1_lower_limit="${-pi}" wrist_1_upper_limit="${pi}"
     wrist_2_lower_limit="${-pi}" wrist_2_upper_limit="${pi}"
-    wrist_3_lower_limit="${-pi}" wrist_3_upper_limit="${pi}"/>
+    wrist_3_lower_limit="${-pi}" wrist_3_upper_limit="${pi}"/> -->
   <link name="o2as_ground" />
   <joint name="world_a_bot_joint" type="fixed">
@@ -64,13 +64,13 @@
     <origin xyz="${a_bot_x} ${a_bot_y} ${a_bot_z}" rpy="0.0 0.0 0.0" />
   </joint>
-  <joint name="world_b_bot_joint" type="fixed">
-    <parent link="o2as_ground" />
-    <child link = "b_bot_base_link" />
-    <origin xyz="${b_bot_x} ${b_bot_y} ${bots_z}" rpy="0.0 0.0 ${b_bot_theta}" />
-  </joint>
+  <!-- <joint name="world_b_bot_joint" type="fixed"> -->
+    <!-- <parent link="o2as_ground" /> -->
+    <!-- <child link = "b_bot_base_link" /> -->
+    <!-- <origin xyz="${b_bot_x} ${b_bot_y} ${bots_z}" rpy="0.0 0.0 ${b_bot_theta}" /> -->
+  <!-- </joint> -->
   <!-- Spawn and attach force sensor -->
   <xacro:include filename="$(find o2as_scene_description)/urdf/ft300.urdf.xacro" />
   <xacro:ft300 prefix="a_bot_" parent="a_bot_ee_link" />
-  <xacro:ft300 prefix="b_bot_" parent="b_bot_ee_link" />
+  <!-- <xacro:ft300 prefix="b_bot_" parent="b_bot_ee_link" /> -->
   <!-- Spawn and attach gripper -->
   <xacro:include filename="$(find o2as_scene_description)/urdf/robotiq_85_gripper_with_tip_link.urdf.xacro" />
@@ -79,36 +79,40 @@
     <origin xyz="0 0 0" rpy="0 0 0"/>
   </xacro:robotiq_85_gripper_with_tip_link>
-  <xacro:include filename="$(find o2as_scene_description)/urdf/single_suction_gripper.urdf.xacro" />
+  <!-- <xacro:include filename="$(find o2as_scene_description)/urdf/single_suction_gripper.urdf.xacro" />
   <xacro:single_suction_gripper_o2as prefix="b_bot_"
   				     parent="b_bot_ft300_frange_link">
     <origin xyz="0 0 0" rpy="0 ${0*pi/180} 0"/>
-  </xacro:single_suction_gripper_o2as>
+  </xacro:single_suction_gripper_o2as> -->
   <!-- <xacro:include filename="$(find aist_scene_description)/urdf/single_suction_gripper_with_ft300.urdf.xacro" /> -->
   <!-- <xacro:single_suction_gripper_with_ft300 prefix="b_bot_" -->
   <!-- 				     parent="b_bot_ee_link"/> -->
+  <!-- Add virtual wall to avoid collision between robot and PhoXi -->
+  <xacro:o2as_box boxname="vwall1" box_w="0.01" box_l="0.5" box_h="1.5" parent="o2as_ground">
+    <origin xyz="0.5 -0.25 0" rpy="0 0 0"/>
+  </xacro:o2as_box>
   <!-- Add PhoXi 3D scanner -->
   <xacro:include filename="$(find o2as_scene_description)/urdf/phoxi_m_camera.urdf.xacro" />
   <xacro:phoxi_m_camera prefix="a_" parent="o2as_ground">
-    <origin xyz="0.679997723974 0.0866831188148 1.46958049634"
+    <origin xyz="0.679997723974 0.5866831188148 1.46958049634"
 	    rpy="${-143.76356757*pi/180}
 		 ${0.312453823638*pi/180} ${85.5565266354*pi/180}"/>
   </xacro:phoxi_m_camera>
   <!-- Add AR markers -->
-  <xacro:include filename="$(find aist_gazebo)/urdf/aist_ar_marker.urdf.xacro"/>
-  <xacro:aist_ar_marker prefix="a_bot_"
+  <!-- <xacro:include filename="$(find aist_gazebo)/urdf/aist_ar_marker.urdf.xacro"/> -->
+  <!-- <xacro:aist_ar_marker prefix="a_bot_"
 			parent="a_bot_robotiq_85_tip_link"
 			marker_id="26">
     <origin xyz="0.0 0.0 0.0185" rpy="0 0 0"/>
-  </xacro:aist_ar_marker>
-  <xacro:aist_ar_marker prefix="b_bot_"
+  </xacro:aist_ar_marker> -->
+  <!-- <xacro:aist_ar_marker prefix="b_bot_"
       parent="b_bot_single_suction_gripper_base_link"
       marker_id="26">
     <origin xyz="0.063 0.0 0.0215" rpy="0 0 0"/>
-  </xacro:aist_ar_marker>
-  <xacro:aist_ar_marker_16cm prefix="workspace_"
+  </xacro:aist_ar_marker> -->
+  <!-- <xacro:aist_ar_marker_16cm prefix="workspace_"
       parent="workspace_center"
       marker_id="32">
     <origin xyz="0.0 0.0 0.0005" rpy="0 0 0"/>
-  </xacro:aist_ar_marker_16cm>
+  </xacro:aist_ar_marker_16cm> -->
   <!-- I would like to remove the "world" link definition, but apparently it is necessary for Gazebo -->
   <link name="world" />
@@ -116,5 +120,5 @@
     <parent link="world" />
     <child link="o2as_ground" />
-    <origin xyz="0.0 0.0 0.0" rpy="0.0 0.0 0.0" />
+    <origin xyz="0.0 0.0 0.01" rpy="0.0 0.0 0.0" />
   </joint>
 </robot>

Commit message: Add virtual table under the base height

File: aist_scene_description/urdf/aist_base_scene.urdf.xacro (robot description, xacro)
@@ -87,5 +87,8 @@
   <!-- <xacro:single_suction_gripper_with_ft300 prefix="b_bot_" -->
   <!-- 				     parent="b_bot_ee_link"/> -->
-  <!-- Add virtual wall to avoid collision between robot and PhoXi -->
+  <!-- Add virtual wall to avoid collisions-->
+  <xacro:o2as_box boxname="vtable" box_w="2" box_l="2" box_h="0.01" parent="world">
+    <origin xyz="-1 0 0" rpy="0 0 0"/>
+  </xacro:o2as_box>
   <xacro:o2as_box boxname="vwall1" box_w="0.01" box_l="0.5" box_h="1.5" parent="o2as_ground">
     <origin xyz="0.5 -0.25 0" rpy="0 0 0"/>

Commit message: Modified launch files of 'aist_moveit_config' to change configurations by arguments

File: aist_scene_description/urdf/aist_base_scene.urdf.xacro (robot description, xacro)
@@ -101,21 +101,4 @@
 		 ${0.312453823638*pi/180} ${85.5565266354*pi/180}"/>
   </xacro:phoxi_m_camera>
-  <!-- Add AR markers -->
-  <!-- <xacro:include filename="$(find aist_gazebo)/urdf/aist_ar_marker.urdf.xacro"/> -->
-  <!-- <xacro:aist_ar_marker prefix="a_bot_"
-			parent="a_bot_robotiq_85_tip_link"
-			marker_id="26">
-    <origin xyz="0.0 0.0 0.0185" rpy="0 0 0"/>
-  </xacro:aist_ar_marker> -->
-  <!-- <xacro:aist_ar_marker prefix="b_bot_"
-      parent="b_bot_single_suction_gripper_base_link"
-      marker_id="26">
-    <origin xyz="0.063 0.0 0.0215" rpy="0 0 0"/>
-  </xacro:aist_ar_marker> -->
-  <!-- <xacro:aist_ar_marker_16cm prefix="workspace_"
-      parent="workspace_center"
-      marker_id="32">
-    <origin xyz="0.0 0.0 0.0005" rpy="0 0 0"/>
-  </xacro:aist_ar_marker_16cm> -->
   <!-- I would like to remove the "world" link definition, but apparently it is necessary for Gazebo -->
   <link name="world" />

Commit message: Moved scene origin to the base of a_bot for checking calibration.

File: aist_scene_description/urdf/aist_base_scene.urdf.xacro (robot description, xacro)
@@ -31,5 +31,5 @@
   <!-- Main workspace -->
   <!-- The surface is 0.01 m below the robot bases and the "workspace_center" frame. -->
-  <xacro:include filename="$(find o2as_scene_description)/urdf/o2as_box.xacro" />
+  <xacro:include filename="$(find o2as_scene_description)/urdf/o2as_box.xacro"/>
   <!-- <xacro:property name="plate_w" value="0.598"/> -->
   <!-- <xacro:property name="plate_l" value="0.899"/> -->
@@ -91,14 +91,22 @@
     <origin xyz="-1 0 0" rpy="0 0 0"/>
   </xacro:o2as_box>
-  <xacro:o2as_box boxname="vwall1" box_w="0.01" box_l="0.5" box_h="1.5" parent="o2as_ground">
-    <origin xyz="0.5 -0.25 0" rpy="0 0 0"/>
+  <xacro:o2as_box boxname="vwall1" box_w="0.01" box_l="0.5" box_h="0.6" parent="o2as_ground">
+    <origin xyz="0.67 0.25 0" rpy="0 0 0"/>
   </xacro:o2as_box>
   <!-- Add PhoXi 3D scanner -->
   <xacro:include filename="$(find o2as_scene_description)/urdf/phoxi_m_camera.urdf.xacro" />
   <xacro:phoxi_m_camera prefix="a_" parent="o2as_ground">
-    <origin xyz="0.679997723974 0.5866831188148 1.46958049634"
-	    rpy="${-143.76356757*pi/180}
-		 ${0.312453823638*pi/180} ${85.5565266354*pi/180}"/>
+    <origin xyz="0.533753808105 0.512093727977 0.904786289459"
+	    rpy="${-152.051675662*pi/180} ${1.32492983016*pi/180} ${88.0374935002*pi/180}"/>
+    <!-- <origin xyz="0.679997723974 0.5 0.7" -->
+    <!-- 	    rpy="${-143.76356757*pi/180} -->
+    <!-- 		 ${0.312453823638*pi/180} ${85.5565266354*pi/180}"/> -->
   </xacro:phoxi_m_camera>
+  <link name="workspace_center"/>
+  <joint name="a_bot_to_workspace_joint" type="fixed">
+    <parent link="o2as_ground"/>
+    <child link="workspace_center"/>
+    <origin xyz="0 0.5 0" rpy="0 0 0"/>
+  </joint>
   <!-- I would like to remove the "world" link definition, but apparently it is necessary for Gazebo -->
   <link name="world" />

File: aist_scene_description/urdf/calibration.urdf.xacro (robot description, xacro)
@@ -12,10 +12,4 @@
     <origin xyz="0.063 0.0 0.0215" rpy="0 0 0"/>
   </xacro:aist_ar_marker> -->
-  <link name="workspace_center"/>
-  <joint name="a_bot_to_workspace_joint" type="fixed">
-    <parent link="a_bot_base_link"/>
-    <child link="workspace_center"/>
-    <origin xyz="0 0.5 0" rpy="0 0 0"/>
-  </joint>
   <xacro:aist_ar_marker_16cm prefix="workspace_" parent="workspace_center" marker_id="32">
     <origin xyz="0.0 0.0 0.0005" rpy="0 0 0"/>

Commit message: Changed robot_base_frame from "xxx_base_link" to "workspace_center".

File: aist_scene_description/urdf/aist_base_scene.urdf.xacro (robot description, xacro)
@@ -12,22 +12,9 @@
   <!-- This is the main file defining our robot arrangement and physical environment. -->
   <!-- common stuff -->
-  <xacro:include filename="$(find ur_description)/urdf/common.gazebo.xacro" />
-  <xacro:include filename="$(find aist_gazebo)/urdf/aist_base_scene.gazebo" />
-  <!-- robots -->
-  <xacro:include filename="$(find o2as_scene_description)/urdf/ur5.urdf.xacro" />
-  <!-- Scene items (trays, bins...) -->
-  <!-- <xacro:include filename="$(find aist_scene_description)/urdf/aist_kitting_scene.xacro" /> -->
-  <!-- Robot bases -->
-  <!-- Putting these at height 0.0 makes them intersect with the ground, so they are elevated. -->
-  <!-- There are some instabilities when the box is big, for some reason. -->
-  <!-- <xacro:include filename="$(find aist_scene_description)/urdf/aist_base.xacro" /> -->
-  <!-- <xacro:aist_base boxname="a_bot_base_smfl" parent="o2as_ground"> -->
-    <!-- <origin xyz="${a_bot_x-0.225/2} ${a_bot_y-0.225/2} 0.72" rpy="0 0 0" /> -->
-  <!-- </xacro:aist_base> -->
-  <!-- <xacro:aist_base boxname="b_bot_base_smfl" parent="o2as_ground"> -->
-    <!-- <origin xyz="${b_bot_x-0.225/2} ${b_bot_y-0.225/2} 0.72" rpy="0 0 0" /> -->
-  <!-- </xacro:aist_base> -->
+  <xacro:include filename="$(find ur_description)/urdf/common.gazebo.xacro"/>
+  <xacro:include filename="$(find aist_gazebo)/urdf/aist_base_scene.gazebo"/>
   <!-- Main workspace -->
   <!-- The surface is 0.01 m below the robot bases and the "workspace_center" frame. -->
+  <link name="o2as_ground"/>
   <xacro:include filename="$(find o2as_scene_description)/urdf/o2as_box.xacro"/>
   <xacro:property name="plate_w" value="0.9"/>
@@ -37,13 +24,14 @@
 		  box_w="${plate_w}" box_l="${plate_l}" box_h="${plate_h}"
 		  parent="o2as_ground">
-    <origin xyz="${-plate_w/2} ${-plate_l/2} ${bots_z - plate_h}" rpy="0 0 0" />
+    <origin xyz="${-plate_w/2} ${-plate_l/2} ${bots_z - plate_h}" rpy="0 0 0"/>
   </xacro:o2as_box>
-  <link name="workspace_center" />
+  <link name="workspace_center"/>
   <joint name="world_to_workspace" type="fixed">
-    <parent link="o2as_ground" />
-    <child link="workspace_center" />
-    <origin xyz="0 0 ${bots_z}" rpy="0 0 0" />
+    <parent link="o2as_ground"/>
+    <child link="workspace_center"/>
+    <origin xyz="0 0 ${bots_z}" rpy="0 0 0"/>
   </joint>
   <!-- robot arms -->
+  <xacro:include filename="$(find o2as_scene_description)/urdf/ur5.urdf.xacro"/>
   <xacro:ur5_robot prefix="a_bot_" joint_limited="false"
     shoulder_pan_lower_limit="${-pi}" shoulder_pan_upper_limit="${pi}"
@@ -60,52 +48,49 @@
     wrist_2_lower_limit="${-pi}" wrist_2_upper_limit="${pi}"
     wrist_3_lower_limit="${-pi}" wrist_3_upper_limit="${pi}"/>
-  <link name="o2as_ground" />
   <joint name="world_a_bot_joint" type="fixed">
-    <parent link="o2as_ground" />
-    <child  link= "a_bot_base_link" />
-    <origin xyz="${a_bot_x} ${a_bot_y} ${bots_z}" rpy="0 0 0" />
+    <parent link="o2as_ground"/>
+    <child  link= "a_bot_base_link"/>
+    <origin xyz="${a_bot_x} ${a_bot_y} ${bots_z}" rpy="0 0 0"/>
   </joint>
   <joint name="world_b_bot_joint" type="fixed">
-    <parent link="o2as_ground" />
-    <child  link= "b_bot_base_link" />
-    <origin xyz="${b_bot_x} ${b_bot_y} ${bots_z}" rpy="0 0 ${b_bot_theta}" />
+    <parent link="o2as_ground"/>
+    <child  link= "b_bot_base_link"/>
+    <origin xyz="${b_bot_x} ${b_bot_y} ${bots_z}" rpy="0 0 ${b_bot_theta}"/>
   </joint>
   <!-- Spawn and attach force sensor -->
-  <xacro:include filename="$(find o2as_scene_description)/urdf/ft300.urdf.xacro" />
-  <xacro:ft300 prefix="a_bot_" parent="a_bot_ee_link" />
-  <xacro:ft300 prefix="b_bot_" parent="b_bot_ee_link" />
+  <xacro:include filename="$(find o2as_scene_description)/urdf/ft300.urdf.xacro"/>
+  <xacro:ft300 prefix="a_bot_" parent="a_bot_ee_link"/>
+  <xacro:ft300 prefix="b_bot_" parent="b_bot_ee_link"/>
   <!-- Spawn and attach gripper -->
-  <xacro:include filename="$(find o2as_scene_description)/urdf/robotiq_85_gripper_with_tip_link.urdf.xacro" />
+  <xacro:include filename="$(find o2as_scene_description)/urdf/robotiq_85_gripper_with_tip_link.urdf.xacro"/>
   <xacro:robotiq_85_gripper_with_tip_link prefix="a_bot_"
 					  parent="a_bot_ft300_frange_link">
     <origin xyz="0 0 0" rpy="0 0 0"/>
   </xacro:robotiq_85_gripper_with_tip_link>
-  <xacro:include filename="$(find o2as_scene_description)/urdf/single_suction_gripper.urdf.xacro" />
+  <xacro:include filename="$(find o2as_scene_description)/urdf/single_suction_gripper.urdf.xacro"/>
   <xacro:single_suction_gripper_o2as prefix="b_bot_"
   				     parent="b_bot_ft300_frange_link">
-    <origin xyz="0 0 0" rpy="0 ${0*pi/180} 0"/>
+    <origin xyz="0 0 0" rpy="0 ${0.8*pi/180} ${-0.5*pi/180}"/>
   </xacro:single_suction_gripper_o2as>
   <!-- Add virtual wall to avoid collisions-->
-  <!-- <xacro:o2as_box boxname="table" box_w="0.9" box_l="0.75" box_h="0.01" parent="o2as_ground"> -->
-  <!--   <origin xyz="-0.45 -0.375 ${bots_z}" rpy="0 0 0"/> -->
-  <!-- </xacro:o2as_box> -->
   <xacro:o2as_box boxname="vwall1" box_w="0.01" box_l="0.5" box_h="0.6" parent="o2as_ground">
     <origin xyz="0.50 -0.25 ${bots_z}" rpy="0 0 0"/>
   </xacro:o2as_box>
   <!-- Add PhoXi 3D scanner -->
-  <xacro:include filename="$(find o2as_scene_description)/urdf/phoxi_m_camera.urdf.xacro" />
+  <xacro:include filename="$(find o2as_scene_description)/urdf/phoxi_m_camera.urdf.xacro"/>
   <xacro:phoxi_m_camera prefix="a_" parent="o2as_ground">
-    <origin xyz="0.533753808105 0.0 1.674786289459"
-	    rpy="${-152.051675662*pi/180} ${1.32492983016*pi/180} ${88.0374935002*pi/180}"/>
-    <!-- <origin xyz="0.679997723974 0.5 0.7" -->
-    <!-- 	    rpy="${-143.76356757*pi/180} -->
-    <!-- 		 ${0.312453823638*pi/180} ${85.5565266354*pi/180}"/> -->
+    <origin xyz="0.547941636523
+		 -0.00827443204237
+		 1.67030171767"
+	    rpy="${-151.493605482*pi/180}
+		 ${0.698490882792*pi/180}
+		 ${85.0482907121*pi/180}"/>
   </xacro:phoxi_m_camera>
   <!-- I would like to remove the "world" link definition, but apparently it is necessary for Gazebo -->
-  <link name="world" />
+  <link name="world"/>
   <joint name="world_o2as_joint" type="fixed">
-    <parent link="world" />
-    <child link="o2as_ground" />
-    <origin xyz="0 0 0" rpy="0 0 0" />
+    <parent link="world"/>
+    <child link="o2as_ground"/>
+    <origin xyz="0 0 0" rpy="0 0 0"/>
   </joint>
 </robot>

File: aist_scene_description/urdf/aist_calibration.urdf.xacro (robot description, xacro)
@@ -1,4 +1,4 @@
 <?xml version="1.0"?>
-<robot xmlns:xacro="http://wiki.ros.org/xacro" name="calibration">
+<robot xmlns:xacro="http://wiki.ros.org/xacro" name="aist_calibration">
   <xacro:include filename="$(find aist_scene_description)/urdf/aist_base_scene.urdf.xacro"/>
   <!-- Add AR markers -->
