Commit message: Precision gripper added for simulation.

File: aist_scene_description/urdf/aist_base_scene.urdf.xacro (robot description, xacro)
@@ -68,4 +68,8 @@
     <origin xyz="0 0 0" rpy="0 0 0"/>
   </xacro:robotiq_85_gripper_with_tip_link>
+  <!-- <xacro:include filename="$(find o2as_scene_description)/urdf/InnerOnlyGripper.xacro" /> -->
+  <!-- <xacro:InnerOnlyGripper prefix="a_bot_"  grippername = "gripper" parent = "a_bot_ft300_frange_link"> -->
+  <!--   <origin xyz="0 0 0" rpy="0 ${90*pi/180} 0"/> -->
+  <!-- </xacro:InnerOnlyGripper> -->
   <xacro:include filename="$(find o2as_scene_description)/urdf/single_suction_gripper.urdf.xacro"/>
   <xacro:single_suction_gripper_o2as prefix="b_bot_"
@@ -74,7 +78,7 @@
   </xacro:single_suction_gripper_o2as>
   <!-- Add virtual wall to avoid collisions-->
-  <xacro:o2as_box boxname="vwall1" box_w="0.01" box_l="0.5" box_h="0.6" parent="o2as_ground">
-    <origin xyz="0.50 -0.25 ${bots_z}" rpy="0 0 0"/>
-  </xacro:o2as_box>
+  <!-- <xacro:o2as_box boxname="vwall1" box_w="0.01" box_l="0.5" box_h="0.6" parent="o2as_ground"> -->
+  <!--   <origin xyz="0.50 -0.25 ${bots_z}" rpy="0 0 0"/> -->
+  <!-- </xacro:o2as_box> -->
   <!-- Add PhoXi 3D scanner -->
   <xacro:include filename="$(find o2as_scene_description)/urdf/phoxi_m_camera.urdf.xacro"/>

File: aist_scene_description/urdf/pgrp_base_scene.urdf.xacro (robot description, xacro)
@@ -1,12 +1,12 @@
 <?xml version="1.0"?>
 <robot xmlns:xacro="http://www.ros.org/wiki/xacro"
-        name="ur5e_base_scene" >
+        name="pgrp_base_scene" >
   <!-- Calibration help: If the robot is not moving far enough to the calibration point, increase these distances -->
-  <xacro:property name="c_bot_x" value="0"/>
-  <xacro:property name="c_bot_y" value="-0.4875"/>
-  <!-- <xacro:property name="c_bot_theta" value="${pi}"/> -->
-  <xacro:property name="d_bot_x" value="0"/>
-  <xacro:property name="d_bot_y" value="0.4875"/>
-  <xacro:property name="d_bot_theta" value="${pi}"/>
+  <xacro:property name="a_bot_x" value="0"/>
+  <xacro:property name="a_bot_y" value="-0.4875"/>
+  <!-- <xacro:property name="a_bot_theta" value="${pi}"/> -->
+  <xacro:property name="b_bot_x" value="0"/>
+  <xacro:property name="b_bot_y" value="0.4875"/>
+  <xacro:property name="b_bot_theta" value="${pi}"/>
   <xacro:property name="bots_z" value="0.77"/>
   <!-- This is the main file defining our robot arrangement and physical environment. -->
@@ -33,6 +33,6 @@
   </joint>
   <!-- robot arms -->
-  <xacro:include filename="$(find o2as_scene_description)/urdf/ur5e.urdf.xacro"/>
-  <xacro:ur5e_robot prefix="c_bot_" joint_limited="false"
+  <xacro:include filename="$(find o2as_scene_description)/urdf/ur5.urdf.xacro"/>
+  <xacro:ur5_robot prefix="a_bot_" joint_limited="false"
     shoulder_pan_lower_limit="${-pi}" shoulder_pan_upper_limit="${pi}"
     shoulder_lift_lower_limit="${-pi}" shoulder_lift_upper_limit="${pi}"
@@ -41,5 +41,5 @@
     wrist_2_lower_limit="${-pi}" wrist_2_upper_limit="${pi}"
     wrist_3_lower_limit="${-pi}" wrist_3_upper_limit="${pi}"/>
-  <xacro:ur5e_robot prefix="d_bot_" joint_limited="false"
+  <xacro:ur5_robot prefix="b_bot_" joint_limited="false"
     shoulder_pan_lower_limit="${-pi}" shoulder_pan_upper_limit="${pi}"
     shoulder_lift_lower_limit="${-pi}" shoulder_lift_upper_limit="${pi}"
@@ -48,33 +48,28 @@
     wrist_2_lower_limit="${-pi}" wrist_2_upper_limit="${pi}"
     wrist_3_lower_limit="${-pi}" wrist_3_upper_limit="${pi}"/>
-  <joint name="world_c_bot_joint" type="fixed">
+  <joint name="world_a_bot_joint" type="fixed">
     <parent link="o2as_ground"/>
-    <child  link= "c_bot_base_link"/>
-    <origin xyz="${c_bot_x} ${c_bot_y} ${bots_z}" rpy="0 0 0"/>
+    <child  link= "a_bot_base_link"/>
+    <origin xyz="${a_bot_x} ${a_bot_y} ${bots_z}" rpy="0 0 0"/>
   </joint>
-  <joint name="world_d_bot_joint" type="fixed">
+  <joint name="world_b_bot_joint" type="fixed">
     <parent link="o2as_ground"/>
-    <child  link= "d_bot_base_link"/>
-    <origin xyz="${d_bot_x} ${d_bot_y} ${bots_z}" rpy="0 0 ${d_bot_theta}"/>
+    <child  link= "b_bot_base_link"/>
+    <origin xyz="${b_bot_x} ${b_bot_y} ${bots_z}" rpy="0 0 ${b_bot_theta}"/>
   </joint>
   <!-- Spawn and attach force sensor -->
   <xacro:include filename="$(find o2as_scene_description)/urdf/ft300.urdf.xacro"/>
-  <xacro:ft300 prefix="c_bot_" parent="c_bot_ee_link"/>
-  <xacro:ft300 prefix="d_bot_" parent="d_bot_ee_link"/>
+  <xacro:ft300 prefix="a_bot_" parent="a_bot_ee_link"/>
+  <xacro:ft300 prefix="b_bot_" parent="b_bot_ee_link"/>
   <!-- Spawn and attach gripper -->
-  <xacro:include filename="$(find o2as_scene_description)/urdf/robotiq_85_gripper_with_tip_link.urdf.xacro"/>
-  <xacro:robotiq_85_gripper_with_tip_link prefix="c_bot_"
-					  parent="c_bot_ft300_frange_link">
-    <origin xyz="0 0 0" rpy="0 0 0"/>
-  </xacro:robotiq_85_gripper_with_tip_link>
-  <!-- <xacro:include filename="$(find o2as_scene_description)/urdf/InnerOnlyGripper.xacro" /> -->
-  <!-- <xacro:InnerOnlyGripper prefix="c_bot_"  grippername = "gripper" parent = "c_bot_ft300_frange_link"> -->
-  <!--   <origin xyz="0 0 0" rpy="0 ${90*pi/180} 0"/> -->
-  <!-- </xacro:InnerOnlyGripper> -->
-  <xacro:include filename="$(find o2as_scene_description)/urdf/dual_suction_gripper.urdf.xacro"/>
-  <xacro:dual_suction_gripper_o2as prefix="d_bot_"
-  				     parent="d_bot_ft300_frange_link">
+  <xacro:include filename="$(find aist_scene_description)/urdf/InnerOnlyGripper.urdf.xacro" />
+  <xacro:InnerOnlyGripper prefix="a_bot_"  grippername = "gripper" parent = "a_bot_ft300_frange_link">
+    <origin xyz="0 0 0" rpy="${-pi/2} 0 0"/>
+  </xacro:InnerOnlyGripper>
+  <xacro:include filename="$(find o2as_scene_description)/urdf/single_suction_gripper.urdf.xacro"/>
+  <xacro:single_suction_gripper_o2as prefix="b_bot_"
+  				     parent="b_bot_ft300_frange_link">
     <origin xyz="0 0 0" rpy="0 ${0.8*pi/180} ${-0.5*pi/180}"/>
-  </xacro:dual_suction_gripper_o2as>
+  </xacro:single_suction_gripper_o2as>
   <!-- Add virtual wall to avoid collisions-->
   <!-- <xacro:o2as_box boxname="vwall1" box_w="0.01" box_l="0.5" box_h="0.6" parent="o2as_ground"> -->
@@ -83,5 +78,5 @@
   <!-- Add PhoXi 3D scanner -->
   <xacro:include filename="$(find o2as_scene_description)/urdf/phoxi_m_camera.urdf.xacro"/>
-  <xacro:phoxi_m_camera prefix="b_" parent="o2as_ground">
+  <xacro:phoxi_m_camera prefix="a_" parent="o2as_ground">
     <origin xyz="0.547941636523
 		 -0.00827443204237

Commit message: Cleaning up.

File: aist_scene_description/urdf/aist_base_scene.urdf.xacro (robot description, xacro)
@@ -68,8 +68,4 @@
     <origin xyz="0 0 0" rpy="0 0 0"/>
   </xacro:robotiq_85_gripper_with_tip_link>
-  <!-- <xacro:include filename="$(find o2as_scene_description)/urdf/InnerOnlyGripper.xacro" /> -->
-  <!-- <xacro:InnerOnlyGripper prefix="a_bot_"  grippername = "gripper" parent = "a_bot_ft300_frange_link"> -->
-  <!--   <origin xyz="0 0 0" rpy="0 ${90*pi/180} 0"/> -->
-  <!-- </xacro:InnerOnlyGripper> -->
   <xacro:include filename="$(find o2as_scene_description)/urdf/single_suction_gripper.urdf.xacro"/>
   <xacro:single_suction_gripper_o2as prefix="b_bot_"

Commit message: Kitting scene modified.

File: aist_scene_description/urdf/aist_base_scene.urdf.xacro (robot description, xacro)
@@ -18,11 +18,11 @@
   <link name="o2as_ground"/>
   <xacro:include filename="$(find o2as_scene_description)/urdf/o2as_box.xacro"/>
-  <xacro:property name="plate_w" value="0.9"/>
-  <xacro:property name="plate_l" value="0.75"/>
-  <xacro:property name="plate_h" value="0.01"/>
+  <xacro:property name="table_w" value="0.9"/>
+  <xacro:property name="table_l" value="0.75"/>
+  <xacro:property name="table_h" value="0.01"/>
   <xacro:o2as_box boxname="workbox"
-		  box_w="${plate_w}" box_l="${plate_l}" box_h="${plate_h}"
+		  box_w="${table_w}" box_l="${table_l}" box_h="${table_h}"
 		  parent="o2as_ground">
-    <origin xyz="${-plate_w/2} ${-plate_l/2} ${bots_z - plate_h}" rpy="0 0 0"/>
+    <origin xyz="${-table_w/2} ${-table_l/2} ${bots_z - table_h}" rpy="0 0 0"/>
   </xacro:o2as_box>
   <link name="workspace_center"/>

File: aist_scene_description/urdf/kitting_bins.xacro (robot description, xacro)
@@ -25,21 +25,31 @@
   <xacro:property name="set2_z" value="0"/>
   <!--bin_2_part_4_-->
-  <xacro:kitting_bin_2 binname="bin_2_part_4" parent="workspace_center" z_origin_offset="-.008">
+  <xacro:kitting_bin_2 binname="bin_2_part_4"
+		       parent="workspace_center"
+		       z_origin_offset="-.008">
     <origin xyz="0 0.04 0.008" rpy="0 0 0" />
   </xacro:kitting_bin_2>
   <!--bin_2_part_7_-->
-  <xacro:kitting_bin_2 binname="bin_2_part_7" parent="workspace_center" z_origin_offset="-.008">
+  <xacro:kitting_bin_2 binname="bin_2_part_7"
+		       parent="workspace_center"
+		       z_origin_offset="-.008">
     <origin xyz="0 -0.072 0.008" rpy="0 0 0" />
   </xacro:kitting_bin_2>
   <!--bin_2_part_8_-->
-  <xacro:kitting_bin_2 binname="bin_2_part_8" parent="workspace_center" z_origin_offset="-.008">
+  <xacro:kitting_bin_2 binname="bin_2_part_8"
+		       parent="workspace_center"
+		       z_origin_offset="-.008">
     <origin xyz="0 -0.184 0.008" rpy="0 0 0" />
   </xacro:kitting_bin_2>
   <!--bin_3_part_15_-->
-  <xacro:kitting_bin_3 binname="bin_3_part_15" parent="workspace_center" z_origin_offset="-.004">
+  <xacro:kitting_bin_3 binname="bin_3_part_15"
+		       parent="workspace_center"
+		       z_origin_offset="-.004">
     <origin xyz="0.25 0.0 0.004" rpy="0 0 0" />
   </xacro:kitting_bin_3>
   <!--bin_3_part_16_-->
-  <xacro:kitting_bin_3 binname="bin_3_part_16" parent="workspace_center" z_origin_offset="-.004">
+  <xacro:kitting_bin_3 binname="bin_3_part_16"
+		       parent="workspace_center"
+		       z_origin_offset="-.004">
     <origin xyz="0.25 -0.192 0.004" rpy="0 0 0" />
   </xacro:kitting_bin_3>

File: aist_scene_description/urdf/pgrp_base_scene.urdf.xacro (robot description, xacro)
@@ -18,11 +18,11 @@
   <link name="o2as_ground"/>
   <xacro:include filename="$(find o2as_scene_description)/urdf/o2as_box.xacro"/>
-  <xacro:property name="plate_w" value="0.9"/>
-  <xacro:property name="plate_l" value="0.75"/>
-  <xacro:property name="plate_h" value="0.01"/>
+  <xacro:property name="table_w" value="0.9"/>
+  <xacro:property name="table_l" value="0.75"/>
+  <xacro:property name="table_h" value="0.01"/>
   <xacro:o2as_box boxname="workbox"
-		  box_w="${plate_w}" box_l="${plate_l}" box_h="${plate_h}"
+		  box_w="${table_w}" box_l="${table_l}" box_h="${table_h}"
 		  parent="o2as_ground">
-    <origin xyz="${-plate_w/2} ${-plate_l/2} ${bots_z - plate_h}" rpy="0 0 0"/>
+    <origin xyz="${-table_w/2} ${-table_l/2} ${bots_z - table_h}" rpy="0 0 0"/>
   </xacro:o2as_box>
   <link name="workspace_center"/>

File: aist_scene_description/urdf/pgrp_kitting.urdf.xacro (robot description, xacro)
@@ -1,8 +1,73 @@
 <?xml version="1.0"?>
-<robot xmlns:xacro="http://www.ros.org/wiki/xacro" name="aist_kitting_scene">
-    <xacro:include filename="$(find aist_scene_description)/urdf/kitting_tray_with_partitions.xacro" />
-  <xacro:include filename="$(find o2as_scene_description)/urdf/o2as_box.xacro" />
-  <xacro:include filename="$(find aist_scene_description)/urdf/kitting_bins.xacro" />
+<robot xmlns:xacro="http://www.ros.org/wiki/xacro" name="pgrp_kitting">
+  <xacro:include filename="$(find aist_scene_description)/urdf/pgrp_base_scene.urdf.xacro" />
+  <!-- base plate -->
+  <xacro:include filename="$(find o2as_scene_description)/urdf/o2as_box.xacro"/>
+  <xacro:property name="plate_w" value="0.4"/>
+  <xacro:property name="plate_l" value="0.75"/>
+  <xacro:property name="plate_h" value="0.015"/>
+  <xacro:o2as_box boxname="plate"
+		  box_w="${plate_w}" box_l="${plate_l}" box_h="${plate_h}"
+		  parent="workspace_center">
+    <origin xyz="${-plate_w/2} ${-plate_l/2} 0" rpy="0 0 0"/>
+  </xacro:o2as_box>
+  <link name="plate_center"/>
+  <joint name="workspace_to_plate" type="fixed">
+    <parent link="workspace_center"/>
+    <child  link="plate_center"/>
+    <origin xyz="0 0 ${plate_h}" rpy="0 0 0"/>
+  </joint>
+  <!-- bin1_definition -->
   <xacro:include filename="$(find o2as_scene_description)/urdf/kitting_bin_macros.xacro" />
+  <xacro:property name="bin_1_width"		value="0.125"/>
+  <xacro:property name="bin_1_length"		value="0.128"/>
+  <xacro:property name="z_origin_offset_1"	value="-.005" />
+  <!-- bin2_definition -->
+  <xacro:property name="bin_2_width"		value="0.112"/>
+  <xacro:property name="bin_2_length"		value="0.201"/>
+  <xacro:property name="z_origin_offset_2"	value="-.008" />
+  <!-- bin3_definition -->
+  <xacro:property name="bin_3_width"		value="0.192"/>
+  <xacro:property name="bin_3_length"		value="0.285"/>
+  <xacro:property name="z_origin_offset_3"	value="-.004" />
+  <!-- A row of bin1 -->
+  <xacro:property name="set1_x"	value="0"/>
+  <xacro:property name="set1_y" value="0.096"/>
+  <xacro:property name="set1_z" value="0"/>
+  <!-- A row of bin2 -->
+  <xacro:property name="set2_x" value="0.25"/>
+  <xacro:property name="set2_y" value="0.096"/>
+  <xacro:property name="set2_z" value="0"/>
+  <!--bin_2_part_4_-->
+  <xacro:kitting_bin_2 binname	      ="bin_2_part_4"
+		       parent	      ="plate_center"
+		       z_origin_offset="-0.008">
+    <origin xyz="0.285  0 0.004" rpy="0 0 0" />
+  </xacro:kitting_bin_2>
+  <!--bin_2_part_7_-->
+  <xacro:kitting_bin_2 binname	      ="bin_2_part_7"
+		       parent	      ="plate_center"
+		       z_origin_offset="-0.008">
+    <origin xyz="0.285 0.112 0.008" rpy="0 0 0" />
+  </xacro:kitting_bin_2>
+  <!--bin_2_part_8_-->
+  <xacro:kitting_bin_2 binname	      ="bin_2_part_8"
+  		       parent	      ="plate_center"
+  		       z_origin_offset="-0.008">
+    <origin xyz="0.285 -0.112 0.008" rpy="0 0 0" />
+  </xacro:kitting_bin_2>
+  <!-- bin_3_part_15_ -->
+  <xacro:kitting_bin_3 binname	      ="bin_3_part_15"
+  		       parent	      ="plate_center"
+  		       z_origin_offset="-0.004">
+    <origin xyz="0 0.096 0.004" rpy="0 0 0" />
+  </xacro:kitting_bin_3>
+  <!-- bin_3_part_16_ -->
+  <xacro:kitting_bin_3 binname	      ="bin_3_part_16"
+  		       parent	      ="plate_center"
+  		       z_origin_offset="-0.004">
+    <origin xyz="0 -0.096 0.004" rpy="0 0 0" />
+  </xacro:kitting_bin_3>
+  <xacro:include filename="$(find aist_scene_description)/urdf/kitting_tray_with_partitions.xacro" />
   <xacro:property name="tray_width" value=".210" />
   <xacro:property name="tray_length" value=".300" />
@@ -13,4 +78,3 @@
   <xacro:property name="bin_rack_length" value=".680" />
   <xacro:property name="bin_rack_height" value=".015" />
-  <xacro:include filename="$(find aist_scene_description)/urdf/pgrp_base_scene.urdf.xacro" />
 </robot>

File: aist_scene_description/urdf/ur5e_base_scene.urdf.xacro (robot description, xacro)
@@ -18,11 +18,11 @@
   <link name="o2as_ground"/>
   <xacro:include filename="$(find o2as_scene_description)/urdf/o2as_box.xacro"/>
-  <xacro:property name="plate_w" value="0.9"/>
-  <xacro:property name="plate_l" value="0.75"/>
-  <xacro:property name="plate_h" value="0.01"/>
+  <xacro:property name="table_w" value="0.9"/>
+  <xacro:property name="table_l" value="0.75"/>
+  <xacro:property name="table_h" value="0.01"/>
   <xacro:o2as_box boxname="workbox"
-		  box_w="${plate_w}" box_l="${plate_l}" box_h="${plate_h}"
+		  box_w="${table_w}" box_l="${table_l}" box_h="${table_h}"
 		  parent="o2as_ground">
-    <origin xyz="${-plate_w/2} ${-plate_l/2} ${bots_z - plate_h}" rpy="0 0 0"/>
+    <origin xyz="${-table_w/2} ${-table_l/2} ${bots_z - table_h}" rpy="0 0 0"/>
   </xacro:o2as_box>
   <link name="workspace_center"/>

Commit message: API changed for o2as_phoxi_camera.Search graspability is now implemented using action lib.

File: aist_scene_description/urdf/aist_base_scene.urdf.xacro (robot description, xacro)
@@ -71,5 +71,6 @@
   <xacro:single_suction_gripper_o2as prefix="b_bot_"
   				     parent="b_bot_ft300_frange_link">
-    <origin xyz="0 0 0" rpy="0 ${0.8*pi/180} ${-0.5*pi/180}"/>
+    <origin xyz="0 0 0" rpy="0 ${-0.1*pi/180} ${0.1*pi/180}"/>
+    <!-- <origin xyz="0 0 0" rpy="0 0 0"/> -->
   </xacro:single_suction_gripper_o2as>
   <!-- Add virtual wall to avoid collisions-->

File: aist_scene_description/urdf/pgrp_base_scene.urdf.xacro (robot description, xacro)
@@ -67,11 +67,11 @@
 			  grippername = "gripper"
 			  parent = "a_bot_ft300_frange_link">
-    <!-- <origin xyz="0 0 0" rpy="${-pi/2} ${-0.9*pi/180} ${-0.5*pi/180}"/> -->
-    <origin xyz="0 0 0" rpy="${-pi/2} 0 0"/>
+    <origin xyz="-0.004 0 0" rpy="${-pi/2} ${-1.0*pi/180} ${-0.5*pi/180}"/>
+    <!-- <origin xyz="-0.004 0 0" rpy="${-pi/2} 0 0"/> -->
   </xacro:InnerOnlyGripper>
   <xacro:include filename="$(find o2as_scene_description)/urdf/single_suction_gripper.urdf.xacro"/>
   <xacro:single_suction_gripper_o2as prefix="b_bot_"
   				     parent="b_bot_ft300_frange_link">
-    <origin xyz="0 0 0" rpy="0 ${0.1*pi/180} ${-0.2*pi/180}"/>
+    <origin xyz="0 0 0" rpy="0 ${-0.1*pi/180} ${0.1*pi/180}"/>
     <!-- <origin xyz="0 0 0" rpy="0 0 0"/> -->
   </xacro:single_suction_gripper_o2as>
@@ -83,10 +83,10 @@
   <xacro:include filename="$(find o2as_scene_description)/urdf/phoxi_m_camera.urdf.xacro"/>
   <xacro:phoxi_m_camera prefix="a_" parent="o2as_ground">
-    <origin xyz="0.521217687458
-		 -0.00508307933619
-		 1.43718368936"
-	    rpy="${-150.749317075*pi/180}
-		 ${0.617210923766*pi/180}
-		 ${88.4045592933*pi/180}"/>
+    <origin xyz="0.523323618924
+		 -0.0127144528585
+		 1.43727836373"
+	    rpy="${-150.824488274*pi/180}
+		 ${-0.392518546798*pi/180}
+		 ${86.9392445854*pi/180}"/>
   </xacro:phoxi_m_camera>
   <!-- Add RealSense camera -->

Commit message: Made callback function non-static.

File: aist_scene_description/urdf/aist_base_scene.urdf.xacro (robot description, xacro)
@@ -71,5 +71,5 @@
   <xacro:single_suction_gripper_o2as prefix="b_bot_"
   				     parent="b_bot_ft300_frange_link">
-    <origin xyz="0 0 0" rpy="0 ${-0.1*pi/180} ${0.1*pi/180}"/>
+    <origin xyz="0 0 0" rpy="0 ${0.7*pi/180} ${-0.9*pi/180}"/>
     <!-- <origin xyz="0 0 0" rpy="0 0 0"/> -->
   </xacro:single_suction_gripper_o2as>

Commit message: Fixed bug in tool_calibration.py.

File: aist_scene_description/urdf/aist_base_scene.urdf.xacro (robot description, xacro)
@@ -71,5 +71,5 @@
   <xacro:single_suction_gripper_o2as prefix="b_bot_"
   				     parent="b_bot_ft300_frange_link">
-    <origin xyz="0 0 0" rpy="0 ${0.7*pi/180} ${-0.9*pi/180}"/>
+    <origin xyz="0 0 0" rpy="0 ${0.4*pi/180} ${-1.1*pi/180}"/>
     <!-- <origin xyz="0 0 0" rpy="0 0 0"/> -->
   </xacro:single_suction_gripper_o2as>
@@ -81,10 +81,10 @@
   <xacro:include filename="$(find o2as_scene_description)/urdf/phoxi_m_camera.urdf.xacro"/>
   <xacro:phoxi_m_camera prefix="a_" parent="o2as_ground">
-    <origin xyz="0.547941636523
-		 -0.00827443204237
-		 1.67030171767"
-	    rpy="${-151.493605482*pi/180}
-		 ${0.698490882792*pi/180}
-		 ${85.0482907121*pi/180}"/>
+    <origin xyz="0.480002181393
+		 -0.0102469021884
+		 1.40147194843"
+	    rpy="${-152.32508021*pi/180}
+		 ${-0.53545059011*pi/180}
+		 ${86.2439460292*pi/180}"/>
   </xacro:phoxi_m_camera>
   <!-- I would like to remove the "world" link definition, but apparently it is necessary for Gazebo -->

File: aist_scene_description/urdf/pgrp_base_scene.urdf.xacro (robot description, xacro)
@@ -67,5 +67,5 @@
 			  grippername = "gripper"
 			  parent = "a_bot_ft300_frange_link">
-    <origin xyz="-0.004 0 0" rpy="${-pi/2} ${-1.0*pi/180} ${-0.5*pi/180}"/>
+    <origin xyz="-0.004 0 0" rpy="${-pi/2} ${-0.2*pi/180} ${1.3*pi/180}"/>
     <!-- <origin xyz="-0.004 0 0" rpy="${-pi/2} 0 0"/> -->
   </xacro:InnerOnlyGripper>
@@ -73,5 +73,5 @@
   <xacro:single_suction_gripper_o2as prefix="b_bot_"
   				     parent="b_bot_ft300_frange_link">
-    <origin xyz="0 0 0" rpy="0 ${-0.1*pi/180} ${0.1*pi/180}"/>
+    <origin xyz="0 0 0" rpy="0 ${0.4*pi/180} ${-1.1*pi/180}"/>
     <!-- <origin xyz="0 0 0" rpy="0 0 0"/> -->
   </xacro:single_suction_gripper_o2as>
@@ -83,10 +83,10 @@
   <xacro:include filename="$(find o2as_scene_description)/urdf/phoxi_m_camera.urdf.xacro"/>
   <xacro:phoxi_m_camera prefix="a_" parent="o2as_ground">
-    <origin xyz="0.523323618924
-		 -0.0127144528585
-		 1.43727836373"
-	    rpy="${-150.824488274*pi/180}
-		 ${-0.392518546798*pi/180}
-		 ${86.9392445854*pi/180}"/>
+    <origin xyz="0.480002181393
+		 -0.0102469021884
+		 1.40147194843"
+	    rpy="${-152.32508021*pi/180}
+		 ${-0.53545059011*pi/180}
+		 ${86.2439460292*pi/180}"/>
   </xacro:phoxi_m_camera>
   <!-- Add RealSense camera -->
