Commit message: Setup hardware from YAML files.

File: aist_scene_description/urdf/aist_kitting.urdf.xacro (robot description, xacro)
@@ -1,16 +1,16 @@
 <?xml version="1.0"?>
 <robot xmlns:xacro="http://www.ros.org/wiki/xacro" name="aist_kitting_scene">
-    <xacro:include filename="$(find aist_scene_description)/urdf/kitting_tray_with_partitions.xacro" />
+  <xacro:include filename="$(find aist_scene_description)/urdf/aist_base_scene.urdf.xacro" />
+  <xacro:include filename="$(find aist_scene_description)/urdf/kitting_tray_with_partitions.xacro" />
   <xacro:include filename="$(find o2as_scene_description)/urdf/o2as_box.xacro" />
   <xacro:include filename="$(find aist_scene_description)/urdf/kitting_bins.xacro" />
   <xacro:include filename="$(find o2as_scene_description)/urdf/kitting_bin_macros.xacro" />
-  <xacro:property name="tray_width" value=".210" />
-  <xacro:property name="tray_length" value=".300" />
-  <xacro:property name="tray_rack_width" value=".210" />
-  <xacro:property name="tray_rack_length" value=".600" />
-  <xacro:property name="tray_rack_height" value=".015" />
-  <xacro:property name="bin_rack_width" value=".420" />
-  <xacro:property name="bin_rack_length" value=".680" />
-  <xacro:property name="bin_rack_height" value=".015" />
-  <xacro:include filename="$(find aist_scene_description)/urdf/aist_base_scene.urdf.xacro" />
+  <!-- <xacro:property name="tray_width" value=".210" /> -->
+  <!-- <xacro:property name="tray_length" value=".300" /> -->
+  <!-- <xacro:property name="tray_rack_width" value=".210" /> -->
+  <!-- <xacro:property name="tray_rack_length" value=".600" /> -->
+  <!-- <xacro:property name="tray_rack_height" value=".015" /> -->
+  <!-- <xacro:property name="bin_rack_width" value=".420" /> -->
+  <!-- <xacro:property name="bin_rack_length" value=".680" /> -->
+  <!-- <xacro:property name="bin_rack_height" value=".015" /> -->
 </robot>

File: aist_scene_description/urdf/ur5e_base_scene.urdf.xacro (robot description, xacro)
@@ -58,17 +58,13 @@
     <origin xyz="${d_bot_x} ${d_bot_y} ${bots_z}" rpy="0 0 ${d_bot_theta}"/>
   </joint>
-  <!-- Spawn and attach force sensor -->
-  <xacro:include filename="$(find aist_ft300)/urdf/ft300.urdf.xacro"/>
-  <xacro:ft300 prefix="c_bot_" parent="c_bot_ee_link"/>
-  <xacro:ft300 prefix="d_bot_" parent="d_bot_ee_link"/>
   <!-- Spawn and attach gripper -->
   <xacro:include filename="$(find o2as_scene_description)/urdf/robotiq_85_gripper_with_tip_link.urdf.xacro"/>
   <xacro:robotiq_85_gripper_with_tip_link prefix="c_bot_"
-					  parent="c_bot_ft300_frange_link">
+					  parent="c_bot_ee_link">
     <origin xyz="0 0 0" rpy="0 0 0"/>
   </xacro:robotiq_85_gripper_with_tip_link>
   <!-- <xacro:include filename="$(find o2as_scene_description)/urdf/dual_suction_gripper.urdf.xacro"/> -->
   <!-- <xacro:dual_suction_gripper_o2as prefix="d_bot_" -->
-  <!-- 				     parent="d_bot_ft300_frange_link"> -->
+  <!-- 				     parent="d_bot_ee_link"> -->
   <!--   <origin xyz="0 0 0" rpy="0 ${0.8*pi/180} ${-0.5*pi/180}"/> -->
   <!-- </xacro:dual_suction_gripper_o2as> -->
@@ -78,5 +74,5 @@
   <!-- </xacro:o2as_box> -->
   <xacro:robotiq_85_gripper_with_tip_link prefix="d_bot_"
-					  parent="d_bot_ft300_frange_link">
+					  parent="d_bot_ee_link">
     <origin xyz="0 0 0" rpy="0 0 0"/>
   </xacro:robotiq_85_gripper_with_tip_link>
