Commit message: Import fetch_ros and fetch_gazebo as sumodules.

File: aist_scene_description/urdf/aist_box.urdf.xacro (robot description, xacro)
@@ -12,5 +12,5 @@
         </geometry>
         <material name="Grey">
-          <color rgba="0.7 0.7 0.7 1.0"/>
+          <color rgba="1.0 1.0 1.0 1.0"/>
         </material>
       </visual>
@@ -31,5 +31,5 @@
     </link>
     <gazebo reference="${name}">
-      <material>Gazebo/Grey</material>
+      <material>Gazebo/White</material>
     </gazebo>
     <joint name="${name}" type="fixed">

File: aist_scene_description/urdf/ceatec_base_scene.urdf (robot description, URDF)
Before this commit: robot aaa, 1 links, 0 joints
Links:
- removed link base_link
- added link a_cabinet_ar_marker; collision box size=0.1 0.1 0.001; visual box size=0.1 0.1 0.001
- added link a_cabinet_back, mass 1.0; collision box size=0.925 0.03 1.711; visual box size=0.925 0.03 1.711
- added link a_cabinet_base, mass 1.0; collision box size=0.925 0.39 0.18; visual box size=0.925 0.39 0.18
- added link a_cabinet_base_origin
- added link a_cabinet_base_origin_center
- added link a_cabinet_shelf1, mass 1.0; collision box size=0.925 0.39 0.03; visual box size=0.925 0.39 0.03
- added link a_cabinet_shelf1_origin
- added link a_cabinet_shelf1_origin_center
- added link a_cabinet_shelf2, mass 1.0; collision box size=0.925 0.39 0.03; visual box size=0.925 0.39 0.03
- added link a_cabinet_shelf3, mass 1.0; collision box size=0.925 0.39 0.03; visual box size=0.925 0.39 0.03
- added link a_table_ar_marker; collision box size=0.1 0.1 0.001; visual box size=0.1 0.1 0.001
- added link a_table_leg0, mass 1.0; collision box size=0.05 0.05 0.58; visual box size=0.05 0.05 0.58
- added link a_table_leg1, mass 1.0; collision box size=0.05 0.05 0.58; visual box size=0.05 0.05 0.58
- added link a_table_leg2, mass 1.0; collision box size=0.05 0.05 0.58; visual box size=0.05 0.05 0.58
- added link a_table_leg3, mass 1.0; collision box size=0.05 0.05 0.58; visual box size=0.05 0.05 0.58
- added link a_table_top, mass 1.0; collision box size=0.53 0.315 0.02; visual box size=0.53 0.315 0.02
- added link a_table_top_origin
- added link a_table_top_origin_center
- added link b_table_leg0, mass 1.0; collision box size=0.05 0.05 0.7; visual box size=0.05 0.05 0.7
- added link b_table_leg1, mass 1.0; collision box size=0.05 0.05 0.7; visual box size=0.05 0.05 0.7
- added link b_table_leg2, mass 1.0; collision box size=0.05 0.05 0.7; visual box size=0.05 0.05 0.7
- added link b_table_leg3, mass 1.0; collision box size=0.05 0.05 0.7; visual box size=0.05 0.05 0.7
- added link b_table_top, mass 1.0; collision box size=0.9 0.9 0.02; visual box size=0.9 0.9 0.02
- added link b_table_top_origin
- added link b_table_top_origin_center
- added link ground
- added link world
Joints:
- added joint a_cabinet_ar_marker_joint: type fixed, parent a_cabinet_shelf1_origin, child a_cabinet_ar_marker, origin xyz=0.875 0.05 0.001 rpy=0 0 0
- added joint a_cabinet_back: type fixed, parent a_cabinet_base, child a_cabinet_back, origin xyz=0 0.39 0 rpy=0 0 0
- added joint a_cabinet_base: type fixed, parent ground, child a_cabinet_base, origin xyz=1.08    -0.075    0 rpy=0 0 -1.57079632679
- added joint a_cabinet_base_origin: type fixed, parent a_cabinet_base, child a_cabinet_base_origin, origin xyz=0 0 0.18 rpy=0 0 0
- added joint a_cabinet_base_origin_center: type fixed, parent a_cabinet_base_origin, child a_cabinet_base_origin_center, origin xyz=0.4625 0.195 0 rpy=0 0 0
- added joint a_cabinet_shelf1: type fixed, parent a_cabinet_base, child a_cabinet_shelf1, origin xyz=0 0 0.712 rpy=0 0 0
- added joint a_cabinet_shelf1_origin: type fixed, parent a_cabinet_shelf1, child a_cabinet_shelf1_origin, origin xyz=0 0 0.03 rpy=0 0 0
- added joint a_cabinet_shelf1_origin_center: type fixed, parent a_cabinet_shelf1_origin, child a_cabinet_shelf1_origin_center, origin xyz=0.4625 0.195 0 rpy=0 0 0
- added joint a_cabinet_shelf2: type fixed, parent a_cabinet_base, child a_cabinet_shelf2, origin xyz=0 0 0.96 rpy=0 0 0
- added joint a_cabinet_shelf3: type fixed, parent a_cabinet_base, child a_cabinet_shelf3, origin xyz=0 0 1.43 rpy=0 0 0
- added joint a_table_ar_marker_joint: type fixed, parent a_table_top_origin, child a_table_ar_marker, origin xyz=0.05 0.05 0.001 rpy=0 0 0
- added joint a_table_leg0: type fixed, parent ground, child a_table_leg0, origin xyz=0.35    0.485    0 rpy=0 0 0
- added joint a_table_leg1: type fixed, parent a_table_leg0, child a_table_leg1, origin xyz=0.48 0 0 rpy=0 0 0
- added joint a_table_leg2: type fixed, parent a_table_leg0, child a_table_leg2, origin xyz=0 0.265 0 rpy=0 0 0
- added joint a_table_leg3: type fixed, parent a_table_leg0, child a_table_leg3, origin xyz=0.48      0.265      0 rpy=0 0 0
- added joint a_table_top: type fixed, parent a_table_leg0, child a_table_top, origin xyz=0 0 0.58 rpy=0 0 0
- added joint a_table_top_origin: type fixed, parent a_table_top, child a_table_top_origin, origin xyz=0 0 0.02 rpy=0 0 0
- added joint a_table_top_origin_center: type fixed, parent a_table_top_origin, child a_table_top_origin_center, origin xyz=0.265 0.1575 0 rpy=0 0 0
- added joint b_table_leg0: type fixed, parent ground, child b_table_leg0, origin xyz=-1.5    0.1    0 rpy=0 0 0
- added joint b_table_leg1: type fixed, parent b_table_leg0, child b_table_leg1, origin xyz=0.85 0 0 rpy=0 0 0
- added joint b_table_leg2: type fixed, parent b_table_leg0, child b_table_leg2, origin xyz=0 0.85 0 rpy=0 0 0
- added joint b_table_leg3: type fixed, parent b_table_leg0, child b_table_leg3, origin xyz=0.85      0.85      0 rpy=0 0 0
- added joint b_table_top: type fixed, parent b_table_leg0, child b_table_top, origin xyz=0 0 0.7 rpy=0 0 0
- added joint b_table_top_origin: type fixed, parent b_table_top, child b_table_top_origin, origin xyz=0 0 0.02 rpy=0 0 0
- added joint b_table_top_origin_center: type fixed, parent b_table_top_origin, child b_table_top_origin_center, origin xyz=0.45 0.45 0 rpy=0 0 0
- added joint world_ground_joint: type fixed, parent world, child ground, origin xyz=0 0 0 rpy=0 0 0

File: aist_scene_description/urdf/ceatec_base_scene.urdf.xacro (robot description, xacro)
@@ -100,14 +100,11 @@
   <!--   <origin xyz="${(b_table_width/2 - tray_width)/2} 0.03 0" rpy="0 0 0"/> -->
   <!-- </xacro:tray> -->
-  <!-- I would like to remove the "world" link definition, but apparently it is necessary for Gazebo -->
-  <!-- <joint name="ground_base_joint" type="planar"> -->
-  <!--   <parent link="ground"/> -->
-  <!--   <child  link="base_link"/> -->
-  <!--   <origin xyz="0 -0.5 0" rpy="0 0 0"/> -->
-  <!-- </joint> -->
-  <joint name="base_ground_joint" type="planar">
-    <parent link="base_link"/>
+  <!-- I would like to remove the "world" link definition, but
+       apparently it is necessary for Gazebo -->
+  <link name="world"/>
+  <joint name="world_ground_joint" type="fixed">
+    <parent link="world"/>
     <child  link="ground"/>
-    <origin xyz="0 0.5 0" rpy="0 0 0"/>
+    <origin xyz="0 0 0" rpy="0 0 0"/>
   </joint>
 </robot>
