Commit message: Cleaning up.

File: aist_scene_description/urdf/ceatec_base_scene.urdf.xacro (robot description, xacro)
@@ -1,110 +1,15 @@
 <?xml version="1.0"?>
 <robot xmlns:xacro="http://www.ros.org/wiki/xacro"
-       name="ceatec_base_scene" >
-  <xacro:property name="workspace_width"	value="3.000"/>
-  <xacro:property name="workspace_length"	value="2.000"/>
-  <xacro:property name="a_table_width"		value="0.530"/>
-  <xacro:property name="a_table_length"		value="0.315"/>
-  <xacro:property name="a_table_height"		value="0.600"/>
-  <xacro:property name="b_table_width"		value="0.900"/>
-  <xacro:property name="b_table_length"		value="0.900"/>
-  <xacro:property name="b_table_height"		value="0.720"/>
-  <xacro:property name="cabinet_width"		value="0.925"/>
-  <xacro:property name="cabinet_length"		value="0.420"/>
-  <xacro:property name="cabinet_base_height"	value="0.180"/>
-  <xacro:property name="cabinet_shelf1_height"	value="0.742"/>
-  <xacro:property name="cabinet_shelf2_height"	value="0.990"/>
-  <xacro:property name="cabinet_shelf3_height"	value="1.460"/>
-  <xacro:property name="cabinet_back_height"	value="1.711"/>
-  <xacro:property name="tray_width"		value="0.340"/>
-  <xacro:property name="tray_length"		value="0.250"/>
-  <xacro:property name="tray_height"		value="0.062"/>
-  <!-- Main workspace -->
-  <link name="ground"/>
+       name="ceatec_base_scene_with_fetch" >
   <!-- Fetch robot -->
-  <!-- <xacro:include filename="$(find fetch_gazebo)/robots/fetch.gazebo.xacro"/> -->
-  <!-- Table -->
-  <xacro:include filename="$(find
-			   aist_scene_description)/urdf/table.urdf.xacro"/>
-  <xacro:table prefix="a_"
-  	       width="${a_table_width}"
-  	       length="${a_table_length}"
-  	       height="${a_table_height}"
-  	       parent="ground">
-    <origin xyz="${workspace_width/2  - cabinet_length - a_table_width - 0.2}
-		 ${workspace_length/2 - a_table_length - 0.2}
-		 0"
-	    rpy="0 0 0"/>
-  </xacro:table>
-  <xacro:table prefix="b_"
-  	       width="${b_table_width}"
-  	       length="${b_table_length}"
-  	       height="${b_table_height}"
-  	       parent="ground">
-    <origin xyz="${-workspace_width/2}
-		 ${workspace_length/2 - b_table_length}
-		 0"
-	    rpy="0 0 0"/>
-  </xacro:table>
-  <!-- Cabinet -->
-  <xacro:include filename="$(find
-			   aist_scene_description)/urdf/cabinet.urdf.xacro"/>
-  <xacro:cabinet prefix="a_"
-		 width="${cabinet_width}"
-		 length="${cabinet_length}"
-		 base_height="${cabinet_base_height}"
-		 shelf1_height="${cabinet_shelf1_height}"
-		 shelf2_height="${cabinet_shelf2_height}"
-		 shelf3_height="${cabinet_shelf3_height}"
-		 back_height="${cabinet_back_height}"
-		 parent="ground">
-    <origin xyz="${workspace_width/2   - cabinet_length}
-		 ${-workspace_length/2 + cabinet_width}
-		 0"
-	    rpy="0 0 ${-pi/2}"/>
-  </xacro:cabinet>
-  <!-- AR markers -->
-  <xacro:include filename="$(find aist_gazebo)/urdf/ar_marker.urdf.xacro"/>
-  <xacro:ar_marker prefix="a_cabinet_"
-  		   parent="a_cabinet_shelf1_origin"
-  		   marker_id="17"
-		   size="0.1"
-		   thickness="0.001">
-    <origin xyz="${cabinet_width - 0.05} 0.05 0.001" rpy="0 0 0"/>
-  </xacro:ar_marker>
-  <xacro:ar_marker prefix="a_table_"
-  		   parent="a_table_top_origin"
-  		   marker_id="26"
-		   size="0.1"
-		   thickness="0.001">
-    <origin xyz="0.05 0.05 0.001" rpy="0 0 0"/>
-  </xacro:ar_marker>
-  <!-- Trays -->
-  <!-- <xacro:include filename="$(find -->
-  <!-- 			   aist_scene_description)/urdf/tray.urdf.xacro"/> -->
-  <!-- <xacro:tray prefix="a_" -->
-  <!-- 	      width="${tray_width}" -->
-  <!-- 	      length="${tray_length}" -->
-  <!-- 	      height="${tray_height}" -->
-  <!-- 	      parent="a_table_top_origin"> -->
-  <!--   <origin xyz="${(a_table_width  - tray_width)/2} -->
-  <!-- 		 ${(a_table_length - tray_length)/2} -->
-  <!-- 		 0" -->
-  <!-- 	    rpy="0 0 0"/> -->
-  <!-- </xacro:tray> -->
-  <!-- <xacro:tray prefix="b_" -->
-  <!-- 	      width="${tray_width}" -->
-  <!-- 	      length="${tray_length}" -->
-  <!-- 	      height="${tray_height}" -->
-  <!-- 	      parent="b_table_top_origin"> -->
-  <!--   <origin xyz="${(b_table_width/2 - tray_width)/2} 0.03 0" rpy="0 0 0"/> -->
-  <!-- </xacro:tray> -->
+  <xacro:include filename="$(find fetch_gazebo)/robots/fetch.gazebo.xacro"/>
+  <!-- CEATEC base scene -->
+  <xacro:include filename="$(find aist_scene_description)/urdf/ceatec_base_scene_without_fetch.urdf.xacro"/>
   <!-- I would like to remove the "world" link definition, but
        apparently it is necessary for Gazebo -->
-  <link name="world"/>
-  <joint name="world_ground_joint" type="fixed">
+  <joint name="world_base_joint" type="planar">
     <parent link="world"/>
-    <child  link="ground"/>
-    <origin xyz="0 0 0" rpy="0 0 0"/>
+    <child  link="base_link"/>
+    <origin xyz="0 -0.5 0" rpy="0 0 0"/>
   </joint>
 </robot>

Commit message: Separate robot and environment urdf files and configurations.

File: aist_scene_description/urdf/ceatec_base_scene.urdf.xacro (robot description, xacro)
@@ -1,15 +1,29 @@
 <?xml version="1.0"?>
 <robot xmlns:xacro="http://www.ros.org/wiki/xacro"
-       name="ceatec_base_scene_with_fetch" >
+       name="ceatec_base_scene" >
   <!-- Fetch robot -->
   <xacro:include filename="$(find fetch_gazebo)/robots/fetch.gazebo.xacro"/>
   <!-- CEATEC base scene -->
-  <xacro:include filename="$(find aist_scene_description)/urdf/ceatec_base_scene_without_fetch.urdf.xacro"/>
+  <xacro:include filename="$(find aist_scene_description)/urdf/ceatec_base_scene_environment.urdf.xacro"/>
   <!-- I would like to remove the "world" link definition, but
        apparently it is necessary for Gazebo -->
-  <joint name="world_base_joint" type="planar">
-    <parent link="world"/>
+  <!-- <link  name="map"/> -->
+  <link  name="odom"/>
+  <!-- <joint name="map_odom_joint" type="planar"> -->
+  <!--   <parent link="map"/> -->
+  <!--   <child  link="odom"/> -->
+  <!--   <origin xyz="0 0 0" rpy="0 0 0"/> -->
+  <!--   <axis   xyz="0 0 1"/> -->
+  <!-- </joint> -->
+  <joint name="odom_base_joint" type="planar">
+    <parent link="odom"/>
     <child  link="base_link"/>
-    <origin xyz="0 -0.5 0" rpy="0 0 0"/>
+    <origin xyz="0 0 0" rpy="0 0 0"/>
+    <axis   xyz="0 0 1"/>
+  </joint>
+  <joint name="odom_world_joint" type="planar">
+    <parent link="odom"/>
+    <child  link="world"/>
+    <origin xyz="0.5 0.5 0" rpy="0 0 0"/>
   </joint>
 </robot>

File: aist_scene_description/urdf/ceatec_base_scene_environment.urdf.xacro (robot description, xacro)
@@ -1,5 +1,5 @@
 <?xml version="1.0"?>
 <robot xmlns:xacro="http://www.ros.org/wiki/xacro"
-       name="ceatec_base_scene" >
+       name="ceatec_base_scene_environment" >
   <xacro:property name="workspace_width"	value="3.000"/>
   <xacro:property name="workspace_length"	value="2.000"/>
@@ -22,6 +22,4 @@
   <!-- Main workspace -->
   <link name="ground"/>
-  <!-- Fetch robot -->
-  <!-- <xacro:include filename="$(find fetch_gazebo)/robots/fetch.gazebo.xacro"/> -->
   <!-- Table -->
   <xacro:include filename="$(find

Commit message: TF tree is now constructed cleanly.

File: aist_scene_description/urdf/ceatec_base_scene.urdf.xacro (robot description, xacro)
@@ -22,5 +22,5 @@
     <axis   xyz="0 0 1"/>
   </joint>
-  <joint name="odom_world_joint" type="planar">
+  <joint name="odom_world_joint" type="fixed">
     <parent link="odom"/>
     <child  link="world"/>

Commit message: Confirmed that fetch robot can be controlled by moveit in gazebo world.

File: aist_scene_description/urdf/ceatec_base_scene.urdf.xacro (robot description, xacro)
@@ -8,20 +8,18 @@
   <!-- I would like to remove the "world" link definition, but
        apparently it is necessary for Gazebo -->
-  <!-- <link  name="map"/> -->
+  <link  name="map"/>
   <link  name="odom"/>
-  <!-- <joint name="map_odom_joint" type="planar"> -->
-  <!--   <parent link="map"/> -->
-  <!--   <child  link="odom"/> -->
-  <!--   <origin xyz="0 0 0" rpy="0 0 0"/> -->
-  <!--   <axis   xyz="0 0 1"/> -->
-  <!-- </joint> -->
+  <joint name="map_odom_joint" type="planar">
+    <parent link="map"/>
+    <child  link="odom"/>
+    <axis   xyz="0 0 1"/>
+  </joint>
   <joint name="odom_base_joint" type="planar">
     <parent link="odom"/>
     <child  link="base_link"/>
-    <origin xyz="0 0 0" rpy="0 0 0"/>
     <axis   xyz="0 0 1"/>
   </joint>
-  <joint name="odom_world_joint" type="fixed">
-    <parent link="odom"/>
+  <joint name="map_world_joint" type="fixed">
+    <parent link="map"/>
     <child  link="world"/>
     <origin xyz="0.5 0.5 0" rpy="0 0 0"/>

Commit message: Added move_base support.

File: aist_scene_description/urdf/ceatec_base_scene.urdf.xacro (robot description, xacro)
@@ -23,5 +23,5 @@
     <parent link="map"/>
     <child  link="world"/>
-    <origin xyz="0.5 0.5 0" rpy="0 0 0"/>
+    <origin xyz="0.3 0.5 0" rpy="0 0 0"/>
   </joint>
 </robot>

File: aist_scene_description/urdf/ceatec_base_scene_environment.urdf.xacro (robot description, xacro)
@@ -107,5 +107,5 @@
     <parent link="a_cabinet_base" />
     <child  link="a_cabinet_standpoint" />
-    <origin xyz="${cabinet_width/2} -0.6 0" rpy="0 0 ${pi/2}" />
+    <origin xyz="${cabinet_width/2} -0.9 0" rpy="0 0 ${pi/2}" />
   </joint>
   <!-- Frames to place items on cabinet -->
