Commit message: GripperClient reorganized but not completed.

File: aist_scene_description/urdf/tray.urdf.xacro (robot description, xacro)
@@ -62,5 +62,5 @@
       <parent link ="b_item_on_${prefix}tray"/>
       <child  link="a_item_on_${prefix}tray"/>
-      <origin xyz="0 ${-width/4 + tray_thickness/2} 0" rpy="0 0 0"/>
+      <origin xyz="0 ${-width/3 + tray_thickness/2} 0" rpy="0 0 0"/>
     </joint>
     <link name="c_item_on_${prefix}tray"/>
@@ -68,5 +68,5 @@
       <parent link ="b_item_on_${prefix}tray"/>
       <child  link="c_item_on_${prefix}tray"/>
-      <origin xyz="0 ${width/4 - tray_thickness/2} 0" rpy="0 0 0"/>
+      <origin xyz="0 ${width/3 - tray_thickness/2} 0" rpy="0 0 0"/>
     </joint>
     <link name="d_item_on_${prefix}tray"/>

Commit message: Changed the name of joint between a tray and its parent.

File: aist_scene_description/urdf/tray.urdf.xacro (robot description, xacro)
@@ -8,5 +8,5 @@
     <xacro:property name="item_radius"		value="0.04" />
     <link name="${prefix}tray"/>
-    <joint name="${prefix}tray" type="floating">
+    <joint name="${prefix}tray_joint" type="floating">
       <parent link="${parent}" />
       <child  link="${prefix}tray" />
