Commit message: Set frames for palcing items.

File: aist_scene_description/urdf/ceatec_base_scene_environment.urdf.xacro (robot description, xacro)
@@ -23,5 +23,5 @@
   <!-- Main workspace -->
   <link name="ground"/>
-  <!-- Table -->
+  <!-- a_table -->
   <xacro:include filename="$(find aist_scene_description)/urdf/table.urdf.xacro"/>
   <xacro:table prefix="a_"
@@ -38,14 +38,24 @@
 	    rpy="0 0 ${-pi/6}"/>
   </xacro:table>
-  <!-- Frame to put box on a_table -->
-  <xacro:property name="box_width"	value="0.340" />
-  <xacro:property name="box_length"	value="0.250" />
-  <xacro:property name="box_height"	value="0.065" />
-  <link name="box_on_pedestral" />
-  <joint name="box_on_pedestral_joint" type="fixed">
+  <!-- Frame to place trays on a_table -->
+  <link name="a_tray_on_a_table" />
+  <joint name="a_tray_on_a_table_joint" type="fixed">
     <parent link="a_table_top_origin_center" />
-    <child link="box_on_pedestral" />
-    <origin xyz="0 ${-box_length/2} ${box_height}" rpy="0 ${pi/2} 0" />
+    <child link="a_tray_on_a_table" />
+    <origin xyz="0 ${-tray_length/2} 0" rpy="0 0 0" />
   </joint>
+  <link name="b_tray_on_a_table" />
+  <joint name="b_tray_on_a_table_joint" type="fixed">
+    <parent link="a_table_top_origin_center" />
+    <child link="b_tray_on_a_table" />
+    <origin xyz="0 ${-tray_length/2} 0" rpy="0 0 0" />
+  </joint>
+  <link name="a_table_standpoint"/>
+  <joint name="a_table_standpoint_joint" type="fixed">
+    <parent link="a_table_leg0" />
+    <child  link="a_table_standpoint" />
+    <origin xyz="${a_table_width/2} -0.4 0" rpy="0 0 ${pi/2}" />
+  </joint>
+  <!-- b_table -->
   <xacro:table prefix="b_"
 	       width="${b_table_width}"
@@ -58,18 +68,22 @@
 	    rpy="0 0 0"/>
   </xacro:table>
-  <!-- Frame to put box on b_table -->
-  <link name="box1_on_b_table" />
-  <joint name="box1_on_b_table_joint" type="fixed">
+  <!-- Frame to place trays on b_table -->
+  <link name="a_tray_on_b_table" />
+  <joint name="a_tray_on_b_table_joint" type="fixed">
     <parent link="b_table_top_origin_center" />
-    <child  link="box1_on_b_table" />
-    <origin xyz="${-(box_width/2+0.05)} ${-box_length/2}
-		 ${box_height}"
-	    rpy="0 ${pi/2} 0"/>
+    <child link="a_tray_on_b_table" />
+    <origin xyz="${-tray_width/2 - 0.05} ${-tray_length/2} 0" rpy="0 0 0" />
   </joint>
-  <link name="box0_on_b_table" />
-  <joint name="box0_on_b_table_joint" type="fixed">
+  <link name="b_tray_on_b_table" />
+  <joint name="b_tray_on_b_table_joint" type="fixed">
     <parent link="b_table_top_origin_center" />
-    <child link="box0_on_b_table" />
-    <origin xyz="${(box_width/2+0.05)} ${-box_length/2} ${box_height}" rpy="0 ${pi/2} 0"/>
+    <child link="b_tray_on_b_table" />
+    <origin xyz="${tray_width/2 + 0.05} ${-tray_length/2} 0" rpy="0 0 0" />
+  </joint>
+  <link name="b_table_standpoint"/>
+  <joint name="b_table_standpoint_joint" type="fixed">
+    <parent link="b_table_leg0" />
+    <child  link="b_table_standpoint" />
+    <origin xyz="${b_table_width/2} -0.4 0" rpy="0 0 ${pi/2}" />
   </joint>
   <!-- Cabinet -->
@@ -80,54 +94,47 @@
 		 0" rpy="0 0 ${-pi/2}"/>
   </xacro:cabinet>
-  <!-- Frames to put noodles on cabinet -->
-  <!-- Have to be described abstractly -->
-  <!-- <xacro:property name="a_noodle_x_origin" value="-0.065" />
-  <xacro:property name="a_noodle_y_origin" value="-${cabinet_length/4-0.002}" />
-  <xacro:property name="a_noodle_z_origin" value="0.100" />
-  <xacro:property name="a_noodle_x_offset" value="-0.130" />
-  <xacro:property name="a_noodle_y_offset" value="0.000" />
-  <xacro:property name="a_noodle_z_offset" value="0.000" />
-  <link name="a_noodle1" />
-  <joint name="a_noodle1_joint" type="fixed">
-    <parent link="a_cabinet_shelf1_origin_center" />
-    <child link="a_noodle1" />
-    <origin rpy="0 0 ${pi/2}" xyz="${a_noodle_x_origin} ${a_noodle_y_origin} ${a_noodle_z_origin}" />
+  <link name="a_cabinet_standpoint"/>
+  <joint name="a_cabinet_standpoint_joint" type="fixed">
+    <parent link="a_cabinet_base" />
+    <child  link="a_cabinet_standpoint" />
+    <origin xyz="${cabinet_width/2} -0.6 0" rpy="0 0 ${pi/2}" />
   </joint>
-  <link name="a_noodle2" />
-  <joint name="a_noodle2_joint" type="fixed">
-    <parent link="a_cabinet_shelf1_origin_center" />
-    <child link="a_noodle2" />
-    <origin rpy="0 0 ${pi/2}" xyz="${a_noodle_x_origin + a_noodle_x_offset*1} ${a_noodle_y_origin + a_noodle_y_offset*1} ${a_noodle_z_origin + a_noodle_z_offset*1}" />
+  <!-- Frames to place items on cabinet -->
+  <link name="a_item_in_cabinet"/>
+  <joint name="a_item_in_cabinet_joint" type="fixed">
+    <parent link="a_cabinet_shelf1_origin" />
+    <child  link="a_item_in_cabinet" />
+    <origin xyz="${cabinet_width/12} 0.1 0.08" rpy="${pi/2} ${pi/2} 0" />
   </joint>
-  <link name="a_noodle3" />
-  <joint name="a_noodle3_joint" type="fixed">
-    <parent link="a_cabinet_shelf1_origin_center" />
-    <child link="a_noodle3" />
-    <origin rpy="0 0 ${pi/2}" xyz="${a_noodle_x_origin + a_noodle_x_offset*2} ${a_noodle_y_origin + a_noodle_y_offset*2} ${a_noodle_z_origin + a_noodle_z_offset*2}" />
+  <link name="b_item_in_cabinet"/>
+  <joint name="b_item_in_cabinet_joint" type="fixed">
+    <parent link="a_item_in_cabinet" />
+    <child  link="b_item_in_cabinet" />
+    <origin xyz="0 ${cabinet_width/6} 0" rpy="0 0 0" />
   </joint>
-  <xacro:property name="b_noodle_x_origin" value="0.065" />
-  <xacro:property name="b_noodle_y_origin" value="-${cabinet_length/4-0.002}" />
-  <xacro:property name="b_noodle_z_origin" value="0.100" />
-  <xacro:property name="b_noodle_x_offset" value="0.130" />
-  <xacro:property name="b_noodle_y_offset" value="0.000" />
-  <xacro:property name="b_noodle_z_offset" value="0.000" />
-  <link name="b_noodle1" />
-  <joint name="b_noodle1_joint" type="fixed">
-    <parent link="a_cabinet_shelf1_origin_center" />
-    <child link="b_noodle1" />
-    <origin rpy="0 0 ${pi/2}" xyz="${b_noodle_x_origin} ${b_noodle_y_origin} ${b_noodle_z_origin}" />
+  <link name="c_item_in_cabinet"/>
+  <joint name="c_item_in_cabinet_joint" type="fixed">
+    <parent link="b_item_in_cabinet" />
+    <child  link="c_item_in_cabinet" />
+    <origin xyz="0 ${cabinet_width/6} 0" rpy="0 0 0" />
   </joint>
-  <link name="b_noodle2" />
-  <joint name="b_noodle2_joint" type="fixed">
-    <parent link="a_cabinet_shelf1_origin_center" />
-    <child link="b_noodle2" />
-    <origin rpy="0 0 ${pi/2}" xyz="${b_noodle_x_origin + b_noodle_x_offset*1} ${b_noodle_y_origin + b_noodle_y_offset*1} ${b_noodle_z_origin + b_noodle_z_offset*1}" />
+  <link name="d_item_in_cabinet"/>
+  <joint name="d_item_in_cabinet_joint" type="fixed">
+    <parent link="c_item_in_cabinet" />
+    <child  link="d_item_in_cabinet" />
+    <origin xyz="0 ${cabinet_width/6} 0" rpy="0 0 0" />
   </joint>
-  <link name="b_noodle3" />
-  <joint name="b_noodle3_joint" type="fixed">
-    <parent link="a_cabinet_shelf1_origin_center" />
-    <child link="b_noodle3" />
-    <origin rpy="0 0 ${pi/2}" xyz="${b_noodle_x_origin + b_noodle_x_offset*2} ${b_noodle_y_origin + b_noodle_y_offset*2} ${b_noodle_z_origin + b_noodle_z_offset*2}" />
-  </joint> -->
+  <link name="e_item_in_cabinet"/>
+  <joint name="e_item_in_cabinet_joint" type="fixed">
+    <parent link="d_item_in_cabinet" />
+    <child  link="e_item_in_cabinet" />
+    <origin xyz="0 ${cabinet_width/6} 0" rpy="0 0 0" />
+  </joint>
+  <link name="f_item_in_cabinet"/>
+  <joint name="f_item_in_cabinet_joint" type="fixed">
+    <parent link="e_item_in_cabinet" />
+    <child  link="f_item_in_cabinet" />
+    <origin xyz="0 ${cabinet_width/6} 0" rpy="0 0 0" />
+  </joint>
   <!-- AR markers -->
   <xacro:include filename="$(find aist_gazebo)/urdf/ar_marker.urdf.xacro"/>

File: aist_scene_description/urdf/tray.urdf.xacro (robot description, xacro)
@@ -3,20 +3,26 @@
        name="table">
   <xacro:include filename="$(find aist_scene_description)/urdf/aist_box.urdf.xacro"/>
-  <xacro:include filename="$(find aist_scene_description)/urdf/aist_floating_box.urdf.xacro"/>
   <xacro:macro name="tray"
 	       params="prefix width length height parent *origin">
     <xacro:property name="tray_thickness"	value="0.005" />
-    <xacro:aist_floating_box name="${prefix}tray"
-			     width="${width}"
-			     length="${length}"
-			     height="${tray_thickness}"
-			     parent="${parent}">
+    <xacro:property name="item_radius"		value="0.04" />
+    <link name="${prefix}tray"/>
+    <joint name="${prefix}tray" type="floating">
+      <parent link="${parent}" />
+      <child  link="${prefix}tray" />
       <xacro:insert_block name="origin"/>
-    </xacro:aist_floating_box>
+    </joint>
+    <xacro:aist_box name="${prefix}tray_bottom"
+		    width="${width}"
+		    length="${length}"
+		    height="${tray_thickness}"
+		    parent="${parent}">
+      <origin xyz="${-width/2} ${-tray_thickness/2} 0" rpy="0 0 0"/>
+    </xacro:aist_box>
     <xacro:aist_box name="${prefix}tray_wall0"
 		    width="${width}"
 		    length="${tray_thickness}"
 		    height="${height - tray_thickness}"
-		    parent="${prefix}tray">
+		    parent="${prefix}tray_bottom">
       <origin xyz="0 0 ${tray_thickness}" rpy="0 0 0"/>
     </xacro:aist_box>
@@ -25,5 +31,5 @@
 		    length="${length - 2*tray_thickness}"
 		    height="${height - tray_thickness}"
-		    parent="${prefix}tray">
+		    parent="${prefix}tray_bottom">
       <origin xyz="0 ${tray_thickness} ${tray_thickness}" rpy="0 0 0"/>
     </xacro:aist_box>
@@ -32,5 +38,5 @@
 		    length="${tray_thickness}"
 		    height="${height - tray_thickness}"
-		    parent="${prefix}tray">
+		    parent="${prefix}tray_bottom">
       <origin xyz="0 ${length - tray_thickness} ${tray_thickness}" rpy="0 0 0"/>
     </xacro:aist_box>
@@ -39,24 +45,47 @@
 		    length="${length - 2*tray_thickness}"
 		    height="${height - tray_thickness}"
-		    parent="${prefix}tray">
+		    parent="${prefix}tray_bottom">
       <origin xyz="${width - tray_thickness} ${tray_thickness} ${tray_thickness}"
 	      rpy="0 0 0"/>
     </xacro:aist_box>
-    <xacro:macro name="auxiliary_frame" params="parent framename *origin">
-      <joint name="${parent}_${framename}" type="fixed">
-	<parent link="${parent}" />
-	<child link = "${parent}_${framename}"/>
-	<xacro:insert_block name="origin"/>
-      </joint>
-      <link name="${parent}_${framename}"/>
-    </xacro:macro>
-    <xacro:auxiliary_frame parent="${prefix}tray" framename="origin">
-      <origin xyz="${tray_thickness} ${tray_thickness} ${tray_thickness}"
-	      rpy="0 0 0"/>
-    </xacro:auxiliary_frame>
-    <xacro:auxiliary_frame parent="${prefix}tray_origin" framename="center">
-      <origin xyz="${width/2 - tray_thickness} ${length/2 - tray_thickness} 0"
-	      rpy="0 0 0"/>
-    </xacro:auxiliary_frame>
+    <link name="b_item_on_${prefix}tray"/>
+    <joint name="b_item_on_${prefix}tray_joint" type="fixed">
+      <parent link ="${prefix}tray_bottom"/>
+      <child  link="b_item_on_${prefix}tray"/>
+      <origin xyz="${width/2}
+		   ${length/2}
+		   ${tray_thickness + item_radius}"
+    	      rpy="0 0 ${-pi/2}"/>
+    </joint>
+    <link name="a_item_on_${prefix}tray"/>
+    <joint name="a_item_on_${prefix}tray_joint" type="fixed">
+      <parent link ="b_item_on_${prefix}tray"/>
+      <child  link="a_item_on_${prefix}tray"/>
+      <origin xyz="0 ${-width/4 + tray_thickness/2} 0" rpy="0 0 0"/>
+    </joint>
+    <link name="c_item_on_${prefix}tray"/>
+    <joint name="c_item_on_${prefix}tray_joint" type="fixed">
+      <parent link ="b_item_on_${prefix}tray"/>
+      <child  link="c_item_on_${prefix}tray"/>
+      <origin xyz="0 ${width/4 - tray_thickness/2} 0" rpy="0 0 0"/>
+    </joint>
+    <link name="d_item_on_${prefix}tray"/>
+    <joint name="d_item_on_${prefix}tray_joint" type="fixed">
+      <parent link ="a_item_on_${prefix}tray"/>
+      <child  link="d_item_on_${prefix}tray"/>
+      <origin xyz="0 0 0" rpy="0 0 0"/>
+    </joint>
+    <link name="e_item_on_${prefix}tray"/>
+    <joint name="e_item_on_${prefix}tray_joint" type="fixed">
+      <parent link ="b_item_on_${prefix}tray"/>
+      <child  link="e_item_on_${prefix}tray"/>
+      <origin xyz="0 0 0" rpy="0 0 0"/>
+    </joint>
+    <link name="f_item_on_${prefix}tray"/>
+    <joint name="f_item_on_${prefix}tray_joint" type="fixed">
+      <parent link ="c_item_on_${prefix}tray"/>
+      <child  link="f_item_on_${prefix}tray"/>
+      <origin xyz="0 0 0" rpy="0 0 0"/>
+    </joint>
   </xacro:macro>
 </robot>

Commit message: Added trays to the environment.

File: aist_scene_description/urdf/ceatec_base_scene_environment.urdf.xacro (robot description, xacro)
@@ -2,23 +2,23 @@
 <robot xmlns:xacro="http://www.ros.org/wiki/xacro"
        name="ceatec_base_scene_environment">
-  <xacro:property name="workspace_width" value="3.000"/>
-  <xacro:property name="workspace_length" value="2.000"/>
-  <xacro:property name="a_table_width" value="0.530"/>
-  <xacro:property name="a_table_length" value="0.315"/>
-  <xacro:property name="a_table_height" value="0.540"/>
-  <xacro:property name="b_table_width" value="0.700"/>
-  <xacro:property name="b_table_length" value="0.350"/>
-  <xacro:property name="b_table_height" value="0.600"/>
-  <xacro:property name="cabinet_width" value="0.925"/>
-  <xacro:property name="cabinet_length" value="0.420"/>
-  <xacro:property name="cabinet_base_height" value="0.180"/>
-  <xacro:property name="cabinet_shelf1_height" value="0.443"/>
-  <xacro:property name="cabinet_shelf2_height" value="0.743"/>
-  <xacro:property name="cabinet_shelf3_height" value="1.043"/>
-  <xacro:property name="cabinet_shelf4_height" value="1.366"/>
-  <xacro:property name="cabinet_back_height" value="1.711"/>
-  <xacro:property name="tray_width" value="0.340"/>
-  <xacro:property name="tray_length" value="0.250"/>
-  <xacro:property name="tray_height" value="0.062"/>
+  <xacro:property name="workspace_width"	value="3.000"/>
+  <xacro:property name="workspace_length"	value="2.000"/>
+  <xacro:property name="a_table_width"		value="0.530"/>
+  <xacro:property name="a_table_length"		value="0.315"/>
+  <xacro:property name="a_table_height"		value="0.540"/>
+  <xacro:property name="b_table_width"		value="0.700"/>
+  <xacro:property name="b_table_length"		value="0.350"/>
+  <xacro:property name="b_table_height"		value="0.600"/>
+  <xacro:property name="cabinet_width"		value="0.925"/>
+  <xacro:property name="cabinet_length"		value="0.420"/>
+  <xacro:property name="cabinet_base_height"	value="0.180"/>
+  <xacro:property name="cabinet_shelf1_height"	value="0.443"/>
+  <xacro:property name="cabinet_shelf2_height"	value="0.743"/>
+  <xacro:property name="cabinet_shelf3_height"	value="1.043"/>
+  <xacro:property name="cabinet_shelf4_height"	value="1.366"/>
+  <xacro:property name="cabinet_back_height"	value="1.711"/>
+  <xacro:property name="tray_width"		value="0.340"/>
+  <xacro:property name="tray_length"		value="0.250"/>
+  <xacro:property name="tray_height"		value="0.062"/>
   <!-- Main workspace -->
   <link name="ground"/>
@@ -42,5 +42,5 @@
   <joint name="a_tray_on_a_table_joint" type="fixed">
     <parent link="a_table_top_origin_center" />
-    <child link="a_tray_on_a_table" />
+    <child  link="a_tray_on_a_table" />
     <origin xyz="0 ${-tray_length/2} 0" rpy="0 0 0" />
   </joint>
@@ -48,5 +48,5 @@
   <joint name="b_tray_on_a_table_joint" type="fixed">
     <parent link="a_table_top_origin_center" />
-    <child link="b_tray_on_a_table" />
+    <child  link="b_tray_on_a_table" />
     <origin xyz="0 ${-tray_length/2} 0" rpy="0 0 0" />
   </joint>
@@ -55,5 +55,5 @@
     <parent link="a_table_leg0" />
     <child  link="a_table_standpoint" />
-    <origin xyz="${a_table_width/2} -0.4 0" rpy="0 0 ${pi/2}" />
+    <origin xyz="${a_table_width/2} -0.7 0" rpy="0 0 ${pi/2}" />
   </joint>
   <!-- b_table -->
@@ -72,5 +72,5 @@
   <joint name="a_tray_on_b_table_joint" type="fixed">
     <parent link="b_table_top_origin_center" />
-    <child link="a_tray_on_b_table" />
+    <child  link="a_tray_on_b_table" />
     <origin xyz="${-tray_width/2 - 0.05} ${-tray_length/2} 0" rpy="0 0 0" />
   </joint>
@@ -78,5 +78,5 @@
   <joint name="b_tray_on_b_table_joint" type="fixed">
     <parent link="b_table_top_origin_center" />
-    <child link="b_tray_on_b_table" />
+    <child  link="b_tray_on_b_table" />
     <origin xyz="${tray_width/2 + 0.05} ${-tray_length/2} 0" rpy="0 0 0" />
   </joint>
@@ -85,12 +85,21 @@
     <parent link="b_table_leg0" />
     <child  link="b_table_standpoint" />
-    <origin xyz="${b_table_width/2} -0.4 0" rpy="0 0 ${pi/2}" />
+    <origin xyz="${b_table_width/2} -0.7 0" rpy="0 0 ${pi/2}" />
   </joint>
   <!-- Cabinet -->
   <xacro:include filename="$(find aist_scene_description)/urdf/cabinet.urdf.xacro"/>
-  <xacro:cabinet prefix="a_" width="${cabinet_width}" length="${cabinet_length}" base_height="${cabinet_base_height}" shelf1_height="${cabinet_shelf1_height}" shelf2_height="${cabinet_shelf2_height}" shelf3_height="${cabinet_shelf3_height}" shelf4_height="${cabinet_shelf4_height}" back_height="${cabinet_back_height}" parent="ground">
+  <xacro:cabinet prefix="a_"
+		 width="${cabinet_width}"
+		 length="${cabinet_length}"
+		 base_height="${cabinet_base_height}"
+		 shelf1_height="${cabinet_shelf1_height}"
+		 shelf2_height="${cabinet_shelf2_height}"
+		 shelf3_height="${cabinet_shelf3_height}"
+		 shelf4_height="${cabinet_shelf4_height}"
+		 back_height="${cabinet_back_height}" parent="ground">
     <origin xyz="${workspace_width/2   - cabinet_length}
 		 ${-workspace_length/2 + cabinet_width}
-		 0" rpy="0 0 ${-pi/2}"/>
+		 0"
+	    rpy="0 0 ${-pi/2}"/>
   </xacro:cabinet>
   <link name="a_cabinet_standpoint"/>
@@ -139,16 +148,28 @@
   <!-- AR markers -->
   <xacro:include filename="$(find aist_gazebo)/urdf/ar_marker.urdf.xacro"/>
-  <xacro:ar_marker prefix="a_cabinet_" parent="a_cabinet_shelf1_origin" marker_id="17" size="0.1" thickness="0.001">
+  <xacro:ar_marker prefix="a_cabinet_" parent="a_cabinet_shelf1_origin"
+		   marker_id="17" size="0.1" thickness="0.001">
     <origin xyz="${cabinet_width - 0.05} 0.05 0.001" rpy="0 0 0"/>
   </xacro:ar_marker>
-  <xacro:ar_marker prefix="a_table_" parent="a_table_top_origin" marker_id="26" size="0.1" thickness="0.001">
+  <xacro:ar_marker prefix="a_table_" parent="a_table_top_origin"
+		   marker_id="26" size="0.1" thickness="0.001">
     <origin xyz="0.05 0.05 0.001" rpy="0 0 0"/>
   </xacro:ar_marker>
-  <!-- I would like to remove the "world" link definition, but apparently it is necessary for Gazebo -->
-  <!-- <joint name="ground_base_joint" type="planar"> -->
-  <!--   <parent link="ground"/> -->
-  <!--   <child link="base_link"/> -->
-  <!--   <origin xyz="0 -0.5 0" rpy="0 0 0"/> -->
-  <!-- </joint> -->
+  <!-- Trays -->
+  <xacro:include filename="$(find aist_scene_description)/urdf/tray.urdf.xacro"/>
+  <xacro:tray prefix="a_"
+	      width="${tray_width}"
+	      length="${tray_length}"
+	      height="${tray_height}"
+	      parent="a_tray_on_a_table">
+    <origin xyz="${-tray_width/2} 0 0" rpy="0 0 0"/>
+  </xacro:tray>
+  <xacro:tray prefix="b_"
+	      width="${tray_width}"
+	      length="${tray_length}"
+	      height="${tray_height}"
+	      parent="b_tray_on_b_table">
+    <origin xyz="${-tray_width/2} 0 0" rpy="0 0 0"/>
+  </xacro:tray>
   <!-- I would like to remove the "world" link definition, but
        apparently it is necessary for Gazebo -->

Commit message: Fixed item coordinate frames.

File: aist_scene_description/urdf/ceatec_base_scene_environment.urdf.xacro (robot description, xacro)
@@ -114,5 +114,5 @@
     <parent link="a_cabinet_shelf1_origin" />
     <child  link="a_item_in_cabinet" />
-    <origin xyz="${cabinet_width/12} 0.1 0.08" rpy="${pi/2} ${pi/2} 0" />
+    <origin xyz="${cabinet_width/12} 0.1 0.08" rpy="${pi/2} ${-pi/2} 0"/>
   </joint>
   <link name="b_item_in_cabinet"/>
@@ -120,5 +120,5 @@
     <parent link="a_item_in_cabinet" />
     <child  link="b_item_in_cabinet" />
-    <origin xyz="0 ${cabinet_width/6} 0" rpy="0 0 0" />
+    <origin xyz="0 ${-cabinet_width/6} 0" rpy="0 0 0" />
   </joint>
   <link name="c_item_in_cabinet"/>
@@ -126,5 +126,5 @@
     <parent link="b_item_in_cabinet" />
     <child  link="c_item_in_cabinet" />
-    <origin xyz="0 ${cabinet_width/6} 0" rpy="0 0 0" />
+    <origin xyz="0 ${-cabinet_width/6} 0" rpy="0 0 0" />
   </joint>
   <link name="d_item_in_cabinet"/>
@@ -132,5 +132,5 @@
     <parent link="c_item_in_cabinet" />
     <child  link="d_item_in_cabinet" />
-    <origin xyz="0 ${cabinet_width/6} 0" rpy="0 0 0" />
+    <origin xyz="0 ${-cabinet_width/6} 0" rpy="0 0 0" />
   </joint>
   <link name="e_item_in_cabinet"/>
@@ -138,5 +138,5 @@
     <parent link="d_item_in_cabinet" />
     <child  link="e_item_in_cabinet" />
-    <origin xyz="0 ${cabinet_width/6} 0" rpy="0 0 0" />
+    <origin xyz="0 ${-cabinet_width/6} 0" rpy="0 0 0" />
   </joint>
   <link name="f_item_in_cabinet"/>
@@ -144,5 +144,5 @@
     <parent link="e_item_in_cabinet" />
     <child  link="f_item_in_cabinet" />
-    <origin xyz="0 ${cabinet_width/6} 0" rpy="0 0 0" />
+    <origin xyz="0 ${-cabinet_width/6} 0" rpy="0 0 0" />
   </joint>
   <!-- AR markers -->

File: aist_scene_description/urdf/tray.urdf.xacro (robot description, xacro)
@@ -56,5 +56,5 @@
 		   ${length/2}
 		   ${tray_thickness + item_radius}"
-    	      rpy="0 0 ${-pi/2}"/>
+    	      rpy="0 0 ${pi/2}"/>
     </joint>
     <link name="a_item_on_${prefix}tray"/>
@@ -62,5 +62,5 @@
       <parent link ="b_item_on_${prefix}tray"/>
       <child  link="a_item_on_${prefix}tray"/>
-      <origin xyz="0 ${-width/3 + tray_thickness/2} 0" rpy="0 0 0"/>
+      <origin xyz="0 ${width/3 + tray_thickness/2} 0" rpy="0 0 0"/>
     </joint>
     <link name="c_item_on_${prefix}tray"/>
@@ -68,5 +68,5 @@
       <parent link ="b_item_on_${prefix}tray"/>
       <child  link="c_item_on_${prefix}tray"/>
-      <origin xyz="0 ${width/3 - tray_thickness/2} 0" rpy="0 0 0"/>
+      <origin xyz="0 ${-width/3 - tray_thickness/2} 0" rpy="0 0 0"/>
     </joint>
     <link name="d_item_on_${prefix}tray"/>
