Commit message: Trying to launch two robots but yet succeeded.

File: aist_scene_description/urdf/dtorobo_base_scene.urdf.xacro (robot description, xacro)
@@ -5,9 +5,7 @@
   <xacro:property name="a_torobo_x" value="0"/>
   <xacro:property name="a_torobo_y" value="-0.4875"/>
-  <!-- <xacro:property name="a_torobo_theta" value="${pi}"/> -->
   <xacro:property name="b_torobo_x" value="0"/>
   <xacro:property name="b_torobo_y" value="0.4875"/>
-  <xacro:property name="b_torobo_theta" value="${pi}"/>
-  <xacro:property name="bots_z" value="0.785"/>
+  <xacro:property name="bots_z"	    value="0.785"/>
   <!-- common stuff -->
   <xacro:include filename="$(find aist_gazebo)/urdf/aist_base_scene.gazebo"/>
@@ -22,26 +20,25 @@
 		  box_w="${table_w}" box_l="${table_l}" box_h="${table_h}"
 		  parent="o2as_ground">
-    <origin xyz="${-table_w/2} ${-table_l/2} ${bots_z - table_h}" rpy="0 0 0"/>
+    <origin xyz="${-table_w/2} ${-table_l/2} ${bots_z -table_h}" rpy="0 0 0"/>
   </xacro:o2as_box>
   <link name="workspace_center"/>
   <joint name="world_to_workspace" type="fixed">
     <parent link="o2as_ground"/>
-    <child link="workspace_center"/>
+    <child  link="workspace_center"/>
     <origin xyz="0 0 ${bots_z}" rpy="0 0 0"/>
   </joint>
   <!-- robot arms -->
   <xacro:include filename="$(find aist_scene_description)/urdf/torobo_arm.urdf.xacro"/>
-  <xacro:torobo_arm_gripper prefix="a_torobo"/>
+  <xacro:torobo_arm_gripper prefix="a_torobo_"/>
   <joint name="world_a_torobo_joint" type="fixed">
     <parent link="o2as_ground"/>
-    <child  link= "a_torobo/base"/>
-    <origin xyz="${a_torobo_x} ${a_torobo_y} ${bots_z}" rpy="0 0 0"/>
+    <child  link= "a_torobo_base"/>
+    <origin xyz="${a_torobo_x} ${a_torobo_y} ${bots_z}" rpy="0 0 ${pi/2}"/>
   </joint>
-  <xacro:torobo_arm_gripper prefix="b_torobo"/>
+  <xacro:torobo_arm_gripper prefix="b_torobo_"/>
   <joint name="world_b_torobo_joint" type="fixed">
     <parent link="o2as_ground"/>
-    <child  link= "b_torobo/base"/>
-    <origin xyz="${b_torobo_x} ${b_torobo_y} ${bots_z}"
-	    rpy="0 0 ${b_torobo_theta}"/>
+    <child  link= "b_torobo_base"/>
+    <origin xyz="${b_torobo_x} ${b_torobo_y} ${bots_z}" rpy="0 0 ${-pi/2}"/>
   </joint>
   <!-- Add PhoXi 3D scanner -->

File: aist_scene_description/urdf/torobo_arm.urdf.xacro (robot description, xacro)
@@ -5,12 +5,12 @@
   <xacro:macro name="torobo_arm" params="prefix">
     <xacro:property name="COL_K" value="1.2"/>
-    <link name="${prefix}/base"/>
+    <link name="${prefix}base"/>
     <!-- =============== Link & Joint =============== -->
-    <joint name="${prefix}/arm/root" type="fixed">
+    <joint name="${prefix}arm/root" type="fixed">
       <origin xyz="0 0 0"/>
-      <parent link="${prefix}/base"/>
-      <child link="${prefix}/arm/link_0"/>
-    </joint>
-    <link name="${prefix}/arm/link_0">
+      <parent link="${prefix}base"/>
+      <child link="${prefix}arm/link_0"/>
+    </joint>
+    <link name="${prefix}arm/link_0">
       <visual>
 	<geometry>
@@ -33,12 +33,12 @@
       </inertial>
     </link>
-    <joint name="${prefix}/arm/joint_1" type="revolute">
-      <parent link="${prefix}/arm/link_0"/>
-      <child link="${prefix}/arm/link_1"/>
+    <joint name="${prefix}arm/joint_1" type="revolute">
+      <parent link="${prefix}arm/link_0"/>
+      <child link="${prefix}arm/link_1"/>
       <origin xyz="0 0 0.220" rpy="0 0 0"/>
       <axis xyz="0 0 1"/>
       <limit lower="${-170*M_PI/180}" upper="${170*M_PI/180}" effort="110" velocity="${100*M_PI/180}"/>
     </joint>
-    <link name="${prefix}/arm/link_1">
+    <link name="${prefix}arm/link_1">
       <visual>
 	<geometry>
@@ -59,12 +59,12 @@
       </inertial>
     </link>
-    <joint name="${prefix}/arm/joint_2" type="revolute">
-      <parent link="${prefix}/arm/link_1"/>
-      <child link="${prefix}/arm/link_2"/>
+    <joint name="${prefix}arm/joint_2" type="revolute">
+      <parent link="${prefix}arm/link_1"/>
+      <child link="${prefix}arm/link_2"/>
       <origin xyz="0 0 0" rpy="${-90*M_PI/180} 0 0"/>
       <axis xyz="0 0 1"/>
       <limit lower="${-110*M_PI/180}" upper="${110*M_PI/180}" effort="110" velocity="${100*M_PI/180}"/>
     </joint>
-    <link name="${prefix}/arm/link_2">
+    <link name="${prefix}arm/link_2">
       <visual>
 	<geometry>
@@ -85,12 +85,12 @@
       </inertial>
     </link>
-    <joint name="${prefix}/arm/joint_3" type="revolute">
-      <parent link="${prefix}/arm/link_2"/>
-      <child link="${prefix}/arm/link_3"/>
+    <joint name="${prefix}arm/joint_3" type="revolute">
+      <parent link="${prefix}arm/link_2"/>
+      <child link="${prefix}arm/link_3"/>
       <origin xyz="0 -0.3 0" rpy="${90*M_PI/180} 0 0"/>
       <axis xyz="0 0 1"/>
       <limit lower="${-165*M_PI/180}" upper="${165*M_PI/180}" effort="70" velocity="${120*M_PI/180}"/>
     </joint>
-    <link name="${prefix}/arm/link_3">
+    <link name="${prefix}arm/link_3">
       <visual>
 	<geometry>
@@ -111,12 +111,12 @@
       </inertial>
     </link>
-    <joint name="${prefix}/arm/joint_4" type="revolute">
-      <parent link="${prefix}/arm/link_3"/>
-      <child link="${prefix}/arm/link_4"/>
+    <joint name="${prefix}arm/joint_4" type="revolute">
+      <parent link="${prefix}arm/link_3"/>
+      <child link="${prefix}arm/link_4"/>
       <origin xyz="0 0 0" rpy="${-90*M_PI/180} 0 0"/>
       <axis xyz="0 0 1"/>
       <limit lower="${-125*M_PI/180}" upper="${125*M_PI/180}" effort="70" velocity="${120*M_PI/180}"/>
     </joint>
-    <link name="${prefix}/arm/link_4">
+    <link name="${prefix}arm/link_4">
       <visual>
 	<geometry>
@@ -137,12 +137,12 @@
       </inertial>
     </link>
-    <joint name="${prefix}/arm/joint_5" type="revolute">
-      <parent link="${prefix}/arm/link_4"/>
-      <child link="${prefix}/arm/link_5"/>
+    <joint name="${prefix}arm/joint_5" type="revolute">
+      <parent link="${prefix}arm/link_4"/>
+      <child link="${prefix}arm/link_5"/>
       <origin xyz="0 -0.3 0" rpy="${90*M_PI/180} 0 0"/>
       <axis xyz="0 0 1"/>
       <limit lower="${-165*M_PI/180}" upper="${165*M_PI/180}" effort="30" velocity="${160*M_PI/180}"/>
     </joint>
-    <link name="${prefix}/arm/link_5">
+    <link name="${prefix}arm/link_5">
       <visual>
 	<geometry>
@@ -163,12 +163,12 @@
       </inertial>
     </link>
-    <joint name="${prefix}/arm/joint_6" type="revolute">
-      <parent link="${prefix}/arm/link_5"/>
-      <child link="${prefix}/arm/link_6"/>
+    <joint name="${prefix}arm/joint_6" type="revolute">
+      <parent link="${prefix}arm/link_5"/>
+      <child link="${prefix}arm/link_6"/>
       <origin xyz="0 0 0" rpy="${-90*M_PI/180} 0 0"/>
       <axis xyz="0 0 1"/>
       <limit lower="${-120*M_PI/180}" upper="${120*M_PI/180}" effort="30" velocity="${160*M_PI/180}"/>
     </joint>
-    <link name="${prefix}/arm/link_6">
+    <link name="${prefix}arm/link_6">
       <visual>
 	<geometry>
@@ -189,12 +189,12 @@
       </inertial>
     </link>
-    <joint name="${prefix}/arm/joint_7" type="revolute">
-      <parent link="${prefix}/arm/link_6"/>
-      <child link="${prefix}/arm/link_7"/>
+    <joint name="${prefix}arm/joint_7" type="revolute">
+      <parent link="${prefix}arm/link_6"/>
+      <child link="${prefix}arm/link_7"/>
       <origin xyz="0 -0.170 0" rpy="${90*M_PI/180} 0 0"/>
       <axis xyz="0 0 1"/>
       <limit lower="${-170*M_PI/180}" upper="${170*M_PI/180}" effort="15" velocity="${240*M_PI/180}"/>
     </joint>
-    <link name="${prefix}/arm/link_7">
+    <link name="${prefix}arm/link_7">
       <visual>
 	<geometry>
@@ -216,43 +216,43 @@
     </link>
     <!-- =============== Transmission =============== -->
-    <simple_transmission name="${prefix}/arm/joint_1" reduction="1"/>
-    <simple_transmission name="${prefix}/arm/joint_2" reduction="1"/>
-    <simple_transmission name="${prefix}/arm/joint_3" reduction="1"/>
-    <simple_transmission name="${prefix}/arm/joint_4" reduction="1"/>
-    <simple_transmission name="${prefix}/arm/joint_5" reduction="1"/>
-    <simple_transmission name="${prefix}/arm/joint_6" reduction="1"/>
-    <simple_transmission name="${prefix}/arm/joint_7" reduction="1"/>
+    <simple_transmission name="${prefix}arm/joint_1" reduction="1"/>
+    <simple_transmission name="${prefix}arm/joint_2" reduction="1"/>
+    <simple_transmission name="${prefix}arm/joint_3" reduction="1"/>
+    <simple_transmission name="${prefix}arm/joint_4" reduction="1"/>
+    <simple_transmission name="${prefix}arm/joint_5" reduction="1"/>
+    <simple_transmission name="${prefix}arm/joint_6" reduction="1"/>
+    <simple_transmission name="${prefix}arm/joint_7" reduction="1"/>
     <!-- Link1 -->
-    <gazebo reference="${prefix}/arm/link_1">
+    <gazebo reference="${prefix}arm/link_1">
       <mu1>0.2</mu1>
       <mu2>0.2</mu2>
     </gazebo>
     <!-- Link2 -->
-    <gazebo reference="${prefix}/arm/link_2">
+    <gazebo reference="${prefix}arm/link_2">
       <mu1>0.2</mu1>
       <mu2>0.2</mu2>
     </gazebo>
     <!-- Link3 -->
-    <gazebo reference="${prefix}/arm/link_3">
+    <gazebo reference="${prefix}arm/link_3">
       <mu1>0.2</mu1>
       <mu2>0.2</mu2>
     </gazebo>
     <!-- Link4 -->
-    <gazebo reference="${prefix}/arm/link_4">
+    <gazebo reference="${prefix}arm/link_4">
       <mu1>0.2</mu1>
       <mu2>0.2</mu2>
     </gazebo>
     <!-- Link5 -->
-    <gazebo reference="${prefix}/arm/link_5">
+    <gazebo reference="${prefix}arm/link_5">
       <mu1>0.2</mu1>
       <mu2>0.2</mu2>
     </gazebo>
     <!-- Link6 -->
-    <gazebo reference="${prefix}/arm/link_6">
+    <gazebo reference="${prefix}arm/link_6">
       <mu1>0.2</mu1>
       <mu2>0.2</mu2>
     </gazebo>
     <!-- Link7 -->
-    <gazebo reference="${prefix}/arm/link_7">
+    <gazebo reference="${prefix}arm/link_7">
       <mu1>0.2</mu1>
       <mu2>0.2</mu2>
@@ -265,14 +265,14 @@
   <xacro:macro name="torobo_arm_gripper" params="prefix">
     <xacro:torobo_arm prefix="${prefix}"/>
-    <xacro:gripper_macro prefix="${prefix}/gripper/"
-			 attach_link="${prefix}/arm/link_7"
+    <xacro:gripper_macro prefix="${prefix}gripper/"
+			 attach_link="${prefix}arm/link_7"
 			 attach_xyz="0 0 0"
 			 attach_rpy="0 0 0" />
-    <xacro:gripper_gazebo_macro prefix="${prefix}/gripper/"
+    <xacro:gripper_gazebo_macro prefix="${prefix}gripper/"
 				use_graspfix="false"/>
-    <link  name="${prefix}/gripper/tip_link"/>
-    <joint name="${prefix}/gripper/tip_joint" type="fixed">
-      <parent link="${prefix}/gripper/grasping_frame"/>
-      <child  link="${prefix}/gripper/tip_link"/>
+    <link  name="${prefix}gripper/tip_link"/>
+    <joint name="${prefix}gripper/tip_joint" type="fixed">
+      <parent link="${prefix}gripper/grasping_frame"/>
+      <child  link="${prefix}gripper/tip_link"/>
       <origin xyz="0 0 0" rpy="0 ${-M_PI/2} 0"/>
     </joint>

Commit message: Confirmed that torobo arms can be controlled by MoveIt.

File: aist_scene_description/urdf/dtorobo_base_scene.urdf.xacro (robot description, xacro)
@@ -30,15 +30,29 @@
   <!-- robot arms -->
   <xacro:include filename="$(find aist_scene_description)/urdf/torobo_arm.urdf.xacro"/>
-  <xacro:torobo_arm_gripper prefix="a_torobo_"/>
+  <xacro:torobo_arm prefix="a_torobo_"/>
   <joint name="world_a_torobo_joint" type="fixed">
     <parent link="o2as_ground"/>
-    <child  link= "a_torobo_base"/>
+    <child  link="a_torobo_base"/>
     <origin xyz="${a_torobo_x} ${a_torobo_y} ${bots_z}" rpy="0 0 ${pi/2}"/>
   </joint>
-  <xacro:torobo_arm_gripper prefix="b_torobo_"/>
+  <xacro:torobo_arm prefix="b_torobo_"/>
   <joint name="world_b_torobo_joint" type="fixed">
     <parent link="o2as_ground"/>
-    <child  link= "b_torobo_base"/>
+    <child  link="b_torobo_base"/>
     <origin xyz="${b_torobo_x} ${b_torobo_y} ${bots_z}" rpy="0 0 ${-pi/2}"/>
+  </joint>
+  <!-- Attach grippers -->
+  <xacro:include filename="$(find aist_scene_description)/urdf/torobo_gripper.urdf.xacro"/>
+  <xacro:torobo_gripper prefix="a_torobo_"/>
+  <joint name="a_torobo_arm_gripper_joint" type="fixed">
+    <parent link="a_torobo_arm/ee_link"/>
+    <child  link="a_torobo_gripper/base_link"/>
+    <origin xyz="0 0 0" rpy="0 0 0"/>
+  </joint>
+  <xacro:torobo_gripper prefix="b_torobo_"/>
+  <joint name="b_torobo_arm_gripper_joint" type="fixed">
+    <parent link="b_torobo_arm/ee_link"/>
+    <child  link="b_torobo_gripper/base_link"/>
+    <origin xyz="0 0 0" rpy="0 0 0"/>
   </joint>
   <!-- Add PhoXi 3D scanner -->

File: aist_scene_description/urdf/torobo_arm.urdf.xacro (robot description, xacro)
@@ -1,10 +1,8 @@
 <?xml version="1.0"?>
 <robot xmlns:xacro="http://ros.org/wiki/xacro">
-  <!-- =============== Constants =============== -->
   <xacro:property name="M_PI" value="3.1415926535897931"/>
   <!-- =============== Load Dependencies =============== -->
   <xacro:include filename="$(find torobo_description)/urdf/torobo.gazebo"/>
-  <xacro:include filename="$(find
-			   torobo_description)/urdf/torobo.transmission.xacro"/>
+  <xacro:include filename="$(find torobo_description)/urdf/torobo.transmission.xacro"/>
   <xacro:macro name="torobo_arm" params="prefix">
     <xacro:property name="COL_K" value="1.2"/>
@@ -219,4 +217,10 @@
       </inertial>
     </link>
+    <link name="${prefix}arm/ee_link"/>
+    <joint name="${prefix}arm/ee_joint" type="fixed">
+      <parent link="${prefix}arm/link_7"/>
+      <child  link="${prefix}arm/ee_link"/>
+      <origin xyz="0 0 0" rpy="0 ${-M_PI/2} 0"/>
+    </joint>
     <!-- =============== Transmission =============== -->
     <simple_transmission name="${prefix}arm/joint_1" reduction="1"/>
@@ -263,22 +267,3 @@
     </gazebo>
   </xacro:macro>
-  <xacro:include filename="$(find torobo_resources
-			   )/TRBG-L-B-001/urdf/gripper.urdf.xacro"/>
-  <xacro:include filename="$(find torobo_resources
-			   )/TRBG-L-B-001/urdf/gripper.gazebo"/>
-  <xacro:macro name="torobo_arm_gripper" params="prefix">
-    <xacro:torobo_arm prefix="${prefix}"/>
-    <xacro:gripper_macro prefix="${prefix}gripper/"
-			 attach_link="${prefix}arm/link_7"
-			 attach_xyz="0 0 0"
-			 attach_rpy="0 0 0" />
-    <xacro:gripper_gazebo_macro prefix="${prefix}gripper/"
-				use_graspfix="false"/>
-    <link  name="${prefix}gripper/tip_link"/>
-    <joint name="${prefix}gripper/tip_joint" type="fixed">
-      <parent link="${prefix}gripper/grasping_frame"/>
-      <child  link="${prefix}gripper/tip_link"/>
-      <origin xyz="0 0 0" rpy="0 ${-M_PI/2} 0"/>
-    </joint>
-  </xacro:macro>
 </robot>
