Commit message: Added Realsense camera to a_bot of pgrp configuration.

File: aist_scene_description/urdf/pgrp_base_scene.urdf.xacro (robot description, xacro)
@@ -86,4 +86,15 @@
 		 ${85.0482907121*pi/180}"/>
   </xacro:phoxi_m_camera>
+  <!-- Add RealSense camerar -->
+  <xacro:include filename="$(find o2as_realsense2_camera)/urdf/_d435.urdf.xacro" />
+  <link name="a_bot_cam_holder_link" />
+  <joint name="a_bot_cam_holder_joint" type="fixed">
+    <parent link="a_bot_wrist_2_link" />
+    <child  link="a_bot_cam_holder_link" />
+    <origin xyz="0.04 -0.06 0.20" rpy="${12*pi/180} 0.0 ${pi/2}" />
+  </joint>
+  <xacro:sensor_d435 prefix="a_bot_" parent="a_bot_cam_holder_link">
+    <origin xyz="0 0 0" rpy="0 0 0"/>
+  </xacro:sensor_d435>
   <!-- I would like to remove the "world" link definition, but apparently it is necessary for Gazebo -->
   <link name="world"/>

File: aist_scene_description/urdf/pgrp_calibration.urdf.xacro (robot description, xacro)
@@ -9,4 +9,9 @@
     <origin xyz="0.063 0.0 0.0215" rpy="0 0 0"/>
   </xacro:aist_ar_marker>
+  <xacro:aist_ar_marker prefix="a_bot_"
+  			parent="a_bot_gripper_base_link"
+  			marker_id="26">
+    <origin xyz="0.08 -0.065 0" rpy="${pi/2} 0 0"/>
+  </xacro:aist_ar_marker>
   <xacro:aist_ar_marker_16cm prefix="workspace_"
 			     parent="workspace_center"

Commit message: COnfirmed that eye_on_hand calibration works with simulation.

File: aist_scene_description/urdf/pgrp_base_scene.urdf.xacro (robot description, xacro)
@@ -92,5 +92,5 @@
     <parent link="a_bot_wrist_2_link" />
     <child  link="a_bot_cam_holder_link" />
-    <origin xyz="0.04 -0.06 0.20" rpy="${0*pi/180} 0.0 ${pi/2}" />
+    <origin xyz="0.0 -0.06 0.20" rpy="${0*pi/180} 0.0 ${pi/2}" />
   </joint>
   <xacro:sensor_d435 prefix="a_bot_" parent="a_bot_cam_holder_link">

Commit message: Cleaning up

File: aist_scene_description/urdf/pgrp_base_scene.urdf.xacro (robot description, xacro)
@@ -88,12 +88,6 @@
   <!-- Add RealSense camerar -->
   <xacro:include filename="$(find o2as_realsense2_camera)/urdf/_d435.urdf.xacro" />
-  <link name="a_bot_cam_holder_link" />
-  <joint name="a_bot_cam_holder_joint" type="fixed">
-    <parent link="a_bot_wrist_2_link" />
-    <child  link="a_bot_cam_holder_link" />
+  <xacro:sensor_d435 prefix="a_bot_" parent="a_bot_wrist_2_link">
     <origin xyz="0.0 -0.06 0.20" rpy="${0*pi/180} 0.0 ${pi/2}" />
-  </joint>
-  <xacro:sensor_d435 prefix="a_bot_" parent="a_bot_cam_holder_link">
-    <origin xyz="0 0 0" rpy="0 0 0"/>
   </xacro:sensor_d435>
   <!-- I would like to remove the "world" link definition, but apparently it is necessary for Gazebo -->

Commit message: Performed first pick experiment.

File: aist_scene_description/urdf/pgrp_base_scene.urdf.xacro (robot description, xacro)
@@ -79,12 +79,12 @@
   <xacro:include filename="$(find o2as_scene_description)/urdf/phoxi_m_camera.urdf.xacro"/>
   <xacro:phoxi_m_camera prefix="a_" parent="o2as_ground">
-    <origin xyz="0.547941636523
-		 -0.00827443204237
-		 1.67030171767"
-	    rpy="${-151.493605482*pi/180}
-		 ${0.698490882792*pi/180}
-		 ${85.0482907121*pi/180}"/>
+    <origin xyz="0.572594862147
+		 -0.0379835306047
+		 1.5494206833"
+	    rpy="${-147.507867496*pi/180}
+		 ${-0.907591630585*pi/180}
+		 ${91.5563307899*pi/180}"/>
   </xacro:phoxi_m_camera>
-  <!-- Add RealSense camerar -->
+  <!-- Add RealSense camera -->
   <xacro:include filename="$(find o2as_realsense2_camera)/urdf/_d435.urdf.xacro" />
   <xacro:sensor_d435 prefix="a_bot_" parent="a_bot_wrist_2_link">

File: aist_scene_description/urdf/pgrp_kitting.urdf.xacro (robot description, xacro)
@@ -12,5 +12,5 @@
 		  box_h="${plate_h}"
 		  parent="workspace_center">
-    <origin xyz="${table_w/2 - plate_w - 0.08} ${-plate_l/2} 0"
+    <origin xyz="${table_w/2 - plate_w - 0.14} ${-plate_l/2} 0"
 	    rpy="0 0 0"/>
   </xacro:o2as_box>
@@ -44,5 +44,5 @@
   <xacro:property name="set2_z" value="0"/>
   <!--bin_1_part_15_-->
-  <xacro:kitting_bin_1 binname	      ="bin_1_part_15"
+  <xacro:kitting_bin_1 binname	      ="bin_1_part_5"
 		       parent	      ="plate_center"
 		       z_origin_offset="${z_origin_offset_1}">
@@ -58,5 +58,5 @@
     <origin xyz="${plate_w/2 - bin_1_length/2}
 		 0
-		 ${-z_origin_offset_2}"
+		 ${-z_origin_offset_1}"
 	    rpy="0 0 0" />
   </xacro:kitting_bin_1>

Commit message: Assign surface normal and finger open direction to graspabilities.

File: aist_scene_description/urdf/pgrp_base_scene.urdf.xacro (robot description, xacro)
@@ -65,10 +65,10 @@
   <xacro:include filename="$(find aist_scene_description)/urdf/InnerOnlyGripper.urdf.xacro" />
   <xacro:InnerOnlyGripper prefix="a_bot_"  grippername = "gripper" parent = "a_bot_ft300_frange_link">
-    <origin xyz="0 0 0" rpy="${-pi/2} ${-1.3*pi/180} ${0.4*pi/180}"/>
+    <origin xyz="0 0 0" rpy="${-pi/2} ${-0.85*pi/180} ${-0.5*pi/180}"/>
   </xacro:InnerOnlyGripper>
   <xacro:include filename="$(find o2as_scene_description)/urdf/single_suction_gripper.urdf.xacro"/>
   <xacro:single_suction_gripper_o2as prefix="b_bot_"
   				     parent="b_bot_ft300_frange_link">
-    <origin xyz="0 0 0" rpy="0 ${0.8*pi/180} ${-0.5*pi/180}"/>
+    <origin xyz="0 0 0" rpy="0 ${0.2*pi/180} ${0.3*pi/180}"/>
   </xacro:single_suction_gripper_o2as>
   <!-- Add virtual wall to avoid collisions-->
@@ -79,10 +79,10 @@
   <xacro:include filename="$(find o2as_scene_description)/urdf/phoxi_m_camera.urdf.xacro"/>
   <xacro:phoxi_m_camera prefix="a_" parent="o2as_ground">
-    <origin xyz="0.572594862147
-		 -0.0379835306047
-		 1.5494206833"
-	    rpy="${-147.507867496*pi/180}
-		 ${-0.907591630585*pi/180}
-		 ${91.5563307899*pi/180}"/>
+    <origin xyz="0.573914993333
+		 -0.0330632805883
+		 1.55311851758"
+	    rpy="${-147.090382646*pi/180}
+		 ${-0.868638780663*pi/180}
+		 ${84.1231285383*pi/180}"/>
   </xacro:phoxi_m_camera>
   <!-- Add RealSense camera -->

File: aist_scene_description/urdf/pgrp_kitting.urdf.xacro (robot description, xacro)
@@ -99,15 +99,15 @@
   <!-- tray_1 -->
   <xacro:kitting_tray1 trayname="tray_1" parent="plate_center">
-    <origin xyz="${plate_w/2 - bin_1_length - bin_2_length - tray_length}
-		 0
+    <origin xyz="${plate_w/2 - bin_1_length - bin_2_length - tray_width}
+		 ${tray_length}
 		 0"
-	    rpy="0 0 0" />
+	    rpy="0 0 ${-pi/2}" />
   </xacro:kitting_tray1>
   <!-- tray_2 -->
   <xacro:kitting_tray2 trayname="tray_2" parent="plate_center">
-    <origin xyz="${plate_w/2 - bin_1_length - bin_2_length - tray_length}
-		 ${-tray_width}
+    <origin xyz="${plate_w/2 - bin_1_length - bin_2_length - tray_width}
+		 0
 		 0"
-	    rpy="0 0 0" />
+	    rpy="0 0 ${-pi/2}" />
   </xacro:kitting_tray2>
 </robot>

Commit message: Use MarkerArray instead of Marker for publishing visualization markers.

File: aist_scene_description/urdf/pgrp_base_scene.urdf.xacro (robot description, xacro)
@@ -73,16 +73,16 @@
   </xacro:single_suction_gripper_o2as>
   <!-- Add virtual wall to avoid collisions-->
-  <!-- <xacro:o2as_box boxname="vwall1" box_w="0.01" box_l="0.5" box_h="0.6" parent="o2as_ground"> -->
-  <!--   <origin xyz="0.50 -0.25 ${bots_z}" rpy="0 0 0"/> -->
-  <!-- </xacro:o2as_box> -->
+  <xacro:o2as_box boxname="vwall1" box_w="0.01" box_l="0.3" box_h="0.6" parent="o2as_ground">
+    <origin xyz="0.45 -0.15 ${bots_z}" rpy="0 0 0"/>
+  </xacro:o2as_box>
   <!-- Add PhoXi 3D scanner -->
   <xacro:include filename="$(find o2as_scene_description)/urdf/phoxi_m_camera.urdf.xacro"/>
   <xacro:phoxi_m_camera prefix="a_" parent="o2as_ground">
-    <origin xyz="0.573914993333
-		 -0.0330632805883
-		 1.55311851758"
-	    rpy="${-147.090382646*pi/180}
-		 ${-0.868638780663*pi/180}
-		 ${84.1231285383*pi/180}"/>
+    <origin xyz="0.571555325522
+		 -0.0254263761312
+		 1.55210350714"
+	    rpy="${-146.961510137*pi/180}
+		 ${-0.588467063736*pi/180}
+		 ${83.8809430549*pi/180}"/>
   </xacro:phoxi_m_camera>
   <!-- Add RealSense camera -->

Commit message: Updated srdf files to add a group all_bots. matlab_graspability_server.m updated to improve handling background and mask images.

File: aist_scene_description/urdf/pgrp_base_scene.urdf.xacro (robot description, xacro)
@@ -64,11 +64,13 @@
   <!-- Spawn and attach gripper -->
   <xacro:include filename="$(find aist_scene_description)/urdf/InnerOnlyGripper.urdf.xacro" />
-  <xacro:InnerOnlyGripper prefix="a_bot_"  grippername = "gripper" parent = "a_bot_ft300_frange_link">
-    <origin xyz="0 0 0" rpy="${-pi/2} ${-0.85*pi/180} ${-0.5*pi/180}"/>
+  <xacro:InnerOnlyGripper prefix="a_bot_"
+			  grippername = "gripper"
+			  parent = "a_bot_ft300_frange_link">
+    <origin xyz="0 0 0" rpy="${-pi/2} ${-0.9*pi/180} ${-0.5*pi/180}"/>
   </xacro:InnerOnlyGripper>
   <xacro:include filename="$(find o2as_scene_description)/urdf/single_suction_gripper.urdf.xacro"/>
   <xacro:single_suction_gripper_o2as prefix="b_bot_"
   				     parent="b_bot_ft300_frange_link">
-    <origin xyz="0 0 0" rpy="0 ${0.2*pi/180} ${0.3*pi/180}"/>
+    <origin xyz="0 0 0" rpy="0 ${-0.5*pi/180} ${-0.3*pi/180}"/>
   </xacro:single_suction_gripper_o2as>
   <!-- Add virtual wall to avoid collisions-->
@@ -79,10 +81,10 @@
   <xacro:include filename="$(find o2as_scene_description)/urdf/phoxi_m_camera.urdf.xacro"/>
   <xacro:phoxi_m_camera prefix="a_" parent="o2as_ground">
-    <origin xyz="0.571555325522
-		 -0.0254263761312
-		 1.55210350714"
-	    rpy="${-146.961510137*pi/180}
-		 ${-0.588467063736*pi/180}
-		 ${83.8809430549*pi/180}"/>
+    <origin xyz="0.564327397092
+		 -0.0280911591052
+		 1.55061967739"
+	    rpy="${-150.214133529*pi/180}
+		 ${-0.641287772221*pi/180}
+		 ${86.0074821612*pi/180}"/>
   </xacro:phoxi_m_camera>
   <!-- Add RealSense camera -->

Commit message: Cleaning up.

File: aist_scene_description/urdf/pgrp_base_scene.urdf.xacro (robot description, xacro)
@@ -67,10 +67,12 @@
 			  grippername = "gripper"
 			  parent = "a_bot_ft300_frange_link">
-    <origin xyz="0 0 0" rpy="${-pi/2} ${-0.9*pi/180} ${-0.5*pi/180}"/>
+    <!-- <origin xyz="0 0 0" rpy="${-pi/2} ${-0.9*pi/180} ${-0.5*pi/180}"/> -->
+    <origin xyz="0 0 0" rpy="${-pi/2} 0 0"/>
   </xacro:InnerOnlyGripper>
   <xacro:include filename="$(find o2as_scene_description)/urdf/single_suction_gripper.urdf.xacro"/>
   <xacro:single_suction_gripper_o2as prefix="b_bot_"
   				     parent="b_bot_ft300_frange_link">
-    <origin xyz="0 0 0" rpy="0 ${-0.5*pi/180} ${-0.3*pi/180}"/>
+    <origin xyz="0 0 0" rpy="0 ${1.1*pi/180} ${-0.6*pi/180}"/>
+    <!-- <origin xyz="0 0 0" rpy="0 0 0"/> -->
   </xacro:single_suction_gripper_o2as>
   <!-- Add virtual wall to avoid collisions-->

Commit message: Fixed bug in reading bg and mask images in matlab_graspability_server.m.

File: aist_scene_description/urdf/pgrp_base_scene.urdf.xacro (robot description, xacro)
@@ -19,5 +19,5 @@
   <xacro:include filename="$(find o2as_scene_description)/urdf/o2as_box.xacro"/>
   <xacro:property name="table_w" value="0.9"/>
-  <xacro:property name="table_l" value="0.75"/>
+  <xacro:property name="table_l" value="1.8"/>
   <xacro:property name="table_h" value="0.01"/>
   <xacro:o2as_box boxname="workbox"

Commit message: check_calibration.py updated to work with move_lin.

File: aist_scene_description/urdf/pgrp_base_scene.urdf.xacro (robot description, xacro)
@@ -34,5 +34,5 @@
   <!-- robot arms -->
   <xacro:include filename="$(find o2as_scene_description)/urdf/ur5.urdf.xacro"/>
-  <xacro:ur5_robot prefix="a_bot_" joint_limited="true"
+  <xacro:ur5_robot prefix="a_bot_" joint_limited="false"
     shoulder_pan_lower_limit="${-pi}" shoulder_pan_upper_limit="${pi}"
     shoulder_lift_lower_limit="${-pi}" shoulder_lift_upper_limit="${pi}"
@@ -41,5 +41,5 @@
     wrist_2_lower_limit="${-pi}" wrist_2_upper_limit="${pi}"
     wrist_3_lower_limit="${-pi}" wrist_3_upper_limit="${pi}"/>
-  <xacro:ur5_robot prefix="b_bot_" joint_limited="true"
+  <xacro:ur5_robot prefix="b_bot_" joint_limited="false"
     shoulder_pan_lower_limit="${-pi}" shoulder_pan_upper_limit="${pi}"
     shoulder_lift_lower_limit="${-pi}" shoulder_lift_upper_limit="${pi}"
@@ -73,10 +73,9 @@
   <xacro:single_suction_gripper_o2as prefix="b_bot_"
   				     parent="b_bot_ft300_frange_link">
-    <origin xyz="0 0 0" rpy="0 ${1.1*pi/180} ${-0.6*pi/180}"/>
+    <origin xyz="0 0 0" rpy="0 ${0.3*pi/180} ${-0.3*pi/180}"/>
     <!-- <origin xyz="0 0 0" rpy="0 0 0"/> -->
   </xacro:single_suction_gripper_o2as>
   <!-- Add virtual wall to avoid collisions-->
-  <xacro:o2as_box boxname="vwall1"
-		  box_w="0.01" box_l="0.3" box_h="0.55" parent="o2as_ground">
+  <xacro:o2as_box boxname="vwall1" box_w="0.01" box_l="0.3" box_h="0.55" parent="o2as_ground">
     <origin xyz="0.45 -0.15 ${bots_z}" rpy="0 0 0"/>
   </xacro:o2as_box>
@@ -84,10 +83,10 @@
   <xacro:include filename="$(find o2as_scene_description)/urdf/phoxi_m_camera.urdf.xacro"/>
   <xacro:phoxi_m_camera prefix="a_" parent="o2as_ground">
-    <origin xyz="0.564327397092
-		 -0.0280911591052
-		 1.55061967739"
-	    rpy="${-150.214133529*pi/180}
-		 ${-0.641287772221*pi/180}
-		 ${86.0074821612*pi/180}"/>
+    <origin xyz="0.520760383355
+		 -0.00603134128121
+		 1.43707943481"
+	    rpy="${-150.73999755*pi/180}
+		 ${0.644901804876*pi/180}
+		 ${88.2535056807*pi/180}"/>
   </xacro:phoxi_m_camera>
   <!-- Add RealSense camera -->

Commit message: Cleaning up.

File: aist_scene_description/urdf/pgrp_base_scene.urdf.xacro (robot description, xacro)
@@ -73,5 +73,5 @@
   <xacro:single_suction_gripper_o2as prefix="b_bot_"
   				     parent="b_bot_ft300_frange_link">
-    <origin xyz="0 0 0" rpy="0 ${0.3*pi/180} ${-0.3*pi/180}"/>
+    <origin xyz="0 0 0" rpy="0 ${0.1*pi/180} ${-0.2*pi/180}"/>
     <!-- <origin xyz="0 0 0" rpy="0 0 0"/> -->
   </xacro:single_suction_gripper_o2as>
@@ -83,10 +83,10 @@
   <xacro:include filename="$(find o2as_scene_description)/urdf/phoxi_m_camera.urdf.xacro"/>
   <xacro:phoxi_m_camera prefix="a_" parent="o2as_ground">
-    <origin xyz="0.520760383355
-		 -0.00603134128121
-		 1.43707943481"
-	    rpy="${-150.73999755*pi/180}
-		 ${0.644901804876*pi/180}
-		 ${88.2535056807*pi/180}"/>
+    <origin xyz="0.521217687458
+		 -0.00508307933619
+		 1.43718368936"
+	    rpy="${-150.749317075*pi/180}
+		 ${0.617210923766*pi/180}
+		 ${88.4045592933*pi/180}"/>
   </xacro:phoxi_m_camera>
   <!-- Add RealSense camera -->

Commit message: Cleaning up tool_calibration.py.

File: aist_scene_description/urdf/pgrp_base_scene.urdf.xacro (robot description, xacro)
@@ -67,6 +67,6 @@
 			  grippername = "gripper"
 			  parent = "a_bot_ft300_frange_link">
-    <origin xyz="-0.004 0 0" rpy="${-pi/2} ${-1.0*pi/180} ${-0.5*pi/180}"/>
-    <!-- <origin xyz="-0.004 0 0" rpy="${-pi/2} 0 0"/> -->
+    <!-- <origin xyz="-0.004 0 0" rpy="${-pi/2} ${-1.0*pi/180} ${-0.5*pi/180}"/> -->
+    <origin xyz="-0.004 0 0" rpy="${-pi/2} 0 0"/>
   </xacro:InnerOnlyGripper>
   <xacro:include filename="$(find o2as_scene_description)/urdf/single_suction_gripper.urdf.xacro"/>

Commit message: Cleaning up tool_calibration.py again.

File: aist_scene_description/urdf/pgrp_base_scene.urdf.xacro (robot description, xacro)
@@ -67,6 +67,6 @@
 			  grippername = "gripper"
 			  parent = "a_bot_ft300_frange_link">
-    <!-- <origin xyz="-0.004 0 0" rpy="${-pi/2} ${-1.0*pi/180} ${-0.5*pi/180}"/> -->
-    <origin xyz="-0.004 0 0" rpy="${-pi/2} 0 0"/>
+    <origin xyz="-0.004 0 0" rpy="${-pi/2} ${-1.0*pi/180} ${-0.5*pi/180}"/>
+    <!-- <origin xyz="-0.004 0 0" rpy="${-pi/2} 0 0"/> -->
   </xacro:InnerOnlyGripper>
   <xacro:include filename="$(find o2as_scene_description)/urdf/single_suction_gripper.urdf.xacro"/>

Commit message: Calibrate PhoXi again.

File: aist_scene_description/urdf/pgrp_base_scene.urdf.xacro (robot description, xacro)
@@ -73,5 +73,5 @@
   <xacro:single_suction_gripper_o2as prefix="b_bot_"
   				     parent="b_bot_ft300_frange_link">
-    <origin xyz="0 0 0" rpy="0 ${0.4*pi/180} ${-1.1*pi/180}"/>
+    <origin xyz="0 0 0" rpy="0 ${0.3*pi/180} ${-1.2*pi/180}"/>
     <!-- <origin xyz="0 0 0" rpy="0 0 0"/> -->
   </xacro:single_suction_gripper_o2as>
@@ -83,10 +83,10 @@
   <xacro:include filename="$(find o2as_scene_description)/urdf/phoxi_m_camera.urdf.xacro"/>
   <xacro:phoxi_m_camera prefix="a_" parent="o2as_ground">
-    <origin xyz="0.480002181393
-		 -0.0102469021884
-		 1.40147194843"
-	    rpy="${-152.32508021*pi/180}
-		 ${-0.53545059011*pi/180}
-		 ${86.2439460292*pi/180}"/>
+    <origin xyz="0.480007829432
+		 -0.0129330709185
+		 1.40113963018"
+	    rpy="${-152.336676298*pi/180}
+		 ${-0.699529445369*pi/180}
+		 ${86.1343226364*pi/180}"/>
   </xacro:phoxi_m_camera>
   <!-- Add RealSense camera -->

Commit message: Modified handeye_calibration reference points for config pgrp. Performed handeye_calibration and saved the results in pgrp_base_scnene.

File: aist_scene_description/urdf/pgrp_base_scene.urdf.xacro (robot description, xacro)
@@ -77,5 +77,5 @@
   <xacro:single_suction_gripper_o2as prefix="b_bot_"
   				     parent="b_bot_ft300_flange_link">
-    <origin xyz="0 0 0" rpy="0 ${0.3*pi/180} ${-1.2*pi/180}"/>
+    <origin xyz="0 0 0" rpy="0 ${0.3*pi/180} ${-0.25*pi/180}"/>
     <!-- <origin xyz="0 0 0" rpy="0 0 0"/> -->
   </xacro:single_suction_gripper_o2as>
@@ -87,10 +87,10 @@
   <xacro:include filename="$(find o2as_scene_description)/urdf/phoxi_m_camera.urdf.xacro"/>
   <xacro:phoxi_m_camera prefix="a_" parent="o2as_ground">
-    <origin xyz="0.480007829432
-		 -0.0129330709185
-		 1.40113963018"
-	    rpy="${-152.336676298*pi/180}
-		 ${-0.699529445369*pi/180}
-		 ${86.1343226364*pi/180}"/>
+    <origin xyz="0.481260423417
+		 -0.0133140326572
+		 1.40237918548"
+	    rpy="${-152.303067811*pi/180}
+		 ${-1.81267714073*pi/180}
+		 ${85.5074280136*pi/180}"/>
   </xacro:phoxi_m_camera>
   <!-- Add RealSense camera -->

Commit message: Fixed bug in base.paramtuples().

File: aist_scene_description/urdf/pgrp_base_scene.urdf.xacro (robot description, xacro)
@@ -77,9 +77,10 @@
   <xacro:single_suction_gripper_o2as prefix="b_bot_"
   				     parent="b_bot_ft300_flange_link">
-    <origin xyz="0 0 0" rpy="0 ${0.3*pi/180} ${-0.25*pi/180}"/>
+    <origin xyz="0 0 0" rpy="0 ${0.25*pi/180} ${-0.3*pi/180}"/>
     <!-- <origin xyz="0 0 0" rpy="0 0 0"/> -->
   </xacro:single_suction_gripper_o2as>
   <!-- Add virtual wall to avoid collisions-->
-  <xacro:o2as_box boxname="vwall1" box_w="0.01" box_l="0.3" box_h="0.5" parent="o2as_ground">
+  <xacro:o2as_box boxname="vwall1" box_w="0.01" box_l="0.3" box_h="0.5"
+		  parent="o2as_ground">
     <origin xyz="0.45 -0.15 ${bots_z}" rpy="0 0 0"/>
   </xacro:o2as_box>
@@ -87,10 +88,10 @@
   <xacro:include filename="$(find o2as_scene_description)/urdf/phoxi_m_camera.urdf.xacro"/>
   <xacro:phoxi_m_camera prefix="a_" parent="o2as_ground">
-    <origin xyz="0.481260423417
-		 -0.0133140326572
-		 1.40237918548"
-	    rpy="${-152.303067811*pi/180}
-		 ${-1.81267714073*pi/180}
-		 ${85.5074280136*pi/180}"/>
+    <origin xyz="0.483495324929
+		 -0.0156195600384
+		 1.4037839232"
+	    rpy="${-152.261551001*pi/180}
+		 ${-1.99751517356*pi/180}
+		 ${86.5856239945*pi/180}"/>
   </xacro:phoxi_m_camera>
   <!-- Add RealSense camera -->

Commit message: Added grasp/release commands to kitting.py. Fixed release offset of part_8.

File: aist_scene_description/urdf/pgrp_base_scene.urdf.xacro (robot description, xacro)
@@ -77,5 +77,5 @@
   <xacro:single_suction_gripper_o2as prefix="b_bot_"
   				     parent="b_bot_ft300_flange_link">
-    <origin xyz="0 0 0" rpy="0 ${0.25*pi/180} ${-0.3*pi/180}"/>
+    <origin xyz="0 0 0" rpy="0 ${-0.2*pi/180} ${-0.9*pi/180}"/>
     <!-- <origin xyz="0 0 0" rpy="0 0 0"/> -->
   </xacro:single_suction_gripper_o2as>
@@ -88,10 +88,10 @@
   <xacro:include filename="$(find o2as_scene_description)/urdf/phoxi_m_camera.urdf.xacro"/>
   <xacro:phoxi_m_camera prefix="a_" parent="o2as_ground">
-    <origin xyz="0.483495324929
-		 -0.0156195600384
-		 1.4037839232"
-	    rpy="${-152.261551001*pi/180}
-		 ${-1.99751517356*pi/180}
-		 ${86.5856239945*pi/180}"/>
+    <origin xyz="0.484295583013
+		 -0.0166431117381
+		 1.40352762972"
+	    rpy="${-152.276420805*pi/180}
+		 ${-2.02008972972*pi/180}
+		 ${86.5892287041*pi/180}"/>
   </xacro:phoxi_m_camera>
   <!-- Add RealSense camera -->

Commit message: Removed uncecessary dependencies.

File: aist_scene_description/urdf/pgrp_base_scene.urdf.xacro (robot description, xacro)
@@ -77,5 +77,5 @@
   <xacro:single_suction_gripper_o2as prefix="b_bot_"
   				     parent="b_bot_ft300_flange_link">
-    <origin xyz="0 0 0" rpy="0 ${-0.2*pi/180} ${-0.9*pi/180}"/>
+    <origin xyz="0 0 0" rpy="0 ${0.2*pi/180} ${-0.4*pi/180}"/>
     <!-- <origin xyz="0 0 0" rpy="0 0 0"/> -->
   </xacro:single_suction_gripper_o2as>
