Commit message: Modified 'aist_gazebo'.

File: aist_gazebo/o2as_gazebo/urdf/aist_ar_marker.urdf.xacro (robot description, xacro)
@@ -1,5 +1,5 @@
 <?xml version="1.0" ?>
-<robot name="o2as_ar_marker" xmlns:xacro="http://www.ros.org/wiki/xacro">
-  <xacro:macro name="o2as_ar_marker" params="marker_id prefix parent *origin">
+<robot name="aist_ar_marker" xmlns:xacro="http://www.ros.org/wiki/xacro">
+  <xacro:macro name="aist_ar_marker" params="marker_id prefix parent *origin">
     <joint name="${prefix}ar_marker_joint" type="fixed">
       <parent link="${parent}" />
@@ -23,5 +23,5 @@
     </link>
     <!-- For Gazebo, material of AR marker is defined in
-         o2as_gazebo/media/material. You also need to export
+         aist_gazebo/media/material. You also need to export
          gazebo_media_path in package.xml. -->
     <gazebo reference="${prefix}ar_marker">
@@ -29,5 +29,5 @@
     </gazebo>
   </xacro:macro>
-  <xacro:macro name="o2as_ar_marker_16cm" params="marker_id prefix parent *origin">
+  <xacro:macro name="aist_ar_marker_16cm" params="marker_id prefix parent *origin">
     <joint name="${prefix}ar_marker_joint" type="fixed">
       <parent link="${parent}" />
@@ -51,5 +51,5 @@
     </link>
     <!-- For Gazebo, material of AR marker is defined in
-         o2as_gazebo/media/material. You also need to export
+         aist_gazebo/media/material. You also need to export
          gazebo_media_path in package.xml. -->
     <gazebo reference="${prefix}ar_marker">

File: aist_gazebo/o2as_gazebo/urdf/aist_ar_marker_16cm.urdf.xacro (robot description, xacro)
@@ -1,5 +1,5 @@
 <?xml version="1.0" ?>
-<robot name="o2as_ar_marker" xmlns:xacro="http://www.ros.org/wiki/xacro">
-  <xacro:macro name="o2as_ar_marker_16cm" params="marker_id prefix parent *origin">
+<robot name="aist_ar_marker" xmlns:xacro="http://www.ros.org/wiki/xacro">
+  <xacro:macro name="aist_ar_marker_16cm" params="marker_id prefix parent *origin">
     <joint name="${prefix}ar_marker_joint" type="fixed">
       <parent link="${parent}" />
@@ -23,5 +23,5 @@
     </link>
     <!-- For Gazebo, material of AR marker is defined in
-         o2as_gazebo/media/material. You also need to export
+         aist_gazebo/media/material. You also need to export
          gazebo_media_path in package.xml. -->
     <gazebo reference="${prefix}ar_marker">

File: aist_gazebo/o2as_gazebo/urdf/d_bot_camera.urdf.xacro (robot description, xacro)
@@ -4,5 +4,5 @@
     <static>true</static>
   </gazebo>
-  <xacro:include filename="$(find o2as_gazebo)/urdf/d_bot_camera.gazebo" />
+  <xacro:include filename="$(find aist_gazebo)/urdf/d_bot_camera.gazebo" />
   <xacro:include filename="$(find realsense2_camera)/urdf/_d435.urdf.xacro" />
   <link name="world" />

File: aist_scene_description/urdf/aist_base_scene.urdf.xacro (robot description, xacro)
@@ -9,6 +9,6 @@
   <!-- This is the main file defining our robot arrangement and physical environment. -->
   <!-- common stuff -->
-  <!-- <xacro:include filename="$(find ur_description)/urdf/common.gazebo.xacro" />
-  <xacro:include filename="$(find o2as_gazebo)/urdf/o2as_base_scene.gazebo" /> -->
+  <xacro:include filename="$(find ur_description)/urdf/common.gazebo.xacro" />
+  <xacro:include filename="$(find aist_gazebo)/urdf/aist_base_scene.gazebo" />
   <!-- robots -->
   <xacro:include filename="$(find o2as_scene_description)/urdf/ur5.urdf.xacro" />
@@ -58,4 +58,15 @@
   <origin xyz="0.64685382925 0.00793354972549 1.47431467674" rpy="${-144.009037015*pi/180} ${0.0354016148982*pi/180} ${85.0410662353*pi/180}"/>
   </xacro:phoxi_m_camera>
+  <xacro:include filename="$(find aist_gazebo)/urdf/aist_ar_marker.urdf.xacro"/>
+  <xacro:aist_ar_marker prefix="b_bot_"
+      parent="b_bot_single_suction_gripper_base_link"
+      marker_id="26">
+    <origin xyz="0.063 0.0 0.0215" rpy="0 0 0"/>
+  </xacro:aist_ar_marker>
+  <xacro:aist_ar_marker_16cm prefix="workspace_"
+      parent="workspace_center"
+      marker_id="32">
+    <origin xyz="0.0 0.0 0.0005" rpy="0 0 0"/>
+  </xacro:aist_ar_marker_16cm>
   <!-- I would like to remove the "world" link definition, but apparently it is necessary for Gazebo -->
   <link name="world" />
