Commit message: Added wrench frame to ft300 sensor. Confirmed that PLAN_FAILURE and PICK_FAILURE work in real bin-picking.

File: aist_ft300/urdf/ft300.urdf.xacro (robot description, xacro)
@@ -31,4 +31,10 @@
       <origin xyz="${ft300_length} 0 0" rpy="0 0 0"/>
     </joint>
+    <link name="${prefix}ft300_wrench_link"/>
+    <joint name="${prefix}ft300_wrench_joint" type="fixed">
+      <parent link="${prefix}ft300_frange_link"/>
+      <child  link="${prefix}ft300_wrench_link"/>
+      <origin xyz="0 0 0" rpy="${-pi/2} 0 ${-pi/2}"/>
+    </joint>
   </xacro:macro>
 </robot>

File: aist_scene_description/urdf/ur5e_base_scene.urdf.xacro (robot description, xacro)
@@ -68,17 +68,17 @@
     <origin xyz="0 0 0" rpy="0 0 0"/>
   </xacro:robotiq_85_gripper_with_tip_link>
-  <!-- <xacro:include filename="$(find o2as_scene_description)/urdf/InnerOnlyGripper.xacro" /> -->
-  <!-- <xacro:InnerOnlyGripper prefix="c_bot_"  grippername = "gripper" parent = "c_bot_ft300_frange_link"> -->
-  <!--   <origin xyz="0 0 0" rpy="0 ${90*pi/180} 0"/> -->
-  <!-- </xacro:InnerOnlyGripper> -->
-  <xacro:include filename="$(find o2as_scene_description)/urdf/dual_suction_gripper.urdf.xacro"/>
-  <xacro:dual_suction_gripper_o2as prefix="d_bot_"
-  				     parent="d_bot_ft300_frange_link">
-    <origin xyz="0 0 0" rpy="0 ${0.8*pi/180} ${-0.5*pi/180}"/>
-  </xacro:dual_suction_gripper_o2as>
+  <!-- <xacro:include filename="$(find o2as_scene_description)/urdf/dual_suction_gripper.urdf.xacro"/> -->
+  <!-- <xacro:dual_suction_gripper_o2as prefix="d_bot_" -->
+  <!-- 				     parent="d_bot_ft300_frange_link"> -->
+  <!--   <origin xyz="0 0 0" rpy="0 ${0.8*pi/180} ${-0.5*pi/180}"/> -->
+  <!-- </xacro:dual_suction_gripper_o2as> -->
   <!-- Add virtual wall to avoid collisions-->
   <!-- <xacro:o2as_box boxname="vwall1" box_w="0.01" box_l="0.5" box_h="0.6" parent="o2as_ground"> -->
   <!--   <origin xyz="0.50 -0.25 ${bots_z}" rpy="0 0 0"/> -->
   <!-- </xacro:o2as_box> -->
+  <xacro:robotiq_85_gripper_with_tip_link prefix="d_bot_"
+					  parent="d_bot_ft300_frange_link">
+    <origin xyz="0 0 0" rpy="0 0 0"/>
+  </xacro:robotiq_85_gripper_with_tip_link>
   <!-- Add PhoXi 3D scanner -->
   <xacro:include filename="$(find o2as_scene_description)/urdf/phoxi_m_camera.urdf.xacro"/>

Commit message: Added mesh file of FT300 force sensor. PLAN_FAILURE has been renamed to MOVE_FAILURE.

File: aist_ft300/urdf/ft300.urdf.xacro (robot description, xacro)
@@ -1,20 +1,30 @@
 <?xml version="1.0"?>
 <robot name="ft300" xmlns:xacro="http://www.ros.org/wiki/xacro">
-  <xacro:property name="ft300_length" value="0.0360"/>
+  <xacro:property name="ft300_radius" value="0.0375"/>
+  <xacro:property name="ft300_length" value="0.0375"/>
   <xacro:macro name="ft300" params="prefix parent">
     <link name="${prefix}ft300_link">
       <visual>
-        <origin xyz="${ft300_length/2} 0 0" rpy="0 ${pi/2} 0"/>
-        <geometry>
-          <cylinder length="${ft300_length}" radius="0.0375"/>
-        </geometry>
-        <material name="Black">
-          <color rgba="0.2 0.2 0.2 1.0"/>
-        </material>
+        <origin xyz="${ft300_length} 0 0" rpy="${pi} ${pi/2} 0"/>
+	<geometry>
+          <mesh filename="package://aist_ft300/meshes/ft300.stl" scale="0.001 0.001 0.001"/>
+	</geometry>
+	<material name="Black">
+	  <color rgba="0.2 0.2 0.2 1"/>
+	</material>
       </visual>
+      <!-- <visual> -->
+      <!--   <origin xyz="${ft300_length/2} 0 0" rpy="0 ${pi/2} 0"/> -->
+      <!--   <geometry> -->
+      <!--     <cylinder length="${ft300_length}" radius="0.0375"/> -->
+      <!--   </geometry> -->
+      <!--   <material name="Black"> -->
+      <!--     <color rgba="0.2 0.2 0.2 1.0"/> -->
+      <!--   </material> -->
+      <!-- </visual> -->
       <collision>
         <origin xyz="${ft300_length/2} 0 0" rpy="0 ${pi/2} 0"/>
         <geometry>
-          <cylinder length="${ft300_length}" radius="0.0375"/>
+          <cylinder length="${ft300_length}" radius="${ft300_radius}"/>
         </geometry>
       </collision>

Commit message: Changed orientation of tray2.

File: aist_ft300/urdf/ft300.urdf.xacro (robot description, xacro)
@@ -2,5 +2,5 @@
 <robot name="ft300" xmlns:xacro="http://www.ros.org/wiki/xacro">
   <xacro:property name="ft300_radius" value="0.0375"/>
-  <xacro:property name="ft300_length" value="0.0375"/>
+  <xacro:property name="ft300_length" value="0.0360"/>
   <xacro:macro name="ft300" params="prefix parent">
     <link name="${prefix}ft300_link">

File: aist_scene_description/urdf/pgrp_kitting.urdf.xacro (robot description, xacro)
@@ -106,8 +106,8 @@
   <!-- tray_2 -->
   <xacro:kitting_tray2 trayname="tray_2" parent="plate_center">
-    <origin xyz="${plate_w/2 - bin_1_length - bin_2_length - tray_width}
-		 0
+    <origin xyz="${plate_w/2 - bin_1_length - bin_2_length}
+		 ${-tray_length}
 		 0"
-	    rpy="0 0 ${-pi/2}" />
+	    rpy="0 0 ${pi/2}" />
   </xacro:kitting_tray2>
 </robot>
