Commit message: MoveGroupCommander is created in the constructor of AISTBaseRoutines.

File: o2as_realsense2_camera/urdf/_d435.urdf.xacro (robot description, xacro)
@@ -40,5 +40,5 @@
         <geometry>
           <!-- <box size="${d435_cam_width} ${d435_cam_height} ${d435_cam_depth}"/> -->
-	        <mesh filename="package://realsense2_camera/meshes/d435.dae" />
+	        <mesh filename="package://realsense2_description/meshes/d435.dae" />
         </geometry>
 	<material name="aluminum">
