Commit message: Moved URDF model of ft300 sensor from aist_ft300 to aist_ftsensor.

File: aist_ftsensor/urdf/ft300.urdf.xacro (robot description, xacro)
@@ -8,5 +8,5 @@
         <origin xyz="${ft300_length} 0 0" rpy="${pi} ${pi/2} 0"/>
 	<geometry>
-          <mesh filename="package://aist_ft300/meshes/ft300.stl" scale="0.001 0.001 0.001"/>
+          <mesh filename="package://aist_ftsensor/meshes/ft300.stl" scale="0.001 0.001 0.001"/>
 	</geometry>
 	<material name="Black">

File: aist_scene_description/urdf/aist_base_scene.urdf.xacro (robot description, xacro)
@@ -59,5 +59,5 @@
   </joint>
   <!-- Spawn and attach force sensor -->
-  <xacro:include filename="$(find aist_ft300)/urdf/ft300.urdf.xacro"/>
+  <xacro:include filename="$(find aist_ftsensor)/urdf/ft300.urdf.xacro"/>
   <xacro:ft300 prefix="a_bot_" parent="a_bot_ee_link"/>
   <xacro:ft300 prefix="b_bot_" parent="b_bot_ee_link"/>

File: aist_scene_description/urdf/pgrp_base_scene.urdf.xacro (robot description, xacro)
@@ -59,5 +59,5 @@
   </joint>
   <!-- Spawn and attach force sensor -->
-  <xacro:include filename="$(find aist_ft300)/urdf/ft300.urdf.xacro"/>
+  <xacro:include filename="$(find aist_ftsensor)/urdf/ft300.urdf.xacro"/>
   <xacro:ft300 prefix="a_bot_" parent="a_bot_ee_link"/>
   <xacro:ft300 prefix="b_bot_" parent="b_bot_ee_link"/>

Commit message: Cleaning up.

File: aist_ftsensor/urdf/ft300.urdf.xacro (robot description, xacro)
@@ -3,5 +3,5 @@
   <xacro:property name="ft300_radius" value="0.0375"/>
   <xacro:property name="ft300_length" value="0.0360"/>
-  <xacro:macro name="ft300" params="prefix parent">
+  <xacro:macro name="ft300" params="prefix parent *origin">
     <link name="${prefix}ft300_link">
       <visual>
@@ -34,14 +34,15 @@
       <parent link="${parent}"/>
       <child  link="${prefix}ft300_link"/>
+      <xacro:insert_block name="origin"/>
     </joint>
-    <link name="${prefix}ft300_frange_link"/>
-    <joint name="${prefix}ft300_frange_joint" type="fixed">
+    <link name="${prefix}ft300_flange_link"/>
+    <joint name="${prefix}ft300_flange_joint" type="fixed">
       <parent link="${prefix}ft300_link"/>
-      <child  link="${prefix}ft300_frange_link"/>
+      <child  link="${prefix}ft300_flange_link"/>
       <origin xyz="${ft300_length} 0 0" rpy="0 0 0"/>
     </joint>
     <link name="${prefix}ft300_wrench_link"/>
     <joint name="${prefix}ft300_wrench_joint" type="fixed">
-      <parent link="${prefix}ft300_frange_link"/>
+      <parent link="${prefix}ft300_flange_link"/>
       <child  link="${prefix}ft300_wrench_link"/>
       <origin xyz="0 0 0" rpy="${-pi/2} 0 ${-pi/2}"/>

File: aist_scene_description/urdf/InnerOnlyGripper.urdf.xacro (robot description, xacro)
@@ -2,73 +2,73 @@
 ">
   <xacro:macro name="InnerOnlyGripper" params="prefix grippername parent *origin">
-  <xacro:property name="mesh_file" value="package://o2as_scene_description/meshes/Assem2.STL" />
-  <link name="${prefix}${grippername}_base_link">
-    <inertial>
-      <origin rpy="0 0 0" xyz="0 0 0"/>
-      <mass value="1.0"/>
-      <inertia ixx="1.0" ixy="0" ixz="0" iyy="1.0" iyz="0" izz="1.0"/>
-    </inertial>
-    <visual>
-      <!-- <origin rpy="0 0 ${pi/2}" xyz="0 0 0"/> -->
-      <origin rpy="${pi/2} 0 ${pi/2}" xyz="0 0 0"/>
-      <geometry>
-        <mesh filename="${mesh_file}" scale="0.001 0.001 0.001"/>
-      </geometry>
+    <xacro:property name="mesh_file" value="package://o2as_scene_description/meshes/Assem2.STL" />
+    <link name="${prefix}${grippername}_base_link">
+      <inertial>
+	<origin rpy="0 0 0" xyz="0 0 0"/>
+	<mass value="1.0"/>
+	<inertia ixx="1.0" ixy="0" ixz="0" iyy="1.0" iyz="0" izz="1.0"/>
+      </inertial>
+      <visual>
+	<!-- <origin rpy="0 0 ${pi/2}" xyz="0 0 0"/> -->
+	<origin rpy="${pi/2} 0 ${pi/2}" xyz="0 0 0"/>
+	<geometry>
+          <mesh filename="${mesh_file}" scale="0.001 0.001 0.001"/>
+	</geometry>
         <material name="darkgrey">
           <color rgba="0.1 0.1 0.1 1"/>
         </material>
-    </visual>
-    <collision>
-      <origin rpy="0 0 0" xyz="0 -0.01 0.062"/>
-      <geometry>
-        <box size="0.07 0.09 0.18"/>
-      </geometry>
-    </collision>
-    <collision>
-      <origin rpy="0 0 0" xyz="0 -0.015 0.116"/>
-      <geometry>
-        <box size=".04 .05 .08"/>
-      </geometry>
-    </collision>
-    <!-- <visual>
-      <origin rpy="0 0 0" xyz="0.0 -0.015 0.062"/>
-      <geometry>
-        <box size="0.07 0.09 0.1"/>
-      </geometry>
-      <material name="green2">
-        <color rgba="0.1 0.8 0.1 0.3"/>
-      </material>
-    </visual>
-    <visual>
-      <origin rpy="0 0 0" xyz="0 -0.015 0.116"/>
-      <geometry>
-        <box size=".04 .05 .08"/>
-      </geometry>
-      <material name="cyan2">
-        <color rgba="0.3 0.5 0.5 0.3"/>
-      </material>
-    </visual> -->
-  </link>
-  <joint name="${prefix}${grippername}" type="fixed">
-    <parent link="${parent}" />
-    <child link = "${prefix}${grippername}_base_link" />
-    <xacro:insert_block name="origin"/>
-  </joint>
-  <!-- Add additional links for us to plan with.-->
-  <joint name="${prefix}${grippername}_tip_link_joint" type="fixed">
-    <parent link="${prefix}${grippername}_base_link"/>
-    <child link="${prefix}${grippername}_tip_link"/>
-    <!-- <origin rpy="0.0 ${-pi/2} 0.0" xyz="0.001 -0.008 .162"/> -->
-    <!-- <origin rpy="0 0 0" xyz="0.162 -0.008 -0.001"/> -->
-    <origin rpy="0 0 0" xyz="0.162 -0.015 -0.001"/>
-    <!-- +y is the same, +x in the new frame is +z in the parent, +z is -x in the parent? -->
-  </joint>
-  <link name="${prefix}${grippername}_tip_link"/>
-  <joint name="${prefix}${grippername}_screw_pickup_joint" type="fixed">
-    <parent link="${prefix}${grippername}_tip_link"/>
-    <child link="${prefix}${grippername}_screw_pickup"/>
-    <origin rpy="0 ${pi/2} 0" xyz="-0.032 0 -0.003"/>
-  </joint>
-  <link name="${prefix}${grippername}_screw_pickup"/>
+      </visual>
+      <collision>
+	<origin rpy="0 0 0" xyz="0 -0.01 0.062"/>
+	<geometry>
+          <box size="0.07 0.09 0.18"/>
+	</geometry>
+      </collision>
+      <collision>
+	<origin rpy="0 0 0" xyz="0 -0.015 0.116"/>
+	<geometry>
+          <box size=".04 .05 .08"/>
+	</geometry>
+      </collision>
+      <!-- <visual>
+	   <origin rpy="0 0 0" xyz="0.0 -0.015 0.062"/>
+	   <geometry>
+           <box size="0.07 0.09 0.1"/>
+	   </geometry>
+	   <material name="green2">
+           <color rgba="0.1 0.8 0.1 0.3"/>
+	   </material>
+	   </visual>
+	   <visual>
+	   <origin rpy="0 0 0" xyz="0 -0.015 0.116"/>
+	   <geometry>
+           <box size=".04 .05 .08"/>
+	   </geometry>
+	   <material name="cyan2">
+           <color rgba="0.3 0.5 0.5 0.3"/>
+	   </material>
+	   </visual> -->
+    </link>
+    <joint name="${prefix}${grippername}" type="fixed">
+      <parent link="${parent}" />
+      <child link = "${prefix}${grippername}_base_link" />
+      <xacro:insert_block name="origin"/>
+    </joint>
+    <!-- Add additional links for us to plan with.-->
+    <joint name="${prefix}${grippername}_tip_link_joint" type="fixed">
+      <parent link="${prefix}${grippername}_base_link"/>
+      <child link="${prefix}${grippername}_tip_link"/>
+      <!-- <origin rpy="0.0 ${-pi/2} 0.0" xyz="0.001 -0.008 .162"/> -->
+      <!-- <origin rpy="0 0 0" xyz="0.162 -0.008 -0.001"/> -->
+      <origin rpy="0 0 0" xyz="0.162 -0.015 -0.001"/>
+      <!-- +y is the same, +x in the new frame is +z in the parent, +z is -x in the parent? -->
+    </joint>
+    <link name="${prefix}${grippername}_tip_link"/>
+    <joint name="${prefix}${grippername}_screw_pickup_joint" type="fixed">
+      <parent link="${prefix}${grippername}_tip_link"/>
+      <child link="${prefix}${grippername}_screw_pickup"/>
+      <origin rpy="0 ${pi/2} 0" xyz="-0.032 0 -0.003"/>
+    </joint>
+    <link name="${prefix}${grippername}_screw_pickup"/>
   </xacro:macro>
 </robot>

File: aist_scene_description/urdf/aist_base_scene.urdf.xacro (robot description, xacro)
@@ -60,15 +60,19 @@
   <!-- Spawn and attach force sensor -->
   <xacro:include filename="$(find aist_ftsensor)/urdf/ft300.urdf.xacro"/>
-  <xacro:ft300 prefix="a_bot_" parent="a_bot_ee_link"/>
-  <xacro:ft300 prefix="b_bot_" parent="b_bot_ee_link"/>
+  <xacro:ft300 prefix="a_bot_" parent="a_bot_ee_link">
+    <origin xyz="0 0 0" rpy="0 0 0"/>
+  </xacro:ft300>
+  <xacro:ft300 prefix="b_bot_" parent="b_bot_ee_link">
+    <origin xyz="0 0 0" rpy="0 0 0"/>
+  </xacro:ft300>
   <!-- Spawn and attach gripper -->
   <xacro:include filename="$(find o2as_scene_description)/urdf/robotiq_85_gripper_with_tip_link.urdf.xacro"/>
   <xacro:robotiq_85_gripper_with_tip_link prefix="a_bot_"
-					  parent="a_bot_ft300_frange_link">
+					  parent="a_bot_ft300_flange_link">
     <origin xyz="0 0 0" rpy="0 0 0"/>
   </xacro:robotiq_85_gripper_with_tip_link>
   <xacro:include filename="$(find o2as_scene_description)/urdf/single_suction_gripper.urdf.xacro"/>
   <xacro:single_suction_gripper_o2as prefix="b_bot_"
-  				     parent="b_bot_ft300_frange_link">
+  				     parent="b_bot_ft300_flange_link">
     <origin xyz="0 0 0" rpy="0 ${0.4*pi/180} ${-1.1*pi/180}"/>
     <!-- <origin xyz="0 0 0" rpy="0 0 0"/> -->

File: aist_scene_description/urdf/pgrp_base_scene.urdf.xacro (robot description, xacro)
@@ -60,11 +60,15 @@
   <!-- Spawn and attach force sensor -->
   <xacro:include filename="$(find aist_ftsensor)/urdf/ft300.urdf.xacro"/>
-  <xacro:ft300 prefix="a_bot_" parent="a_bot_ee_link"/>
-  <xacro:ft300 prefix="b_bot_" parent="b_bot_ee_link"/>
+  <xacro:ft300 prefix="a_bot_" parent="a_bot_ee_link">
+    <origin xyz="0 0 0" rpy="0 0 0"/>
+  </xacro:ft300>
+  <xacro:ft300 prefix="b_bot_" parent="b_bot_ee_link">
+    <origin xyz="0 0 0" rpy="0 0 0"/>
+  </xacro:ft300>
   <!-- Spawn and attach gripper -->
   <xacro:include filename="$(find aist_scene_description)/urdf/InnerOnlyGripper.urdf.xacro" />
   <xacro:InnerOnlyGripper prefix="a_bot_"
 			  grippername = "gripper"
-			  parent = "a_bot_ft300_frange_link">
+			  parent = "a_bot_ft300_flange_link">
     <origin xyz="-0.004 0 0" rpy="${-pi/2} ${-0.2*pi/180} ${1.3*pi/180}"/>
     <!-- <origin xyz="-0.004 0 0" rpy="${-pi/2} 0 0"/> -->
@@ -72,5 +76,5 @@
   <xacro:include filename="$(find o2as_scene_description)/urdf/single_suction_gripper.urdf.xacro"/>
   <xacro:single_suction_gripper_o2as prefix="b_bot_"
-  				     parent="b_bot_ft300_frange_link">
+  				     parent="b_bot_ft300_flange_link">
     <origin xyz="0 0 0" rpy="0 ${0.3*pi/180} ${-1.2*pi/180}"/>
     <!-- <origin xyz="0 0 0" rpy="0 0 0"/> -->
