Commit message: Add AR markers to aist_description package.

File: aist_description/device/urdf/_d435.urdf.xacro (robot description, xacro)
@@ -112,4 +112,48 @@
     </joint>
     <link name="${prefix}camera_fisheye_optical_frame"/>
+    <gazebo reference="${prefix}camera_depth_frame">
+      <sensor type="depth" name="${prefix}camera">
+	<always_on>true</always_on>
+	<visualize>true</visualize>
+	<camera>
+          <horizontal_fov>1.047</horizontal_fov>
+          <image>
+            <width>640</width>
+            <height>480</height>
+            <format>R8G8B8</format>
+          </image>
+          <depth_camera>
+          </depth_camera>
+          <clip>
+            <near>0.1</near>
+            <far>100</far>
+          </clip>
+	</camera>
+	<plugin name="${prefix}cam_controller"
+		filename="libgazebo_ros_openni_kinect.so">
+          <baseline>0.2</baseline>
+          <alwaysOn>true</alwaysOn>
+          <updateRate>10.0</updateRate>
+          <cameraName>${prefix}camera</cameraName>
+          <frameName>${prefix}camera_color_optical_frame</frameName>
+          <imageTopicName>color/image_raw</imageTopicName>
+          <cameraInfoTopicName>color/camera_info</cameraInfoTopicName>
+          <depthImageTopicName>aligned_depth_to_color/image_raw</depthImageTopicName>
+          <depthImageCameraInfoTopicName>depth/camera_info</depthImageCameraInfoTopicName>
+          <pointCloudTopicName>depth/points</pointCloudTopicName>
+          <pointCloudCutoff>0.4</pointCloudCutoff>
+          <!-- <hackBaseline>0.07</hackBaseline> -->
+          <distortionK1>0.0</distortionK1>
+          <distortionK2>0.0</distortionK2>
+          <distortionK3>0.0</distortionK3>
+          <distortionT1>0.0</distortionT1>
+          <distortionT2>0.0</distortionT2>
+          <CxPrime>0.0</CxPrime>
+          <Cx>0.0</Cx>
+          <Cy>0.0</Cy>
+          <focalLength>0.0</focalLength>
+	</plugin>
+      </sensor>
+    </gazebo>
   </xacro:macro>
 </robot>

File: aist_description/scene/urdf/aist_base_scene.urdf.xacro (robot description, xacro)
@@ -11,7 +11,4 @@
   <xacro:property name="bots_z" value="0.77"/>
   <!-- This is the main file defining our robot arrangement and physical environment. -->
-  <!-- common stuff -->
-  <xacro:include filename="$(find ur_description)/urdf/common.gazebo.xacro"/>
-  <xacro:include filename="$(find aist_gazebo)/urdf/aist_base_scene.gazebo"/>
   <!-- Main workspace -->
   <!-- The surface is 0.01 m below the robot bases and the "workspace_center" frame. -->
@@ -33,4 +30,5 @@
   </joint>
   <!-- robot arms -->
+  <xacro:include filename="$(find ur_description)/urdf/common.gazebo.xacro"/>
   <xacro:include filename="$(find aist_description)/device/urdf/ur5.urdf.xacro"/>
   <xacro:ur5_robot prefix="a_bot_" joint_limited="false"
@@ -50,10 +48,10 @@
   <joint name="world_a_bot_joint" type="fixed">
     <parent link="world"/>
-    <child  link= "a_bot_base_link"/>
+    <child  link="a_bot_base_link"/>
     <origin xyz="${a_bot_x} ${a_bot_y} ${bots_z}" rpy="0 0 0"/>
   </joint>
   <joint name="world_b_bot_joint" type="fixed">
     <parent link="world"/>
-    <child  link= "b_bot_base_link"/>
+    <child  link="b_bot_base_link"/>
     <origin xyz="${b_bot_x} ${b_bot_y} ${bots_z}" rpy="0 0 ${b_bot_theta}"/>
   </joint>

File: aist_description/scene/urdf/aist_calibration.urdf.xacro (robot description, xacro)
@@ -3,19 +3,19 @@
   <xacro:include filename="$(find aist_description)/scene/urdf/aist_base_scene.urdf.xacro"/>
   <!-- Add AR markers -->
-  <xacro:include filename="$(find aist_gazebo)/urdf/aist_ar_marker.urdf.xacro"/>
-  <xacro:aist_ar_marker prefix="a_bot_"
-			parent="a_bot_robotiq_85_tip_link"
-			marker_id="26">
+  <xacro:include filename="$(find aist_description)/object/urdf/ar_markers.urdf.xacro"/>
+  <xacro:ar_marker_70_5_5 prefix="a_bot_"
+			  parent="a_bot_robotiq_85_tip_link"
+			  marker_id="26">
     <origin xyz="0.0 0.0 0.0185" rpy="0 0 0"/>
-  </xacro:aist_ar_marker>
-  <xacro:aist_ar_marker prefix="b_bot_"
-  			parent="b_bot_single_suction_gripper_base_link"
-  			marker_id="26">
+  </xacro:ar_marker_70_5_5>
+  <xacro:ar_marker_70_5_5 prefix="b_bot_"
+  			  parent="b_bot_single_suction_gripper_base_link"
+  			  marker_id="26">
     <origin xyz="0.063 0.0 0.0215" rpy="0 0 0"/>
-  </xacro:aist_ar_marker>
-  <xacro:aist_ar_marker_16cm prefix="workspace_"
-			     parent="workspace_center"
-			     marker_id="32">
+  </xacro:ar_marker_70_5_5>
+  <xacro:ar_marker_160_10_1 prefix="workspace_"
+			    parent="workspace_center"
+			    marker_id="32">
     <origin xyz="0.0 0.0 0.005" rpy="0 0 0"/>
-  </xacro:aist_ar_marker_16cm>
+  </xacro:ar_marker_160_10_1>
 </robot>

File: aist_description/scene/urdf/ceatec_base_scene.urdf.xacro (robot description, xacro)
@@ -4,5 +4,5 @@
   <!-- Fetch robot -->
   <xacro:include filename="$(find fetch_gazebo)/robots/fetch.gazebo.xacro"/>
-  <!-- CEATEC base scene -->
+  <!-- Environment of CEATEC base scene -->
   <xacro:include filename="$(find aist_description)/scene/urdf/ceatec_base_scene_environment.urdf.xacro"/>
   <!-- I would like to remove the "world" link definition, but

File: aist_description/scene/urdf/ceatec_base_scene_environment.urdf.xacro (robot description, xacro)
@@ -147,12 +147,16 @@
   </joint>
   <!-- AR markers -->
-  <xacro:include filename="$(find aist_gazebo)/urdf/ar_marker.urdf.xacro"/>
+  <xacro:include filename="$(find aist_description)/object/urdf/ar_markers.urdf.xacro"/>
   <xacro:ar_marker prefix="a_cabinet_" parent="a_cabinet_shelf1_origin"
-		   marker_id="17" size="0.1" thickness="0.001">
-    <origin xyz="${cabinet_width - 0.05} 0.05 0.001" rpy="0 0 0"/>
+		   marker_id="17" size="0.1" margin="0.005" thickness="0.001">
+    <origin xyz="${cabinet_width - size/2 - margin}
+		 ${size/2 + margin}
+		 ${thickness}"
+	    rpy="0 0 0"/>
   </xacro:ar_marker>
   <xacro:ar_marker prefix="a_table_" parent="a_table_top_origin"
-		   marker_id="26" size="0.1" thickness="0.001">
-    <origin xyz="0.05 0.05 0.001" rpy="0 0 0"/>
+		   marker_id="26" size="0.1" margin="0.005" thickness="0.001">
+    <origin xyz="${size/2 + margin} ${size/2 + margin} ${thickness}"
+	    rpy="0 0 0"/>
   </xacro:ar_marker>
   <!-- Trays -->

File: aist_description/scene/urdf/dtorobo_base_scene.urdf.xacro (robot description, xacro)
@@ -8,6 +8,4 @@
   <xacro:property name="b_torobo_y" value="0.4875"/>
   <xacro:property name="bots_z"	    value="0.785"/>
-  <!-- common stuff -->
-  <xacro:include filename="$(find aist_gazebo)/urdf/aist_base_scene.gazebo"/>
   <!-- Main workspace -->
   <!-- The surface is 0.01 m below the robot bases and the "workspace_center" frame. -->

File: aist_description/scene/urdf/mocap_base_scene.urdf.xacro (robot description, xacro)
@@ -8,7 +8,4 @@
   <xacro:property name="bots_z" value="0.77"/>
   <!-- This is the main file defining our robot arrangement and physical environment. -->
-  <!-- common stuff -->
-  <xacro:include filename="$(find ur_description)/urdf/common.gazebo.xacro"/>
-  <xacro:include filename="$(find aist_gazebo)/urdf/aist_base_scene.gazebo"/>
   <!-- Main workspace -->
   <!-- The surface is 0.01 m below the robot bases and the "workspace_center" frame. -->
@@ -26,8 +23,9 @@
   <joint name="world_to_workspace" type="fixed">
     <parent link="world"/>
-    <child link="workspace_center"/>
+    <child  link="workspace_center"/>
     <origin xyz="0 0 ${bots_z}" rpy="0 0 0"/>
   </joint>
   <!-- robot arms -->
+  <xacro:include filename="$(find ur_description)/urdf/common.gazebo.xacro"/>
   <xacro:include filename="$(find aist_description)/device/urdf/ur5e.urdf.xacro"/>
   <xacro:ur5e_robot prefix="c_bot_" joint_limited="false"
@@ -40,5 +38,5 @@
   <joint name="world_c_bot_joint" type="fixed">
     <parent link="world"/>
-    <child  link= "c_bot_base_link"/>
+    <child  link="c_bot_base_link"/>
     <origin xyz="${c_bot_x} ${c_bot_y} ${bots_z}" rpy="0 0 0"/>
   </joint>

File: aist_description/scene/urdf/pgrp_base_scene.urdf.xacro (robot description, xacro)
@@ -11,7 +11,4 @@
   <xacro:property name="bots_z" value="0.77"/>
   <!-- This is the main file defining our robot arrangement and physical environment. -->
-  <!-- common stuff -->
-  <xacro:include filename="$(find ur_description)/urdf/common.gazebo.xacro"/>
-  <xacro:include filename="$(find aist_gazebo)/urdf/aist_base_scene.gazebo"/>
   <!-- Main workspace -->
   <!-- The surface is 0.01 m below the robot bases and the "workspace_center" frame. -->
@@ -29,8 +26,9 @@
   <joint name="world_to_workspace" type="fixed">
     <parent link="world"/>
-    <child link="workspace_center"/>
+    <child  link="workspace_center"/>
     <origin xyz="0 0 ${bots_z}" rpy="0 0 0"/>
   </joint>
   <!-- robot arms -->
+  <xacro:include filename="$(find ur_description)/urdf/common.gazebo.xacro"/>
   <xacro:include filename="$(find aist_description)/device/urdf/ur5.urdf.xacro"/>
   <xacro:ur5_robot prefix="a_bot_" joint_limited="false"
@@ -69,6 +67,6 @@
   <xacro:include filename="$(find o2as_precision_gripper)/urdf/precision_gripper.urdf.xacro" />
   <xacro:precision_gripper prefix="a_bot_"
-			   grippername = "gripper"
-			   parent = "a_bot_ft300_flange_link">
+			   grippername="gripper"
+			   parent="a_bot_ft300_flange_link">
     <origin xyz="-0.004 0 0" rpy="${-pi/2} ${-0.2*pi/180} ${1.3*pi/180}"/>
     <!-- <origin xyz="-0.004 0 0" rpy="${-pi/2} 0 0"/> -->

File: aist_description/scene/urdf/pgrp_calibration.urdf.xacro (robot description, xacro)
@@ -3,19 +3,19 @@
   <xacro:include filename="$(find aist_description)/scene/urdf/pgrp_base_scene.urdf.xacro"/>
   <!-- Add AR markers -->
-  <xacro:include filename="$(find aist_gazebo)/urdf/aist_ar_marker.urdf.xacro"/>
-  <xacro:aist_ar_marker prefix="b_bot_"
-  			parent="b_bot_single_suction_gripper_base_link"
-  			marker_id="26">
+  <xacro:include filename="$(find aist_description)/object/urdf/ar_markers.urdf.xacro"/>
+  <xacro:ar_marker_70_5_5 prefix="a_bot_"
+  			  parent="a_bot_gripper_base_link"
+  			  marker_id="26">
+    <origin xyz="0.08 -0.065 0" rpy="${pi/2} 0 0"/>
+  </xacro:ar_marker_70_5_5>
+  <xacro:ar_marker_70_5_5 prefix="b_bot_"
+  			  parent="b_bot_single_suction_gripper_base_link"
+  			  marker_id="26">
     <origin xyz="0.063 0.0 0.0215" rpy="0 0 0"/>
-  </xacro:aist_ar_marker>
-  <xacro:aist_ar_marker prefix="a_bot_"
-  			parent="a_bot_gripper_base_link"
-  			marker_id="26">
-    <origin xyz="0.08 -0.065 0" rpy="${pi/2} 0 0"/>
-  </xacro:aist_ar_marker>
-  <xacro:aist_ar_marker_16cm prefix="workspace_"
-			     parent="workspace_center"
-			     marker_id="32">
+  </xacro:ar_marker_70_5_5>
+  <xacro:ar_marker_160_10_1 prefix="workspace_"
+			    parent="workspace_center"
+			    marker_id="32">
     <origin xyz="0.0 0.0 0.005" rpy="0 0 0"/>
-  </xacro:aist_ar_marker_16cm>
+  </xacro:ar_marker_160_10_1>
 </robot>

File: aist_description/scene/urdf/ur5e_base_scene.urdf.xacro (robot description, xacro)
@@ -1,9 +1,7 @@
 <?xml version="1.0"?>
-<robot xmlns:xacro="http://www.ros.org/wiki/xacro"
-        name="ur5e_base_scene" >
+<robot xmlns:xacro="http://www.ros.org/wiki/xacro" name="ur5e_base_scene" >
   <!-- Calibration help: If the robot is not moving far enough to the calibration point, increase these distances -->
   <xacro:property name="c_bot_x" value="0"/>
   <xacro:property name="c_bot_y" value="-0.4875"/>
-  <!-- <xacro:property name="c_bot_theta" value="${pi}"/> -->
   <xacro:property name="d_bot_x" value="0"/>
   <xacro:property name="d_bot_y" value="0.4875"/>
@@ -11,7 +9,4 @@
   <xacro:property name="bots_z" value="0.77"/>
   <!-- This is the main file defining our robot arrangement and physical environment. -->
-  <!-- common stuff -->
-  <xacro:include filename="$(find ur_description)/urdf/common.gazebo.xacro"/>
-  <xacro:include filename="$(find aist_gazebo)/urdf/aist_base_scene.gazebo"/>
   <!-- Main workspace -->
   <!-- The surface is 0.01 m below the robot bases and the "workspace_center" frame. -->
@@ -33,4 +28,5 @@
   </joint>
   <!-- robot arms -->
+  <xacro:include filename="$(find ur_description)/urdf/common.gazebo.xacro"/>
   <xacro:include filename="$(find aist_description)/device/urdf/ur5e.urdf.xacro"/>
   <xacro:ur5e_robot prefix="c_bot_" joint_limited="false"

File: aist_description/scene/urdf/ur5e_calibration.urdf.xacro (robot description, xacro)
@@ -3,19 +3,14 @@
   <xacro:include filename="$(find aist_description)/scene/urdf/ur5e_base_scene.urdf.xacro"/>
   <!-- Add AR markers -->
-  <xacro:include filename="$(find aist_gazebo)/urdf/aist_ar_marker.urdf.xacro"/>
-  <xacro:aist_ar_marker prefix="c_bot_"
-			parent="c_bot_robotiq_85_tip_link"
-			marker_id="26">
+  <xacro:include filename="$(find aist_description)/object/urdf/ar_markers.urdf.xacro"/>
+  <xacro:ar_marker_70_5_5 prefix="c_bot_"
+			  parent="c_bot_robotiq_85_tip_link"
+			  marker_id="26">
     <origin xyz="0.0 0.0 0.0185" rpy="0 0 0"/>
-  </xacro:aist_ar_marker>
-  <xacro:aist_ar_marker prefix="d_bot_"
-  			parent="d_bot_dual_suction_gripper_base_link"
-  			marker_id="26">
+  </xacro:ar_marker_70_5_5>
+  <xacro:ar_marker_70_5_5 prefix="d_bot_"
+  			  parent="d_bot_dual_suction_gripper_base_link"
+  			  marker_id="26">
     <origin xyz="0.063 0.0 0.0215" rpy="0 0 0"/>
-  </xacro:aist_ar_marker>
-  <!-- <xacro:aist_ar_marker_16cm prefix="workspace_" -->
-  <!-- 			     parent="workspace_center" -->
-  <!-- 			     marker_id="32"> -->
-  <!--   <origin xyz="0.0 0.0 0.005" rpy="0 0 0"/> -->
-  <!-- </xacro:aist_ar_marker_16cm> -->
+  </xacro:ar_marker_70_5_5>
 </robot>
