Commit message: Confirmed that kitting works under aist_descriptions.

File: aist_description/device/urdf/_d435.urdf.xacro (robot description, xacro)
@@ -6,5 +6,5 @@
 aluminum peripherial evaluation case.
 -->
-<robot name="sensor_d435" xmlns:xacro="http://ros.org/wiki/xacro">
+<robot name="sensor_d435" xmlns:xacro="http://wiki.ros.org/xacro">
   <xacro:macro name="sensor_d435" params="prefix parent *origin">
     <xacro:property name="M_PI" value="3.1415926535897931" />

File: aist_description/device/urdf/_r410.urdf.xacro (robot description, xacro)
@@ -6,5 +6,5 @@
 aluminum peripherial evalution case.
 -->
-<robot name="sensor_r410" xmlns:xacro="http://ros.org/wiki/xacro">
+<robot name="sensor_r410" xmlns:xacro="http://wiki.ros.org/xacro">
   <xacro:property name="M_PI" value="3.1415926535897931" />
   <!-- The following values are approximate, and the camera node

File: aist_description/device/urdf/_r430.urdf.xacro (robot description, xacro)
@@ -6,5 +6,5 @@
 aluminum peripherial evaluation case.
 -->
-<robot name="sensor_r430" xmlns:xacro="http://ros.org/wiki/xacro">
+<robot name="sensor_r430" xmlns:xacro="http://wiki.ros.org/xacro">
   <xacro:property name="M_PI" value="3.1415926535897931" />
   <!-- The following values are approximate, and the camera node

File: aist_description/device/urdf/dual_suction_gripper.urdf.xacro (robot description, xacro)
@@ -1,5 +1,5 @@
 <?xml version="1.0"?>
 <robot name="dual_suction_gripper"
-       xmlns:xacro="http://ros.org/wiki/xacro">
+       xmlns:xacro="http://wiki.ros.org/xacro">
   <xacro:macro name="dual_suction_gripper"
 	       params="prefix parent *origin">

File: aist_description/device/urdf/robotiq_85_gripper_with_tip_link.urdf.xacro (robot description, xacro)
@@ -3,5 +3,5 @@
 <!-- The position of the TF frame has not been measured at all and needs to be calibrated. -->
 <robot name="robotiq_85_gripper_with_tip_link"
-       xmlns:xacro="http://www.ros.org/wiki/xacro">
+       xmlns:xacro="http://wiki.ros.org/xacro">
   <xacro:macro name="robotiq_85_gripper_with_tip_link"
 	       params="prefix parent *origin">

File: aist_description/device/urdf/robotiq_hande_with_tip_link.urdf.xacro (robot description, xacro)
@@ -3,5 +3,5 @@
 <!-- The position of the TF frame has not been measured at all and needs to be calibrated. -->
 <robot name="robotiq_hande_with_tip_link"
-       xmlns:xacro="http://www.ros.org/wiki/xacro">
+       xmlns:xacro="http://wiki.ros.org/xacro">
   <xacro:macro name="robotiq_hande_with_tip_link"
 	       params="prefix parent *origin">

File: aist_description/device/urdf/single_suction_gripper.urdf.xacro (robot description, xacro)
@@ -1,5 +1,5 @@
 <?xml version="1.0"?>
 <robot name="single_suction_gripper"
-       xmlns:xacro="http://ros.org/wiki/xacro">
+       xmlns:xacro="http://wiki.ros.org/xacro">
   <xacro:macro name="single_suction_gripper"
 	       params="prefix parent *origin">

File: aist_description/device/urdf/torobo_arm.urdf.xacro (robot description, xacro)
@@ -1,4 +1,4 @@
 <?xml version="1.0"?>
-<robot xmlns:xacro="http://ros.org/wiki/xacro">
+<robot xmlns:xacro="http://wiki.ros.org/xacro">
   <xacro:property name="M_PI" value="3.1415926535897931"/>
   <!-- =============== Load Dependencies =============== -->

File: aist_description/device/urdf/torobo_gripper.urdf.xacro (robot description, xacro)
@@ -1,4 +1,4 @@
 <?xml version="1.0"?>
-<robot xmlns:xacro="http://ros.org/wiki/xacro">
+<robot xmlns:xacro="http://wiki.ros.org/xacro">
   <xacro:property name="M_PI" value="3.1415926535897931"/>
   <xacro:include filename="$(find torobo_resources

File: aist_description/device/urdf/ur10.urdf.xacro (robot description, xacro)
@@ -1,4 +1,4 @@
 <?xml version="1.0"?>
-<robot xmlns:xacro="http://ros.org/wiki/xacro">
+<robot xmlns:xacro="http://wiki.ros.org/xacro">
 <!--
   Author: Kelsey Hawkins

File: aist_description/device/urdf/ur3.urdf.xacro (robot description, xacro)
@@ -1,4 +1,4 @@
 <?xml version="1.0"?>
-<robot xmlns:xacro="http://ros.org/wiki/xacro">
+<robot xmlns:xacro="http://wiki.ros.org/xacro">
 <!--
   Author: Felix Messmer

File: aist_description/device/urdf/ur5.urdf.xacro (robot description, xacro)
@@ -1,4 +1,4 @@
 <?xml version="1.0"?>
-<robot xmlns:xacro="http://ros.org/wiki/xacro">
+<robot xmlns:xacro="http://wiki.ros.org/xacro">
   <xacro:include filename="$(find ur_description)/urdf/ur.transmission.xacro" />
   <xacro:include filename="$(find ur_description)/urdf/ur.gazebo.xacro" />

File: aist_description/device/urdf/ur5e.urdf.xacro (robot description, xacro)
@@ -1,4 +1,4 @@
 <?xml version="1.0"?>
-<robot xmlns:xacro="http://ros.org/wiki/xacro">
+<robot xmlns:xacro="http://wiki.ros.org/xacro">
   <xacro:include filename="$(find ur_e_description)/urdf/ur.transmission.xacro" />
   <xacro:include filename="$(find ur_e_description)/urdf/ur.gazebo.xacro" />

File: aist_description/object/urdf/aist_box.urdf.xacro (robot description, xacro)
@@ -1,4 +1,4 @@
 <?xml version="1.0"?>
-<robot xmlns:xacro="http://www.ros.org/wiki/xacro">
+<robot xmlns:xacro="http://wiki.ros.org/xacro">
   <xacro:macro name="aist_box"
 	       params="name width length height parent *origin">
@@ -12,5 +12,5 @@
         </geometry>
         <material name="Grey">
-          <color rgba="1.0 1.0 1.0 1.0"/>
+          <color rgba="0.7 0.7 0.7 1.0"/>
         </material>
       </visual>
@@ -23,5 +23,5 @@
       <!-- This is required for Gazebo. -->
       <inertial>
-        <mass value="1.0" />
+        <mass value="1.0"/>
         <!-- <origin xyz="${width/2} ${length} ${height/2}" rpy="0 0 0"/> -->
         <inertia ixx="0.0" ixy="0.0" ixz="0.0" iyy="0.0" iyz="0.0" izz="0.0"/>
@@ -29,9 +29,9 @@
     </link>
     <gazebo reference="${name}">
-      <material>Gazebo/White</material>
+      <material>Gazebo/Grey</material>
     </gazebo>
     <joint name="${name}" type="fixed">
-      <parent link="${parent}" />
-      <child link = "${name}" />
+      <parent link="${parent}"/>
+      <child  link="${name}"/>
       <xacro:insert_block name="origin"/>
     </joint>

File: aist_description/object/urdf/ar_markers.urdf.xacro (robot description, xacro)
@@ -1,4 +1,4 @@
 <?xml version="1.0" ?>
-<robot name="ar_marker" xmlns:xacro="http://www.ros.org/wiki/xacro">
+<robot name="ar_marker" xmlns:xacro="http://wiki.ros.org/xacro">
   <xacro:macro name="ar_marker"
 	       params="prefix parent marker_id size margin thickness *origin">
@@ -26,28 +26,28 @@
          gazebo_media_path in package.xml. -->
     <gazebo reference="${prefix}ar_marker">
-      <material>Aruco/marker-${marker_id}-${1000*size}-${1000*margin}</material>
+      <material>Aruco/marker-${marker_id}-${int(1000*size)}-${int(1000*margin)}</material>
     </gazebo>
   </xacro:macro>
-  <xacro:macro name="ar_marker_70_5_5"
-	       params="prefix parent marker_id *origin">
+  <xacro:macro name="ar_marker_70_5"
+	       params="prefix parent marker_id thickness *origin">
     <xacro:ar_marker prefix="${prefix}" parent="${parent}"
 		     marker_id="${marker_id}" size="0.07"
-		     margin="0.005" thickness="0.005">
+		     margin="0.005" thickness="${thickness}">
       <xacro:insert_block name="origin"/>
     </xacro:ar_marker>
   </xacro:macro>
-  <xacro:macro name="ar_marker_80_10_5"
-	       params="prefix parent marker_id *origin">
+  <xacro:macro name="ar_marker_80_10"
+	       params="prefix parent marker_id thickness *origin">
     <xacro:ar_marker prefix="${prefix}" parent="${parent}"
 		     marker_id="${marker_id}" size="0.08"
-		     margin="0.01" thickness="0.005">
+		     margin="0.01" thickness="${thickness}">
       <xacro:insert_block name="origin"/>
     </xacro:ar_marker>
   </xacro:macro>
-  <xacro:macro name="ar_marker_160_10_1"
-	       params="prefix parent marker_id *origin">
+  <xacro:macro name="ar_marker_160_10"
+	       params="prefix parent marker_id thickness *origin">
     <xacro:ar_marker prefix="${prefix}" parent="${parent}"
 		     marker_id="${marker_id}" size="0.16"
-		     margin="0.01" thickness="0.001">
+		     margin="0.01" thickness="${thickness}">
       <xacro:insert_block name="origin"/>
     </xacro:ar_marker>

File: aist_description/object/urdf/cabinet.urdf.xacro (robot description, xacro)
@@ -1,5 +1,4 @@
 <?xml version="1.0" ?>
-<robot xmlns:xacro="http://ros.org/wiki/xacro"
-       name="cabinet">
+<robot xmlns:xacro="http://wiki.ros.org/xacro" name="cabinet">
   <xacro:include filename="$(find aist_description)/object/urdf/aist_box.urdf.xacro"/>
   <xacro:macro name="cabinet"

File: aist_description/object/urdf/table.urdf.xacro (robot description, xacro)
@@ -1,5 +1,4 @@
 <?xml version="1.0" ?>
-<robot xmlns:xacro="http://ros.org/wiki/xacro"
-       name="table">
+<robot xmlns:xacro="http://wiki.ros.org/xacro" name="table">
   <xacro:include filename="$(find aist_description)/object/urdf/aist_box.urdf.xacro"/>
   <xacro:macro name="table"

File: aist_description/object/urdf/tray.urdf.xacro (robot description, xacro)
@@ -1,5 +1,4 @@
 <?xml version="1.0" ?>
-<robot xmlns:xacro="http://ros.org/wiki/xacro"
-       name="table">
+<robot xmlns:xacro="http://wiki.ros.org/xacro" name="table">
   <xacro:include filename="$(find aist_description)/object/urdf/aist_box.urdf.xacro"/>
   <xacro:macro name="tray"

File: aist_description/scene/urdf/aist_base_scene.urdf.xacro (robot description, xacro)
@@ -1,4 +1,4 @@
 <?xml version="1.0"?>
-<robot xmlns:xacro="http://www.ros.org/wiki/xacro"
+<robot xmlns:xacro="http://wiki.ros.org/xacro"
         name="aist_base_scene" >
   <!-- Calibration help: If the robot is not moving far enough to the calibration point, increase these distances -->
@@ -13,17 +13,17 @@
   <!-- Main workspace -->
   <!-- The surface is 0.01 m below the robot bases and the "workspace_center" frame. -->
-  <link name="world"/>
-  <xacro:include filename="$(find aist_description)/object/urdf/aist_box.xacro"/>
+  <link name="ground"/>
+  <xacro:include filename="$(find aist_description)/object/urdf/aist_box.urdf.xacro"/>
   <xacro:property name="table_w" value="0.9"/>
   <xacro:property name="table_l" value="0.75"/>
   <xacro:property name="table_h" value="0.01"/>
-  <xacro:aist_box boxname="workbox"
-		  box_w="${table_w}" box_l="${table_l}" box_h="${table_h}"
-		  parent="world">
+  <xacro:aist_box name="workbox"
+		  width="${table_w}" length="${table_l}" height="${table_h}"
+		  parent="ground">
     <origin xyz="${-table_w/2} ${-table_l/2} ${bots_z - table_h}" rpy="0 0 0"/>
   </xacro:aist_box>
   <link name="workspace_center"/>
-  <joint name="world_to_workspace" type="fixed">
-    <parent link="world"/>
+  <joint name="ground_to_workspace" type="fixed">
+    <parent link="ground"/>
     <child link="workspace_center"/>
     <origin xyz="0 0 ${bots_z}" rpy="0 0 0"/>
@@ -46,11 +46,11 @@
     wrist_2_lower_limit="${-pi}" wrist_2_upper_limit="${pi}"
     wrist_3_lower_limit="${-pi}" wrist_3_upper_limit="${pi}"/>
-  <joint name="world_a_bot_joint" type="fixed">
-    <parent link="world"/>
+  <joint name="ground_a_bot_joint" type="fixed">
+    <parent link="ground"/>
     <child  link="a_bot_base_link"/>
     <origin xyz="${a_bot_x} ${a_bot_y} ${bots_z}" rpy="0 0 0"/>
   </joint>
-  <joint name="world_b_bot_joint" type="fixed">
-    <parent link="world"/>
+  <joint name="ground_b_bot_joint" type="fixed">
+    <parent link="ground"/>
     <child  link="b_bot_base_link"/>
     <origin xyz="${b_bot_x} ${b_bot_y} ${bots_z}" rpy="0 0 ${b_bot_theta}"/>
@@ -76,11 +76,7 @@
     <!-- <origin xyz="0 0 0" rpy="0 0 0"/> -->
   </xacro:single_suction_gripper>
-  <!-- Add virtual wall to avoid collisions-->
-  <!-- <xacro:aist_box boxname="vwall1" box_w="0.01" box_l="0.5" box_h="0.6" parent="world"> -->
-  <!--   <origin xyz="0.50 -0.25 ${bots_z}" rpy="0 0 0"/> -->
-  <!-- </xacro:aist_box> -->
   <!-- Add PhoXi 3D scanner -->
   <xacro:include filename="$(find o2as_phoxi_camera)/urdf/phoxi_m_camera.urdf.xacro"/>
-  <xacro:phoxi_m_camera prefix="a_" parent="world">
+  <xacro:phoxi_m_camera prefix="a_" parent="ground">
     <origin xyz="0.480002181393
 		 -0.0102469021884
@@ -90,3 +86,10 @@
 		 ${86.2439460292*pi/180}"/>
   </xacro:phoxi_m_camera>
+  <!-- I would like to remove the "world" link definition, but apparently it is necessary for Gazebo -->
+  <link name="world"/>
+  <joint name="world_ground_joint" type="fixed">
+    <parent link="world"/>
+    <child  link="ground"/>
+    <origin xyz="0 0 0" rpy="0 0 0"/>
+  </joint>
 </robot>

File: aist_description/scene/urdf/aist_calibration.urdf.xacro (robot description, xacro)
@@ -4,18 +4,21 @@
   <!-- Add AR markers -->
   <xacro:include filename="$(find aist_description)/object/urdf/ar_markers.urdf.xacro"/>
-  <xacro:ar_marker_70_5_5 prefix="a_bot_"
-			  parent="a_bot_robotiq_85_tip_link"
-			  marker_id="26">
+  <xacro:ar_marker_70_5 prefix="a_bot_"
+			parent="a_bot_robotiq_85_tip_link"
+			marker_id="26"
+			thickness="0.005">
     <origin xyz="0.0 0.0 0.0185" rpy="0 0 0"/>
-  </xacro:ar_marker_70_5_5>
-  <xacro:ar_marker_70_5_5 prefix="b_bot_"
-  			  parent="b_bot_single_suction_gripper_base_link"
-  			  marker_id="26">
+  </xacro:ar_marker_70_5>
+  <xacro:ar_marker_70_5 prefix="b_bot_"
+  			parent="b_bot_single_suction_gripper_base_link"
+  			marker_id="26"
+			thickness="0.005">
     <origin xyz="0.063 0.0 0.0215" rpy="0 0 0"/>
-  </xacro:ar_marker_70_5_5>
-  <xacro:ar_marker_160_10_1 prefix="workspace_"
-			    parent="workspace_center"
-			    marker_id="32">
-    <origin xyz="0.0 0.0 0.005" rpy="0 0 0"/>
-  </xacro:ar_marker_160_10_1>
+  </xacro:ar_marker_70_5>
+  <xacro:ar_marker_160_10 prefix="workspace_"
+			  parent="workspace_center"
+			  marker_id="32"
+			  thickness="0.001">
+    <origin xyz="0.0 0.0 0.0005" rpy="0 0 0"/>
+  </xacro:ar_marker_160_10>
 </robot>
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