Commit message: Moved WRC-related urdf and meshes to independent subdiretories.

File: aist_description/scene/urdf/pgrp_kitting.urdf.xacro (robot description, xacro)
@@ -21,6 +21,6 @@
     <origin xyz="${plate_w/2} ${plate_l/2} ${plate_h}" rpy="0 0 0"/>
   </joint>
-  <xacro:include filename="$(find aist_description)/object/urdf/kitting_bins.urdf.xacro"/>
-  <xacro:include filename="$(find aist_description)/object/urdf/kitting_trays.urdf.xacro"/>
+  <xacro:include filename="$(find aist_description)/wrc/urdf/kitting_bins.urdf.xacro"/>
+  <xacro:include filename="$(find aist_description)/wrc/urdf/kitting_trays.urdf.xacro"/>
   <!-- bin_1_definition -->
   <xacro:property name="bin_1_width"		value="0.125"/>

File: aist_description/wrc/urdf/kitting_bins.urdf.xacro (robot description, xacro)
@@ -5,7 +5,7 @@
 	       params="binname parent filename z_origin_offset *origin">
     <xacro:property name="mesh_file"
-		    value="package://aist_description/object/meshes/${filename}.stl"/>
+		    value="package://aist_description/wrc/meshes/${filename}.stl"/>
     <xacro:property name="mesh_file_col"
-		    value="package://aist_description/object/meshes/${filename}.vhacd.dae"/>
+		    value="package://aist_description/wrc/meshes/${filename}.vhacd.dae"/>
     <link name="${binname}">
       <inertial>

File: aist_description/wrc/urdf/kitting_trays.urdf.xacro (robot description, xacro)
@@ -9,6 +9,6 @@
   <!-- ========== The basic tray, without partitions -->
   <xacro:macro name="kitting_tray" params="trayname parent *origin">
-    <xacro:property name="mesh_file" value="package://aist_description/object/meshes/tray_PZ-0006-B.stl" />
-    <xacro:property name="mesh_file_col" value="package://aist_description/object/meshes/tray_PZ-0006-B.vhacd.dae" />
+    <xacro:property name="mesh_file" value="package://aist_description/wrc/meshes/tray_PZ-0006-B.stl" />
+    <xacro:property name="mesh_file_col" value="package://aist_description/wrc/meshes/tray_PZ-0006-B.vhacd.dae" />
     <link name="${trayname}">
       <inertial>
@@ -48,5 +48,5 @@
 	<xacro:insert_block name="origin"/>
 	<geometry>
-          <mesh filename="package://aist_description/object/meshes/${contents}.stl" scale="0.001 0.001 0.001" />
+          <mesh filename="package://aist_description/wrc/meshes/${contents}.stl" scale="0.001 0.001 0.001" />
 	</geometry>
 	<material name="white">
@@ -57,5 +57,5 @@
         <xacro:insert_block name="origin"/>
         <geometry>
-          <mesh filename="package://aist_description/object/meshes/${contents}.stl" scale="0.001 0.001 0.001" />
+          <mesh filename="package://aist_description/wrc/meshes/${contents}.stl" scale="0.001 0.001 0.001" />
         </geometry>
       </collision>
