Commit message: Changed fix direction of the precision gripper.

File: aist_description/scene/urdf/pgrp_base_scene.urdf.xacro (robot description, xacro)
@@ -68,5 +68,5 @@
 			   grippername="gripper"
 			   parent="a_bot_ft300_flange_link">
-    <origin xyz="-0.004 0 0" rpy="${-pi/2} ${-0.2*pi/180} ${1.3*pi/180}"/>
+    <origin xyz="0 -0.004 0" rpy="0 ${0.4*pi/180} ${1.3*pi/180}"/>
     <!-- <origin xyz="-0.004 0 0" rpy="${-pi/2} 0 0"/> -->
   </xacro:precision_gripper>
@@ -74,5 +74,5 @@
   <xacro:single_suction_gripper prefix="b_bot_"
   				parent="b_bot_ft300_flange_link">
-    <origin xyz="0 0 0" rpy="0 ${0.4*pi/180} ${-0.4*pi/180}"/>
+    <origin xyz="0 0 0" rpy="0 ${0.5*pi/180} ${-0.5*pi/180}"/>
     <!-- <origin xyz="0 0 0" rpy="0 0 0"/> -->
   </xacro:single_suction_gripper>
@@ -85,10 +85,10 @@
   <xacro:include filename="$(find o2as_phoxi_camera)/urdf/phoxi_m_camera.urdf.xacro"/>
   <xacro:phoxi_m_camera prefix="a_" parent="ground">
-    <origin xyz="0.484129483132
-		 -0.0151601080731
-		 1.40426350958"
-	    rpy="${-152.311809234*pi/180}
-		 ${-1.94191632711*pi/180}
-		 ${86.6469459386*pi/180}"/>
+    <origin xyz="0.483504569548
+		 -0.0136152151543
+		 1.40415528784"
+	    rpy="${-152.318075493*pi/180}
+		 ${-1.92295891376*pi/180}
+		 ${86.8018873041*pi/180}"/>
   </xacro:phoxi_m_camera>
   <!-- Add RealSense camera -->

File: aist_description/scene/urdf/pgrp_calibration.urdf.xacro (robot description, xacro)
@@ -8,5 +8,5 @@
   			marker_id="26"
 			thickness="0.005">
-    <origin xyz="0.08 -0.065 0" rpy="${pi/2} 0 0"/>
+    <origin xyz="0.08 0 0.02" rpy="0 0 0"/>
   </xacro:ar_marker_70_5>
   <xacro:ar_marker_70_5 prefix="b_bot_"

File: o2as_precision_gripper/urdf/precision_gripper.urdf.xacro (robot description, xacro)
@@ -12,5 +12,5 @@
       <visual>
 	<!-- <origin rpy="0 0 ${pi/2}" xyz="0 0 0"/> -->
-	<origin rpy="${pi/2} 0 ${pi/2}" xyz="0 0 0"/>
+	<origin rpy="${-pi/2} 0 ${-pi/2}" xyz="0 0 0"/>
 	<geometry>
           <mesh filename="${mesh_file}" scale="0.001 0.001 0.001"/>

Commit message: Changed calibration points for a_bot_camera.

File: aist_description/scene/urdf/pgrp_base_scene.urdf.xacro (robot description, xacro)
@@ -95,5 +95,10 @@
   <xacro:include filename="$(find aist_description)/device/urdf/_d435.urdf.xacro" />
   <xacro:sensor_d435 prefix="a_bot_" parent="a_bot_wrist_2_link">
-    <origin xyz="0.0 -0.06 0.20" rpy="${0*pi/180} 0.0 ${pi/2}" />
+    <origin xyz="0.0136772228487
+		 -0.0680299757021
+		 0.198556563348"
+	    rpy="${-1.97302363932*pi/180}
+		 ${10.5114862531*pi/180}
+		 ${94.8091668854*pi/180}"/>
   </xacro:sensor_d435>
   <!-- I would like to remove the "world" link definition, but apparently it is necessary for Gazebo -->

Commit message: Fixed frame definition of the precision gripper.

File: aist_description/scene/urdf/pgrp_base_scene.urdf.xacro (robot description, xacro)
@@ -68,5 +68,5 @@
 			   grippername="gripper"
 			   parent="a_bot_ft300_flange_link">
-    <origin xyz="0 -0.004 0" rpy="0 ${0.4*pi/180} ${1.3*pi/180}"/>
+    <origin xyz="-0.005 0 0" rpy="0 ${0.4*pi/180} ${0.5*pi/180}"/>
     <!-- <origin xyz="-0.004 0 0" rpy="${-pi/2} 0 0"/> -->
   </xacro:precision_gripper>

File: o2as_precision_gripper/urdf/precision_gripper.urdf.xacro (robot description, xacro)
@@ -62,5 +62,5 @@
       <!-- <origin rpy="0.0 ${-pi/2} 0.0" xyz="0.001 -0.008 .162"/> -->
       <!-- <origin rpy="0 0 0" xyz="0.162 -0.008 -0.001"/> -->
-      <origin rpy="0 0 0" xyz="0.162 -0.015 -0.001"/>
+      <origin rpy="0 0 0" xyz="0.160 0.015 0.000"/>
       <!-- +y is the same, +x in the new frame is +z in the parent, +z is -x in the parent? -->
     </joint>
@@ -69,5 +69,6 @@
       <parent link="${prefix}${grippername}_tip_link"/>
       <child  link="${prefix}${grippername}_screw_pickup"/>
-      <origin rpy="0 ${pi/2} 0" xyz="-0.032 0 -0.003"/>
+      <!-- <origin rpy="0 ${pi/2} 0" xyz="-0.032 0 -0.003"/> -->
+      <origin rpy="0 0 0" xyz="-0.032 0 -0.003"/>
     </joint>
     <link name="${prefix}${grippername}_screw_pickup"/>

Commit message: Added Realsense SR305 support. Fixed tip_link of precision gripper. Fixed orientation of the marker frame when detected without depth image.

File: aist_description/scene/urdf/pgrp_base_scene.urdf.xacro (robot description, xacro)
@@ -74,5 +74,5 @@
   <xacro:single_suction_gripper prefix="b_bot_"
   				parent="b_bot_ft300_flange_link">
-    <origin xyz="0 0 0" rpy="0 ${0.5*pi/180} ${-0.5*pi/180}"/>
+    <origin xyz="0 0 0" rpy="0 ${0.9*pi/180} ${0.4*pi/180}"/>
     <!-- <origin xyz="0 0 0" rpy="0 0 0"/> -->
   </xacro:single_suction_gripper>
@@ -93,13 +93,13 @@
   </xacro:phoxi_m_camera>
   <!-- Add RealSense camera -->
-  <xacro:include filename="$(find aist_description)/device/urdf/_d435.urdf.xacro" />
-  <xacro:sensor_d435 prefix="a_bot_" parent="a_bot_wrist_2_link">
-    <origin xyz="0.0136772228487
-		 -0.0680299757021
-		 0.198556563348"
-	    rpy="${-1.97302363932*pi/180}
-		 ${10.5114862531*pi/180}
-		 ${94.8091668854*pi/180}"/>
-  </xacro:sensor_d435>
+  <xacro:include filename="$(find aist_description)/device/urdf/_sr305.urdf.xacro" />
+  <xacro:sensor_sr305 prefix="a_bot_" parent="a_bot_wrist_2_link">
+    <origin xyz="0.0326671856774
+		 -0.063887034743
+		 0.194855923541"
+	    rpy="${-1.9802935144*pi/180}
+		 ${10.1226491078*pi/180}
+		 ${94.4366841644*pi/180}"/>
+  </xacro:sensor_sr305>
   <!-- I would like to remove the "world" link definition, but apparently it is necessary for Gazebo -->
   <link name="world"/>

File: o2as_precision_gripper/urdf/precision_gripper.urdf.xacro (robot description, xacro)
@@ -62,5 +62,5 @@
       <!-- <origin rpy="0.0 ${-pi/2} 0.0" xyz="0.001 -0.008 .162"/> -->
       <!-- <origin rpy="0 0 0" xyz="0.162 -0.008 -0.001"/> -->
-      <origin rpy="0 0 0" xyz="0.160 0.015 0.000"/>
+      <origin rpy="0 0 0" xyz="0.160 0.016 0.000"/>
       <!-- +y is the same, +x in the new frame is +z in the parent, +z is -x in the parent? -->
     </joint>

Commit message: Added a new kitting demo routine.

File: aist_description/scene/urdf/pgrp_base_scene.urdf.xacro (robot description, xacro)
@@ -74,6 +74,5 @@
   <xacro:single_suction_gripper prefix="b_bot_"
   				parent="b_bot_ft300_flange_link">
-    <origin xyz="0 0 0" rpy="0 ${0.9*pi/180} ${0.4*pi/180}"/>
-    <!-- <origin xyz="0 0 0" rpy="0 0 0"/> -->
+    <origin xyz="0 0 0" rpy="0 ${0.3*pi/180} ${-0.6*pi/180}"/>
   </xacro:single_suction_gripper>
   <!-- Add virtual wall to avoid collisions-->
@@ -85,10 +84,10 @@
   <xacro:include filename="$(find aist_phoxi_camera)/urdf/phoxi_m_camera.urdf.xacro"/>
   <xacro:phoxi_m_camera prefix="a_" parent="ground">
-    <origin xyz="0.483504569548
-		 -0.0136152151543
-		 1.40415528784"
-	    rpy="${-152.318075493*pi/180}
-		 ${-1.92295891376*pi/180}
-		 ${86.8018873041*pi/180}"/>
+    <origin xyz="0.481198965059
+		 -0.0135554880428
+		 1.40325326014"
+	    rpy="${-152.362593503*pi/180}
+		 ${-1.91385632258*pi/180}
+		 ${86.7760807485*pi/180}"/>
   </xacro:phoxi_m_camera>
   <!-- Add RealSense camera -->
