Commit message: Add new devices: grippers and TRanbo

File: aist_description/scenes/urdf/skhi_base_scene.urdf.xacro (robot description, xacro)
@@ -3,5 +3,5 @@
   <!-- Calibration help: If the robot is not moving far enough to the calibration point, increase these distances -->
   <xacro:property name="a_khi_x" value="0"/>
-  <xacro:property name="a_khi_y" value="0.4875"/>
+  <xacro:property name="a_khi_y" value="-0.4875"/>
   <xacro:property name="bots_z"	 value="0.785"/>
   <!-- Main workspace -->
@@ -27,5 +27,5 @@
 			   )/devices/urdf/rs007l.urdf.xacro"/>
   <xacro:rs007l prefix="a_khi_" parent="ground">
-    <origin xyz="${a_khi_x} ${a_khi_y} ${bots_z}" rpy="0 0 ${pi}"/>
+    <origin xyz="${a_khi_x} ${a_khi_y} ${bots_z}" rpy="0 0 0"/>
   </xacro:rs007l>
   <!-- Attach grippers -->

Commit message: Attach magripper to a_khi robot

File: aist_description/scenes/urdf/skhi_base_scene.urdf.xacro (robot description, xacro)
@@ -30,14 +30,13 @@
   </xacro:rs007l>
   <!-- Attach grippers -->
-  <!-- Add PhoXi 3D scanner -->
-  <xacro:include filename="$(find aist_phoxi_camera)/urdf/phoxi_m_camera.urdf.xacro"/>
-  <xacro:phoxi_m_camera prefix="b_" parent="ground">
-    <origin xyz="0.547941636523
-		 -0.00827443204237
-		 1.67030171767"
-	    rpy="${-151.493605482*pi/180}
-		 ${0.698490882792*pi/180}
-		 ${85.0482907121*pi/180}"/>
-  </xacro:phoxi_m_camera>
+  <xacro:include filename="$(find aist_description)/devices/urdf/magripper.urdf.xacro" />
+  <xacro:magripper2 prefix="" parent="a_khi_ee_link">
+    <origin xyz="0 0 0" rpy="0 0 0"/>
+  </xacro:magripper2>
+  <!-- Required because package robot_controllers is used for
+       driving lehz40k2_30 gripper -->
+  <!-- <gazebo> -->
+  <!--   <plugin name="fetch_gazebo_plugin" filename="libfetch_gazebo_plugin.so"/> -->
+  <!-- </gazebo> -->
   <!-- I would like to remove the "world" link definition, but apparently it is necessary for Gazebo -->
   <link name="world"/>
