Commit message: Recovered suffix of scene urdf files

File: aist_description/scenes/urdf/aist_calibration.urdf.xacro (robot description, xacro)
@@ -1,12 +1,12 @@
 <?xml version="1.0"?>
-<robot xmlns:xacro="http://wiki.ros.org/xacro" name="pgrp_calibration">
-  <xacro:include filename="$(find aist_description)/scenes/urdf/pgrp_base_scene.urdf"/>
+<robot xmlns:xacro="http://wiki.ros.org/xacro" name="aist_calibration">
+  <xacro:include filename="$(find aist_description)/scenes/urdf/aist_base_scene.urdf.xacro"/>
   <!-- Add AR markers -->
   <xacro:include filename="$(find aist_description)/objects/urdf/ar_markers.urdf.xacro"/>
   <xacro:ar_marker_70_5 prefix="a_bot_"
-  			parent="a_bot_gripper_base_link"
-  			marker_id="26"
+			parent="a_bot_robotiq_85_tip_link"
+			marker_id="26"
 			thickness="0.005">
-    <origin xyz="0.08 0 0.02" rpy="0 0 0"/>
+    <origin xyz="0.0 0.0 0.0185" rpy="0 0 0"/>
   </xacro:ar_marker_70_5>
   <xacro:ar_marker_70_5 prefix="b_bot_"
@@ -17,7 +17,7 @@
   </xacro:ar_marker_70_5>
   <xacro:ar_marker_160_10 prefix="workspace_"
-			    parent="workspace_center"
-			    marker_id="32"
-			    thickness="0.001">
+			  parent="workspace_center"
+			  marker_id="32"
+			  thickness="0.001">
     <origin xyz="0.0 0.0 0.0005" rpy="0 0 0"/>
   </xacro:ar_marker_160_10>

File: aist_description/scenes/urdf/aist_kitting.urdf.xacro (robot description, xacro)
@@ -1,5 +1,5 @@
 <?xml version="1.0"?>
 <robot xmlns:xacro="http://wiki.ros.org/xacro" name="aist_kitting">
-  <xacro:include filename="$(find aist_description)/scenes/urdf/aist_base_scene.urdf"/>
+  <xacro:include filename="$(find aist_description)/scenes/urdf/aist_base_scene.urdf.xacro"/>
   <xacro:property name="plate_w" value="0.68"/>
   <xacro:property name="plate_l" value="0.42"/>

File: aist_description/scenes/urdf/ceatec.urdf.xacro (robot description, xacro)
@@ -2,7 +2,7 @@
 <robot xmlns:xacro="http://wiki.ros.org/xacro" name="ceatec" >
   <!-- Fetch robot in empty scene (root = "map") -->
-  <xacro:include filename="$(find aist_description)/scenes/urdf/fetch_base_scene.urdf"/>
+  <xacro:include filename="$(find aist_description)/scenes/urdf/fetch_base_scene.urdf.xacro"/>
   <!-- Environment of "ceatec" scene (root = "world") -->
-  <xacro:include filename="$(find aist_description)/scenes/urdf/ceatec_environment.urdf"/>
+  <xacro:include filename="$(find aist_description)/scenes/urdf/ceatec_environment.urdf.xacro"/>
   <!-- Make "map" frame a child of "world" frame -->
   <joint name="world_map_joint" type="fixed">

File: aist_description/scenes/urdf/pgrp_calibration.urdf.xacro (robot description, xacro)
@@ -1,12 +1,12 @@
 <?xml version="1.0"?>
-<robot xmlns:xacro="http://wiki.ros.org/xacro" name="aist_calibration">
-  <xacro:include filename="$(find aist_description)/scenes/urdf/aist_base_scene.urdf"/>
+<robot xmlns:xacro="http://wiki.ros.org/xacro" name="pgrp_calibration">
+  <xacro:include filename="$(find aist_description)/scenes/urdf/pgrp_base_scene.urdf.xacro"/>
   <!-- Add AR markers -->
   <xacro:include filename="$(find aist_description)/objects/urdf/ar_markers.urdf.xacro"/>
   <xacro:ar_marker_70_5 prefix="a_bot_"
-			parent="a_bot_robotiq_85_tip_link"
-			marker_id="26"
+  			parent="a_bot_gripper_base_link"
+  			marker_id="26"
 			thickness="0.005">
-    <origin xyz="0.0 0.0 0.0185" rpy="0 0 0"/>
+    <origin xyz="0.08 0 0.02" rpy="0 0 0"/>
   </xacro:ar_marker_70_5>
   <xacro:ar_marker_70_5 prefix="b_bot_"
@@ -17,7 +17,7 @@
   </xacro:ar_marker_70_5>
   <xacro:ar_marker_160_10 prefix="workspace_"
-			  parent="workspace_center"
-			  marker_id="32"
-			  thickness="0.001">
+			    parent="workspace_center"
+			    marker_id="32"
+			    thickness="0.001">
     <origin xyz="0.0 0.0 0.0005" rpy="0 0 0"/>
   </xacro:ar_marker_160_10>

File: aist_description/scenes/urdf/pgrp_kitting.urdf.xacro (robot description, xacro)
@@ -1,5 +1,5 @@
 <?xml version="1.0"?>
 <robot xmlns:xacro="http://wiki.ros.org/xacro" name="pgrp_kitting">
-  <xacro:include filename="$(find aist_description)/scenes/urdf/pgrp_base_scene.urdf"/>
+  <xacro:include filename="$(find aist_description)/scenes/urdf/pgrp_base_scene.urdf.xacro"/>
   <xacro:property name="plate_w" value="0.68"/>
   <xacro:property name="plate_l" value="0.42"/>
