Commit message: Cleaning up and improved calibration points for wrist cameras

File: aist_description/scenes/urdf/calibration.urdf.xacro (robot description, xacro)
@@ -3,10 +3,10 @@
   <!-- Add AR markers -->
   <xacro:include filename="$(find aist_description)/objects/urdf/ar_markers.urdf.xacro"/>
-  <xacro:ar_marker_70_5 prefix="a_bot_"
-			parent="a_bot_robotiq_85_tip_link"
-			marker_id="26"
-			thickness="0.005">
-    <origin xyz="0.0 0.0 0.0185" rpy="0 0 0"/>
-  </xacro:ar_marker_70_5>
+  <!-- <xacro:ar_marker_70_5 prefix="a_bot_" -->
+  <!-- 			parent="a_bot_robotiq_85_tip_link" -->
+  <!-- 			marker_id="26" -->
+  <!-- 			thickness="0.005"> -->
+  <!--   <origin xyz="0.0 0.0 0.0185" rpy="0 0 0"/> -->
+  <!-- </xacro:ar_marker_70_5> -->
   <xacro:ar_marker_70_5 prefix="b_bot_"
   			parent="b_bot_single_suction_gripper_base_link"
