Commit message: Add missing launch files

File: aist_description/scenes/urdf/ur10e_calibration.urdf.xacro (robot description, xacro)
@@ -3,10 +3,4 @@
   <!-- Add AR markers -->
   <xacro:include filename="$(find aist_description)/objects/urdf/ar_markers.urdf.xacro"/>
-  <!-- <xacro:ar_marker_70_5 prefix="a_bot_" -->
-  <!-- 			parent="a_bot_robotiq_85_tip_link" -->
-  <!-- 			marker_id="26" -->
-  <!-- 			thickness="0.005"> -->
-  <!--   <origin xyz="0.0 0.0 0.0185" rpy="0 0 0"/> -->
-  <!-- </xacro:ar_marker_70_5> -->
   <xacro:ar_marker_70_5 prefix="workspace_"
 			parent="workspace_center"
