Commit message: Improve support for nodelet

File: aist_description/scenes/urdf/aist_base_scene.urdf.xacro (robot description, xacro)
@@ -83,10 +83,10 @@
   <xacro:include filename="$(find aist_phoxi_camera)/urdf/phoxi_m_camera.urdf.xacro"/>
   <xacro:phoxi_m_camera prefix="a_" parent="ground">
-    <origin xyz="0.481198965059
-		 -0.0135554880428
-		 1.40325326014"
-	    rpy="${-152.362593503*pi/180}
-		 ${-1.91385632258*pi/180}
-		 ${86.7760807485*pi/180}"/>
+    <origin xyz="0.483473761574
+		 -0.0146268275279
+		 1.4038624572"
+	    rpy="${-152.299482977*pi/180}
+		 ${-1.97595651456*pi/180}
+		 ${86.7431680432*pi/180}"/>
   </xacro:phoxi_m_camera>
   <!-- Add RealSense camera -->

Commit message: Cleaning up

File: aist_description/scenes/urdf/aist_base_scene.urdf.xacro (robot description, xacro)
@@ -83,11 +83,11 @@
   <xacro:include filename="$(find
 			   aist_phoxi_camera)/urdf/phoxi_m_camera.urdf.xacro"/>
-  <xacro:phoxi_m_camera prefix="a_phoxi_m_" parent="ground">
-    <origin xyz="0.483473761574
-		 -0.0146268275279
-		 1.4038624572"
-	    rpy="${-152.299482977*pi/180}
-		 ${-1.97595651456*pi/180}
-		 ${86.7431680432*pi/180}"/>
+  <xacro:phoxi_m_camera prefix="a_phoxi_m_" parent="workspace_center">
+    <origin xyz="0.483543436025
+		 -0.0149511700982
+		 0.633792706454"
+	    rpy="${-152.286950706*pi/180}
+		 ${-2.00315281361*pi/180}
+		 ${86.7522427304*pi/180}"/>
   </xacro:phoxi_m_camera>
   <!-- Add RealSense camera -->

Commit message: Make tool_calibration.py and interactive.py be invoked through launch files

File: aist_description/scenes/urdf/aist_base_scene.urdf.xacro (robot description, xacro)
@@ -73,5 +73,5 @@
   <xacro:single_suction_gripper prefix="b_bot_"
   				parent="b_bot_ft300_flange_link">
-    <origin xyz="0 0 0" rpy="0 ${0.3*pi/180} ${-0.6*pi/180}"/>
+    <origin xyz="0 0 0" rpy="0 ${0.0*pi/180} ${-0.1*pi/180}"/>
   </xacro:single_suction_gripper>
   <!-- Add virtual wall to avoid collisions-->

Commit message: Make aist_camera_multiplexer not use message_filter

File: aist_description/scenes/urdf/aist_base_scene.urdf.xacro (robot description, xacro)
@@ -73,5 +73,5 @@
   <xacro:single_suction_gripper prefix="b_bot_"
   				parent="b_bot_ft300_flange_link">
-    <origin xyz="0 0 0" rpy="0 ${0.0*pi/180} ${-0.1*pi/180}"/>
+    <origin xyz="0 0 0" rpy="0 ${0.4*pi/180} ${0.1*pi/180}"/>
   </xacro:single_suction_gripper>
   <!-- Add virtual wall to avoid collisions-->

Commit message: Update tool calibration of b_bot_suction_gripper

File: aist_description/scenes/urdf/aist_base_scene.urdf.xacro (robot description, xacro)
@@ -77,5 +77,5 @@
   <xacro:single_suction_gripper prefix="b_bot_"
   				parent="b_bot_ft300_flange_link">
-    <origin xyz="0 0 0" rpy="0 ${0.4*pi/180} ${0.1*pi/180}"/>
+    <origin xyz="0 0 0" rpy="0 ${0.2*pi/180} ${-1.2*pi/180}"/>
   </xacro:single_suction_gripper>
   <!-- Add virtual wall to avoid collisions-->

Commit message: Updated tool calibration

File: aist_description/scenes/urdf/aist_base_scene.urdf.xacro (robot description, xacro)
@@ -77,5 +77,6 @@
   <xacro:single_suction_gripper prefix="b_bot_"
   				parent="b_bot_ft300_flange_link">
-    <origin xyz="0 0 0" rpy="0 ${0.2*pi/180} ${-1.2*pi/180}"/>
+    <!-- <origin xyz="0 0 0" rpy="0 ${0.2*pi/180} ${-1.2*pi/180}"/> -->
+    <origin xyz="0 0 0" rpy="0 ${0.5*pi/180} ${-0.2*pi/180}"/>
   </xacro:single_suction_gripper>
   <!-- Add virtual wall to avoid collisions-->

Commit message: Add feedback to pickOrPlaceAction

File: aist_description/scenes/urdf/aist_base_scene.urdf.xacro (robot description, xacro)
@@ -78,5 +78,5 @@
   				parent="b_bot_ft300_flange_link">
     <!-- <origin xyz="0 0 0" rpy="0 ${0.2*pi/180} ${-1.2*pi/180}"/> -->
-    <origin xyz="0 0 0" rpy="0 ${0.5*pi/180} ${-0.2*pi/180}"/>
+    <origin xyz="0 0 0" rpy="0 ${0.0*pi/180} ${-0.2*pi/180}"/>
   </xacro:single_suction_gripper>
   <!-- Add virtual wall to avoid collisions-->

Commit message: Update tool calibration and modified graspability parameters

File: aist_description/scenes/urdf/aist_base_scene.urdf.xacro (robot description, xacro)
@@ -78,5 +78,5 @@
   				parent="b_bot_ft300_flange_link">
     <!-- <origin xyz="0 0 0" rpy="0 ${0.2*pi/180} ${-1.2*pi/180}"/> -->
-    <origin xyz="0 0 0" rpy="0 ${0.0*pi/180} ${-0.2*pi/180}"/>
+    <origin xyz="0 0 0" rpy="0 ${-0.1*pi/180} ${0.45*pi/180}"/>
   </xacro:single_suction_gripper>
   <!-- Add virtual wall to avoid collisions-->
