Commit message: Cleaning up tranbo.urdf.xacro

File: aist_description/devices/urdf/tranbo.urdf.xacro (robot description, xacro)
@@ -52,4 +52,55 @@
       <child  link="${prefix}caster_link" />
     </joint>
+  </xacro:macro>
+  <!-- ========= Wheel ========= -->
+  <xacro:macro name="tranbo_wheel" params="prefix parent left">
+    <link name="${prefix}wheel_link">
+      <inertial>
+    	<origin xyz="0 0 0" rpy="0 0 0"/>
+    	<mass value="4.3542"/>
+    	<inertia ixx="0.0045" ixy="0" ixz="0"
+		 iyy="0.005"  iyz="0" izz="0.0045"/>
+      </inertial>
+      <visual>
+    	<origin xyz="0 0 0" rpy="${pi/2} 0 0"/>
+    	<geometry>
+	  <cylinder radius="${tranbo_wheel_radius}"
+		    length="${tranbo_wheel_length}"/>
+    	</geometry>
+    	<material name="">
+          <color rgba="0.086 0.506 0.767 1" />
+    	</material>
+      </visual>
+      <collision>
+    	<origin xyz="0 0 0" rpy="${pi/2} 0 0"/>
+    	<geometry>
+	  <cylinder radius="${tranbo_wheel_radius}"
+		    length="${tranbo_wheel_length}"/>
+    	</geometry>
+      </collision>
+    </link>
+    <gazebo reference="${prefix}wheel_link">
+      <kp>500000.0</kp>
+      <kd>10.0</kd>
+      <mu1>10</mu1>
+      <mu2>10</mu2>
+      <fdir1>1 0 0</fdir1>
+      <maxVel>1.0</maxVel>
+      <minDepth>0.003</minDepth>
+      <material>Gazebo/Black</material>
+    </gazebo>
+    <joint name="${prefix}wheel_joint" type="continuous">
+      <origin xyz="0
+		   ${tranbo_tread/2 if left else -tranbo_tread/2}
+		   ${tranbo_wheel_radius}"
+	      rpy="0 0 0"/>
+      <parent link="${parent}" />
+      <child  link="${prefix}wheel_link" />
+      <axis xyz="0 1 0" />
+      <limit effort="8.85" velocity="34.8" />
+    </joint>
+    <gazebo reference="${prefix}wheel_joint">
+      <implicitSpringDamper>1</implicitSpringDamper>
+    </gazebo>
   </xacro:macro>
   <!-- ========= Tranbo ========= -->
@@ -114,95 +165,11 @@
 			 front="False" left="False"/>
     <!-- Left wheel -->
-    <link name="${prefix}l_wheel_link">
-      <inertial>
-    	<origin xyz="0 0 0" rpy="0 0 0"/>
-    	<mass value="4.3542"/>
-    	<inertia ixx="0.0045" ixy="0" ixz="0"
-		 iyy="0.005" iyz="0" izz="0.0045"/>
-      </inertial>
-      <visual>
-    	<origin xyz="0 0 0" rpy="${pi/2} 0 0"/>
-    	<geometry>
-	  <cylinder radius="${tranbo_wheel_radius}"
-		    length="${tranbo_wheel_length}"/>
-    	</geometry>
-    	<material name="">
-          <color rgba="0.086 0.506 0.767 1" />
-    	</material>
-      </visual>
-      <collision>
-    	<origin xyz="0 0 0" rpy="${pi/2} 0 0"/>
-    	<geometry>
-	  <cylinder radius="${tranbo_wheel_radius}"
-		    length="${tranbo_wheel_length}"/>
-    	</geometry>
-      </collision>
-    </link>
-    <gazebo reference="${prefix}l_wheel_link">
-      <kp>500000.0</kp>
-      <kd>10.0</kd>
-      <mu1>10</mu1>
-      <mu2>10</mu2>
-      <fdir1>1 0 0</fdir1>
-      <maxVel>1.0</maxVel>
-      <minDepth>0.003</minDepth>
-      <material>Gazebo/Black</material>
-    </gazebo>
-    <joint name="${prefix}l_wheel_joint" type="continuous">
-      <origin xyz="0 ${tranbo_tread/2} ${tranbo_wheel_radius}" rpy="0 0 0"/>
-      <parent link="${prefix}base_link" />
-      <child  link="${prefix}l_wheel_link" />
-      <axis xyz="0 1 0" />
-      <limit effort="8.85" velocity="34.8" />
-    </joint>
-    <gazebo reference="${prefix}l_wheel_joint">
-      <implicitSpringDamper>1</implicitSpringDamper>
-    </gazebo>
+    <xacro:tranbo_wheel prefix="${prefix}l_"
+			parent="${prefix}base_link"
+			left="True"/>
     <!-- Right wheel -->
-    <link name="${prefix}r_wheel_link">
-      <inertial>
-    	<origin xyz="0 0 0" rpy="0 0 0"/>
-    	<mass value="4.3542"/>
-    	<inertia ixx="0.0045" ixy="0" ixz="0"
-		 iyy="0.005" iyz="0" izz="0.0045"/>
-      </inertial>
-      <visual>
-    	<origin xyz="0 0 0" rpy="${pi/2} 0 0"/>
-    	<geometry>
-	  <cylinder radius="${tranbo_wheel_radius}"
-		    length="${tranbo_wheel_length}"/>
-    	</geometry>
-    	<material name="">
-          <color rgba="0.086 0.506 0.767 1" />
-    	</material>
-      </visual>
-      <collision>
-    	<origin xyz="0 0 0" rpy="${pi/2} 0 0"/>
-    	<geometry>
-	  <cylinder radius="${tranbo_wheel_radius}"
-		    length="${tranbo_wheel_length}"/>
-    	</geometry>
-      </collision>
-    </link>
-    <gazebo reference="${prefix}r_wheel_link">
-      <kp>500000.0</kp>
-      <kd>10.0</kd>
-      <mu1>10</mu1>
-      <mu2>10</mu2>
-      <fdir1>1 0 0</fdir1>
-      <maxVel>1.0</maxVel>
-      <minDepth>0.003</minDepth>
-      <material>Gazebo/Black</material>
-    </gazebo>
-    <joint name="${prefix}r_wheel_joint" type="continuous">
-      <origin xyz="0 ${-tranbo_tread/2} ${tranbo_wheel_radius}" rpy="0 0 0"/>
-      <parent link="${prefix}base_link" />
-      <child  link="${prefix}r_wheel_link" />
-      <axis xyz="0 1 0" />
-      <limit effort="8.85" velocity="34.8" />
-    </joint>
-    <gazebo reference="${prefix}r_wheel_joint">
-      <implicitSpringDamper>1</implicitSpringDamper>
-    </gazebo>
+    <xacro:tranbo_wheel prefix="${prefix}r_"
+			parent="${prefix}base_link"
+			left="False"/>
   </xacro:macro>
 </robot>

Commit message: Cleaning up URDF of tranbo

File: aist_description/devices/urdf/tranbo.urdf.xacro (robot description, xacro)
@@ -1,20 +1,10 @@
 <?xml version="1.0"?>
 <robot name="tranbo" xmlns:xacro="http://ros.org/wiki/xacro">
-  <!-- Tranbo constants -->
-  <xacro:property name="tranbo_length"		value="1.050"/>
-  <xacro:property name="tranbo_width"		value="0.595"/>
-  <!-- <xacro:property name="tranbo_height"	value="0.8788"/> -->
-  <xacro:property name="tranbo_height"		value="0.882"/>
-  <xacro:property name="tranbo_offset"		value="-0.225"/>
-  <xacro:property name="tranbo_tread"		value="0.441"/>
-  <xacro:property name="tranbo_wheel_mass"	value="2.0"/>
-  <xacro:property name="tranbo_wheel_radius"	value="0.075"/>
-  <xacro:property name="tranbo_wheel_length"	value="0.05"/>
-  <xacro:property name="tranbo_caster_base"	value="0.840"/>
-  <xacro:property name="tranbo_caster_radius"	value="0.065"/>
-  <xacro:property name="tranbo_caster_length"	value="0.05"/>
-  <xacro:property name="tranbo_caster_tread"	value="0.385"/>
   <!-- ========= Catser ========= -->
   <xacro:macro name="tranbo_caster" params="prefix parent front left">
+    <xacro:property name="tranbo_caster_base"	value="0.840"/>
+    <xacro:property name="tranbo_caster_radius"	value="0.065"/>
+    <xacro:property name="tranbo_caster_length"	value="0.050"/>
+    <xacro:property name="tranbo_caster_tread"	value="0.385"/>
     <link name="${prefix}caster_link">
       <inertial>
@@ -29,5 +19,5 @@
 	</geometry>
 	<material name="">
-          <color rgba="0 0 0 1" />
+          <color rgba="0 0 0 1"/>
 	</material>
       </visual>
@@ -47,12 +37,15 @@
       <origin xyz="${tranbo_caster_base/2 if front else -tranbo_caster_base/2}
 		   ${tranbo_caster_tread/2 if left else -tranbo_caster_tread/2}
-		   ${tranbo_caster_radius + 0.005}"
-	      rpy="${pi/2} 0 0" />
-      <parent link="${parent}" />
-      <child  link="${prefix}caster_link" />
+		   ${tranbo_caster_radius + 0.002}"
+	      rpy="${pi/2} 0 0"/>
+      <parent link="${parent}"/>
+      <child  link="${prefix}caster_link"/>
     </joint>
   </xacro:macro>
   <!-- ========= Wheel ========= -->
   <xacro:macro name="tranbo_wheel" params="prefix parent left">
+    <xacro:property name="tranbo_tread"		value="0.441"/>
+    <xacro:property name="tranbo_wheel_radius"	value="0.075"/>
+    <xacro:property name="tranbo_wheel_length"	value="0.050"/>
     <link name="${prefix}wheel_link">
       <inertial>
@@ -69,5 +62,5 @@
     	</geometry>
     	<material name="">
-          <color rgba="0.086 0.506 0.767 1" />
+          <color rgba="0.086 0.506 0.767 1"/>
     	</material>
       </visual>
@@ -83,6 +76,6 @@
       <kp>500000.0</kp>
       <kd>10.0</kd>
-      <mu1>10</mu1>
-      <mu2>10</mu2>
+      <mu1>100.0</mu1>
+      <mu2>100.0</mu2>
       <fdir1>1 0 0</fdir1>
       <maxVel>1.0</maxVel>
@@ -95,8 +88,8 @@
 		   ${tranbo_wheel_radius}"
 	      rpy="0 0 0"/>
-      <parent link="${parent}" />
-      <child  link="${prefix}wheel_link" />
-      <axis xyz="0 1 0" />
-      <limit effort="8.85" velocity="34.8" />
+      <parent link="${parent}"/>
+      <child  link="${prefix}wheel_link"/>
+      <axis xyz="0 1 0"/>
+      <limit effort="8.85" velocity="34.8"/>
     </joint>
     <gazebo reference="${prefix}wheel_joint">
@@ -106,9 +99,14 @@
   <!-- ========= Tranbo ========= -->
   <xacro:macro name="tranbo" params="prefix">
+    <xacro:property name="tranbo_length"		value="1.050"/>
+    <xacro:property name="tranbo_width"			value="0.595"/>
+    <xacro:property name="tranbo_height"		value="0.8788"/>
+    <xacro:property name="tranbo_offset"		value="-0.225"/>
+    <xacro:property name="tranbo_ground_clearance"	value="0.040"/>
     <!-- Body -->
     <link name="${prefix}base_link">
       <inertial>
-	<origin xyz="-0.0036 0.0 0.0014" rpy="0 0 0"/>
-	<mass value="70.1294" />
+	<origin xyz="0 0 ${tranbo_height/2}" rpy="0 0 0"/>
+	<mass value="70.1294"/>
 	<inertia ixx="1.225"  ixy="0.0099"  ixz="0.0062"
 		 iyy="1.2853" iyz="-0.0034" izz="0.987"/>
@@ -126,7 +124,10 @@
       </visual>
       <collision>
-        <origin xyz="0 0 ${tranbo_height/2 + 0.04}" rpy="0 0 0" />
+        <origin xyz="0 0
+		     ${tranbo_height/2 + tranbo_ground_clearance}"
+		rpy="0 0 0" />
 	<geometry>
-	  <box size="${tranbo_length} ${tranbo_width} ${tranbo_height - 0.04}"/>
+	  <box size="${tranbo_length} ${tranbo_width}
+		     ${tranbo_height - tranbo_ground_clearance}"/>
 	</geometry>
       </collision>

Commit message: updaded tranbo paramters

File: aist_description/devices/urdf/tranbo.urdf.xacro (robot description, xacro)
@@ -9,5 +9,5 @@
     <link name="${prefix}caster_link">
       <inertial>
-    	<mass value="4.3542"/>
+    	<mass value="1.5"/>
     	<inertia ixx="0.0045" ixy="0" ixz="0"
 		 iyy="0.005" iyz="0" izz="0.0045"/>
@@ -30,6 +30,6 @@
     </link>
     <gazebo reference="${prefix}caster_link">
-      <mu1>0.0</mu1>
-      <mu2>0.0</mu2>
+      <mu1>0.01</mu1>
+      <mu2>0.01</mu2>
       <material>Gazebo/Black</material>
     </gazebo>
@@ -37,5 +37,5 @@
       <origin xyz="${tranbo_caster_base/2 if front else -tranbo_caster_base/2}
 		   ${tranbo_caster_tread/2 if left else -tranbo_caster_tread/2}
-		   ${tranbo_caster_radius + 0.002}"
+		   ${tranbo_caster_radius + 0.004}"
 	      rpy="${pi/2} 0 0"/>
       <parent link="${parent}"/>
@@ -76,6 +76,6 @@
       <kp>500000.0</kp>
       <kd>10.0</kd>
-      <mu1>100.0</mu1>
-      <mu2>100.0</mu2>
+      <mu1>10</mu1>
+      <mu2>10</mu2>
       <fdir1>1 0 0</fdir1>
       <maxVel>1.0</maxVel>
@@ -103,9 +103,9 @@
     <xacro:property name="tranbo_height"		value="0.8788"/>
     <xacro:property name="tranbo_offset"		value="-0.225"/>
-    <xacro:property name="tranbo_ground_clearance"	value="0.040"/>
+    <xacro:property name="tranbo_ground_clearance"	value="0.04"/>
     <!-- Body -->
     <link name="${prefix}base_link">
       <inertial>
-	<origin xyz="0 0 ${tranbo_height/2}" rpy="0 0 0"/>
+	<origin xyz="0 0 0" rpy="0 0 0"/>
 	<mass value="70.1294"/>
 	<inertia ixx="1.225"  ixy="0.0099"  ixz="0.0062"
@@ -136,6 +136,6 @@
       <kp>100000000.0</kp>
       <kd>10.0</kd>
-      <mu1>0.1</mu1>
-      <mu2>0.1</mu2>
+      <mu1>0.01</mu1>
+      <mu2>0.01</mu2>
       <fdir1>1 0 0</fdir1>
       <maxVel>10.0</maxVel>

Commit message: Spawn relay and mux nodes of topic_tools package within fetch_controller.launch

File: aist_description/devices/urdf/tranbo.urdf.xacro (robot description, xacro)
@@ -30,6 +30,6 @@
     </link>
     <gazebo reference="${prefix}caster_link">
-      <mu1>0.01</mu1>
-      <mu2>0.01</mu2>
+      <mu1>0.1</mu1>
+      <mu2>0.1</mu2>
       <material>Gazebo/Black</material>
     </gazebo>
@@ -108,5 +108,6 @@
       <inertial>
 	<origin xyz="0 0 0" rpy="0 0 0"/>
-	<mass value="70.1294"/>
+	<!-- <mass value="70.1294"/> -->
+	<mass value="150.0"/>
 	<inertia ixx="1.225"  ixy="0.0099"  ixz="0.0062"
 		 iyy="1.2853" iyz="-0.0034" izz="0.987"/>
@@ -124,6 +125,5 @@
       </visual>
       <collision>
-        <origin xyz="0 0
-		     ${tranbo_height/2 + tranbo_ground_clearance}"
+        <origin xyz="0 0 ${tranbo_height/2 + tranbo_ground_clearance}"
 		rpy="0 0 0" />
 	<geometry>
@@ -136,6 +136,6 @@
       <kp>100000000.0</kp>
       <kd>10.0</kd>
-      <mu1>0.01</mu1>
-      <mu2>0.01</mu2>
+      <mu1>0.1</mu1>
+      <mu2>0.1</mu2>
       <fdir1>1 0 0</fdir1>
       <maxVel>10.0</maxVel>
