Commit message: Add dual wrist cameras to a_bot

File: aist_description/devices/urdf/_sr305.urdf.xacro (robot description, xacro)
@@ -1,52 +1,77 @@
 <?xml version="1.0"?>
 <!--
-License: Apache 2.0. See LICENSE file in root directory.
-Copyright(c) 2017 Intel Corporation. All Rights Reserved
-This is the URDF model for the Intel RealSense 430 camera, in it's
-aluminum peripherial evaluation case.
+This file is based on the d435 urdf from the realsense package.
+The origin of the mesh is at the center of the back mount.
 -->
-<robot name="sensor_sr305" xmlns:xacro="http://wiki.ros.org/xacro">
-  <xacro:macro name="sensor_sr305" params="prefix parent *origin">
+<robot name="sensor_sr305" xmlns:xacro="http://ros.org/wiki/xacro">
+  <xacro:macro name="sensor_sr305" params="prefix parent use_bottom_mount:=false *origin">
+    <!-- TODO: Allow placing the camera using bottom mount or back mount -->
     <xacro:property name="M_PI" value="3.1415926535897931" />
-    <!-- The following values are approximate, and the camera node
-    publishing TF values with actual calibrated camera extrinsic values -->
-    <xacro:property name="sr305_cam_depth_to_color_offset" value="0.02403"/>
-    <xacro:property name="sr305_cam_depth_to_projector_offset" value="0.04785"/>
-    <!-- The following values model the aluminum peripherial case for the
-      SR305 camera, with the camera joint represented by the actual
-      peripheral camera tripod mount -->
+    <!-- The following values are approximate -->
+    <xacro:property name="sr305_cam_depth_to_left_ir_offset" value="0.0"/>
+    <xacro:property name="sr305_cam_depth_to_right_ir_offset" value="0.040"/>
+    <xacro:property name="sr305_cam_depth_to_color_offset" value="0.015"/>
+    <!-- The following values model the aluminum case of the
+  	sr305 camera, with the camera joint represented by the actual
+  	peripherial camera tripod mount -->
     <xacro:property name="sr305_cam_width" value="0.140"/>
-    <xacro:property name="sr305_cam_height" value="0.0255"/>
-    <xacro:property name="sr305_cam_depth" value="0.0095"/>
-    <xacro:property name="sr305_cam_mount_from_center_offset" value="0.0160"/>
-    <!-- The following offset is relative to the physical SR305 camera peripherial
-      camera tripod mount -->
-    <xacro:property name="sr305_cam_depth_px"
-		    value="${sr305_cam_mount_from_center_offset}"/>
-    <xacro:property name="sr305_cam_depth_py" value="-0.00754"/>
-    <xacro:property name="sr305_cam_depth_pz" value="${sr305_cam_height/2}"/>
-    <!-- <material name="aluminum"> -->
-    <!--   <color rgba="0.5 0.5 0.5 1"/> -->
-    <!-- </material> -->
+    <xacro:property name="sr305_cam_height" value="0.023"/>
+    <xacro:property name="sr305_cam_depth" value="0.012"/>
+    <!-- <xacro:property name="sr305_cam_mount_from_center_offset" value="0.0149"/> -->
+    <xacro:property name="sr305_cam_mount_from_center_offset" value="0.004"/>
+    <!-- Left sensor (looking from front):  -7.54 mm, 0, -3.721 mm -->
+    <!-- Right sensor (RGB?)(looking from front): 16.492 mm, 0, -3.721 mm -->
+    <!-- 24.033 mm distance between the camera centers, apparently -->
+    <!-- camera mount to origin: 4mm; cameras to origin: 3.721 mm. = 7.721 mm offset? -->
+    <!-- The following offset is relative to the physical sr305 camera peripheral
+  	camera tripod mount -->
+    <xacro:property name="sr305_cam_depth_px" value="${sr305_cam_mount_from_center_offset}"/>
+    <xacro:property name="sr305_cam_depth_py" value="0.0"/>
+    <xacro:property name="sr305_cam_depth_pz" value=".013063"/>
     <!-- camera body, with origin at bottom screw mount -->
-    <joint name="${prefix}camera_joint" type="fixed">
-      <xacro:insert_block name="origin" />
-      <parent link="${parent}"/>
-      <child link="${prefix}camera_link" />
-    </joint>
+    <xacro:if value="${use_bottom_mount}">
+      <joint name="${prefix}camera_joint" type="fixed">
+        <xacro:insert_block name="origin" />
+        <parent link="${parent}"/>
+        <child link="${prefix}camera_bottom_screw_frame" />
+      </joint>
+      <link name="${prefix}camera_bottom_screw_frame"/>
+      <joint name="${prefix}camera_link_joint" type="fixed">
+        <origin xyz="${sr305_cam_depth_px} ${sr305_cam_depth_py} ${sr305_cam_depth_pz}" rpy="0 0 0"/>
+        <parent link="${prefix}camera_bottom_screw_frame"/>
+        <child link="${prefix}camera_link" />
+      </joint>
+    </xacro:if>
+    <xacro:if value="${not use_bottom_mount}">
+      <!-- I forgot which conventions exist for "camera_joint" and "camera_link_joint" so I hesitate to delete one. -->
+      <joint name="${prefix}camera_joint" type="fixed">
+        <xacro:insert_block name="origin" />
+        <parent link="${parent}"/>
+        <child link="${prefix}camera_connector_link" />
+      </joint>
+      <link name="${prefix}camera_connector_link"/>
+      <joint name="${prefix}camera_link_joint" type="fixed">
+        <origin xyz="0 0 0" rpy="0 0 0"/>
+        <parent link="${prefix}camera_connector_link"/>
+        <child link="${prefix}camera_link" />
+      </joint>
+    </xacro:if>
     <link name="${prefix}camera_link">
       <visual>
-      <origin xyz="${sr305_cam_mount_from_center_offset} 0.0 ${sr305_cam_height/2}" rpy="${M_PI/2} 0 ${M_PI/2}"/>
+      <origin xyz="${0} ${-sr305_cam_depth_py} 0" rpy="${M_PI/2} 0 ${M_PI/2}"/>
         <geometry>
-	  <mesh filename="package://aist_description/devices/meshes/SR305.stl"
-		scale="0.001 0.001 0.001"/>
+          <xacro:if value="${use_bottom_mount}">
+	          <mesh filename="package://aist_description/devices/meshes/sr305_simplified.stl" scale=".001 .001 .001" />
+          </xacro:if>
+          <xacro:if value="${not use_bottom_mount}">
+	          <mesh filename="package://aist_description/devices/meshes/sr305_simplified_body.stl" scale=".001 .001 .001" />
+          </xacro:if>
         </geometry>
-	<material name="aluminum">
-	  <color rgba="0.5 0.5 0.5 1"/>
-	</material>
-        <!-- <material name="aluminum"/> -->
+        <material name="sr305_aluminum">
+          <color rgba="0.5 0.5 0.5 1"/>
+        </material>
       </visual>
       <collision>
-        <origin xyz="0.0 0.0 ${sr305_cam_height/2}" rpy="0 0 0"/>
+        <origin xyz="${sr305_cam_depth/2} ${-sr305_cam_depth_py} 0" rpy="0 0 0"/>
         <geometry>
           <box size="${sr305_cam_depth} ${sr305_cam_width} ${sr305_cam_height}"/>
@@ -62,5 +87,5 @@
     <!-- camera depth joints and links -->
     <joint name="${prefix}camera_depth_joint" type="fixed">
-      <origin xyz="${sr305_cam_depth_px} ${sr305_cam_depth_py} ${sr305_cam_depth_pz}" rpy="0 0 0"/>
+      <origin xyz=".003721 0 0" rpy="0 0 0"/>
       <parent link="${prefix}camera_link"/>
       <child link="${prefix}camera_depth_frame" />
@@ -73,17 +98,30 @@
     </joint>
     <link name="${prefix}camera_depth_optical_frame"/>
-    <!-- camera IR joints and links -->
-    <joint name="${prefix}camera_infra1_joint" type="fixed">
-      <origin xyz="0 0 0" rpy="0 0 0" />
+    <!-- camera left IR joints and links -->
+    <joint name="${prefix}camera_left_ir_joint" type="fixed">
+      <origin xyz="0 ${sr305_cam_depth_to_left_ir_offset} 0" rpy="0 0 0" />
       <parent link="${prefix}camera_depth_frame" />
-      <child link="${prefix}camera_infra1_frame" />
+      <child link="${prefix}camera_left_ir_frame" />
     </joint>
-    <link name="${prefix}camera_infra1_frame"/>
-    <joint name="${prefix}camera_infra1_optical_joint" type="fixed">
+    <link name="${prefix}camera_left_ir_frame"/>
+    <joint name="${prefix}camera_left_ir_optical_joint" type="fixed">
       <origin xyz="0 0 0" rpy="${-M_PI/2} 0 ${-M_PI/2}" />
-      <parent link="${prefix}camera_infra1_frame" />
-      <child link="${prefix}camera_infra1_optical_frame" />
+      <parent link="${prefix}camera_left_ir_frame" />
+      <child link="${prefix}camera_left_ir_optical_frame" />
     </joint>
-    <link name="${prefix}camera_infra1_optical_frame"/>
+    <link name="${prefix}camera_left_ir_optical_frame"/>
+    <!-- camera right IR joints and links -->
+    <joint name="${prefix}camera_right_ir_joint" type="fixed">
+      <origin xyz="0 ${sr305_cam_depth_to_right_ir_offset} 0" rpy="0 0 0" />
+      <parent link="${prefix}camera_depth_frame" />
+      <child link="${prefix}camera_right_ir_frame" />
+    </joint>
+    <link name="${prefix}camera_right_ir_frame"/>
+    <joint name="${prefix}camera_right_ir_optical_joint" type="fixed">
+      <origin xyz="0 0 0" rpy="${-M_PI/2} 0 ${-M_PI/2}" />
+      <parent link="${prefix}camera_right_ir_frame" />
+      <child link="${prefix}camera_right_ir_optical_frame" />
+    </joint>
+    <link name="${prefix}camera_right_ir_optical_frame"/>
     <!-- camera color joints and links -->
     <joint name="${prefix}camera_color_joint" type="fixed">
@@ -99,11 +137,4 @@
     </joint>
     <link name="${prefix}camera_color_optical_frame"/>
-    <!-- camera projector joints and links -->
-    <joint name="${prefix}camera_projector_joint" type="fixed">
-      <origin xyz="0 ${sr305_cam_depth_to_projector_offset} 0" rpy="0 0 0" />
-      <parent link="${prefix}camera_depth_frame" />
-      <child link="${prefix}camera_projector_frame" />
-    </joint>
-    <link name="${prefix}camera_projector_frame"/>
     <gazebo reference="${prefix}camera_depth_frame">
       <sensor type="depth" name="${prefix}camera">

File: aist_description/devices/urdf/wrist_cameras.urdf.xacro (robot description, xacro)
@@ -1,9 +1,13 @@
 <?xml version="1.0"?>
+<!-- This macro adds a convenient TF frame at the tip of the closed gripper. -->
+<!-- The position of the TF frame has not been measured at all and needs to be calibrated. -->
 <robot name="robotiq_85_gripper_o2ac" xmlns:xacro="http://www.ros.org/wiki/xacro">
   <xacro:macro name="wrist_cameras" params="prefix parent">
-    <xacro:include filename="$(find aist_description)/devices/urdf/_sr305.urdf.xacro" />
+    <xacro:include filename="$(find aist_description
+			     )/devices/urdf/_sr305.urdf.xacro"/>
       <!-- Add the holder and two SR305 cameras -->
-    <xacro:property name="mount_mesh_file" value="package://aist_description/devices/meshes/sr305_mount.stl" />
-    <link name="${prefix}cam_mount">
+      <xacro:property name="mount_mesh_file"
+		      value="package://aist_description/devices/meshes/sr305_mount.stl"/>
+    <link name="${prefix}camera_mount">
       <inertial>
         <origin rpy="${pi} 0 ${pi/2}" xyz="0 0 0.0"/>
@@ -27,26 +31,14 @@
       </collision>
     </link>
-    <joint name="${prefix}cam_mount_joint" type="fixed">
+    <joint name="${prefix}camera_mount_joint" type="fixed">
       <parent link="${parent}" />
-      <child link = "${prefix}cam_mount" />
+      <child link = "${prefix}camera_mount" />
       <origin xyz="0.035 0.0 0.025" rpy="0 0 0"/>
     </joint>
-    <link name="${prefix}cam_1_link" />
-    <joint name="${prefix}cam_1_joint" type="fixed">
-      <parent link="${parent}" />
-      <child link="${prefix}cam_1_link" />
+    <xacro:sensor_sr305 prefix="${prefix}inside_" parent="${parent}">
       <origin xyz="0.026 0 0.0595" rpy="0 ${20.0*pi/180.0} 0" />
-    </joint>
-    <xacro:sensor_sr305 prefix="${prefix}_cam_1_" parent="${prefix}cam_1_link">
-      <origin xyz="0 0 0" rpy="0 0 0"/>
     </xacro:sensor_sr305>
-    <link name="${prefix}cam_2_link" />
-    <joint name="${prefix}cam_2_joint" type="fixed">
-      <parent link="${parent}" />
-      <child link="${prefix}cam_2_link" />
+    <xacro:sensor_sr305 prefix="${prefix}outside_" parent="${parent}">
       <origin xyz="0.026 0 ${0.0595+.024}" rpy="0 ${-15.0*pi/180.0} 0" />
-    </joint>
-    <xacro:sensor_sr305 prefix="${prefix}_cam_2_" parent="${prefix}cam_2_link">
-      <origin xyz="0 0 0" rpy="0 0 0"/>
     </xacro:sensor_sr305>
   </xacro:macro>

File: aist_description/scenes/urdf/aist_base_scene.urdf.xacro (robot description, xacro)
@@ -91,13 +91,8 @@
   </xacro:phoxi_m_camera>
   <!-- Add RealSense camera -->
-  <xacro:include filename="$(find aist_description)/devices/urdf/_sr305.urdf.xacro" />
-  <xacro:sensor_sr305 prefix="a_bot_" parent="a_bot_wrist_2_link">
-    <origin xyz="0.0326671856774
-		 -0.063887034743
-		 0.194855923541"
-	    rpy="${-1.9802935144*pi/180}
-		 ${10.1226491078*pi/180}
-		 ${94.4366841644*pi/180}"/>
-  </xacro:sensor_sr305>
+  <xacro:include filename="$(find aist_description
+			   )/devices/urdf/wrist_cameras.urdf.xacro" />
+  <xacro:wrist_cameras prefix="a_bot_"
+		       parent="a_bot_robotiq_85_base_link"/>
   <!-- I would like to remove the "world" link definition, but apparently it is necessary for Gazebo -->
   <link name="world"/>
