Commit message: Change joint name of pillar of magripper

File: aist_description/devices/urdf/magripper.urdf.xacro (robot description, xacro)
@@ -5,5 +5,5 @@
   <xacro:include filename="$(find aist_description)/devices/urdf/lehz40k2_30.urdf.xacro" />
   <xacro:macro name="pillar" params="name length diameter parent *origin">
-    <joint name="${name}" type="fixed">
+    <joint name="${name}_joint" type="fixed">
       <parent link="${parent}"/>
       <child  link="${name}"/>

Commit message: Cleaning up urdfs and added launch script for KHI robot

File: aist_description/devices/urdf/magripper.urdf.xacro (robot description, xacro)
@@ -27,5 +27,5 @@
       </collision>
       <inertial>
-        <mass value="1.0"/>
+        <mass value="0.3"/>
         <inertia ixx="0.0" ixy="0.0" ixz="0.0" iyy="0.0" iyz="0.0" izz="0.0"/>
       </inertial>

File: aist_description/devices/urdf/tranbo.urdf.xacro (robot description, xacro)
@@ -1,15 +1,58 @@
 <?xml version="1.0"?>
 <robot name="tranbo" xmlns:xacro="http://ros.org/wiki/xacro">
+  <!-- Tranbo constants -->
+  <xacro:property name="tranbo_length"		value="1.050"/>
+  <xacro:property name="tranbo_width"		value="0.595"/>
+  <!-- <xacro:property name="tranbo_height"	value="0.8788"/> -->
+  <xacro:property name="tranbo_height"		value="0.882"/>
+  <xacro:property name="tranbo_offset"		value="-0.225"/>
+  <xacro:property name="tranbo_tread"		value="0.441"/>
+  <xacro:property name="tranbo_wheel_mass"	value="2.0"/>
+  <xacro:property name="tranbo_wheel_radius"	value="0.075"/>
+  <xacro:property name="tranbo_wheel_length"	value="0.05"/>
+  <xacro:property name="tranbo_caster_base"	value="0.840"/>
+  <xacro:property name="tranbo_caster_radius"	value="0.065"/>
+  <xacro:property name="tranbo_caster_length"	value="0.05"/>
+  <xacro:property name="tranbo_caster_tread"	value="0.385"/>
+  <!-- ========= Catser ========= -->
+  <xacro:macro name="tranbo_caster" params="prefix parent front left">
+    <link name="${prefix}caster_link">
+      <inertial>
+    	<mass value="4.3542"/>
+    	<inertia ixx="0.0045" ixy="0" ixz="0"
+		 iyy="0.005" iyz="0" izz="0.0045"/>
+      </inertial>
+      <visual>
+	<geometry>
+	  <cylinder radius="${tranbo_caster_radius}"
+		    length="${tranbo_caster_length}"/>
+	</geometry>
+	<material name="">
+          <color rgba="0 0 0 1" />
+	</material>
+      </visual>
+      <collision>
+	<geometry>
+	  <cylinder radius="${tranbo_caster_radius}"
+		    length="${tranbo_caster_length}"/>
+	</geometry>
+      </collision>
+    </link>
+    <gazebo reference="${prefix}caster_link">
+      <mu1>0.0</mu1>
+      <mu2>0.0</mu2>
+      <material>Gazebo/Black</material>
+    </gazebo>
+    <joint name="${prefix}caster_joint" type="fixed">
+      <origin xyz="${tranbo_caster_base/2 if front else -tranbo_caster_base/2}
+		   ${tranbo_caster_tread/2 if left else -tranbo_caster_tread/2}
+		   ${tranbo_caster_radius + 0.005}"
+	      rpy="${pi/2} 0 0" />
+      <parent link="${parent}" />
+      <child  link="${prefix}caster_link" />
+    </joint>
+  </xacro:macro>
+  <!-- ========= Tranbo ========= -->
   <xacro:macro name="tranbo" params="prefix">
-    <!-- Tranbo constants -->
-    <xacro:property name="tranbo_length"	value="1.050"/>
-    <xacro:property name="tranbo_width"		value="0.595"/>
-    <!-- <xacro:property name="tranbo_height"	value="0.8788"/> -->
-    <xacro:property name="tranbo_height"	value="0.882"/>
-    <xacro:property name="tranbo_offset"	value="-0.225"/>
-    <xacro:property name="tranbo_tread"		value="0.441"/>
-    <xacro:property name="tranbo_wheel_mass"	value="2.0"/>
-    <xacro:property name="tranbo_wheel_radius"	value="0.075"/>
-    <xacro:property name="tranbo_wheel_length"	value="0.05"/>
     <!-- Body -->
     <link name="${prefix}base_link">
@@ -17,5 +60,6 @@
 	<origin xyz="-0.0036 0.0 0.0014" rpy="0 0 0"/>
 	<mass value="70.1294" />
-	<inertia ixx="1.225" ixy="0.0099" ixz="0.0062" iyy="1.2853" iyz="-0.0034" izz="0.987"/>
+	<inertia ixx="1.225"  ixy="0.0099"  ixz="0.0062"
+		 iyy="1.2853" iyz="-0.0034" izz="0.987"/>
       </inertial>
       <visual>
@@ -23,5 +67,6 @@
 		rpy="0 0 ${-pi/2}" />
 	<geometry>
-          <mesh filename="package://aist_description/devices/meshes/TRanbo.stl" scale="0.001 0.001 0.001"/>
+          <mesh filename="package://aist_description/devices/meshes/TRanbo.stl"
+		scale="0.001 0.001 0.001"/>
 	</geometry>
 	<material name="">
@@ -30,7 +75,7 @@
       </visual>
       <collision>
-        <origin xyz="0 0 ${tranbo_height/2 + 0.005}" rpy="0 0 0" />
-	<geometry>
-	  <box size="${tranbo_length} ${tranbo_width} ${tranbo_height}"/>
+        <origin xyz="0 0 ${tranbo_height/2 + 0.04}" rpy="0 0 0" />
+	<geometry>
+	  <box size="${tranbo_length} ${tranbo_width} ${tranbo_height - 0.04}"/>
 	</geometry>
       </collision>
@@ -52,4 +97,20 @@
     </joint>
     <link name="${prefix}basement_link"/>
+    <!-- Front-left caster -->
+    <xacro:tranbo_caster prefix="${prefix}front_left_"
+			 parent="${prefix}base_link"
+			 front="True" left="True"/>
+    <!-- Front-right caster -->
+    <xacro:tranbo_caster prefix="${prefix}front_right_"
+			 parent="${prefix}base_link"
+			 front="True" left="False"/>
+    <!-- Rear-left caster -->
+    <xacro:tranbo_caster prefix="${prefix}rear_left_"
+			 parent="${prefix}base_link"
+			 front="False" left="True"/>
+    <!-- Front-right caster -->
+    <xacro:tranbo_caster prefix="${prefix}rear_right_"
+			 parent="${prefix}base_link"
+			 front="False" left="False"/>
     <!-- Left wheel -->
     <link name="${prefix}l_wheel_link">
@@ -57,8 +118,9 @@
     	<origin xyz="0 0 0" rpy="0 0 0"/>
     	<mass value="4.3542"/>
-    	<inertia ixx="0.0045" ixy="0" ixz="0" iyy="0.005" iyz="0" izz="0.0045"/>
-      </inertial>
-      <visual>
-    	<origin xyz="0 0 0" rpy="${-pi/2} 0 0"/>
+    	<inertia ixx="0.0045" ixy="0" ixz="0"
+		 iyy="0.005" iyz="0" izz="0.0045"/>
+      </inertial>
+      <visual>
+    	<origin xyz="0 0 0" rpy="${pi/2} 0 0"/>
     	<geometry>
 	  <cylinder radius="${tranbo_wheel_radius}"
@@ -70,5 +132,5 @@
       </visual>
       <collision>
-    	<origin xyz="0 0 0" rpy="${-pi/2} 0 0"/>
+    	<origin xyz="0 0 0" rpy="${pi/2} 0 0"/>
     	<geometry>
 	  <cylinder radius="${tranbo_wheel_radius}"
@@ -102,8 +164,9 @@
     	<origin xyz="0 0 0" rpy="0 0 0"/>
     	<mass value="4.3542"/>
-    	<inertia ixx="0.0045" ixy="0" ixz="0" iyy="0.005" iyz="0" izz="0.0045"/>
-      </inertial>
-      <visual>
-    	<origin xyz="0 0 0" rpy="${-pi/2} 0 0"/>
+    	<inertia ixx="0.0045" ixy="0" ixz="0"
+		 iyy="0.005" iyz="0" izz="0.0045"/>
+      </inertial>
+      <visual>
+    	<origin xyz="0 0 0" rpy="${pi/2} 0 0"/>
     	<geometry>
 	  <cylinder radius="${tranbo_wheel_radius}"
@@ -115,5 +178,5 @@
       </visual>
       <collision>
-    	<origin xyz="0 0 0" rpy="${-pi/2} 0 0"/>
+    	<origin xyz="0 0 0" rpy="${pi/2} 0 0"/>
     	<geometry>
 	  <cylinder radius="${tranbo_wheel_radius}"

Commit message: Add model of magripper made by KHI

File: aist_description/devices/urdf/magripper.urdf.xacro (robot description, xacro)
@@ -122,3 +122,94 @@
     </xacro:lehz40k2_30>
   </xacro:macro>
+  <xacro:macro name="magripper3" params="prefix parent *origin">
+    <xacro:property name="gripper_x_offset" value="0.075"/>
+    <xacro:property name="gripper_y_offset" value="-0.050"/>
+    <xacro:property name="gripper_z_offset" value="0.050"/>
+    <xacro:property name="magnet_y_offset" value="-0.174"/>
+    <!-- <xacro:property name="camera_x_offset" value="0.298"/> -->
+    <xacro:property name="camera_x_offset" value="0.180"/>
+    <xacro:property name="camera_y_offset" value="-0.1145"/>
+    <xacro:property name="camera_z_offset" value="-0.0355"/>
+    <joint name="${prefix}magripper_base_joint" type="fixed">
+      <parent link="${parent}"/>
+      <child link="${prefix}magripper_base_link"/>
+      <xacro:insert_block name="origin"/>
+    </joint>
+    <link name="${prefix}magripper_base_link">
+      <visual>
+        <origin xyz="0 0 0" rpy="0 0 0" />
+        <geometry>
+          <mesh filename="package://aist_description/devices/meshes/magripper_base.stl" scale="0.001 0.001 0.001"/>
+        </geometry>
+        <material name="Gazebo/Grey">
+          <color rgba="0.7 0.7 0.7 1" />
+        </material>
+      </visual>
+      <collision>
+        <origin xyz="$0 0 0" rpy="0 0 0" />
+        <geometry>
+          <mesh filename="package://aist_description/devices/meshes/collision/magripper_base.stl" scale="0.001 0.001 0.001"/>
+        </geometry>
+      </collision>
+      <!-- Required for Gazebo -->
+      <inertial>
+	<mass value="1.5"/>
+	<inertia ixx="0.0" ixy="0.0" ixz="0.0" iyy="0.0" iyz="0.0" izz="0.0"/>
+      </inertial>
+    </link>
+    <!-- <gazebo reference="${prefix}magripper_base_link"> -->
+    <!--   <material>Gazebo/Grey</material> -->
+    <!--   <selfCollide>True</selfCollide> -->
+    <!-- </gazebo> -->
+    <!-- Magswitch_E30 magnet hand -->
+    <joint name="${prefix}magripper_magnet_axis_joint" type="fixed">
+      <parent link="${prefix}magripper_base_link"/>
+      <child  link="${prefix}magripper_magnet_axis_link"/>
+      <origin xyz="${gripper_x_offset} 0 0"
+	      rpy="${-pi/4} 0 0"/>
+    </joint>
+    <link name="${prefix}magripper_magnet_axis_link"/>
+    <joint name="${prefix}magripper_magnet_flange_joint" type="fixed">
+      <parent link="${prefix}magripper_magnet_axis_link"/>
+      <child  link="${prefix}magripper_magnet_flange"/>
+      <origin xyz="0 ${magnet_y_offset} ${gripper_z_offset}"
+	      rpy="0 0 ${-pi/2}"/>
+    </joint>
+    <link name="${prefix}magripper_magnet_flange"/>
+    <xacro:magswitch_e30 prefix="${prefix}"
+    			 parent="${prefix}magripper_magnet_flange">
+      <origin xyz="0 0 0" rpy="0 0 0"/>
+    </xacro:magswitch_e30>
+    <!-- LEHZ40K2-30 two-finger gripper -->
+    <joint name="${prefix}magripper_gripper_axis_joint" type="fixed">
+      <parent link="${prefix}magripper_base_link"/>
+      <child  link="${prefix}magripper_gripper_axis_link"/>
+      <origin xyz="${gripper_x_offset} 0 0"
+	      rpy="${pi/4} 0 0"/>
+    </joint>
+    <link name="${prefix}magripper_gripper_axis_link"/>
+    <joint name="${prefix}magripper_gripper_flange_joint" type="fixed">
+      <parent link="${prefix}magripper_gripper_axis_link"/>
+      <child  link="${prefix}magripper_gripper_flange"/>
+      <origin xyz="0 ${gripper_y_offset} ${-gripper_z_offset}"
+	      rpy="0 0 ${-pi/2}"/>
+    </joint>
+    <link name="${prefix}magripper_gripper_flange"/>
+    <xacro:lehz40k2_30 prefix="${prefix}"
+    		       parent="${prefix}magripper_gripper_flange">
+      <origin xyz="0 0 0" rpy="0 0 0"/>
+    </xacro:lehz40k2_30>
+    <!-- PhoXi camera -->
+    <joint name="${prefix}magripper_camera_flange_joint" type="fixed">
+      <parent link="${prefix}magripper_base_link"/>
+      <child  link="${prefix}magripper_camera_flange"/>
+      <origin xyz="${camera_x_offset} ${camera_y_offset} ${camera_z_offset}"
+	      rpy="${-pi/2} 0 ${pi}"/>
+    </joint>
+    <link name="${prefix}magripper_camera_flange"/>
+    <xacro:phoxi_m_camera prefix="${prefix}"
+    			  parent="${prefix}magripper_camera_flange">
+      <origin xyz="0 0 0" rpy="0 0 0"/>
+    </xacro:phoxi_m_camera>
+  </xacro:macro>
 </robot>

Commit message: Confirmed that real KHI robot works

File: aist_description/devices/urdf/magripper.urdf.xacro (robot description, xacro)
@@ -147,5 +147,5 @@
       </visual>
       <collision>
-        <origin xyz="$0 0 0" rpy="0 0 0" />
+        <origin xyz="0 0 0" rpy="0 0 0" />
         <geometry>
           <mesh filename="package://aist_description/devices/meshes/collision/magripper_base.stl" scale="0.001 0.001 0.001"/>

File: aist_description/devices/urdf/rs007l.urdf.xacro (robot description, xacro)
@@ -14,5 +14,5 @@
       <parent link="${prefix}link6"/>
       <child  link="${prefix}ee_link"/>
-      <origin xyz="0 0 0" rpy="${pi/2} ${-pi/2} 0"/>
+      <origin xyz="0 0 0" rpy="${pi} ${-pi/2} 0"/>
     </joint>
   </xacro:macro>
