Commit message: Changed finger frames of the LEHZ40K2 gripper

File: aist_description/devices/urdf/lehz40k2_30.urdf.xacro (robot description, xacro)
@@ -2,8 +2,8 @@
 <robot xmlns:xacro="http://ros.org/wiki/xacro">
   <xacro:macro name="lehz40k2_30"  params="prefix parent *origin">
-    <xacro:property name="length" value="0.1959"/>
-    <xacro:property name="x_offset" value="0.1084"/>
+    <xacro:property name="length"	   value="0.1959"/>
+    <xacro:property name="x_offset"	   value="0.1084"/>
     <xacro:property name="x_finger_offset" value="-0.0465"/>
-    <xacro:property name="z_offset" value="0.0238"/>
+    <xacro:property name="z_offset"	   value="0.0238"/>
     <!-- Body -->
     <joint name="${prefix}gripper_base_joint" type="fixed">
@@ -52,9 +52,9 @@
       <child  link="${prefix}l_finger_link"/>
       <axis xyz="0 -1 0"/>
-      <limit lower="0" upper="0.03125" effort="130" velocity="0.15"/>
+      <limit lower="0.015" upper="0.030" effort="130" velocity="0.15"/>
     </joint>
     <link name="${prefix}l_finger_link">
       <visual>
-        <origin xyz="${x_finger_offset} 0 ${z_offset}"
+        <origin xyz="${x_finger_offset} 0.015 ${z_offset}"
 		rpy="${pi/2} 0 ${pi/2}" />
         <geometry>
@@ -66,5 +66,5 @@
       </visual>
       <collision>
-        <origin xyz="${x_finger_offset} 0 ${z_offset}"
+        <origin xyz="${x_finger_offset} 0.015 ${z_offset}"
 		rpy="${pi/2} 0 ${pi/2}" />
         <geometry>
@@ -92,9 +92,9 @@
       <child  link="${prefix}r_finger_link"/>
       <axis xyz="0 1 0"/>
-      <limit lower="0" upper="0.03125" effort="130" velocity="0.15"/>
+      <limit lower="0.015" upper="0.030" effort="130" velocity="0.15"/>
     </joint>
     <link name="${prefix}r_finger_link">
       <visual>
-        <origin xyz="${x_finger_offset} 0 ${z_offset}"
+        <origin xyz="${x_finger_offset} -0.015 ${z_offset}"
 		rpy="${pi/2} 0 ${pi/2}" />
         <geometry>
@@ -106,5 +106,5 @@
       </visual>
       <collision>
-        <origin xyz="${x_finger_offset} 0 ${z_offset}"
+        <origin xyz="${x_finger_offset} -0.015 ${z_offset}"
 		rpy="${pi/2} 0 ${pi/2}" />
         <geometry>

Commit message: Change tip link of LEHZ40K2 gripper

File: aist_description/devices/urdf/lehz40k2_30.urdf.xacro (robot description, xacro)
@@ -3,4 +3,5 @@
   <xacro:macro name="lehz40k2_30"  params="prefix parent *origin">
     <xacro:property name="length"	   value="0.1959"/>
+    <xacro:property name="nail_length"	   value="0.1200"/>
     <xacro:property name="x_offset"	   value="0.1084"/>
     <xacro:property name="x_finger_offset" value="-0.0465"/>
@@ -43,5 +44,5 @@
       <parent link="${prefix}gripper_base_link"/>
       <child  link="${prefix}gripper_link"/>
-      <origin xyz="${length} 0 0" rpy="0 0 0"/>
+      <origin xyz="${length + nail_length} 0 0" rpy="0 0 0"/>
     </joint>
     <link name="${prefix}gripper_link"/>
