Commit message: Add ur10e configuration

File: aist_description/devices/urdf/robotiq_140_gripper_with_tip_link.urdf.xacro (robot description, xacro)
@@ -15,5 +15,5 @@
       <parent link="${prefix}robotiq_140_base_link"/>
       <child link="${prefix}robotiq_140_tip_link"/>
-      <origin rpy="0.0 0.0 0.0" xyz=".163 0.0 0.0"/>
+      <origin rpy="0.0 0.0 0.0" xyz=".233 0.0 0.0"/>
     </joint>
   </xacro:macro>

File: aist_description/scenes/urdf/ur10e_base_scene.urdf.xacro (robot description, xacro)
@@ -43,9 +43,9 @@
   </joint>
   <!-- Spawn and attach gripper -->
-  <xacro:include filename="$(find aist_description)/devices/urdf/robotiq_85_gripper_with_tip_link.urdf.xacro"/>
-  <xacro:robotiq_85_gripper_with_tip_link prefix="a_bot_"
-					  parent="a_bot_ee_link">
+  <xacro:include filename="$(find aist_description)/devices/urdf/robotiq_140_gripper_with_tip_link.urdf.xacro"/>
+  <xacro:robotiq_140_gripper_with_tip_link prefix="a_bot_"
+					   parent="a_bot_ee_link">
     <origin xyz="0 0 0" rpy="0 0 0"/>
-  </xacro:robotiq_85_gripper_with_tip_link>
+  </xacro:robotiq_140_gripper_with_tip_link>
   <!-- I would like to remove the "world" link definition, but apparently it is necessary for Gazebo -->
   <link name="world"/>
