Commit message: Add missing launch file for calibration under ur10e econfiguration

File: aist_description/devices/urdf/_d435.urdf.xacro (robot description, xacro)
@@ -6,49 +6,50 @@
 aluminum peripherial evaluation case.
 -->
-<robot name="sensor_d435" xmlns:xacro="http://wiki.ros.org/xacro">
-  <xacro:macro name="sensor_d435" params="prefix parent *origin">
+<robot name="sensor_d435" xmlns:xacro="http://ros.org/wiki/xacro">
+  <!-- Includes -->
+  <xacro:include filename="$(find realsense2_description)/urdf/_materials.urdf.xacro" />
+  <xacro:macro name="sensor_d435" params="parent *origin prefix">
     <xacro:property name="M_PI" value="3.1415926535897931" />
     <!-- The following values are approximate, and the camera node
-    publishing TF values with actual calibrated camera extrinsic values -->
-    <xacro:property name="d435_cam_depth_to_left_ir_offset" value="-0.025"/>
-    <xacro:property name="d435_cam_depth_to_right_ir_offset" value="0.025"/>
-    <xacro:property name="d435_cam_depth_to_fisheye_offset" value="0.040"/>
+     publishing TF values with actual calibrated camera extrinsic values -->
+    <xacro:property name="d435_cam_depth_to_infra1_offset" value="0.0"/>
+    <xacro:property name="d435_cam_depth_to_infra2_offset" value="-0.050"/>
+    <xacro:property name="d435_cam_depth_to_color_offset" value="0.015"/>
     <!-- The following values model the aluminum peripherial case for the
-      D435 camera, with the camera joint represented by the actual
-      peripheral camera tripod mount -->
+  	D435 camera, with the camera joint represented by the actual
+  	peripherial camera tripod mount -->
     <xacro:property name="d435_cam_width" value="0.090"/>
     <xacro:property name="d435_cam_height" value="0.025"/>
     <xacro:property name="d435_cam_depth" value="0.02505"/>
     <xacro:property name="d435_cam_mount_from_center_offset" value="0.0149"/>
-    <!-- The following offset is relative to the physical D435 camera peripherial
-      camera tripod mount -->
+    <!-- The following offset is relative the the physical D435 camera peripherial
+  	camera tripod mount -->
     <xacro:property name="d435_cam_depth_px" value="${d435_cam_mount_from_center_offset}"/>
-    <xacro:property name="d435_cam_depth_py" value="-0.0075"/>
+    <xacro:property name="d435_cam_depth_py" value="0.0175"/>
     <xacro:property name="d435_cam_depth_pz" value="${d435_cam_height/2}"/>
-    <!-- <material name="aluminum"> -->
-    <!--   <color rgba="0.5 0.5 0.5 1"/> -->
-    <!-- </material> -->
     <!-- camera body, with origin at bottom screw mount -->
     <joint name="${prefix}camera_joint" type="fixed">
       <xacro:insert_block name="origin" />
       <parent link="${parent}"/>
+      <child link="${prefix}camera_bottom_screw_frame" />
+    </joint>
+    <link name="${prefix}camera_bottom_screw_frame"/>
+    <joint name="${prefix}camera_link_joint" type="fixed">
+      <origin xyz="0 ${d435_cam_depth_py} ${d435_cam_depth_pz}" rpy="0 0 0"/>
+      <parent link="${prefix}camera_bottom_screw_frame"/>
       <child link="${prefix}camera_link" />
     </joint>
     <link name="${prefix}camera_link">
       <visual>
-      <origin xyz="${d435_cam_mount_from_center_offset} 0.0 ${d435_cam_height/2}" rpy="${M_PI/2} 0 ${M_PI/2}"/>
+        <origin xyz="${d435_cam_mount_from_center_offset} ${-d435_cam_depth_py} 0" rpy="${M_PI/2} 0 ${M_PI/2}"/>
         <geometry>
           <!-- <box size="${d435_cam_width} ${d435_cam_height} ${d435_cam_depth}"/> -->
-	        <mesh filename="package://realsense2_description/meshes/d435.dae" />
+	  <mesh filename="package://realsense2_description/meshes/d435.dae" />
         </geometry>
-	<material name="aluminum">
-	  <color rgba="0.5 0.5 0.5 1"/>
-	</material>
-        <!-- <material name="aluminum"/> -->
       </visual>
       <collision>
-        <origin xyz="0.0 0.0 ${d435_cam_height/2}" rpy="0 0 0"/>
+        <origin xyz="0 ${-d435_cam_depth_py} 0" rpy="0 0 0"/>
         <geometry>
-        <box size="${d435_cam_depth} ${d435_cam_width} ${d435_cam_height}"/>
+          <box size="${d435_cam_depth} ${d435_cam_width} ${d435_cam_height}"/>
         </geometry>
       </collision>
@@ -62,5 +63,5 @@
     <!-- camera depth joints and links -->
     <joint name="${prefix}camera_depth_joint" type="fixed">
-      <origin xyz="${d435_cam_depth_px} ${d435_cam_depth_py} ${d435_cam_depth_pz}" rpy="0 0 0"/>
+      <origin xyz="0 0 0" rpy="0 0 0"/>
       <parent link="${prefix}camera_link"/>
       <child link="${prefix}camera_depth_frame" />
@@ -74,42 +75,42 @@
     <link name="${prefix}camera_depth_optical_frame"/>
     <!-- camera left IR joints and links -->
-    <joint name="${prefix}camera_left_ir_joint" type="fixed">
-      <origin xyz="0 ${d435_cam_depth_to_left_ir_offset} 0" rpy="0 0 0" />
-      <parent link="${prefix}camera_depth_frame" />
-      <child link="${prefix}camera_left_ir_frame" />
+    <joint name="${prefix}camera_infra1_joint" type="fixed">
+      <origin xyz="0 ${d435_cam_depth_to_infra1_offset} 0" rpy="0 0 0" />
+      <parent link="${prefix}camera_link" />
+      <child link="${prefix}camera_infra1_frame" />
     </joint>
-    <link name="${prefix}camera_left_ir_frame"/>
-    <joint name="${prefix}camera_left_ir_optical_joint" type="fixed">
+    <link name="${prefix}camera_infra1_frame"/>
+    <joint name="${prefix}camera_infra1_optical_joint" type="fixed">
       <origin xyz="0 0 0" rpy="${-M_PI/2} 0 ${-M_PI/2}" />
-      <parent link="${prefix}camera_left_ir_frame" />
-      <child link="${prefix}camera_left_ir_optical_frame" />
+      <parent link="${prefix}camera_infra1_frame" />
+      <child link="${prefix}camera_infra1_optical_frame" />
     </joint>
-    <link name="${prefix}camera_left_ir_optical_frame"/>
+    <link name="${prefix}camera_infra1_optical_frame"/>
     <!-- camera right IR joints and links -->
-    <joint name="${prefix}camera_right_ir_joint" type="fixed">
-      <origin xyz="0 ${d435_cam_depth_to_right_ir_offset} 0" rpy="0 0 0" />
-      <parent link="${prefix}camera_depth_frame" />
-      <child link="${prefix}camera_right_ir_frame" />
+    <joint name="${prefix}camera_infra2_joint" type="fixed">
+      <origin xyz="0 ${d435_cam_depth_to_infra2_offset} 0" rpy="0 0 0" />
+      <parent link="${prefix}camera_link" />
+      <child link="${prefix}camera_infra2_frame" />
     </joint>
-    <link name="${prefix}camera_right_ir_frame"/>
-    <joint name="${prefix}camera_right_ir_optical_joint" type="fixed">
+    <link name="${prefix}camera_infra2_frame"/>
+    <joint name="${prefix}camera_infra2_optical_joint" type="fixed">
       <origin xyz="0 0 0" rpy="${-M_PI/2} 0 ${-M_PI/2}" />
-      <parent link="${prefix}camera_right_ir_frame" />
-      <child link="${prefix}camera_right_ir_optical_frame" />
+      <parent link="${prefix}camera_infra2_frame" />
+      <child link="${prefix}camera_infra2_optical_frame" />
     </joint>
-    <link name="${prefix}camera_right_ir_optical_frame"/>
-    <!-- camera fisheye joints and links -->
-    <joint name="${prefix}camera_fisheye_joint" type="fixed">
-      <origin xyz="0 ${d435_cam_depth_to_fisheye_offset} 0" rpy="0 0 0" />
-      <parent link="${prefix}camera_depth_frame" />
-      <child link="${prefix}camera_fisheye_frame" />
+    <link name="${prefix}camera_infra2_optical_frame"/>
+    <!-- camera color joints and links -->
+    <joint name="${prefix}camera_color_joint" type="fixed">
+      <origin xyz="0 ${d435_cam_depth_to_color_offset} 0" rpy="0 0 0" />
+      <parent link="${prefix}camera_link" />
+      <child link="${prefix}camera_color_frame" />
     </joint>
-    <link name="${prefix}camera_fisheye_frame"/>
-    <joint name="${prefix}camera_fisheye_optical_joint" type="fixed">
+    <link name="${prefix}camera_color_frame"/>
+    <joint name="${prefix}camera_color_optical_joint" type="fixed">
       <origin xyz="0 0 0" rpy="${-M_PI/2} 0 ${-M_PI/2}" />
-      <parent link="${prefix}camera_fisheye_frame" />
-      <child link="${prefix}camera_fisheye_optical_frame" />
+      <parent link="${prefix}camera_color_frame" />
+      <child link="${prefix}camera_color_optical_frame" />
     </joint>
-    <link name="${prefix}camera_fisheye_optical_frame"/>
+    <link name="${prefix}camera_color_optical_frame"/>
     <gazebo reference="${prefix}camera_depth_frame">
       <sensor type="depth" name="${prefix}camera">
@@ -117,5 +118,5 @@
 	<visualize>true</visualize>
 	<camera>
-          <horizontal_fov>1.047</horizontal_fov>
+          <horizontal_fov>1.034</horizontal_fov>
           <image>
             <width>640</width>
@@ -142,5 +143,5 @@
           <depthImageCameraInfoTopicName>depth/camera_info</depthImageCameraInfoTopicName>
           <pointCloudTopicName>depth/points</pointCloudTopicName>
-          <pointCloudCutoff>0.4</pointCloudCutoff>
+          <pointCloudCutoff>0.1</pointCloudCutoff>
           <!-- <hackBaseline>0.07</hackBaseline> -->
           <distortionK1>0.0</distortionK1>

File: aist_description/scenes/urdf/ur10e_base_scene.urdf.xacro (robot description, xacro)
@@ -1,5 +1,5 @@
 <?xml version="1.0"?>
 <robot xmlns:xacro="http://wiki.ros.org/xacro" name="ur10e_base_scene" >
-  <xacro:arg name="scene" default=""/>
+  <xacro:arg name="scene" default="ur10e_calibration"/>
   <!-- Calibration help: If the robot is not moving far enough to the calibration point, increase these distances -->
   <xacro:property name="a_bot_x" value="0"/>
@@ -48,4 +48,8 @@
     <origin xyz="0 0 0" rpy="0 0 0"/>
   </xacro:robotiq_140_gripper_with_tip_link>
+  <!-- Add RealSense camera -->
+  <xacro:include filename="$(find aist_description
+			   )/devices/urdf/wrist_d435.urdf.xacro" />
+  <xacro:wrist_d435 prefix="a_bot_" parent="a_bot_robotiq_140_base_link"/>
   <!-- I would like to remove the "world" link definition, but apparently it is necessary for Gazebo -->
   <link name="world"/>

Commit message: Setup handeye calibration for mocap configuration

File: aist_description/devices/urdf/_d435.urdf.xacro (robot description, xacro)
@@ -7,112 +7,14 @@
 -->
 <robot name="sensor_d435" xmlns:xacro="http://ros.org/wiki/xacro">
-  <!-- Includes -->
-  <xacro:include filename="$(find realsense2_description)/urdf/_materials.urdf.xacro" />
-  <xacro:macro name="sensor_d435" params="parent *origin prefix">
-    <xacro:property name="M_PI" value="3.1415926535897931" />
-    <!-- The following values are approximate, and the camera node
-     publishing TF values with actual calibrated camera extrinsic values -->
-    <xacro:property name="d435_cam_depth_to_infra1_offset" value="0.0"/>
-    <xacro:property name="d435_cam_depth_to_infra2_offset" value="-0.050"/>
-    <xacro:property name="d435_cam_depth_to_color_offset" value="0.015"/>
-    <!-- The following values model the aluminum peripherial case for the
-  	D435 camera, with the camera joint represented by the actual
-  	peripherial camera tripod mount -->
-    <xacro:property name="d435_cam_width" value="0.090"/>
-    <xacro:property name="d435_cam_height" value="0.025"/>
-    <xacro:property name="d435_cam_depth" value="0.02505"/>
-    <xacro:property name="d435_cam_mount_from_center_offset" value="0.0149"/>
-    <!-- The following offset is relative the the physical D435 camera peripherial
-  	camera tripod mount -->
-    <xacro:property name="d435_cam_depth_px" value="${d435_cam_mount_from_center_offset}"/>
-    <xacro:property name="d435_cam_depth_py" value="0.0175"/>
-    <xacro:property name="d435_cam_depth_pz" value="${d435_cam_height/2}"/>
-    <!-- camera body, with origin at bottom screw mount -->
-    <joint name="${prefix}camera_joint" type="fixed">
-      <xacro:insert_block name="origin" />
-      <parent link="${parent}"/>
-      <child link="${prefix}camera_bottom_screw_frame" />
-    </joint>
-    <link name="${prefix}camera_bottom_screw_frame"/>
-    <joint name="${prefix}camera_link_joint" type="fixed">
-      <origin xyz="0 ${d435_cam_depth_py} ${d435_cam_depth_pz}" rpy="0 0 0"/>
-      <parent link="${prefix}camera_bottom_screw_frame"/>
-      <child link="${prefix}camera_link" />
-    </joint>
-    <link name="${prefix}camera_link">
-      <visual>
-        <origin xyz="${d435_cam_mount_from_center_offset} ${-d435_cam_depth_py} 0" rpy="${M_PI/2} 0 ${M_PI/2}"/>
-        <geometry>
-          <!-- <box size="${d435_cam_width} ${d435_cam_height} ${d435_cam_depth}"/> -->
-	  <mesh filename="package://realsense2_description/meshes/d435.dae" />
-        </geometry>
-      </visual>
-      <collision>
-        <origin xyz="0 ${-d435_cam_depth_py} 0" rpy="0 0 0"/>
-        <geometry>
-          <box size="${d435_cam_depth} ${d435_cam_width} ${d435_cam_height}"/>
-        </geometry>
-      </collision>
-      <inertial>
-        <!-- The following are not reliable values, and should not be used for modeling -->
-        <mass value="0.564" />
-        <origin xyz="0 0 0" />
-        <inertia ixx="0.003881243" ixy="0.0" ixz="0.0" iyy="0.000498940" iyz="0.0" izz="0.003879257" />
-      </inertial>
-    </link>
-    <!-- camera depth joints and links -->
-    <joint name="${prefix}camera_depth_joint" type="fixed">
-      <origin xyz="0 0 0" rpy="0 0 0"/>
-      <parent link="${prefix}camera_link"/>
-      <child link="${prefix}camera_depth_frame" />
-    </joint>
-    <link name="${prefix}camera_depth_frame"/>
-    <joint name="${prefix}camera_depth_optical_joint" type="fixed">
-      <origin xyz="0 0 0" rpy="${-M_PI/2} 0 ${-M_PI/2}" />
-      <parent link="${prefix}camera_depth_frame" />
-      <child link="${prefix}camera_depth_optical_frame" />
-    </joint>
-    <link name="${prefix}camera_depth_optical_frame"/>
-    <!-- camera left IR joints and links -->
-    <joint name="${prefix}camera_infra1_joint" type="fixed">
-      <origin xyz="0 ${d435_cam_depth_to_infra1_offset} 0" rpy="0 0 0" />
-      <parent link="${prefix}camera_link" />
-      <child link="${prefix}camera_infra1_frame" />
-    </joint>
-    <link name="${prefix}camera_infra1_frame"/>
-    <joint name="${prefix}camera_infra1_optical_joint" type="fixed">
-      <origin xyz="0 0 0" rpy="${-M_PI/2} 0 ${-M_PI/2}" />
-      <parent link="${prefix}camera_infra1_frame" />
-      <child link="${prefix}camera_infra1_optical_frame" />
-    </joint>
-    <link name="${prefix}camera_infra1_optical_frame"/>
-    <!-- camera right IR joints and links -->
-    <joint name="${prefix}camera_infra2_joint" type="fixed">
-      <origin xyz="0 ${d435_cam_depth_to_infra2_offset} 0" rpy="0 0 0" />
-      <parent link="${prefix}camera_link" />
-      <child link="${prefix}camera_infra2_frame" />
-    </joint>
-    <link name="${prefix}camera_infra2_frame"/>
-    <joint name="${prefix}camera_infra2_optical_joint" type="fixed">
-      <origin xyz="0 0 0" rpy="${-M_PI/2} 0 ${-M_PI/2}" />
-      <parent link="${prefix}camera_infra2_frame" />
-      <child link="${prefix}camera_infra2_optical_frame" />
-    </joint>
-    <link name="${prefix}camera_infra2_optical_frame"/>
-    <!-- camera color joints and links -->
-    <joint name="${prefix}camera_color_joint" type="fixed">
-      <origin xyz="0 ${d435_cam_depth_to_color_offset} 0" rpy="0 0 0" />
-      <parent link="${prefix}camera_link" />
-      <child link="${prefix}camera_color_frame" />
-    </joint>
-    <link name="${prefix}camera_color_frame"/>
-    <joint name="${prefix}camera_color_optical_joint" type="fixed">
-      <origin xyz="0 0 0" rpy="${-M_PI/2} 0 ${-M_PI/2}" />
-      <parent link="${prefix}camera_color_frame" />
-      <child link="${prefix}camera_color_optical_frame" />
-    </joint>
-    <link name="${prefix}camera_color_optical_frame"/>
-    <gazebo reference="${prefix}camera_depth_frame">
-      <sensor type="depth" name="${prefix}camera">
+  <xacro:macro name="sensor_d435"
+  	       params="parent *origin name:=camera use_nominal_extrinsics:=false">
+    <xacro:include filename="$(find realsense2_description
+			     )/urdf/_d435.urdf.xacro" />
+    <xacro:sensor_d435 parent="${parent}" name="${name}"
+		       use_nominal_extrinsics="${use_nominal_extrinsics}">
+      <xacro:insert_block name="origin"/>
+    </xacro:sensor_d435>
+    <gazebo reference="${name}_depth_frame">
+      <sensor type="depth" name="${name}">
 	<always_on>true</always_on>
 	<visualize>true</visualize>
@@ -131,11 +33,11 @@
           </clip>
 	</camera>
-	<plugin name="${prefix}cam_controller"
+	<plugin name="${name}_controller"
 		filename="libgazebo_ros_openni_kinect.so">
           <baseline>0.2</baseline>
           <alwaysOn>true</alwaysOn>
           <updateRate>10.0</updateRate>
-          <cameraName>${prefix}camera</cameraName>
-          <frameName>${prefix}camera_color_optical_frame</frameName>
+          <cameraName>${name}</cameraName>
+          <frameName>${name}_color_optical_frame</frameName>
           <imageTopicName>color/image_raw</imageTopicName>
           <cameraInfoTopicName>color/camera_info</cameraInfoTopicName>

File: aist_description/scenes/urdf/aist_calibration.urdf.xacro (robot description, xacro)
@@ -1,4 +1,4 @@
 <?xml version="1.0"?>
-<robot xmlns:xacro="http://wiki.ros.org/xacro" name="calibration">
+<robot xmlns:xacro="http://wiki.ros.org/xacro" name="aist_calibration">
   <!-- Add AR markers -->
   <xacro:include filename="$(find aist_description)/objects/urdf/ar_markers.urdf.xacro"/>

File: aist_description/scenes/urdf/mocap_base_scene.urdf.xacro (robot description, xacro)
@@ -41,9 +41,18 @@
   </joint>
   <!-- Spawn and attach gripper -->
-  <xacro:include filename="$(find aist_description)/devices/urdf/robotiq_85_gripper_with_tip_link.urdf.xacro"/>
+  <xacro:include filename="$(find aist_description
+			   )/devices/urdf/robotiq_85_gripper_with_tip_link.urdf.xacro"/>
   <xacro:robotiq_85_gripper_with_tip_link prefix="c_bot_"
 					  parent="c_bot_ee_link">
     <origin xyz="0 0 0" rpy="0 0 0"/>
   </xacro:robotiq_85_gripper_with_tip_link>
+  <!-- Add RealSense camera -->
+  <xacro:include filename="$(find aist_description
+			   )/devices/urdf/_d435.urdf.xacro"/>
+  <xacro:sensor_d435 name="realsenseD435" parent="workspace_center"
+		     use_nominal_extrinsics="true">
+    <origin xyz="0.0 0.7 0.6"
+	    rpy="${0*pi/180} ${30*pi/180} ${-90*pi/180}"/>
+  </xacro:sensor_d435>
   <!-- I would like to remove the "world" link definition, but apparently it is necessary for Gazebo -->
   <link name="world"/>
