Commit message: Make indivisual scene urdf file included into base_scene urdf file

File: aist_description/objects/urdf/ar_markers.urdf.xacro (robot description, xacro)
@@ -23,5 +23,5 @@
     </link>
     <!-- For Gazebo, material of AR marker is defined in
-         aist_gazebo/media/material. You also need to export
+         aist_description/media/material. You also need to export
          gazebo_media_path in package.xml. -->
     <gazebo reference="${prefix}ar_marker">

File: aist_description/scenes/urdf/aist_base_scene.urdf.xacro (robot description, xacro)
@@ -1,4 +1,5 @@
 <?xml version="1.0"?>
 <robot xmlns:xacro="http://wiki.ros.org/xacro" name="aist_base_scene" >
+  <xacro:arg name="scene" default=""/>
   <!-- Calibration help: If the robot is not moving far enough to the calibration point, increase these distances -->
   <xacro:property name="a_bot_x" value="0"/>
@@ -106,3 +107,9 @@
     <origin xyz="0 0 0" rpy="0 0 0"/>
   </joint>
+  <!-- Include indivisual scene file -->
+  <xacro:property name="scene_name" value="$(arg scene)"/>
+  <xacro:if value="${scene_name != ''}">
+    <xacro:include filename="$(find aist_description)/scenes/urdf/$(arg
+			     scene).urdf.xacro"/>
+  </xacro:if>
 </robot>

File: aist_description/scenes/urdf/calibration.urdf.xacro (robot description, xacro)
@@ -1,5 +1,4 @@
 <?xml version="1.0"?>
-<robot xmlns:xacro="http://wiki.ros.org/xacro" name="aist_calibration">
-  <xacro:include filename="$(find aist_description)/scenes/urdf/aist_base_scene.urdf.xacro"/>
+<robot xmlns:xacro="http://wiki.ros.org/xacro" name="calibration">
   <!-- Add AR markers -->
   <xacro:include filename="$(find aist_description)/objects/urdf/ar_markers.urdf.xacro"/>

File: aist_description/scenes/urdf/ceatec.urdf.xacro (robot description, xacro)
@@ -1,6 +1,4 @@
 <?xml version="1.0"?>
 <robot xmlns:xacro="http://wiki.ros.org/xacro" name="ceatec" >
-  <!-- Fetch robot in empty scene (root = "map") -->
-  <xacro:include filename="$(find aist_description)/scenes/urdf/fetch_base_scene.urdf.xacro"/>
   <!-- Environment of "ceatec" scene (root = "world") -->
   <xacro:include filename="$(find aist_description)/scenes/urdf/ceatec_environment.urdf.xacro"/>

File: aist_description/scenes/urdf/diiwa_base_scene.urdf.xacro (robot description, xacro)
@@ -1,4 +1,5 @@
 <?xml version="1.0"?>
 <robot xmlns:xacro="http://wiki.ros.org/xacro" name="diiwa_base_scene" >
+  <xacro:arg name="scene"		default=""/>
   <xacro:arg name="hardware_interface"	default="PositionJointInterface"/>
   <!-- Calibration help: If the robot is not moving far enough to the calibration point, increase these distances -->
@@ -68,3 +69,9 @@
     <origin xyz="0 0 0" rpy="0 0 0"/>
   </joint>
+  <!-- Include indivisual scene file -->
+  <xacro:property name="scene_name" value="$(arg scene)"/>
+  <xacro:if value="${scene_name != ''}">
+    <xacro:include filename="$(find aist_description)/scenes/urdf/$(arg
+			     scene).urdf.xacro"/>
+  </xacro:if>
 </robot>

File: aist_description/scenes/urdf/dkhi_base_scene.urdf.xacro (robot description, xacro)
@@ -1,4 +1,5 @@
 <?xml version="1.0"?>
 <robot xmlns:xacro="http://wiki.ros.org/xacro" name="dkhi_base_scene" >
+  <xacro:arg name="scene" default=""/>
   <!-- Calibration help: If the robot is not moving far enough to the calibration point, increase these distances -->
   <xacro:property name="a_khi_x" value="0"/>
@@ -55,3 +56,9 @@
     <origin xyz="0 0 0" rpy="0 0 0"/>
   </joint>
+  <!-- Include indivisual scene file -->
+  <xacro:property name="scene_name" value="$(arg scene)"/>
+  <xacro:if value="${scene_name != ''}">
+    <xacro:include filename="$(find aist_description)/scenes/urdf/$(arg
+			     scene).urdf.xacro"/>
+  </xacro:if>
 </robot>

File: aist_description/scenes/urdf/dtorobo_base_scene.urdf.xacro (robot description, xacro)
@@ -1,4 +1,5 @@
 <?xml version="1.0"?>
 <robot xmlns:xacro="http://wiki.ros.org/xacro" name="dtorobo_base_scene" >
+  <xacro:arg name="scene" default=""/>
   <!-- Calibration help: If the robot is not moving far enough to the calibration point, increase these distances -->
   <xacro:property name="a_torobo_x" value="0"/>
@@ -62,3 +63,9 @@
     <origin xyz="0 0 0" rpy="0 0 0"/>
   </joint>
+  <!-- Include indivisual scene file -->
+  <xacro:property name="scene_name" value="$(arg scene)"/>
+  <xacro:if value="${scene_name != ''}">
+    <xacro:include filename="$(find aist_description)/scenes/urdf/$(arg
+			     scene).urdf.xacro"/>
+  </xacro:if>
 </robot>

File: aist_description/scenes/urdf/fetch_base_scene.urdf.xacro (robot description, xacro)
@@ -1,4 +1,5 @@
 <?xml version="1.0"?>
-<robot xmlns:xacro="http://wiki.ros.org/xacro" name="fetch_base_scene" >
+<robot xmlns:xacro="http://wiki.ros.org/xacro" name="fetch_base_scene">
+  <xacro:arg name="scene" default=""/>
   <!-- Fetch robot (root = "base_link") -->
   <xacro:include filename="$(find fetch_gazebo)/robots/fetch.gazebo.xacro"/>
@@ -15,3 +16,9 @@
     <axis   xyz="0 0 1"/>
   </joint>
+  <!-- Include indivisual scene file -->
+  <xacro:property name="scene_name" value="$(arg scene)"/>
+  <xacro:if value="${scene_name != ''}">
+    <xacro:include filename="$(find aist_description)/scenes/urdf/$(arg
+			     scene).urdf.xacro"/>
+  </xacro:if>
 </robot>

File: aist_description/scenes/urdf/kitting.urdf.xacro (robot description, xacro)
@@ -1,5 +1,4 @@
 <?xml version="1.0"?>
-<robot xmlns:xacro="http://wiki.ros.org/xacro" name="pgrp_kitting">
-  <xacro:include filename="$(find aist_description)/scenes/urdf/pgrp_base_scene.urdf.xacro"/>
+<robot xmlns:xacro="http://wiki.ros.org/xacro" name="kitting">
   <xacro:property name="plate_w" value="0.68"/>
   <xacro:property name="plate_l" value="0.42"/>

File: aist_description/scenes/urdf/mocap_base_scene.urdf.xacro (robot description, xacro)
@@ -1,5 +1,5 @@
 <?xml version="1.0"?>
-<robot xmlns:xacro="http://wiki.ros.org/xacro"
-        name="mocap_base_scene" >
+<robot xmlns:xacro="http://wiki.ros.org/xacro" name="mocap_base_scene">
+  <xacro:arg name="scene" default=""/>
   <!-- Calibration help: If the robot is not moving far enough to the calibration point, increase these distances -->
   <xacro:property name="c_bot_x" value="0"/>
@@ -64,3 +64,9 @@
     <origin xyz="0 0 0" rpy="0 0 0"/>
   </joint>
+  <!-- Include indivisual scene file -->
+  <xacro:property name="scene_name" value="$(arg scene)"/>
+  <xacro:if value="${scene_name != ''}">
+    <xacro:include filename="$(find aist_description)/scenes/urdf/$(arg
+			     scene).urdf.xacro"/>
+  </xacro:if>
 </robot>

File: aist_description/scenes/urdf/pgrp_base_scene.urdf.xacro (robot description, xacro)
@@ -1,4 +1,5 @@
 <?xml version="1.0"?>
 <robot xmlns:xacro="http://wiki.ros.org/xacro" name="pgrp_base_scene" >
+  <xacro:arg name="scene" default=""/>
   <!-- Calibration help: If the robot is not moving far enough to the calibration point, increase these distances -->
   <xacro:property name="a_bot_x" value="0"/>
@@ -108,3 +109,9 @@
     <origin xyz="0 0 0" rpy="0 0 0"/>
   </joint>
+  <!-- Include indivisual scene file -->
+  <xacro:property name="scene_name" value="$(arg scene)"/>
+  <xacro:if value="${scene_name != ''}">
+    <xacro:include filename="$(find aist_description)/scenes/urdf/$(arg
+			     scene).urdf.xacro"/>
+  </xacro:if>
 </robot>

File: aist_description/scenes/urdf/skhi_base_scene.urdf.xacro (robot description, xacro)
@@ -1,4 +1,5 @@
 <?xml version="1.0"?>
 <robot xmlns:xacro="http://wiki.ros.org/xacro" name="skhi_base_scene" >
+  <xacro:arg name="scene" default=""/>
   <!-- Calibration help: If the robot is not moving far enough to the calibration point, increase these distances -->
   <xacro:property name="a_khi_x" value="0"/>
@@ -50,3 +51,9 @@
     <origin xyz="0 0 0" rpy="0 0 0"/>
   </joint>
+  <!-- Include indivisual scene file -->
+  <xacro:property name="scene_name" value="$(arg scene)"/>
+  <xacro:if value="${scene_name != ''}">
+    <xacro:include filename="$(find aist_description)/scenes/urdf/$(arg
+			     scene).urdf.xacro"/>
+  </xacro:if>
 </robot>

File: aist_description/scenes/urdf/ur5e_base_scene.urdf.xacro (robot description, xacro)
@@ -1,4 +1,5 @@
 <?xml version="1.0"?>
 <robot xmlns:xacro="http://wiki.ros.org/xacro" name="ur5e_base_scene" >
+  <xacro:arg name="scene" default=""/>
   <!-- Calibration help: If the robot is not moving far enough to the calibration point, increase these distances -->
   <xacro:property name="c_bot_x" value="0"/>
@@ -94,3 +95,9 @@
     <origin xyz="0 0 0" rpy="0 0 0"/>
   </joint>
+  <!-- Include indivisual scene file -->
+  <xacro:property name="scene_name" value="$(arg scene)"/>
+  <xacro:if value="${scene_name != ''}">
+    <xacro:include filename="$(find aist_description)/scenes/urdf/$(arg
+			     scene).urdf.xacro"/>
+  </xacro:if>
 </robot>
