Commit message: Add transparency flag to aist_box xacro

File: aist_description/objects/urdf/aist_box.urdf.xacro (robot description, xacro)
@@ -2,6 +2,15 @@
 <robot xmlns:xacro="http://wiki.ros.org/xacro">
   <xacro:macro name="aist_box"
-	       params="name width length height parent *origin">
+	       params="name width length height parent transparent:=false
+		       *origin">
     <!-- This creates a box with the origin in the bottom corner, fixed to the world link. -->
+    <xacro:unless value="${transparent}">
+      <xacro:property name="rgba"	value="0.7 0.7 0.7 1"/>
+      <xacro:property name="color_name" value="Grey"/>
+    </xacro:unless>
+    <xacro:if value="${transparent}">
+      <xacro:property name="rgba"	value="0 0 0 0"/>
+      <xacro:property name="color_name"	value="Transparent"/>
+    </xacro:if>
     <link name="${name}">
       <!-- w is in x, l is in y, h is in z -->
@@ -11,6 +20,6 @@
           <box size="${width} ${length} ${height}"/>
         </geometry>
-        <material name="Grey">
-          <color rgba="0.7 0.7 0.7 1.0"/>
+        <material name="${color_name}">
+          <color rgba="${rgba}"/>
         </material>
       </visual>
@@ -29,5 +38,5 @@
     </link>
     <gazebo reference="${name}">
-      <material>Gazebo/Grey</material>
+      <material>Gazebo/${color_name}</material>
     </gazebo>
     <joint name="${name}" type="fixed">

File: aist_description/scenes/urdf/aist_base_scene.urdf.xacro (robot description, xacro)
@@ -77,5 +77,5 @@
   <!-- Add virtual wall to avoid collisions-->
   <xacro:aist_box name="vwall1" width="0.01" length="0.3" height="0.5"
-		  parent="ground">
+		  parent="ground" transparent="true">
     <origin xyz="0.45 -0.15 ${bots_z}" rpy="0 0 0"/>
   </xacro:aist_box>
