Commit message: Reorganize package

File: aist_robotiq/urdf/robotiq_85_gripper.urdf.xacro (robot description, xacro)
@@ -1,22 +1,16 @@
 <?xml version="1.0"?>
 <robot xmlns:xacro="http://ros.org/wiki/xacro">
-  <xacro:include filename="$(find aist_robotiq_description)/urdf/robotiq_arg2f_transmission.xacro" />
+  <xacro:include filename="$(find aist_robotiq)/urdf/robotiq_arg2f_transmission.xacro" />
   <xacro:macro name="outer_knuckle" params="prefix fingerprefix stroke">
     <link name="${prefix}${fingerprefix}_outer_knuckle">
-      <inertial>
+      <!--<inertial>
         <origin xyz="-0.000200000000003065 0.0199435877845359 0.0292245259211331" rpy="0 0 0" />
         <mass value="0.00853198276973456" />
-        <inertia
-            ixx="2.89328108496468E-06"
-            ixy="-1.57935047237397E-19"
-            ixz="-1.93980378593255E-19"
-            iyy="1.86719750325683E-06"
-            iyz="-1.21858577871576E-06"
-            izz="1.21905238907251E-06" />
-      </inertial>
-      <visual>
-        <origin xyz="0 0 0" rpy="0 0 0" />
-        <geometry>
-          <mesh filename="package://aist_robotiq_description/meshes/visual/robotiq_arg2f_${stroke}_outer_knuckle.stl" />
+        <inertia ixx="2.89328108496468E-06" ixy="-1.57935047237397E-19" ixz="-1.93980378593255E-19" iyy="1.86719750325683E-06" iyz="-1.21858577871576E-06" izz="1.21905238907251E-06" />
+        </inertial> -->
+      <visual>
+        <origin xyz="0 0 0" rpy="0 0 0" />
+        <geometry>
+          <mesh filename="package://aist_robotiq/meshes/visual/robotiq_arg2f_85_outer_knuckle.dae" scale="0.001 0.001 0.001"/>
         </geometry>
         <material name="">
@@ -27,5 +21,5 @@
         <origin xyz="0 0 0" rpy="0 0 0" />
         <geometry>
-          <mesh filename="package://aist_robotiq_description/meshes/collision/robotiq_arg2f_${stroke}_outer_knuckle.stl" />
+          <mesh filename="package://aist_robotiq/meshes/collision/robotiq_arg2f_85_outer_knuckle.dae" scale="0.001 0.001 0.001"/>
         </geometry>
       </collision>
@@ -37,19 +31,13 @@
   <xacro:macro name="outer_finger" params="prefix fingerprefix stroke">
     <link name="${prefix}${fingerprefix}_outer_finger">
-      <inertial>
+      <!--<inertial>
         <origin xyz="0.00030115855001899 0.0373907951953854 -0.0208027427000385" rpy="0 0 0" />
         <mass value="0.022614240507152" />
-        <inertia
-            ixx="1.52518312458174E-05"
-            ixy="9.76583423954399E-10"
-            ixz="-5.43838577022588E-10"
-            iyy="6.17694243867776E-06"
-            iyz="6.78636130740228E-06"
-            izz="1.16494917907219E-05" />
-      </inertial>
-      <visual>
-        <origin xyz="0 0 0" rpy="0 0 0" />
-        <geometry>
-          <mesh filename="package://aist_robotiq_description/meshes/visual/robotiq_arg2f_${stroke}_outer_finger.stl" />
+        <inertia ixx="1.52518312458174E-05" ixy="9.76583423954399E-10" ixz="-5.43838577022588E-10" iyy="6.17694243867776E-06" iyz="6.78636130740228E-06" izz="1.16494917907219E-05" />
+        </inertial> -->
+      <visual>
+        <origin xyz="0 0 0" rpy="0 0 0" />
+        <geometry>
+          <mesh filename="package://aist_robotiq/meshes/visual/robotiq_arg2f_85_outer_finger.dae" scale="0.001 0.001 0.001"/>
         </geometry>
         <material name="">
@@ -60,5 +48,5 @@
         <origin xyz="0 0 0" rpy="0 0 0" />
         <geometry>
-          <mesh filename="package://aist_robotiq_description/meshes/collision/robotiq_arg2f_${stroke}_outer_finger.stl" />
+          <mesh filename="package://aist_robotiq/meshes/collision/robotiq_arg2f_85_outer_finger.dae" scale="0.001 0.001 0.001"/>
         </geometry>
       </collision>
@@ -70,19 +58,13 @@
   <xacro:macro name="inner_knuckle" params="prefix fingerprefix stroke">
     <link name="${prefix}${fingerprefix}_inner_knuckle">
-      <inertial>
+      <!--<inertial>
         <origin xyz="0.000123011831763771 0.0507850843201817 0.00103968640075166" rpy="0 0 0" />
-        <mass value="0.0271177346495152" />
-        <inertia
-            ixx="2.61910379223783E-05"
-            ixy="-2.43616858946494E-07"
-            ixz="-6.37789906117123E-09"
-            iyy="2.8270243746167E-06"
-            iyz="-5.37200748039765E-07"
-            izz="2.83695868220296E-05" />
-      </inertial>
-      <visual>
-        <origin xyz="0 0 0" rpy="0 0 0" />
-        <geometry>
-          <mesh filename="package://aist_robotiq_description/meshes/visual/robotiq_arg2f_${stroke}_inner_knuckle.stl" />
+       <mass value="0.0271177346495152" />
+        <inertia ixx="2.61910379223783E-05" ixy="-2.43616858946494E-07" ixz="-6.37789906117123E-09" iyy="2.8270243746167E-06" iyz="-5.37200748039765E-07" izz="2.83695868220296E-05" />
+        </inertial> -->
+      <visual>
+        <origin xyz="0 0 0" rpy="0 0 0" />
+        <geometry>
+          <mesh filename="package://aist_robotiq/meshes/visual/robotiq_arg2f_85_inner_knuckle.dae" scale="0.001 0.001 0.001"/>
         </geometry>
         <material name="">
@@ -93,5 +75,5 @@
         <origin xyz="0 0 0" rpy="0 0 0" />
         <geometry>
-          <mesh filename="package://aist_robotiq_description/meshes/collision/robotiq_arg2f_${stroke}_inner_knuckle.stl" />
+          <mesh filename="package://aist_robotiq/meshes/collision/robotiq_arg2f_85_inner_knuckle.dae" scale="0.001 0.001 0.001"/>
         </geometry>
       </collision>
@@ -103,19 +85,13 @@
   <xacro:macro name="inner_finger" params="prefix fingerprefix stroke">
     <link name="${prefix}${fingerprefix}_inner_finger">
-      <inertial>
+      <!--<inertial>
         <origin xyz="0.000299999999999317 0.0160078233491243 -0.0136945669206257" rpy="0 0 0" />
         <mass value="0.0104003125914103" />
-        <inertia
-            ixx="2.71909453810972E-06"
-            ixy="1.35402465472579E-21"
-            ixz="-7.1817349065269E-22"
-            iyy="7.69100314106116E-07"
-            iyz="6.74715432769696E-07"
-            izz="2.30315190420171E-06" />
-      </inertial>
-      <visual>
-        <origin xyz="0 0 0" rpy="0 0 0" />
-        <geometry>
-          <mesh filename="package://aist_robotiq_description/meshes/visual/robotiq_arg2f_${stroke}_inner_finger.stl" />
+        <inertia ixx="2.71909453810972E-06" ixy="1.35402465472579E-21" ixz="-7.1817349065269E-22" iyy="7.69100314106116E-07" iyz="6.74715432769696E-07" izz="2.30315190420171E-06" />
+        </inertial> -->
+      <visual>
+        <origin xyz="0 0 0" rpy="0 0 0" />
+        <geometry>
+          <mesh filename="package://aist_robotiq/meshes/visual/robotiq_arg2f_85_inner_finger.dae" scale="0.001 0.001 0.001"/>
         </geometry>
         <material name="">
@@ -126,5 +102,5 @@
         <origin xyz="0 0 0" rpy="0 0 0" />
         <geometry>
-          <mesh filename="package://aist_robotiq_description/meshes/collision/robotiq_arg2f_${stroke}_inner_finger.stl" />
+          <mesh filename="package://aist_robotiq/meshes/collision/robotiq_arg2f_85_inner_finger.dae" scale="0.001 0.001 0.001" />
         </geometry>
       </collision>
@@ -134,5 +110,5 @@
     </gazebo>
   </xacro:macro>
-  <!-- Finger pad link, the default are the "big pads" with rubber-->
+   <!-- Finger pad link, the default are the "big pads" with rubber-->
   <xacro:macro name="inner_finger_pad" params="prefix fingerprefix">
     <link name="${prefix}${fingerprefix}_inner_finger_pad">
@@ -140,5 +116,5 @@
         <origin xyz="0 0 0" rpy="0 0 0" />
         <geometry>
-          <box size="0.027 0.065 0.0075"/>
+          <box size="0.022 0.00635 0.0375"/>
         </geometry>
         <material name="">
@@ -149,5 +125,5 @@
         <origin xyz="0 0 0" rpy="0 0 0" />
         <geometry>
-           <box size="0.03 0.07 0.0075"/>
+           <box size="0.022 0.00635 0.0375"/>
         </geometry>
         <material name="">
@@ -162,5 +138,5 @@
   <xacro:macro name="outer_finger_joint" params="prefix fingerprefix">
     <joint name="${prefix}${fingerprefix}_outer_finger_joint" type="fixed">
-      <origin xyz="0 0.01821998610742 0.0260018192872234" rpy="0 0 0" />
+      <origin xyz="0 0.0315 -0.0041" rpy="0 0 0"/>
       <parent link="${prefix}${fingerprefix}_outer_knuckle" />
       <child link="${prefix}${fingerprefix}_outer_finger" />
@@ -170,25 +146,26 @@
   <xacro:macro name="inner_knuckle_joint" params="prefix fingerprefix reflect">
     <joint name="${prefix}${fingerprefix}_inner_knuckle_joint" type="revolute">
-      <origin xyz="0 ${reflect * -0.0127} 0.06142" rpy="${pi / 2 + .725} 0 ${(reflect - 1) * pi / 2}" />
+      <!-- <origin xyz="0 ${reflect * -0.0127} 0.06142" rpy="${pi / 2 + .725} 0 ${(reflect - 1) * pi / 2}" /> -->
+      <origin xyz="0 ${reflect * -0.0127} 0.06142" rpy="0 0 ${(1 + reflect) * pi / 2}"/>
       <parent link="${prefix}robotiq_arg2f_base_link" />
       <child link="${prefix}${fingerprefix}_inner_knuckle" />
       <axis xyz="1 0 0" />
-      <limit lower="-0.8757" upper="0.8757" velocity="2.0" effort="1000" />
-      <mimic joint="${prefix}finger_joint" multiplier="-1" offset="0" />
+      <limit lower="0" upper="0.8757" velocity="2.0" effort="1000" />
+      <mimic joint="${prefix}finger_joint" multiplier="1" offset="0" />
     </joint>
   </xacro:macro>
   <xacro:macro name="inner_finger_joint" params="prefix fingerprefix">
     <joint name="${prefix}${fingerprefix}_inner_finger_joint" type="revolute">
-      <origin xyz="0 0.0817554015893473 -0.0282203446692936" rpy="-0.725 0 0" />
+      <origin xyz="0 0.0061 0.0471" rpy="0 0 0"/>
       <parent link="${prefix}${fingerprefix}_outer_finger" />
       <child link="${prefix}${fingerprefix}_inner_finger" />
       <axis xyz="1 0 0" />
-      <limit lower="-0.8757" upper="0.8757" velocity="2.0" effort="1000" />
-      <mimic joint="${prefix}finger_joint" multiplier="1" offset="0" />
+      <limit lower="0" upper="0.8757" velocity="2.0" effort="1000" />
+      <mimic joint="${prefix}finger_joint" multiplier="-1" offset="0" />
     </joint>
   </xacro:macro>
   <xacro:macro name="inner_finger_pad_joint" params="prefix fingerprefix">
     <joint name="${prefix}${fingerprefix}_inner_finger_pad_joint" type="fixed">
-      <origin xyz="0 0.0457554015893473 -0.0272203446692936" rpy="0 0 0" />
+      <origin xyz="0 -0.0220203446692936 0.03242" rpy="0 0 0"/>
       <parent link="${prefix}${fingerprefix}_inner_finger" />
       <child link="${prefix}${fingerprefix}_inner_finger_pad" />
@@ -196,12 +173,12 @@
     </joint>
   </xacro:macro>
-  <xacro:include filename="$(find aist_robotiq_description)/urdf/robotiq_arg2f.xacro" />
+  <xacro:include filename="$(find aist_robotiq)/urdf/robotiq_arg2f.xacro" />
   <xacro:macro name="finger_joint" params="prefix">
     <joint name="${prefix}finger_joint" type="revolute">
-      <origin xyz="0 -0.030601 0.054905" rpy="${pi / 2 + .725} 0 0" />
+      <origin xyz="0 -0.0306011 0.054904" rpy="0 0 ${pi}"/>
       <parent link="${prefix}robotiq_arg2f_base_link" />
       <child link="${prefix}left_outer_knuckle" />
-      <axis xyz="-1 0 0" />
-      <limit lower="0" upper="0.7" velocity="2.0" effort="1000" />
+      <axis xyz="1 0 0" />
+      <limit lower="0" upper="0.8" velocity="2.0" effort="1000" />
     </joint>
     <xacro:finger_joints prefix="${prefix}" fingerprefix="left" reflect="1.0"/>
@@ -209,34 +186,35 @@
   <xacro:macro name="right_outer_knuckle_joint" params="prefix">
     <joint name="${prefix}right_outer_knuckle_joint" type="revolute">
-      <origin xyz="0 0.030601 0.054905" rpy="${pi / 2 + .725} 0 ${pi}" />
+      <origin xyz="0 0.0306011 0.054904" rpy="0 0 0"/>
       <parent link="${prefix}robotiq_arg2f_base_link" />
       <child link="${prefix}right_outer_knuckle" />
       <axis xyz="1 0 0" />
-      <limit lower="-0.725" upper="0.725" velocity="2.0" effort="1000" />
-    <mimic joint="${prefix}finger_joint" multiplier="-1" offset="0" />
+      <limit lower="0" upper="0.81" velocity="2.0" effort="1000" />
+      <mimic joint="${prefix}finger_joint" multiplier="1" offset="0" />
     </joint>
     <xacro:finger_joints prefix="${prefix}" fingerprefix="right" reflect="-1.0"/>
   </xacro:macro>
-  <xacro:macro name="robotiq_140_gripper" params="prefix parent *origin">
-    <joint name="${prefix}robotiq_140_base_joint" type="fixed">
+  <!-- Initialization of all joints and links -->
+  <xacro:macro name="robotiq_85_gripper" params="prefix parent *origin">
+    <joint name="${prefix}base_joint" type="fixed">
       <parent link="${parent}"/>
-      <child link="${prefix}robotiq_140_base_link"/>
+      <child link="${prefix}base_link"/>
       <xacro:insert_block name="origin"/>
     </joint>
-    <link name="${prefix}robotiq_140_base_link"/>
+    <link name="${prefix}base_link"/>
     <joint name="${prefix}robotiq_arg2f_base_joint" type="fixed">
-      <parent link="${prefix}robotiq_140_base_link"/>
+      <parent link="${prefix}base_link"/>
       <child link="${prefix}robotiq_arg2f_base_link"/>
       <origin xyz="0 0 0" rpy="${pi} ${-pi/2} 0" />
     </joint>
-    <link name="${prefix}robotiq_140_tip_link"/>
-    <joint name="${prefix}robotiq_140_tip_link_joint" type="fixed">
-      <parent link="${prefix}robotiq_140_base_link"/>
-      <child link="${prefix}robotiq_140_tip_link"/>
-      <origin rpy="0.0 0.0 0.0" xyz=".2333 0.0 0.0"/>
+    <link name="${prefix}tip_link"/>
+    <joint name="${prefix}tip_link_joint" type="fixed">
+      <parent link="${prefix}base_link"/>
+      <child link="${prefix}tip_link"/>
+      <origin rpy="0.0 0.0 0.0" xyz=".1628 0.0 0.0"/>
     </joint>
     <xacro:robotiq_arg2f_base_link prefix="${prefix}"/>
-    <xacro:finger_links prefix="${prefix}" fingerprefix="left" stroke="140"/>
-    <xacro:finger_links prefix="${prefix}" fingerprefix="right" stroke="140"/>
+    <xacro:finger_links prefix="${prefix}" fingerprefix="left" stroke="85"/>
+    <xacro:finger_links prefix="${prefix}" fingerprefix="right" stroke="85"/>
     <xacro:finger_joint prefix="${prefix}"/>
     <xacro:right_outer_knuckle_joint prefix="${prefix}"/>
@@ -244,17 +222,17 @@
     <!-- Mimic joints -->
     <gazebo>
-      <plugin filename="libgazebo_mimic_joint_plugin.so" name="${prefix}mimic_robotiq_85_1">
+      <plugin filename="libgazebo_mimic_joint_plugin.so" name="${prefix}mimic_1">
         <joint>${prefix}finger_joint</joint>
         <mimicJoint>${prefix}right_outer_knuckle_joint</mimicJoint>
       </plugin>
-      <plugin filename="libgazebo_mimic_joint_plugin.so" name="${prefix}mimic_robotiq_85_2">
+      <plugin filename="libgazebo_mimic_joint_plugin.so" name="${prefix}mimic_2">
         <joint>${prefix}finger_joint</joint>
         <mimicJoint>${prefix}left_inner_knuckle_joint</mimicJoint>
       </plugin>
-      <plugin filename="libgazebo_mimic_joint_plugin.so" name="${prefix}mimic_robotiq_85_3">
+      <plugin filename="libgazebo_mimic_joint_plugin.so" name="${prefix}mimic_3">
         <joint>${prefix}finger_joint</joint>
         <mimicJoint>${prefix}right_inner_knuckle_joint</mimicJoint>
       </plugin>
-      <plugin filename="libgazebo_mimic_joint_plugin.so" name="${prefix}mimic_robotiq_85_4">
+      <plugin filename="libgazebo_mimic_joint_plugin.so" name="${prefix}mimic_4">
         <joint>${prefix}finger_joint</joint>
         <mimicJoint>${prefix}left_inner_finger_joint</mimicJoint>
@@ -262,5 +240,5 @@
         <offset>0.0</offset>
       </plugin>
-      <plugin filename="libgazebo_mimic_joint_plugin.so" name="${prefix}mimic_robotiq_85_5">
+      <plugin filename="libgazebo_mimic_joint_plugin.so" name="${prefix}mimic_5">
         <joint>${prefix}finger_joint</joint>
         <mimicJoint>${prefix}right_inner_finger_joint</mimicJoint>

File: aist_robotiq/urdf/robotiq_hande.urdf.xacro (robot description, xacro)
@@ -2,10 +2,10 @@
 <robot xmlns:xacro="http://ros.org/wiki/xacro">
   <xacro:macro name="robotiq_hande"  params="prefix parent *origin">
-    <joint name="${prefix}robotiq_hande_base_joint" type="fixed">
+    <joint name="${prefix}base_joint" type="fixed">
       <parent link="${parent}"/>
-      <child link="${prefix}robotiq_hande_base_link"/>
+      <child link="${prefix}base_link"/>
       <xacro:insert_block name="origin"/>
     </joint>
-    <link name="${prefix}robotiq_hande_base_link">
+    <link name="${prefix}base_link">
       <inertial>
         <origin xyz="0 0 0.04607" rpy="${pi/2} 0 ${pi/2}" />
@@ -16,5 +16,5 @@
         <origin xyz="0 0 0" rpy="${pi/2} 0 ${pi/2}" />
         <geometry>
-          <mesh filename="package://aist_robotiq_description/meshes/visual/hand-e.dae" scale="0.001 0.001 0.001"/>
+          <mesh filename="package://aist_robotiq/meshes/visual/hand-e.dae" scale="0.001 0.001 0.001"/>
         </geometry>
         <material name="Gazebo/Black">
@@ -25,13 +25,13 @@
         <origin xyz="0 0 0" rpy="${pi/2} 0 ${pi/2}" />
         <geometry>
-          <mesh filename="package://aist_robotiq_description/meshes/visual/hand-e.dae" scale="0.001 0.001 0.001"/>
+          <mesh filename="package://aist_robotiq/meshes/visual/hand-e.dae" scale="0.001 0.001 0.001"/>
         </geometry>
       </collision>
     </link>
-    <gazebo reference="${prefix}robotiq_hande_base_link">
+    <gazebo reference="${prefix}base_link">
       <material>Gazebo/Black</material>
       <selfCollide>True</selfCollide>
     </gazebo>
-    <link name="${prefix}robotiq_hande_left_finger">
+    <link name="${prefix}left_finger">
       <inertial>
         <origin xyz="0.02262 -0.00759 0.00738" rpy="${pi/2} 0 ${pi/2}"/>
@@ -42,5 +42,5 @@
         <origin xyz="0 0 0" rpy="${pi/2} 0 ${pi/2}"/>
         <geometry>
-          <mesh filename="package://aist_robotiq_description/meshes/visual/hand-e_finger_1.dae" scale="0.001 0.001 0.001"/>
+          <mesh filename="package://aist_robotiq/meshes/visual/hand-e_finger_1.dae" scale="0.001 0.001 0.001"/>
         </geometry>
         <material name="Gazebo/Grey">
@@ -51,13 +51,13 @@
         <origin xyz="0 0 0" rpy="${pi/2} 0 ${pi/2}"/>
         <geometry>
-          <mesh filename="package://aist_robotiq_description/meshes/visual/hand-e_finger_1.dae" scale="0.001 0.001 0.001"/>
+          <mesh filename="package://aist_robotiq/meshes/visual/hand-e_finger_1.dae" scale="0.001 0.001 0.001"/>
         </geometry>
       </collision>
     </link>
-    <gazebo reference="${prefix}robotiq_hande_left_finger">
+    <gazebo reference="${prefix}left_finger">
       <material>Gazebo/Grey</material>
       <selfCollide>True</selfCollide>
     </gazebo>
-    <link name="${prefix}robotiq_hande_right_finger">
+    <link name="${prefix}right_finger">
       <inertial>
         <origin xyz="-0.02262 0.00759 0.00738" rpy="${pi/2} 0 ${pi/2}"/>
@@ -68,5 +68,5 @@
         <origin xyz="0 0 0" rpy="${pi/2} 0 ${pi/2}"/>
         <geometry>
-          <mesh filename="package://aist_robotiq_description/meshes/visual/hand-e_finger_2.dae" scale="0.001 0.001 0.001"/>
+          <mesh filename="package://aist_robotiq/meshes/visual/hand-e_finger_2.dae" scale="0.001 0.001 0.001"/>
         </geometry>
         <material name="Gazebo/Grey">
@@ -77,40 +77,40 @@
         <origin xyz="0 0 0" rpy="${pi/2} 0 ${pi/2}"/>
         <geometry>
-          <mesh filename="package://aist_robotiq_description/meshes/visual/hand-e_finger_2.dae" scale="0.001 0.001 0.001"/>
+          <mesh filename="package://aist_robotiq/meshes/visual/hand-e_finger_2.dae" scale="0.001 0.001 0.001"/>
         </geometry>
       </collision>
     </link>
-    <gazebo reference="${prefix}robotiq_hande_right_finger">
+    <gazebo reference="${prefix}right_finger">
       <material>Gazebo/Grey</material>
       <selfCollide>True</selfCollide>
     </gazebo>
-    <joint name="${prefix}robotiq_hande_joint_finger" type="prismatic">
+    <joint name="${prefix}joint_finger" type="prismatic">
       <origin xyz="0.099 0 0" rpy="0 0 0"/>
-      <parent link="${prefix}robotiq_hande_base_link"/>
-      <child link="${prefix}robotiq_hande_left_finger"/>
+      <parent link="${prefix}base_link"/>
+      <child link="${prefix}left_finger"/>
       <axis xyz="0 -1 0"/>
       <limit effort="130" lower="0" upper="0.025" velocity="0.15"/>
     </joint>
-    <joint name="${prefix}robotiq_hande_base_to_right_finger" type="prismatic">
+    <joint name="${prefix}base_to_right_finger" type="prismatic">
       <origin xyz="0.099 0 0" rpy="0 0 0"/>
-      <parent link="${prefix}robotiq_hande_base_link"/>
-      <child link="${prefix}robotiq_hande_right_finger"/>
+      <parent link="${prefix}base_link"/>
+      <child link="${prefix}right_finger"/>
       <axis xyz="0 1 0"/>
       <limit effort="130" lower="0" upper="0.025" velocity="0.15"/>
-      <mimic joint="${prefix}robotiq_hande_joint_finger" multiplier="1" offset="0"/>
+      <mimic joint="${prefix}joint_finger" multiplier="1" offset="0"/>
     </joint>
     <!-- Add additional links for us to plan with. Oriented like the UR frame. -->
-    <link name="${prefix}robotiq_hande_tip_link"/>
-    <joint name="${prefix}robotiq_hande_tip_link_joint" type="fixed">
-      <parent link="${prefix}robotiq_hande_base_link"/>
-      <child link="${prefix}robotiq_hande_tip_link"/>
+    <link name="${prefix}tip_link"/>
+    <joint name="${prefix}tip_link_joint" type="fixed">
+      <parent link="${prefix}base_link"/>
+      <child link="${prefix}tip_link"/>
       <origin rpy="0.0 0.0 0.0" xyz=".146 0.0 0.0"/>
     </joint>
-    <transmission name="${prefix}robotiq_hande_joint_finger_trans">
+    <transmission name="${prefix}joint_finger_trans">
       <type>transmission_interface/SimpleTransmission</type>
-      <joint name="${prefix}robotiq_hande_joint_finger">
+      <joint name="${prefix}joint_finger">
         <hardwareInterface>hardware_interface/PositionJointInterface</hardwareInterface>
       </joint>
-      <actuator name="${prefix}robotiq_hande_joint_finger_motor">
+      <actuator name="${prefix}joint_finger_motor">
         <mechanicalReduction>1</mechanicalReduction>
         <hardwareInterface>hardware_interface/PositionJointInterface</hardwareInterface>
@@ -120,6 +120,6 @@
       <plugin filename="libgazebo_mimic_joint_plugin.so"
 	      name="${prefix}mimic_robotiq_hande">
-        <joint>${prefix}robotiq_hande_joint_finger</joint>
-        <mimicJoint>${prefix}robotiq_hande_base_to_right_finger</mimicJoint>
+        <joint>${prefix}joint_finger</joint>
+        <mimicJoint>${prefix}base_to_right_finger</mimicJoint>
       </plugin>
     </gazebo>
